Commit message: remove absolute pathes

File: urdflbriiwa7/urdf/urdflbriiwa7.urdf (robot description, URDF)
Before this commit: robot urdflbriiwa7, 10 links, 9 joints
Links:
- link URDFLBRiiwa7Axis1: geometry collision mesh filename=package://urdflbriiwa7/meshes/collision/iiwa_r820_link_1_co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; visual mesh filename=package://urdflbriiwa7/meshes/visual/iiwa_r820_link_1_hull_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
- link URDFLBRiiwa7Axis2: geometry collision mesh filename=package://urdflbriiwa7/meshes/collision/iiwa_r820_link_2_co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; visual mesh filename=package://urdflbriiwa7/meshes/visual/iiwa_r820_link_2_hull_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
- link URDFLBRiiwa7RobotBase: geometry collision mesh filename=package://urdflbriiwa7/meshes/collision/iiwa_r820_link_0_co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; visual mesh filename=package://urdflbriiwa7/meshes/visual/iiwa_r820_link_0_hull_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
- link URDFLBRiiwaAxis3: geometry collision mesh filename=package://urdflbriiwa7/meshes/collision/iiwa_r820_link_3_co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; visual mesh filename=package://urdflbriiwa7/meshes/visual/iiwa_r820_link_3_hull_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
- link URDFLBRiiwaAxis4: geometry collision mesh filename=package://urdflbriiwa7/meshes/collision/iiwa_r820_link_4_co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; visual mesh filename=package://urdflbriiwa7/meshes/visual/iiwa_r820_link_4_hull_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
- link URDFLBRiiwaAxis5: geometry collision mesh filename=package://urdflbriiwa7/meshes/collision/iiwa_r820_link_5_co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; visual mesh filename=package://urdflbriiwa7/meshes/visual/iiwa_r820_link_5_hull_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
- link URDFLBRiiwaAxis6: geometry collision mesh filename=package://urdflbriiwa7/meshes/collision/iiwa_r820_link_6_co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; visual mesh filename=package://urdflbriiwa7/meshes/visual/iiwa_r820_link_6_hull_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
- link URDFLBRiiwaAxis7: geometry collision mesh filename=package://urdflbriiwa7/meshes/collision/iiwa_r820_link_7_co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; visual mesh filename=package://urdflbriiwa7/meshes/visual/iiwa_r820_link_7_hull_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
