Commit message: rename package and fix names

File: kuka_lbr_iiwa7_support/urdf/urdflbriiwa7.urdf (robot description, URDF)
Before this commit: robot urdflbriiwa7, 10 links, 9 joints
Links:
- link URDFLBRiiwa7Axis1: geometry collision mesh filename=package://kuka_lbr_iiwa7_support/meshes/collision/iiwa_r820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; visual mesh filename=package://kuka_lbr_iiwa7_support/meshes/visual/iiwa_r820_li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
- link URDFLBRiiwa7Axis2: geometry collision mesh filename=package://kuka_lbr_iiwa7_support/meshes/collision/iiwa_r820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; visual mesh filename=package://kuka_lbr_iiwa7_support/meshes/visual/iiwa_r820_li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
- link URDFLBRiiwa7RobotBase: geometry collision mesh filename=package://kuka_lbr_iiwa7_support/meshes/collision/iiwa_r820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; visual mesh filename=package://kuka_lbr_iiwa7_support/meshes/visual/iiwa_r820_li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
- link URDFLBRiiwaAxis3: geometry collision mesh filename=package://kuka_lbr_iiwa7_support/meshes/collision/iiwa_r820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; visual mesh filename=package://kuka_lbr_iiwa7_support/meshes/visual/iiwa_r820_li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
- link URDFLBRiiwaAxis4: geometry collision mesh filename=package://kuka_lbr_iiwa7_support/meshes/collision/iiwa_r820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; visual mesh filename=package://kuka_lbr_iiwa7_support/meshes/visual/iiwa_r820_li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
- link URDFLBRiiwaAxis5: geometry collision mesh filename=package://kuka_lbr_iiwa7_support/meshes/collision/iiwa_r820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; visual mesh filename=package://kuka_lbr_iiwa7_support/meshes/visual/iiwa_r820_li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
- link URDFLBRiiwaAxis6: geometry collision mesh filename=package://kuka_lbr_iiwa7_support/meshes/collision/iiwa_r820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; visual mesh filename=package://kuka_lbr_iiwa7_support/meshes/visual/iiwa_r820_li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
- link URDFLBRiiwaAxis7: geometry collision mesh filename=package://kuka_lbr_iiwa7_support/meshes/collision/iiwa_r820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; visual mesh filename=package://kuka_lbr_iiwa7_support/meshes/visual/iiwa_r820_li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

Commit message: remove urdf from robot name

File: kuka_lbr_iiwa7_support/urdf/urdflbriiwa7.urdf (robot description, URDF)
Before this commit: robot lbriiwa7, 10 links, 9 joints
Links:
- removed link URDFLBRiiwa7Axis1
- removed link URDFLBRiiwa7Axis2
- removed link URDFLBRiiwa7RobotBase
- removed link URDFLBRiiwaAxis3
- removed link URDFLBRiiwaAxis4
- removed link URDFLBRiiwaAxis5
- removed link URDFLBRiiwaAxis6
- removed link URDFLBRiiwaAxis7
- removed link URDFLBRiiwaFlange
- added link LBRiiwa7Axis1, mass 6.495; collision mesh filename=package://kuka_lbr_iiwa7_support/meshes/collision/iiwa_r820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; visual mesh filename=package://kuka_lbr_iiwa7_support/meshes/visual/iiwa_r820_li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
- added link LBRiiwa7Axis2, mass 8.365; collision mesh filename=package://kuka_lbr_iiwa7_support/meshes/collision/iiwa_r820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; visual mesh filename=package://kuka_lbr_iiwa7_support/meshes/visual/iiwa_r820_li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
- added link LBRiiwa7RobotBase, mass 3.2832; collision mesh filename=package://kuka_lbr_iiwa7_support/meshes/collision/iiwa_r820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; visual mesh filename=package://kuka_lbr_iiwa7_support/meshes/visual/iiwa_r820_li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
- added link LBRiiwaAxis3, mass 2.5697; collision mesh filename=package://kuka_lbr_iiwa7_support/meshes/collision/iiwa_r820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; visual mesh filename=package://kuka_lbr_iiwa7_support/meshes/visual/iiwa_r820_li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
- added link LBRiiwaAxis4, mass 5.41; collision mesh filename=package://kuka_lbr_iiwa7_support/meshes/collision/iiwa_r820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; visual mesh filename=package://kuka_lbr_iiwa7_support/meshes/visual/iiwa_r820_li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
- added link LBRiiwaAxis5, mass 1.867; collision mesh filename=package://kuka_lbr_iiwa7_support/meshes/collision/iiwa_r820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; visual mesh filename=package://kuka_lbr_iiwa7_support/meshes/visual/iiwa_r820_li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
- added link LBRiiwaAxis6, mass 2.458; collision mesh filename=package://kuka_lbr_iiwa7_support/meshes/collision/iiwa_r820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; visual mesh filename=package://kuka_lbr_iiwa7_support/meshes/visual/iiwa_r820_li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
- added link LBRiiwaAxis7, mass 0.627; collision mesh filename=package://kuka_lbr_iiwa7_support/meshes/collision/iiwa_r820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; visual mesh filename=package://kuka_lbr_iiwa7_support/meshes/visual/iiwa_r820_li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
- added link LBRiiwaFlange
Joints:
- removed joint URDFLBRiiwa7Joint1
- removed joint URDFLBRiiwa7Joint2
- removed joint URDFLBRiiwa7RobotBaseJoint
- removed joint URDFLBRiiwaJoint3
- removed joint URDFLBRiiwaJoint4
- removed joint URDFLBRiiwaJoint5
- removed joint URDFLBRiiwaJoint6
- removed joint URDFLBRiiwaJoint7
- removed joint URDFLBRiiwaTCP
- added joint LBRiiwa7Joint1: type revolute, parent LBRiiwa7RobotBase, child LBRiiwa7Axis1, origin xyz=0.0 0.0 0.1375 rpy=-0.0 0.0 0.0, axis 0.0 0.0 1.0, limit lower=-2.67035 upper=2.67035 effort=158.4 velocity=6.283
- added joint LBRiiwa7Joint2: type revolute, parent LBRiiwa7Axis1, child LBRiiwa7Axis2, origin xyz=0.0 0.0 0.2025 rpy=-0.0 0.0 0.0, axis 0.0 1.0 0.0, limit lower=-1.8849 upper=1.8849 effort=158.4 velocity=6.283
- added joint LBRiiwa7RobotBaseJoint: type fixed, parent world, child LBRiiwa7RobotBase
- added joint LBRiiwaJoint3: type revolute, parent LBRiiwa7Axis2, child LBRiiwaAxis3, origin xyz=0.0 0.0 0.1845 rpy=-0.0 0.0 0.0, axis 0.0 0.0 1.0, limit lower=-2.67035 upper=2.67035 effort=99 velocity=6.283
- added joint LBRiiwaJoint4: type revolute, parent LBRiiwaAxis3, child LBRiiwaAxis4, origin xyz=0.0 0.0 0.2155 rpy=-0.0 0.0 0.0, axis 0.0 -1.0 0.0, limit lower=-1.8849 upper=1.8849 effort=99 velocity=6.283
- added joint LBRiiwaJoint5: type revolute, parent LBRiiwaAxis4, child LBRiiwaAxis5, origin xyz=0.0 0.0 0.1845 rpy=-0.0 0.0 0.0, axis 0.0 0.0 1.0, limit lower=-2.67035 upper=2.67035 effort=99 velocity=6.283
- added joint LBRiiwaJoint6: type revolute, parent LBRiiwaAxis5, child LBRiiwaAxis6, origin xyz=0.0 0.0 0.2155 rpy=-0.0 0.0 0.0, axis 0.0 1.0 0.0, limit lower=-1.8849 upper=1.8849 effort=36 velocity=6.283
- added joint LBRiiwaJoint7: type revolute, parent LBRiiwaAxis6, child LBRiiwaAxis7, origin xyz=0.0 0.0 0.081 rpy=-0.0 0.0 0.0, axis 0.0 0.0 1.0, limit lower=-2.74889 upper=2.74889 effort=36 velocity=6.283
- added joint LBRiiwaTCP: type fixed, parent LBRiiwaAxis7, child LBRiiwaFlange, origin xyz=0.0 0.0 0.071 rpy=-0.0 0.0 0.0, axis 0.0 0.0 1.0
