Commit message: move gpio config to kuka_sunrise package

File: kuka_lbr_iiwa7_support/urdf/lbriiwa7_macro.xacro (robot description, xacro)
@@ -1,4 +1,5 @@
 <?xml version="1.0"?>
-<robot name="lbriiwa7">
+<robot xmlns:xacro="http://wiki.ros.org/xacro">
+  <xacro:macro name="kuka_lbr_iiwa7" params="io_access">
   <ros2_control name="iiwa_hardware" type="system">
     <hardware>
@@ -98,46 +99,11 @@
     </joint>
     <!-- TODO(Svastits): update GPIO list from config file-->
-    <gpio name="gpio">
-      <command_interface name="Input1" data_type="boolean">
-         <param name="initial_value">0</param>
-      </command_interface>
-      <command_interface name="Input2" data_type="boolean">
-         <param name="initial_value">0</param>
-      </command_interface>
-      <command_interface name="Input3" data_type="boolean">
-         <param name="initial_value">0</param>
-      </command_interface>
-      <command_interface name="Input4" data_type="boolean">
-         <param name="initial_value">0</param>
-      </command_interface>
-      <command_interface name="Input5" data_type="boolean">
-         <param name="initial_value">0</param>
-      </command_interface>
-      <command_interface name="Input6" data_type="boolean">
-         <param name="initial_value">0</param>
-      </command_interface>
-      <command_interface name="Input7" data_type="boolean">
-         <param name="initial_value">0</param>
-      </command_interface>
-      <command_interface name="Input8" data_type="boolean">
-         <param name="initial_value">0</param>
-      </command_interface>
-      <command_interface name="Input9" data_type="boolean">
-         <param name="initial_value">0</param>
-      </command_interface>
-      <command_interface name="Input10" data_type="boolean">
-         <param name="initial_value">0</param>
-      </command_interface>
-      <state_interface name="Output1" data_type="boolean"/>
-      <state_interface name="Output2" data_type="boolean"/>
-      <state_interface name="Output3" data_type="boolean"/>
-      <state_interface name="Output4" data_type="boolean"/>
-      <state_interface name="Output5" data_type="boolean"/>
-      <state_interface name="Output6" data_type="boolean"/>
-      <state_interface name="Output7" data_type="boolean"/>
-      <state_interface name="Output8" data_type="boolean"/>
-      <state_interface name="Output9" data_type="boolean"/>
-      <state_interface name="Output10" data_type="boolean"/>
-    </gpio>
+    <xacro:if value="${io_access}">
+      <xacro:include filename="$(find kuka_sunrise)/config/gpio_config.xacro" />
+      <xacro:fri_gpio_config/>
+    </xacro:if>
+    <xacro:unless value="${io_access}">
+      <gpio name="gpio"/>
+    </xacro:unless>
   </ros2_control>
   <gazebo>
@@ -145,5 +111,5 @@
       <robotNamespace>/lbriiwa7</robotNamespace>
       <robotSimType>gazebo_ros2_control/DefaultRobotHWSim</robotSimType>
-      <parameters>$(find lbriiwa7)/config/lbriiwa7_control.yaml</parameters>
+      <parameters>$(find kuka_lbr_iiwa7_support)/config/lbriiwa7_control.yaml</parameters>
     </plugin>
   </gazebo>
@@ -463,3 +429,4 @@
     </actuator>
   </transmission>
+  </xacro:macro>
 </robot>

Commit message: fix iiwa joint and axis names

File: kuka_lbr_iiwa7_support/urdf/lbriiwa7_macro.xacro (robot description, xacro)
@@ -126,21 +126,21 @@
     <material>Gazebo/Orange</material>
   </gazebo>
-  <gazebo reference="LBRiiwaAxis3">
-    <selfCollide>true</selfCollide>
-    <material>Gazebo/Orange</material>
-  </gazebo>
-  <gazebo reference="LBRiiwaAxis4">
-    <selfCollide>true</selfCollide>
-    <material>Gazebo/Orange</material>
-  </gazebo>
-  <gazebo reference="LBRiiwaAxis5">
-    <selfCollide>true</selfCollide>
-    <material>Gazebo/Orange</material>
-  </gazebo>
-  <gazebo reference="LBRiiwaAxis6">
-    <selfCollide>true</selfCollide>
-    <material>Gazebo/Orange</material>
-  </gazebo>
-  <gazebo reference="LBRiiwaAxis7">
+  <gazebo reference="LBRiiwa7Axis3">
+    <selfCollide>true</selfCollide>
+    <material>Gazebo/Orange</material>
+  </gazebo>
+  <gazebo reference="LBRiiwa7Axis4">
+    <selfCollide>true</selfCollide>
+    <material>Gazebo/Orange</material>
+  </gazebo>
+  <gazebo reference="LBRiiwa7Axis5">
+    <selfCollide>true</selfCollide>
+    <material>Gazebo/Orange</material>
+  </gazebo>
+  <gazebo reference="LBRiiwa7Axis6">
+    <selfCollide>true</selfCollide>
+    <material>Gazebo/Orange</material>
+  </gazebo>
+  <gazebo reference="LBRiiwa7Axis7">
     <selfCollide>true</selfCollide>
     <material>Gazebo/Orange</material>
@@ -204,5 +204,5 @@
     </inertial>
   </link>
-  <link name="LBRiiwaAxis3">
+  <link name="LBRiiwa7Axis3">
     <visual>
       <geometry>
@@ -223,5 +223,5 @@
     </inertial>
   </link>
-  <link name="LBRiiwaAxis4">
+  <link name="LBRiiwa7Axis4">
     <visual>
       <geometry>
@@ -242,5 +242,5 @@
     </inertial>
   </link>
-  <link name="LBRiiwaAxis5">
+  <link name="LBRiiwa7Axis5">
     <visual>
       <geometry>
@@ -261,5 +261,5 @@
     </inertial>
   </link>
-  <link name="LBRiiwaAxis6">
+  <link name="LBRiiwa7Axis6">
     <visual>
       <geometry>
@@ -280,5 +280,5 @@
     </inertial>
   </link>
-  <link name="LBRiiwaAxis7">
+  <link name="LBRiiwa7Axis7">
     <visual>
       <geometry>
@@ -318,35 +318,35 @@
     <limit effort="158.4" lower="-1.8849" upper="1.8849" velocity="6.283"/>
   </joint>
-  <joint name="LBRiiwaJoint3" type="revolute">
+  <joint name="LBRiiwa7Joint3" type="revolute">
     <parent link="LBRiiwa7Axis2"/>
-    <child link="LBRiiwaAxis3"/>
+    <child link="LBRiiwa7Axis3"/>
     <origin rpy="-0.0 0.0 0.0" xyz="0.0 0.0 0.1845"/>
     <axis xyz="0.0 0.0 1.0"/>
     <limit effort="99" lower="-2.67035" upper="2.67035" velocity="6.283"/>
   </joint>
-  <joint name="LBRiiwaJoint4" type="revolute">
-    <parent link="LBRiiwaAxis3"/>
-    <child link="LBRiiwaAxis4"/>
+  <joint name="LBRiiwa7Joint4" type="revolute">
+    <parent link="LBRiiwa7Axis3"/>
+    <child link="LBRiiwa7Axis4"/>
     <origin rpy="-0.0 0.0 0.0" xyz="0.0 0.0 0.2155"/>
     <axis xyz="0.0 -1.0 0.0"/>
     <limit effort="99" lower="-1.8849" upper="1.8849" velocity="6.283"/>
   </joint>
-  <joint name="LBRiiwaJoint5" type="revolute">
-    <parent link="LBRiiwaAxis4"/>
-    <child link="LBRiiwaAxis5"/>
+  <joint name="LBRiiwa7Joint5" type="revolute">
+    <parent link="LBRiiwa7Axis4"/>
+    <child link="LBRiiwa7Axis5"/>
     <origin rpy="-0.0 0.0 0.0" xyz="0.0 0.0 0.1845"/>
     <axis xyz="0.0 0.0 1.0"/>
     <limit effort="99" lower="-2.67035" upper="2.67035" velocity="6.283"/>
   </joint>
-  <joint name="LBRiiwaJoint6" type="revolute">
-    <parent link="LBRiiwaAxis5"/>
-    <child link="LBRiiwaAxis6"/>
+  <joint name="LBRiiwa7Joint6" type="revolute">
+    <parent link="LBRiiwa7Axis5"/>
+    <child link="LBRiiwa7Axis6"/>
     <origin rpy="-0.0 0.0 0.0" xyz="0.0 0.0 0.2155"/>
     <axis xyz="0.0 1.0 0.0"/>
     <limit effort="36" lower="-1.8849" upper="1.8849" velocity="6.283"/>
   </joint>
-  <joint name="LBRiiwaJoint7" type="revolute">
-    <parent link="LBRiiwaAxis6"/>
-    <child link="LBRiiwaAxis7"/>
+  <joint name="LBRiiwa7Joint7" type="revolute">
+    <parent link="LBRiiwa7Axis6"/>
+    <child link="LBRiiwa7Axis7"/>
     <origin rpy="-0.0 0.0 0.0" xyz="0.0 0.0 0.081"/>
     <axis xyz="0.0 0.0 1.0"/>
@@ -354,5 +354,5 @@
   </joint>
   <joint name="LBRiiwaTCP" type="fixed">
-    <parent link="LBRiiwaAxis7"/>
+    <parent link="LBRiiwa7Axis7"/>
     <child link="LBRiiwaFlange"/>
     <origin rpy="-0.0 0.0 0.0" xyz="0.0 0.0 0.071"/>
@@ -379,50 +379,50 @@
     </actuator>
   </transmission>
-  <transmission name="Transmission_LBRiiwaJoint3">
-    <type>transmission_interface/SimpleTransmission</type>
-    <joint name="LBRiiwaJoint3">
-      <hardwareInterface>hardware_interface/EffortJointInterface</hardwareInterface>
-    </joint>
-    <actuator name="motor_LBRiiwaJoint3">
-      <hardwareInterface>EffortJointInterface</hardwareInterface>
-      <mechanicalReduction>1.0</mechanicalReduction>
-    </actuator>
-  </transmission>
-  <transmission name="Transmission_LBRiiwaJoint4">
-    <type>transmission_interface/SimpleTransmission</type>
-    <joint name="LBRiiwaJoint4">
-      <hardwareInterface>hardware_interface/EffortJointInterface</hardwareInterface>
-    </joint>
-    <actuator name="motor_LBRiiwaJoint4">
-      <hardwareInterface>EffortJointInterface</hardwareInterface>
-      <mechanicalReduction>1.0</mechanicalReduction>
-    </actuator>
-  </transmission>
-  <transmission name="Transmission_LBRiiwaJoint5">
-    <type>transmission_interface/SimpleTransmission</type>
-    <joint name="LBRiiwaJoint5">
-      <hardwareInterface>hardware_interface/EffortJointInterface</hardwareInterface>
-    </joint>
-    <actuator name="motor_LBRiiwaJoint5">
-      <hardwareInterface>EffortJointInterface</hardwareInterface>
-      <mechanicalReduction>1.0</mechanicalReduction>
-    </actuator>
-  </transmission>
-  <transmission name="Transmission_LBRiiwaJoint6">
-    <type>transmission_interface/SimpleTransmission</type>
-    <joint name="LBRiiwaJoint6">
-      <hardwareInterface>hardware_interface/EffortJointInterface</hardwareInterface>
-    </joint>
-    <actuator name="motor_LBRiiwaJoint6">
-      <hardwareInterface>EffortJointInterface</hardwareInterface>
-      <mechanicalReduction>1.0</mechanicalReduction>
-    </actuator>
-  </transmission>
-  <transmission name="Transmission_LBRiiwaJoint7">
-    <type>transmission_interface/SimpleTransmission</type>
-    <joint name="LBRiiwaJoint7">
-      <hardwareInterface>hardware_interface/EffortJointInterface</hardwareInterface>
-    </joint>
-    <actuator name="motor_LBRiiwaJoint7">
+  <transmission name="Transmission_LBRiiwa7Joint3">
+    <type>transmission_interface/SimpleTransmission</type>
+    <joint name="LBRiiwa7Joint3">
+      <hardwareInterface>hardware_interface/EffortJointInterface</hardwareInterface>
+    </joint>
+    <actuator name="motor_LBRiiwa7Joint3">
+      <hardwareInterface>EffortJointInterface</hardwareInterface>
+      <mechanicalReduction>1.0</mechanicalReduction>
+    </actuator>
+  </transmission>
+  <transmission name="Transmission_LBRiiwa7Joint4">
+    <type>transmission_interface/SimpleTransmission</type>
+    <joint name="LBRiiwa7Joint4">
+      <hardwareInterface>hardware_interface/EffortJointInterface</hardwareInterface>
+    </joint>
+    <actuator name="motor_LBRiiwa7Joint4">
+      <hardwareInterface>EffortJointInterface</hardwareInterface>
+      <mechanicalReduction>1.0</mechanicalReduction>
+    </actuator>
+  </transmission>
+  <transmission name="Transmission_LBRiiwa7Joint5">
+    <type>transmission_interface/SimpleTransmission</type>
+    <joint name="LBRiiwa7Joint5">
+      <hardwareInterface>hardware_interface/EffortJointInterface</hardwareInterface>
+    </joint>
+    <actuator name="motor_LBRiiwa7Joint5">
+      <hardwareInterface>EffortJointInterface</hardwareInterface>
+      <mechanicalReduction>1.0</mechanicalReduction>
+    </actuator>
+  </transmission>
+  <transmission name="Transmission_LBRiiwa7Joint6">
+    <type>transmission_interface/SimpleTransmission</type>
+    <joint name="LBRiiwa7Joint6">
+      <hardwareInterface>hardware_interface/EffortJointInterface</hardwareInterface>
+    </joint>
+    <actuator name="motor_LBRiiwa7Joint6">
+      <hardwareInterface>EffortJointInterface</hardwareInterface>
+      <mechanicalReduction>1.0</mechanicalReduction>
+    </actuator>
+  </transmission>
+  <transmission name="Transmission_LBRiiwa7Joint7">
+    <type>transmission_interface/SimpleTransmission</type>
+    <joint name="LBRiiwa7Joint7">
+      <hardwareInterface>hardware_interface/EffortJointInterface</hardwareInterface>
+    </joint>
+    <actuator name="motor_LBRiiwa7Joint7">
       <hardwareInterface>EffortJointInterface</hardwareInterface>
       <mechanicalReduction>1.0</mechanicalReduction>
