Commit message: reorganize config files

File: kuka_iisy_support/urdf/iisy.urdf (robot description, URDF)
Before this commit: robot LBR3R760iisy, 8 links, 7 joints
Links:
- link LBR3R760_iisy_axis1: mass 3.471E0 -> 3.2492E0
Joints:
- joint joint_a1: limit lower=-3.05432619E0 upper=3.05432619E0 effort=5.0E0 velocity=2.0E0 -> lower=-3.2288591E0 upper=3.2288591E0 effort=5.0E0 velocity=2.0E0
- joint joint_a2: origin xyz=0.0 -0.0829 0.0886 rpy=-0.0 1.570796 -0.0 -> xyz=0.0 -0.0829 0.0886 rpy=-0.0 0.0 -0.0
- joint joint_a3: origin xyz=0.0 0.0 0.3 rpy=-0.0 -1.570796 -0.0 -> xyz=0.0 0.0 0.3 rpy=-0.0 0.0 -0.0

File: kuka_iisy_support/urdf/iisy.urdf.xacro (robot description, xacro)
@@ -1,5 +1,5 @@
 <?xml version="1.0"?>
 <robot xmlns:xacro="http://www.ros.org/wiki/xacro" name="LBR3R760iisy">
-    <!-- Import panda urdf file -->
+    <!-- Import iisy urdf file -->
     <xacro:include filename="iisy.urdf" />
 </robot>

File: kuka_iisy_support/urdf/iisy_arm.srdf.xacro (robot description, xacro)
@@ -5,5 +5,5 @@
 -->
 <robot xmlns:xacro="http://www.ros.org/wiki/xacro" name="LBR3R760iisy">
-  <xacro:include filename="$(find kuka_iisy_moveit_config)/config/iisy_arm.xacro" />
+  <xacro:include filename="$(find kuka_iisy_support)/urdf/iisy_arm.xacro" />
   <xacro:iisy_arm />
 </robot>

File: kuka_iisy_support/urdf/iisy_arm.xacro (robot description, xacro)
@@ -8,5 +8,5 @@
     <!--SUBGROUPS: Groups can also be formed by referencing to already defined group names-->
     <group name="iisy_arm">
-      <chain base_link="base_link" tip_link="LBR3R760_iisy_axis6" />
+      <chain base_link="LBR3R760_iisy_fixedbase" tip_link="LBR3R760_iisy_axis6" />
     </group>
     <!--GROUP STATES: Purpose: Define a named state for a particular group, in terms of joint values. This is useful to define states like 'folded arms'-->
@@ -20,11 +20,12 @@
     </group_state>
     <!--VIRTUAL JOINT: Purpose: this element defines a virtual joint between a robot link and an external frame of reference (considered fixed with respect to the robot)-->
-    <virtual_joint name="virtual_joint" type="floating" parent_frame="world" child_link="base_link" />
+    <virtual_joint name="virtual_joint" type="floating" parent_frame="base_link" child_link="LBR3R760_iisy_fixedbase" />
     <!--DISABLE COLLISIONS: By default it is assumed that any link of the robot could potentially come into collision with any other link in the robot. This tag disables collision checking between a specified pair of links. -->
-    <disable_collisions link1="joint_a1" link2="joint_a2" reason="Adjacent" />
-    <disable_collisions link1="joint_a2" link2="joint_a3" reason="Adjacent" />
-    <disable_collisions link1="joint_a3" link2="joint_a4" reason="Adjacent" />
-    <disable_collisions link1="joint_a4" link2="joint_a5" reason="Adjacent" />
-    <disable_collisions link1="joint_a5" link2="joint_a6" reason="Adjacent" />
+    <disable_collisions link1="LBR3R760_iisy_fixedbase" link2="LBR3R760_iisy_axis1" reason="Adjacent"/>
+    <disable_collisions link1="LBR3R760_iisy_axis1" link2="LBR3R760_iisy_axis2" reason="Adjacent"/>
+    <disable_collisions link1="LBR3R760_iisy_axis2" link2="LBR3R760_iisy_axis3" reason="Adjacent"/>
+    <disable_collisions link1="LBR3R760_iisy_axis3" link2="LBR3R760_iisy_axis4" reason="Adjacent"/>
+    <disable_collisions link1="LBR3R760_iisy_axis4" link2="LBR3R760_iisy_axis5" reason="Adjacent"/>
+    <disable_collisions link1="LBR3R760_iisy_axis5" link2="LBR3R760_iisy_axis6" reason="Adjacent"/>
   </xacro:macro>
 </robot>

Commit message: rollback to old model

File: kuka_iisy_support/urdf/iisy.urdf (robot description, URDF)
Before this commit: robot LBR3R760iisy, 8 links, 7 joints
Links:
- link LBR3R760_iisy_axis1: mass 3.2492E0 -> 3.471E0
Joints:
- joint joint_a1: limit lower=-3.2288591E0 upper=3.2288591E0 effort=5.0E0 velocity=2.0E0 -> lower=-3.05432619E0 upper=3.05432619E0 effort=5.0E0 velocity=2.0E0
- joint joint_a2: origin xyz=0.0 -0.0829 0.0886 rpy=-0.0 0.0 -0.0 -> xyz=0.0 -0.0829 0.0886 rpy=-0.0 1.570796 -0.0
- joint joint_a3: origin xyz=0.0 0.0 0.3 rpy=-0.0 0.0 -0.0 -> xyz=0.0 0.0 0.3 rpy=-0.0 -1.570796 -0.0

Commit message: update to new urdf

File: kuka_iisy_support/urdf/iisy.urdf (robot description, URDF)
Before this commit: robot LBR3R760iisy, 8 links, 7 joints
Links:
- link LBR3R760_iisy_axis1: mass 3.471E0 -> 3.2492E0
Joints:
- joint joint_a1: axis 0.0 0.0 1.0 -> 0.0 0.0 -1.0; limit lower=-3.05432619E0 upper=3.05432619E0 effort=5.0E0 velocity=2.0E0 -> lower=-3.2288591E0 upper=3.2288591E0 effort=5.0E0 velocity=2.0E0
- joint joint_a2: axis 0.0 1.0 0.0 -> 0.0 0.0 1.0; origin xyz=0.0 -0.0829 0.0886 rpy=-0.0 1.570796 -0.0 -> xyz=0.0 0.0 0.0886 rpy=-1.5707963267948963 0.0 -0.0
- joint joint_a3: axis 0.0 1.0 0.0 -> 0.0 0.0 1.0; origin xyz=0.0 0.0 0.3 rpy=-0.0 -1.570796 -0.0 -> xyz=0.3 0.0 0.0 rpy=0.0 0.0 -1.5707963267948963
- joint joint_a4: axis 1.0 0.0 0.0 -> 0.0 0.0 1.0; origin xyz=0.1292 0.0829 0.0 rpy=-0.0 0.0 -0.0 -> xyz=0.0 0.0 0.0 rpy=1.5707963267948963 0.0 -0.0
- joint joint_a5: axis 0.0 1.0 0.0 -> 0.0 0.0 1.0; origin xyz=0.1708 0.0382 0.0 rpy=-0.0 0.0 -0.0 -> xyz=0.0 0.0 -0.3 rpy=-1.5707963267948963 0.0 -0.0
- joint joint_a6: axis 1.0 0.0 0.0 -> 0.0 0.0 1.0; origin xyz=0.0682 -0.0382 0.0 rpy=-0.0 0.0 -0.0 -> xyz=0.0 0.0 0.0 rpy=1.5707963267948963 0.0 -0.0
