Commit message: get params from config file

File: kuka_iisy_support/urdf/iisy.ros2_control.urdf.xacro (robot description, xacro)
@@ -1,7 +1,11 @@
 <?xml version="1.0" encoding="UTF-8"?>
-<robot name="LBR3R760iisy">
+<robot name="LBR3R760iisy" xmlns:xacro="http://www.ros.org/wiki/xacro">
+  <xacro:macro name="eci_config" params="client_ip controller_ip control_mode">
   <ros2_control name="iisy_hardware" type="system">
     <hardware>
       <plugin>kuka_rox::KukaRoXHardwareInterface</plugin>
+      <param name="client_ip">${client_ip}</param>
+      <param name="controller_ip">${controller_ip}</param>
+      <param name="control_mode">${control_mode}</param>
     </hardware>
     <!-- define joints and command/state interfaces for each joint -->
@@ -301,3 +305,4 @@
     <type>transmission_interface/SimpleTransmission</type>
   </transmission>
+  </xacro:macro>
 </robot>

File: kuka_iisy_support/urdf/iisy.urdf.xacro (robot description, xacro)
@@ -1,5 +1,8 @@
 <?xml version="1.0"?>
 <robot xmlns:xacro="http://www.ros.org/wiki/xacro" name="LBR3R760iisy">
-    <!-- Import iisy urdf file -->
-    <xacro:include filename="iisy.urdf" />
+<!-- Import iisy urdf file  -->
+<xacro:include filename="$(find kuka_iisy_support)/urdf/iisy.ros2_control.urdf.xacro"/>
+<xacro:eci_config client_ip="10.36.60.228"
+                  controller_ip="10.36.60.227"
+                  control_mode="position_control"/>
 </robot>

Commit message: add qos params to xacro

File: kuka_iisy_support/urdf/iisy.ros2_control.urdf.xacro (robot description, xacro)
@@ -1,5 +1,5 @@
 <?xml version="1.0" encoding="UTF-8"?>
 <robot name="LBR3R760iisy" xmlns:xacro="http://www.ros.org/wiki/xacro">
-  <xacro:macro name="eci_config" params="client_ip controller_ip control_mode">
+  <xacro:macro name="eci_config" params="client_ip controller_ip control_mode consequent_lost_packets lost_packets_in_timeframe timeframe_ms">
   <ros2_control name="iisy_hardware" type="system">
     <hardware>
@@ -8,4 +8,7 @@
       <param name="controller_ip">${controller_ip}</param>
       <param name="control_mode">${control_mode}</param>
+      <param name="consequent_lost_packets">${consequent_lost_packets}</param>
+      <param name="lost_packets_in_timeframe">${lost_packets_in_timeframe}</param>
+      <param name="timeframe_ms">${timeframe_ms}</param>
     </hardware>
     <!-- define joints and command/state interfaces for each joint -->

File: kuka_iisy_support/urdf/iisy.urdf.xacro (robot description, xacro)
@@ -3,11 +3,21 @@
 <!-- Import iisy urdf file  -->
 <xacro:include filename="$(find kuka_iisy_support)/urdf/iisy.ros2_control.urdf.xacro"/>
+<!-- Read parameters from eci_config  -->
 <xacro:property name="eci_config" value="$(find kuka_rox_hw_interface)/config/eci_config.yaml" />
-<xacro:property name="config_dict" value="${xacro.load_yaml(eci_config)}"/>
-<xacro:property name="control_mode" value="${config_dict['robot_manager']['ros__parameters']['control_mode']}" />
-<xacro:property name="client_ip" value="${config_dict['robot_manager']['ros__parameters']['client_ip']}" />
-<xacro:property name="controller_ip" value="${config_dict['robot_manager']['ros__parameters']['controller_ip']}" />
+<xacro:property name="eci_config_dict" value="${xacro.load_yaml(eci_config)}"/>
+<xacro:property name="control_mode" value="${eci_config_dict['robot_manager']['ros__parameters']['control_mode']}" />
+<xacro:property name="client_ip" value="${eci_config_dict['robot_manager']['ros__parameters']['client_ip']}" />
+<xacro:property name="controller_ip" value="${eci_config_dict['robot_manager']['ros__parameters']['controller_ip']}" />
+<!-- Read QoS profile parameters  -->
+<xacro:property name="qos_config" value="$(find kuka_rox_hw_interface)/config/qos_profiles.yaml" />
+<xacro:property name="qos_config_dict" value="${xacro.load_yaml(qos_config)}"/>
+<xacro:property name="consequent_lost_packets" value="${qos_config_dict['rt_packet_loss_profile']['consequent_lost_packets']}" />
+<xacro:property name="lost_packets_in_timeframe" value="${qos_config_dict['rt_packet_loss_profile']['lost_packets_in_timeframe']}" />
+<xacro:property name="timeframe_ms" value="${qos_config_dict['rt_packet_loss_profile']['timeframe_ms']}" />
 <xacro:eci_config client_ip="${client_ip}"
                   controller_ip="${controller_ip}"
-                  control_mode="${control_mode}"/>
+                  control_mode="${control_mode}"
+                  consequent_lost_packets="${consequent_lost_packets}"
+                  lost_packets_in_timeframe="${lost_packets_in_timeframe}"
+                  timeframe_ms="${timeframe_ms}"/>
 </robot>

Commit message: add link6-flange tf

File: kuka_iisy_support/urdf/iisy.ros2_control.urdf.xacro (robot description, xacro)
@@ -196,4 +196,5 @@
     </visual>
   </link>
+  <link name="LBR3R760_iisy_flange" />
   <joint name="base_joint" type="fixed">
     <parent link="base_link" />
@@ -242,4 +243,9 @@
     <parent link="LBR3R760_iisy_axis5"/>
   </joint>
+  <joint name="link6-flange" type="fixed">
+    <child link="LBR3R760_iisy_flange"/>
+    <origin rpy="0 1.5707963267948963 -0.0" xyz="0.0 0.0 -0.1605"/>
+    <parent link="LBR3R760_iisy_axis6"/>
+  </joint>
   <transmission name="trans_LBR3R760iisy_Urdf_Joint1_name">
     <actuator name="LBR3R760iisy_Urdf_Joint1_name_motor">
