Commit message: mesh file conventions

File: kuka_iisy_support/urdf/iisy_macro.xacro (robot description, xacro)
@@ -17,5 +17,5 @@
       <collision>
         <geometry>
-          <mesh filename="package://kuka_iisy_support/meshes/robotbase.stl" />
+          <mesh filename="package://kuka_iisy_support/meshes/LBR3R760/collision/base_link.stl" />
         </geometry>
         <origin rpy="-0.0 0.0 -0.0" xyz="0.0 0.0 0.0" />
@@ -28,5 +28,5 @@
       <visual>
         <geometry>
-          <mesh filename="package://kuka_iisy_support/meshes/robotbase.stl" />
+          <mesh filename="package://kuka_iisy_support/meshes/LBR3R760/visual/base_link.stl" />
         </geometry>
         <origin rpy="-0.0 0.0 -0.0" xyz="0.0 0.0 0.0" />
@@ -36,5 +36,5 @@
       <collision>
         <geometry>
-          <mesh filename="package://kuka_iisy_support/meshes/link1.stl" />
+          <mesh filename="package://kuka_iisy_support/meshes/LBR3R760/collision/link_1.stl" />
         </geometry>
         <origin rpy="-0.0 0.0 -0.0" xyz="0.0 0.0 0.0" />
@@ -47,5 +47,5 @@
       <visual>
         <geometry>
-          <mesh filename="package://kuka_iisy_support/meshes/link1.stl" />
+          <mesh filename="package://kuka_iisy_support/meshes/LBR3R760/visual/link_1.stl" />
         </geometry>
         <origin rpy="-0.0 0.0 -0.0" xyz="0.0 0.0 0.0" />
@@ -55,5 +55,5 @@
       <collision>
         <geometry>
-          <mesh filename="package://kuka_iisy_support/meshes/link2.stl" />
+          <mesh filename="package://kuka_iisy_support/meshes/LBR3R760/collision/link_2.stl" />
         </geometry>
         <origin rpy="-0.0 0.0 -0.0" xyz="0.0 0.0 0.0" />
@@ -66,5 +66,5 @@
       <visual>
         <geometry>
-          <mesh filename="package://kuka_iisy_support/meshes/link2.stl" />
+          <mesh filename="package://kuka_iisy_support/meshes/LBR3R760/visual/link_2.stl" />
         </geometry>
         <origin rpy="-0.0 0.0 -0.0" xyz="0.0 0.0 0.0" />
@@ -74,5 +74,5 @@
       <collision>
         <geometry>
-          <mesh filename="package://kuka_iisy_support/meshes/link3.stl" />
+          <mesh filename="package://kuka_iisy_support/meshes/LBR3R760/collision/link_3.stl" />
         </geometry>
         <origin rpy="-0.0 0.0 -0.0" xyz="0.0 0.0 0.0" />
@@ -85,5 +85,5 @@
       <visual>
         <geometry>
-          <mesh filename="package://kuka_iisy_support/meshes/link3.stl" />
+          <mesh filename="package://kuka_iisy_support/meshes/LBR3R760/visual/link_3.stl" />
         </geometry>
         <origin rpy="-0.0 0.0 -0.0" xyz="0.0 0.0 0.0" />
@@ -93,5 +93,5 @@
       <collision>
         <geometry>
-          <mesh filename="package://kuka_iisy_support/meshes/link4.stl" />
+          <mesh filename="package://kuka_iisy_support/meshes/LBR3R760/collision/link_4.stl" />
         </geometry>
         <origin rpy="-0.0 0.0 -0.0" xyz="0.0 0.0 0.0" />
@@ -104,5 +104,5 @@
       <visual>
         <geometry>
-          <mesh filename="package://kuka_iisy_support/meshes/link4.stl" />
+          <mesh filename="package://kuka_iisy_support/meshes/LBR3R760/visual/link_4.stl" />
         </geometry>
         <origin rpy="-0.0 0.0 -0.0" xyz="0.0 0.0 0.0" />
@@ -112,5 +112,5 @@
       <collision>
         <geometry>
-          <mesh filename="package://kuka_iisy_support/meshes/link5.stl" />
+          <mesh filename="package://kuka_iisy_support/meshes/LBR3R760/collision/link_5.stl" />
         </geometry>
         <origin rpy="-0.0 0.0 -0.0" xyz="0.0 0.0 0.0" />
@@ -123,5 +123,5 @@
       <visual>
         <geometry>
-          <mesh filename="package://kuka_iisy_support/meshes/link5.stl" />
+          <mesh filename="package://kuka_iisy_support/meshes/LBR3R760/visual/link_5.stl" />
         </geometry>
         <origin rpy="-0.0 0.0 -0.0" xyz="0.0 0.0 0.0" />
@@ -131,5 +131,5 @@
       <collision>
         <geometry>
-          <mesh filename="package://kuka_iisy_support/meshes/link6.stl" />
+          <mesh filename="package://kuka_iisy_support/meshes/LBR3R760/collision/link_6.stl" />
         </geometry>
         <origin rpy="-0.0 0.0 -0.0" xyz="0.0 0.0 0.0" />
@@ -142,5 +142,5 @@
       <visual>
         <geometry>
-          <mesh filename="package://kuka_iisy_support/meshes/link6.stl" />
+          <mesh filename="package://kuka_iisy_support/meshes/LBR3R760/visual/link_6.stl" />
         </geometry>
         <origin rpy="-0.0 0.0 -0.0" xyz="0.0 0.0 0.0" />
