Commit message: moveit config package conventions

File: kuka_lbr_iisy_moveit_config/srdf/lbr_iisy_arm.srdf.xacro (robot description, xacro)
@@ -4,6 +4,6 @@
     A URDF file must exist for this robot as well, where the joints and the links that are referenced are defined
 -->
-<robot xmlns:xacro="http://www.ros.org/wiki/xacro" name="LBR3R760iisy">
-  <xacro:include filename="iisy_arm.xacro" />
-  <xacro:iisy_arm />
+<robot xmlns:xacro="http://www.ros.org/wiki/xacro" name="LBRiisy3R760">
+  <xacro:include filename="lbr_iisy_arm.xacro" />
+  <xacro:kuka_lbr_iisy_arm />
 </robot>

File: kuka_lbr_iisy_moveit_config/srdf/lbr_iisy_arm.xacro (robot description, xacro)
@@ -1,5 +1,5 @@
 <?xml version="1.0" ?>
-<robot xmlns:xacro="http://www.ros.org/wiki/xacro" name="LBR3R760iisy">
-  <xacro:macro name="iisy_arm">
+<robot xmlns:xacro="http://www.ros.org/wiki/xacro" name="LBRiisy3R760">
+  <xacro:macro name="kuka_lbr_iisy_arm">
     <!--GROUPS: Representation of a set of joints and links. This can be useful for specifying DOF to plan for, defining arms, end effectors, etc-->
     <!--LINKS: When a link is specified, the parent joint of that link (if it exists) is automatically included-->
@@ -7,6 +7,6 @@
     <!--CHAINS: When a chain is specified, all the links along the chain (including endpoints) are included in the group. Additionally, all the joints that are parents to included links are also included. This means that joints along the chain and the parent joint of the base link are included in the group-->
     <!--SUBGROUPS: Groups can also be formed by referencing to already defined group names-->
-    <group name="iisy_arm">
-      <chain base_link="LBR3R760_iisy_fixedbase" tip_link="LBR3R760_iisy_flange" />
+    <group name="lbr_iisy_arm">
+      <chain base_link="base_link" tip_link="tool0" />
     </group>
     <!--GROUP STATES: Purpose: Define a named state for a particular group, in terms of joint values. This is useful to define states like 'folded arms'-->
@@ -20,13 +20,12 @@
     </group_state>
     <!--VIRTUAL JOINT: Purpose: this element defines a virtual joint between a robot link and an external frame of reference (considered fixed with respect to the robot)-->
-    <virtual_joint name="virtual_joint" type="floating" parent_frame="base_link" child_link="LBR3R760_iisy_fixedbase" />
+    <virtual_joint name="world_joint" type="fixed" parent_frame="world" child_link="base_link" />
     <!--DISABLE COLLISIONS: By default it is assumed that any link of the robot could potentially come into collision with any other link in the robot. This tag disables collision checking between a specified pair of links. -->
-    <disable_collisions link1="LBR3R760_iisy_fixedbase" link2="LBR3R760_iisy_axis1" reason="Adjacent"/>
-    <disable_collisions link1="LBR3R760_iisy_axis1" link2="LBR3R760_iisy_axis2" reason="Adjacent"/>
-    <disable_collisions link1="LBR3R760_iisy_axis2" link2="LBR3R760_iisy_axis3" reason="Adjacent"/>
-    <disable_collisions link1="LBR3R760_iisy_axis3" link2="LBR3R760_iisy_axis4" reason="Adjacent"/>
-    <disable_collisions link1="LBR3R760_iisy_axis4" link2="LBR3R760_iisy_axis5" reason="Adjacent"/>
-    <disable_collisions link1="LBR3R760_iisy_axis5" link2="LBR3R760_iisy_axis6" reason="Adjacent"/>
-    <disable_collisions link1="LBR3R760_iisy_axis6" link2="LBR3R760_iisy_flange" reason="Adjacent"/>
+    <disable_collisions link1="base_link" link2="link_1" reason="Adjacent"/>
+    <disable_collisions link1="link_1" link2="link_2" reason="Adjacent"/>
+    <disable_collisions link1="link_2" link2="link_3" reason="Adjacent"/>
+    <disable_collisions link1="link_3" link2="link_4" reason="Adjacent"/>
+    <disable_collisions link1="link_4" link2="link_5" reason="Adjacent"/>
+    <disable_collisions link1="link_5" link2="link_6" reason="Adjacent"/>
   </xacro:macro>
 </robot>
