Commit message: fix tool0 parent frame

File: kuka_lbr_iisy_moveit_config/srdf/lbr_iisy_arm.xacro (robot description, xacro)
@@ -11,5 +11,5 @@
     </group>
     <!--GROUP STATES: Purpose: Define a named state for a particular group, in terms of joint values. This is useful to define states like 'folded arms'-->
-    <group_state name="null_pos" group="iisy_arm">
+    <group_state name="null_pos" group="lbr_iisy_arm">
       <joint name="joint_a1" value="0" />
       <joint name="joint_a2" value="0" />
@@ -20,5 +20,5 @@
     </group_state>
     <!--VIRTUAL JOINT: Purpose: this element defines a virtual joint between a robot link and an external frame of reference (considered fixed with respect to the robot)-->
-    <virtual_joint name="world_joint" type="fixed" parent_frame="world" child_link="base_link" />
+    <!-- <virtual_joint name="world_joint" type="fixed" parent_frame="world" child_link="base_link" /> -->
     <!--DISABLE COLLISIONS: By default it is assumed that any link of the robot could potentially come into collision with any other link in the robot. This tag disables collision checking between a specified pair of links. -->
     <disable_collisions link1="base_link" link2="link_1" reason="Adjacent"/>

File: kuka_lbr_iisy_support/urdf/lbr_iisy3_r760_macro.xacro (robot description, xacro)
@@ -223,8 +223,8 @@
     <!-- ROS-Industrial 'tool0' frame - all-zeros tool frame -->
     <link name="${prefix}tool0" />
-    <joint name="${prefix}flange-tool0" type="fixed">
+    <joint name="${prefix}link6-tool0" type="fixed">
       <child link="${prefix}tool0" />
-      <origin rpy="0.0 0.0 0.0" xyz="0.0 0.0 0.0" />
-      <parent link="${prefix}flange" />
+      <origin rpy="0 ${pi} -0.0" xyz="0.0 0.0 -0.1605" />
+      <parent link="${prefix}link_6" />
     </joint>
   </xacro:macro>
