Commit message: add prefix to srdf

File: kuka_lbr_iisy_moveit_config/srdf/lbr_iisy_arm.macro.xacro (robot description, xacro)
@@ -1,5 +1,5 @@
 <?xml version="1.0" ?>
 <robot xmlns:xacro="http://www.ros.org/wiki/xacro" name="LBRiisy3R760">
-  <xacro:macro name="kuka_lbr_iisy_arm">
+  <xacro:macro name="kuka_lbr_iisy_arm" params="prefix">
     <!--GROUPS: Representation of a set of joints and links. This can be useful for specifying DOF to plan for, defining arms, end effectors, etc-->
     <!--LINKS: When a link is specified, the parent joint of that link (if it exists) is automatically included-->
@@ -8,24 +8,24 @@
     <!--SUBGROUPS: Groups can also be formed by referencing to already defined group names-->
     <group name="lbr_iisy_arm">
-      <chain base_link="base_link" tip_link="tool0" />
+      <chain base_link="${prefix}base_link" tip_link="${prefix}tool0" />
     </group>
     <!--GROUP STATES: Purpose: Define a named state for a particular group, in terms of joint values. This is useful to define states like 'folded arms'-->
     <group_state name="null_pos" group="lbr_iisy_arm">
-      <joint name="joint_a1" value="0" />
-      <joint name="joint_a2" value="0" />
-      <joint name="joint_a3" value="0" />
-      <joint name="joint_a4" value="0" />
-      <joint name="joint_a5" value="0" />
-      <joint name="joint_a6" value="0" />
+      <joint name="${prefix}joint_a1" value="0" />
+      <joint name="${prefix}joint_a2" value="0" />
+      <joint name="${prefix}joint_a3" value="0" />
+      <joint name="${prefix}joint_a4" value="0" />
+      <joint name="${prefix}joint_a5" value="0" />
+      <joint name="${prefix}joint_a6" value="0" />
     </group_state>
     <!--VIRTUAL JOINT: Purpose: this element defines a virtual joint between a robot link and an external frame of reference (considered fixed with respect to the robot)-->
     <!-- <virtual_joint name="world_joint" type="fixed" parent_frame="world" child_link="base_link" /> -->
     <!--DISABLE COLLISIONS: By default it is assumed that any link of the robot could potentially come into collision with any other link in the robot. This tag disables collision checking between a specified pair of links. -->
-    <disable_collisions link1="base_link_inertia" link2="link_1" reason="Adjacent"/>
-    <disable_collisions link1="link_1" link2="link_2" reason="Adjacent"/>
-    <disable_collisions link1="link_2" link2="link_3" reason="Adjacent"/>
-    <disable_collisions link1="link_3" link2="link_4" reason="Adjacent"/>
-    <disable_collisions link1="link_4" link2="link_5" reason="Adjacent"/>
-    <disable_collisions link1="link_5" link2="link_6" reason="Adjacent"/>
+    <disable_collisions link1="${prefix}base_link_inertia" link2="${prefix}link_1" reason="Adjacent"/>
+    <disable_collisions link1="${prefix}link_1" link2="${prefix}link_2" reason="Adjacent"/>
+    <disable_collisions link1="${prefix}link_2" link2="${prefix}link_3" reason="Adjacent"/>
+    <disable_collisions link1="${prefix}link_3" link2="${prefix}link_4" reason="Adjacent"/>
+    <disable_collisions link1="${prefix}link_4" link2="${prefix}link_5" reason="Adjacent"/>
+    <disable_collisions link1="${prefix}link_5" link2="${prefix}link_6" reason="Adjacent"/>
   </xacro:macro>
 </robot>

File: kuka_lbr_iisy_moveit_config/srdf/lbr_iisy_arm.srdf.xacro (robot description, xacro)
@@ -6,4 +6,4 @@
 <robot xmlns:xacro="http://www.ros.org/wiki/xacro" name="LBRiisy3R760">
   <xacro:include filename="lbr_iisy_arm.macro.xacro" />
-  <xacro:kuka_lbr_iisy_arm />
+  <xacro:kuka_lbr_iisy_arm prefix=""/>
 </robot>

Commit message: update rviz config and srdf

File: kuka_lbr_iisy_moveit_config/srdf/lbr_iisy_arm.macro.xacro (robot description, xacro)
@@ -8,5 +8,9 @@
     <!--SUBGROUPS: Groups can also be formed by referencing to already defined group names-->
     <group name="lbr_iisy_arm">
-      <chain base_link="${prefix}base_link" tip_link="${prefix}tool0" />
+      <chain base_link="${prefix}base_link" tip_link="${prefix}flange" />
+    </group>
+    <!--Add flange as end effector to be able to use moveit_visual_tools for visualising end effector path-->
+    <group name="end_effector">
+      <link name="${prefix}flange"/>
     </group>
     <!--GROUP STATES: Purpose: Define a named state for a particular group, in terms of joint values. This is useful to define states like 'folded arms'-->
@@ -21,4 +25,6 @@
     <!--VIRTUAL JOINT: Purpose: this element defines a virtual joint between a robot link and an external frame of reference (considered fixed with respect to the robot)-->
     <!-- <virtual_joint name="world_joint" type="fixed" parent_frame="world" child_link="base_link" /> -->
+    <!--END EFFECTOR: Purpose: Represent information about an end effector.-->
+    <end_effector name="flange" parent_link="${prefix}flange" group="end_effector" parent_group="lbr_iisy_arm"/>
     <!--DISABLE COLLISIONS: By default it is assumed that any link of the robot could potentially come into collision with any other link in the robot. This tag disables collision checking between a specified pair of links. -->
     <disable_collisions link1="${prefix}base_link_inertia" link2="${prefix}link_1" reason="Adjacent"/>
