Commit message: use lower case letters

File: kuka_lbr_iisy_moveit_config/srdf/lbr_iisy11_r1300_arm.srdf.xacro (robot description, xacro)
@@ -4,5 +4,5 @@
     A URDF file must exist for this robot as well, where the joints and the links that are referenced are defined
 -->
-<robot xmlns:xacro="http://www.ros.org/wiki/xacro" name="LBRiisy11R1300">
+<robot xmlns:xacro="http://www.ros.org/wiki/xacro" name="lbr_iisy11_r1300">
   <xacro:include filename="lbr_iisy_arm.macro.xacro" />
   <xacro:kuka_lbr_iisy_arm prefix=""/>

File: kuka_lbr_iisy_moveit_config/srdf/lbr_iisy15_r930_arm.srdf.xacro (robot description, xacro)
@@ -4,5 +4,5 @@
     A URDF file must exist for this robot as well, where the joints and the links that are referenced are defined
 -->
-<robot xmlns:xacro="http://www.ros.org/wiki/xacro" name="LBRiisy15R930">
+<robot xmlns:xacro="http://www.ros.org/wiki/xacro" name="lbr_iisy15_r930">
   <xacro:include filename="lbr_iisy_arm.macro.xacro" />
   <xacro:kuka_lbr_iisy_arm prefix=""/>

File: kuka_lbr_iisy_moveit_config/srdf/lbr_iisy3_r760_arm.srdf.xacro (robot description, xacro)
@@ -4,5 +4,5 @@
     A URDF file must exist for this robot as well, where the joints and the links that are referenced are defined
 -->
-<robot xmlns:xacro="http://www.ros.org/wiki/xacro" name="LBRiisy3R760">
+<robot xmlns:xacro="http://www.ros.org/wiki/xacro" name="lbr_iisy3_r760">
   <xacro:include filename="lbr_iisy_arm.macro.xacro" />
   <xacro:kuka_lbr_iisy_arm prefix=""/>

File: kuka_lbr_iisy_support/urdf/lbr_iisy11_r1300.urdf.xacro (robot description, xacro)
@@ -1,4 +1,4 @@
 <?xml version="1.0"?>
-<robot xmlns:xacro="http://www.ros.org/wiki/xacro" name="LBRiisy11R1300">
+<robot xmlns:xacro="http://www.ros.org/wiki/xacro" name="lbr_iisy11_r1300">
 <!-- Import iisy urdf file  -->
 <xacro:include filename="$(find kuka_lbr_iisy_support)/urdf/lbr_iisy11_r1300_macro.xacro"/>

File: kuka_lbr_iisy_support/urdf/lbr_iisy11_r1300_macro.xacro (robot description, xacro)
@@ -1,4 +1,4 @@
 <?xml version="1.0" encoding="UTF-8"?>
-<robot xmlns:xacro="http://www.ros.org/wiki/xacro" name="LBRiisy11R1300">
+<robot xmlns:xacro="http://www.ros.org/wiki/xacro" name="lbr_iisy11_r1300">
   <!-- include helper xacros -->
   <xacro:include filename="$(find kuka_lbr_iisy_support)/urdf/lbr_iisy_ros2_control.xacro" />
@@ -8,5 +8,5 @@
     <!-- ros2 control instance -->
     <xacro:kuka_lbr_iisy_ros2_control
-    name="LBRiisy11R1300"
+    name="lbr_iisy11_r1300"
     prefix="${prefix}"
     client_ip="${client_ip}"
@@ -22,5 +22,5 @@
       <collision>
         <geometry>
-          <mesh filename="package://kuka_lbr_iisy_support/meshes/LBRiisy11R1300/collision/base_link.stl" />
+          <mesh filename="package://kuka_lbr_iisy_support/meshes/lbr_iisy11_r1300/collision/base_link.stl" />
         </geometry>
         <origin rpy="-0.0 0.0 -0.0" xyz="0.0 0.0 0.0" />
@@ -33,5 +33,5 @@
       <visual>
         <geometry>
-          <mesh filename="package://kuka_lbr_iisy_support/meshes/LBRiisy11R1300/visual/base_link.stl" />
+          <mesh filename="package://kuka_lbr_iisy_support/meshes/lbr_iisy11_r1300/visual/base_link.stl" />
         </geometry>
         <origin rpy="-0.0 0.0 -0.0" xyz="0.0 0.0 0.0" />
@@ -42,5 +42,5 @@
       <collision>
         <geometry>
-          <mesh filename="package://kuka_lbr_iisy_support/meshes/LBRiisy11R1300/collision/link_1.stl" />
+          <mesh filename="package://kuka_lbr_iisy_support/meshes/lbr_iisy11_r1300/collision/link_1.stl" />
         </geometry>
         <origin rpy="-0.0 0.0 -0.0" xyz="0.0 0.0 0.0" />
@@ -53,5 +53,5 @@
       <visual>
         <geometry>
-          <mesh filename="package://kuka_lbr_iisy_support/meshes/LBRiisy11R1300/visual/link_1.stl" />
+          <mesh filename="package://kuka_lbr_iisy_support/meshes/lbr_iisy11_r1300/visual/link_1.stl" />
         </geometry>
         <origin rpy="-0.0 0.0 -0.0" xyz="0.0 0.0 0.0" />
@@ -62,5 +62,5 @@
       <collision>
         <geometry>
-          <mesh filename="package://kuka_lbr_iisy_support/meshes/LBRiisy11R1300/collision/link_2.stl" />
+          <mesh filename="package://kuka_lbr_iisy_support/meshes/lbr_iisy11_r1300/collision/link_2.stl" />
         </geometry>
         <origin rpy="-0.0 0.0 -0.0" xyz="0.0 0.0 0.0" />
@@ -73,5 +73,5 @@
       <visual>
         <geometry>
-          <mesh filename="package://kuka_lbr_iisy_support/meshes/LBRiisy11R1300/visual/link_2.stl" />
+          <mesh filename="package://kuka_lbr_iisy_support/meshes/lbr_iisy11_r1300/visual/link_2.stl" />
         </geometry>
         <origin rpy="-0.0 0.0 -0.0" xyz="0.0 0.0 0.0" />
@@ -82,5 +82,5 @@
       <collision>
         <geometry>
-          <mesh filename="package://kuka_lbr_iisy_support/meshes/LBRiisy11R1300/collision/link_3.stl" />
+          <mesh filename="package://kuka_lbr_iisy_support/meshes/lbr_iisy11_r1300/collision/link_3.stl" />
         </geometry>
         <origin rpy="-0.0 0.0 -0.0" xyz="0.0 0.0 0.0" />
@@ -93,5 +93,5 @@
       <visual>
         <geometry>
-          <mesh filename="package://kuka_lbr_iisy_support/meshes/LBRiisy11R1300/visual/link_3.stl" />
+          <mesh filename="package://kuka_lbr_iisy_support/meshes/lbr_iisy11_r1300/visual/link_3.stl" />
         </geometry>
         <origin rpy="-0.0 0.0 -0.0" xyz="0.0 0.0 0.0" />
@@ -102,5 +102,5 @@
       <collision>
         <geometry>
-          <mesh filename="package://kuka_lbr_iisy_support/meshes/LBRiisy11R1300/collision/link_4.stl" />
+          <mesh filename="package://kuka_lbr_iisy_support/meshes/lbr_iisy11_r1300/collision/link_4.stl" />
         </geometry>
         <origin rpy="-0.0 0.0 -0.0" xyz="0.0 0.0 0.0" />
@@ -113,5 +113,5 @@
       <visual>
         <geometry>
-          <mesh filename="package://kuka_lbr_iisy_support/meshes/LBRiisy11R1300/visual/link_4.stl" />
+          <mesh filename="package://kuka_lbr_iisy_support/meshes/lbr_iisy11_r1300/visual/link_4.stl" />
         </geometry>
         <origin rpy="-0.0 0.0 -0.0" xyz="0.0 0.0 0.0" />
@@ -122,5 +122,5 @@
       <collision>
         <geometry>
-          <mesh filename="package://kuka_lbr_iisy_support/meshes/LBRiisy11R1300/collision/link_5.stl" />
+          <mesh filename="package://kuka_lbr_iisy_support/meshes/lbr_iisy11_r1300/collision/link_5.stl" />
         </geometry>
         <origin rpy="-0.0 0.0 -0.0" xyz="0.0 0.0 0.0" />
@@ -133,5 +133,5 @@
       <visual>
         <geometry>
-          <mesh filename="package://kuka_lbr_iisy_support/meshes/LBRiisy11R1300/visual/link_5.stl" />
+          <mesh filename="package://kuka_lbr_iisy_support/meshes/lbr_iisy11_r1300/visual/link_5.stl" />
         </geometry>
         <origin rpy="-0.0 0.0 -0.0" xyz="0.0 0.0 0.0" />
@@ -142,5 +142,5 @@
       <collision>
         <geometry>
-          <mesh filename="package://kuka_lbr_iisy_support/meshes/LBRiisy11R1300/collision/link_6.stl" />
+          <mesh filename="package://kuka_lbr_iisy_support/meshes/lbr_iisy11_r1300/collision/link_6.stl" />
         </geometry>
         <origin rpy="-0.0 0.0 -0.0" xyz="0.0 0.0 0.0" />
@@ -153,5 +153,5 @@
       <visual>
         <geometry>
-          <mesh filename="package://kuka_lbr_iisy_support/meshes/LBRiisy11R1300/visual/link_6.stl" />
+          <mesh filename="package://kuka_lbr_iisy_support/meshes/lbr_iisy11_r1300/visual/link_6.stl" />
         </geometry>
         <origin rpy="-0.0 0.0 -0.0" xyz="0.0 0.0 0.0" />

File: kuka_lbr_iisy_support/urdf/lbr_iisy15_r930.urdf.xacro (robot description, xacro)
@@ -1,4 +1,4 @@
 <?xml version="1.0"?>
-<robot xmlns:xacro="http://www.ros.org/wiki/xacro" name="LBRiisy15R930">
+<robot xmlns:xacro="http://www.ros.org/wiki/xacro" name="lbr_iisy15_r930">
 <!-- Import iisy urdf file  -->
 <xacro:include filename="$(find kuka_lbr_iisy_support)/urdf/lbr_iisy15_r930_macro.xacro"/>

File: kuka_lbr_iisy_support/urdf/lbr_iisy15_r930_macro.xacro (robot description, xacro)
@@ -1,4 +1,4 @@
 <?xml version="1.0" encoding="UTF-8"?>
-<robot xmlns:xacro="http://www.ros.org/wiki/xacro" name="LBRiisy15R930">
+<robot xmlns:xacro="http://www.ros.org/wiki/xacro" name="lbr_iisy15_r930">
   <!-- include helper xacros -->
   <xacro:include filename="$(find kuka_lbr_iisy_support)/urdf/lbr_iisy_ros2_control.xacro" />
@@ -8,5 +8,5 @@
     <!-- ros2 control instance -->
     <xacro:kuka_lbr_iisy_ros2_control
-    name="LBRiisy15R930"
+    name="lbr_iisy15_r930"
     prefix="${prefix}"
     client_ip="${client_ip}"
@@ -22,5 +22,5 @@
       <collision>
         <geometry>
-          <mesh filename="package://kuka_lbr_iisy_support/meshes/LBRiisy15R930/collision/base_link.stl" />
+          <mesh filename="package://kuka_lbr_iisy_support/meshes/lbr_iisy15_r930/collision/base_link.stl" />
         </geometry>
         <origin rpy="-0.0 0.0 -0.0" xyz="0.0 0.0 0.0" />
@@ -33,5 +33,5 @@
       <visual>
         <geometry>
-          <mesh filename="package://kuka_lbr_iisy_support/meshes/LBRiisy15R930/visual/base_link.stl" />
+          <mesh filename="package://kuka_lbr_iisy_support/meshes/lbr_iisy15_r930/visual/base_link.stl" />
         </geometry>
         <origin rpy="-0.0 0.0 -0.0" xyz="0.0 0.0 0.0" />
@@ -42,5 +42,5 @@
       <collision>
         <geometry>
-          <mesh filename="package://kuka_lbr_iisy_support/meshes/LBRiisy15R930/collision/link_1.stl" />
+          <mesh filename="package://kuka_lbr_iisy_support/meshes/lbr_iisy15_r930/collision/link_1.stl" />
         </geometry>
         <origin rpy="-0.0 0.0 -0.0" xyz="0.0 0.0 0.0" />
@@ -53,5 +53,5 @@
       <visual>
         <geometry>
-          <mesh filename="package://kuka_lbr_iisy_support/meshes/LBRiisy15R930/visual/link_1.stl" />
+          <mesh filename="package://kuka_lbr_iisy_support/meshes/lbr_iisy15_r930/visual/link_1.stl" />
         </geometry>
         <origin rpy="-0.0 0.0 -0.0" xyz="0.0 0.0 0.0" />
@@ -62,5 +62,5 @@
       <collision>
         <geometry>
-          <mesh filename="package://kuka_lbr_iisy_support/meshes/LBRiisy15R930/collision/link_2.stl" />
+          <mesh filename="package://kuka_lbr_iisy_support/meshes/lbr_iisy15_r930/collision/link_2.stl" />
         </geometry>
         <origin rpy="-0.0 0.0 -0.0" xyz="0.0 0.0 0.0" />
@@ -73,5 +73,5 @@
       <visual>
         <geometry>
-          <mesh filename="package://kuka_lbr_iisy_support/meshes/LBRiisy15R930/visual/link_2.stl" />
+          <mesh filename="package://kuka_lbr_iisy_support/meshes/lbr_iisy15_r930/visual/link_2.stl" />
         </geometry>
         <origin rpy="-0.0 0.0 -0.0" xyz="0.0 0.0 0.0" />
@@ -82,5 +82,5 @@
       <collision>
         <geometry>
-          <mesh filename="package://kuka_lbr_iisy_support/meshes/LBRiisy15R930/collision/link_3.stl" />
+          <mesh filename="package://kuka_lbr_iisy_support/meshes/lbr_iisy15_r930/collision/link_3.stl" />
         </geometry>
         <origin rpy="-0.0 0.0 -0.0" xyz="0.0 0.0 0.0" />
@@ -93,5 +93,5 @@
       <visual>
         <geometry>
-          <mesh filename="package://kuka_lbr_iisy_support/meshes/LBRiisy15R930/visual/link_3.stl" />
+          <mesh filename="package://kuka_lbr_iisy_support/meshes/lbr_iisy15_r930/visual/link_3.stl" />
         </geometry>
         <origin rpy="-0.0 0.0 -0.0" xyz="0.0 0.0 0.0" />
@@ -102,5 +102,5 @@
       <collision>
         <geometry>
-          <mesh filename="package://kuka_lbr_iisy_support/meshes/LBRiisy15R930/collision/link_4.stl" />
+          <mesh filename="package://kuka_lbr_iisy_support/meshes/lbr_iisy15_r930/collision/link_4.stl" />
         </geometry>
         <origin rpy="-0.0 0.0 -0.0" xyz="0.0 0.0 0.0" />
@@ -113,5 +113,5 @@
       <visual>
         <geometry>
-          <mesh filename="package://kuka_lbr_iisy_support/meshes/LBRiisy15R930/visual/link_4.stl" />
+          <mesh filename="package://kuka_lbr_iisy_support/meshes/lbr_iisy15_r930/visual/link_4.stl" />
         </geometry>
         <origin rpy="-0.0 0.0 -0.0" xyz="0.0 0.0 0.0" />
@@ -122,5 +122,5 @@
       <collision>
         <geometry>
-          <mesh filename="package://kuka_lbr_iisy_support/meshes/LBRiisy15R930/collision/link_5.stl" />
+          <mesh filename="package://kuka_lbr_iisy_support/meshes/lbr_iisy15_r930/collision/link_5.stl" />
         </geometry>
         <origin rpy="-0.0 0.0 -0.0" xyz="0.0 0.0 0.0" />
@@ -133,5 +133,5 @@
       <visual>
         <geometry>
-          <mesh filename="package://kuka_lbr_iisy_support/meshes/LBRiisy15R930/visual/link_5.stl" />
+          <mesh filename="package://kuka_lbr_iisy_support/meshes/lbr_iisy15_r930/visual/link_5.stl" />
         </geometry>
         <origin rpy="-0.0 0.0 -0.0" xyz="0.0 0.0 0.0" />
@@ -142,5 +142,5 @@
       <collision>
         <geometry>
-          <mesh filename="package://kuka_lbr_iisy_support/meshes/LBRiisy15R930/collision/link_6.stl" />
+          <mesh filename="package://kuka_lbr_iisy_support/meshes/lbr_iisy15_r930/collision/link_6.stl" />
         </geometry>
         <origin rpy="-0.0 0.0 -0.0" xyz="0.0 0.0 0.0" />
@@ -153,5 +153,5 @@
       <visual>
         <geometry>
-          <mesh filename="package://kuka_lbr_iisy_support/meshes/LBRiisy15R930/visual/link_6.stl" />
+          <mesh filename="package://kuka_lbr_iisy_support/meshes/lbr_iisy15_r930/visual/link_6.stl" />
         </geometry>
         <origin rpy="-0.0 0.0 -0.0" xyz="0.0 0.0 0.0" />

File: kuka_lbr_iisy_support/urdf/lbr_iisy3_r760.urdf.xacro (robot description, xacro)
@@ -1,4 +1,4 @@
 <?xml version="1.0"?>
-<robot xmlns:xacro="http://www.ros.org/wiki/xacro" name="LBRiisy3R760">
+<robot xmlns:xacro="http://www.ros.org/wiki/xacro" name="lbr_iisy3_r760">
 <!-- Import iisy urdf file  -->
 <xacro:include filename="$(find kuka_lbr_iisy_support)/urdf/lbr_iisy3_r760_macro.xacro"/>

File: kuka_lbr_iisy_support/urdf/lbr_iisy3_r760_macro.xacro (robot description, xacro)
@@ -1,4 +1,4 @@
 <?xml version="1.0" encoding="UTF-8"?>
-<robot xmlns:xacro="http://www.ros.org/wiki/xacro" name="LBRiisy3R760">
+<robot xmlns:xacro="http://www.ros.org/wiki/xacro" name="lbr_iisy3_r760">
   <!-- include helper xacros -->
   <xacro:include filename="$(find kuka_lbr_iisy_support)/urdf/lbr_iisy_ros2_control.xacro" />
@@ -8,5 +8,5 @@
     <!-- ros2 control instance -->
     <xacro:kuka_lbr_iisy_ros2_control
-    name="LBRiisy3R760"
+    name="lbr_iisy3_r760"
     prefix="${prefix}"
     client_ip="${client_ip}"
@@ -23,5 +23,5 @@
       <collision>
         <geometry>
-          <mesh filename="package://kuka_lbr_iisy_support/meshes/LBRiisy3R760/collision/base_link.stl" />
+          <mesh filename="package://kuka_lbr_iisy_support/meshes/lbr_iisy3_r760/collision/base_link.stl" />
         </geometry>
         <origin rpy="-0.0 0.0 -0.0" xyz="0.0 0.0 0.0" />
@@ -34,5 +34,5 @@
       <visual>
         <geometry>
-          <mesh filename="package://kuka_lbr_iisy_support/meshes/LBRiisy3R760/visual/base_link.stl" />
+          <mesh filename="package://kuka_lbr_iisy_support/meshes/lbr_iisy3_r760/visual/base_link.stl" />
         </geometry>
         <origin rpy="-0.0 0.0 -0.0" xyz="0.0 0.0 0.0" />
@@ -43,5 +43,5 @@
       <collision>
         <geometry>
-          <mesh filename="package://kuka_lbr_iisy_support/meshes/LBRiisy3R760/collision/link_1.stl" />
+          <mesh filename="package://kuka_lbr_iisy_support/meshes/lbr_iisy3_r760/collision/link_1.stl" />
         </geometry>
         <origin rpy="-0.0 0.0 -0.0" xyz="0.0 0.0 0.0" />
@@ -54,5 +54,5 @@
       <visual>
         <geometry>
-          <mesh filename="package://kuka_lbr_iisy_support/meshes/LBRiisy3R760/visual/link_1.stl" />
+          <mesh filename="package://kuka_lbr_iisy_support/meshes/lbr_iisy3_r760/visual/link_1.stl" />
         </geometry>
         <origin rpy="-0.0 0.0 -0.0" xyz="0.0 0.0 0.0" />
@@ -63,5 +63,5 @@
       <collision>
         <geometry>
-          <mesh filename="package://kuka_lbr_iisy_support/meshes/LBRiisy3R760/collision/link_2.stl" />
+          <mesh filename="package://kuka_lbr_iisy_support/meshes/lbr_iisy3_r760/collision/link_2.stl" />
         </geometry>
         <origin rpy="-0.0 0.0 -0.0" xyz="0.0 0.0 0.0" />
@@ -74,5 +74,5 @@
       <visual>
         <geometry>
-          <mesh filename="package://kuka_lbr_iisy_support/meshes/LBRiisy3R760/visual/link_2.stl" />
+          <mesh filename="package://kuka_lbr_iisy_support/meshes/lbr_iisy3_r760/visual/link_2.stl" />
         </geometry>
         <origin rpy="-0.0 0.0 -0.0" xyz="0.0 0.0 0.0" />
@@ -83,5 +83,5 @@
       <collision>
         <geometry>
-          <mesh filename="package://kuka_lbr_iisy_support/meshes/LBRiisy3R760/collision/link_3.stl" />
+          <mesh filename="package://kuka_lbr_iisy_support/meshes/lbr_iisy3_r760/collision/link_3.stl" />
         </geometry>
         <origin rpy="-0.0 0.0 -0.0" xyz="0.0 0.0 0.0" />
@@ -94,5 +94,5 @@
       <visual>
         <geometry>
-          <mesh filename="package://kuka_lbr_iisy_support/meshes/LBRiisy3R760/visual/link_3.stl" />
+          <mesh filename="package://kuka_lbr_iisy_support/meshes/lbr_iisy3_r760/visual/link_3.stl" />
         </geometry>
         <origin rpy="-0.0 0.0 -0.0" xyz="0.0 0.0 0.0" />
@@ -103,5 +103,5 @@
       <collision>
         <geometry>
-          <mesh filename="package://kuka_lbr_iisy_support/meshes/LBRiisy3R760/collision/link_4.stl" />
+          <mesh filename="package://kuka_lbr_iisy_support/meshes/lbr_iisy3_r760/collision/link_4.stl" />
         </geometry>
         <origin rpy="-0.0 0.0 -0.0" xyz="0.0 0.0 0.0" />
@@ -114,5 +114,5 @@
       <visual>
         <geometry>
-          <mesh filename="package://kuka_lbr_iisy_support/meshes/LBRiisy3R760/visual/link_4.stl" />
+          <mesh filename="package://kuka_lbr_iisy_support/meshes/lbr_iisy3_r760/visual/link_4.stl" />
         </geometry>
         <origin rpy="-0.0 0.0 -0.0" xyz="0.0 0.0 0.0" />
@@ -123,5 +123,5 @@
       <collision>
         <geometry>
-          <mesh filename="package://kuka_lbr_iisy_support/meshes/LBRiisy3R760/collision/link_5.stl" />
+          <mesh filename="package://kuka_lbr_iisy_support/meshes/lbr_iisy3_r760/collision/link_5.stl" />
         </geometry>
         <origin rpy="-0.0 0.0 -0.0" xyz="0.0 0.0 0.0" />
@@ -134,5 +134,5 @@
       <visual>
         <geometry>
-          <mesh filename="package://kuka_lbr_iisy_support/meshes/LBRiisy3R760/visual/link_5.stl" />
+          <mesh filename="package://kuka_lbr_iisy_support/meshes/lbr_iisy3_r760/visual/link_5.stl" />
         </geometry>
         <origin rpy="-0.0 0.0 -0.0" xyz="0.0 0.0 0.0" />
@@ -143,5 +143,5 @@
       <collision>
         <geometry>
-          <mesh filename="package://kuka_lbr_iisy_support/meshes/LBRiisy3R760/collision/link_6.stl" />
+          <mesh filename="package://kuka_lbr_iisy_support/meshes/lbr_iisy3_r760/collision/link_6.stl" />
         </geometry>
         <origin rpy="-0.0 0.0 -0.0" xyz="0.0 0.0 0.0" />
@@ -154,5 +154,5 @@
       <visual>
         <geometry>
-          <mesh filename="package://kuka_lbr_iisy_support/meshes/LBRiisy3R760/visual/link_6.stl" />
+          <mesh filename="package://kuka_lbr_iisy_support/meshes/lbr_iisy3_r760/visual/link_6.stl" />
         </geometry>
         <origin rpy="-0.0 0.0 -0.0" xyz="0.0 0.0 0.0" />
