Commit message: modified urdf and launch to support rviz visual

File: kuka_mobile_robot_support/urdf/DifferentialMR.urdf (robot description, URDF)
Before this commit: robot genericMR_37146123288, 11 links, 10 joints
Links:
- added link generic_mr_body_dummy
- link caster_base_bl_link: geometry collision mesh filename=package://kuka_mobile_robot_support/meshes/37152976775.stl; visual mesh filename=package://kuka_mobile_robot_support/meshes/37152984509.stl
- link caster_base_br_link: geometry collision mesh filename=package://kuka_mobile_robot_support/meshes/37153311411.stl; visual mesh filename=package://kuka_mobile_robot_support/meshes/37153318102.stl
- link caster_base_fl_link: geometry collision mesh filename=package://kuka_mobile_robot_support/meshes/37153528620.stl; visual mesh filename=package://kuka_mobile_robot_support/meshes/37153537063.stl
- link caster_base_rl_link: geometry collision mesh filename=package://kuka_mobile_robot_support/meshes/37153636399.stl; visual mesh filename=package://kuka_mobile_robot_support/meshes/37153643851.stl
- link caster_wheel_bl_link: geometry collision mesh filename=package://kuka_mobile_robot_support/meshes/37149321854.stl; visual mesh filename=package://kuka_mobile_robot_support/meshes/37149329314.stl
- link caster_wheel_br_link: geometry collision mesh filename=package://kuka_mobile_robot_support/meshes/37149321854.stl; visual mesh filename=package://kuka_mobile_robot_support/meshes/37149329314.stl
- link caster_wheel_rl_link: geometry collision mesh filename=package://kuka_mobile_robot_support/meshes/37149321854.stl; visual mesh filename=package://kuka_mobile_robot_support/meshes/37149329314.stl
- link left_wheel: geometry collision mesh filename=package://kuka_mobile_robot_support/meshes/37153975930.stl; visual mesh filename=package://kuka_mobile_robot_support/meshes/37153983406.stl
- link right_wheel: geometry collision mesh filename=package://kuka_mobile_robot_support/meshes/37154306984.stl; visual mesh filename=package://kuka_mobile_robot_support/meshes/37154317878.stl
Joints:
- added joint generic_mr_body_dummy: type fixed, parent generic_mr_body_dummy, child generic_mr_body, origin xyz=0 0 0 rpy=0 0 0

File: kuka_mobile_robot_support/urdf/diffbot_kuka_macro.xacro (robot description, xacro)
@@ -17,5 +17,282 @@
     <!-- Include and instatiate diffbot description urdf file-->
     <xacro:include filename="$(find kuka_mobile_robot_support)/urdf/diffbot_description.urdf.xacro" />
-    <xacro:diffbot prefix="${prefix}" />
+    <!--xacro:genericMR_37146123288 prefix="${prefix}" /-->
+      <joint name="generic_mr_body_dummy" type="fixed">
+            <parent link="generic_mr_body_dummy" />
+            <child link="generic_mr_body" />
+            <origin xyz="0 0 0" rpy="0 0 0" />
+          </joint>
+        <joint name="caster_wheel_br_joint" type="fixed">
+          <axis xyz="0.0 1.0 0.0"/>
+          <child link="caster_wheel_br_link"/>
+          <origin rpy="-0.0 0.0 -0.0" xyz="-0.015 0.0 -0.026"/>
+          <parent link="caster_base_br_link"/>
+        </joint>
+        <joint name="left_wheel_motor" type="continuous">
+          <axis xyz="0.0 1.0 0.0"/>
+          <child link="left_wheel"/>
+          <limit effort="5.0E2" velocity="1.0E2"/>
+          <origin rpy="-0.0 0.0 -0.0" xyz="0.0 0.325 0.06"/>
+          <parent link="generic_mr_body"/>
+        </joint>
+        <joint name="right_wheel_motor" type="continuous">
+          <axis xyz="0.0 1.0 0.0"/>
+          <child link="right_wheel"/>
+          <limit effort="5.0E2" velocity="1.0E1"/>
+          <origin rpy="-0.0 0.0 -0.0" xyz="0.0 -0.325 0.0"/>
+          <parent link="generic_mr_body"/>
+        </joint>
+        <joint name="caster_base_fl_joint" type="fixed">
+          <axis xyz="0.0 0.0 1.0"/>
+          <child link="caster_base_fl_link"/>
+          <origin rpy="-0.0 0.0 -0.0" xyz="0.48 0.27 0.055"/>
+          <parent link="generic_mr_body"/>
+        </joint>
+        <joint name="caster_base_rl_joint" type="fixed">
+          <axis xyz="0.0 0.0 1.0"/>
+          <child link="caster_base_rl_link"/>
+          <origin rpy="-0.0 0.0 -0.0" xyz="0.48 -0.27 0.055"/>
+          <parent link="generic_mr_body"/>
+        </joint>
+        <joint name="caster_base_bl_joint" type="fixed">
+          <axis xyz="0.0 0.0 1.0"/>
+          <child link="caster_base_bl_link"/>
+          <origin rpy="-0.0 0.0 -0.0" xyz="-0.48 0.27 0.055"/>
+          <parent link="generic_mr_body"/>
+        </joint>
+        <joint name="caster_base_br_joint" type="fixed">
+          <axis xyz="0.0 0.0 1.0"/>
+          <child link="caster_base_br_link"/>
+          <origin rpy="-0.0 0.0 -0.0" xyz="-0.48 -0.27 0.055"/>
+          <parent link="generic_mr_body"/>
+        </joint>
+        <joint name="caster_wheel_fl_joint" type="fixed">
+          <axis xyz="0.0 1.0 0.0"/>
+          <child link="caster_wheel_fl_link"/>
+          <origin rpy="-0.0 0.0 -0.0" xyz="-0.015 0.0 -0.026"/>
+          <parent link="caster_base_fl_link"/>
+        </joint>
+        <joint name="caster_wheel_rl_joint" type="fixed">
+          <axis xyz="0.0 1.0 0.0"/>
+          <child link="caster_wheel_rl_link"/>
+          <origin rpy="-0.0 0.0 -0.0" xyz="-0.015 0.0 -0.026"/>
+          <parent link="caster_base_rl_link"/>
+        </joint>
+        <joint name="caster_wheel_bl_joint" type="fixed">
+          <axis xyz="0.0 1.0 0.0"/>
+          <child link="caster_wheel_bl_link"/>
+          <origin rpy="-0.0 0.0 -0.0" xyz="-0.015 0.0 -0.026"/>
+          <parent link="caster_base_bl_link"/>
+        </joint>
+        <link name="generic_mr_body_dummy"/>
+        <link name="generic_mr_body">
+          <collision>
+            <geometry>
+              <mesh filename="package://kuka_mobile_robot_support/meshes/37156934227.stl"/>
+            </geometry>
+            <origin rpy="-0.0 0.0 -0.0" xyz="0.0 0.0 0.0"/>
+          </collision>
+          <inertial>
+            <inertia ixx="5.0" ixy="0.0" ixz="0.0" iyy="10.0" iyz="0.0" izz="10.0"/>
+            <mass value="1.0E1"/>
+            <origin rpy="-0.0 0.0 -0.0" xyz="0.0 0.0 0.325"/>
+          </inertial>
+          <visual>
+            <geometry>
+              <mesh filename="package://kuka_mobile_robot_support/meshes/37156942086.stl"/>
+            </geometry>
+            <origin rpy="-0.0 0.0 -0.0" xyz="0.0 0.0 0.0"/>
+          </visual>
+        </link>
+        <link name="caster_wheel_fl_link">
+          <collision>
+            <geometry>
+              <mesh filename="package://kuka_mobile_robot_support/meshes/37149321854.stl"/>
+            </geometry>
+            <origin rpy="1.5707963267948963 0.0 -0.0" xyz="0.0 0.0 0.0"/>
+          </collision>
+          <inertial>
+            <inertia ixx="1.0E-4" ixy="0.0" ixz="0.0" iyy="1.0E-4" iyz="0.0" izz="1.0E-4"/>
+            <mass value="1.0E-1"/>
+            <origin rpy="-0.0 0.0 -0.0" xyz="0.0 0.0 0.0"/>
+          </inertial>
+          <visual>
+            <geometry>
+              <mesh filename="package://kuka_mobile_robot_support/meshes/37149329314.stl"/>
+            </geometry>
+            <origin rpy="1.5707963267948963 0.0 -0.0" xyz="0.0 0.0 0.0"/>
+          </visual>
+        </link>
+        <link name="left_wheel">
+          <collision>
+            <geometry>
+              <mesh filename="package://kuka_mobile_robot_support/meshes/37153975930.stl"/>
+            </geometry>
+            <origin rpy="1.5707963267948963 0.0 -0.0" xyz="0.0 0.0 0.0"/>
+          </collision>
+          <inertial>
+            <inertia ixx="5.0E-4" ixy="0.0" ixz="0.0" iyy="5.0E-4" iyz="0.0" izz="5.0E-4"/>
+            <mass value="3.0E0"/>
+            <origin rpy="-0.0 0.0 -0.0" xyz="0.0 0.0 0.0"/>
+          </inertial>
+          <visual>
+            <geometry>
+              <mesh filename="package://kuka_mobile_robot_support/meshes/37153983406.stl"/>
+            </geometry>
+            <origin rpy="0.0 0.0 -1.5707963267948963" xyz="0.0 -0.02 0.0"/>
+          </visual>
+        </link>
+        <link name="caster_base_fl_link">
+          <collision>
+            <geometry>
+              <mesh filename="package://kuka_mobile_robot_support/meshes/37153528620.stl"/>
+            </geometry>
+            <origin rpy="-0.0 0.0 -0.0" xyz="0.0 0.0 0.0"/>
+          </collision>
+          <inertial>
+            <inertia ixx="1.0E-4" ixy="0.0" ixz="0.0" iyy="1.0E-4" iyz="0.0" izz="1.0E-4"/>
+            <mass value="1.0E-1"/>
+            <origin rpy="-0.0 0.0 -0.0" xyz="0.0 0.0 0.0"/>
+          </inertial>
+          <visual>
+            <geometry>
+              <mesh filename="package://kuka_mobile_robot_support/meshes/37153537063.stl"/>
+            </geometry>
+            <origin rpy="-0.0 0.0 -0.0" xyz="0.0 0.0 0.0"/>
+          </visual>
+        </link>
+        <link name="caster_wheel_rl_link">
+          <collision>
+            <geometry>
+              <mesh filename="package://kuka_mobile_robot_support/meshes/37149321854.stl"/>
+            </geometry>
+            <origin rpy="1.5707963267948963 0.0 -0.0" xyz="0.0 0.0 0.0"/>
+          </collision>
+          <inertial>
+            <inertia ixx="1.0E-4" ixy="0.0" ixz="0.0" iyy="1.0E-4" iyz="0.0" izz="1.0E-4"/>
+            <mass value="1.0E-1"/>
+            <origin rpy="-0.0 0.0 -0.0" xyz="0.0 0.0 0.0"/>
+          </inertial>
+          <visual>
+            <geometry>
+              <mesh filename="package://kuka_mobile_robot_support/meshes/37149329314.stl"/>
+            </geometry>
+            <origin rpy="1.5707963267948963 0.0 -0.0" xyz="0.0 0.0 0.0"/>
+          </visual>
+        </link>
+        <link name="caster_base_rl_link">
+          <collision>
+            <geometry>
+              <mesh filename="package://kuka_mobile_robot_support/meshes/37153636399.stl"/>
+            </geometry>
+            <origin rpy="-0.0 0.0 -0.0" xyz="0.0 0.0 0.0"/>
+          </collision>
+          <inertial>
+            <inertia ixx="1.0E-4" ixy="0.0" ixz="0.0" iyy="1.0E-4" iyz="0.0" izz="1.0E-4"/>
+            <mass value="1.0E-1"/>
+            <origin rpy="-0.0 0.0 -0.0" xyz="0.0 0.0 0.0"/>
+          </inertial>
+          <visual>
+            <geometry>
+              <mesh filename="package://kuka_mobile_robot_support/meshes/37153643851.stl"/>
+            </geometry>
+            <origin rpy="-0.0 0.0 -0.0" xyz="0.0 0.0 0.0"/>
+          </visual>
+        </link>
+        <link name="right_wheel">
+          <collision>
+            <geometry>
+              <mesh filename="package://kuka_mobile_robot_support/meshes/37154306984.stl"/>
+            </geometry>
+            <origin rpy="1.5707963267948963 0.0 -0.0" xyz="0.0 0.0 0.0"/>
+          </collision>
+          <inertial>
+            <inertia ixx="5.0E-4" ixy="0.0" ixz="0.0" iyy="5.0E-4" iyz="0.0" izz="5.0E-4"/>
+            <mass value="3.0E0"/>
+            <origin rpy="-0.0 0.0 -0.0" xyz="0.0 0.0 0.0"/>
+          </inertial>
+          <visual>
+            <geometry>
+              <mesh filename="package://kuka_mobile_robot_support/meshes/37154317878.stl"/>
+            </geometry>
+            <origin rpy="-0.0 0.0 1.5707963267948963" xyz="0.0 0.02 0.0"/>
+          </visual>
+        </link>
+        <link name="caster_wheel_bl_link">
+          <collision>
+            <geometry>
+              <mesh filename="package://kuka_mobile_robot_support/meshes/37149321854.stl"/>
+            </geometry>
+            <origin rpy="1.5707963267948963 0.0 -0.0" xyz="0.0 0.0 0.0"/>
+          </collision>
+          <inertial>
+            <inertia ixx="1.0E-4" ixy="0.0" ixz="0.0" iyy="1.0E-4" iyz="0.0" izz="1.0E-4"/>
+            <mass value="1.0E-1"/>
+            <origin rpy="-0.0 0.0 -0.0" xyz="0.0 0.0 0.0"/>
+          </inertial>
+          <visual>
+            <geometry>
+              <mesh filename="package://kuka_mobile_robot_support/meshes/37149329314.stl"/>
+            </geometry>
+            <origin rpy="1.5707963267948963 0.0 -0.0" xyz="0.0 0.0 0.0"/>
+          </visual>
+        </link>
+        <link name="caster_base_bl_link">
+          <collision>
+            <geometry>
+              <mesh filename="package://kuka_mobile_robot_support/meshes/37152976775.stl"/>
+            </geometry>
+            <origin rpy="-0.0 0.0 -0.0" xyz="0.0 0.0 0.0"/>
+          </collision>
+          <inertial>
+            <inertia ixx="1.0E-4" ixy="0.0" ixz="0.0" iyy="1.0E-4" iyz="0.0" izz="1.0E-4"/>
+            <mass value="1.0E-1"/>
+            <origin rpy="-0.0 0.0 -0.0" xyz="0.0 0.0 0.0"/>
+          </inertial>
+          <visual>
+            <geometry>
+              <mesh filename="package://kuka_mobile_robot_support/meshes/37152984509.stl"/>
+            </geometry>
+            <origin rpy="-0.0 0.0 -0.0" xyz="0.0 0.0 0.0"/>
+          </visual>
+        </link>
+        <link name="caster_wheel_br_link">
+          <collision>
+            <geometry>
+              <mesh filename="package://kuka_mobile_robot_support/meshes/37149321854.stl"/>
+            </geometry>
+            <origin rpy="1.5707963267948963 0.0 -0.0" xyz="0.0 0.0 0.0"/>
+          </collision>
+          <inertial>
+            <inertia ixx="1.0E-4" ixy="0.0" ixz="0.0" iyy="1.0E-4" iyz="0.0" izz="1.0E-4"/>
+            <mass value="1.0E-1"/>
+            <origin rpy="-0.0 0.0 -0.0" xyz="0.0 0.0 0.0"/>
+          </inertial>
+          <visual>
+            <geometry>
+              <mesh filename="package://kuka_mobile_robot_support/meshes/37149329314.stl"/>
+            </geometry>
+            <origin rpy="1.5707963267948963 0.0 -0.0" xyz="0.0 0.0 0.0"/>
+          </visual>
+        </link>
+        <link name="caster_base_br_link">
+          <collision>
+            <geometry>
+              <mesh filename="package://kuka_mobile_robot_support/meshes/37153311411.stl"/>
+            </geometry>
+            <origin rpy="-0.0 0.0 -0.0" xyz="0.0 0.0 0.0"/>
+          </collision>
+          <inertial>
+            <inertia ixx="1.0E-4" ixy="0.0" ixz="0.0" iyy="1.0E-4" iyz="0.0" izz="1.0E-4"/>
+            <mass value="1.0E-1"/>
+            <origin rpy="-0.0 0.0 -0.0" xyz="0.0 0.0 0.0"/>
+          </inertial>
+          <visual>
+            <geometry>
+              <mesh filename="package://kuka_mobile_robot_support/meshes/37153318102.stl"/>
+            </geometry>
+            <origin rpy="-0.0 0.0 -0.0" xyz="0.0 0.0 0.0"/>
+          </visual>
+        </link>
   </xacro:macro>
 </robot>
