Commit message: add odom joint, fix wheels

File: kuka_mobile_robot_support/urdf/mrob_kuka_macro.xacro (robot description, xacro)
@@ -17,7 +17,10 @@
       use_fake_hardware="${use_fake_hardware}"
       gazebo_sim="${gazebo_sim}"/>
-    <!-- Include and instatiate diffbot description urdf file-->
-    <xacro:include filename="$(find kuka_mobile_robot_support)/urdf/diffbot_description.urdf.xacro" />
-    <!--xacro:genericMR_37146123288 prefix="${prefix}" /-->
+     <joint name="odom_joint" type="planar">
+            <axis xyz="0.0 1.0 0.0"/>
+            <parent link="odom" />
+            <child link="generic_mr_body_dummy" />
+            <origin xyz="0 0 0" rpy="0 0 0" />
+          </joint>
       <joint name="generic_mr_body_dummy" type="fixed">
             <parent link="generic_mr_body_dummy" />
@@ -31,5 +34,5 @@
           <parent link="caster_base_br_link"/>
         </joint>
-        <joint name="left_wheel_motor" type="continuous">
+        <joint name="left_wheel_motor" type="fixed">
           <axis xyz="0.0 1.0 0.0"/>
           <child link="left_wheel"/>
@@ -38,5 +41,5 @@
           <parent link="generic_mr_body"/>
         </joint>
-        <joint name="right_wheel_motor" type="continuous">
+        <joint name="right_wheel_motor" type="fixed">
           <axis xyz="0.0 1.0 0.0"/>
           <child link="right_wheel"/>
@@ -88,4 +91,5 @@
         </joint>
         <link name="generic_mr_body_dummy"/>
+        <link name="odom"/>
         <link name="generic_mr_body">
           <collision>
