Commit message: mesh dir rename

File: kuka_lbr_iisy_support/urdf/lbr_iisy3_r760_macro.xacro (robot description, xacro)
@@ -1,8 +1,9 @@
 <?xml version="1.0" encoding="UTF-8"?>
-<robot xmlns:xacro="http://www.ros.org/wiki/xacro" name="LBR3R760iisy">
+<robot xmlns:xacro="http://www.ros.org/wiki/xacro" name="LBRiisy3R760">
   <xacro:macro name="kuka_lbr3_r760_robot" params="prefix client_ip controller_ip control_mode consequent_lost_packets lost_packets_in_timeframe timeframe_ms">
     <xacro:include filename="$(find kuka_lbr_iisy_support)/urdf/lbr_iisy_ros2_control.xacro" />
     <!-- ros2 control instance -->
     <xacro:kuka_lbr_iisy_ros2_control
+    name="LBRiisy3R760"
     prefix="${prefix}"
     client_ip="${client_ip}"
@@ -17,5 +18,5 @@
       <collision>
         <geometry>
-          <mesh filename="package://kuka_lbr_iisy_support/meshes/LBR3R760/collision/base_link.stl" />
+          <mesh filename="package://kuka_lbr_iisy_support/meshes/LBRiisy3R760/collision/base_link.stl" />
         </geometry>
         <origin rpy="-0.0 0.0 -0.0" xyz="0.0 0.0 0.0" />
@@ -28,5 +29,5 @@
       <visual>
         <geometry>
-          <mesh filename="package://kuka_lbr_iisy_support/meshes/LBR3R760/visual/base_link.stl" />
+          <mesh filename="package://kuka_lbr_iisy_support/meshes/LBRiisy3R760/visual/base_link.stl" />
         </geometry>
         <origin rpy="-0.0 0.0 -0.0" xyz="0.0 0.0 0.0" />
@@ -36,5 +37,5 @@
       <collision>
         <geometry>
-          <mesh filename="package://kuka_lbr_iisy_support/meshes/LBR3R760/collision/link_1.stl" />
+          <mesh filename="package://kuka_lbr_iisy_support/meshes/LBRiisy3R760/collision/link_1.stl" />
         </geometry>
         <origin rpy="-0.0 0.0 -0.0" xyz="0.0 0.0 0.0" />
@@ -47,5 +48,5 @@
       <visual>
         <geometry>
-          <mesh filename="package://kuka_lbr_iisy_support/meshes/LBR3R760/visual/link_1.stl" />
+          <mesh filename="package://kuka_lbr_iisy_support/meshes/LBRiisy3R760/visual/link_1.stl" />
         </geometry>
         <origin rpy="-0.0 0.0 -0.0" xyz="0.0 0.0 0.0" />
@@ -55,5 +56,5 @@
       <collision>
         <geometry>
-          <mesh filename="package://kuka_lbr_iisy_support/meshes/LBR3R760/collision/link_2.stl" />
+          <mesh filename="package://kuka_lbr_iisy_support/meshes/LBRiisy3R760/collision/link_2.stl" />
         </geometry>
         <origin rpy="-0.0 0.0 -0.0" xyz="0.0 0.0 0.0" />
@@ -66,5 +67,5 @@
       <visual>
         <geometry>
-          <mesh filename="package://kuka_lbr_iisy_support/meshes/LBR3R760/visual/link_2.stl" />
+          <mesh filename="package://kuka_lbr_iisy_support/meshes/LBRiisy3R760/visual/link_2.stl" />
         </geometry>
         <origin rpy="-0.0 0.0 -0.0" xyz="0.0 0.0 0.0" />
@@ -74,5 +75,5 @@
       <collision>
         <geometry>
-          <mesh filename="package://kuka_lbr_iisy_support/meshes/LBR3R760/collision/link_3.stl" />
+          <mesh filename="package://kuka_lbr_iisy_support/meshes/LBRiisy3R760/collision/link_3.stl" />
         </geometry>
         <origin rpy="-0.0 0.0 -0.0" xyz="0.0 0.0 0.0" />
@@ -85,5 +86,5 @@
       <visual>
         <geometry>
-          <mesh filename="package://kuka_lbr_iisy_support/meshes/LBR3R760/visual/link_3.stl" />
+          <mesh filename="package://kuka_lbr_iisy_support/meshes/LBRiisy3R760/visual/link_3.stl" />
         </geometry>
         <origin rpy="-0.0 0.0 -0.0" xyz="0.0 0.0 0.0" />
@@ -93,5 +94,5 @@
       <collision>
         <geometry>
-          <mesh filename="package://kuka_lbr_iisy_support/meshes/LBR3R760/collision/link_4.stl" />
+          <mesh filename="package://kuka_lbr_iisy_support/meshes/LBRiisy3R760/collision/link_4.stl" />
         </geometry>
         <origin rpy="-0.0 0.0 -0.0" xyz="0.0 0.0 0.0" />
@@ -104,5 +105,5 @@
       <visual>
         <geometry>
-          <mesh filename="package://kuka_lbr_iisy_support/meshes/LBR3R760/visual/link_4.stl" />
+          <mesh filename="package://kuka_lbr_iisy_support/meshes/LBRiisy3R760/visual/link_4.stl" />
         </geometry>
         <origin rpy="-0.0 0.0 -0.0" xyz="0.0 0.0 0.0" />
@@ -112,5 +113,5 @@
       <collision>
         <geometry>
-          <mesh filename="package://kuka_lbr_iisy_support/meshes/LBR3R760/collision/link_5.stl" />
+          <mesh filename="package://kuka_lbr_iisy_support/meshes/LBRiisy3R760/collision/link_5.stl" />
         </geometry>
         <origin rpy="-0.0 0.0 -0.0" xyz="0.0 0.0 0.0" />
@@ -123,5 +124,5 @@
       <visual>
         <geometry>
-          <mesh filename="package://kuka_lbr_iisy_support/meshes/LBR3R760/visual/link_5.stl" />
+          <mesh filename="package://kuka_lbr_iisy_support/meshes/LBRiisy3R760/visual/link_5.stl" />
         </geometry>
         <origin rpy="-0.0 0.0 -0.0" xyz="0.0 0.0 0.0" />
@@ -131,5 +132,5 @@
       <collision>
         <geometry>
-          <mesh filename="package://kuka_lbr_iisy_support/meshes/LBR3R760/collision/link_6.stl" />
+          <mesh filename="package://kuka_lbr_iisy_support/meshes/LBRiisy3R760/collision/link_6.stl" />
         </geometry>
         <origin rpy="-0.0 0.0 -0.0" xyz="0.0 0.0 0.0" />
@@ -142,5 +143,5 @@
       <visual>
         <geometry>
-          <mesh filename="package://kuka_lbr_iisy_support/meshes/LBR3R760/visual/link_6.stl" />
+          <mesh filename="package://kuka_lbr_iisy_support/meshes/LBRiisy3R760/visual/link_6.stl" />
         </geometry>
         <origin rpy="-0.0 0.0 -0.0" xyz="0.0 0.0 0.0" />

File: kuka_lbr_iisy_support/urdf/lbr_iisy_ros2_control.xacro (robot description, xacro)
@@ -1,6 +1,6 @@
 <?xml version="1.0" encoding="UTF-8"?>
-<robot name="LBR3R760iisy" xmlns:xacro="http://www.ros.org/wiki/xacro">
-  <xacro:macro name="kuka_lbr_iisy_ros2_control" params="prefix client_ip controller_ip control_mode consequent_lost_packets lost_packets_in_timeframe timeframe_ms">
-    <ros2_control name="iisy_hardware" type="system">
+<robot xmlns:xacro="http://www.ros.org/wiki/xacro">
+  <xacro:macro name="kuka_lbr_iisy_ros2_control" params="name prefix client_ip controller_ip control_mode consequent_lost_packets lost_packets_in_timeframe timeframe_ms">
+    <ros2_control name=${name} type="system">
       <hardware>
         <plugin>kuka_rox::KukaRoXHardwareInterface</plugin>

Commit message: link conventions

File: kuka_lbr_iisy_support/urdf/lbr_iisy3_r760_macro.xacro (robot description, xacro)
@@ -14,6 +14,5 @@
     timeframe_ms="${timeframe_ms}" />
     <!-- links - main serial chain -->
-    <link name="${prefix}base_link" />
-    <link name="${prefix}LBR3R760_iisy_fixedbase">
+    <link name="${prefix}base_link">
       <collision>
         <geometry>
@@ -34,5 +33,5 @@
       </visual>
     </link>
-    <link name="${prefix}LBR3R760_iisy_axis1">
+    <link name="${prefix}link_1">
       <collision>
         <geometry>
@@ -53,5 +52,5 @@
       </visual>
     </link>
-    <link name="${prefix}LBR3R760_iisy_axis2">
+    <link name="${prefix}link_2">
       <collision>
         <geometry>
@@ -72,5 +71,5 @@
       </visual>
     </link>
-    <link name="${prefix}LBR3R760_iisy_axis3">
+    <link name="${prefix}link_3">
       <collision>
         <geometry>
@@ -91,5 +90,5 @@
       </visual>
     </link>
-    <link name="${prefix}LBR3R760_iisy_axis4">
+    <link name="${prefix}link_4">
       <collision>
         <geometry>
@@ -110,5 +109,5 @@
       </visual>
     </link>
-    <link name="${prefix}LBR3R760_iisy_axis5">
+    <link name="${prefix}link_5">
       <collision>
         <geometry>
@@ -129,5 +128,5 @@
       </visual>
     </link>
-    <link name="${prefix}LBR3R760_iisy_axis6">
+    <link name="${prefix}link_6">
       <collision>
         <geometry>
@@ -148,65 +147,67 @@
       </visual>
     </link>
-    <!-- fix base to environment -->
-    <joint name="${prefix}base_joint" type="fixed">
-      <parent link="${prefix}base_link" />
-      <child link="${prefix}LBR3R760_iisy_fixedbase" />
-    </joint>
     <!-- joints - main serial chain -->
     <joint name="${prefix}joint_a1" type="revolute">
       <axis xyz="0.0 0.0 -1.0" />
-      <child link="${prefix}LBR3R760_iisy_axis1" />
+      <child link="${prefix}link_1" />
       <limit effort="5.0E0" lower="-3.2288591E0" upper="3.2288591E0" velocity="2.0E0" />
       <origin rpy="-0.0 0.0 -0.0" xyz="0.0 0.0 0.1264" />
-      <parent link="${prefix}LBR3R760_iisy_fixedbase" />
+      <parent link="${prefix}base_link" />
     </joint>
     <joint name="${prefix}joint_a2" type="revolute">
       <axis xyz="0.0 0.0 1.0" />
-      <child link="${prefix}LBR3R760_iisy_axis2" />
+      <child link="${prefix}link_2" />
       <limit effort="5.0E0" lower="-4.0142572796E0" upper="8.726646E-1" velocity="2.0E0" />
       <origin rpy="-1.5707963267948963 0.0 -0.0" xyz="0.0 0.0 0.0886" />
-      <parent link="${prefix}LBR3R760_iisy_axis1" />
+      <parent link="${prefix}link_1" />
     </joint>
     <joint name="${prefix}joint_a3" type="revolute">
       <axis xyz="0.0 0.0 1.0" />
-      <child link="${prefix}LBR3R760_iisy_axis3" />
+      <child link="${prefix}link_3" />
       <limit effort="5.0E0" lower="-2.61799387799E0" upper="2.61799387799E0" velocity="2.0E0" />
       <origin rpy="0.0 0.0 -1.5707963267948963" xyz="0.3 0.0 0.0" />
-      <parent link="${prefix}LBR3R760_iisy_axis2" />
+      <parent link="${prefix}link_2" />
     </joint>
     <joint name="${prefix}joint_a4" type="revolute">
       <axis xyz="0.0 0.0 1.0" />
-      <child link="${prefix}LBR3R760_iisy_axis4" />
+      <child link="${prefix}link_4" />
       <limit effort="5.0E0" lower="-3.05432619E0" upper="3.05432619E0" velocity="2.0E0" />
       <origin rpy="1.5707963267948963 0.0 -0.0" xyz="0.0 0.0 0.0" />
-      <parent link="${prefix}LBR3R760_iisy_axis3" />
+      <parent link="${prefix}link_3" />
     </joint>
     <joint name="${prefix}joint_a5" type="revolute">
       <axis xyz="0.0 0.0 1.0" />
-      <child link="${prefix}LBR3R760_iisy_axis5" />
+      <child link="${prefix}link_5" />
       <limit effort="5.0E0" lower="-1.919862177E0" upper="1.919862177E0" velocity="2.0E0" />
       <origin rpy="-1.5707963267948963 0.0 -0.0" xyz="0.0 0.0 -0.3" />
-      <parent link="${prefix}LBR3R760_iisy_axis4" />
+      <parent link="${prefix}link_4" />
     </joint>
     <joint name="${prefix}joint_a6" type="revolute">
       <axis xyz="0.0 0.0 1.0" />
-      <child link="${prefix}LBR3R760_iisy_axis6" />
+      <child link="${prefix}link_6" />
       <limit effort="5.0E0" lower="-3.839724354E0" upper="3.839724354E0" velocity="2.0E0" />
       <origin rpy="1.5707963267948963 0.0 -0.0" xyz="0.0 0.0 0.0" />
-      <parent link="${prefix}LBR3R760_iisy_axis5" />
+      <parent link="${prefix}link_5" />
+    </joint>
+    <!-- ROS-Industrial 'base' frame - equivalent of 'KUKA ROBROOT'-->
+    <link name="${prefix}base" />
+    <joint name="${prefix}base_link-base" type="fixed">
+      <origin xyz="0 0 0" rpy="0 0 0"/>
+      <parent link="${prefix}base_link"/>
+      <child link="${prefix}base"/>
     </joint>
     <!-- ROS-Industrial 'flange' frame - attachment point for EEF models -->
-    <link name="${prefix}LBR3R760_iisy_flange" />
+    <link name="${prefix}flange" />
     <joint name="${prefix}link6-flange" type="fixed">
-      <child link="${prefix}LBR3R760_iisy_flange" />
+      <child link="${prefix}flange" />
       <origin rpy="0 3.14159265359  -0.0" xyz="0.0 0.0 -0.1605" />
-      <parent link="${prefix}LBR3R760_iisy_axis6" />
+      <parent link="${prefix}link_6" />
     </joint>
     <!-- ROS-Industrial 'tool0' frame - all-zeros tool frame -->
-    <link name="${prefix}LBR3R760_iisy_tool0" />
+    <link name="${prefix}tool0" />
     <joint name="${prefix}flange-tool0" type="fixed">
-      <child link="${prefix}LBR3R760_iisy_tool0" />
+      <child link="${prefix}tool0" />
       <origin rpy="0.0 0.0 0.0" xyz="0.0 0.0 0.0" />
-      <parent link="${prefix}LBR3R760_iisy_flange" />
+      <parent link="${prefix}flange" />
     </joint>
     <xacro:include filename="$(find kuka_lbr_iisy_support)/urdf/lbr_iisy_transmission.xacro" />

Commit message: add pi and color macros

File: kuka_lbr_iisy_support/urdf/lbr_iisy3_r760_macro.xacro (robot description, xacro)
@@ -1,6 +1,9 @@
 <?xml version="1.0" encoding="UTF-8"?>
 <robot xmlns:xacro="http://www.ros.org/wiki/xacro" name="LBRiisy3R760">
+  <!-- include helper xacros -->
+  <xacro:include filename="$(find kuka_lbr_iisy_support)/urdf/lbr_iisy_ros2_control.xacro" />
+  <xacro:include filename="$(find kuka_resources)/urdf/common_materials.xacro"/>
+  <xacro:include filename="$(find kuka_lbr_iisy_support)/urdf/lbr_iisy_transmission.xacro" />
   <xacro:macro name="kuka_lbr3_r760_robot" params="prefix client_ip controller_ip control_mode consequent_lost_packets lost_packets_in_timeframe timeframe_ms">
-    <xacro:include filename="$(find kuka_lbr_iisy_support)/urdf/lbr_iisy_ros2_control.xacro" />
     <!-- ros2 control instance -->
     <xacro:kuka_lbr_iisy_ros2_control
@@ -31,4 +34,5 @@
         </geometry>
         <origin rpy="-0.0 0.0 -0.0" xyz="0.0 0.0 0.0" />
+        <xacro:material_kuka_ral_pure_white />
       </visual>
     </link>
@@ -50,4 +54,5 @@
         </geometry>
         <origin rpy="-0.0 0.0 -0.0" xyz="0.0 0.0 0.0" />
+        <xacro:material_kuka_ral_pure_white />
       </visual>
     </link>
@@ -69,4 +74,5 @@
         </geometry>
         <origin rpy="-0.0 0.0 -0.0" xyz="0.0 0.0 0.0" />
+        <xacro:material_kuka_ral_pure_white />
       </visual>
     </link>
@@ -88,4 +94,5 @@
         </geometry>
         <origin rpy="-0.0 0.0 -0.0" xyz="0.0 0.0 0.0" />
+        <xacro:material_kuka_ral_pure_white />
       </visual>
     </link>
@@ -107,4 +114,5 @@
         </geometry>
         <origin rpy="-0.0 0.0 -0.0" xyz="0.0 0.0 0.0" />
+        <xacro:material_kuka_ral_pure_white />
       </visual>
     </link>
@@ -126,4 +134,5 @@
         </geometry>
         <origin rpy="-0.0 0.0 -0.0" xyz="0.0 0.0 0.0" />
+        <xacro:material_kuka_ral_pure_white />
       </visual>
     </link>
@@ -145,4 +154,5 @@
         </geometry>
         <origin rpy="-0.0 0.0 -0.0" xyz="0.0 0.0 0.0" />
+        <xacro:material_kuka_ral_pure_white />
       </visual>
     </link>
@@ -159,5 +169,5 @@
       <child link="${prefix}link_2" />
       <limit effort="5.0E0" lower="-4.0142572796E0" upper="8.726646E-1" velocity="2.0E0" />
-      <origin rpy="-1.5707963267948963 0.0 -0.0" xyz="0.0 0.0 0.0886" />
+      <origin rpy="${-pi/2.0} 0.0 -0.0" xyz="0.0 0.0 0.0886" />
       <parent link="${prefix}link_1" />
     </joint>
@@ -166,5 +176,5 @@
       <child link="${prefix}link_3" />
       <limit effort="5.0E0" lower="-2.61799387799E0" upper="2.61799387799E0" velocity="2.0E0" />
-      <origin rpy="0.0 0.0 -1.5707963267948963" xyz="0.3 0.0 0.0" />
+      <origin rpy="0.0 0.0 ${-pi/2.0}" xyz="0.3 0.0 0.0" />
       <parent link="${prefix}link_2" />
     </joint>
@@ -173,5 +183,5 @@
       <child link="${prefix}link_4" />
       <limit effort="5.0E0" lower="-3.05432619E0" upper="3.05432619E0" velocity="2.0E0" />
-      <origin rpy="1.5707963267948963 0.0 -0.0" xyz="0.0 0.0 0.0" />
+      <origin rpy="${pi/2.0} 0.0 -0.0" xyz="0.0 0.0 0.0" />
       <parent link="${prefix}link_3" />
     </joint>
@@ -180,5 +190,5 @@
       <child link="${prefix}link_5" />
       <limit effort="5.0E0" lower="-1.919862177E0" upper="1.919862177E0" velocity="2.0E0" />
-      <origin rpy="-1.5707963267948963 0.0 -0.0" xyz="0.0 0.0 -0.3" />
+      <origin rpy="${-pi/2.0} 0.0 -0.0" xyz="0.0 0.0 -0.3" />
       <parent link="${prefix}link_4" />
     </joint>
@@ -187,5 +197,5 @@
       <child link="${prefix}link_6" />
       <limit effort="5.0E0" lower="-3.839724354E0" upper="3.839724354E0" velocity="2.0E0" />
-      <origin rpy="1.5707963267948963 0.0 -0.0" xyz="0.0 0.0 0.0" />
+      <origin rpy="${pi/2.0} 0.0 -0.0" xyz="0.0 0.0 0.0" />
       <parent link="${prefix}link_5" />
     </joint>
@@ -201,5 +211,5 @@
     <joint name="${prefix}link6-flange" type="fixed">
       <child link="${prefix}flange" />
-      <origin rpy="0 3.14159265359  -0.0" xyz="0.0 0.0 -0.1605" />
+      <origin rpy="0 ${pi} -0.0" xyz="0.0 0.0 -0.1605" />
       <parent link="${prefix}link_6" />
     </joint>
@@ -211,5 +221,4 @@
       <parent link="${prefix}flange" />
     </joint>
-    <xacro:include filename="$(find kuka_lbr_iisy_support)/urdf/lbr_iisy_transmission.xacro" />
   </xacro:macro>
 </robot>

Commit message: add base_link_inertia

File: kuka_lbr_iisy_support/urdf/lbr_iisy3_r760_macro.xacro (robot description, xacro)
@@ -17,5 +17,7 @@
     timeframe_ms="${timeframe_ms}" />
     <!-- links - main serial chain -->
-    <link name="${prefix}base_link">
+    <!-- links - root element cannot have inertia, therefore a dummy base_link is needed -->
+    <link name="${prefix}base_link"/>
+    <link name="${prefix}base_link_inertia">
       <collision>
         <geometry>
@@ -158,4 +160,9 @@
     </link>
     <!-- joints - main serial chain -->
+    <joint name="${prefix}base_link-base_link_inertia" type="fixed">
+      <parent link="${prefix}base_link" />
+      <child link="${prefix}base_link_inertia" />
+      <origin xyz="0 0 0" rpy="0 0 0" />
+    </joint>
     <joint name="${prefix}joint_a1" type="revolute">
       <axis xyz="0.0 0.0 -1.0" />
@@ -163,5 +170,5 @@
       <limit effort="5.0E0" lower="-3.2288591E0" upper="3.2288591E0" velocity="2.0E0" />
       <origin rpy="-0.0 0.0 -0.0" xyz="0.0 0.0 0.1264" />
-      <parent link="${prefix}base_link" />
+      <parent link="${prefix}base_link_inertia" />
     </joint>
     <joint name="${prefix}joint_a2" type="revolute">

Commit message: fix iisy3 mass data

File: kuka_lbr_iisy_support/urdf/lbr_iisy3_r760_macro.xacro (robot description, xacro)
@@ -27,6 +27,6 @@
       </collision>
       <inertial>
-        <inertia ixx="5.0E-4" ixy="0.0" ixz="0.0" iyy="5.0E-4" iyz="0.0" izz="5.0E-4" />
-        <mass value="3.6832E0" />
+        <inertia ixx="0.00865396" ixy="0.0" ixz="0.0" iyy="0.0057294" iyz="0.0" izz="0.00975485"/>
+        <mass value="3.6896E0"/>
         <origin rpy="-0.0 0.0 -0.0" xyz="0.0 0.0 0.0" />
       </inertial>
@@ -47,6 +47,6 @@
       </collision>
       <inertial>
-        <inertia ixx="0.00864540353780418" ixy="0.0" ixz="0.0" iyy="0.00573103463618732" iyz="0.0" izz="0.00974792600424334" />
-        <mass value="3.2492E0" />
+        <inertia ixx="0.05207611" ixy="0.0" ixz="0.0" iyy="0.00423" iyz="0.0" izz="0.05335256"/>
+        <mass value="3.2536E0"/>
         <origin rpy="-0.0 0.0 -0.0" xyz="0.0 0.0 0.0" />
       </inertial>
@@ -67,6 +67,6 @@
       </collision>
       <inertial>
-        <inertia ixx="0.0521692170047944" ixy="0.0" ixz="0.0" iyy="0.0042331111850977" iyz="0.0" izz="0.0534425693052013" />
-        <mass value="3.212E0" />
+        <inertia ixx="0.01136164" ixy="0.0" ixz="0.0" iyy="0.0056706" iyz="0.0" izz="0.01338145"/>
+        <mass value="3.208E0"/>
         <origin rpy="-0.0 0.0 -0.0" xyz="0.0 0.0 0.0" />
       </inertial>
@@ -87,6 +87,6 @@
       </collision>
       <inertial>
-        <inertia ixx="0.0113804888378926" ixy="0.0" ixz="0.0" iyy="0.00566536942404497" iyz="0.0" izz="0.0133950588482047" />
-        <mass value="3.471E0" />
+        <inertia ixx="0.00244685" ixy="0.0" ixz="0.0" iyy="0.00929301" iyz="0.0" izz="0.00957903"/>
+        <mass value="3.4737E0"/>
         <origin rpy="-0.0 0.0 -0.0" xyz="0.0 0.0 0.0" />
       </inertial>
@@ -107,6 +107,6 @@
       </collision>
       <inertial>
-        <inertia ixx="0.00244684891934666" ixy="0.0" ixz="0.0" iyy="0.00929300990970133" iyz="0.0" izz="0.00957902612033654" />
-        <mass value="2.0138E0" />
+        <inertia ixx="0.00235422" ixy="0.0" ixz="0.0" iyy="0.00141662" iyz="0.0" izz="0.00257108"/>
+        <mass value="2.0138E0"/>
         <origin rpy="-0.0 0.0 -0.0" xyz="0.0 0.0 0.0" />
       </inertial>
@@ -127,6 +127,6 @@
       </collision>
       <inertial>
-        <inertia ixx="0.00236252846105637" ixy="0.0" ixz="0.0" iyy="0.00141854396142661" iyz="0.0" izz="0.0025813096143987" />
-        <mass value="1.4418E0" />
+        <inertia ixx="0.00146739" ixy="0.0" ixz="0.0" iyy="0.00112132" iyz="0.0" izz="0.0015816"/>
+        <mass value="1.4344E0"/>
         <origin rpy="-0.0 0.0 -0.0" xyz="0.0 0.0 0.0" />
       </inertial>
@@ -147,6 +147,6 @@
       </collision>
       <inertial>
-        <inertia ixx="0.0014673917002994" ixy="0.0" ixz="0.0" iyy="0.00112131520678352" iyz="0.0" izz="0.00158160486913488" />
-        <mass value="8.43E-1" />
+        <inertia ixx="0.00146739" ixy="0.0" ixz="0.0" iyy="0.00112132" iyz="0.0" izz="0.0015816"/>
+        <mass value="8.43E-1"/>
         <origin rpy="-0.0 0.0 -0.0" xyz="0.0 0.0 0.0" />
       </inertial>

Commit message: iisy3 limit fix

File: kuka_lbr_iisy_support/urdf/lbr_iisy3_r760_macro.xacro (robot description, xacro)
@@ -168,5 +168,5 @@
       <axis xyz="0.0 0.0 -1.0" />
       <child link="${prefix}link_1" />
-      <limit effort="5.0E0" lower="-3.2288591E0" upper="3.2288591E0" velocity="2.0E0" />
+      <limit effort="74.930405" lower="-3.2288591E0" upper="3.2288591E0" velocity="3.490656" />
       <origin rpy="-0.0 0.0 -0.0" xyz="0.0 0.0 0.1264" />
       <parent link="${prefix}base_link_inertia" />
@@ -175,5 +175,5 @@
       <axis xyz="0.0 0.0 1.0" />
       <child link="${prefix}link_2" />
-      <limit effort="5.0E0" lower="-4.0142572796E0" upper="8.726646E-1" velocity="2.0E0" />
+      <limit effort="74.472453" lower="-4.0142572796E0" upper="8.726646E-1" velocity="3.490656" />
       <origin rpy="${-pi/2.0} 0.0 -0.0" xyz="0.0 0.0 0.0886" />
       <parent link="${prefix}link_1" />
@@ -182,5 +182,5 @@
       <axis xyz="0.0 0.0 1.0" />
       <child link="${prefix}link_3" />
-      <limit effort="5.0E0" lower="-2.61799387799E0" upper="2.61799387799E0" velocity="2.0E0" />
+      <limit effort="43.393430" lower="-2.61799387799E0" upper="2.61799387799E0" velocity="3.490656" />
       <origin rpy="0.0 0.0 ${-pi/2.0}" xyz="0.3 0.0 0.0" />
       <parent link="${prefix}link_2" />
@@ -189,5 +189,5 @@
       <axis xyz="0.0 0.0 1.0" />
       <child link="${prefix}link_4" />
-      <limit effort="5.0E0" lower="-3.05432619E0" upper="3.05432619E0" velocity="2.0E0" />
+      <limit effort="14.767719" lower="-3.05432619E0" upper="3.05432619E0" velocity="5.235988" />
       <origin rpy="${pi/2.0} 0.0 -0.0" xyz="0.0 0.0 0.0" />
       <parent link="${prefix}link_3" />
@@ -196,5 +196,5 @@
       <axis xyz="0.0 0.0 1.0" />
       <child link="${prefix}link_5" />
-      <limit effort="5.0E0" lower="-1.919862177E0" upper="1.919862177E0" velocity="2.0E0" />
+      <limit effort="13.187655" lower="-1.919862177E0" upper="1.919862177E0" velocity="5.235988" />
       <origin rpy="${-pi/2.0} 0.0 -0.0" xyz="0.0 0.0 -0.3" />
       <parent link="${prefix}link_4" />
@@ -203,5 +203,5 @@
       <axis xyz="0.0 0.0 1.0" />
       <child link="${prefix}link_6" />
-      <limit effort="5.0E0" lower="-3.839724354E0" upper="3.839724354E0" velocity="2.0E0" />
+      <limit effort="4.834440" lower="-3.839724354E0" upper="3.839724354E0" velocity="6.981310" />
       <origin rpy="${pi/2.0} 0.0 -0.0" xyz="0.0 0.0 0.0" />
       <parent link="${prefix}link_5" />
