Commit message: fix mass properties

File: kuka_lbr_iisy_support/urdf/lbr_iisy15_r930_macro.xacro (robot description, xacro)
@@ -27,6 +27,6 @@
       </collision>
       <inertial>
-        <inertia ixx="0.05163236" ixy="0.0" ixz="0.0" iyy="0.03961305" iyz="0.0" izz="0.05515706"/>
-        <mass value="8.865E0"/>
+        <inertia ixx="0.0489108" ixy="0.0" ixz="0.0" iyy="0.03837059" iyz="0.0" izz="0.05221216"/>
+        <mass value="8.666E0"/>
         <origin rpy="-0.0 0.0 -0.0" xyz="0.0 0.0 0.0" />
       </inertial>
@@ -47,6 +47,6 @@
       </collision>
       <inertial>
-        <inertia ixx="0.62408426" ixy="0.0" ixz="0.0" iyy="0.03943643" iyz="0.0" izz="0.63132936"/>
-        <mass value="9.87E0"/>
+        <inertia ixx="0.03061686" ixy="0.0" ixz="0.0" iyy="0.25204709" iyz="0.0" izz="0.25865036"/>
+        <mass value="9.62E0"/>
         <origin rpy="-0.0 0.0 -0.0" xyz="0.0 0.0 0.0" />
       </inertial>
@@ -67,6 +67,6 @@
       </collision>
       <inertial>
-        <inertia ixx="0.01739898" ixy="0.0" ixz="0.0" iyy="0.03354988" iyz="0.0" izz="0.0366683"/>
-        <mass value="1.0139E1"/>
+        <inertia ixx="0.0181557" ixy="0.0" ixz="0.0" iyy="0.03469164" iyz="0.0" izz="0.03777695"/>
+        <mass value="8.079E0"/>
         <origin rpy="-0.0 0.0 -0.0" xyz="0.0 0.0 0.0" />
       </inertial>
@@ -87,6 +87,6 @@
       </collision>
       <inertial>
-        <inertia ixx="0.02748508" ixy="0.0" ixz="0.0" iyy="0.16186323" iyz="0.0" izz="0.1694282"/>
-        <mass value="7.5014E0"/>
+        <inertia ixx="0.02087716" ixy="0.0" ixz="0.0" iyy="0.05261357" iyz="0.0" izz="0.05874859"/>
+        <mass value="7.6604E0"/>
         <origin rpy="-0.0 0.0 -0.0" xyz="0.0 0.0 0.0" />
       </inertial>
@@ -107,6 +107,6 @@
       </collision>
       <inertial>
-        <inertia ixx="0.00716767" ixy="0.0" ixz="0.0" iyy="0.00536601" iyz="0.0" izz="0.0089832"/>
-        <mass value="6.9744E0"/>
+        <inertia ixx="0.00667163" ixy="0.0" ixz="0.0" iyy="0.00503488" iyz="0.0" izz="0.00840869"/>
+        <mass value="5.7014E0"/>
         <origin rpy="-0.0 0.0 -0.0" xyz="0.0 0.0 0.0" />
       </inertial>
@@ -127,6 +127,6 @@
       </collision>
       <inertial>
-        <inertia ixx="0.00396428" ixy="0.0" ixz="0.0" iyy="0.00292738" iyz="0.0" izz="0.00410763"/>
-        <mass value="2.509E0"/>
+        <inertia ixx="0.00390274" ixy="0.0" ixz="0.0" iyy="0.00286931" iyz="0.0" izz="0.00403512"/>
+        <mass value="2.381E0"/>
         <origin rpy="-0.0 0.0 -0.0" xyz="0.0 0.0 0.0" />
       </inertial>
@@ -147,6 +147,6 @@
       </collision>
       <inertial>
-        <inertia ixx="0.00396428" ixy="0.0" ixz="0.0" iyy="0.00292738" iyz="0.0" izz="0.00410763"/>
-        <mass value="1.527E0"/>
+        <inertia ixx="0.00390274" ixy="0.0" ixz="0.0" iyy="0.00286931" iyz="0.0" izz="0.00403512"/>
+        <mass value="1.509E0"/>
         <origin rpy="-0.0 0.0 -0.0" xyz="0.0 0.0 0.0" />
       </inertial>

Commit message: fix tool transform

File: kuka_lbr_iisy_support/urdf/lbr_iisy15_r930_macro.xacro (robot description, xacro)
@@ -67,6 +67,6 @@
       </collision>
       <inertial>
-        <inertia ixx="0.0181557" ixy="0.0" ixz="0.0" iyy="0.03469164" iyz="0.0" izz="0.03777695"/>
-        <mass value="8.079E0"/>
+      <inertia ixx="0.0181557" ixy="0.0" ixz="0.0" iyy="0.03469164" iyz="0.0" izz="0.03777695"/>
+      <mass value="8.079E0"/>
         <origin rpy="-0.0 0.0 -0.0" xyz="0.0 0.0 0.0" />
       </inertial>
@@ -218,5 +218,5 @@
     <joint name="${prefix}link6-flange" type="fixed">
       <child link="${prefix}flange" />
-      <origin rpy="0 ${pi} -0.0" xyz="0.0 0.0 -0.18" /> <!--TODO-->
+      <origin rpy="0 ${pi} -0.0" xyz="0.0 0.0 -0.178" />
       <parent link="${prefix}link_6" />
     </joint>
@@ -225,5 +225,5 @@
     <joint name="${prefix}link6-tool0" type="fixed">
       <child link="${prefix}tool0" />
-      <origin rpy="0 ${pi} -0.0" xyz="0.0 0.0 -0.18" /> <!--TODO-->
+      <origin rpy="0 ${pi} -0.0" xyz="0.0 0.0 -0.178" />
       <parent link="${prefix}link_6" />
     </joint>

Commit message: iisy15 limits

File: kuka_lbr_iisy_support/urdf/lbr_iisy15_r930_macro.xacro (robot description, xacro)
@@ -168,5 +168,5 @@
       <axis xyz="0.0 0.0 1.0" />
       <child link="${prefix}link_1" />
-      <limit effort="1.0E1" lower="-3.2288591161895095E0" upper="3.2288591161895095E0" velocity="8.001E3"/>
+      <limit effort="398.011277" lower="-3.2288591161895095E0" upper="3.2288591161895095E0" velocity="3.490656"/>
       <origin rpy="${-pi} 0.0 -0.0" xyz="0.0 0.0 0.0"/>
       <parent link="${prefix}base_link_inertia" />
@@ -175,5 +175,5 @@
       <axis xyz="0.0 0.0 1.0" />
       <child link="${prefix}link_2" />
-      <limit effort="1.0E1" lower="-4.014257279586958E0" upper="8.726646259971648E-1" velocity="8.001E3"/>
+      <limit effort="286.529873" lower="-4.014257279586958E0" upper="8.726646259971648E-1" velocity="3.490656"/>
       <origin rpy="${pi/2.0} 0.0 -0.0" xyz="0.0 0.0 -0.3"/>
       <parent link="${prefix}link_1" />
@@ -182,5 +182,5 @@
       <axis xyz="0.0 0.0 1.0" />
       <child link="${prefix}link_3" />
-      <limit effort="1.0E1" lower="-2.6179938779914944E0" upper="2.6179938779914944E0" velocity="8.001E3"/>
+      <limit effort="137.666701" lower="-2.6179938779914944E0" upper="2.6179938779914944E0" velocity="3.490656"/>
       <origin rpy="0.0 0.0 ${-pi/2.0}" xyz="0.385 0.0 0.0"/>
       <parent link="${prefix}link_2" />
@@ -189,5 +189,5 @@
       <axis xyz="0.0 0.0 1.0" />
       <child link="${prefix}link_4" />
-      <limit effort="1.0E1" lower="-3.141592653589793E0" upper="3.141592653589793E0" velocity="8.001E3"/>
+      <limit effort="63.574238" lower="-3.141592653589793E0" upper="3.141592653589793E0" velocity="4.014255"/>
       <origin rpy="${pi/2.0} 0.0 -0.0" xyz="0.0 0.0 0.0"/>
       <parent link="${prefix}link_3" />
@@ -196,5 +196,5 @@
       <axis xyz="0.0 0.0 1.0" />
       <child link="${prefix}link_5" />
-      <limit effort="1.0E1" lower="-1.9198621771937625E0" upper="1.9198621771937625E0" velocity="8.001E3"/>
+      <limit effort="58.580298" lower="-1.9198621771937625E0" upper="1.9198621771937625E0" velocity="4.537856"/>
       <origin rpy="${-pi/2.0} 0.0 -0.0" xyz="0.0 0.0 -0.367"/>
       <parent link="${prefix}link_4" />
@@ -203,5 +203,5 @@
       <axis xyz="0.0 0.0 1.0" />
       <child link="${prefix}link_6" />
-      <limit effort="1.0E1" lower="-3.839724354387525E0" upper="3.839724354387525E0" velocity="8.001E3"/>
+      <limit effort="15.927568" lower="-3.839724354387525E0" upper="3.839724354387525E0" velocity="7.504909"/>
       <origin rpy="${pi/2.0} 0.0 -0.0" xyz="0.0 0.0 0.0"/>
       <parent link="${prefix}link_5" />
