Commit message: package and macro renames

File: kuka_lbr_iisy_support/urdf/lbr_iisy3_r760.urdf.xacro (robot description, xacro)
@@ -2,5 +2,5 @@
 <robot xmlns:xacro="http://www.ros.org/wiki/xacro" name="LBR3R760iisy">
 <!-- Import iisy urdf file  -->
-<xacro:include filename="$(find kuka_iisy_support)/urdf/iisy_macro.xacro"/>
+<xacro:include filename="$(find kuka_lbr_iisy_support)/urdf/lbr_iisy3_r760_macro.xacro"/>
 <!-- Read parameters from eci_config  -->
 <xacro:property name="eci_config" value="$(find kuka_rox_hw_interface)/config/eci_config.yaml" />
@@ -15,5 +15,5 @@
 <xacro:property name="lost_packets_in_timeframe" value="${qos_config_dict['rt_packet_loss_profile']['lost_packets_in_timeframe']}" />
 <xacro:property name="timeframe_ms" value="${qos_config_dict['rt_packet_loss_profile']['timeframe_ms']}" />
-<xacro:iisy_robot prefix=""
+<xacro:kuka_lbr3_r760_robot prefix=""
                   client_ip="${client_ip}"
                   controller_ip="${controller_ip}"

File: kuka_lbr_iisy_support/urdf/lbr_iisy3_r760_macro.xacro (robot description, xacro)
@@ -1,8 +1,8 @@
 <?xml version="1.0" encoding="UTF-8"?>
 <robot xmlns:xacro="http://www.ros.org/wiki/xacro" name="LBR3R760iisy">
-  <xacro:macro name="iisy_robot" params="prefix client_ip controller_ip control_mode consequent_lost_packets lost_packets_in_timeframe timeframe_ms">
-    <xacro:include filename="$(find kuka_iisy_support)/urdf/iisy_ros2_control.xacro" />
+  <xacro:macro name="kuka_lbr3_r760_robot" params="prefix client_ip controller_ip control_mode consequent_lost_packets lost_packets_in_timeframe timeframe_ms">
+    <xacro:include filename="$(find kuka_lbr_iisy_support)/urdf/lbr_iisy_ros2_control.xacro" />
     <!-- ros2 control instance -->
-    <xacro:iisy_ros2_control
+    <xacro:kuka_lbr_iisy_ros2_control
     prefix="${prefix}"
     client_ip="${client_ip}"
@@ -17,5 +17,5 @@
       <collision>
         <geometry>
-          <mesh filename="package://kuka_iisy_support/meshes/LBR3R760/collision/base_link.stl" />
+          <mesh filename="package://kuka_lbr_iisy_support/meshes/LBR3R760/collision/base_link.stl" />
         </geometry>
         <origin rpy="-0.0 0.0 -0.0" xyz="0.0 0.0 0.0" />
@@ -28,5 +28,5 @@
       <visual>
         <geometry>
-          <mesh filename="package://kuka_iisy_support/meshes/LBR3R760/visual/base_link.stl" />
+          <mesh filename="package://kuka_lbr_iisy_support/meshes/LBR3R760/visual/base_link.stl" />
         </geometry>
         <origin rpy="-0.0 0.0 -0.0" xyz="0.0 0.0 0.0" />
@@ -36,5 +36,5 @@
       <collision>
         <geometry>
-          <mesh filename="package://kuka_iisy_support/meshes/LBR3R760/collision/link_1.stl" />
+          <mesh filename="package://kuka_lbr_iisy_support/meshes/LBR3R760/collision/link_1.stl" />
         </geometry>
         <origin rpy="-0.0 0.0 -0.0" xyz="0.0 0.0 0.0" />
@@ -47,5 +47,5 @@
       <visual>
         <geometry>
-          <mesh filename="package://kuka_iisy_support/meshes/LBR3R760/visual/link_1.stl" />
+          <mesh filename="package://kuka_lbr_iisy_support/meshes/LBR3R760/visual/link_1.stl" />
         </geometry>
         <origin rpy="-0.0 0.0 -0.0" xyz="0.0 0.0 0.0" />
@@ -55,5 +55,5 @@
       <collision>
         <geometry>
-          <mesh filename="package://kuka_iisy_support/meshes/LBR3R760/collision/link_2.stl" />
+          <mesh filename="package://kuka_lbr_iisy_support/meshes/LBR3R760/collision/link_2.stl" />
         </geometry>
         <origin rpy="-0.0 0.0 -0.0" xyz="0.0 0.0 0.0" />
@@ -66,5 +66,5 @@
       <visual>
         <geometry>
-          <mesh filename="package://kuka_iisy_support/meshes/LBR3R760/visual/link_2.stl" />
+          <mesh filename="package://kuka_lbr_iisy_support/meshes/LBR3R760/visual/link_2.stl" />
         </geometry>
         <origin rpy="-0.0 0.0 -0.0" xyz="0.0 0.0 0.0" />
@@ -74,5 +74,5 @@
       <collision>
         <geometry>
-          <mesh filename="package://kuka_iisy_support/meshes/LBR3R760/collision/link_3.stl" />
+          <mesh filename="package://kuka_lbr_iisy_support/meshes/LBR3R760/collision/link_3.stl" />
         </geometry>
         <origin rpy="-0.0 0.0 -0.0" xyz="0.0 0.0 0.0" />
@@ -85,5 +85,5 @@
       <visual>
         <geometry>
-          <mesh filename="package://kuka_iisy_support/meshes/LBR3R760/visual/link_3.stl" />
+          <mesh filename="package://kuka_lbr_iisy_support/meshes/LBR3R760/visual/link_3.stl" />
         </geometry>
         <origin rpy="-0.0 0.0 -0.0" xyz="0.0 0.0 0.0" />
@@ -93,5 +93,5 @@
       <collision>
         <geometry>
-          <mesh filename="package://kuka_iisy_support/meshes/LBR3R760/collision/link_4.stl" />
+          <mesh filename="package://kuka_lbr_iisy_support/meshes/LBR3R760/collision/link_4.stl" />
         </geometry>
         <origin rpy="-0.0 0.0 -0.0" xyz="0.0 0.0 0.0" />
@@ -104,5 +104,5 @@
       <visual>
         <geometry>
-          <mesh filename="package://kuka_iisy_support/meshes/LBR3R760/visual/link_4.stl" />
+          <mesh filename="package://kuka_lbr_iisy_support/meshes/LBR3R760/visual/link_4.stl" />
         </geometry>
         <origin rpy="-0.0 0.0 -0.0" xyz="0.0 0.0 0.0" />
@@ -112,5 +112,5 @@
       <collision>
         <geometry>
-          <mesh filename="package://kuka_iisy_support/meshes/LBR3R760/collision/link_5.stl" />
+          <mesh filename="package://kuka_lbr_iisy_support/meshes/LBR3R760/collision/link_5.stl" />
         </geometry>
         <origin rpy="-0.0 0.0 -0.0" xyz="0.0 0.0 0.0" />
@@ -123,5 +123,5 @@
       <visual>
         <geometry>
-          <mesh filename="package://kuka_iisy_support/meshes/LBR3R760/visual/link_5.stl" />
+          <mesh filename="package://kuka_lbr_iisy_support/meshes/LBR3R760/visual/link_5.stl" />
         </geometry>
         <origin rpy="-0.0 0.0 -0.0" xyz="0.0 0.0 0.0" />
@@ -131,5 +131,5 @@
       <collision>
         <geometry>
-          <mesh filename="package://kuka_iisy_support/meshes/LBR3R760/collision/link_6.stl" />
+          <mesh filename="package://kuka_lbr_iisy_support/meshes/LBR3R760/collision/link_6.stl" />
         </geometry>
         <origin rpy="-0.0 0.0 -0.0" xyz="0.0 0.0 0.0" />
@@ -142,5 +142,5 @@
       <visual>
         <geometry>
-          <mesh filename="package://kuka_iisy_support/meshes/LBR3R760/visual/link_6.stl" />
+          <mesh filename="package://kuka_lbr_iisy_support/meshes/LBR3R760/visual/link_6.stl" />
         </geometry>
         <origin rpy="-0.0 0.0 -0.0" xyz="0.0 0.0 0.0" />
@@ -209,5 +209,5 @@
       <parent link="${prefix}LBR3R760_iisy_flange" />
     </joint>
-    <xacro:include filename="$(find kuka_iisy_support)/urdf/iisy_transmission.xacro" />
+    <xacro:include filename="$(find kuka_lbr_iisy_support)/urdf/lbr_iisy_transmission.xacro" />
   </xacro:macro>
 </robot>

File: kuka_lbr_iisy_support/urdf/lbr_iisy_ros2_control.xacro (robot description, xacro)
@@ -1,5 +1,5 @@
 <?xml version="1.0" encoding="UTF-8"?>
 <robot name="LBR3R760iisy" xmlns:xacro="http://www.ros.org/wiki/xacro">
-  <xacro:macro name="iisy_ros2_control" params="prefix client_ip controller_ip control_mode consequent_lost_packets lost_packets_in_timeframe timeframe_ms">
+  <xacro:macro name="kuka_lbr_iisy_ros2_control" params="prefix client_ip controller_ip control_mode consequent_lost_packets lost_packets_in_timeframe timeframe_ms">
     <ros2_control name="iisy_hardware" type="system">
       <hardware>

File: kuka_lbr_iisy_support/urdf/lbr_iisy_transmission.xacro (robot description, xacro)
@@ -1,5 +1,5 @@
 <?xml version="1.0" encoding="UTF-8"?>
 <robot xmlns:xacro="http://wiki.ros.org/xacro">
-  <xacro:macro name="kuka_iisy_transmission" params="prefix">
+  <xacro:macro name="kuka_lbr_iisy_transmission" params="prefix">
     <transmission name="${prefix}joint_a1_trans">
       <actuator name="${prefix}joint_a1_motor">

Commit message: Add mock hardware option to LBR iisy ros2_control file

File: kuka_lbr_iisy_support/urdf/lbr_iisy3_r760.urdf.xacro (robot description, xacro)
@@ -15,4 +15,6 @@
 <xacro:property name="lost_packets_in_timeframe" value="${qos_config_dict['rt_packet_loss_profile']['lost_packets_in_timeframe']}" />
 <xacro:property name="timeframe_ms" value="${qos_config_dict['rt_packet_loss_profile']['timeframe_ms']}" />
+<!-- Read additional arguments  -->
+<xacro:arg name="use_fake_hardware" default="false" />
 <xacro:kuka_lbr3_r760_robot prefix=""
                   client_ip="${client_ip}"
@@ -21,4 +23,5 @@
                   consequent_lost_packets="${consequent_lost_packets}"
                   lost_packets_in_timeframe="${lost_packets_in_timeframe}"
-                  timeframe_ms="${timeframe_ms}"/>
+                  timeframe_ms="${timeframe_ms}"
+                  use_fake_hardware="$(arg use_fake_hardware)"/>
 </robot>

File: kuka_lbr_iisy_support/urdf/lbr_iisy3_r760_macro.xacro (robot description, xacro)
@@ -5,5 +5,5 @@
   <xacro:include filename="$(find kuka_resources)/urdf/common_materials.xacro"/>
   <xacro:include filename="$(find kuka_lbr_iisy_support)/urdf/lbr_iisy_transmission.xacro" />
-  <xacro:macro name="kuka_lbr3_r760_robot" params="prefix client_ip controller_ip control_mode consequent_lost_packets lost_packets_in_timeframe timeframe_ms">
+  <xacro:macro name="kuka_lbr3_r760_robot" params="prefix client_ip controller_ip control_mode consequent_lost_packets lost_packets_in_timeframe timeframe_ms use_fake_hardware:=false">
     <!-- ros2 control instance -->
     <xacro:kuka_lbr_iisy_ros2_control
@@ -15,5 +15,6 @@
     consequent_lost_packets="${consequent_lost_packets}"
     lost_packets_in_timeframe="${lost_packets_in_timeframe}"
-    timeframe_ms="${timeframe_ms}" />
+    timeframe_ms="${timeframe_ms}"
+    use_fake_hardware="${use_fake_hardware}" />
     <!-- links - main serial chain -->
     <!-- links - root element cannot have inertia, therefore a dummy base_link is needed -->

File: kuka_lbr_iisy_support/urdf/lbr_iisy_ros2_control.xacro (robot description, xacro)
@@ -1,14 +1,21 @@
 <?xml version="1.0" encoding="UTF-8"?>
 <robot xmlns:xacro="http://www.ros.org/wiki/xacro">
-  <xacro:macro name="kuka_lbr_iisy_ros2_control" params="name prefix client_ip controller_ip control_mode consequent_lost_packets lost_packets_in_timeframe timeframe_ms">
+  <xacro:macro name="kuka_lbr_iisy_ros2_control" params="name prefix client_ip controller_ip control_mode consequent_lost_packets lost_packets_in_timeframe timeframe_ms use_fake_hardware:=false">
     <ros2_control name="${name}" type="system">
       <hardware>
-        <plugin>kuka_rox::KukaRoXHardwareInterface</plugin>
-        <param name="client_ip">${client_ip}</param>
-        <param name="controller_ip">${controller_ip}</param>
-        <param name="control_mode">${control_mode}</param>
-        <param name="consequent_lost_packets">${consequent_lost_packets}</param>
-        <param name="lost_packets_in_timeframe">${lost_packets_in_timeframe}</param>
-        <param name="timeframe_ms">${timeframe_ms}</param>
+        <xacro:if value="${use_fake_hardware}">
+          <plugin>mock_components/GenericSystem</plugin>
+          <param name="fake_sensor_commands">false</param>
+          <param name="state_following_offset">0.0</param>
+        </xacro:if>
+        <xacro:unless value="${use_fake_hardware}">
+          <plugin>kuka_rox::KukaRoXHardwareInterface</plugin>
+          <param name="client_ip">${client_ip}</param>
+          <param name="controller_ip">${controller_ip}</param>
+          <param name="control_mode">${control_mode}</param>
+          <param name="consequent_lost_packets">${consequent_lost_packets}</param>
+          <param name="lost_packets_in_timeframe">${lost_packets_in_timeframe}</param>
+          <param name="timeframe_ms">${timeframe_ms}</param>
+        </xacro:unless>
       </hardware>
       <!-- define joints and command/state interfaces for each joint -->

Commit message: add gazebo support to urdf

File: kuka_lbr_iisy_support/urdf/lbr_iisy3_r760.urdf.xacro (robot description, xacro)
@@ -17,4 +17,5 @@
 <!-- Read additional arguments  -->
 <xacro:arg name="use_fake_hardware" default="false" />
+<xacro:arg name="gazebo_sim" default="false" />
 <xacro:kuka_lbr3_r760_robot prefix=""
                   client_ip="${client_ip}"
@@ -24,4 +25,5 @@
                   lost_packets_in_timeframe="${lost_packets_in_timeframe}"
                   timeframe_ms="${timeframe_ms}"
-                  use_fake_hardware="$(arg use_fake_hardware)"/>
+                  use_fake_hardware="$(arg use_fake_hardware)"
+                  gazebo_sim="$(arg gazebo_sim)"/>
 </robot>

File: kuka_lbr_iisy_support/urdf/lbr_iisy3_r760_macro.xacro (robot description, xacro)
@@ -5,5 +5,5 @@
   <xacro:include filename="$(find kuka_resources)/urdf/common_materials.xacro"/>
   <xacro:include filename="$(find kuka_lbr_iisy_support)/urdf/lbr_iisy_transmission.xacro" />
-  <xacro:macro name="kuka_lbr3_r760_robot" params="prefix client_ip controller_ip control_mode consequent_lost_packets lost_packets_in_timeframe timeframe_ms use_fake_hardware:=false">
+  <xacro:macro name="kuka_lbr3_r760_robot" params="prefix client_ip controller_ip control_mode consequent_lost_packets lost_packets_in_timeframe timeframe_ms use_fake_hardware:=false gazebo_sim:=false">
     <!-- ros2 control instance -->
     <xacro:kuka_lbr_iisy_ros2_control
@@ -16,5 +16,6 @@
     lost_packets_in_timeframe="${lost_packets_in_timeframe}"
     timeframe_ms="${timeframe_ms}"
-    use_fake_hardware="${use_fake_hardware}" />
+    use_fake_hardware="${use_fake_hardware}"
+    gazebo_sim="${gazebo_sim}" />
     <!-- links - main serial chain -->
     <!-- links - root element cannot have inertia, therefore a dummy base_link is needed -->

File: kuka_lbr_iisy_support/urdf/lbr_iisy_ros2_control.xacro (robot description, xacro)
@@ -1,5 +1,5 @@
 <?xml version="1.0" encoding="UTF-8"?>
 <robot xmlns:xacro="http://www.ros.org/wiki/xacro">
-  <xacro:macro name="kuka_lbr_iisy_ros2_control" params="name prefix client_ip controller_ip control_mode consequent_lost_packets lost_packets_in_timeframe timeframe_ms use_fake_hardware:=false">
+  <xacro:macro name="kuka_lbr_iisy_ros2_control" params="name prefix client_ip controller_ip control_mode consequent_lost_packets lost_packets_in_timeframe timeframe_ms use_fake_hardware:=false gazebo_sim:=false">
     <ros2_control name="${name}" type="system">
       <hardware>
@@ -10,12 +10,18 @@
         </xacro:if>
         <xacro:unless value="${use_fake_hardware}">
-          <plugin>kuka_rox::KukaRoXHardwareInterface</plugin>
-          <param name="client_ip">${client_ip}</param>
-          <param name="controller_ip">${controller_ip}</param>
-          <param name="control_mode">${control_mode}</param>
-          <param name="consequent_lost_packets">${consequent_lost_packets}</param>
-          <param name="lost_packets_in_timeframe">${lost_packets_in_timeframe}</param>
-          <param name="timeframe_ms">${timeframe_ms}</param>
+          <xacro:if value="${gazebo_sim}">
+            <plugin>gazebo_ros2_control/GazeboSystem</plugin>
+          </xacro:if>
+          <xacro:unless value="${gazebo_sim}">
+            <plugin>kuka_rox::KukaRoXHardwareInterface</plugin>
+            <param name="client_ip">${client_ip}</param>
+            <param name="controller_ip">${controller_ip}</param>
+            <param name="control_mode">${control_mode}</param>
+            <param name="consequent_lost_packets">${consequent_lost_packets}</param>
+            <param name="lost_packets_in_timeframe">${lost_packets_in_timeframe}</param>
+            <param name="timeframe_ms">${timeframe_ms}</param>
+          </xacro:unless>
         </xacro:unless>
+        <plugin>gazebo_ros2_control/GazeboSystem</plugin>
       </hardware>
       <!-- define joints and command/state interfaces for each joint -->
@@ -69,4 +75,12 @@
       </joint>
     </ros2_control>
+    <gazebo>
+      <plugin filename="libgazebo_ros2_control.so" name="gazebo_ros2_control">
+        <robot_param>robot_description</robot_param>
+        <robot_param_node>robot_state_publisher</robot_param_node>
+        <parameters>$(find kuka_rox_hw_interface)/config/ros2_controller_config.yaml</parameters>
+        <parameters>$(find kuka_rox_hw_interface)/config/joint_trajectory_controller_config.yaml</parameters>
+      </plugin>
+    </gazebo>
   </xacro:macro>
 </robot>

Commit message: fix origin

File: kuka_lbr_iisy_support/urdf/lbr_iisy3_r760.urdf.xacro (robot description, xacro)
@@ -13,5 +13,5 @@
         client_ip="$(arg client_ip)"
         use_fake_hardware="$(arg use_fake_hardware)">
-        <origin xyz="10 0 0" rpy="0 0 0" />
+        <origin xyz="0 0 0" rpy="0 0 0" />
     </xacro:kuka_lbr_iisy3_r760_robot>
 </robot>
