Commit message: Fixed URDF

File: kuka_lbr_iisy_support/urdf/lbr_iisy3_r760_gazebo.urdf.xacro (robot description, xacro)
@@ -2,6 +2,5 @@
 <robot xmlns:xacro="http://www.ros.org/wiki/xacro" name="lbr_iisy3_r760">
   <!-- Import iisy gazebo urdf file  -->
-  <!-- <xacro:include filename="$(find kuka_lbr_iisy_support)/urdf/lbr_iisy3_r760_gazebo_macro.xacro"/> -->
-  <xacro:include filename="$(find kuka_irl_project)/urdf/gazebo_lbr_macro.xacro"/>
+  <xacro:include filename="$(find kuka_lbr_iisy_support)/urdf/lbr_iisy3_r760_gazebo_macro.xacro"/>
   <!-- Read additional arguments  -->
   <xacro:arg name="prefix" default=""/>
@@ -12,10 +11,7 @@
   <xacro:arg name="pitch" default="0"/>
   <xacro:arg name="yaw" default="0"/>
-  <!-- <xacro:lbr_iisy3_r760_gazebo_macro prefix="$(arg prefix)">
+  <xacro:lbr_iisy3_r760_gazebo_macro prefix="$(arg prefix)">
     <origin xyz="$(arg x) $(arg y) $(arg z)" rpy="$(arg roll) $(arg pitch) $(arg yaw)"/>
-  </xacro:lbr_iisy3_r760_gazebo_macro> -->
-  <xacro:gazebo_lbr_macro prefix="$(arg prefix)">
-      <origin xyz="$(arg x) $(arg y) $(arg z)" rpy="$(arg roll) $(arg pitch) $(arg yaw)"/>
-  </xacro:gazebo_lbr_macro>
+  </xacro:lbr_iisy3_r760_gazebo_macro>
   <xacro:include filename="$(find kuka_lbr_iisy_support)/urdf/gazebo_plugin_macro.xacro" />
   <xacro:gazebo_plugin_macro/>
