Commit message: Added Gazebo URDF's for other lbr_iisy robots
- Created new URDF's for lbr_iisy11_r1300 and lbr_iisy15_930 for Gazebo simulation

- Removed unnecessary arguments from Launch file

- Fixed formatting issues

File: kuka_lbr_iisy_support/urdf/gazebo_plugin_macro.xacro (robot description, xacro)
@@ -1,15 +1,14 @@
 <?xml version="1.0"?>
 <robot xmlns:xacro="http://www.ros.org/wiki/xacro">
-    <xacro:macro name="gazebo_plugin_macro">
-        <!-- ros_control-plugin -->
-        <gazebo>
-            <plugin name="gz_ros2_control::GazeboSimROS2ControlPlugin"
-                filename="gz_ros2_control-system">
-                <parameters>$(find kuka_lbr_iisy_moveit_config)/config/lbr_controllers.yaml</parameters>
-                <ros>
-                    <namespace>/</namespace>
-                </ros>
-            </plugin>
-        </gazebo>
-    </xacro:macro>
+  <xacro:macro name="gazebo_plugin_macro">
+    <!-- ros_control-plugin -->
+    <gazebo>
+      <plugin name="gz_ros2_control::GazeboSimROS2ControlPlugin" filename="gz_ros2_control-system">
+        <parameters>$(find kuka_lbr_iisy_moveit_config)/config/lbr_controllers.yaml</parameters>
+        <ros>
+          <namespace>/</namespace>
+        </ros>
+      </plugin>
+    </gazebo>
+  </xacro:macro>
 </robot>

File: kuka_lbr_iisy_support/urdf/lbr_iisy11_r1300_gazebo.urdf.xacro (robot description, xacro)
@@ -1,6 +1,6 @@
 <?xml version="1.0"?>
-<robot xmlns:xacro="http://www.ros.org/wiki/xacro" name="lbr_iisy3_r760">
+<robot xmlns:xacro="http://www.ros.org/wiki/xacro" name="lbr_iisy11_r1300">
   <!-- Import iisy gazebo urdf file  -->
-  <xacro:include filename="$(find kuka_lbr_iisy_support)/urdf/lbr_iisy3_r760_gazebo_macro.xacro"/>
+  <xacro:include filename="$(find kuka_lbr_iisy_support)/urdf/lbr_iisy11_r1300_gazebo_macro.xacro"/>
   <!-- Read additional arguments  -->
   <xacro:arg name="prefix" default=""/>
@@ -11,7 +11,7 @@
   <xacro:arg name="pitch" default="0"/>
   <xacro:arg name="yaw" default="0"/>
-  <xacro:lbr_iisy3_r760_gazebo prefix="$(arg prefix)">
+  <xacro:kuka_lbr_iisy11_r1300_gazebo prefix="$(arg prefix)">
     <origin xyz="$(arg x) $(arg y) $(arg z)" rpy="$(arg roll) $(arg pitch) $(arg yaw)"/>
-  </xacro:lbr_iisy3_r760_gazebo>
+  </xacro:kuka_lbr_iisy11_r1300_gazebo>
   <xacro:include filename="$(find kuka_lbr_iisy_support)/urdf/gazebo_plugin_macro.xacro"/>
   <xacro:gazebo_plugin_macro/>

File: kuka_lbr_iisy_support/urdf/lbr_iisy11_r1300_gazebo_macro.xacro (robot description, xacro)
@@ -1,12 +1,12 @@
 <?xml version="1.0" encoding="UTF-8"?>
-<robot xmlns:xacro="http://www.ros.org/wiki/xacro" name="lbr_iisy3_r760_gazebo">
-  <!-- Include helper xacros -->
+<robot xmlns:xacro="http://www.ros.org/wiki/xacro" name="lbr_iisy11_r1300_gazebo">
+  <!-- include helper xacros -->
   <xacro:include filename="$(find kuka_lbr_iisy_support)/urdf/gazebo_control_macro.xacro"/>
   <xacro:include filename="$(find kuka_resources)/urdf/common_materials.xacro"/>
   <xacro:include filename="$(find kuka_lbr_iisy_support)/urdf/lbr_iisy_transmission.xacro"/>
-  <xacro:macro name="lbr_iisy3_r760_gazebo" params="prefix *origin">
+  <xacro:macro name="kuka_lbr_iisy11_r1300_gazebo" params="prefix *origin">
     <!-- Gazebo Control Macro -->
     <xacro:gazebo_control_macro prefix="${prefix}"/>
-    <!-- Links - main serial chain -->
+    <!-- links - main serial chain -->
     <link name="world"/>
     <link name="${prefix}base_link">
@@ -18,11 +18,11 @@
       <collision>
         <geometry>
-          <mesh filename="package://kuka_lbr_iisy_support/meshes/lbr_iisy3_r760/collision/base_link.stl"/>
-        </geometry>
-        <origin rpy="-0.0 0.0 -0.0" xyz="0.0 0.0 0.0"/>
-      </collision>
-      <visual>
-        <geometry>
-          <mesh filename="package://kuka_lbr_iisy_support/meshes/lbr_iisy3_r760/visual/base_link.stl"/>
+          <mesh filename="package://kuka_lbr_iisy_support/meshes/lbr_iisy11_r1300/collision/base_link.stl"/>
+        </geometry>
+        <origin rpy="-0.0 0.0 -0.0" xyz="0.0 0.0 0.0"/>
+      </collision>
+      <visual>
+        <geometry>
+          <mesh filename="package://kuka_lbr_iisy_support/meshes/lbr_iisy11_r1300/visual/base_link.stl"/>
         </geometry>
         <origin rpy="-0.0 0.0 -0.0" xyz="0.0 0.0 0.0"/>
@@ -38,11 +38,16 @@
       <collision>
         <geometry>
-          <mesh filename="package://kuka_lbr_iisy_support/meshes/lbr_iisy3_r760/collision/link_1.stl"/>
-        </geometry>
-        <origin rpy="-0.0 0.0 -0.0" xyz="0.0 0.0 0.0"/>
-      </collision>
-      <visual>
-        <geometry>
-          <mesh filename="package://kuka_lbr_iisy_support/meshes/lbr_iisy3_r760/visual/link_1.stl"/>
+          <mesh filename="package://kuka_lbr_iisy_support/meshes/lbr_iisy11_r1300/collision/link_1.stl"/>
+        </geometry>
+        <origin rpy="-0.0 0.0 -0.0" xyz="0.0 0.0 0.0"/>
+      </collision>
+      <inertial>
+        <inertia ixx="0.0489108039022503" ixy="0.0" ixz="0.0" iyy="0.038370593540088" iyz="0.0" izz="0.0522121642769911"/>
+        <mass value="9.62E0"/>
+        <origin rpy="-1.3035636348359196 -0.7815781053554712 1.2529437882898178" xyz="0.00344301039501039 0.0191980353430353 -0.08662803846153849"/>
+      </inertial>
+      <visual>
+        <geometry>
+          <mesh filename="package://kuka_lbr_iisy_support/meshes/lbr_iisy11_r1300/visual/link_1.stl"/>
         </geometry>
         <origin rpy="-0.0 0.0 -0.0" xyz="0.0 0.0 0.0"/>
@@ -58,11 +63,16 @@
       <collision>
         <geometry>
-          <mesh filename="package://kuka_lbr_iisy_support/meshes/lbr_iisy3_r760/collision/link_2.stl"/>
-        </geometry>
-        <origin rpy="-0.0 0.0 -0.0" xyz="0.0 0.0 0.0"/>
-      </collision>
-      <visual>
-        <geometry>
-          <mesh filename="package://kuka_lbr_iisy_support/meshes/lbr_iisy3_r760/visual/link_2.stl"/>
+          <mesh filename="package://kuka_lbr_iisy_support/meshes/lbr_iisy11_r1300/collision/link_2.stl"/>
+        </geometry>
+        <origin rpy="-0.0 0.0 -0.0" xyz="0.0 0.0 0.0"/>
+      </collision>
+      <inertial>
+        <inertia ixx="0.609923712050298" ixy="0.0" ixz="0.0" iyy="0.0385097671170806" iyz="0.0" izz="0.617803845441985"/>
+        <mass value="9.86515786038357E0"/>
+        <origin rpy="-0.0037282594736534596 -0.018939981545576166 -1.569953728930981" xyz="0.249085185084359 -0.00442629366790902 -0.0535128397562821"/>
+      </inertial>
+      <visual>
+        <geometry>
+          <mesh filename="package://kuka_lbr_iisy_support/meshes/lbr_iisy11_r1300/visual/link_2.stl"/>
         </geometry>
         <origin rpy="-0.0 0.0 -0.0" xyz="0.0 0.0 0.0"/>
@@ -78,11 +88,16 @@
       <collision>
         <geometry>
-          <mesh filename="package://kuka_lbr_iisy_support/meshes/lbr_iisy3_r760/collision/link_3.stl"/>
-        </geometry>
-        <origin rpy="-0.0 0.0 -0.0" xyz="0.0 0.0 0.0"/>
-      </collision>
-      <visual>
-        <geometry>
-          <mesh filename="package://kuka_lbr_iisy_support/meshes/lbr_iisy3_r760/visual/link_3.stl"/>
+          <mesh filename="package://kuka_lbr_iisy_support/meshes/lbr_iisy11_r1300/collision/link_3.stl"/>
+        </geometry>
+        <origin rpy="-0.0 0.0 -0.0" xyz="0.0 0.0 0.0"/>
+      </collision>
+      <inertial>
+        <inertia ixx="0.0181557035426496" ixy="0.0" ixz="0.0" iyy="0.0346916391676837" iyz="0.0" izz="0.037776951242458"/>
+        <mass value="7.49283573690527E0"/>
+        <origin rpy="0.1692981167548117 0.5271433699021747 -2.9605806714357508" xyz="0.0438696763639649 -0.00482189531013714 0.044913251068375"/>
+      </inertial>
+      <visual>
+        <geometry>
+          <mesh filename="package://kuka_lbr_iisy_support/meshes/lbr_iisy11_r1300/visual/link_3.stl"/>
         </geometry>
         <origin rpy="-0.0 0.0 -0.0" xyz="0.0 0.0 0.0"/>
@@ -98,11 +113,16 @@
       <collision>
         <geometry>
-          <mesh filename="package://kuka_lbr_iisy_support/meshes/lbr_iisy3_r760/collision/link_4.stl"/>
-        </geometry>
-        <origin rpy="-0.0 0.0 -0.0" xyz="0.0 0.0 0.0"/>
-      </collision>
-      <visual>
-        <geometry>
-          <mesh filename="package://kuka_lbr_iisy_support/meshes/lbr_iisy3_r760/visual/link_4.stl"/>
+          <mesh filename="package://kuka_lbr_iisy_support/meshes/lbr_iisy11_r1300/collision/link_4.stl"/>
+        </geometry>
+        <origin rpy="-0.0 0.0 -0.0" xyz="0.0 0.0 0.0"/>
+      </collision>
+      <inertial>
+        <inertia ixx="0.0283133115058557" ixy="0.0" ixz="0.0" iyy="0.15625788909506" iyz="0.0" izz="0.163792683235523"/>
+        <mass value="7.09182257561761E0"/>
+        <origin rpy="1.4927296069780172 -1.403978512066052 -1.5036439267584298" xyz="-7.163989476214221E-5 0.0445982847464326 -0.175445521620292"/>
+      </inertial>
+      <visual>
+        <geometry>
+          <mesh filename="package://kuka_lbr_iisy_support/meshes/lbr_iisy11_r1300/visual/link_4.stl"/>
         </geometry>
         <origin rpy="-0.0 0.0 -0.0" xyz="0.0 0.0 0.0"/>
@@ -118,11 +138,16 @@
       <collision>
         <geometry>
-          <mesh filename="package://kuka_lbr_iisy_support/meshes/lbr_iisy3_r760/collision/link_5.stl"/>
-        </geometry>
-        <origin rpy="-0.0 0.0 -0.0" xyz="0.0 0.0 0.0"/>
-      </collision>
-      <visual>
-        <geometry>
-          <mesh filename="package://kuka_lbr_iisy_support/meshes/lbr_iisy3_r760/visual/link_5.stl"/>
+          <mesh filename="package://kuka_lbr_iisy_support/meshes/lbr_iisy11_r1300/collision/link_5.stl"/>
+        </geometry>
+        <origin rpy="-0.0 0.0 -0.0" xyz="0.0 0.0 0.0"/>
+      </collision>
+      <inertial>
+        <inertia ixx="0.00667288072123254" ixy="0.0" ixz="0.0" iyy="0.00503543168148481" iyz="0.0" izz="0.00841044585602456"/>
+        <mass value="2.4516241997261E0"/>
+        <origin rpy="0.4256203528755516 0.14544264795709014 1.2195648324165669" xyz="0.0384076101043046 0.00235993465013012 -0.0244545111288499"/>
+      </inertial>
+      <visual>
+        <geometry>
+          <mesh filename="package://kuka_lbr_iisy_support/meshes/lbr_iisy11_r1300/visual/link_5.stl"/>
         </geometry>
         <origin rpy="-0.0 0.0 -0.0" xyz="0.0 0.0 0.0"/>
@@ -138,17 +163,22 @@
       <collision>
         <geometry>
-          <mesh filename="package://kuka_lbr_iisy_support/meshes/lbr_iisy3_r760/collision/link_6.stl"/>
-        </geometry>
-        <origin rpy="-0.0 0.0 -0.0" xyz="0.0 0.0 0.0"/>
-      </collision>
-      <visual>
-        <geometry>
-          <mesh filename="package://kuka_lbr_iisy_support/meshes/lbr_iisy3_r760/visual/link_6.stl"/>
-        </geometry>
-        <origin rpy="-0.0 0.0 -0.0" xyz="0.0 0.0 0.0"/>
-        <xacro:material_kuka_ral_pure_white/>
-      </visual>
-    </link>
-    <!-- Joints - main serial chain -->
+          <mesh filename="package://kuka_lbr_iisy_support/meshes/lbr_iisy11_r1300/collision/link_6.stl"/>
+        </geometry>
+        <origin rpy="-0.0 0.0 -0.0" xyz="0.0 0.0 0.0"/>
+      </collision>
+      <inertial>
+        <inertia ixx="0.00390274036654823" ixy="0.0" ixz="0.0" iyy="0.00286930887521153" iyz="0.0" izz="0.00403512413298348"/>
+        <mass value="1.23566751268437E0"/>
+        <origin rpy="-0.051936335875096745 -0.1296523529795729 -0.0038347791577379832" xyz="0.00315856028595676 0.0135678555121583 -0.038876254431844504"/>
+      </inertial>
+      <visual>
+        <geometry>
+          <mesh filename="package://kuka_lbr_iisy_support/meshes/lbr_iisy11_r1300/visual/link_6.stl"/>
+        </geometry>
+        <origin rpy="-0.0 0.0 -0.0" xyz="0.0 0.0 0.0"/>
+        <xacro:material_kuka_ral_pure_white/>
+      </visual>
+    </link>
+    <!-- joints - main serial chain -->
     <joint name="${prefix}world-base_link" type="fixed">
       <parent link="world"/>
@@ -157,8 +187,8 @@
     </joint>
     <joint name="${prefix}joint_1" type="revolute">
-      <axis xyz="0.0 0.0 -1.0"/>
+      <axis xyz="0.0 0.0 1.0"/>
       <child link="${prefix}link_1"/>
-      <limit effort="74.930405" lower="-3.2288591E0" upper="3.2288591E0" velocity="3.490656"/>
-      <origin rpy="-0.0 0.0 -0.0" xyz="0.0 0.0 0.1264"/>
+      <limit effort="4.0584E2" lower="-3.2288591125E0" upper="3.2288591125E0" velocity="3.49065850398866E0"/>
+      <origin rpy="${pi} -0.0 0.0" xyz="0.0 0.0 0.1845"/>
       <parent link="${prefix}base_link"/>
     </joint>
@@ -166,6 +196,6 @@
       <axis xyz="0.0 0.0 1.0"/>
       <child link="${prefix}link_2"/>
-      <limit effort="74.472453" lower="-4.0142572796E0" upper="8.726646E-1" velocity="3.490656"/>
-      <origin rpy="${-pi/2.0} 0.0 -0.0" xyz="0.0 0.0 0.0886"/>
+      <limit effort="366.247685" lower="-4.014257279586958E0" upper="8.726646259971648E-1" velocity="3.490656"/>
+      <origin rpy="${pi/2.0} 0.0 -0.0" xyz="0.0 0.1011 -0.1155"/>
       <parent link="${prefix}link_1"/>
     </joint>
@@ -173,6 +203,6 @@
       <axis xyz="0.0 0.0 1.0"/>
       <child link="${prefix}link_3"/>
-      <limit effort="43.393430" lower="-2.61799387799E0" upper="2.61799387799E0" velocity="3.490656"/>
-      <origin rpy="0.0 0.0 ${-pi/2.0}" xyz="0.3 0.0 0.0"/>
+      <limit effort="1.47189439778934E2" lower="-2.617993875E0" upper="2.617993875E0" velocity="3.49065850398866E0"/>
+      <origin rpy="0.0 -0.0 0.0" xyz="0.59 0.0 0.0237"/>
       <parent link="${prefix}link_2"/>
     </joint>
@@ -180,6 +210,6 @@
       <axis xyz="0.0 0.0 1.0"/>
       <child link="${prefix}link_4"/>
-      <limit effort="14.767719" lower="-3.05432619E0" upper="3.05432619E0" velocity="5.235988"/>
-      <origin rpy="${pi/2.0} 0.0 -0.0" xyz="0.0 0.0 0.0"/>
+      <limit effort="6.54825468125571E1" lower="-3.14159265E0" upper="3.14159265E0" velocity="4.01425727958696E0"/>
+      <origin rpy="${pi/2} -0.0 ${-pi/2}" xyz="0.1139 0.0 0.0774"/>
       <parent link="${prefix}link_3"/>
     </joint>
@@ -187,6 +217,6 @@
       <axis xyz="0.0 0.0 1.0"/>
       <child link="${prefix}link_5"/>
-      <limit effort="13.187655" lower="-1.919862177E0" upper="1.919862177E0" velocity="5.235988"/>
-      <origin rpy="${-pi/2.0} 0.0 -0.0" xyz="0.0 0.0 -0.3"/>
+      <limit effort="6.46576468348751E1" lower="-1.919862175E0" upper="1.919862175E0" velocity="4.53785605518526E0"/>
+      <origin rpy="0.0 ${pi/2} ${pi/2}" xyz="0.0 0.0507 -0.4181"/>
       <parent link="${prefix}link_4"/>
     </joint>
@@ -194,6 +224,6 @@
       <axis xyz="0.0 0.0 1.0"/>
       <child link="${prefix}link_6"/>
-      <limit effort="4.834440" lower="-3.839724354E0" upper="3.839724354E0" velocity="6.981310"/>
-      <origin rpy="${pi/2.0} 0.0 -0.0" xyz="0.0 0.0 0.0"/>
+      <limit effort="1.57202326869092E1" lower="-3.83972435E0" upper="3.83972435E0" velocity="7.50491578357562E0"/>
+      <origin rpy="${pi/2} -0.0 ${-pi/2}" xyz="0.0837 0.0 -0.0507"/>
       <parent link="${prefix}link_5"/>
     </joint>
@@ -209,5 +239,5 @@
     <joint name="${prefix}link6-flange" type="fixed">
       <child link="${prefix}flange"/>
-      <origin rpy="0 ${pi/2} -0.0" xyz="0.0 0.0 -0.1605"/>
+      <origin rpy="0.0 ${pi/2} 0.0" xyz="0.0 0.0 -0.0943"/>
       <parent link="${prefix}link_6"/>
     </joint>
@@ -216,5 +246,5 @@
     <joint name="${prefix}link6-tool0" type="fixed">
       <child link="${prefix}tool0"/>
-      <origin rpy="0 ${pi} -0.0" xyz="0.0 0.0 -0.1605"/>
+      <origin rpy="0.0 ${pi} 0.0" xyz="0.0 0.0 -0.0943"/>
       <parent link="${prefix}link_6"/>
     </joint>

File: kuka_lbr_iisy_support/urdf/lbr_iisy15_r930_gazebo.urdf.xacro (robot description, xacro)
@@ -1,6 +1,6 @@
 <?xml version="1.0"?>
-<robot xmlns:xacro="http://www.ros.org/wiki/xacro" name="lbr_iisy3_r760">
+<robot xmlns:xacro="http://www.ros.org/wiki/xacro" name="lbr_iisy15_r930">
   <!-- Import iisy gazebo urdf file  -->
-  <xacro:include filename="$(find kuka_lbr_iisy_support)/urdf/lbr_iisy3_r760_gazebo_macro.xacro"/>
+  <xacro:include filename="$(find kuka_lbr_iisy_support)/urdf/lbr_iisy15_r930_gazebo_macro.xacro"/>
   <!-- Read additional arguments  -->
   <xacro:arg name="prefix" default=""/>
@@ -11,7 +11,7 @@
   <xacro:arg name="pitch" default="0"/>
   <xacro:arg name="yaw" default="0"/>
-  <xacro:lbr_iisy3_r760_gazebo prefix="$(arg prefix)">
+  <xacro:kuka_lbr_iisy15_r930_gazebo prefix="$(arg prefix)">
     <origin xyz="$(arg x) $(arg y) $(arg z)" rpy="$(arg roll) $(arg pitch) $(arg yaw)"/>
-  </xacro:lbr_iisy3_r760_gazebo>
+  </xacro:kuka_lbr_iisy15_r930_gazebo>
   <xacro:include filename="$(find kuka_lbr_iisy_support)/urdf/gazebo_plugin_macro.xacro"/>
   <xacro:gazebo_plugin_macro/>
