Commit message: Added Gazebo URDF's for other lbr_iisy robots
- Created new URDF's for lbr_iisy11_r1300 and lbr_iisy15_930 for Gazebo simulation

- Removed unnecessary arguments from Launch file

- Fixed formatting issues

File: kuka_lbr_iisy_support/urdf/lbr_iisy15_r930_gazebo_macro.xacro (robot description, xacro)
@@ -1,12 +1,12 @@
 <?xml version="1.0" encoding="UTF-8"?>
-<robot xmlns:xacro="http://www.ros.org/wiki/xacro" name="lbr_iisy3_r760_gazebo">
-  <!-- Include helper xacros -->
+<robot xmlns:xacro="http://www.ros.org/wiki/xacro" name="lbr_iisy15_r930_gazebo">
+  <!-- include helper xacros -->
   <xacro:include filename="$(find kuka_lbr_iisy_support)/urdf/gazebo_control_macro.xacro"/>
   <xacro:include filename="$(find kuka_resources)/urdf/common_materials.xacro"/>
   <xacro:include filename="$(find kuka_lbr_iisy_support)/urdf/lbr_iisy_transmission.xacro"/>
-  <xacro:macro name="lbr_iisy3_r760_gazebo" params="prefix *origin">
+  <xacro:macro name="kuka_lbr_iisy15_r930_gazebo" params="prefix *origin">
     <!-- Gazebo Control Macro -->
     <xacro:gazebo_control_macro prefix="${prefix}"/>
-    <!-- Links - main serial chain -->
+    <!-- links - main serial chain -->
     <link name="world"/>
     <link name="${prefix}base_link">
@@ -18,11 +18,11 @@
       <collision>
         <geometry>
-          <mesh filename="package://kuka_lbr_iisy_support/meshes/lbr_iisy3_r760/collision/base_link.stl"/>
-        </geometry>
-        <origin rpy="-0.0 0.0 -0.0" xyz="0.0 0.0 0.0"/>
-      </collision>
-      <visual>
-        <geometry>
-          <mesh filename="package://kuka_lbr_iisy_support/meshes/lbr_iisy3_r760/visual/base_link.stl"/>
+          <mesh filename="package://kuka_lbr_iisy_support/meshes/lbr_iisy15_r930/collision/base_link.stl"/>
+        </geometry>
+        <origin rpy="-0.0 0.0 -0.0" xyz="0.0 0.0 0.0"/>
+      </collision>
+      <visual>
+        <geometry>
+          <mesh filename="package://kuka_lbr_iisy_support/meshes/lbr_iisy15_r930/visual/base_link.stl"/>
         </geometry>
         <origin rpy="-0.0 0.0 -0.0" xyz="0.0 0.0 0.0"/>
@@ -38,11 +38,11 @@
       <collision>
         <geometry>
-          <mesh filename="package://kuka_lbr_iisy_support/meshes/lbr_iisy3_r760/collision/link_1.stl"/>
-        </geometry>
-        <origin rpy="-0.0 0.0 -0.0" xyz="0.0 0.0 0.0"/>
-      </collision>
-      <visual>
-        <geometry>
-          <mesh filename="package://kuka_lbr_iisy_support/meshes/lbr_iisy3_r760/visual/link_1.stl"/>
+          <mesh filename="package://kuka_lbr_iisy_support/meshes/lbr_iisy15_r930/collision/link_1.stl"/>
+        </geometry>
+        <origin rpy="-0.0 0.0 -0.0" xyz="0.0 0.0 0.0"/>
+      </collision>
+      <visual>
+        <geometry>
+          <mesh filename="package://kuka_lbr_iisy_support/meshes/lbr_iisy15_r930/visual/link_1.stl"/>
         </geometry>
         <origin rpy="-0.0 0.0 -0.0" xyz="0.0 0.0 0.0"/>
@@ -58,11 +58,11 @@
       <collision>
         <geometry>
-          <mesh filename="package://kuka_lbr_iisy_support/meshes/lbr_iisy3_r760/collision/link_2.stl"/>
-        </geometry>
-        <origin rpy="-0.0 0.0 -0.0" xyz="0.0 0.0 0.0"/>
-      </collision>
-      <visual>
-        <geometry>
-          <mesh filename="package://kuka_lbr_iisy_support/meshes/lbr_iisy3_r760/visual/link_2.stl"/>
+          <mesh filename="package://kuka_lbr_iisy_support/meshes/lbr_iisy15_r930/collision/link_2.stl"/>
+        </geometry>
+        <origin rpy="-0.0 0.0 -0.0" xyz="0.0 0.0 0.0"/>
+      </collision>
+      <visual>
+        <geometry>
+          <mesh filename="package://kuka_lbr_iisy_support/meshes/lbr_iisy15_r930/visual/link_2.stl"/>
         </geometry>
         <origin rpy="-0.0 0.0 -0.0" xyz="0.0 0.0 0.0"/>
@@ -78,11 +78,11 @@
       <collision>
         <geometry>
-          <mesh filename="package://kuka_lbr_iisy_support/meshes/lbr_iisy3_r760/collision/link_3.stl"/>
-        </geometry>
-        <origin rpy="-0.0 0.0 -0.0" xyz="0.0 0.0 0.0"/>
-      </collision>
-      <visual>
-        <geometry>
-          <mesh filename="package://kuka_lbr_iisy_support/meshes/lbr_iisy3_r760/visual/link_3.stl"/>
+          <mesh filename="package://kuka_lbr_iisy_support/meshes/lbr_iisy15_r930/collision/link_3.stl"/>
+        </geometry>
+        <origin rpy="-0.0 0.0 -0.0" xyz="0.0 0.0 0.0"/>
+      </collision>
+      <visual>
+        <geometry>
+          <mesh filename="package://kuka_lbr_iisy_support/meshes/lbr_iisy15_r930/visual/link_3.stl"/>
         </geometry>
         <origin rpy="-0.0 0.0 -0.0" xyz="0.0 0.0 0.0"/>
@@ -98,11 +98,11 @@
       <collision>
         <geometry>
-          <mesh filename="package://kuka_lbr_iisy_support/meshes/lbr_iisy3_r760/collision/link_4.stl"/>
-        </geometry>
-        <origin rpy="-0.0 0.0 -0.0" xyz="0.0 0.0 0.0"/>
-      </collision>
-      <visual>
-        <geometry>
-          <mesh filename="package://kuka_lbr_iisy_support/meshes/lbr_iisy3_r760/visual/link_4.stl"/>
+          <mesh filename="package://kuka_lbr_iisy_support/meshes/lbr_iisy15_r930/collision/link_4.stl"/>
+        </geometry>
+        <origin rpy="-0.0 0.0 -0.0" xyz="0.0 0.0 0.0"/>
+      </collision>
+      <visual>
+        <geometry>
+          <mesh filename="package://kuka_lbr_iisy_support/meshes/lbr_iisy15_r930/visual/link_4.stl"/>
         </geometry>
         <origin rpy="-0.0 0.0 -0.0" xyz="0.0 0.0 0.0"/>
@@ -118,11 +118,11 @@
       <collision>
         <geometry>
-          <mesh filename="package://kuka_lbr_iisy_support/meshes/lbr_iisy3_r760/collision/link_5.stl"/>
-        </geometry>
-        <origin rpy="-0.0 0.0 -0.0" xyz="0.0 0.0 0.0"/>
-      </collision>
-      <visual>
-        <geometry>
-          <mesh filename="package://kuka_lbr_iisy_support/meshes/lbr_iisy3_r760/visual/link_5.stl"/>
+          <mesh filename="package://kuka_lbr_iisy_support/meshes/lbr_iisy15_r930/collision/link_5.stl"/>
+        </geometry>
+        <origin rpy="-0.0 0.0 -0.0" xyz="0.0 0.0 0.0"/>
+      </collision>
+      <visual>
+        <geometry>
+          <mesh filename="package://kuka_lbr_iisy_support/meshes/lbr_iisy15_r930/visual/link_5.stl"/>
         </geometry>
         <origin rpy="-0.0 0.0 -0.0" xyz="0.0 0.0 0.0"/>
@@ -138,17 +138,17 @@
       <collision>
         <geometry>
-          <mesh filename="package://kuka_lbr_iisy_support/meshes/lbr_iisy3_r760/collision/link_6.stl"/>
-        </geometry>
-        <origin rpy="-0.0 0.0 -0.0" xyz="0.0 0.0 0.0"/>
-      </collision>
-      <visual>
-        <geometry>
-          <mesh filename="package://kuka_lbr_iisy_support/meshes/lbr_iisy3_r760/visual/link_6.stl"/>
-        </geometry>
-        <origin rpy="-0.0 0.0 -0.0" xyz="0.0 0.0 0.0"/>
-        <xacro:material_kuka_ral_pure_white/>
-      </visual>
-    </link>
-    <!-- Joints - main serial chain -->
+          <mesh filename="package://kuka_lbr_iisy_support/meshes/lbr_iisy15_r930/collision/link_6.stl"/>
+        </geometry>
+        <origin rpy="-0.0 0.0 -0.0" xyz="0.0 0.0 0.0"/>
+      </collision>
+      <visual>
+        <geometry>
+          <mesh filename="package://kuka_lbr_iisy_support/meshes/lbr_iisy15_r930/visual/link_6.stl"/>
+        </geometry>
+        <origin rpy="-0.0 0.0 -0.0" xyz="0.0 0.0 0.0"/>
+        <xacro:material_kuka_ral_pure_white/>
+      </visual>
+    </link>
+    <!-- joints - main serial chain -->
     <joint name="${prefix}world-base_link" type="fixed">
       <parent link="world"/>
@@ -157,8 +157,8 @@
     </joint>
     <joint name="${prefix}joint_1" type="revolute">
-      <axis xyz="0.0 0.0 -1.0"/>
+      <axis xyz="0.0 0.0 1.0"/>
       <child link="${prefix}link_1"/>
-      <limit effort="74.930405" lower="-3.2288591E0" upper="3.2288591E0" velocity="3.490656"/>
-      <origin rpy="-0.0 0.0 -0.0" xyz="0.0 0.0 0.1264"/>
+      <limit effort="398.011277" lower="-3.2288591161895095E0" upper="3.2288591161895095E0" velocity="3.490656"/>
+      <origin rpy="${-pi} 0.0 -0.0" xyz="0.0 0.0 0.0"/>
       <parent link="${prefix}base_link"/>
     </joint>
@@ -166,6 +166,6 @@
       <axis xyz="0.0 0.0 1.0"/>
       <child link="${prefix}link_2"/>
-      <limit effort="74.472453" lower="-4.0142572796E0" upper="8.726646E-1" velocity="3.490656"/>
-      <origin rpy="${-pi/2.0} 0.0 -0.0" xyz="0.0 0.0 0.0886"/>
+      <limit effort="286.529873" lower="-4.014257279586958E0" upper="8.726646259971648E-1" velocity="3.490656"/>
+      <origin rpy="${pi/2.0} 0.0 -0.0" xyz="0.0 0.0 -0.3"/>
       <parent link="${prefix}link_1"/>
     </joint>
@@ -173,6 +173,6 @@
       <axis xyz="0.0 0.0 1.0"/>
       <child link="${prefix}link_3"/>
-      <limit effort="43.393430" lower="-2.61799387799E0" upper="2.61799387799E0" velocity="3.490656"/>
-      <origin rpy="0.0 0.0 ${-pi/2.0}" xyz="0.3 0.0 0.0"/>
+      <limit effort="137.666701" lower="-2.6179938779914944E0" upper="2.6179938779914944E0" velocity="3.490656"/>
+      <origin rpy="0.0 0.0 ${-pi/2.0}" xyz="0.385 0.0 0.0"/>
       <parent link="${prefix}link_2"/>
     </joint>
@@ -180,5 +180,5 @@
       <axis xyz="0.0 0.0 1.0"/>
       <child link="${prefix}link_4"/>
-      <limit effort="14.767719" lower="-3.05432619E0" upper="3.05432619E0" velocity="5.235988"/>
+      <limit effort="63.574238" lower="-3.141592653589793E0" upper="3.141592653589793E0" velocity="4.014255"/>
       <origin rpy="${pi/2.0} 0.0 -0.0" xyz="0.0 0.0 0.0"/>
       <parent link="${prefix}link_3"/>
@@ -187,6 +187,6 @@
       <axis xyz="0.0 0.0 1.0"/>
       <child link="${prefix}link_5"/>
-      <limit effort="13.187655" lower="-1.919862177E0" upper="1.919862177E0" velocity="5.235988"/>
-      <origin rpy="${-pi/2.0} 0.0 -0.0" xyz="0.0 0.0 -0.3"/>
+      <limit effort="58.580298" lower="-1.9198621771937625E0" upper="1.9198621771937625E0" velocity="4.537856"/>
+      <origin rpy="${-pi/2.0} 0.0 -0.0" xyz="0.0 0.0 -0.367"/>
       <parent link="${prefix}link_4"/>
     </joint>
@@ -194,5 +194,5 @@
       <axis xyz="0.0 0.0 1.0"/>
       <child link="${prefix}link_6"/>
-      <limit effort="4.834440" lower="-3.839724354E0" upper="3.839724354E0" velocity="6.981310"/>
+      <limit effort="15.927568" lower="-3.839724354387525E0" upper="3.839724354387525E0" velocity="7.504909"/>
       <origin rpy="${pi/2.0} 0.0 -0.0" xyz="0.0 0.0 0.0"/>
       <parent link="${prefix}link_5"/>
@@ -209,5 +209,5 @@
     <joint name="${prefix}link6-flange" type="fixed">
       <child link="${prefix}flange"/>
-      <origin rpy="0 ${pi/2} -0.0" xyz="0.0 0.0 -0.1605"/>
+      <origin rpy="0 ${pi/2} -0.0" xyz="0.0 0.0 -0.178"/>
       <parent link="${prefix}link_6"/>
     </joint>
@@ -216,5 +216,5 @@
     <joint name="${prefix}link6-tool0" type="fixed">
       <child link="${prefix}tool0"/>
-      <origin rpy="0 ${pi} -0.0" xyz="0.0 0.0 -0.1605"/>
+      <origin rpy="0 ${pi} -0.0" xyz="0.0 0.0 -0.178"/>
       <parent link="${prefix}link_6"/>
     </joint>
