Commit message: start iiwa renamings (not working yet)

File: kuka_lbr_iisy_support/urdf/lbr_iisy11_r1300.urdf.xacro (robot description, xacro)
@@ -15,5 +15,5 @@
 <xacro:property name="lost_packets_in_timeframe" value="${qos_config_dict['rt_packet_loss_profile']['lost_packets_in_timeframe']}" />
 <xacro:property name="timeframe_ms" value="${qos_config_dict['rt_packet_loss_profile']['timeframe_ms']}" />
-<xacro:kuka_lbr11_r1300_robot prefix=""
+<xacro:kuka_lbr_iisy11_r1300_robot prefix=""
                   client_ip="${client_ip}"
                   controller_ip="${controller_ip}"

File: kuka_lbr_iisy_support/urdf/lbr_iisy11_r1300_macro.xacro (robot description, xacro)
@@ -5,5 +5,5 @@
   <xacro:include filename="$(find kuka_resources)/urdf/common_materials.xacro"/>
   <xacro:include filename="$(find kuka_lbr_iisy_support)/urdf/lbr_iisy_transmission.xacro" />
-  <xacro:macro name="kuka_lbr11_r1300_robot" params="prefix client_ip controller_ip control_mode consequent_lost_packets lost_packets_in_timeframe timeframe_ms">
+  <xacro:macro name="kuka_lbr_iisy11_r1300_robot" params="prefix client_ip controller_ip control_mode consequent_lost_packets lost_packets_in_timeframe timeframe_ms">
     <!-- ros2 control instance -->
     <xacro:kuka_lbr_iisy_ros2_control

File: kuka_lbr_iisy_support/urdf/lbr_iisy15_r930.urdf.xacro (robot description, xacro)
@@ -15,5 +15,5 @@
 <xacro:property name="lost_packets_in_timeframe" value="${qos_config_dict['rt_packet_loss_profile']['lost_packets_in_timeframe']}" />
 <xacro:property name="timeframe_ms" value="${qos_config_dict['rt_packet_loss_profile']['timeframe_ms']}" />
-<xacro:kuka_lbr15_r930_robot prefix=""
+<xacro:kuka_lbr_iisy15_r930_robot prefix=""
                   client_ip="${client_ip}"
                   controller_ip="${controller_ip}"

File: kuka_lbr_iisy_support/urdf/lbr_iisy15_r930_macro.xacro (robot description, xacro)
@@ -5,5 +5,5 @@
   <xacro:include filename="$(find kuka_resources)/urdf/common_materials.xacro"/>
   <xacro:include filename="$(find kuka_lbr_iisy_support)/urdf/lbr_iisy_transmission.xacro" />
-  <xacro:macro name="kuka_lbr15_r930_robot" params="prefix client_ip controller_ip control_mode consequent_lost_packets lost_packets_in_timeframe timeframe_ms">
+  <xacro:macro name="kuka_lbr_iisy15_r930_robot" params="prefix client_ip controller_ip control_mode consequent_lost_packets lost_packets_in_timeframe timeframe_ms">
     <!-- ros2 control instance -->
     <xacro:kuka_lbr_iisy_ros2_control

File: kuka_lbr_iisy_support/urdf/lbr_iisy3_r760.urdf.xacro (robot description, xacro)
@@ -17,5 +17,5 @@
 <!-- Read additional arguments  -->
 <xacro:arg name="use_fake_hardware" default="false" />
-<xacro:kuka_lbr3_r760_robot prefix=""
+<xacro:kuka_lbr_iisy3_r760_robot prefix=""
                   client_ip="${client_ip}"
                   controller_ip="${controller_ip}"

File: kuka_lbr_iisy_support/urdf/lbr_iisy3_r760_macro.xacro (robot description, xacro)
@@ -5,5 +5,5 @@
   <xacro:include filename="$(find kuka_resources)/urdf/common_materials.xacro"/>
   <xacro:include filename="$(find kuka_lbr_iisy_support)/urdf/lbr_iisy_transmission.xacro" />
-  <xacro:macro name="kuka_lbr3_r760_robot" params="prefix client_ip controller_ip control_mode consequent_lost_packets lost_packets_in_timeframe timeframe_ms use_fake_hardware:=false">
+  <xacro:macro name="kuka_lbr_iisy3_r760_robot" params="prefix client_ip controller_ip control_mode consequent_lost_packets lost_packets_in_timeframe timeframe_ms use_fake_hardware:=false">
     <!-- ros2 control instance -->
     <xacro:kuka_lbr_iisy_ros2_control

File: kuka_lbr_iiwa_support/urdf/lbr_iiwa14_r820_macro.xacro (robot description, xacro)
@@ -1,5 +1,5 @@
 <?xml version="1.0"?>
 <robot xmlns:xacro="http://wiki.ros.org/xacro">
-  <xacro:macro name="kuka_lbr_iiwa7" params="io_access">
+  <xacro:macro name="kuka_lbr_iiwa14_r820_robot" params="io_access">
   <ros2_control name="iiwa_hardware" type="system">
     <hardware>
@@ -7,83 +7,83 @@
     </hardware>
     <!-- define joints and command/state interfaces for each joint -->
-    <joint name="LBRiiwa7Joint1">
-      <command_interface name="position">
-        <param name="min">-1</param>
-        <param name="max"> 1</param>
-      </command_interface>
-      <command_interface name="effort">
-        <param name="min">-1</param>
-        <param name="max"> 1</param>
-      </command_interface>
-      <state_interface name="position"/>
-      <state_interface name="effort"/>
-      <state_interface name="external_torque"/>
-    </joint>
-    <joint name="LBRiiwa7Joint2">
-      <command_interface name="position">
-        <param name="min">-1</param>
-        <param name="max"> 1</param>
-      </command_interface>
-      <command_interface name="effort">
-        <param name="min">-1</param>
-        <param name="max"> 1</param>
-      </command_interface>
-      <state_interface name="position"/>
-      <state_interface name="effort"/>
-      <state_interface name="external_torque"/>
-    </joint>
-    <joint name="LBRiiwa7Joint3">
-      <command_interface name="position">
-        <param name="min">-1</param>
-        <param name="max"> 1</param>
-      </command_interface>
-      <command_interface name="effort">
-        <param name="min">-1</param>
-        <param name="max"> 1</param>
-      </command_interface>
-      <state_interface name="position"/>
-      <state_interface name="effort"/>
-      <state_interface name="external_torque"/>
-    </joint>
-    <joint name="LBRiiwa7Joint4">
-      <command_interface name="position">
-        <param name="min">-1</param>
-        <param name="max"> 1</param>
-      </command_interface>
-      <command_interface name="effort">
-        <param name="min">-1</param>
-        <param name="max"> 1</param>
-      </command_interface>
-      <state_interface name="position"/>
-      <state_interface name="effort"/>
-      <state_interface name="external_torque"/>
-    </joint>
-    <joint name="LBRiiwa7Joint5">
-      <command_interface name="position">
-        <param name="min">-1</param>
-        <param name="max"> 1</param>
-      </command_interface>
-      <command_interface name="effort">
-        <param name="min">-1</param>
-        <param name="max"> 1</param>
-      </command_interface>
-      <state_interface name="position"/>
-      <state_interface name="effort"/>
-      <state_interface name="external_torque"/>
-    </joint>
-    <joint name="LBRiiwa7Joint6">
-      <command_interface name="position">
-        <param name="min">-1</param>
-        <param name="max"> 1</param>
-      </command_interface>
-      <command_interface name="effort">
-        <param name="min">-1</param>
-        <param name="max"> 1</param>
-      </command_interface>
-      <state_interface name="position"/>
-      <state_interface name="effort"/>
-      <state_interface name="external_torque"/>
-    </joint>
-    <joint name="LBRiiwa7Joint7">
+    <joint name="${prefix}joint_a1">
+      <command_interface name="position">
+        <param name="min">-1</param>
+        <param name="max"> 1</param>
+      </command_interface>
+      <command_interface name="effort">
+        <param name="min">-1</param>
+        <param name="max"> 1</param>
+      </command_interface>
+      <state_interface name="position"/>
+      <state_interface name="effort"/>
+      <state_interface name="external_torque"/>
+    </joint>
+    <joint name="${prefix}joint_a2">
+      <command_interface name="position">
+        <param name="min">-1</param>
+        <param name="max"> 1</param>
+      </command_interface>
+      <command_interface name="effort">
+        <param name="min">-1</param>
+        <param name="max"> 1</param>
+      </command_interface>
+      <state_interface name="position"/>
+      <state_interface name="effort"/>
+      <state_interface name="external_torque"/>
+    </joint>
+    <joint name="${prefix}joint_a3">
+      <command_interface name="position">
+        <param name="min">-1</param>
+        <param name="max"> 1</param>
+      </command_interface>
+      <command_interface name="effort">
+        <param name="min">-1</param>
+        <param name="max"> 1</param>
+      </command_interface>
+      <state_interface name="position"/>
+      <state_interface name="effort"/>
+      <state_interface name="external_torque"/>
+    </joint>
+    <joint name="${prefix}joint_a4">
+      <command_interface name="position">
+        <param name="min">-1</param>
+        <param name="max"> 1</param>
+      </command_interface>
+      <command_interface name="effort">
+        <param name="min">-1</param>
+        <param name="max"> 1</param>
+      </command_interface>
+      <state_interface name="position"/>
+      <state_interface name="effort"/>
+      <state_interface name="external_torque"/>
+    </joint>
+    <joint name="${prefix}joint_a5">
+      <command_interface name="position">
+        <param name="min">-1</param>
+        <param name="max"> 1</param>
+      </command_interface>
+      <command_interface name="effort">
+        <param name="min">-1</param>
+        <param name="max"> 1</param>
+      </command_interface>
+      <state_interface name="position"/>
+      <state_interface name="effort"/>
+      <state_interface name="external_torque"/>
+    </joint>
+    <joint name="${prefix}joint_a6">
+      <command_interface name="position">
+        <param name="min">-1</param>
+        <param name="max"> 1</param>
+      </command_interface>
+      <command_interface name="effort">
+        <param name="min">-1</param>
+        <param name="max"> 1</param>
+      </command_interface>
+      <state_interface name="position"/>
+      <state_interface name="effort"/>
+      <state_interface name="external_torque"/>
+    </joint>
+    <joint name="${prefix}joint_a7">
       <command_interface name="position">
         <param name="min">-1</param>
@@ -109,53 +109,52 @@
   <gazebo>
     <plugin name="gazebo_ros2_control" filename="libgazebo_ros2_control.so">
-      <robotNamespace>/lbriiwa7</robotNamespace>
       <robotSimType>gazebo_ros2_control/DefaultRobotHWSim</robotSimType>
-      <parameters>$(find kuka_lbr_iiwa7_support)/config/lbriiwa7_control.yaml</parameters>
+      <parameters>$(find kuka_lbr_iiwa_support)/config/lbriiwa_control.yaml</parameters>
     </plugin>
   </gazebo>
-  <gazebo reference="LBRiiwa7RobotBase">
-    <selfCollide>true</selfCollide>
-    <material>Gazebo/Orange</material>
-  </gazebo>
-  <gazebo reference="LBRiiwa7Axis1">
-    <selfCollide>true</selfCollide>
-    <material>Gazebo/Orange</material>
-  </gazebo>
-  <gazebo reference="LBRiiwa7Axis2">
-    <selfCollide>true</selfCollide>
-    <material>Gazebo/Orange</material>
-  </gazebo>
-  <gazebo reference="LBRiiwa7Axis3">
-    <selfCollide>true</selfCollide>
-    <material>Gazebo/Orange</material>
-  </gazebo>
-  <gazebo reference="LBRiiwa7Axis4">
-    <selfCollide>true</selfCollide>
-    <material>Gazebo/Orange</material>
-  </gazebo>
-  <gazebo reference="LBRiiwa7Axis5">
-    <selfCollide>true</selfCollide>
-    <material>Gazebo/Orange</material>
-  </gazebo>
-  <gazebo reference="LBRiiwa7Axis6">
-    <selfCollide>true</selfCollide>
-    <material>Gazebo/Orange</material>
-  </gazebo>
-  <gazebo reference="LBRiiwa7Axis7">
+  <gazebo reference="${prefix}base_link">
+    <selfCollide>true</selfCollide>
+    <material>Gazebo/Orange</material>
+  </gazebo>
+  <gazebo reference="${prefix}link_1">
+    <selfCollide>true</selfCollide>
+    <material>Gazebo/Orange</material>
+  </gazebo>
+  <gazebo reference="${prefix}link_2">
+    <selfCollide>true</selfCollide>
+    <material>Gazebo/Orange</material>
+  </gazebo>
+  <gazebo reference="${prefix}link_3">
+    <selfCollide>true</selfCollide>
+    <material>Gazebo/Orange</material>
+  </gazebo>
+  <gazebo reference="${prefix}link_4">
+    <selfCollide>true</selfCollide>
+    <material>Gazebo/Orange</material>
+  </gazebo>
+  <gazebo reference="${prefix}link_5">
+    <selfCollide>true</selfCollide>
+    <material>Gazebo/Orange</material>
+  </gazebo>
+  <gazebo reference="${prefix}link_6">
+    <selfCollide>true</selfCollide>
+    <material>Gazebo/Orange</material>
+  </gazebo>
+  <gazebo reference="${prefix}link_7">
     <selfCollide>true</selfCollide>
     <material>Gazebo/Orange</material>
   </gazebo>
   <link name="world"/>
-  <link name="LBRiiwa7RobotBase">
-    <visual>
-      <geometry>
-        <mesh filename="package://kuka_lbr_iiwa7_support/meshes/visual/iiwa_r820_link_0_hull_v0.1_iiwa_r820_link_0_hull.stl"/>
-      </geometry>
-      <origin rpy="-0.0 0.0 0.0" xyz="0.0 0.0 0.0"/>
-    </visual>
-    <collision>
-      <origin rpy="-0.0 0.0 0.0" xyz="0.0 0.0 0.0"/>
-      <geometry>
-        <mesh filename="package://kuka_lbr_iiwa7_support/meshes/collision/iiwa_r820_link_0_collision_v0.1_iiwa_r820_link_0_collision.stl"/>
+  <link name="${prefix}base_link">
+    <visual>
+      <geometry>
+        <mesh filename="package://kuka_lbr_iiwa_support/meshes/visual/iiwa_r820_link_0_hull_v0.1_iiwa_r820_link_0_hull.stl"/>
+      </geometry>
+      <origin rpy="-0.0 0.0 0.0" xyz="0.0 0.0 0.0"/>
+    </visual>
+    <collision>
+      <origin rpy="-0.0 0.0 0.0" xyz="0.0 0.0 0.0"/>
+      <geometry>
+        <mesh filename="package://kuka_lbr_iiwa_support/meshes/collision/iiwa_r820_link_0_collision_v0.1_iiwa_r820_link_0_collision.stl"/>
       </geometry>
     </collision>
@@ -166,15 +165,15 @@
     </inertial>
   </link>
-  <link name="LBRiiwa7Axis1">
-    <visual>
-      <geometry>
-        <mesh filename="package://kuka_lbr_iiwa7_support/meshes/visual/iiwa_r820_link_1_hull_v0.1_iiwa_r820_link_1_hull.stl"/>
-      </geometry>
-      <origin rpy="-0.0 0.0 0.0" xyz="0.0 0.0 0.0"/>
-    </visual>
-    <collision>
-      <origin rpy="-0.0 0.0 0.0" xyz="0.0 0.0 0.0"/>
-      <geometry>
-        <mesh filename="package://kuka_lbr_iiwa7_support/meshes/collision/iiwa_r820_link_1_collision_v0.1_iiwa_r820_link_1_collision.stl"/>
+  <link name="${prefix}link_1">
+    <visual>
+      <geometry>
+        <mesh filename="package://kuka_lbr_iiwa_support/meshes/visual/iiwa_r820_link_1_hull_v0.1_iiwa_r820_link_1_hull.stl"/>
+      </geometry>
+      <origin rpy="-0.0 0.0 0.0" xyz="0.0 0.0 0.0"/>
+    </visual>
+    <collision>
+      <origin rpy="-0.0 0.0 0.0" xyz="0.0 0.0 0.0"/>
+      <geometry>
+        <mesh filename="package://kuka_lbr_iiwa_support/meshes/collision/iiwa_r820_link_1_collision_v0.1_iiwa_r820_link_1_collision.stl"/>
       </geometry>
     </collision>
@@ -185,15 +184,15 @@
     </inertial>
   </link>
-  <link name="LBRiiwa7Axis2">
-    <visual>
-      <geometry>
-        <mesh filename="package://kuka_lbr_iiwa7_support/meshes/visual/iiwa_r820_link_2_hull_v0.1_iiwa_r820_link_2_hull.stl"/>
-      </geometry>
-      <origin rpy="-0.0 0.0 0.0" xyz="0.0 0.0 0.0"/>
-    </visual>
-    <collision>
-      <origin rpy="-0.0 0.0 0.0" xyz="0.0 0.0 0.0"/>
-      <geometry>
-        <mesh filename="package://kuka_lbr_iiwa7_support/meshes/collision/iiwa_r820_link_2_collision_v0.1_iiwa_r820_link_2_collision.stl"/>
+  <link name="${prefix}link_2">
+    <visual>
+      <geometry>
+        <mesh filename="package://kuka_lbr_iiwa_support/meshes/visual/iiwa_r820_link_2_hull_v0.1_iiwa_r820_link_2_hull.stl"/>
+      </geometry>
+      <origin rpy="-0.0 0.0 0.0" xyz="0.0 0.0 0.0"/>
+    </visual>
+    <collision>
+      <origin rpy="-0.0 0.0 0.0" xyz="0.0 0.0 0.0"/>
+      <geometry>
+        <mesh filename="package://kuka_lbr_iiwa_support/meshes/collision/iiwa_r820_link_2_collision_v0.1_iiwa_r820_link_2_collision.stl"/>
       </geometry>
     </collision>
@@ -204,15 +203,15 @@
     </inertial>
   </link>
-  <link name="LBRiiwa7Axis3">
-    <visual>
-      <geometry>
-        <mesh filename="package://kuka_lbr_iiwa7_support/meshes/visual/iiwa_r820_link_3_hull_v0.1_iiwa_r820_link_3_hull.stl"/>
-      </geometry>
-      <origin rpy="-0.0 0.0 0.0" xyz="0.0 0.0 0.0"/>
-    </visual>
-    <collision>
-      <origin rpy="-0.0 0.0 0.0" xyz="0.0 0.0 0.0"/>
-      <geometry>
-        <mesh filename="package://kuka_lbr_iiwa7_support/meshes/collision/iiwa_r820_link_3_collision_v0.1_iiwa_r820_link_3_collision.stl"/>
+  <link name="${prefix}link_3">
+    <visual>
+      <geometry>
+        <mesh filename="package://kuka_lbr_iiwa_support/meshes/visual/iiwa_r820_link_3_hull_v0.1_iiwa_r820_link_3_hull.stl"/>
+      </geometry>
+      <origin rpy="-0.0 0.0 0.0" xyz="0.0 0.0 0.0"/>
+    </visual>
+    <collision>
+      <origin rpy="-0.0 0.0 0.0" xyz="0.0 0.0 0.0"/>
+      <geometry>
+        <mesh filename="package://kuka_lbr_iiwa_support/meshes/collision/iiwa_r820_link_3_collision_v0.1_iiwa_r820_link_3_collision.stl"/>
       </geometry>
     </collision>
@@ -223,15 +222,15 @@
     </inertial>
   </link>
-  <link name="LBRiiwa7Axis4">
-    <visual>
-      <geometry>
-        <mesh filename="package://kuka_lbr_iiwa7_support/meshes/visual/iiwa_r820_link_4_hull_v0.1_iiwa_r820_link_4_hull.stl"/>
-      </geometry>
-      <origin rpy="-0.0 0.0 0.0" xyz="0.0 0.0 0.0"/>
-    </visual>
-    <collision>
-      <origin rpy="-0.0 0.0 0.0" xyz="0.0 0.0 0.0"/>
-      <geometry>
-        <mesh filename="package://kuka_lbr_iiwa7_support/meshes/collision/iiwa_r820_link_4_collision_v0.1_iiwa_r820_link_4_collision.stl"/>
+  <link name="${prefix}link_4">
+    <visual>
+      <geometry>
+        <mesh filename="package://kuka_lbr_iiwa_support/meshes/visual/iiwa_r820_link_4_hull_v0.1_iiwa_r820_link_4_hull.stl"/>
+      </geometry>
+      <origin rpy="-0.0 0.0 0.0" xyz="0.0 0.0 0.0"/>
+    </visual>
+    <collision>
+      <origin rpy="-0.0 0.0 0.0" xyz="0.0 0.0 0.0"/>
+      <geometry>
+        <mesh filename="package://kuka_lbr_iiwa_support/meshes/collision/iiwa_r820_link_4_collision_v0.1_iiwa_r820_link_4_collision.stl"/>
       </geometry>
     </collision>
@@ -242,15 +241,15 @@
     </inertial>
   </link>
-  <link name="LBRiiwa7Axis5">
-    <visual>
-      <geometry>
-        <mesh filename="package://kuka_lbr_iiwa7_support/meshes/visual/iiwa_r820_link_5_hull_v0.1_iiwa_r820_link_5_hull.stl"/>
-      </geometry>
-      <origin rpy="-0.0 0.0 0.0" xyz="0.0 0.0 0.0"/>
-    </visual>
-    <collision>
-      <origin rpy="-0.0 0.0 0.0" xyz="0.0 0.0 0.0"/>
-      <geometry>
-        <mesh filename="package://kuka_lbr_iiwa7_support/meshes/collision/iiwa_r820_link_5_collision_v0.1_iiwa_r820_link_5_collision.stl"/>
+  <link name="${prefix}link_5">
+    <visual>
+      <geometry>
+        <mesh filename="package://kuka_lbr_iiwa_support/meshes/visual/iiwa_r820_link_5_hull_v0.1_iiwa_r820_link_5_hull.stl"/>
+      </geometry>
+      <origin rpy="-0.0 0.0 0.0" xyz="0.0 0.0 0.0"/>
+    </visual>
+    <collision>
+      <origin rpy="-0.0 0.0 0.0" xyz="0.0 0.0 0.0"/>
+      <geometry>
+        <mesh filename="package://kuka_lbr_iiwa_support/meshes/collision/iiwa_r820_link_5_collision_v0.1_iiwa_r820_link_5_collision.stl"/>
       </geometry>
     </collision>
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