Commit message: test launch files with fake hw

File: kuka_lbr_iisy_support/urdf/lbr_iisy11_r1300.urdf.xacro (robot description, xacro)
@@ -1,24 +1,8 @@
 <?xml version="1.0"?>
 <robot xmlns:xacro="http://www.ros.org/wiki/xacro" name="lbr_iisy11_r1300">
-<!-- Import iisy urdf file  -->
-<xacro:include filename="$(find kuka_lbr_iisy_support)/urdf/lbr_iisy11_r1300_macro.xacro"/>
-<!-- Read parameters from eci_config  -->
-<xacro:property name="eci_config" value="$(find kuka_rox_hw_interface)/config/eci_config.yaml" />
-<xacro:property name="eci_config_dict" value="${xacro.load_yaml(eci_config)}"/>
-<xacro:property name="control_mode" value="${eci_config_dict['robot_manager']['ros__parameters']['control_mode']}" />
-<xacro:property name="client_ip" value="${eci_config_dict['robot_manager']['ros__parameters']['client_ip']}" />
-<xacro:property name="controller_ip" value="${eci_config_dict['robot_manager']['ros__parameters']['controller_ip']}" />
-<!-- Read QoS profile parameters  -->
-<xacro:property name="qos_config" value="$(find kuka_rox_hw_interface)/config/qos_profiles.yaml" />
-<xacro:property name="qos_config_dict" value="${xacro.load_yaml(qos_config)}"/>
-<xacro:property name="consequent_lost_packets" value="${qos_config_dict['rt_packet_loss_profile']['consequent_lost_packets']}" />
-<xacro:property name="lost_packets_in_timeframe" value="${qos_config_dict['rt_packet_loss_profile']['lost_packets_in_timeframe']}" />
-<xacro:property name="timeframe_ms" value="${qos_config_dict['rt_packet_loss_profile']['timeframe_ms']}" />
-<xacro:kuka_lbr_iisy11_r1300_robot prefix=""
-                  client_ip="${client_ip}"
-                  controller_ip="${controller_ip}"
-                  control_mode="${control_mode}"
-                  consequent_lost_packets="${consequent_lost_packets}"
-                  lost_packets_in_timeframe="${lost_packets_in_timeframe}"
-                  timeframe_ms="${timeframe_ms}"/>
+    <!-- Import iisy urdf file  -->
+    <xacro:include filename="$(find kuka_lbr_iisy_support)/urdf/lbr_iisy11_r1300_macro.xacro"/>
+    <!-- Read additional arguments  -->
+    <xacro:arg name="use_fake_hardware" default="false" />
+    <xacro:kuka_lbr_iisy11_r1300_robot prefix="" use_fake_hardware="$(arg use_fake_hardware)"/>
 </robot>

File: kuka_lbr_iisy_support/urdf/lbr_iisy11_r1300_macro.xacro (robot description, xacro)
@@ -5,15 +5,10 @@
   <xacro:include filename="$(find kuka_resources)/urdf/common_materials.xacro"/>
   <xacro:include filename="$(find kuka_lbr_iisy_support)/urdf/lbr_iisy_transmission.xacro" />
-  <xacro:macro name="kuka_lbr_iisy11_r1300_robot" params="prefix client_ip controller_ip control_mode consequent_lost_packets lost_packets_in_timeframe timeframe_ms">
+  <xacro:macro name="kuka_lbr_iisy11_r1300_robot" params="prefix use_fake_hardware:=false">
     <!-- ros2 control instance -->
     <xacro:kuka_lbr_iisy_ros2_control
     name="lbr_iisy11_r1300"
     prefix="${prefix}"
-    client_ip="${client_ip}"
-    controller_ip="${controller_ip}"
-    control_mode="${control_mode}"
-    consequent_lost_packets="${consequent_lost_packets}"
-    lost_packets_in_timeframe="${lost_packets_in_timeframe}"
-    timeframe_ms="${timeframe_ms}" />
+    use_fake_hardware="${use_fake_hardware}" />
     <!-- links - main serial chain -->
     <!-- links - root element cannot have inertia, therefore a dummy base_link is needed -->

File: kuka_lbr_iisy_support/urdf/lbr_iisy15_r930.urdf.xacro (robot description, xacro)
@@ -1,24 +1,8 @@
 <?xml version="1.0"?>
 <robot xmlns:xacro="http://www.ros.org/wiki/xacro" name="lbr_iisy15_r930">
-<!-- Import iisy urdf file  -->
-<xacro:include filename="$(find kuka_lbr_iisy_support)/urdf/lbr_iisy15_r930_macro.xacro"/>
-<!-- Read parameters from eci_config  -->
-<xacro:property name="eci_config" value="$(find kuka_rox_hw_interface)/config/eci_config.yaml" />
-<xacro:property name="eci_config_dict" value="${xacro.load_yaml(eci_config)}"/>
-<xacro:property name="control_mode" value="${eci_config_dict['robot_manager']['ros__parameters']['control_mode']}" />
-<xacro:property name="client_ip" value="${eci_config_dict['robot_manager']['ros__parameters']['client_ip']}" />
-<xacro:property name="controller_ip" value="${eci_config_dict['robot_manager']['ros__parameters']['controller_ip']}" />
-<!-- Read QoS profile parameters  -->
-<xacro:property name="qos_config" value="$(find kuka_rox_hw_interface)/config/qos_profiles.yaml" />
-<xacro:property name="qos_config_dict" value="${xacro.load_yaml(qos_config)}"/>
-<xacro:property name="consequent_lost_packets" value="${qos_config_dict['rt_packet_loss_profile']['consequent_lost_packets']}" />
-<xacro:property name="lost_packets_in_timeframe" value="${qos_config_dict['rt_packet_loss_profile']['lost_packets_in_timeframe']}" />
-<xacro:property name="timeframe_ms" value="${qos_config_dict['rt_packet_loss_profile']['timeframe_ms']}" />
-<xacro:kuka_lbr_iisy15_r930_robot prefix=""
-                  client_ip="${client_ip}"
-                  controller_ip="${controller_ip}"
-                  control_mode="${control_mode}"
-                  consequent_lost_packets="${consequent_lost_packets}"
-                  lost_packets_in_timeframe="${lost_packets_in_timeframe}"
-                  timeframe_ms="${timeframe_ms}"/>
+    <!-- Import iisy urdf file  -->
+    <xacro:include filename="$(find kuka_lbr_iisy_support)/urdf/lbr_iisy15_r930_macro.xacro"/>
+    <!-- Read additional arguments  -->
+    <xacro:arg name="use_fake_hardware" default="false" />
+    <xacro:kuka_lbr_iisy15_r930_robot prefix="" use_fake_hardware="$(arg use_fake_hardware)"/>
 </robot>

File: kuka_lbr_iisy_support/urdf/lbr_iisy15_r930_macro.xacro (robot description, xacro)
@@ -5,15 +5,10 @@
   <xacro:include filename="$(find kuka_resources)/urdf/common_materials.xacro"/>
   <xacro:include filename="$(find kuka_lbr_iisy_support)/urdf/lbr_iisy_transmission.xacro" />
-  <xacro:macro name="kuka_lbr_iisy15_r930_robot" params="prefix client_ip controller_ip control_mode consequent_lost_packets lost_packets_in_timeframe timeframe_ms">
+  <xacro:macro name="kuka_lbr_iisy15_r930_robot" params="prefix use_fake_hardware:=false">
     <!-- ros2 control instance -->
     <xacro:kuka_lbr_iisy_ros2_control
     name="lbr_iisy15_r930"
     prefix="${prefix}"
-    client_ip="${client_ip}"
-    controller_ip="${controller_ip}"
-    control_mode="${control_mode}"
-    consequent_lost_packets="${consequent_lost_packets}"
-    lost_packets_in_timeframe="${lost_packets_in_timeframe}"
-    timeframe_ms="${timeframe_ms}" />
+    use_fake_hardware="${use_fake_hardware}" />
     <!-- links - main serial chain -->
     <!-- links - root element cannot have inertia, therefore a dummy base_link is needed -->

File: kuka_lbr_iisy_support/urdf/lbr_iisy3_r760.urdf.xacro (robot description, xacro)
@@ -1,27 +1,8 @@
 <?xml version="1.0"?>
 <robot xmlns:xacro="http://www.ros.org/wiki/xacro" name="lbr_iisy3_r760">
-<!-- Import iisy urdf file  -->
-<xacro:include filename="$(find kuka_lbr_iisy_support)/urdf/lbr_iisy3_r760_macro.xacro"/>
-<!-- Read parameters from eci_config  -->
-<xacro:property name="eci_config" value="$(find kuka_rox_hw_interface)/config/eci_config.yaml" />
-<xacro:property name="eci_config_dict" value="${xacro.load_yaml(eci_config)}"/>
-<xacro:property name="control_mode" value="${eci_config_dict['robot_manager']['ros__parameters']['control_mode']}" />
-<xacro:property name="client_ip" value="${eci_config_dict['robot_manager']['ros__parameters']['client_ip']}" />
-<xacro:property name="controller_ip" value="${eci_config_dict['robot_manager']['ros__parameters']['controller_ip']}" />
-<!-- Read QoS profile parameters  -->
-<xacro:property name="qos_config" value="$(find kuka_rox_hw_interface)/config/qos_profiles.yaml" />
-<xacro:property name="qos_config_dict" value="${xacro.load_yaml(qos_config)}"/>
-<xacro:property name="consequent_lost_packets" value="${qos_config_dict['rt_packet_loss_profile']['consequent_lost_packets']}" />
-<xacro:property name="lost_packets_in_timeframe" value="${qos_config_dict['rt_packet_loss_profile']['lost_packets_in_timeframe']}" />
-<xacro:property name="timeframe_ms" value="${qos_config_dict['rt_packet_loss_profile']['timeframe_ms']}" />
-<!-- Read additional arguments  -->
-<xacro:arg name="use_fake_hardware" default="false" />
-<xacro:kuka_lbr_iisy3_r760_robot prefix=""
-                  client_ip="${client_ip}"
-                  controller_ip="${controller_ip}"
-                  control_mode="${control_mode}"
-                  consequent_lost_packets="${consequent_lost_packets}"
-                  lost_packets_in_timeframe="${lost_packets_in_timeframe}"
-                  timeframe_ms="${timeframe_ms}"
-                  use_fake_hardware="$(arg use_fake_hardware)"/>
+    <!-- Import iisy urdf file  -->
+    <xacro:include filename="$(find kuka_lbr_iisy_support)/urdf/lbr_iisy3_r760_macro.xacro"/>
+    <!-- Read additional arguments  -->
+    <xacro:arg name="use_fake_hardware" default="false" />
+    <xacro:kuka_lbr_iisy3_r760_robot prefix="" use_fake_hardware="$(arg use_fake_hardware)"/>
 </robot>

File: kuka_lbr_iisy_support/urdf/lbr_iisy3_r760_macro.xacro (robot description, xacro)
@@ -5,15 +5,9 @@
   <xacro:include filename="$(find kuka_resources)/urdf/common_materials.xacro"/>
   <xacro:include filename="$(find kuka_lbr_iisy_support)/urdf/lbr_iisy_transmission.xacro" />
-  <xacro:macro name="kuka_lbr_iisy3_r760_robot" params="prefix client_ip controller_ip control_mode consequent_lost_packets lost_packets_in_timeframe timeframe_ms use_fake_hardware:=false">
+  <xacro:macro name="kuka_lbr_iisy3_r760_robot" params="prefix use_fake_hardware:=false">
     <!-- ros2 control instance -->
     <xacro:kuka_lbr_iisy_ros2_control
     name="lbr_iisy3_r760"
     prefix="${prefix}"
-    client_ip="${client_ip}"
-    controller_ip="${controller_ip}"
-    control_mode="${control_mode}"
-    consequent_lost_packets="${consequent_lost_packets}"
-    lost_packets_in_timeframe="${lost_packets_in_timeframe}"
-    timeframe_ms="${timeframe_ms}"
     use_fake_hardware="${use_fake_hardware}" />
     <!-- links - main serial chain -->

File: kuka_lbr_iisy_support/urdf/lbr_iisy_ros2_control.xacro (robot description, xacro)
@@ -1,5 +1,5 @@
 <?xml version="1.0" encoding="UTF-8"?>
 <robot xmlns:xacro="http://www.ros.org/wiki/xacro">
-  <xacro:macro name="kuka_lbr_iisy_ros2_control" params="name prefix client_ip controller_ip control_mode consequent_lost_packets lost_packets_in_timeframe timeframe_ms use_fake_hardware:=false">
+  <xacro:macro name="kuka_lbr_iisy_ros2_control" params="name prefix use_fake_hardware:=false">
     <ros2_control name="${name}" type="system">
       <hardware>
@@ -10,4 +10,16 @@
         </xacro:if>
         <xacro:unless value="${use_fake_hardware}">
+          <!-- Read parameters from eci_config  -->
+          <xacro:property name="eci_config" value="$(find kuka_rox_hw_interface)/config/eci_config.yaml" />
+          <xacro:property name="eci_config_dict" value="${xacro.load_yaml(eci_config)}"/>
+          <xacro:property name="control_mode" value="${eci_config_dict['robot_manager']['ros__parameters']['control_mode']}" />
+          <xacro:property name="client_ip" value="${eci_config_dict['robot_manager']['ros__parameters']['client_ip']}" />
+          <xacro:property name="controller_ip" value="${eci_config_dict['robot_manager']['ros__parameters']['controller_ip']}" />
+          <!-- Read QoS profile parameters  -->
+          <xacro:property name="qos_config" value="$(find kuka_rox_hw_interface)/config/qos_profiles.yaml" />
+          <xacro:property name="qos_config_dict" value="${xacro.load_yaml(qos_config)}"/>
+          <xacro:property name="consequent_lost_packets" value="${qos_config_dict['rt_packet_loss_profile']['consequent_lost_packets']}" />
+          <xacro:property name="lost_packets_in_timeframe" value="${qos_config_dict['rt_packet_loss_profile']['lost_packets_in_timeframe']}" />
+          <xacro:property name="timeframe_ms" value="${qos_config_dict['rt_packet_loss_profile']['timeframe_ms']}" />
           <plugin>kuka_rox::KukaRoXHardwareInterface</plugin>
           <param name="client_ip">${client_ip}</param>

Commit message: add ips as xacro arg

File: kuka_lbr_iisy_support/urdf/lbr_iisy11_r1300.urdf.xacro (robot description, xacro)
@@ -4,5 +4,8 @@
     <xacro:include filename="$(find kuka_lbr_iisy_support)/urdf/lbr_iisy11_r1300_macro.xacro"/>
     <!-- Read additional arguments  -->
+    <xacro:arg name="prefix" default="" />
+    <xacro:arg name="controller_ip" default="0.0.0.0" />
+    <xacro:arg name="client_ip" default="0.0.0.0" />
     <xacro:arg name="use_fake_hardware" default="false" />
-    <xacro:kuka_lbr_iisy11_r1300_robot prefix="" use_fake_hardware="$(arg use_fake_hardware)"/>
+    <xacro:kuka_lbr_iisy11_r1300_robot prefix="$(arg prefix)" controller_ip="$(arg controller_ip)" client_ip="$(arg client_ip)" use_fake_hardware="$(arg use_fake_hardware)"/>
 </robot>

File: kuka_lbr_iisy_support/urdf/lbr_iisy11_r1300_macro.xacro (robot description, xacro)
@@ -5,9 +5,11 @@
   <xacro:include filename="$(find kuka_resources)/urdf/common_materials.xacro"/>
   <xacro:include filename="$(find kuka_lbr_iisy_support)/urdf/lbr_iisy_transmission.xacro" />
-  <xacro:macro name="kuka_lbr_iisy11_r1300_robot" params="prefix use_fake_hardware:=false">
+  <xacro:macro name="kuka_lbr_iisy11_r1300_robot" params="prefix controller_ip client_ip use_fake_hardware">
     <!-- ros2 control instance -->
     <xacro:kuka_lbr_iisy_ros2_control
     name="lbr_iisy11_r1300"
     prefix="${prefix}"
+    client_ip="${client_ip}"
+    controller_ip="${controller_ip}"
     use_fake_hardware="${use_fake_hardware}" />
     <!-- links - main serial chain -->

File: kuka_lbr_iisy_support/urdf/lbr_iisy15_r930.urdf.xacro (robot description, xacro)
@@ -4,5 +4,8 @@
     <xacro:include filename="$(find kuka_lbr_iisy_support)/urdf/lbr_iisy15_r930_macro.xacro"/>
     <!-- Read additional arguments  -->
+    <xacro:arg name="prefix" default="" />
+    <xacro:arg name="controller_ip" default="0.0.0.0" />
+    <xacro:arg name="client_ip" default="0.0.0.0" />
     <xacro:arg name="use_fake_hardware" default="false" />
-    <xacro:kuka_lbr_iisy15_r930_robot prefix="" use_fake_hardware="$(arg use_fake_hardware)"/>
+    <xacro:kuka_lbr_iisy15_r930_robot prefix="$(arg prefix)" controller_ip="$(arg controller_ip)" client_ip="$(arg client_ip)" use_fake_hardware="$(arg use_fake_hardware)"/>
 </robot>

File: kuka_lbr_iisy_support/urdf/lbr_iisy15_r930_macro.xacro (robot description, xacro)
@@ -5,9 +5,11 @@
   <xacro:include filename="$(find kuka_resources)/urdf/common_materials.xacro"/>
   <xacro:include filename="$(find kuka_lbr_iisy_support)/urdf/lbr_iisy_transmission.xacro" />
-  <xacro:macro name="kuka_lbr_iisy15_r930_robot" params="prefix use_fake_hardware:=false">
+  <xacro:macro name="kuka_lbr_iisy15_r930_robot" params="prefix controller_ip client_ip use_fake_hardware">
     <!-- ros2 control instance -->
     <xacro:kuka_lbr_iisy_ros2_control
     name="lbr_iisy15_r930"
     prefix="${prefix}"
+    client_ip="${client_ip}"
+    controller_ip="${controller_ip}"
     use_fake_hardware="${use_fake_hardware}" />
     <!-- links - main serial chain -->

File: kuka_lbr_iisy_support/urdf/lbr_iisy3_r760.urdf.xacro (robot description, xacro)
@@ -4,5 +4,8 @@
     <xacro:include filename="$(find kuka_lbr_iisy_support)/urdf/lbr_iisy3_r760_macro.xacro"/>
     <!-- Read additional arguments  -->
+    <xacro:arg name="prefix" default="" />
+    <xacro:arg name="controller_ip" default="0.0.0.0" />
+    <xacro:arg name="client_ip" default="0.0.0.0" />
     <xacro:arg name="use_fake_hardware" default="false" />
-    <xacro:kuka_lbr_iisy3_r760_robot prefix="" use_fake_hardware="$(arg use_fake_hardware)"/>
+    <xacro:kuka_lbr_iisy3_r760_robot prefix="$(arg prefix)" controller_ip="$(arg controller_ip)" client_ip="$(arg client_ip)" use_fake_hardware="$(arg use_fake_hardware)"/>
 </robot>

File: kuka_lbr_iisy_support/urdf/lbr_iisy3_r760_macro.xacro (robot description, xacro)
@@ -5,9 +5,11 @@
   <xacro:include filename="$(find kuka_resources)/urdf/common_materials.xacro"/>
   <xacro:include filename="$(find kuka_lbr_iisy_support)/urdf/lbr_iisy_transmission.xacro" />
-  <xacro:macro name="kuka_lbr_iisy3_r760_robot" params="prefix use_fake_hardware:=false">
+  <xacro:macro name="kuka_lbr_iisy3_r760_robot" params="prefix controller_ip client_ip use_fake_hardware">
     <!-- ros2 control instance -->
     <xacro:kuka_lbr_iisy_ros2_control
     name="lbr_iisy3_r760"
     prefix="${prefix}"
+    client_ip="${client_ip}"
+    controller_ip="${controller_ip}"
     use_fake_hardware="${use_fake_hardware}" />
     <!-- links - main serial chain -->

File: kuka_lbr_iisy_support/urdf/lbr_iisy_ros2_control.xacro (robot description, xacro)
@@ -1,5 +1,5 @@
 <?xml version="1.0" encoding="UTF-8"?>
 <robot xmlns:xacro="http://www.ros.org/wiki/xacro">
-  <xacro:macro name="kuka_lbr_iisy_ros2_control" params="name prefix use_fake_hardware:=false">
+  <xacro:macro name="kuka_lbr_iisy_ros2_control" params="name prefix client_ip controller_ip use_fake_hardware">
     <ros2_control name="${name}" type="system">
       <hardware>
@@ -10,10 +10,4 @@
         </xacro:if>
         <xacro:unless value="${use_fake_hardware}">
-          <!-- Read parameters from driver_config  -->
-          <xacro:property name="driver_config" value="$(find kuka_iiqka_eac_driver)/config/driver_config.yaml" />
-          <xacro:property name="driver_config_dict" value="${xacro.load_yaml(driver_config)}"/>
-          <xacro:property name="control_mode" value="${driver_config_dict['robot_manager']['ros__parameters']['control_mode']}" />
-          <xacro:property name="client_ip" value="${driver_config_dict['robot_manager']['ros__parameters']['client_ip']}" />
-          <xacro:property name="controller_ip" value="${driver_config_dict['robot_manager']['ros__parameters']['controller_ip']}" />
           <!-- Read QoS profile parameters  -->
           <xacro:property name="qos_config" value="$(find kuka_iiqka_eac_driver)/config/qos_profiles.yaml" />
@@ -25,5 +19,4 @@
           <param name="client_ip">${client_ip}</param>
           <param name="controller_ip">${controller_ip}</param>
-          <param name="control_mode">${control_mode}</param>
           <param name="consequent_lost_packets">${consequent_lost_packets}</param>
           <param name="lost_packets_in_timeframe">${lost_packets_in_timeframe}</param>
