Commit message: remove prefix from base_link

File: kuka_lbr_iisy_support/urdf/lbr_iisy11_r1300.urdf.xacro (robot description, xacro)
@@ -8,4 +8,10 @@
     <xacro:arg name="client_ip" default="0.0.0.0" />
     <xacro:arg name="use_fake_hardware" default="false" />
-    <xacro:kuka_lbr_iisy11_r1300_robot prefix="$(arg prefix)" controller_ip="$(arg controller_ip)" client_ip="$(arg client_ip)" use_fake_hardware="$(arg use_fake_hardware)"/>
+    <xacro:kuka_lbr_iisy11_r1300_robot
+        prefix="$(arg prefix)"
+        controller_ip="$(arg controller_ip)"
+        client_ip="$(arg client_ip)"
+        use_fake_hardware="$(arg use_fake_hardware)">
+        <origin xyz="0 0 0" rpy="0 0 0" />
+    </xacro:kuka_lbr_iisy11_r1300_robot>
 </robot>

File: kuka_lbr_iisy_support/urdf/lbr_iisy11_r1300_macro.xacro (robot description, xacro)
@@ -5,8 +5,8 @@
   <xacro:include filename="$(find kuka_resources)/urdf/common_materials.xacro"/>
   <xacro:include filename="$(find kuka_lbr_iisy_support)/urdf/lbr_iisy_transmission.xacro" />
-  <xacro:macro name="kuka_lbr_iisy11_r1300_robot" params="prefix controller_ip client_ip use_fake_hardware">
+  <xacro:macro name="kuka_lbr_iisy11_r1300_robot" params="prefix controller_ip client_ip use_fake_hardware *origin">
     <!-- ros2 control instance -->
     <xacro:kuka_lbr_iisy_ros2_control
-    name="lbr_iisy11_r1300"
+    name="${prefix}lbr_iisy11_r1300"
     prefix="${prefix}"
     client_ip="${client_ip}"
@@ -15,5 +15,5 @@
     <!-- links - main serial chain -->
     <!-- links - root element cannot have inertia, therefore a dummy base_link is needed -->
-    <link name="${prefix}base_link"/>
+    <link name="base_link"/>
     <link name="${prefix}base_link_inertia">
       <collision>
@@ -158,7 +158,7 @@
     <!-- joints - main serial chain -->
     <joint name="${prefix}base_link-base_link_inertia" type="fixed">
-      <parent link="${prefix}base_link" />
+      <parent link="base_link" />
       <child link="${prefix}base_link_inertia" />
-      <origin xyz="0 0 0" rpy="0 0 0" />
+      <xacro:insert_block name="origin" />
     </joint>
     <joint name="${prefix}joint_1" type="revolute">
@@ -208,5 +208,5 @@
     <joint name="${prefix}base_link-base" type="fixed">
       <origin xyz="0 0 0" rpy="0 0 0"/>
-      <parent link="${prefix}base_link"/>
+      <parent link="${prefix}base_link_inertia"/>
       <child link="${prefix}base"/>
     </joint>

File: kuka_lbr_iisy_support/urdf/lbr_iisy15_r930.urdf.xacro (robot description, xacro)
@@ -8,4 +8,10 @@
     <xacro:arg name="client_ip" default="0.0.0.0" />
     <xacro:arg name="use_fake_hardware" default="false" />
-    <xacro:kuka_lbr_iisy15_r930_robot prefix="$(arg prefix)" controller_ip="$(arg controller_ip)" client_ip="$(arg client_ip)" use_fake_hardware="$(arg use_fake_hardware)"/>
+    <xacro:kuka_lbr_iisy15_r930_robot
+        prefix="$(arg prefix)"
+        controller_ip="$(arg controller_ip)"
+        client_ip="$(arg client_ip)"
+        use_fake_hardware="$(arg use_fake_hardware)">
+        <origin xyz="10 0 0" rpy="0 0 0" />
+    </xacro:kuka_lbr_iisy15_r930_robot>
 </robot>

File: kuka_lbr_iisy_support/urdf/lbr_iisy15_r930_macro.xacro (robot description, xacro)
@@ -5,8 +5,8 @@
   <xacro:include filename="$(find kuka_resources)/urdf/common_materials.xacro"/>
   <xacro:include filename="$(find kuka_lbr_iisy_support)/urdf/lbr_iisy_transmission.xacro" />
-  <xacro:macro name="kuka_lbr_iisy15_r930_robot" params="prefix controller_ip client_ip use_fake_hardware">
+  <xacro:macro name="kuka_lbr_iisy15_r930_robot" params="prefix controller_ip client_ip use_fake_hardware *origin">
     <!-- ros2 control instance -->
     <xacro:kuka_lbr_iisy_ros2_control
-    name="lbr_iisy15_r930"
+    name="${prefix}lbr_iisy15_r930"
     prefix="${prefix}"
     client_ip="${client_ip}"
@@ -15,5 +15,5 @@
     <!-- links - main serial chain -->
     <!-- links - root element cannot have inertia, therefore a dummy base_link is needed -->
-    <link name="${prefix}base_link"/>
+    <link name="base_link"/>
     <link name="${prefix}base_link_inertia">
       <collision>
@@ -158,7 +158,7 @@
     <!-- joints - main serial chain -->
     <joint name="${prefix}base_link-base_link_inertia" type="fixed">
-      <parent link="${prefix}base_link" />
+      <parent link="base_link" />
       <child link="${prefix}base_link_inertia" />
-      <origin xyz="0 0 0" rpy="0 0 0" />
+      <xacro:insert_block name="origin" />
     </joint>
     <joint name="${prefix}joint_1" type="revolute">
@@ -208,5 +208,5 @@
     <joint name="${prefix}base_link-base" type="fixed">
       <origin xyz="0 0 0" rpy="0 0 0"/>
-      <parent link="${prefix}base_link"/>
+      <parent link="${prefix}base_link_inertia"/>
       <child link="${prefix}base"/>
     </joint>

File: kuka_lbr_iisy_support/urdf/lbr_iisy3_r760.urdf.xacro (robot description, xacro)
@@ -8,4 +8,10 @@
     <xacro:arg name="client_ip" default="0.0.0.0" />
     <xacro:arg name="use_fake_hardware" default="false" />
-    <xacro:kuka_lbr_iisy3_r760_robot prefix="$(arg prefix)" controller_ip="$(arg controller_ip)" client_ip="$(arg client_ip)" use_fake_hardware="$(arg use_fake_hardware)"/>
+    <xacro:kuka_lbr_iisy3_r760_robot
+        prefix="$(arg prefix)"
+        controller_ip="$(arg controller_ip)"
+        client_ip="$(arg client_ip)"
+        use_fake_hardware="$(arg use_fake_hardware)">
+        <origin xyz="10 0 0" rpy="0 0 0" />
+    </xacro:kuka_lbr_iisy3_r760_robot>
 </robot>

File: kuka_lbr_iisy_support/urdf/lbr_iisy3_r760_macro.xacro (robot description, xacro)
@@ -5,8 +5,8 @@
   <xacro:include filename="$(find kuka_resources)/urdf/common_materials.xacro"/>
   <xacro:include filename="$(find kuka_lbr_iisy_support)/urdf/lbr_iisy_transmission.xacro" />
-  <xacro:macro name="kuka_lbr_iisy3_r760_robot" params="prefix controller_ip client_ip use_fake_hardware">
+  <xacro:macro name="kuka_lbr_iisy3_r760_robot" params="prefix controller_ip client_ip use_fake_hardware *origin">
     <!-- ros2 control instance -->
     <xacro:kuka_lbr_iisy_ros2_control
-    name="lbr_iisy3_r760"
+    name="${prefix}lbr_iisy3_r760"
     prefix="${prefix}"
     client_ip="${client_ip}"
@@ -15,5 +15,5 @@
     <!-- links - main serial chain -->
     <!-- links - root element cannot have inertia, therefore a dummy base_link is needed -->
-    <link name="${prefix}base_link"/>
+    <link name="base_link"/>
     <link name="${prefix}base_link_inertia">
       <collision>
@@ -158,7 +158,7 @@
     <!-- joints - main serial chain -->
     <joint name="${prefix}base_link-base_link_inertia" type="fixed">
-      <parent link="${prefix}base_link" />
+      <parent link="base_link" />
       <child link="${prefix}base_link_inertia" />
-      <origin xyz="0 0 0" rpy="0 0 0" />
+      <xacro:insert_block name="origin" />
     </joint>
     <joint name="${prefix}joint_1" type="revolute">
@@ -208,5 +208,5 @@
     <joint name="${prefix}base_link-base" type="fixed">
       <origin xyz="0 0 0" rpy="0 0 0"/>
-      <parent link="${prefix}base_link"/>
+      <parent link="${prefix}base_link_inertia"/>
       <child link="${prefix}base"/>
     </joint>

Commit message: add all dofs to all iisys

File: kuka_lbr_iisy_support/urdf/lbr_iisy11_r1300.urdf.xacro (robot description, xacro)
@@ -8,4 +8,7 @@
     <xacro:arg name="client_ip" default="0.0.0.0" />
     <xacro:arg name="use_fake_hardware" default="false" />
+    <xacro:arg name="roll" default="0" />
+    <xacro:arg name="pitch" default="0" />
+    <xacro:arg name="yaw" default="0" />
     <xacro:kuka_lbr_iisy11_r1300_robot
         prefix="$(arg prefix)"
@@ -13,5 +16,5 @@
         client_ip="$(arg client_ip)"
         use_fake_hardware="$(arg use_fake_hardware)">
-        <origin xyz="0 0 0" rpy="0 0 0" />
+        <origin xyz="$(arg x) $(arg y) $(arg z)" rpy="$(arg roll) $(arg pitch) $(arg yaw)" />
     </xacro:kuka_lbr_iisy11_r1300_robot>
 </robot>

File: kuka_lbr_iisy_support/urdf/lbr_iisy15_r930.urdf.xacro (robot description, xacro)
@@ -8,4 +8,10 @@
     <xacro:arg name="client_ip" default="0.0.0.0" />
     <xacro:arg name="use_fake_hardware" default="false" />
+    <xacro:arg name="x" default="0" />
+    <xacro:arg name="y" default="0" />
+    <xacro:arg name="z" default="0" />
+    <xacro:arg name="roll" default="0" />
+    <xacro:arg name="pitch" default="0" />
+    <xacro:arg name="yaw" default="0" />
     <xacro:kuka_lbr_iisy15_r930_robot
         prefix="$(arg prefix)"
@@ -13,5 +19,5 @@
         client_ip="$(arg client_ip)"
         use_fake_hardware="$(arg use_fake_hardware)">
-        <origin xyz="10 0 0" rpy="0 0 0" />
+        <origin xyz="$(arg x) $(arg y) $(arg z)" rpy="$(arg roll) $(arg pitch) $(arg yaw)" />
     </xacro:kuka_lbr_iisy15_r930_robot>
 </robot>

File: kuka_lbr_iisy_support/urdf/lbr_iisy3_r760.urdf.xacro (robot description, xacro)
@@ -8,4 +8,10 @@
     <xacro:arg name="client_ip" default="0.0.0.0" />
     <xacro:arg name="use_fake_hardware" default="false" />
+    <xacro:arg name="x" default="0" />
+    <xacro:arg name="y" default="0" />
+    <xacro:arg name="z" default="0" />
+    <xacro:arg name="roll" default="0" />
+    <xacro:arg name="pitch" default="0" />
+    <xacro:arg name="yaw" default="0" />
     <xacro:kuka_lbr_iisy3_r760_robot
         prefix="$(arg prefix)"
@@ -13,5 +19,5 @@
         client_ip="$(arg client_ip)"
         use_fake_hardware="$(arg use_fake_hardware)">
-        <origin xyz="0 0 0" rpy="0 0 0" />
+        <origin xyz="$(arg x) $(arg y) $(arg z)" rpy="$(arg roll) $(arg pitch) $(arg yaw)" />
     </xacro:kuka_lbr_iisy3_r760_robot>
 </robot>

Commit message: add qos config file arg

File: kuka_lbr_iisy_support/urdf/lbr_iisy11_r1300.urdf.xacro (robot description, xacro)
@@ -8,4 +8,5 @@
     <xacro:arg name="client_ip" default="0.0.0.0" />
     <xacro:arg name="use_fake_hardware" default="false" />
+    <xacro:arg name="qos_config_file" default="$(find kuka_iiqka_eac_driver)/config/qos_profiles.yaml">
     <xacro:arg name="x" default="0" />
     <xacro:arg name="y" default="0" />
@@ -18,5 +19,6 @@
         controller_ip="$(arg controller_ip)"
         client_ip="$(arg client_ip)"
-        use_fake_hardware="$(arg use_fake_hardware)">
+        use_fake_hardware="$(arg use_fake_hardware)"
+        qos_config_file="$(arg qos_config_file)">
         <origin xyz="$(arg x) $(arg y) $(arg z)" rpy="$(arg roll) $(arg pitch) $(arg yaw)" />
     </xacro:kuka_lbr_iisy11_r1300_robot>

File: kuka_lbr_iisy_support/urdf/lbr_iisy11_r1300_macro.xacro (robot description, xacro)
@@ -5,5 +5,5 @@
   <xacro:include filename="$(find kuka_resources)/urdf/common_materials.xacro"/>
   <xacro:include filename="$(find kuka_lbr_iisy_support)/urdf/lbr_iisy_transmission.xacro" />
-  <xacro:macro name="kuka_lbr_iisy11_r1300_robot" params="prefix controller_ip client_ip use_fake_hardware *origin">
+  <xacro:macro name="kuka_lbr_iisy11_r1300_robot" params="prefix controller_ip client_ip use_fake_hardware qos_config_file *origin">
     <!-- ros2 control instance -->
     <xacro:kuka_lbr_iisy_ros2_control
@@ -12,5 +12,6 @@
     client_ip="${client_ip}"
     controller_ip="${controller_ip}"
-    use_fake_hardware="${use_fake_hardware}" />
+    use_fake_hardware="${use_fake_hardware}"
+    qos_config_file="${qos_config_file}" />
     <!-- links - main serial chain -->
     <!-- links - root element cannot have inertia, therefore a dummy base_link is needed -->

File: kuka_lbr_iisy_support/urdf/lbr_iisy15_r930.urdf.xacro (robot description, xacro)
@@ -8,4 +8,5 @@
     <xacro:arg name="client_ip" default="0.0.0.0" />
     <xacro:arg name="use_fake_hardware" default="false" />
+    <xacro:arg name="qos_config_file" default="$(find kuka_iiqka_eac_driver)/config/qos_profiles.yaml">
     <xacro:arg name="x" default="0" />
     <xacro:arg name="y" default="0" />
@@ -18,5 +19,6 @@
         controller_ip="$(arg controller_ip)"
         client_ip="$(arg client_ip)"
-        use_fake_hardware="$(arg use_fake_hardware)">
+        use_fake_hardware="$(arg use_fake_hardware)"
+        qos_config_file="$(arg qos_config_file)">
         <origin xyz="$(arg x) $(arg y) $(arg z)" rpy="$(arg roll) $(arg pitch) $(arg yaw)" />
     </xacro:kuka_lbr_iisy15_r930_robot>

File: kuka_lbr_iisy_support/urdf/lbr_iisy15_r930_macro.xacro (robot description, xacro)
@@ -5,5 +5,5 @@
   <xacro:include filename="$(find kuka_resources)/urdf/common_materials.xacro"/>
   <xacro:include filename="$(find kuka_lbr_iisy_support)/urdf/lbr_iisy_transmission.xacro" />
-  <xacro:macro name="kuka_lbr_iisy15_r930_robot" params="prefix controller_ip client_ip use_fake_hardware *origin">
+  <xacro:macro name="kuka_lbr_iisy15_r930_robot" params="prefix controller_ip client_ip use_fake_hardware qos_config_file *origin">
     <!-- ros2 control instance -->
     <xacro:kuka_lbr_iisy_ros2_control
@@ -12,5 +12,6 @@
     client_ip="${client_ip}"
     controller_ip="${controller_ip}"
-    use_fake_hardware="${use_fake_hardware}" />
+    use_fake_hardware="${use_fake_hardware}"
+    qos_config_file="${qos_config_file}" />
     <!-- links - main serial chain -->
     <!-- links - root element cannot have inertia, therefore a dummy base_link is needed -->

File: kuka_lbr_iisy_support/urdf/lbr_iisy3_r760.urdf.xacro (robot description, xacro)
@@ -8,4 +8,5 @@
     <xacro:arg name="client_ip" default="0.0.0.0" />
     <xacro:arg name="use_fake_hardware" default="false" />
+    <xacro:arg name="qos_config_file" default="$(find kuka_iiqka_eac_driver)/config/qos_profiles.yaml">
     <xacro:arg name="x" default="0" />
     <xacro:arg name="y" default="0" />
@@ -18,5 +19,6 @@
         controller_ip="$(arg controller_ip)"
         client_ip="$(arg client_ip)"
-        use_fake_hardware="$(arg use_fake_hardware)">
+        use_fake_hardware="$(arg use_fake_hardware)"
+        qos_config_file="$(arg qos_config_file)">
         <origin xyz="$(arg x) $(arg y) $(arg z)" rpy="$(arg roll) $(arg pitch) $(arg yaw)" />
     </xacro:kuka_lbr_iisy3_r760_robot>

File: kuka_lbr_iisy_support/urdf/lbr_iisy3_r760_macro.xacro (robot description, xacro)
@@ -5,5 +5,5 @@
   <xacro:include filename="$(find kuka_resources)/urdf/common_materials.xacro"/>
   <xacro:include filename="$(find kuka_lbr_iisy_support)/urdf/lbr_iisy_transmission.xacro" />
-  <xacro:macro name="kuka_lbr_iisy3_r760_robot" params="prefix controller_ip client_ip use_fake_hardware *origin">
+  <xacro:macro name="kuka_lbr_iisy3_r760_robot" params="prefix controller_ip client_ip use_fake_hardware qos_config_file *origin">
     <!-- ros2 control instance -->
     <xacro:kuka_lbr_iisy_ros2_control
@@ -12,5 +12,6 @@
     client_ip="${client_ip}"
     controller_ip="${controller_ip}"
-    use_fake_hardware="${use_fake_hardware}" />
+    use_fake_hardware="${use_fake_hardware}"
+    qos_config_file="${qos_config_file}" />
     <!-- links - main serial chain -->
     <!-- links - root element cannot have inertia, therefore a dummy base_link is needed -->

File: kuka_lbr_iisy_support/urdf/lbr_iisy_ros2_control.xacro (robot description, xacro)
@@ -1,5 +1,5 @@
 <?xml version="1.0" encoding="UTF-8"?>
 <robot xmlns:xacro="http://www.ros.org/wiki/xacro">
-  <xacro:macro name="kuka_lbr_iisy_ros2_control" params="name prefix client_ip controller_ip use_fake_hardware">
+  <xacro:macro name="kuka_lbr_iisy_ros2_control" params="name prefix client_ip controller_ip use_fake_hardware qos_config_file">
     <ros2_control name="${name}" type="system">
       <hardware>
@@ -11,5 +11,5 @@
         <xacro:unless value="${use_fake_hardware}">
           <!-- Read QoS profile parameters  -->
-          <xacro:property name="qos_config" value="$(find kuka_iiqka_eac_driver)/config/qos_profiles.yaml" />
+          <xacro:property name="qos_config" value="${qos_config_file}" />
           <xacro:property name="qos_config_dict" value="${xacro.load_yaml(qos_config)}"/>
           <xacro:property name="consequent_lost_packets" value="${qos_config_dict['rt_packet_loss_profile']['consequent_lost_packets']}" />

Commit message: workaround for  kuka_iiqka_eac_driver

File: kuka_lbr_iisy_support/urdf/lbr_iisy11_r1300.urdf.xacro (robot description, xacro)
@@ -8,5 +8,5 @@
     <xacro:arg name="client_ip" default="0.0.0.0" />
     <xacro:arg name="use_fake_hardware" default="false" />
-    <xacro:arg name="qos_config_file" default="$(find kuka_iiqka_eac_driver)/config/qos_config.yaml"/>
+    <xacro:arg name="qos_config_file" default=""/>
     <xacro:arg name="x" default="0" />
     <xacro:arg name="y" default="0" />

File: kuka_lbr_iisy_support/urdf/lbr_iisy15_r930.urdf.xacro (robot description, xacro)
@@ -8,5 +8,5 @@
     <xacro:arg name="client_ip" default="0.0.0.0" />
     <xacro:arg name="use_fake_hardware" default="false" />
-    <xacro:arg name="qos_config_file" default="$(find kuka_iiqka_eac_driver)/config/qos_config.yaml"/>
+    <xacro:arg name="qos_config_file" default=""/>
     <xacro:arg name="x" default="0" />
     <xacro:arg name="y" default="0" />

File: kuka_lbr_iisy_support/urdf/lbr_iisy3_r760.urdf.xacro (robot description, xacro)
@@ -8,5 +8,5 @@
     <xacro:arg name="client_ip" default="0.0.0.0" />
     <xacro:arg name="use_fake_hardware" default="false" />
-    <xacro:arg name="qos_config_file" default="$(find kuka_iiqka_eac_driver)/config/qos_config.yaml"/>
+    <xacro:arg name="qos_config_file" default=""/>
     <xacro:arg name="x" default="0" />
     <xacro:arg name="y" default="0" />

File: kuka_lbr_iisy_support/urdf/lbr_iisy_ros2_control.xacro (robot description, xacro)
@@ -11,5 +11,10 @@
         <xacro:unless value="${use_fake_hardware}">
           <!-- Read QoS profile parameters  -->
-          <xacro:property name="qos_config" value="${qos_config_file}" />
+          <xacro:if value="${qos_config_file == ''}">
+            <xacro:property name="qos_config" value="$(find kuka_iiqka_eac_driver)/config/qos_config.yaml"/>
+          </xacro:if>
+          <xacro:unless value="${qos_config_file == ''}">
+            <xacro:property name="qos_config" value="${qos_config_file}"/>
+          </xacro:unless>
           <xacro:property name="qos_config_dict" value="${xacro.load_yaml(qos_config)}"/>
           <xacro:property name="consequent_lost_packets" value="${qos_config_dict['rt_packet_loss_profile']['consequent_lost_packets']}" />
