Commit message: rm unnec macro if-else, add default qos_config_file value

File: kuka_lbr_iisy_support/urdf/lbr_iisy_ros2_control_macro.xacro (robot description, xacro)
@@ -1,5 +1,5 @@
 <?xml version="1.0" encoding="UTF-8"?>
 <robot xmlns:xacro="http://www.ros.org/wiki/xacro">
-  <xacro:macro name="kuka_lbr_iisy_ros2_control" params="name driver_version prefix client_ip client_port mxa_client_port controller_ip use_gpio mode qos_config_file roundtrip_time verify_robot_model rsi_xml_config_file gazebo_controller_config_path:=config/fake_hardware_config_6_axis.yaml **ext_axes_ros2_control_joints">
+  <xacro:macro name="kuka_lbr_iisy_ros2_control" params="name driver_version prefix client_ip client_port mxa_client_port controller_ip use_gpio mode qos_config_file='' roundtrip_time verify_robot_model rsi_xml_config_file gazebo_controller_config_path:=config/fake_hardware_config_6_axis.yaml **ext_axes_ros2_control_joints">
     <!-- gazebo -->
     <xacro:if value="${mode == 'gazebo'}">

File: kuka_resources/urdf/robot_with_external_axis_template.urdf.xacro (robot description, xacro)
@@ -52,18 +52,9 @@
   <xacro:include filename="${kl_support_urdf_dir}/$(arg kl_ros2_control_macro_file)"/>
   <!-- ros2 control configuration -->
-  <xacro:if value="${robot_ros2_control_macro_name == 'kuka_lbr_iisy_ros2_control'}">
-    <xacro:call macro="${robot_ros2_control_macro_name}" name="$(arg prefix)$(arg composed_model)" driver_version="$(arg driver_version)" client_ip="$(arg client_ip)" client_port="$(arg client_port)" mxa_client_port="$(arg mxa_client_port)" controller_ip="$(arg controller_ip)" prefix="$(arg prefix)" use_gpio="$(arg use_gpio)" mode="$(arg mode)" qos_config_file="" roundtrip_time="$(arg roundtrip_time)" verify_robot_model="$(arg verify_robot_model)" rsi_xml_config_file="$(arg rsi_xml_config_file)" gazebo_controller_config_path="$(arg gazebo_controller_config_path)">
-      <ext_axes_ros2_control_joints>
-        <xacro:call macro="${kl_ros2_control_joints_macro_name}" prefix="${kl_full_prefix}" mode="$(arg mode)"/>
-      </ext_axes_ros2_control_joints>
-    </xacro:call>
-  </xacro:if>
-  <xacro:unless value="${robot_ros2_control_macro_name == 'kuka_lbr_iisy_ros2_control'}">
-    <xacro:call macro="${robot_ros2_control_macro_name}" name="$(arg prefix)$(arg composed_model)" driver_version="$(arg driver_version)" client_ip="$(arg client_ip)" client_port="$(arg client_port)" mxa_client_port="$(arg mxa_client_port)" controller_ip="$(arg controller_ip)" prefix="$(arg prefix)" use_gpio="$(arg use_gpio)" mode="$(arg mode)" roundtrip_time="$(arg roundtrip_time)" verify_robot_model="$(arg verify_robot_model)" rsi_xml_config_file="$(arg rsi_xml_config_file)" gazebo_controller_config_path="$(arg gazebo_controller_config_path)">
-      <ext_axes_ros2_control_joints>
-        <xacro:call macro="${kl_ros2_control_joints_macro_name}" prefix="${kl_full_prefix}" mode="$(arg mode)"/>
-      </ext_axes_ros2_control_joints>
-    </xacro:call>
-  </xacro:unless>
+  <xacro:call macro="${robot_ros2_control_macro_name}" name="$(arg prefix)$(arg composed_model)" driver_version="$(arg driver_version)" client_ip="$(arg client_ip)" client_port="$(arg client_port)" mxa_client_port="$(arg mxa_client_port)" controller_ip="$(arg controller_ip)" prefix="$(arg prefix)" use_gpio="$(arg use_gpio)" mode="$(arg mode)" roundtrip_time="$(arg roundtrip_time)" verify_robot_model="$(arg verify_robot_model)" rsi_xml_config_file="$(arg rsi_xml_config_file)" gazebo_controller_config_path="$(arg gazebo_controller_config_path)">
+    <ext_axes_ros2_control_joints>
+      <xacro:call macro="${kl_ros2_control_joints_macro_name}" prefix="${kl_full_prefix}" mode="$(arg mode)"/>
+    </ext_axes_ros2_control_joints>
+  </xacro:call>
   <!-- world link -->
   <link name="world"/>
