Commit message: added omnimove model

File: kuka_omnimove_e575_support/urdf/omnimove_with_arm.xacro (robot description, xacro)
@@ -2,4 +2,9 @@
 <robot name="kuka_kr6r700sixx" xmlns:xacro="http://wiki.ros.org/xacro">
   <xacro:include filename="$(find kuka_agilus_support)/urdf/kr6_r700_sixx.urdf.xacro"/>
- <!-- <xacro:kuka_kr6_r700_sixx_robot prefix=""/> -->
+  <xacro:include filename="$(find kuka_omnimove_e575_support)/urdf/omnimove.xacro"/>
+  <xacro:omnimove prefix="omnimove_"/>
+  <joint name="omnibase" type="fixed">
+    <parent link="omnimove_base"/>
+    <child link="base_link"/>
+  </joint>
 </robot>
