Commit message: created omnimove.xacro which uses ros2_control plugin forward_controller not yet working

File: kuka_omnimove_e575_support/urdf/omnimove.xacro (robot description, xacro)
@@ -19,3 +19,16 @@
       </link>
   </xacro:macro>
+  <xacro:macro name="omnimove_ros2_control" params="name">
+      <ros2_control name="omnimove" type="system">
+            <hardware>
+                <plugin>omnimove::OmnimoveExternalControl</plugin>
+            </hardware>
+            <joint name="move">
+                <command_interface name="velocity">
+                </command_interface>
+                <state_interface name="position"/>
+                <state_interface name="velocity"/>
+            </joint>
+      </ros2_control>
+  </xacro:macro>
 </robot>

File: kuka_omnimove_e575_support/urdf/omnimove_with_arm.xacro (robot description, xacro)
@@ -4,4 +4,5 @@
   <xacro:include filename="$(find kuka_omnimove_e575_support)/urdf/omnimove.xacro"/>
   <xacro:omnimove prefix="omnimove_"/>
+  <xacro:omnimove_ros2_control name="omnimove"/>
   <joint name="omnibase" type="fixed">
     <parent link="omnimove_base"/>

Commit message: added joints per axis to the omnimove. makes adding extra fields only a configuration. created dummy forward_contrller for testing.

File: kuka_omnimove_e575_support/urdf/omnimove.xacro (robot description, xacro)
@@ -24,7 +24,21 @@
                 <plugin>omnimove::OmnimoveExternalControl</plugin>
             </hardware>
-            <joint name="move">
-                <command_interface name="velocity">
-                </command_interface>
+            <joint name="move_x">
+                <command_interface name="velocity"/>
+                <state_interface name="position"/>
+                <state_interface name="velocity"/>
+            </joint>
+            <joint name="move_y">
+                <command_interface name="velocity"/>
+                <state_interface name="position"/>
+                <state_interface name="velocity"/>
+            </joint>
+            <joint name="move_theta">
+                <command_interface name="velocity"/>
+                <state_interface name="position"/>
+                <state_interface name="velocity"/>
+            </joint>
+            <joint name="move_lift">
+                <command_interface name="velocity"/>
                 <state_interface name="position"/>
                 <state_interface name="velocity"/>

Commit message: added correct parameters for external control

File: kuka_omnimove_e575_support/urdf/omnimove.xacro (robot description, xacro)
@@ -9,5 +9,4 @@
             <mesh filename="package://kuka_omnimove_e575_support/meshes/omnimove_simplified.dae" />
           </geometry>
-          <!--<xacro:material_kuka_pedestal /> -->
         </visual>
         <collision>
@@ -19,8 +18,10 @@
       </link>
   </xacro:macro>
-  <xacro:macro name="omnimove_ros2_control" params="name">
-      <ros2_control name="omnimove" type="system">
+   <xacro:macro name="omnimove_ros2_control" params="name">
+	    <ros2_control name="omnimove" type="system">
             <hardware>
                 <plugin>omnimove::OmnimoveExternalControl</plugin>
+                <param name ="host">127.0.0.1</param>
+                <param name="port">24000</param>
             </hardware>
             <joint name="move_x">
@@ -44,5 +45,5 @@
                 <state_interface name="velocity"/>
             </joint>
-      </ros2_control>
+	   </ros2_control>
   </xacro:macro>
 </robot>

Commit message: added caterpillar support in urdf

File: kuka_omnimove_e575_support/urdf/omnimove.xacro (robot description, xacro)
@@ -27,20 +27,12 @@
             <joint name="move_x">
                 <command_interface name="velocity"/>
-                <state_interface name="position"/>
                 <state_interface name="velocity"/>
             </joint>
             <joint name="move_y">
                 <command_interface name="velocity"/>
-                <state_interface name="position"/>
                 <state_interface name="velocity"/>
             </joint>
             <joint name="move_theta">
                 <command_interface name="velocity"/>
-                <state_interface name="position"/>
-                <state_interface name="velocity"/>
-            </joint>
-            <joint name="move_lift">
-                <command_interface name="velocity"/>
-                <state_interface name="position"/>
                 <state_interface name="velocity"/>
             </joint>
