Commit message: removed all joints from urdf, and replaced with agv_type

File: kuka_omnimove_e575_support/urdf/caterpillar.xacro (robot description, xacro)
@@ -24,47 +24,6 @@
                 <param name ="host">127.0.0.1</param>
                 <param name="port">24000</param>
+                <param name="agv_type">caterpillar</param>
             </hardware>
-            <joint name="move_x">
-                <command_interface name="velocity"/>
-                <state_interface name="velocity"/>
-            </joint>
-<!--            <joint name="move_y">
-                <command_interface name="velocity"/>
-                <state_interface name="velocity"/>
-            </joint> -->
-            <joint name="move_theta">
-                <command_interface name="velocity"/>
-                <state_interface name="velocity"/>
-            </joint>
-            <joint name="pillar1">
-                <command_interface name="velocity"/>
-                <command_interface name="position"/>
-                <state_interface name="position"/>
-                <state_interface name="velocity"/>
-            </joint>
-            <joint name="pillar2">
-                <command_interface name="velocity"/>
-                <command_interface name="position"/>
-                <state_interface name="position"/>
-                <state_interface name="velocity"/>
-            </joint>
-            <joint name="pillar3">
-                <command_interface name="velocity"/>
-                <command_interface name="position"/>
-                <state_interface name="position"/>
-                <state_interface name="velocity"/>
-            </joint>
-            <joint name="pillar4">
-                <command_interface name="velocity"/>
-                <command_interface name="position"/>
-                <state_interface name="position"/>
-                <state_interface name="velocity"/>
-            </joint>
-            <joint name="shield">
-                <command_interface name="velocity"/>
-                <command_interface name="position"/>
-                <state_interface name="position"/>
-                <state_interface name="velocity"/>
-            </joint>
            </ros2_control>
   </xacro:macro>

File: kuka_omnimove_e575_support/urdf/omnimove.xacro (robot description, xacro)
@@ -24,17 +24,6 @@
                 <param name ="host">127.0.0.1</param>
                 <param name="port">24000</param>
+                <param name="agv_type">omnimove</param>
             </hardware>
-            <joint name="move_x">
-                <command_interface name="velocity"/>
-                <state_interface name="velocity"/>
-            </joint>
-            <joint name="move_y">
-                <command_interface name="velocity"/>
-                <state_interface name="velocity"/>
-            </joint>
-            <joint name="move_theta">
-                <command_interface name="velocity"/>
-                <state_interface name="velocity"/>
-            </joint>
 	   </ros2_control>
   </xacro:macro>

Commit message: using new caterpillar and omnimove model publishing transform between platform and robot

File: kuka_omnimove_e575_support/urdf/caterpillar.xacro (robot description, xacro)
@@ -7,5 +7,5 @@
           <origin xyz="0 0 0" rpy="0 0 0" />
           <geometry>
-            <mesh filename="package://kuka_omnimove_e575_support/meshes/omnimove_simplified.dae" />
+            <mesh filename="package://kuka_omnimove_e575_support/meshes/caterpillar_simplified.dae" />
           </geometry>
         </visual>
@@ -13,5 +13,5 @@
           <origin xyz="0 0 0" rpy="0 0 0" />
           <geometry>
-            <mesh filename="package://kuka_omnimove_e575_support/meshes/omnimove_simplified.stl" />
+            <mesh filename="package://kuka_omnimove_e575_support/meshes/caterpillar_simplified.stl" />
           </geometry>
         </collision>

File: kuka_omnimove_e575_support/urdf/omnimove.xacro (robot description, xacro)
@@ -7,5 +7,5 @@
           <origin xyz="0 0 0" rpy="0 0 0" />
           <geometry>
-            <mesh filename="package://kuka_omnimove_e575_support/meshes/omnimove_simplified.dae" />
+            <mesh filename="package://kuka_omnimove_e575_support/meshes/omnimove_simplified_2.dae" />
           </geometry>
         </visual>
@@ -13,5 +13,5 @@
           <origin xyz="0 0 0" rpy="0 0 0" />
           <geometry>
-            <mesh filename="package://kuka_omnimove_e575_support/meshes/omnimove_simplified.stl" />
+            <mesh filename="package://kuka_omnimove_e575_support/meshes/omnimove_simplified_2.stl" />
           </geometry>
         </collision>
