Commit message: add base_link_inertia

File: kuka_cybertech_support/urdf/kr16_r2010-2_macro.xacro (robot description, xacro)
@@ -11,5 +11,6 @@
     client_port="${client_port}"
     use_fake_hardware="${use_fake_hardware}" />
-    <link name="${prefix}base_link">
+    <link name="${prefix}base_link"/>
+    <link name="${prefix}base_link_inertia">
       <collision>
         <geometry>
@@ -144,4 +145,9 @@
       </visual>
     </link>
+    <joint name="${prefix}base_link-base_link_inertia" type="fixed">
+      <parent link="${prefix}base_link" />
+      <child link="${prefix}base_link_inertia" />
+      <origin xyz="0 0 0" rpy="0 0 0" />
+    </joint>
     <joint name="${prefix}joint_a1" type="revolute">
       <axis xyz="0.0 0.0 1.0"/>
@@ -149,5 +155,5 @@
       <limit effort="0.0E0" lower="-3.2288591162E0" upper="3.2288591161895095E0" velocity="4.801E3"/>
       <origin rpy="-3.141592653589793 0.0 -0.0" xyz="0.0 0.0 0.0"/>
-      <parent link="${prefix}base_link"/>
+      <parent link="${prefix}base_link_inertia"/>
     </joint>
     <joint name="${prefix}joint_a2" type="revolute">

Commit message: add effort and velocity limits

File: kuka_cybertech_support/urdf/kr16_r2010-2_macro.xacro (robot description, xacro)
@@ -153,5 +153,5 @@
       <axis xyz="0.0 0.0 1.0"/>
       <child link="${prefix}link_1"/>
-      <limit effort="0.0E0" lower="-3.2288591162E0" upper="3.2288591161895095E0" velocity="4.801E3"/>
+      <limit effort="1905.3" lower="-3.2288591162E0" upper="3.2288591161895095E0" velocity="${radians(200)}"/>
       <origin rpy="-3.141592653589793 0.0 -0.0" xyz="0.0 0.0 0.0"/>
       <parent link="${prefix}base_link_inertia"/>
@@ -160,5 +160,5 @@
       <axis xyz="0.0 0.0 1.0"/>
       <child link="${prefix}link_2"/>
-      <limit effort="0.0E0" lower="-3.2288591161895095E0" upper="1.1344640137963142E0" velocity="4.801E3"/>
+      <limit effort="1633.6259859" lower="-3.2288591161895095E0" upper="1.1344640137963142E0" velocity="${radians(175)}"/>
       <origin rpy="1.5707963267948963 0.0 -0.0" xyz="0.16 0.0 -0.52"/>
       <parent link="${prefix}link_1"/>
@@ -167,5 +167,5 @@
       <axis xyz="0.0 0.0 1.0"/>
       <child link="${prefix}link_3"/>
-      <limit effort="0.0E0" lower="-2.4085543677521746E0" upper="3.0543261909900767E0" velocity="6.001E3"/>
+      <limit effort="850.58019869" lower="-2.4085543677521746E0" upper="3.0543261909900767E0" velocity="${radians(190)}"/>
       <origin rpy="0.0 0.0 -1.5707963267948963" xyz="0.98 0.0 0.0"/>
       <parent link="${prefix}link_2"/>
@@ -174,5 +174,5 @@
       <axis xyz="0.0 0.0 1.0"/>
       <child link="${prefix}link_4"/>
-      <limit effort="0.0E0" lower="-6.1086523819801535E0" upper="6.1086523819801535E0" velocity="6.001E3"/>
+      <limit effort="266.21043332" lower="-6.1086523819801535E0" upper="6.1086523819801535E0" velocity="${radians(430)}"/>
       <origin rpy="1.5707963267948963 0.0 -0.0" xyz="0.15 0.0 0.0"/>
       <parent link="${prefix}link_3"/>
@@ -181,5 +181,5 @@
       <axis xyz="0.0 0.0 1.0"/>
       <child link="${prefix}link_5"/>
-      <limit effort="0.0E0" lower="-2.268928027593E0" upper="2.2689280275926285E0" velocity="6.001E3"/>
+      <limit effort="255.43776663" lower="-2.268928027593E0" upper="2.2689280275926285E0" velocity="${radians(430)}"/>
       <origin rpy="-1.5707963267948963 0.0 -0.0" xyz="0.0 0.0 -0.86"/>
       <parent link="${prefix}link_4"/>
@@ -188,5 +188,5 @@
       <axis xyz="0.0 0.0 1.0"/>
       <child link="${prefix}link_6"/>
-      <limit effort="0.0E0" lower="-6.1086523819801535E0" upper="6.1086523819801535E0" velocity="6.001E3"/>
+      <limit effort="111.65796" lower="-6.1086523819801535E0" upper="6.1086523819801535E0" velocity="${radians(630)}"/>
       <origin rpy="1.5707963267948963 0.0 -0.0" xyz="0.0 0.0 0.0"/>
       <parent link="${prefix}link_5"/>

Commit message: update link6-tcp

File: kuka_cybertech_support/urdf/kr16_r2010-2_macro.xacro (robot description, xacro)
@@ -203,5 +203,5 @@
     <joint name="${prefix}link6-flange" type="fixed">
       <child link="${prefix}flange" />
-      <origin rpy="0 ${pi} -0.0" xyz="0.0 0.0 -0.1605" /> <!-- TODO -->
+      <origin rpy="0 ${pi} -0.0" xyz="0.0 0.0 -0.153" /> <!-- TODO -->
       <parent link="${prefix}link_6" />
     </joint>
@@ -210,5 +210,5 @@
     <joint name="${prefix}link6-tool0" type="fixed">
       <child link="${prefix}tool0" />
-      <origin rpy="0 ${pi} -0.0" xyz="0.0 0.0 -0.1605" /> <!-- TODO -->
+      <origin rpy="0 ${pi} -0.0" xyz="0.0 0.0 -0.153" /> <!-- TODO -->
       <parent link="${prefix}link_6" />
     </joint>

Commit message: remove todo  flags

File: kuka_cybertech_support/urdf/kr16_r2010-2_macro.xacro (robot description, xacro)
@@ -203,5 +203,5 @@
     <joint name="${prefix}link6-flange" type="fixed">
       <child link="${prefix}flange" />
-      <origin rpy="0 ${pi} -0.0" xyz="0.0 0.0 -0.153" /> <!-- TODO -->
+      <origin rpy="0 ${pi} -0.0" xyz="0.0 0.0 -0.153" />
       <parent link="${prefix}link_6" />
     </joint>
@@ -210,5 +210,5 @@
     <joint name="${prefix}link6-tool0" type="fixed">
       <child link="${prefix}tool0" />
-      <origin rpy="0 ${pi} -0.0" xyz="0.0 0.0 -0.153" /> <!-- TODO -->
+      <origin rpy="0 ${pi} -0.0" xyz="0.0 0.0 -0.153" />
       <parent link="${prefix}link_6" />
     </joint>

Commit message: use pi macro

File: kuka_cybertech_support/urdf/kr16_r2010-2_macro.xacro (robot description, xacro)
@@ -154,5 +154,5 @@
       <child link="${prefix}link_1"/>
       <limit effort="1905.3" lower="-3.2288591162E0" upper="3.2288591161895095E0" velocity="${radians(200)}"/>
-      <origin rpy="-3.141592653589793 0.0 -0.0" xyz="0.0 0.0 0.0"/>
+      <origin rpy="${-pi} 0.0 -0.0" xyz="0.0 0.0 0.0"/>
       <parent link="${prefix}base_link_inertia"/>
     </joint>
@@ -161,5 +161,5 @@
       <child link="${prefix}link_2"/>
       <limit effort="1633.6259859" lower="-3.2288591161895095E0" upper="1.1344640137963142E0" velocity="${radians(175)}"/>
-      <origin rpy="1.5707963267948963 0.0 -0.0" xyz="0.16 0.0 -0.52"/>
+      <origin rpy="${pi/2.0} 0.0 -0.0" xyz="0.16 0.0 -0.52"/>
       <parent link="${prefix}link_1"/>
     </joint>
@@ -168,5 +168,5 @@
       <child link="${prefix}link_3"/>
       <limit effort="850.58019869" lower="-2.4085543677521746E0" upper="3.0543261909900767E0" velocity="${radians(190)}"/>
-      <origin rpy="0.0 0.0 -1.5707963267948963" xyz="0.98 0.0 0.0"/>
+      <origin rpy="0.0 0.0 ${-pi/2.0}" xyz="0.98 0.0 0.0"/>
       <parent link="${prefix}link_2"/>
     </joint>
@@ -175,5 +175,5 @@
       <child link="${prefix}link_4"/>
       <limit effort="266.21043332" lower="-6.1086523819801535E0" upper="6.1086523819801535E0" velocity="${radians(430)}"/>
-      <origin rpy="1.5707963267948963 0.0 -0.0" xyz="0.15 0.0 0.0"/>
+      <origin rpy="${pi/2.0} 0.0 -0.0" xyz="0.15 0.0 0.0"/>
       <parent link="${prefix}link_3"/>
     </joint>
@@ -182,5 +182,5 @@
       <child link="${prefix}link_5"/>
       <limit effort="255.43776663" lower="-2.268928027593E0" upper="2.2689280275926285E0" velocity="${radians(430)}"/>
-      <origin rpy="-1.5707963267948963 0.0 -0.0" xyz="0.0 0.0 -0.86"/>
+      <origin rpy="${-pi/2.0} 0.0 -0.0" xyz="0.0 0.0 -0.86"/>
       <parent link="${prefix}link_4"/>
     </joint>
@@ -189,5 +189,5 @@
       <child link="${prefix}link_6"/>
       <limit effort="111.65796" lower="-6.1086523819801535E0" upper="6.1086523819801535E0" velocity="${radians(630)}"/>
-      <origin rpy="1.5707963267948963 0.0 -0.0" xyz="0.0 0.0 0.0"/>
+      <origin rpy="${pi/2.0} 0.0 -0.0" xyz="0.0 0.0 0.0"/>
       <parent link="${prefix}link_5"/>
     </joint>
