Commit message: fix auto replace

File: kuka_cybertech_support/urdf/kr16_r2010_2_macro.xacro (robot description, xacro)
@@ -3,8 +3,8 @@
   <xacro:include filename="$(find kuka_cybertech_support)/urdf/kr_cybertech_ros2_control.xacro" />
   <xacro:include filename="$(find kuka_cybertech_support)/urdf/kr_cybertech_transmission.xacro" />
-  <xacro:macro name="kuka__sixxkr16_r2010_2_robot" params="prefix use_fake_hardware">
+  <xacro:macro name="kuka_kr16_r2010_2_robot" params="prefix use_fake_hardware">
     <!-- ros2 control instance -->
     <xacro:kuka_cybertech_ros2_control
-    name="_sixxkr16_r2010_2"
+    name="kr16_r2010_2"
     prefix="${prefix}"
     use_fake_hardware="${use_fake_hardware}" />
@@ -13,5 +13,5 @@
       <collision>
         <geometry>
-          <mesh filename="package://kuka_cybertech_support/meshes/_sixxkr16_r2010_2/collision/base_link.stl"/>
+          <mesh filename="package://kuka_cybertech_support/meshes/kr16_r2010_2/collision/base_link.stl"/>
         </geometry>
         <origin rpy="-0.0 0.0 -0.0" xyz="0.0 0.0 0.0"/>
@@ -24,5 +24,5 @@
       <visual>
         <geometry>
-          <mesh filename="package://kuka_cybertech_support/meshes/_sixxkr16_r2010_2/visual/base_link.stl"/>
+          <mesh filename="package://kuka_cybertech_support/meshes/kr16_r2010_2/visual/base_link.stl"/>
         </geometry>
         <origin rpy="-0.0 0.0 -0.0" xyz="0.0 0.0 0.0"/>
@@ -32,5 +32,5 @@
       <collision>
         <geometry>
-          <mesh filename="package://kuka_cybertech_support/meshes/_sixxkr16_r2010_2/collision/link_1.stl"/>
+          <mesh filename="package://kuka_cybertech_support/meshes/kr16_r2010_2/collision/link_1.stl"/>
         </geometry>
         <origin rpy="-0.0 0.0 -0.0" xyz="0.0 0.0 0.0"/>
@@ -43,5 +43,5 @@
       <visual>
         <geometry>
-          <mesh filename="package://kuka_cybertech_support/meshes/_sixxkr16_r2010_2/visual/link_1.stl"/>
+          <mesh filename="package://kuka_cybertech_support/meshes/kr16_r2010_2/visual/link_1.stl"/>
         </geometry>
         <origin rpy="-0.0 0.0 -0.0" xyz="0.0 0.0 0.0"/>
@@ -51,5 +51,5 @@
       <collision>
         <geometry>
-          <mesh filename="package://kuka_cybertech_support/meshes/_sixxkr16_r2010_2/collision/link_2.stl"/>
+          <mesh filename="package://kuka_cybertech_support/meshes/kr16_r2010_2/collision/link_2.stl"/>
         </geometry>
         <origin rpy="-0.0 0.0 -0.0" xyz="0.0 0.0 0.0"/>
@@ -62,5 +62,5 @@
       <visual>
         <geometry>
-          <mesh filename="package://kuka_cybertech_support/meshes/_sixxkr16_r2010_2/visual/link_2.stl"/>
+          <mesh filename="package://kuka_cybertech_support/meshes/kr16_r2010_2/visual/link_2.stl"/>
         </geometry>
         <origin rpy="-0.0 0.0 -0.0" xyz="0.0 0.0 0.0"/>
@@ -70,5 +70,5 @@
       <collision>
         <geometry>
-          <mesh filename="package://kuka_cybertech_support/meshes/_sixxkr16_r2010_2/collision/link_3.stl"/>
+          <mesh filename="package://kuka_cybertech_support/meshes/kr16_r2010_2/collision/link_3.stl"/>
         </geometry>
         <origin rpy="-0.0 0.0 -0.0" xyz="0.0 0.0 0.0"/>
@@ -81,5 +81,5 @@
       <visual>
         <geometry>
-          <mesh filename="package://kuka_cybertech_support/meshes/_sixxkr16_r2010_2/visual/link_3.stl"/>
+          <mesh filename="package://kuka_cybertech_support/meshes/kr16_r2010_2/visual/link_3.stl"/>
         </geometry>
         <origin rpy="-0.0 0.0 -0.0" xyz="0.0 0.0 0.0"/>
@@ -89,5 +89,5 @@
       <collision>
         <geometry>
-          <mesh filename="package://kuka_cybertech_support/meshes/_sixxkr16_r2010_2/collision/link_4.stl"/>
+          <mesh filename="package://kuka_cybertech_support/meshes/kr16_r2010_2/collision/link_4.stl"/>
         </geometry>
         <origin rpy="-0.0 0.0 -0.0" xyz="0.0 0.0 0.0"/>
@@ -100,5 +100,5 @@
       <visual>
         <geometry>
-          <mesh filename="package://kuka_cybertech_support/meshes/_sixxkr16_r2010_2/visual/link_4.stl"/>
+          <mesh filename="package://kuka_cybertech_support/meshes/kr16_r2010_2/visual/link_4.stl"/>
         </geometry>
         <origin rpy="-0.0 0.0 -0.0" xyz="0.0 0.0 0.0"/>
@@ -108,5 +108,5 @@
       <collision>
         <geometry>
-          <mesh filename="package://kuka_cybertech_support/meshes/_sixxkr16_r2010_2/collision/link_5.stl"/>
+          <mesh filename="package://kuka_cybertech_support/meshes/kr16_r2010_2/collision/link_5.stl"/>
         </geometry>
         <origin rpy="-0.0 0.0 -0.0" xyz="0.0 0.0 0.0"/>
@@ -119,5 +119,5 @@
       <visual>
         <geometry>
-          <mesh filename="package://kuka_cybertech_support/meshes/_sixxkr16_r2010_2/visual/link_5.stl"/>
+          <mesh filename="package://kuka_cybertech_support/meshes/kr16_r2010_2/visual/link_5.stl"/>
         </geometry>
         <origin rpy="-0.0 0.0 -0.0" xyz="0.0 0.0 0.0"/>
@@ -127,5 +127,5 @@
       <collision>
         <geometry>
-          <mesh filename="package://kuka_cybertech_support/meshes/_sixxkr16_r2010_2/collision/link_6.stl"/>
+          <mesh filename="package://kuka_cybertech_support/meshes/kr16_r2010_2/collision/link_6.stl"/>
         </geometry>
         <origin rpy="-0.0 0.0 -0.0" xyz="0.0 0.0 0.0"/>
@@ -138,5 +138,5 @@
       <visual>
         <geometry>
-          <mesh filename="package://kuka_cybertech_support/meshes/_sixxkr16_r2010_2/visual/link_6.stl"/>
+          <mesh filename="package://kuka_cybertech_support/meshes/kr16_r2010_2/visual/link_6.stl"/>
         </geometry>
         <origin rpy="-0.0 0.0 -0.0" xyz="0.0 0.0 0.0"/>

Commit message: fix flange ros-in convention

File: kuka_cybertech_support/urdf/kr16_r2010_2_macro.xacro (robot description, xacro)
@@ -201,5 +201,5 @@
     <joint name="${prefix}link6-flange" type="fixed">
       <child link="${prefix}flange" />
-      <origin rpy="0 ${pi} -0.0" xyz="0.0 0.0 -0.153" />
+      <origin rpy="0 ${pi/2} -0.0" xyz="0.0 0.0 -0.153" />
       <parent link="${prefix}link_6" />
     </joint>

File: kuka_lbr_iisy_support/urdf/lbr_iisy11_r1300_macro.xacro (robot description, xacro)
@@ -213,5 +213,5 @@
     <joint name="${prefix}link6-flange" type="fixed">
       <child link="${prefix}flange" />
-      <origin rpy="0 ${pi} -0.0" xyz="0.0 0.0 -0.178" />
+      <origin rpy="0 ${pi/2} -0.0" xyz="0.0 0.0 -0.178" />
       <parent link="${prefix}link_6" />
     </joint>

File: kuka_lbr_iisy_support/urdf/lbr_iisy15_r930_macro.xacro (robot description, xacro)
@@ -213,5 +213,5 @@
     <joint name="${prefix}link6-flange" type="fixed">
       <child link="${prefix}flange" />
-      <origin rpy="0 ${pi} -0.0" xyz="0.0 0.0 -0.178" />
+      <origin rpy="0 ${pi/2} -0.0" xyz="0.0 0.0 -0.178" />
       <parent link="${prefix}link_6" />
     </joint>

File: kuka_lbr_iisy_support/urdf/lbr_iisy3_r760_macro.xacro (robot description, xacro)
@@ -213,5 +213,5 @@
     <joint name="${prefix}link6-flange" type="fixed">
       <child link="${prefix}flange" />
-      <origin rpy="0 ${pi} -0.0" xyz="0.0 0.0 -0.1605" />
+      <origin rpy="0 ${pi/2} -0.0" xyz="0.0 0.0 -0.1605" />
       <parent link="${prefix}link_6" />
     </joint>

File: kuka_quantec_support/urdf/kr210_r2700_2_macro.xacro (robot description, xacro)
@@ -201,5 +201,5 @@
     <joint name="${prefix}link6-flange" type="fixed">
       <child link="${prefix}flange" />
-      <origin rpy="0 ${pi} -0.0" xyz="0.0 0.0 -0.215" />
+      <origin rpy="0 ${pi/2} -0.0" xyz="0.0 0.0 -0.215" />
       <parent link="${prefix}link_6" />
     </joint>

File: kuka_quantec_support/urdf/kr210_r3100_2_macro.xacro (robot description, xacro)
@@ -201,5 +201,5 @@
     <joint name="${prefix}link6-flange" type="fixed">
       <child link="${prefix}flange" />
-      <origin rpy="0 ${pi} -0.0" xyz="0.0 0.0 -0.240" />
+      <origin rpy="0 ${pi/2} -0.0" xyz="0.0 0.0 -0.240" />
       <parent link="${prefix}link_6" />
     </joint>

Commit message: Add documentation for support packages (#38)
* readme skeleton

* rviz config cleanup

* add moveit config launch files in readme

* move rsi simulator to drivers

* update skeleton

* joint limits readme

* add xacro ros-in conventions to readme

* update readme

* add table about verified data

* central alignment

* fix special chars

* move rsi simulator to drivers

* joint_ai-> joint_i

* Update README.md

Co-authored-by: G.A. vd. Hoorn <g.a.vanderhoorn@tudelft.nl>

* Update README.md

Co-authored-by: G.A. vd. Hoorn <g.a.vanderhoorn@tudelft.nl>

* MoveIt,checkmark

* use ` for all names

* fix version

* change to gui version in test launch files

* update readme about test launch files

* remove starting spaces

* Update README.md

Co-authored-by: G.A. vd. Hoorn <g.a.vanderhoorn@tudelft.nl>

* `

* lint

* frame conventions

* fix

* fix2

* includes

* fix typo

* fix flange ros-in convention

---------

Co-authored-by: Aron Svastits <svastits1@gmail.com>
Co-authored-by: G.A. vd. Hoorn <g.a.vanderhoorn@tudelft.nl>

File: kuka_cybertech_support/urdf/kr16_r2010_2_macro.xacro (robot description, xacro)
@@ -148,5 +148,5 @@
       <origin xyz="0 0 0" rpy="0 0 0" />
     </joint>
-    <joint name="${prefix}joint_a1" type="revolute">
+    <joint name="${prefix}joint_1" type="revolute">
       <axis xyz="0.0 0.0 1.0"/>
       <child link="${prefix}link_1"/>
@@ -155,5 +155,5 @@
       <parent link="${prefix}base_link_inertia"/>
     </joint>
-    <joint name="${prefix}joint_a2" type="revolute">
+    <joint name="${prefix}joint_2" type="revolute">
       <axis xyz="0.0 0.0 1.0"/>
       <child link="${prefix}link_2"/>
@@ -162,5 +162,5 @@
       <parent link="${prefix}link_1"/>
     </joint>
-    <joint name="${prefix}joint_a3" type="revolute">
+    <joint name="${prefix}joint_3" type="revolute">
       <axis xyz="0.0 0.0 1.0"/>
       <child link="${prefix}link_3"/>
@@ -169,5 +169,5 @@
       <parent link="${prefix}link_2"/>
     </joint>
-    <joint name="${prefix}joint_a4" type="revolute">
+    <joint name="${prefix}joint_4" type="revolute">
       <axis xyz="0.0 0.0 1.0"/>
       <child link="${prefix}link_4"/>
@@ -176,5 +176,5 @@
       <parent link="${prefix}link_3"/>
     </joint>
-    <joint name="${prefix}joint_a5" type="revolute">
+    <joint name="${prefix}joint_5" type="revolute">
       <axis xyz="0.0 0.0 1.0"/>
       <child link="${prefix}link_5"/>
@@ -183,5 +183,5 @@
       <parent link="${prefix}link_4"/>
     </joint>
-    <joint name="${prefix}joint_a6" type="revolute">
+    <joint name="${prefix}joint_6" type="revolute">
       <axis xyz="0.0 0.0 1.0"/>
       <child link="${prefix}link_6"/>
@@ -201,5 +201,5 @@
     <joint name="${prefix}link6-flange" type="fixed">
       <child link="${prefix}flange" />
-      <origin rpy="0 ${pi} -0.0" xyz="0.0 0.0 -0.153" />
+      <origin rpy="0 ${pi/2} -0.0" xyz="0.0 0.0 -0.153" />
       <parent link="${prefix}link_6" />
     </joint>

File: kuka_lbr_iisy_support/urdf/lbr_iisy_ros2_control.xacro (robot description, xacro)
@@ -22,5 +22,5 @@
           <xacro:property name="lost_packets_in_timeframe" value="${qos_config_dict['rt_packet_loss_profile']['lost_packets_in_timeframe']}" />
           <xacro:property name="timeframe_ms" value="${qos_config_dict['rt_packet_loss_profile']['timeframe_ms']}" />
-          <plugin>kuka_rox::KukaRoXHardwareInterface</plugin>
+          <plugin>kuka_eac::KukaEACHardwareInterface</plugin>
           <param name="client_ip">${client_ip}</param>
           <param name="controller_ip">${controller_ip}</param>
@@ -32,5 +32,5 @@
       </hardware>
       <!-- define joints and command/state interfaces for each joint -->
-      <joint name="${prefix}joint_a1">
+      <joint name="${prefix}joint_1">
         <command_interface name="position"/>
         <command_interface name="stiffness"/>
@@ -40,5 +40,5 @@
         <state_interface name="effort"/>
       </joint>
-      <joint name="${prefix}joint_a2">
+      <joint name="${prefix}joint_2">
         <command_interface name="position"/>
         <command_interface name="stiffness"/>
@@ -48,5 +48,5 @@
         <state_interface name="effort"/>
       </joint>
-      <joint name="${prefix}joint_a3">
+      <joint name="${prefix}joint_3">
         <command_interface name="position"/>
         <command_interface name="stiffness"/>
@@ -56,5 +56,5 @@
         <state_interface name="effort"/>
       </joint>
-      <joint name="${prefix}joint_a4">
+      <joint name="${prefix}joint_4">
         <command_interface name="position"/>
         <command_interface name="stiffness"/>
@@ -64,5 +64,5 @@
         <state_interface name="effort"/>
       </joint>
-      <joint name="${prefix}joint_a5">
+      <joint name="${prefix}joint_5">
         <command_interface name="position"/>
         <command_interface name="stiffness"/>
@@ -72,5 +72,5 @@
         <state_interface name="effort"/>
       </joint>
-      <joint name="${prefix}joint_a6">
+      <joint name="${prefix}joint_6">
         <command_interface name="position"/>
         <command_interface name="stiffness"/>

File: kuka_lbr_iiwa_support/urdf/lbr_iiwa_ros2_control.xacro (robot description, xacro)
@@ -10,9 +10,9 @@
         </xacro:if>
         <xacro:unless value="${use_fake_hardware}">
-          <plugin>kuka_sunrise_fri_driver::KUKAFRIHardwareInterface</plugin>
+          <plugin>kuka_sunrise_fri_driver::KukaFRIHardwareInterface</plugin>
         </xacro:unless>
       </hardware>
       <!-- define joints and command/state interfaces for each joint -->
-      <joint name="${prefix}joint_a1">
+      <joint name="${prefix}joint_1">
         <command_interface name="position"/>
         <command_interface name="effort"/>
@@ -21,5 +21,5 @@
         <state_interface name="external_torque"/>
       </joint>
-      <joint name="${prefix}joint_a2">
+      <joint name="${prefix}joint_2">
         <command_interface name="position"/>
         <command_interface name="effort"/>
@@ -28,5 +28,5 @@
         <state_interface name="external_torque"/>
       </joint>
-      <joint name="${prefix}joint_a3">
+      <joint name="${prefix}joint_3">
         <command_interface name="position"/>
         <command_interface name="effort"/>
@@ -35,5 +35,5 @@
         <state_interface name="external_torque"/>
       </joint>
-      <joint name="${prefix}joint_a4">
+      <joint name="${prefix}joint_4">
         <command_interface name="position"/>
         <command_interface name="effort"/>
@@ -42,5 +42,5 @@
         <state_interface name="external_torque"/>
       </joint>
-      <joint name="${prefix}joint_a5">
+      <joint name="${prefix}joint_5">
         <command_interface name="position"/>
         <command_interface name="effort"/>
@@ -49,5 +49,5 @@
         <state_interface name="external_torque"/>
       </joint>
-      <joint name="${prefix}joint_a6">
+      <joint name="${prefix}joint_6">
         <command_interface name="position"/>
         <command_interface name="effort"/>
@@ -56,5 +56,5 @@
         <state_interface name="external_torque"/>
       </joint>
-      <joint name="${prefix}joint_a7">
+      <joint name="${prefix}joint_7">
         <command_interface name="position"/>
         <command_interface name="effort"/>

Commit message: try out coll box

File: kuka_cybertech_support/urdf/kr16_r2010_2_macro.xacro (robot description, xacro)
@@ -10,7 +10,7 @@
       <collision>
         <geometry>
-          <mesh filename="package://kuka_cybertech_support/meshes/kr16_r2010_2/collision/base_link.stl"/>
-        </geometry>
-        <origin rpy="-0.0 0.0 -0.0" xyz="0.0 0.0 0.0"/>
+          <box size="0.6545662432909012 0.37630656361579895 0.28446903824806224"/>
+        </geometry>
+        <origin rpy="0.0 0.0 0.0" xyz="-0.1380831003189087 0.0 0.14223451912403107"/>
       </collision>
       <inertial>
@@ -29,7 +29,7 @@
       <collision>
         <geometry>
-          <mesh filename="package://kuka_cybertech_support/meshes/kr16_r2010_2/collision/link_1.stl"/>
-        </geometry>
-        <origin rpy="-0.0 0.0 -0.0" xyz="0.0 0.0 0.0"/>
+          <box size="0.4838663190603256 0.5623050630092621 0.4337000250816345"/>
+        </geometry>
+        <origin rpy="0.0 0.0 0.0" xyz="0.0559331551194191 -0.0335475318133831 -0.47484999895095825"/>
       </collision>
       <inertial>
@@ -48,7 +48,7 @@
       <collision>
         <geometry>
-          <mesh filename="package://kuka_cybertech_support/meshes/kr16_r2010_2/collision/link_2.stl"/>
-        </geometry>
-        <origin rpy="-0.0 0.0 -0.0" xyz="0.0 0.0 0.0"/>
+           <box size="1.2043238580226898 0.2157236412167549 0.18066882342100143" />
+        </geometry>
+        <origin rpy="-0.0 0.0 -0.0" xyz="0.4583 -0.0005 -0.1718"/>
       </collision>
       <inertial>
@@ -67,7 +67,7 @@
       <collision>
         <geometry>
-          <mesh filename="package://kuka_cybertech_support/meshes/kr16_r2010_2/collision/link_3.stl"/>
-        </geometry>
-        <origin rpy="-0.0 0.0 -0.0" xyz="0.0 0.0 0.0"/>
+          <box size="0.3508647680282593 0.5482000410556793 0.509911298751831"/>
+        </geometry>
+        <origin rpy="0.0 0.0 0.0" xyz="0.04656773805618286 0.03590010106563568 -0.021755695343017578"/>
       </collision>
       <inertial>
@@ -86,7 +86,7 @@
       <collision>
         <geometry>
-          <mesh filename="package://kuka_cybertech_support/meshes/kr16_r2010_2/collision/link_4.stl"/>
-        </geometry>
-        <origin rpy="-0.0 0.0 -0.0" xyz="0.0 0.0 0.0"/>
+          <box size="0.1380000114440918 0.16130001097917557 0.6190000772476196"/>
+        </geometry>
+        <origin rpy="0.0 0.0 0.0" xyz="1.1920928955078125e-07 0.011649999767541885 -0.6095001101493835"/>
       </collision>
       <inertial>
@@ -105,7 +105,7 @@
       <collision>
         <geometry>
-          <mesh filename="package://kuka_cybertech_support/meshes/kr16_r2010_2/collision/link_5.stl"/>
-        </geometry>
-        <origin rpy="-0.0 0.0 -0.0" xyz="0.0 0.0 0.0"/>
+          <box size="0.11500000953674316 0.20200002193450928 0.2007358893752098"/>
+        </geometry>
+        <origin rpy="0.0 0.0 0.0" xyz="1.1920928955078125e-07 0.04350012540817261 0.007631983608007431"/>
       </collision>
       <inertial>
@@ -124,7 +124,7 @@
       <collision>
         <geometry>
-          <mesh filename="package://kuka_cybertech_support/meshes/kr16_r2010_2/collision/link_6.stl"/>
-        </geometry>
-        <origin rpy="-0.0 0.0 -0.0" xyz="0.0 0.0 0.0"/>
+          <box size="0.06693124771118164 0.06696557998657227 0.0140000581741333"/>
+        </geometry>
+        <origin rpy="0.0 0.0 0.0" xyz="-3.4332275390625e-05 0.0 -0.1460002064704895"/>
       </collision>
       <inertial>
