Commit message: add gazebo hw tags to cybertech and iiwa models

File: kuka_cybertech_support/urdf/kr_cybertech_ros2_control_macro.xacro (robot description, xacro)
@@ -2,4 +2,9 @@
 <robot xmlns:xacro="http://www.ros.org/wiki/xacro">
   <xacro:macro name="kuka_cybertech_ros2_control" params="name client_ip client_port controller_ip prefix mode roundtrip_time">
+    <!-- gazebo -->
+    <xacro:if value="${mode == 'gazebo'}">
+      <xacro:include filename="$(find kuka_gazebo)/gazebo/kuka_gazebo.xacro"/>
+      <xacro:kuka_gazebo controller_config_package="kuka_resources" controller_config_path="config/fake_hardware_config_6_axis.yaml"/>
+    </xacro:if>
     <!-- ros2 control -->
     <ros2_control name="${name}" type="system">
@@ -17,4 +22,7 @@
           <param name="client_port">${client_port}</param>
           <param name="controller_ip">${controller_ip}</param>
+        </xacro:if>
+        <xacro:if value="${mode == 'gazebo'}">
+          <plugin>gz_ros2_control/GazeboSimSystem</plugin>
         </xacro:if>
       </hardware>

File: kuka_lbr_iiwa_support/urdf/lbr_iiwa14_r820_macro.xacro (robot description, xacro)
@@ -9,5 +9,5 @@
       <visual>
         <geometry>
-          <mesh filename="package://kuka_lbr_iiwa_support/meshes/lbr_iiwa14_r820/visual/base_link.stl"/>
+          <mesh filename="package://${package_name}/meshes/lbr_iiwa14_r820/visual/base_link.stl"/>
         </geometry>
         <origin rpy="-0.0 0.0 0.0" xyz="0.0 0.0 0.0"/>
@@ -16,5 +16,5 @@
         <origin rpy="-0.0 0.0 0.0" xyz="0.0 0.0 0.0"/>
         <geometry>
-          <mesh filename="package://kuka_lbr_iiwa_support/meshes/lbr_iiwa14_r820/collision/base_link.stl"/>
+          <mesh filename="package://${package_name}/meshes/lbr_iiwa14_r820/collision/base_link.stl"/>
         </geometry>
       </collision>
@@ -23,5 +23,5 @@
       <visual>
         <geometry>
-          <mesh filename="package://kuka_lbr_iiwa_support/meshes/lbr_iiwa14_r820/visual/link_1.stl"/>
+          <mesh filename="package://${package_name}/meshes/lbr_iiwa14_r820/visual/link_1.stl"/>
         </geometry>
         <origin rpy="-0.0 0.0 0.0" xyz="0.0 0.0 0.0"/>
@@ -30,5 +30,5 @@
         <origin rpy="-0.0 0.0 0.0" xyz="0.0 0.0 0.0"/>
         <geometry>
-          <mesh filename="package://kuka_lbr_iiwa_support/meshes/lbr_iiwa14_r820/collision/link_1.stl"/>
+          <mesh filename="package://${package_name}/meshes/lbr_iiwa14_r820/collision/link_1.stl"/>
         </geometry>
       </collision>
@@ -37,5 +37,5 @@
       <visual>
         <geometry>
-          <mesh filename="package://kuka_lbr_iiwa_support/meshes/lbr_iiwa14_r820/visual/link_2.stl"/>
+          <mesh filename="package://${package_name}/meshes/lbr_iiwa14_r820/visual/link_2.stl"/>
         </geometry>
         <origin rpy="-0.0 0.0 0.0" xyz="0.0 0.0 0.0"/>
@@ -44,5 +44,5 @@
         <origin rpy="-0.0 0.0 0.0" xyz="0.0 0.0 0.0"/>
         <geometry>
-          <mesh filename="package://kuka_lbr_iiwa_support/meshes/lbr_iiwa14_r820/collision/link_2.stl"/>
+          <mesh filename="package://${package_name}/meshes/lbr_iiwa14_r820/collision/link_2.stl"/>
         </geometry>
       </collision>
@@ -51,5 +51,5 @@
       <visual>
         <geometry>
-          <mesh filename="package://kuka_lbr_iiwa_support/meshes/lbr_iiwa14_r820/visual/link_3.stl"/>
+          <mesh filename="package://${package_name}/meshes/lbr_iiwa14_r820/visual/link_3.stl"/>
         </geometry>
         <origin rpy="-0.0 0.0 0.0" xyz="0.0 0.0 0.0"/>
@@ -58,5 +58,5 @@
         <origin rpy="-0.0 0.0 0.0" xyz="0.0 0.0 0.0"/>
         <geometry>
-          <mesh filename="package://kuka_lbr_iiwa_support/meshes/lbr_iiwa14_r820/collision/link_3.stl"/>
+          <mesh filename="package://${package_name}/meshes/lbr_iiwa14_r820/collision/link_3.stl"/>
         </geometry>
       </collision>
@@ -65,5 +65,5 @@
       <visual>
         <geometry>
-          <mesh filename="package://kuka_lbr_iiwa_support/meshes/lbr_iiwa14_r820/visual/link_4.stl"/>
+          <mesh filename="package://${package_name}/meshes/lbr_iiwa14_r820/visual/link_4.stl"/>
         </geometry>
         <origin rpy="-0.0 0.0 0.0" xyz="0.0 0.0 0.0"/>
@@ -72,5 +72,5 @@
         <origin rpy="-0.0 0.0 0.0" xyz="0.0 0.0 0.0"/>
         <geometry>
-          <mesh filename="package://kuka_lbr_iiwa_support/meshes/lbr_iiwa14_r820/collision/link_4.stl"/>
+          <mesh filename="package://${package_name}/meshes/lbr_iiwa14_r820/collision/link_4.stl"/>
         </geometry>
       </collision>
@@ -79,5 +79,5 @@
       <visual>
         <geometry>
-          <mesh filename="package://kuka_lbr_iiwa_support/meshes/lbr_iiwa14_r820/visual/link_5.stl"/>
+          <mesh filename="package://${package_name}/meshes/lbr_iiwa14_r820/visual/link_5.stl"/>
         </geometry>
         <origin rpy="-0.0 0.0 0.0" xyz="0.0 0.0 0.0"/>
@@ -86,5 +86,5 @@
         <origin rpy="-0.0 0.0 0.0" xyz="0.0 0.0 0.0"/>
         <geometry>
-          <mesh filename="package://kuka_lbr_iiwa_support/meshes/lbr_iiwa14_r820/collision/link_5.stl"/>
+          <mesh filename="package://${package_name}/meshes/lbr_iiwa14_r820/collision/link_5.stl"/>
         </geometry>
       </collision>
@@ -93,5 +93,5 @@
       <visual>
         <geometry>
-          <mesh filename="package://kuka_lbr_iiwa_support/meshes/lbr_iiwa14_r820/visual/link_6.stl"/>
+          <mesh filename="package://${package_name}/meshes/lbr_iiwa14_r820/visual/link_6.stl"/>
         </geometry>
         <origin rpy="-0.0 0.0 0.0" xyz="0.0 0.0 0.0"/>
@@ -100,5 +100,5 @@
         <origin rpy="-0.0 0.0 0.0" xyz="0.0 0.0 0.0"/>
         <geometry>
-          <mesh filename="package://kuka_lbr_iiwa_support/meshes/lbr_iiwa14_r820/collision/link_6.stl"/>
+          <mesh filename="package://${package_name}/meshes/lbr_iiwa14_r820/collision/link_6.stl"/>
         </geometry>
       </collision>
@@ -107,5 +107,5 @@
       <visual>
         <geometry>
-          <mesh filename="package://kuka_lbr_iiwa_support/meshes/lbr_iiwa14_r820/visual/link_7.stl"/>
+          <mesh filename="package://${package_name}/meshes/lbr_iiwa14_r820/visual/link_7.stl"/>
         </geometry>
         <origin rpy="-0.0 0.0 0.0" xyz="0.0 0.0 0.0"/>
@@ -114,5 +114,5 @@
         <origin rpy="-0.0 0.0 0.0" xyz="0.0 0.0 0.0"/>
         <geometry>
-          <mesh filename="package://kuka_lbr_iiwa_support/meshes/lbr_iiwa14_r820/collision/link_7.stl"/>
+          <mesh filename="package://${package_name}/meshes/lbr_iiwa14_r820/collision/link_7.stl"/>
         </geometry>
       </collision>

File: kuka_lbr_iiwa_support/urdf/lbr_iiwa_ros2_control_macro.xacro (robot description, xacro)
@@ -2,4 +2,9 @@
 <robot xmlns:xacro="http://www.ros.org/wiki/xacro">
   <xacro:macro name="kuka_lbr_iiwa_ros2_control" params="name prefix io_access mode roundtrip_time controller_ip client_ip client_port">
+    <!-- gazebo -->
+    <xacro:if value="${mode == 'gazebo'}">
+      <xacro:include filename="$(find kuka_gazebo)/gazebo/kuka_gazebo.xacro"/>
+      <xacro:kuka_gazebo controller_config_package="kuka_resources" controller_config_path="config/fake_hardware_config_7_axis.yaml"/>
+    </xacro:if>
     <!-- ros2 control -->
     <ros2_control name="${name}" type="system">
@@ -18,11 +23,16 @@
           <param name="client_port">${client_port}</param>
         </xacro:if>
+        <xacro:if value="${mode == 'gazebo'}">
+          <plugin>gz_ros2_control/GazeboSimSystem</plugin>
+        </xacro:if>
       </hardware>
       <!-- define joints and command/state interfaces for each joint -->
       <joint name="${prefix}joint_1">
         <command_interface name="position"/>
-        <command_interface name="stiffness"/>
-        <command_interface name="damping"/>
-        <command_interface name="effort"/>
+        <xacro:unless value="${mode == 'gazebo'}">
+          <command_interface name="stiffness"/>
+          <command_interface name="damping"/>
+          <command_interface name="effort"/>
+        </xacro:unless>
         <state_interface name="position">
           <param name="initial_value">0.0</param>
@@ -37,7 +47,9 @@
       <joint name="${prefix}joint_2">
         <command_interface name="position"/>
-        <command_interface name="stiffness"/>
-        <command_interface name="damping"/>
-        <command_interface name="effort"/>
+        <xacro:unless value="${mode == 'gazebo'}">
+          <command_interface name="stiffness"/>
+          <command_interface name="damping"/>
+          <command_interface name="effort"/>
+        </xacro:unless>
         <state_interface name="position">
           <param name="initial_value">0.0</param>
@@ -52,7 +64,9 @@
       <joint name="${prefix}joint_3">
         <command_interface name="position"/>
-        <command_interface name="stiffness"/>
-        <command_interface name="damping"/>
-        <command_interface name="effort"/>
+        <xacro:unless value="${mode == 'gazebo'}">
+          <command_interface name="stiffness"/>
+          <command_interface name="damping"/>
+          <command_interface name="effort"/>
+        </xacro:unless>
         <state_interface name="position">
           <param name="initial_value">0.0</param>
@@ -67,7 +81,9 @@
       <joint name="${prefix}joint_4">
         <command_interface name="position"/>
-        <command_interface name="stiffness"/>
-        <command_interface name="damping"/>
-        <command_interface name="effort"/>
+        <xacro:unless value="${mode == 'gazebo'}">
+          <command_interface name="stiffness"/>
+          <command_interface name="damping"/>
+          <command_interface name="effort"/>
+        </xacro:unless>
         <state_interface name="position">
           <param name="initial_value">0.0</param>
@@ -82,7 +98,9 @@
       <joint name="${prefix}joint_5">
         <command_interface name="position"/>
-        <command_interface name="stiffness"/>
-        <command_interface name="damping"/>
-        <command_interface name="effort"/>
+        <xacro:unless value="${mode == 'gazebo'}">
+          <command_interface name="stiffness"/>
+          <command_interface name="damping"/>
+          <command_interface name="effort"/>
+        </xacro:unless>
         <state_interface name="position">
           <param name="initial_value">0.0</param>
@@ -97,7 +115,9 @@
       <joint name="${prefix}joint_6">
         <command_interface name="position"/>
-        <command_interface name="stiffness"/>
-        <command_interface name="damping"/>
-        <command_interface name="effort"/>
+        <xacro:unless value="${mode == 'gazebo'}">
+          <command_interface name="stiffness"/>
+          <command_interface name="damping"/>
+          <command_interface name="effort"/>
+        </xacro:unless>
         <state_interface name="position">
           <param name="initial_value">0.0</param>
@@ -112,7 +132,9 @@
       <joint name="${prefix}joint_7">
         <command_interface name="position"/>
-        <command_interface name="stiffness"/>
-        <command_interface name="damping"/>
-        <command_interface name="effort"/>
+        <xacro:unless value="${mode == 'gazebo'}">
+          <command_interface name="stiffness"/>
+          <command_interface name="damping"/>
+          <command_interface name="effort"/>
+        </xacro:unless>
         <state_interface name="position">
           <param name="initial_value">0.0</param>
