Commit message: Fix pre-commit

File: kuka_cybertech_support/urdf/kr20_r1810_2.urdf.xacro (robot description, xacro)
@@ -2,30 +2,25 @@
 <robot xmlns:xacro="http://ros.org/wiki/xacro" name="kr20_r1810_2">
   <!-- Import macro files  -->
-  <xacro:include filename="$(find kuka_cybertech_support)/urdf/kr20_r1810_2_macro.xacro" />
-  <xacro:include
-    filename="$(find kuka_cybertech_support)/urdf/kr_cybertech_ros2_control_macro.xacro" />
+  <xacro:include filename="$(find kuka_cybertech_support)/urdf/kr20_r1810_2_macro.xacro"/>
+  <xacro:include filename="$(find kuka_cybertech_support)/urdf/kr_cybertech_ros2_control_macro.xacro"/>
   <!-- Read additional arguments  -->
-  <xacro:arg name="driver_version" default="eki_rsi" />
-  <xacro:arg name="mode" default="hardware" />
-  <xacro:arg name="use_gpio" default="false" />
-  <xacro:arg name="roundtrip_time" default="0" />
-  <xacro:arg name="client_ip" default="0.0.0.0" />
-  <xacro:arg name="client_port" default="59152" />
-  <xacro:arg name="controller_ip" default="0.0.0.0" />
-  <xacro:arg name="verify_robot_model" default="true" />
-  <xacro:arg name="prefix" default="" />
-  <xacro:arg name="x" default="0" />
-  <xacro:arg name="y" default="0" />
-  <xacro:arg name="z" default="0" />
-  <xacro:arg name="roll" default="0" />
-  <xacro:arg name="pitch" default="0" />
-  <xacro:arg name="yaw" default="0" />
-  <xacro:kuka_cybertech_ros2_control name="$(arg prefix)kr20_r1810_2"
-    driver_version="$(arg driver_version)" client_ip="$(arg client_ip)"
-    client_port="$(arg client_port)" controller_ip="$(arg controller_ip)" prefix="$(arg prefix)"
-    mode="$(arg mode)" use_gpio="$(arg use_gpio)" roundtrip_time="$(arg roundtrip_time)"
-    verify_robot_model="$(arg verify_robot_model)" />
+  <xacro:arg name="driver_version" default="eki_rsi"/>
+  <xacro:arg name="mode" default="hardware"/>
+  <xacro:arg name="use_gpio" default="false"/>
+  <xacro:arg name="roundtrip_time" default="0"/>
+  <xacro:arg name="client_ip" default="0.0.0.0"/>
+  <xacro:arg name="client_port" default="59152"/>
+  <xacro:arg name="controller_ip" default="0.0.0.0"/>
+  <xacro:arg name="verify_robot_model" default="true"/>
+  <xacro:arg name="prefix" default=""/>
+  <xacro:arg name="x" default="0"/>
+  <xacro:arg name="y" default="0"/>
+  <xacro:arg name="z" default="0"/>
+  <xacro:arg name="roll" default="0"/>
+  <xacro:arg name="pitch" default="0"/>
+  <xacro:arg name="yaw" default="0"/>
+  <xacro:kuka_cybertech_ros2_control name="$(arg prefix)kr20_r1810_2" driver_version="$(arg driver_version)" client_ip="$(arg client_ip)" client_port="$(arg client_port)" controller_ip="$(arg controller_ip)" prefix="$(arg prefix)" mode="$(arg mode)" use_gpio="$(arg use_gpio)" roundtrip_time="$(arg roundtrip_time)" verify_robot_model="$(arg verify_robot_model)"/>
   <xacro:kuka_kr20_r1810_2_robot prefix="$(arg prefix)" package_name="kuka_cybertech_support">
-    <origin xyz="$(arg x) $(arg y) $(arg z)" rpy="$(arg roll) $(arg pitch) $(arg yaw)" />
+    <origin xyz="$(arg x) $(arg y) $(arg z)" rpy="$(arg roll) $(arg pitch) $(arg yaw)"/>
   </xacro:kuka_kr20_r1810_2_robot>
 </robot>

File: kuka_cybertech_support/urdf/kr20_r1810_2_macro.xacro (robot description, xacro)
@@ -1,3 +1,3 @@
-<?xml version='1.0' encoding='UTF-8'?>
+<?xml version="1.0" encoding="UTF-8"?>
 <robot xmlns:xacro="http://www.ros.org/wiki/xacro" name="kr20_r1810_2">
   <xacro:macro name="kuka_kr20_r1810_2_robot" params="prefix package_name *origin">
