Commit message: Change robot description to new convention

File: kuka_cybertech_support/urdf/kr12_r1450_3_hw.urdf.xacro (robot description, xacro)
@@ -20,7 +20,16 @@
   <xacro:arg name="pitch" default="0"/>
   <xacro:arg name="yaw" default="0"/>
-  <xacro:kuka_cybertech_ros2_control name="$(arg prefix)kr12_r1450_3_hw" driver_version="$(arg driver_version)" client_ip="$(arg client_ip)" client_port="$(arg client_port)" controller_ip="$(arg controller_ip)" prefix="$(arg prefix)" mode="$(arg mode)" use_gpio="$(arg use_gpio)" roundtrip_time="$(arg roundtrip_time)" verify_robot_model="$(arg verify_robot_model)"/>
-  <xacro:kuka_kr12_r1450_3_hw_robot prefix="$(arg prefix)" package_name="kuka_cybertech_support">
+  <xacro:kuka_cybertech_ros2_control name="$(arg prefix)kr12_r1450_3_hw" driver_version="$(arg driver_version)" client_ip="$(arg client_ip)" client_port="$(arg client_port)" controller_ip="$(arg controller_ip)" prefix="$(arg prefix)" mode="$(arg mode)" use_gpio="$(arg use_gpio)" roundtrip_time="$(arg roundtrip_time)" verify_robot_model="$(arg verify_robot_model)">
+    <ext_axis_ros2_control_joints/>
+  </xacro:kuka_cybertech_ros2_control>
+  <!-- world link -->
+  <link name="world"/>
+  <!-- robot links, joints -->
+  <xacro:kuka_kr12_r1450_3_hw_robot prefix="$(arg prefix)" package_name="kuka_cybertech_support"/>
+  <!-- default world - base_link joint -->
+  <joint name="$(arg prefix)world-base_link" type="fixed">
+    <parent link="world"/>
+    <child link="$(arg prefix)base_link"/>
     <origin xyz="$(arg x) $(arg y) $(arg z)" rpy="$(arg roll) $(arg pitch) $(arg yaw)"/>
-  </xacro:kuka_kr12_r1450_3_hw_robot>
+  </joint>
 </robot>

File: kuka_cybertech_support/urdf/kr20_r1810_2.urdf.xacro (robot description, xacro)
@@ -20,7 +20,16 @@
   <xacro:arg name="pitch" default="0"/>
   <xacro:arg name="yaw" default="0"/>
-  <xacro:kuka_cybertech_ros2_control name="$(arg prefix)kr20_r1810_2" driver_version="$(arg driver_version)" client_ip="$(arg client_ip)" client_port="$(arg client_port)" controller_ip="$(arg controller_ip)" prefix="$(arg prefix)" mode="$(arg mode)" use_gpio="$(arg use_gpio)" roundtrip_time="$(arg roundtrip_time)" verify_robot_model="$(arg verify_robot_model)"/>
-  <xacro:kuka_kr20_r1810_2_robot prefix="$(arg prefix)" package_name="kuka_cybertech_support">
+  <xacro:kuka_cybertech_ros2_control name="$(arg prefix)kr20_r1810_2" driver_version="$(arg driver_version)" client_ip="$(arg client_ip)" client_port="$(arg client_port)" controller_ip="$(arg controller_ip)" prefix="$(arg prefix)" mode="$(arg mode)" use_gpio="$(arg use_gpio)" roundtrip_time="$(arg roundtrip_time)" verify_robot_model="$(arg verify_robot_model)">
+    <ext_axis_ros2_control_joints/>
+  </xacro:kuka_cybertech_ros2_control>
+  <!-- world link -->
+  <link name="world"/>
+  <!-- robot links, joints -->
+  <xacro:kuka_kr20_r1810_2_robot prefix="$(arg prefix)" package_name="kuka_cybertech_support"/>
+  <!-- default world - base_link joint -->
+  <joint name="$(arg prefix)world-base_link" type="fixed">
+    <parent link="world"/>
+    <child link="$(arg prefix)base_link"/>
     <origin xyz="$(arg x) $(arg y) $(arg z)" rpy="$(arg roll) $(arg pitch) $(arg yaw)"/>
-  </xacro:kuka_kr20_r1810_2_robot>
+  </joint>
 </robot>

File: kuka_cybertech_support/urdf/kr8_r1440_2_arc_hw.urdf.xacro (robot description, xacro)
@@ -20,7 +20,16 @@
   <xacro:arg name="pitch" default="0"/>
   <xacro:arg name="yaw" default="0"/>
-  <xacro:kuka_cybertech_ros2_control name="$(arg prefix)kr8_r1440_2_arc_hw" driver_version="$(arg driver_version)" client_ip="$(arg client_ip)" client_port="$(arg client_port)" controller_ip="$(arg controller_ip)" prefix="$(arg prefix)" mode="$(arg mode)" use_gpio="$(arg use_gpio)" roundtrip_time="$(arg roundtrip_time)" verify_robot_model="$(arg verify_robot_model)"/>
-  <xacro:kuka_kr8_r1440_2_arc_hw_robot prefix="$(arg prefix)" package_name="kuka_cybertech_support">
+  <xacro:kuka_cybertech_ros2_control name="$(arg prefix)kr8_r1440_2_arc_hw" driver_version="$(arg driver_version)" client_ip="$(arg client_ip)" client_port="$(arg client_port)" controller_ip="$(arg controller_ip)" prefix="$(arg prefix)" mode="$(arg mode)" use_gpio="$(arg use_gpio)" roundtrip_time="$(arg roundtrip_time)" verify_robot_model="$(arg verify_robot_model)">
+    <ext_axis_ros2_control_joints/>
+  </xacro:kuka_cybertech_ros2_control>
+  <!-- world link -->
+  <link name="world"/>
+  <!-- robot links, joints -->
+  <xacro:kuka_kr8_r1440_2_arc_hw_robot prefix="$(arg prefix)" package_name="kuka_cybertech_support"/>
+  <!-- default world - base_link joint -->
+  <joint name="$(arg prefix)world-base_link" type="fixed">
+    <parent link="world"/>
+    <child link="$(arg prefix)base_link"/>
     <origin xyz="$(arg x) $(arg y) $(arg z)" rpy="$(arg roll) $(arg pitch) $(arg yaw)"/>
-  </xacro:kuka_kr8_r1440_2_arc_hw_robot>
+  </joint>
 </robot>

File: kuka_cybertech_support/urdf/kr8_r2100_2_arc_hw.urdf.xacro (robot description, xacro)
@@ -20,7 +20,16 @@
   <xacro:arg name="pitch" default="0"/>
   <xacro:arg name="yaw" default="0"/>
-  <xacro:kuka_cybertech_ros2_control name="$(arg prefix)kr8_r2100_2_arc_hw" driver_version="$(arg driver_version)" client_ip="$(arg client_ip)" client_port="$(arg client_port)" controller_ip="$(arg controller_ip)" prefix="$(arg prefix)" mode="$(arg mode)" use_gpio="$(arg use_gpio)" roundtrip_time="$(arg roundtrip_time)" verify_robot_model="$(arg verify_robot_model)"/>
-  <xacro:kuka_kr8_r2100_2_arc_hw_robot prefix="$(arg prefix)" package_name="kuka_cybertech_support">
+  <xacro:kuka_cybertech_ros2_control name="$(arg prefix)kr8_r2100_2_arc_hw" driver_version="$(arg driver_version)" client_ip="$(arg client_ip)" client_port="$(arg client_port)" controller_ip="$(arg controller_ip)" prefix="$(arg prefix)" mode="$(arg mode)" use_gpio="$(arg use_gpio)" roundtrip_time="$(arg roundtrip_time)" verify_robot_model="$(arg verify_robot_model)">
+    <ext_axis_ros2_control_joints/>
+  </xacro:kuka_cybertech_ros2_control>
+  <!-- world link -->
+  <link name="world"/>
+  <!-- robot links, joints -->
+  <xacro:kuka_kr8_r2100_2_arc_hw_robot prefix="$(arg prefix)" package_name="kuka_cybertech_support"/>
+  <!-- default world - base_link joint -->
+  <joint name="$(arg prefix)world-base_link" type="fixed">
+    <parent link="world"/>
+    <child link="$(arg prefix)base_link"/>
     <origin xyz="$(arg x) $(arg y) $(arg z)" rpy="$(arg roll) $(arg pitch) $(arg yaw)"/>
-  </xacro:kuka_kr8_r2100_2_arc_hw_robot>
+  </joint>
 </robot>

File: kuka_fortec_support/urdf/kr240_r3330.urdf.xacro (robot description, xacro)
@@ -20,7 +20,16 @@
   <xacro:arg name="pitch" default="0"/>
   <xacro:arg name="yaw" default="0"/>
-  <xacro:kuka_fortec_ros2_control name="$(arg prefix)kr240_r3330" driver_version="$(arg driver_version)" client_ip="$(arg client_ip)" client_port="$(arg client_port)" controller_ip="$(arg controller_ip)" prefix="$(arg prefix)" mode="$(arg mode)" use_gpio="$(arg use_gpio)" roundtrip_time="$(arg roundtrip_time)" verify_robot_model="$(arg verify_robot_model)"/>
-  <xacro:kuka_kr240_r3330_robot prefix="$(arg prefix)" package_name="kuka_fortec_support">
+  <xacro:kuka_fortec_ros2_control name="$(arg prefix)kr240_r3330" driver_version="$(arg driver_version)" client_ip="$(arg client_ip)" client_port="$(arg client_port)" controller_ip="$(arg controller_ip)" prefix="$(arg prefix)" mode="$(arg mode)" use_gpio="$(arg use_gpio)" roundtrip_time="$(arg roundtrip_time)" verify_robot_model="$(arg verify_robot_model)">
+    <ext_axis_ros2_control_joints/>
+  </xacro:kuka_fortec_ros2_control>
+  <!-- world link -->
+  <link name="world"/>
+  <!-- robot links, joints -->
+  <xacro:kuka_kr240_r3330_robot prefix="$(arg prefix)" package_name="kuka_fortec_support"/>
+  <!-- default world - base_link joint -->
+  <joint name="$(arg prefix)world-base_link" type="fixed">
+    <parent link="world"/>
+    <child link="$(arg prefix)base_link"/>
     <origin xyz="$(arg x) $(arg y) $(arg z)" rpy="$(arg roll) $(arg pitch) $(arg yaw)"/>
-  </xacro:kuka_kr240_r3330_robot>
+  </joint>
 </robot>

File: kuka_fortec_support/urdf/kr300_r2800_2_mt.urdf.xacro (robot description, xacro)
@@ -20,7 +20,16 @@
   <xacro:arg name="pitch" default="0"/>
   <xacro:arg name="yaw" default="0"/>
-  <xacro:kuka_fortec_ros2_control name="$(arg prefix)kr300_r2800_2_mt" driver_version="$(arg driver_version)" client_ip="$(arg client_ip)" client_port="$(arg client_port)" controller_ip="$(arg controller_ip)" prefix="$(arg prefix)" mode="$(arg mode)" use_gpio="$(arg use_gpio)" roundtrip_time="$(arg roundtrip_time)" verify_robot_model="$(arg verify_robot_model)"/>
-  <xacro:kuka_kr300_r2800_2_mt_robot prefix="$(arg prefix)" package_name="kuka_fortec_support">
+  <xacro:kuka_fortec_ros2_control name="$(arg prefix)kr300_r2800_2_mt" driver_version="$(arg driver_version)" client_ip="$(arg client_ip)" client_port="$(arg client_port)" controller_ip="$(arg controller_ip)" prefix="$(arg prefix)" mode="$(arg mode)" use_gpio="$(arg use_gpio)" roundtrip_time="$(arg roundtrip_time)" verify_robot_model="$(arg verify_robot_model)">
+    <ext_axis_ros2_control_joints/>
+  </xacro:kuka_fortec_ros2_control>
+  <!-- world link -->
+  <link name="world"/>
+  <!-- robot links, joints -->
+  <xacro:kuka_kr300_r2800_2_mt_robot prefix="$(arg prefix)" package_name="kuka_fortec_support"/>
+  <!-- default world - base_link joint -->
+  <joint name="$(arg prefix)world-base_link" type="fixed">
+    <parent link="world"/>
+    <child link="$(arg prefix)base_link"/>
     <origin xyz="$(arg x) $(arg y) $(arg z)" rpy="$(arg roll) $(arg pitch) $(arg yaw)"/>
-  </xacro:kuka_kr300_r2800_2_mt_robot>
+  </joint>
 </robot>

File: kuka_fortec_support/urdf/kr560_r3100_2.urdf.xacro (robot description, xacro)
@@ -20,7 +20,16 @@
   <xacro:arg name="pitch" default="0"/>
   <xacro:arg name="yaw" default="0"/>
-  <xacro:kuka_fortec_ros2_control name="$(arg prefix)kr560_r3100_2" driver_version="$(arg driver_version)" client_ip="$(arg client_ip)" client_port="$(arg client_port)" controller_ip="$(arg controller_ip)" prefix="$(arg prefix)" mode="$(arg mode)" use_gpio="$(arg use_gpio)" roundtrip_time="$(arg roundtrip_time)" verify_robot_model="$(arg verify_robot_model)"/>
-  <xacro:kuka_kr560_r3100_2_robot prefix="$(arg prefix)" package_name="kuka_fortec_support">
+  <xacro:kuka_fortec_ros2_control name="$(arg prefix)kr560_r3100_2" driver_version="$(arg driver_version)" client_ip="$(arg client_ip)" client_port="$(arg client_port)" controller_ip="$(arg controller_ip)" prefix="$(arg prefix)" mode="$(arg mode)" use_gpio="$(arg use_gpio)" roundtrip_time="$(arg roundtrip_time)" verify_robot_model="$(arg verify_robot_model)">
+    <ext_axes_ros2_control_joints/>
+  </xacro:kuka_fortec_ros2_control>
+  <!-- world link -->
+  <link name="world"/>
+  <!-- robot links, joints -->
+  <xacro:kuka_kr560_r3100_2_robot prefix="$(arg prefix)" package_name="kuka_fortec_support"/>
+  <!-- default world - base_link joint -->
+  <joint name="$(arg prefix)world-base_link" type="fixed">
+    <parent link="world"/>
+    <child link="$(arg prefix)base_link"/>
     <origin xyz="$(arg x) $(arg y) $(arg z)" rpy="$(arg roll) $(arg pitch) $(arg yaw)"/>
-  </xacro:kuka_kr560_r3100_2_robot>
+  </joint>
 </robot>

File: kuka_fortec_support/urdf/kr_fortec_ros2_control_macro.xacro (robot description, xacro)
@@ -1,5 +1,5 @@
 <?xml version="1.0" encoding="UTF-8"?>
 <robot xmlns:xacro="http://www.ros.org/wiki/xacro">
-  <xacro:macro name="kuka_fortec_ros2_control" params="name driver_version client_ip client_port controller_ip prefix mode use_gpio roundtrip_time verify_robot_model">
+  <xacro:macro name="kuka_fortec_ros2_control" params="name driver_version client_ip client_port controller_ip prefix mode use_gpio roundtrip_time verify_robot_model **ext_axes_ros2_control_joints">
     <!-- gazebo -->
     <xacro:if value="${mode == 'gazebo'}">
@@ -32,4 +32,5 @@
         </xacro:if>
       </hardware>
+      <xacro:insert_block name="ext_axes_ros2_control_joints"/>
       <joint name="${prefix}joint_1">
         <command_interface name="position"/>

File: kuka_iontec_support/urdf/kr70_r2100.urdf.xacro (robot description, xacro)
@@ -20,7 +20,16 @@
   <xacro:arg name="pitch" default="0"/>
   <xacro:arg name="yaw" default="0"/>
-  <xacro:kuka_iontec_ros2_control name="$(arg prefix)kr70_r2100" driver_version="$(arg driver_version)" client_ip="$(arg client_ip)" controller_ip="$(arg controller_ip)" client_port="$(arg client_port)" prefix="$(arg prefix)" mode="$(arg mode)" use_gpio="$(arg use_gpio)" roundtrip_time="$(arg roundtrip_time)" verify_robot_model="$(arg verify_robot_model)"/>
-  <xacro:kuka_kr70_r2100_robot prefix="$(arg prefix)" package_name="kuka_iontec_support">
+  <xacro:kuka_iontec_ros2_control name="$(arg prefix)kr70_r2100" driver_version="$(arg driver_version)" client_ip="$(arg client_ip)" controller_ip="$(arg controller_ip)" client_port="$(arg client_port)" prefix="$(arg prefix)" mode="$(arg mode)" use_gpio="$(arg use_gpio)" roundtrip_time="$(arg roundtrip_time)" verify_robot_model="$(arg verify_robot_model)">
+    <ext_axes_ros2_control_joints/>
+  </xacro:kuka_iontec_ros2_control>
+  <!-- world link -->
+  <link name="world"/>
+  <!-- robot links, joints -->
+  <xacro:kuka_kr70_r2100_robot prefix="$(arg prefix)" package_name="kuka_iontec_support"/>
+  <!-- default world - base_link joint -->
+  <joint name="$(arg prefix)world-base_link" type="fixed">
+    <parent link="world"/>
+    <child link="$(arg prefix)base_link"/>
     <origin xyz="$(arg x) $(arg y) $(arg z)" rpy="$(arg roll) $(arg pitch) $(arg yaw)"/>
-  </xacro:kuka_kr70_r2100_robot>
+  </joint>
 </robot>

File: kuka_iontec_support/urdf/kr70_r2100_macro.xacro (robot description, xacro)
@@ -1,7 +1,6 @@
 <?xml version="1.0"?>
 <robot xmlns:xacro="http://wiki.ros.org/xacro">
-  <xacro:macro name="kuka_kr70_r2100_robot" params="prefix package_name *origin">
+  <xacro:macro name="kuka_kr70_r2100_robot" params="prefix package_name">
     <!-- links - main serial chain -->
-    <link name="world"/>
     <link name="${prefix}base_link">
       <collision>
@@ -137,9 +136,4 @@
       </visual>
     </link>
-    <joint name="${prefix}world-base_link" type="fixed">
-      <parent link="world"/>
-      <child link="${prefix}base_link"/>
-      <xacro:insert_block name="origin"/>
-    </joint>
     <joint name="${prefix}joint_1" type="revolute">
       <axis xyz="0.0 0.0 1.0"/>

File: kuka_iontec_support/urdf/kr_iontec_ros2_control_macro.xacro (robot description, xacro)
@@ -1,5 +1,5 @@
 <?xml version="1.0" encoding="UTF-8"?>
 <robot xmlns:xacro="http://www.ros.org/wiki/xacro">
-  <xacro:macro name="kuka_iontec_ros2_control" params="name driver_version client_ip client_port controller_ip prefix mode use_gpio roundtrip_time verify_robot_model">
+  <xacro:macro name="kuka_iontec_ros2_control" params="name driver_version client_ip client_port controller_ip prefix mode use_gpio roundtrip_time verify_robot_model **ext_axes_ros2_control_joints">
     <!-- gazebo -->
     <xacro:if value="${mode == 'gazebo'}">
@@ -32,4 +32,5 @@
         </xacro:if>
       </hardware>
+      <xacro:insert_block name="ext_axes_ros2_control_joints"/>
       <joint name="${prefix}joint_1">
         <command_interface name="position"/>

File: kuka_kl_support/urdf/kl100_2_macro.xacro (robot description, xacro)
@@ -1,15 +1,15 @@
 <?xml version="1.0" encoding="UTF-8"?>
 <robot xmlns:xacro="http://www.ros.org/wiki/xacro">
-  <xacro:macro name="kl100_links" params="">
+  <xacro:macro name="kl100_2_links" params="">
     <!-- links -->
     <link name="rail_base_link">
       <visual>
         <geometry>
-          <mesh filename="package://kuka_kl_support/meshes/kl100/visual/rail_base_link.dae"/>
+          <mesh filename="package://kuka_kl_support/meshes/kl100_2/visual/rail_base_link.dae"/>
         </geometry>
       </visual>
       <collision>
         <geometry>
-          <mesh filename="package://kuka_kl_support/meshes/kl100/collision/rail_base_link.stl"/>
+          <mesh filename="package://kuka_kl_support/meshes/kl100_2/collision/rail_base_link.stl"/>
         </geometry>
       </collision>
@@ -18,15 +18,15 @@
       <visual>
         <geometry>
-          <mesh filename="package://kuka_kl_support/meshes/kl100/visual/rail_moving_link.dae"/>
+          <mesh filename="package://kuka_kl_support/meshes/kl100_2/visual/rail_moving_link.dae"/>
         </geometry>
       </visual>
       <collision>
         <geometry>
-          <mesh filename="package://kuka_kl_support/meshes/kl100/collision/rail_moving_link.stl"/>
+          <mesh filename="package://kuka_kl_support/meshes/kl100_2/collision/rail_moving_link.stl"/>
         </geometry>
       </collision>
     </link>
   </xacro:macro>
-  <xacro:macro name="kl100_joints" params="robot_base_link *origin">
+  <xacro:macro name="kl100_2_joints" params="robot_base_link *origin">
     <!-- joints -->
     <joint name="world-rail_base" type="fixed">
@@ -40,10 +40,10 @@
       <origin rpy="0.0 0.0 0.0" xyz="0.0 0.0 0.0"/>
       <axis xyz="1 0 0"/>
-      <limit lower="-1" upper="1" effort="100.0" velocity="1.0"/>
+      <limit lower="-1.0" upper="1.0" effort="702.0" velocity="2.5"/>
     </joint>
     <joint name="rail-robot_base" type="fixed">
       <parent link="rail_moving_link"/>
       <child link="${robot_base_link}"/>
-      <origin rpy="0.0 0.0 0.0" xyz="0.0 0.0 0.35"/>
+      <origin rpy="0.0 0.0 0.0" xyz="0.0 0.0 0.356"/>
     </joint>
   </xacro:macro>

File: kuka_lbr_iisy_support/urdf/lbr_iisy11_r1300.urdf.xacro (robot description, xacro)
@@ -17,7 +17,16 @@
   <xacro:arg name="pitch" default="0"/>
   <xacro:arg name="yaw" default="0"/>
-  <xacro:kuka_lbr_iisy_ros2_control name="$(arg prefix)lbr_iisy11_r1300" prefix="$(arg prefix)" controller_ip="$(arg controller_ip)" client_ip="$(arg client_ip)" mode="$(arg mode)" roundtrip_time="$(arg roundtrip_time)" qos_config_file="$(arg qos_config_file)"/>
-  <xacro:kuka_lbr_iisy11_r1300_robot prefix="$(arg prefix)" package_name="kuka_lbr_iisy_support">
+  <xacro:kuka_lbr_iisy_ros2_control name="$(arg prefix)lbr_iisy11_r1300" prefix="$(arg prefix)" controller_ip="$(arg controller_ip)" client_ip="$(arg client_ip)" mode="$(arg mode)" roundtrip_time="$(arg roundtrip_time)" qos_config_file="$(arg qos_config_file)">
+    <ext_axis_ros2_control_joints/>
+  </xacro:kuka_lbr_iisy_ros2_control>
+  <!-- world link -->
+  <link name="world"/>
+  <!-- robot links, joints -->
+  <xacro:kuka_lbr_iisy11_r1300_robot prefix="$(arg prefix)" package_name="kuka_lbr_iisy_support"/>
+  <!-- default world - base_link joint -->
+  <joint name="$(arg prefix)world-base_link" type="fixed">
+    <parent link="world"/>
+    <child link="$(arg prefix)base_link"/>
     <origin xyz="$(arg x) $(arg y) $(arg z)" rpy="$(arg roll) $(arg pitch) $(arg yaw)"/>
-  </xacro:kuka_lbr_iisy11_r1300_robot>
+  </joint>
 </robot>

File: kuka_lbr_iisy_support/urdf/lbr_iisy15_r930.urdf.xacro (robot description, xacro)
@@ -17,7 +17,16 @@
   <xacro:arg name="pitch" default="0"/>
   <xacro:arg name="yaw" default="0"/>
-  <xacro:kuka_lbr_iisy_ros2_control name="$(arg prefix)lbr_iisy15_r930" prefix="$(arg prefix)" controller_ip="$(arg controller_ip)" client_ip="$(arg client_ip)" mode="$(arg mode)" roundtrip_time="$(arg roundtrip_time)" qos_config_file="$(arg qos_config_file)"/>
-  <xacro:kuka_lbr_iisy15_r930_robot prefix="$(arg prefix)" package_name="kuka_lbr_iisy_support">
+  <xacro:kuka_lbr_iisy_ros2_control name="$(arg prefix)lbr_iisy15_r930" prefix="$(arg prefix)" controller_ip="$(arg controller_ip)" client_ip="$(arg client_ip)" mode="$(arg mode)" roundtrip_time="$(arg roundtrip_time)" qos_config_file="$(arg qos_config_file)">
+    <ext_axis_ros2_control_joints/>
+  </xacro:kuka_lbr_iisy_ros2_control>
+  <!-- world link -->
+  <link name="world"/>
+  <!-- robot links, joints -->
+  <xacro:kuka_lbr_iisy15_r930_robot prefix="$(arg prefix)" package_name="kuka_lbr_iisy_support"/>
+  <!-- default world - base_link joint -->
+  <joint name="$(arg prefix)world-base_link" type="fixed">
+    <parent link="world"/>
+    <child link="$(arg prefix)base_link"/>
     <origin xyz="$(arg x) $(arg y) $(arg z)" rpy="$(arg roll) $(arg pitch) $(arg yaw)"/>
-  </xacro:kuka_lbr_iisy15_r930_robot>
+  </joint>
 </robot>

File: kuka_lbr_iisy_support/urdf/lbr_iisy3_r760.urdf.xacro (robot description, xacro)
@@ -17,7 +17,16 @@
   <xacro:arg name="pitch" default="0"/>
   <xacro:arg name="yaw" default="0"/>
-  <xacro:kuka_lbr_iisy_ros2_control name="$(arg prefix)lbr_iisy3_r760" prefix="$(arg prefix)" controller_ip="$(arg controller_ip)" client_ip="$(arg client_ip)" mode="$(arg mode)" roundtrip_time="$(arg roundtrip_time)" qos_config_file="$(arg qos_config_file)"/>
-  <xacro:kuka_lbr_iisy3_r760_robot prefix="$(arg prefix)" package_name="kuka_lbr_iisy_support">
+  <xacro:kuka_lbr_iisy_ros2_control name="$(arg prefix)lbr_iisy3_r760" prefix="$(arg prefix)" controller_ip="$(arg controller_ip)" client_ip="$(arg client_ip)" mode="$(arg mode)" roundtrip_time="$(arg roundtrip_time)" qos_config_file="$(arg qos_config_file)">
+    <ext_axis_ros2_control_joints/>
+  </xacro:kuka_lbr_iisy_ros2_control>
+  <!-- world link -->
+  <link name="world"/>
+  <!-- robot links, joints -->
+  <xacro:kuka_lbr_iisy3_r760_robot prefix="$(arg prefix)" package_name="kuka_lbr_iisy_support"/>
+  <!-- default world - base_link joint -->
+  <joint name="$(arg prefix)world-base_link" type="fixed">
+    <parent link="world"/>
+    <child link="$(arg prefix)base_link"/>
     <origin xyz="$(arg x) $(arg y) $(arg z)" rpy="$(arg roll) $(arg pitch) $(arg yaw)"/>
-  </xacro:kuka_lbr_iisy3_r760_robot>
+  </joint>
 </robot>

File: kuka_lbr_iisy_support/urdf/lbr_iisy_ros2_control_macro.xacro (robot description, xacro)
@@ -1,5 +1,5 @@
 <?xml version="1.0" encoding="UTF-8"?>
 <robot xmlns:xacro="http://www.ros.org/wiki/xacro">
-  <xacro:macro name="kuka_lbr_iisy_ros2_control" params="name prefix client_ip controller_ip mode qos_config_file roundtrip_time">
+  <xacro:macro name="kuka_lbr_iisy_ros2_control" params="name prefix client_ip controller_ip mode qos_config_file roundtrip_time **ext_axes_ros2_control_joints">
     <!-- gazebo -->
     <xacro:if value="${mode == 'gazebo'}">
@@ -40,4 +40,5 @@
         </xacro:if>
       </hardware>
+      <xacro:insert_block name="ext_axes_ros2_control_joints"/>
       <!-- define joints and command/state interfaces for each joint -->
       <joint name="${prefix}joint_1">
