Commit message: Change robot description to new convention

File: kuka_lbr_iiwa_support/urdf/lbr_iiwa14_r820.urdf.xacro (robot description, xacro)
@@ -17,7 +17,16 @@
   <xacro:arg name="yaw" default="0"/>
   <xacro:arg name="prefix" default=""/>
-  <xacro:kuka_lbr_iiwa_ros2_control name="$(arg prefix)lbr_iiwa14_r820" prefix="$(arg prefix)" io_access="false" mode="$(arg mode)" roundtrip_time="$(arg roundtrip_time)" controller_ip="$(arg controller_ip)" client_ip="$(arg client_ip)" client_port="$(arg client_port)"/>
-  <xacro:kuka_lbr_iiwa14_r820_robot prefix="$(arg prefix)" package_name="kuka_lbr_iiwa_support">
+  <xacro:kuka_lbr_iiwa_ros2_control name="$(arg prefix)lbr_iiwa14_r820" prefix="$(arg prefix)" io_access="false" mode="$(arg mode)" roundtrip_time="$(arg roundtrip_time)" controller_ip="$(arg controller_ip)" client_ip="$(arg client_ip)" client_port="$(arg client_port)">
+    <ext_axis_ros2_control_joints/>
+  </xacro:kuka_lbr_iiwa_ros2_control>
+  <!-- world link -->
+  <link name="world"/>
+  <!-- robot links, joints -->
+  <xacro:kuka_lbr_iiwa14_r820_robot prefix="$(arg prefix)" package_name="kuka_lbr_iiwa_support"/>
+  <!-- default world - base_link joint -->
+  <joint name="$(arg prefix)world-base_link" type="fixed">
+    <parent link="world"/>
+    <child link="$(arg prefix)base_link"/>
     <origin xyz="$(arg x) $(arg y) $(arg z)" rpy="$(arg roll) $(arg pitch) $(arg yaw)"/>
-  </xacro:kuka_lbr_iiwa14_r820_robot>
+  </joint>
 </robot>

File: kuka_lbr_iiwa_support/urdf/lbr_iiwa_ros2_control_macro.xacro (robot description, xacro)
@@ -1,5 +1,5 @@
 <?xml version="1.0" encoding="UTF-8"?>
 <robot xmlns:xacro="http://www.ros.org/wiki/xacro">
-  <xacro:macro name="kuka_lbr_iiwa_ros2_control" params="name prefix io_access mode roundtrip_time controller_ip client_ip client_port">
+  <xacro:macro name="kuka_lbr_iiwa_ros2_control" params="name prefix io_access mode roundtrip_time controller_ip client_ip client_port **ext_axes_ros2_control_joints">
     <!-- gazebo -->
     <xacro:if value="${mode == 'gazebo'}">
@@ -27,4 +27,5 @@
         </xacro:if>
       </hardware>
+      <xacro:insert_block name="ext_axes_ros2_control_joints"/>
       <!-- define joints and command/state interfaces for each joint -->
       <joint name="${prefix}joint_1">

File: kuka_quantec_support/urdf/kr150_r3100_2.urdf.xacro (robot description, xacro)
@@ -20,7 +20,16 @@
   <xacro:arg name="pitch" default="0"/>
   <xacro:arg name="yaw" default="0"/>
-  <xacro:kuka_quantec_ros2_control name="$(arg prefix)kr150_r3100_2" driver_version="$(arg driver_version)" client_ip="$(arg client_ip)" client_port="$(arg client_port)" controller_ip="$(arg controller_ip)" prefix="$(arg prefix)" mode="$(arg mode)" use_gpio="$(arg use_gpio)" roundtrip_time="$(arg roundtrip_time)" verify_robot_model="$(arg verify_robot_model)"/>
-  <xacro:kuka_kr150_r3100_2_robot prefix="$(arg prefix)" package_name="kuka_quantec_support">
+  <xacro:kuka_quantec_ros2_control name="$(arg prefix)kr150_r3100_2" driver_version="$(arg driver_version)" client_ip="$(arg client_ip)" client_port="$(arg client_port)" controller_ip="$(arg controller_ip)" prefix="$(arg prefix)" mode="$(arg mode)" use_gpio="$(arg use_gpio)" roundtrip_time="$(arg roundtrip_time)" verify_robot_model="$(arg verify_robot_model)">
+    <ext_axis_ros2_control_joints/>
+  </xacro:kuka_quantec_ros2_control>
+  <!-- world link -->
+  <link name="world"/>
+  <!-- robot links, joints -->
+  <xacro:kuka_kr150_r3100_2_robot prefix="$(arg prefix)" package_name="kuka_quantec_support"/>
+  <!-- default world - base_link joint -->
+  <joint name="$(arg prefix)world-base_link" type="fixed">
+    <parent link="world"/>
+    <child link="$(arg prefix)base_link"/>
     <origin xyz="$(arg x) $(arg y) $(arg z)" rpy="$(arg roll) $(arg pitch) $(arg yaw)"/>
-  </xacro:kuka_kr150_r3100_2_robot>
+  </joint>
 </robot>

File: kuka_quantec_support/urdf/kr210_r2700_2.urdf.xacro (robot description, xacro)
@@ -20,7 +20,16 @@
   <xacro:arg name="pitch" default="0"/>
   <xacro:arg name="yaw" default="0"/>
-  <xacro:kuka_quantec_ros2_control name="$(arg prefix)kr210_r2700_2" driver_version="$(arg driver_version)" client_ip="$(arg client_ip)" client_port="$(arg client_port)" controller_ip="$(arg controller_ip)" prefix="$(arg prefix)" mode="$(arg mode)" use_gpio="$(arg use_gpio)" roundtrip_time="$(arg roundtrip_time)" verify_robot_model="$(arg verify_robot_model)"/>
-  <xacro:kuka_kr210_r2700_2_robot prefix="$(arg prefix)" package_name="kuka_quantec_support">
+  <xacro:kuka_quantec_ros2_control name="$(arg prefix)kr210_r2700_2" driver_version="$(arg driver_version)" client_ip="$(arg client_ip)" client_port="$(arg client_port)" controller_ip="$(arg controller_ip)" prefix="$(arg prefix)" mode="$(arg mode)" use_gpio="$(arg use_gpio)" roundtrip_time="$(arg roundtrip_time)" verify_robot_model="$(arg verify_robot_model)">
+    <ext_axis_ros2_control_joints/>
+  </xacro:kuka_quantec_ros2_control>
+  <!-- world link -->
+  <link name="world"/>
+  <!-- robot links, joints -->
+  <xacro:kuka_kr210_r2700_2_robot prefix="$(arg prefix)" package_name="kuka_quantec_support"/>
+  <!-- default world - base_link joint -->
+  <joint name="$(arg prefix)world-base_link" type="fixed">
+    <parent link="world"/>
+    <child link="$(arg prefix)base_link"/>
     <origin xyz="$(arg x) $(arg y) $(arg z)" rpy="$(arg roll) $(arg pitch) $(arg yaw)"/>
-  </xacro:kuka_kr210_r2700_2_robot>
+  </joint>
 </robot>
