Commit message: add general kr support package for moveit

File: kuka_kr_moveit_config/srdf/kr_arm.srdf.xacro (robot description, xacro)
@@ -4,6 +4,7 @@
     A URDF file must exist for this robot as well, where the joints and the links that are referenced are defined
 -->
-<robot xmlns:xacro="http://www.ros.org/wiki/xacro" name="kuka_kr16_r2010-2">
-  <xacro:include filename="cybertech_arm.macro.xacro" />
-  <xacro:kuka_cybertech_arm prefix=""/>
+<!--TODO(Svastits): add an argument for the robot name instead of kr, as srdf model parsers logs an error now-->
+<robot xmlns:xacro="http://www.ros.org/wiki/xacro" name="kr">
+  <xacro:include filename="kr_arm_macro.xacro" />
+  <xacro:kuka_kr_arm prefix=""/>
 </robot>

File: kuka_kr_moveit_config/srdf/kr_arm_macro.xacro (robot description, xacro)
@@ -1,5 +1,5 @@
 <?xml version="1.0" ?>
 <robot xmlns:xacro="http://www.ros.org/wiki/xacro">
-  <xacro:macro name="kuka_cybertech_arm" params="prefix">
+  <xacro:macro name="kuka_kr_arm" params="prefix">
     <!--GROUPS: Representation of a set of joints and links. This can be useful for specifying DOF to plan for, defining arms, end effectors, etc-->
     <!--LINKS: When a link is specified, the parent joint of that link (if it exists) is automatically included-->
@@ -7,13 +7,13 @@
     <!--CHAINS: When a chain is specified, all the links along the chain (including endpoints) are included in the group. Additionally, all the joints that are parents to included links are also included. This means that joints along the chain and the parent joint of the base link are included in the group-->
     <!--SUBGROUPS: Groups can also be formed by referencing to already defined group names-->
-    <group name="cybertech_arm">
-      <chain base_link="${prefix}base_link" tip_link="${prefix}flange" />
+    <group name="${prefix}kr_arm">
+      <chain base_link="${prefix}base_link" tip_link="${prefix}tool0" />
     </group>
-    <!--Add flange as end effector to be able to use moveit_visual_tools for visualising end effector path-->
-    <group name="end_effector">
-      <link name="${prefix}flange"/>
+    <!--Add tool0 as end effector to be able to use moveit_visual_tools for visualising end effector path-->
+    <group name="${prefix}end_effector">
+      <link name="${prefix}tool0"/>
     </group>
     <!--GROUP STATES: Purpose: Define a named state for a particular group, in terms of joint values. This is useful to define states like 'folded arms'-->
-    <group_state name="null_pos" group="cybertech_arm">
+    <group_state name="null_pos" group="${prefix}kr_arm">
       <joint name="${prefix}joint_a1" value="0" />
       <joint name="${prefix}joint_a2" value="0" />
@@ -23,8 +23,6 @@
       <joint name="${prefix}joint_a6" value="0" />
     </group_state>
-    <!--VIRTUAL JOINT: Purpose: this element defines a virtual joint between a robot link and an external frame of reference (considered fixed with respect to the robot)-->
-    <!-- <virtual_joint name="world_joint" type="fixed" parent_frame="world" child_link="base_link" /> -->
     <!--END EFFECTOR: Purpose: Represent information about an end effector.-->
-    <end_effector name="flange" parent_link="${prefix}flange" group="end_effector" parent_group="cybertech_arm"/>
+    <end_effector name="${prefix}eef" parent_link="${prefix}tool0" group="${prefix}end_effector" parent_group="${prefix}kr_arm"/>
     <!--DISABLE COLLISIONS: By default it is assumed that any link of the robot could potentially come into collision with any other link in the robot. This tag disables collision checking between a specified pair of links. -->
     <disable_collisions link1="${prefix}base_link_inertia" link2="${prefix}link_1" reason="Adjacent"/>
