Commit message: update home in srdf

File: kuka_kr_moveit_config/srdf/kr_arm_macro.xacro (robot description, xacro)
@@ -15,8 +15,8 @@
     </group>
     <!--GROUP STATES: Purpose: Define a named state for a particular group, in terms of joint values. This is useful to define states like 'folded arms'-->
-    <group_state name="null_pos" group="${prefix}kr_arm">
+    <group_state name="home" group="${prefix}kr_arm">
       <joint name="${prefix}joint_a1" value="0" />
-      <joint name="${prefix}joint_a2" value="0" />
-      <joint name="${prefix}joint_a3" value="0" />
+      <joint name="${prefix}joint_a2" value="${-pi/2}" />
+      <joint name="${prefix}joint_a3" value="${pi/2}" />
       <joint name="${prefix}joint_a4" value="0" />
       <joint name="${prefix}joint_a5" value="0" />

Commit message: manipulator for group name in srdf

File: kuka_kr_moveit_config/srdf/kr_arm_macro.xacro (robot description, xacro)
@@ -7,9 +7,9 @@
     <!--CHAINS: When a chain is specified, all the links along the chain (including endpoints) are included in the group. Additionally, all the joints that are parents to included links are also included. This means that joints along the chain and the parent joint of the base link are included in the group-->
     <!--SUBGROUPS: Groups can also be formed by referencing to already defined group names-->
-    <group name="${prefix}kr_arm">
+    <group name="${prefix}manipulator">
       <chain base_link="${prefix}base_link" tip_link="${prefix}tool0" />
     </group>
     <!--Add tool0 as end effector to be able to use moveit_visual_tools for visualising end effector path-->
-    <group name="${prefix}end_effector">
+    <group name="end_effector">
       <link name="${prefix}tool0"/>
     </group>

File: kuka_lbr_iisy_moveit_config/srdf/lbr_iisy_arm.macro.xacro (robot description, xacro)
@@ -7,10 +7,10 @@
     <!--CHAINS: When a chain is specified, all the links along the chain (including endpoints) are included in the group. Additionally, all the joints that are parents to included links are also included. This means that joints along the chain and the parent joint of the base link are included in the group-->
     <!--SUBGROUPS: Groups can also be formed by referencing to already defined group names-->
-    <group name="lbr_iisy_arm">
-      <chain base_link="${prefix}base_link" tip_link="${prefix}flange" />
+    <group name="${prefix}manipulator">
+      <chain base_link="${prefix}base_link" tip_link="${prefix}tool0" />
     </group>
-    <!--Add flange as end effector to be able to use moveit_visual_tools for visualising end effector path-->
+    <!--Add tool0 as end effector to be able to use moveit_visual_tools for visualising end effector path-->
     <group name="end_effector">
-      <link name="${prefix}flange"/>
+      <link name="${prefix}tool0"/>
     </group>
     <!--GROUP STATES: Purpose: Define a named state for a particular group, in terms of joint values. This is useful to define states like 'folded arms'-->

File: kuka_lbr_iiwa_moveit_config/srdf/lbr_iiwa_arm.macro.xacro (robot description, xacro)
@@ -7,10 +7,10 @@
     <!--CHAINS: When a chain is specified, all the links along the chain (including endpoints) are included in the group. Additionally, all the joints that are parents to included links are also included. This means that joints along the chain and the parent joint of the base link are included in the group-->
     <!--SUBGROUPS: Groups can also be formed by referencing to already defined group names-->
-    <group name="lbr_iiwa_arm">
-      <chain base_link="${prefix}base_link" tip_link="${prefix}flange" />
+    <group name="${prefix}manipulator">
+      <chain base_link="${prefix}base_link" tip_link="${prefix}tool0" />
     </group>
-    <!--Add flange as end effector to be able to use moveit_visual_tools for visualising end effector path-->
+    <!--Add tool0 as end effector to be able to use moveit_visual_tools for visualising end effector path-->
     <group name="end_effector">
-      <link name="${prefix}flange"/>
+      <link name="${prefix}tool0"/>
     </group>
     <!--GROUP STATES: Purpose: Define a named state for a particular group, in terms of joint values. This is useful to define states like 'folded arms'-->

Commit message: working dual robot prototype setup

File: kuka_kr_moveit_config/srdf/kr_arm_macro.xacro (robot description, xacro)
@@ -7,35 +7,35 @@
     <!--CHAINS: When a chain is specified, all the links along the chain (including endpoints) are included in the group. Additionally, all the joints that are parents to included links are also included. This means that joints along the chain and the parent joint of the base link are included in the group-->
     <!--SUBGROUPS: Groups can also be formed by referencing to already defined group names-->
-    <group name="${prefix}manipulator">
-      <chain base_link="${prefix}base_link" tip_link="${prefix}tool0"/>
+    <group name="manipulator">
+      <chain base_link="test2_base_link" tip_link="test2_tool0"/>
     </group>
     <!--Add tool0 as end effector to be able to use moveit_visual_tools for visualising end effector path-->
     <group name="end_effector">
-      <link name="${prefix}tool0"/>
+      <link name="test2_tool0"/>
     </group>
     <!--GROUP STATES: Purpose: Define a named state for a particular group, in terms of joint values. This is useful to define states like 'folded arms'-->
-    <group_state name="home" group="${prefix}manipulator">
-      <joint name="${prefix}joint_1" value="0"/>
-      <joint name="${prefix}joint_2" value="${-pi/2}"/>
-      <joint name="${prefix}joint_3" value="${pi/2}"/>
-      <joint name="${prefix}joint_4" value="0"/>
-      <joint name="${prefix}joint_5" value="0"/>
-      <joint name="${prefix}joint_6" value="0"/>
+    <group_state name="home" group="manipulator">
+      <joint name="test2_joint_1" value="0"/>
+      <joint name="test2_joint_2" value="${-pi/2}"/>
+      <joint name="test2_joint_3" value="${pi/2}"/>
+      <joint name="test2_joint_4" value="0"/>
+      <joint name="test2_joint_5" value="0"/>
+      <joint name="test2_joint_6" value="0"/>
     </group_state>
     <!--END EFFECTOR: Purpose: Represent information about an end effector.-->
-    <end_effector name="${prefix}eef" parent_link="${prefix}tool0" group="${prefix}end_effector" parent_group="${prefix}manipulator"/>
+    <end_effector name="test2_eef" parent_link="test2_tool0" group="end_effector" parent_group="manipulator"/>
     <!--DISABLE COLLISIONS: By default it is assumed that any link of the robot could potentially come into collision with any other link in the robot. This tag disables collision checking between a specified pair of links. -->
-    <disable_collisions link1="${prefix}base_link" link2="${prefix}link_1" reason="Adjacent"/>
-    <disable_collisions link1="${prefix}link_1" link2="${prefix}link_2" reason="Adjacent"/>
-    <disable_collisions link1="${prefix}link_2" link2="${prefix}link_3" reason="Adjacent"/>
-    <disable_collisions link1="${prefix}link_3" link2="${prefix}link_4" reason="Adjacent"/>
-    <disable_collisions link1="${prefix}link_4" link2="${prefix}link_5" reason="Adjacent"/>
-    <disable_collisions link1="${prefix}link_5" link2="${prefix}link_6" reason="Adjacent"/>
-    <disable_collisions link1="${prefix}link_1" link2="${prefix}link_3" reason="Never"/>
-    <disable_collisions link1="${prefix}link_2" link2="${prefix}link_5" reason="Never"/>
-    <disable_collisions link1="${prefix}link_2" link2="${prefix}link_6" reason="Never"/>
-    <disable_collisions link1="${prefix}link_3" link2="${prefix}link_5" reason="Never"/>
-    <disable_collisions link1="${prefix}link_3" link2="${prefix}link_6" reason="Never"/>
-    <disable_collisions link1="${prefix}link_4" link2="${prefix}link_6" reason="Never"/>
+    <disable_collisions link1="test2_base_link" link2="test2_link_1" reason="Adjacent"/>
+    <disable_collisions link1="test2_link_1" link2="test2_link_2" reason="Adjacent"/>
+    <disable_collisions link1="test2_link_2" link2="test2_link_3" reason="Adjacent"/>
+    <disable_collisions link1="test2_link_3" link2="test2_link_4" reason="Adjacent"/>
+    <disable_collisions link1="test2_link_4" link2="test2_link_5" reason="Adjacent"/>
+    <disable_collisions link1="test2_link_5" link2="test2_link_6" reason="Adjacent"/>
+    <disable_collisions link1="test2_link_1" link2="test2_link_3" reason="Never"/>
+    <disable_collisions link1="test2_link_2" link2="test2_link_5" reason="Never"/>
+    <disable_collisions link1="test2_link_2" link2="test2_link_6" reason="Never"/>
+    <disable_collisions link1="test2_link_3" link2="test2_link_5" reason="Never"/>
+    <disable_collisions link1="test2_link_3" link2="test2_link_6" reason="Never"/>
+    <disable_collisions link1="test2_link_4" link2="test2_link_6" reason="Never"/>
   </xacro:macro>
 </robot>

File: kuka_lbr_iisy_moveit_config/srdf/lbr_iisy_arm.macro.xacro (robot description, xacro)
@@ -7,31 +7,31 @@
     <!--CHAINS: When a chain is specified, all the links along the chain (including endpoints) are included in the group. Additionally, all the joints that are parents to included links are also included. This means that joints along the chain and the parent joint of the base link are included in the group-->
     <!--SUBGROUPS: Groups can also be formed by referencing to already defined group names-->
-    <group name="${prefix}manipulator">
-      <chain base_link="${prefix}base_link" tip_link="${prefix}tool0"/>
+    <group name="manipulator">
+      <chain base_link="test1_base_link" tip_link="test1_tool0"/>
     </group>
     <!--Add tool0 as end effector to be able to use moveit_visual_tools for visualising end effector path-->
-    <group name="${prefix}end_effector">
-      <link name="${prefix}tool0"/>
+    <group name="end_effector">
+      <link name="test1_tool0"/>
     </group>
     <!--GROUP STATES: Purpose: Define a named state for a particular group, in terms of joint values. This is useful to define states like 'folded arms'-->
-    <group_state name="null_pos" group="${prefix}manipulator">
-      <joint name="${prefix}joint_1" value="0"/>
-      <joint name="${prefix}joint_2" value="0"/>
-      <joint name="${prefix}joint_3" value="0"/>
-      <joint name="${prefix}joint_4" value="0"/>
-      <joint name="${prefix}joint_5" value="0"/>
-      <joint name="${prefix}joint_6" value="0"/>
+    <group_state name="null_pos" group="manipulator">
+      <joint name="test1_joint_1" value="0"/>
+      <joint name="test1_joint_2" value="0"/>
+      <joint name="test1_joint_3" value="0"/>
+      <joint name="test1_joint_4" value="0"/>
+      <joint name="test1_joint_5" value="0"/>
+      <joint name="test1_joint_6" value="0"/>
     </group_state>
     <!--VIRTUAL JOINT: Purpose: this element defines a virtual joint between a robot link and an external frame of reference (considered fixed with respect to the robot)-->
     <!-- <virtual_joint name="world_joint" type="fixed" parent_frame="world" child_link="world" /> -->
     <!--END EFFECTOR: Purpose: Represent information about an end effector.-->
-    <end_effector name="${prefix}tool0" parent_link="${prefix}tool0" group="${prefix}end_effector" parent_group="${prefix}manipulator"/>
+    <end_effector name="test1_tool0" parent_link="test1_tool0" group="end_effector" parent_group="manipulator"/>
     <!--DISABLE COLLISIONS: By default it is assumed that any link of the robot could potentially come into collision with any other link in the robot. This tag disables collision checking between a specified pair of links. -->
-    <disable_collisions link1="${prefix}base_link" link2="${prefix}link_1" reason="Adjacent"/>
-    <disable_collisions link1="${prefix}link_1" link2="${prefix}link_2" reason="Adjacent"/>
-    <disable_collisions link1="${prefix}link_2" link2="${prefix}link_3" reason="Adjacent"/>
-    <disable_collisions link1="${prefix}link_3" link2="${prefix}link_4" reason="Adjacent"/>
-    <disable_collisions link1="${prefix}link_4" link2="${prefix}link_5" reason="Adjacent"/>
-    <disable_collisions link1="${prefix}link_5" link2="${prefix}link_6" reason="Adjacent"/>
+    <disable_collisions link1="test1_base_link" link2="test1_link_1" reason="Adjacent"/>
+    <disable_collisions link1="test1_link_1" link2="test1_link_2" reason="Adjacent"/>
+    <disable_collisions link1="test1_link_2" link2="test1_link_3" reason="Adjacent"/>
+    <disable_collisions link1="test1_link_3" link2="test1_link_4" reason="Adjacent"/>
+    <disable_collisions link1="test1_link_4" link2="test1_link_5" reason="Adjacent"/>
+    <disable_collisions link1="test1_link_5" link2="test1_link_6" reason="Adjacent"/>
   </xacro:macro>
 </robot>
