Commit message: fix flange trafo

File: kuka_agilus_support/urdf/kr10_r1100-2_macro.xacro (robot description, xacro)
@@ -215,5 +215,5 @@
     <joint name="${prefix}link6-flange" type="fixed">
       <child link="${prefix}flange" />
-      <origin rpy="0 ${pi} -0.0" xyz="0.0 0.0 -0.1605" />
+      <origin rpy="0 ${pi} -0.0" xyz="0.0 0.0 -0.09" />
       <parent link="${prefix}link_6" />
     </joint>
@@ -222,5 +222,5 @@
     <joint name="${prefix}link6-tool0" type="fixed">
       <child link="${prefix}tool0" />
-      <origin rpy="0 ${pi} -0.0" xyz="0.0 0.0 -0.1605" />
+      <origin rpy="0 ${pi} -0.0" xyz="0.0 0.0 -0.09" />
       <parent link="${prefix}link_6" />
     </joint>
