Commit message: test launc file with fake hw

File: kuka_agilus_support/urdf/kr6_r700-sixx_macro.xacro (robot description, xacro)
@@ -5,11 +5,9 @@
   <xacro:include filename="$(find kuka_agilus_support)/urdf/kr_agilus_ros2_control.xacro" />
   <xacro:include filename="$(find kuka_agilus_support)/urdf/kr_agilus_transmission.xacro" />
-  <xacro:macro name="kuka_kr6_r700-sixx_robot" params="prefix client_ip client_port use_fake_hardware">
+  <xacro:macro name="kuka_kr6_r700-sixx_robot" params="prefix use_fake_hardware">
     <!-- ros2 control instance -->
     <xacro:kuka_agilus_ros2_control
     name="kr6_r700-sixx"
     prefix="${prefix}"
-    client_ip="${client_ip}"
-    client_port="${client_port}"
     use_fake_hardware="${use_fake_hardware}" />
     <link name="${prefix}base_link"/>

File: kuka_agilus_support/urdf/kr6_r900-sixx_macro.xacro (robot description, xacro)
@@ -5,11 +5,9 @@
   <xacro:include filename="$(find kuka_agilus_support)/urdf/kr_agilus_ros2_control.xacro" />
   <xacro:include filename="$(find kuka_agilus_support)/urdf/kr_agilus_transmission.xacro" />
-  <xacro:macro name="kuka_kr6_r900-sixx_robot" params="prefix client_ip client_port use_fake_hardware">
+  <xacro:macro name="kuka_kr6_r900-sixx_robot" params="prefix use_fake_hardware">
     <!-- ros2 control instance -->
     <xacro:kuka_agilus_ros2_control
     name="kr6_r900-sixx"
     prefix="${prefix}"
-    client_ip="${client_ip}"
-    client_port="${client_port}"
     use_fake_hardware="${use_fake_hardware}" />
     <link name="${prefix}base_link"/>

File: kuka_agilus_support/urdf/kr_agilus_ros2_control.xacro (robot description, xacro)
@@ -1,5 +1,5 @@
 <?xml version="1.0" encoding="UTF-8"?>
 <robot xmlns:xacro="http://www.ros.org/wiki/xacro">
-  <xacro:macro name="kuka_agilus_ros2_control" params="name prefix client_ip client_port use_fake_hardware:=false">
+  <xacro:macro name="kuka_agilus_ros2_control" params="name prefix use_fake_hardware:=false">
     <ros2_control name="${name}" type="system">
       <hardware>
@@ -10,4 +10,9 @@
         </xacro:if>
         <xacro:unless value="${use_fake_hardware}">
+          <!-- Read parameters from rsi_config  -->
+          <xacro:property name="rsi_config" value="$(find kuka_rsi_hw_interface)/config/rsi_config.yaml" />
+          <xacro:property name="rsi_config_dict" value="${xacro.load_yaml(rsi_config)}"/>
+          <xacro:property name="client_ip" value="${rsi_config_dict['client_ip']}" />
+          <xacro:property name="client_port" value="${rsi_config_dict['client_port']}" />
           <plugin>kuka_rsi_hw_interface::KukaRSIHardwareInterface</plugin>
           <param name="client_ip">${client_ip}</param>

File: kuka_cybertech_support/urdf/kr16_r2010-2.urdf.xacro (robot description, xacro)
@@ -1,16 +1,8 @@
 <?xml version="1.0"?>
 <robot xmlns:xacro="http://www.ros.org/wiki/xacro" name="kr16_r2010-2">
-<!-- Import urdf file  -->
-<xacro:include filename="$(find kuka_cybertech_support)/urdf/kr16_r2010-2_macro.xacro"/>
-<!-- Read parameters from rsi_config  -->
-<xacro:property name="rsi_config" value="$(find kuka_rsi_hw_interface)/config/rsi_config.yaml" />
-<xacro:property name="rsi_config_dict" value="${xacro.load_yaml(rsi_config)}"/>
-<xacro:property name="client_ip" value="${rsi_config_dict['client_ip']}" />
-<xacro:property name="client_port" value="${rsi_config_dict['client_port']}" />
-<!-- Read additional arguments  -->
-<xacro:arg name="use_fake_hardware" default="false" />
-<xacro:kuka_kr16_r2010-2_robot prefix=""
-                  client_ip="${client_ip}"
-                  client_port="${client_port}"
-                  use_fake_hardware="$(arg use_fake_hardware)"/>
+  <!-- Import urdf file  -->
+  <xacro:include filename="$(find kuka_cybertech_support)/urdf/kr16_r2010-2_macro.xacro"/>
+  <!-- Read additional arguments  -->
+  <xacro:arg name="use_fake_hardware" default="false" />
+  <xacro:kuka_kr16_r2010-2_robot prefix="" use_fake_hardware="$(arg use_fake_hardware)"/>
 </robot>

File: kuka_cybertech_support/urdf/kr16_r2010-2_macro.xacro (robot description, xacro)
@@ -3,11 +3,9 @@
   <xacro:include filename="$(find kuka_cybertech_support)/urdf/kr_cybertech_ros2_control.xacro" />
   <xacro:include filename="$(find kuka_cybertech_support)/urdf/kr_cybertech_transmission.xacro" />
-  <xacro:macro name="kuka_kr16_r2010-2_robot" params="prefix client_ip client_port use_fake_hardware">
+  <xacro:macro name="kuka_kr16_r2010-2_robot" params="prefix use_fake_hardware">
     <!-- ros2 control instance -->
     <xacro:kuka_cybertech_ros2_control
     name="kr16_r2010-2"
     prefix="${prefix}"
-    client_ip="${client_ip}"
-    client_port="${client_port}"
     use_fake_hardware="${use_fake_hardware}" />
     <link name="${prefix}base_link"/>

File: kuka_cybertech_support/urdf/kr_cybertech_ros2_control.xacro (robot description, xacro)
@@ -1,5 +1,5 @@
 <?xml version="1.0" encoding="UTF-8"?>
 <robot xmlns:xacro="http://www.ros.org/wiki/xacro">
-  <xacro:macro name="kuka_cybertech_ros2_control" params="name prefix client_ip client_port use_fake_hardware:=false">
+  <xacro:macro name="kuka_cybertech_ros2_control" params="name prefix use_fake_hardware:=false">
     <ros2_control name="${name}" type="system">
       <hardware>
@@ -10,4 +10,9 @@
         </xacro:if>
         <xacro:unless value="${use_fake_hardware}">
+          <!-- Read parameters from rsi_config  -->
+          <xacro:property name="rsi_config" value="$(find kuka_rsi_hw_interface)/config/rsi_config.yaml" />
+          <xacro:property name="rsi_config_dict" value="${xacro.load_yaml(rsi_config)}"/>
+          <xacro:property name="client_ip" value="${rsi_config_dict['client_ip']}" />
+          <xacro:property name="client_port" value="${rsi_config_dict['client_port']}" />
           <plugin>kuka_rsi_hw_interface::KukaRSIHardwareInterface</plugin>
           <param name="client_ip">${client_ip}</param>

File: kuka_lbr_iiwa_support/urdf/lbr_iiwa14_r820.urdf.xacro (robot description, xacro)
@@ -5,5 +5,4 @@
 <!-- Read additional arguments  -->
 <xacro:arg name="use_fake_hardware" default="false" />
-<xacro:arg name="gazebo_sim" default="false" />
-<xacro:kuka_lbr_iiwa14_r820_robot prefix="" io_access="false" use_fake_hardware="$(arg use_fake_hardware)" gazebo_sim="$(arg gazebo_sim)"/>
+<xacro:kuka_lbr_iiwa14_r820_robot prefix="" io_access="false" use_fake_hardware="$(arg use_fake_hardware)"/>
 </robot>

File: kuka_lbr_iiwa_support/urdf/lbr_iiwa14_r820_macro.xacro (robot description, xacro)
@@ -5,5 +5,5 @@
   <xacro:include filename="$(find kuka_resources)/urdf/common_materials.xacro"/>
   <xacro:include filename="$(find kuka_lbr_iiwa_support)/urdf/lbr_iiwa_transmission.xacro" />
-  <xacro:macro name="kuka_lbr_iiwa14_r820_robot" params="io_access prefix use_fake_hardware:=false gazebo_sim:=false">
+  <xacro:macro name="kuka_lbr_iiwa14_r820_robot" params="io_access prefix use_fake_hardware:=false">
     <!-- ros2 control instance -->
     <xacro:kuka_lbr_iiwa_ros2_control
@@ -11,6 +11,5 @@
     prefix="${prefix}"
     io_access = "${io_access}"
-    use_fake_hardware="${use_fake_hardware}"
-    gazebo_sim="${gazebo_sim}" />
+    use_fake_hardware="${use_fake_hardware}" />
     <!-- links - main serial chain -->
     <!-- links - root element cannot have inertia, therefore a dummy base_link is needed -->

File: kuka_lbr_iiwa_support/urdf/lbr_iiwa_ros2_control.xacro (robot description, xacro)
@@ -1,16 +1,11 @@
 <?xml version="1.0" encoding="UTF-8"?>
 <robot xmlns:xacro="http://www.ros.org/wiki/xacro">
-  <xacro:macro name="kuka_lbr_iiwa_ros2_control" params="name prefix io_access use_fake_hardware:=false gazebo_sim:=false">
+  <xacro:macro name="kuka_lbr_iiwa_ros2_control" params="name prefix io_access use_fake_hardware:=false">
     <ros2_control name="${name}" type="system">
       <hardware>
         <xacro:if value="${use_fake_hardware}">
-          <xacro:if value="${gazebo_sim}">
-            <plugin>gazebo_ros2_control/GazeboSystem</plugin>
-          </xacro:if>
-          <xacro:unless value="${gazebo_sim}">
-            <plugin>mock_components/GenericSystem</plugin>
-            <param name="fake_sensor_commands">false</param>
-            <param name="state_following_offset">0.0</param>
-          </xacro:unless>
+          <plugin>mock_components/GenericSystem</plugin>
+          <param name="fake_sensor_commands">false</param>
+          <param name="state_following_offset">0.0</param>
         </xacro:if>
         <xacro:unless value="${use_fake_hardware}">
@@ -69,20 +64,14 @@
       </joint>
       <!-- TODO(Svastits): update GPIO list from config file-->
-      <xacro:if value="${io_access}">
-        <xacro:include filename="$(find kuka_sunrise)/config/gpio_config.xacro" />
-        <xacro:fri_gpio_config/>
-      </xacro:if>
-      <xacro:unless value="${io_access}">
-        <gpio name="gpio"/>
+      <xacro:unless value="${use_fake_hardware}">
+        <xacro:if value="${io_access}">
+          <xacro:include filename="$(find kuka_sunrise)/config/gpio_config.xacro" />
+          <xacro:fri_gpio_config/>
+        </xacro:if>
+        <xacro:unless value="${io_access}">
+          <gpio name="gpio"/>
+        </xacro:unless>
       </xacro:unless>
     </ros2_control>
-    <gazebo>
-      <plugin filename="libgazebo_ros2_control.so" name="gazebo_ros2_control">
-        <robot_param>robot_description</robot_param>
-        <robot_param_node>robot_state_publisher</robot_param_node>
-        <parameters>$(find kuka_sunrise)/config/ros2_controller_config.yaml</parameters>
-        <parameters>$(find kuka_sunrise)/config/joint_trajectory_controller_config.yaml</parameters>
-      </plugin>
-    </gazebo>
   </xacro:macro>
 </robot>

File: kuka_quantec_support/urdf/kr210_r2700-2.urdf.xacro (robot description, xacro)
@@ -1,16 +1,8 @@
 <?xml version="1.0"?>
 <robot xmlns:xacro="http://www.ros.org/wiki/xacro" name="kr210_r2700-2">
-<!-- Import urdf file  -->
-<xacro:include filename="$(find kuka_quantec_support)/urdf/kr210_r2700-2_macro.xacro"/>
-<!-- Read parameters from rsi_config  -->
-<xacro:property name="rsi_config" value="$(find kuka_rsi_hw_interface)/config/rsi_config.yaml" />
-<xacro:property name="rsi_config_dict" value="${xacro.load_yaml(rsi_config)}"/>
-<xacro:property name="client_ip" value="${rsi_config_dict['client_ip']}" />
-<xacro:property name="client_port" value="${rsi_config_dict['client_port']}" />
-<!-- Read additional arguments  -->
-<xacro:arg name="use_fake_hardware" default="false" />
-<xacro:kuka_kr210_r2700-2_robot prefix=""
-                  client_ip="${client_ip}"
-                  client_port="${client_port}"
-                  use_fake_hardware="$(arg use_fake_hardware)"/>
+  <!-- Import urdf file  -->
+  <xacro:include filename="$(find kuka_quantec_support)/urdf/kr210_r2700-2_macro.xacro"/>
+  <!-- Read additional arguments  -->
+  <xacro:arg name="use_fake_hardware" default="false" />
+  <xacro:kuka_kr210_r2700-2_robot prefix="" use_fake_hardware="$(arg use_fake_hardware)"/>
 </robot>

File: kuka_quantec_support/urdf/kr210_r2700-2_macro.xacro (robot description, xacro)
@@ -3,11 +3,9 @@
   <xacro:include filename="$(find kuka_quantec_support)/urdf/kr_quantec_ros2_control.xacro" />
   <xacro:include filename="$(find kuka_quantec_support)/urdf/kr_quantec_transmission.xacro" />
-  <xacro:macro name="kuka_kr210_r2700-2_robot" params="prefix client_ip client_port use_fake_hardware">
+  <xacro:macro name="kuka_kr210_r2700-2_robot" params="prefix use_fake_hardware">
     <!-- ros2 control instance -->
     <xacro:kuka_quantec_ros2_control
     name="kr210_r2700-2"
     prefix="${prefix}"
-    client_ip="${client_ip}"
-    client_port="${client_port}"
     use_fake_hardware="${use_fake_hardware}" />
     <link name="${prefix}base_link"/>

File: kuka_quantec_support/urdf/kr210_r3100-2.urdf.xacro (robot description, xacro)
@@ -1,16 +1,8 @@
 <?xml version="1.0"?>
 <robot xmlns:xacro="http://www.ros.org/wiki/xacro" name="kr210_r3100-2">
-<!-- Import urdf file  -->
-<xacro:include filename="$(find kuka_quantec_support)/urdf/kr210_r3100-2_macro.xacro"/>
-<!-- Read parameters from rsi_config  -->
-<xacro:property name="rsi_config" value="$(find kuka_rsi_hw_interface)/config/rsi_config.yaml" />
-<xacro:property name="rsi_config_dict" value="${xacro.load_yaml(rsi_config)}"/>
-<xacro:property name="client_ip" value="${rsi_config_dict['client_ip']}" />
-<xacro:property name="client_port" value="${rsi_config_dict['client_port']}" />
-<!-- Read additional arguments  -->
-<xacro:arg name="use_fake_hardware" default="false" />
-<xacro:kuka_kr210_r3100-2_robot prefix=""
-                  client_ip="${client_ip}"
-                  client_port="${client_port}"
-                  use_fake_hardware="$(arg use_fake_hardware)"/>
+  <!-- Import urdf file  -->
+  <xacro:include filename="$(find kuka_quantec_support)/urdf/kr210_r3100-2_macro.xacro"/>
+  <!-- Read additional arguments  -->
+  <xacro:arg name="use_fake_hardware" default="false" />
+  <xacro:kuka_kr210_r3100-2_robot prefix="" use_fake_hardware="$(arg use_fake_hardware)"/>
 </robot>

File: kuka_quantec_support/urdf/kr210_r3100-2_macro.xacro (robot description, xacro)
@@ -3,11 +3,9 @@
   <xacro:include filename="$(find kuka_quantec_support)/urdf/kr_quantec_ros2_control.xacro" />
   <xacro:include filename="$(find kuka_quantec_support)/urdf/kr_quantec_transmission.xacro" />
-  <xacro:macro name="kuka_kr210_r3100-2_robot" params="prefix client_ip client_port use_fake_hardware">
+  <xacro:macro name="kuka_kr210_r3100-2_robot" params="prefix use_fake_hardware">
     <!-- ros2 control instance -->
     <xacro:kuka_quantec_ros2_control
     name="kr210_r3100-2"
     prefix="${prefix}"
-    client_ip="${client_ip}"
-    client_port="${client_port}"
     use_fake_hardware="${use_fake_hardware}" />
     <link name="${prefix}base_link"/>

File: kuka_quantec_support/urdf/kr_quantec_ros2_control.xacro (robot description, xacro)
@@ -1,5 +1,5 @@
 <?xml version="1.0" encoding="UTF-8"?>
 <robot xmlns:xacro="http://www.ros.org/wiki/xacro">
-  <xacro:macro name="kuka_quantec_ros2_control" params="name prefix client_ip client_port use_fake_hardware:=false">
+  <xacro:macro name="kuka_quantec_ros2_control" params="name prefix use_fake_hardware:=false">
     <ros2_control name="${name}" type="system">
       <hardware>
@@ -10,4 +10,9 @@
         </xacro:if>
         <xacro:unless value="${use_fake_hardware}">
+          <!-- Read parameters from rsi_config  -->
+          <xacro:property name="rsi_config" value="$(find kuka_rsi_hw_interface)/config/rsi_config.yaml" />
+          <xacro:property name="rsi_config_dict" value="${xacro.load_yaml(rsi_config)}"/>
+          <xacro:property name="client_ip" value="${rsi_config_dict['client_ip']}" />
+          <xacro:property name="client_port" value="${rsi_config_dict['client_port']}" />
           <plugin>kuka_rsi_hw_interface::KukaRSIHardwareInterface</plugin>
           <param name="client_ip">${client_ip}</param>
