Commit message: adapt to driver changes

File: kuka_agilus_support/urdf/kr_agilus_ros2_control.xacro (robot description, xacro)
@@ -11,9 +11,9 @@
         <xacro:unless value="${use_fake_hardware}">
           <!-- Read parameters from rsi_config  -->
-          <xacro:property name="rsi_config" value="$(find kuka_rsi_hw_interface)/config/rsi_config.yaml" />
+          <xacro:property name="rsi_config" value="$(find kuka_kss_rsi_driver)/config/rsi_config.yaml" />
           <xacro:property name="rsi_config_dict" value="${xacro.load_yaml(rsi_config)}"/>
           <xacro:property name="client_ip" value="${rsi_config_dict['client_ip']}" />
           <xacro:property name="client_port" value="${rsi_config_dict['client_port']}" />
-          <plugin>kuka_rsi_hw_interface::KukaRSIHardwareInterface</plugin>
+          <plugin>kuka_kss_rsi_driver::KukaRSIHardwareInterface</plugin>
           <param name="client_ip">${client_ip}</param>
           <param name="client_port">${client_port}</param>

File: kuka_cybertech_support/urdf/kr_cybertech_ros2_control.xacro (robot description, xacro)
@@ -11,9 +11,9 @@
         <xacro:unless value="${use_fake_hardware}">
           <!-- Read parameters from rsi_config  -->
-          <xacro:property name="rsi_config" value="$(find kuka_rsi_hw_interface)/config/rsi_config.yaml" />
+          <xacro:property name="rsi_config" value="$(find kuka_kss_rsi_driver)/config/rsi_config.yaml" />
           <xacro:property name="rsi_config_dict" value="${xacro.load_yaml(rsi_config)}"/>
           <xacro:property name="client_ip" value="${rsi_config_dict['client_ip']}" />
           <xacro:property name="client_port" value="${rsi_config_dict['client_port']}" />
-          <plugin>kuka_rsi_hw_interface::KukaRSIHardwareInterface</plugin>
+          <plugin>kuka_kss_rsi_driver::KukaRSIHardwareInterface</plugin>
           <param name="client_ip">${client_ip}</param>
           <param name="client_port">${client_port}</param>

File: kuka_lbr_iisy_support/urdf/lbr_iisy_ros2_control.xacro (robot description, xacro)
@@ -11,5 +11,5 @@
         <xacro:unless value="${use_fake_hardware}">
           <!-- Read parameters from eci_config  -->
-          <xacro:property name="eci_config" value="$(find kuka_rox_hw_interface)/config/eci_config.yaml" />
+          <xacro:property name="eci_config" value="$(find kuka_iiqka_eac_driver)/config/eci_config.yaml" />
           <xacro:property name="eci_config_dict" value="${xacro.load_yaml(eci_config)}"/>
           <xacro:property name="control_mode" value="${eci_config_dict['robot_manager']['ros__parameters']['control_mode']}" />
@@ -17,5 +17,5 @@
           <xacro:property name="controller_ip" value="${eci_config_dict['robot_manager']['ros__parameters']['controller_ip']}" />
           <!-- Read QoS profile parameters  -->
-          <xacro:property name="qos_config" value="$(find kuka_rox_hw_interface)/config/qos_profiles.yaml" />
+          <xacro:property name="qos_config" value="$(find kuka_iiqka_eac_driver)/config/qos_profiles.yaml" />
           <xacro:property name="qos_config_dict" value="${xacro.load_yaml(qos_config)}"/>
           <xacro:property name="consequent_lost_packets" value="${qos_config_dict['rt_packet_loss_profile']['consequent_lost_packets']}" />

File: kuka_lbr_iiwa_support/urdf/lbr_iiwa_ros2_control.xacro (robot description, xacro)
@@ -10,5 +10,5 @@
         </xacro:if>
         <xacro:unless value="${use_fake_hardware}">
-          <plugin>kuka_sunrise::KUKAFRIHardwareInterface</plugin>
+          <plugin>kuka_sunrise_fri_driver::KUKAFRIHardwareInterface</plugin>
         </xacro:unless>
       </hardware>
@@ -66,5 +66,5 @@
       <xacro:unless value="${use_fake_hardware}">
         <xacro:if value="${io_access}">
-          <xacro:include filename="$(find kuka_sunrise)/config/gpio_config.xacro" />
+          <xacro:include filename="$(find kuka_sunrise_fri_driver)/config/gpio_config.xacro" />
           <xacro:fri_gpio_config/>
         </xacro:if>

File: kuka_quantec_support/urdf/kr_quantec_ros2_control.xacro (robot description, xacro)
@@ -11,9 +11,9 @@
         <xacro:unless value="${use_fake_hardware}">
           <!-- Read parameters from rsi_config  -->
-          <xacro:property name="rsi_config" value="$(find kuka_rsi_hw_interface)/config/rsi_config.yaml" />
+          <xacro:property name="rsi_config" value="$(find kuka_kss_rsi_driver)/config/rsi_config.yaml" />
           <xacro:property name="rsi_config_dict" value="${xacro.load_yaml(rsi_config)}"/>
           <xacro:property name="client_ip" value="${rsi_config_dict['client_ip']}" />
           <xacro:property name="client_port" value="${rsi_config_dict['client_port']}" />
-          <plugin>kuka_rsi_hw_interface::KukaRSIHardwareInterface</plugin>
+          <plugin>kuka_kss_rsi_driver::KukaRSIHardwareInterface</plugin>
           <param name="client_ip">${client_ip}</param>
           <param name="client_port">${client_port}</param>

Commit message: fix driver config files

File: kuka_agilus_support/urdf/kr_agilus_ros2_control.xacro (robot description, xacro)
@@ -11,5 +11,5 @@
         <xacro:unless value="${use_fake_hardware}">
           <!-- Read parameters from rsi_config  -->
-          <xacro:property name="rsi_config" value="$(find kuka_kss_rsi_driver)/config/rsi_config.yaml" />
+          <xacro:property name="rsi_config" value="$(find kuka_kss_rsi_driver)/config/driver_config.yaml" />
           <xacro:property name="rsi_config_dict" value="${xacro.load_yaml(rsi_config)}"/>
           <xacro:property name="client_ip" value="${rsi_config_dict['client_ip']}" />

File: kuka_cybertech_support/urdf/kr_cybertech_ros2_control.xacro (robot description, xacro)
@@ -11,5 +11,5 @@
         <xacro:unless value="${use_fake_hardware}">
           <!-- Read parameters from rsi_config  -->
-          <xacro:property name="rsi_config" value="$(find kuka_kss_rsi_driver)/config/rsi_config.yaml" />
+          <xacro:property name="rsi_config" value="$(find kuka_kss_rsi_driver)/config/driver_config.yaml" />
           <xacro:property name="rsi_config_dict" value="${xacro.load_yaml(rsi_config)}"/>
           <xacro:property name="client_ip" value="${rsi_config_dict['client_ip']}" />

File: kuka_lbr_iisy_support/urdf/lbr_iisy_ros2_control.xacro (robot description, xacro)
@@ -10,10 +10,10 @@
         </xacro:if>
         <xacro:unless value="${use_fake_hardware}">
-          <!-- Read parameters from eci_config  -->
-          <xacro:property name="eci_config" value="$(find kuka_iiqka_eac_driver)/config/eci_config.yaml" />
-          <xacro:property name="eci_config_dict" value="${xacro.load_yaml(eci_config)}"/>
-          <xacro:property name="control_mode" value="${eci_config_dict['robot_manager']['ros__parameters']['control_mode']}" />
-          <xacro:property name="client_ip" value="${eci_config_dict['robot_manager']['ros__parameters']['client_ip']}" />
-          <xacro:property name="controller_ip" value="${eci_config_dict['robot_manager']['ros__parameters']['controller_ip']}" />
+          <!-- Read parameters from driver_config  -->
+          <xacro:property name="driver_config" value="$(find kuka_iiqka_eac_driver)/config/driver_config.yaml" />
+          <xacro:property name="driver_config_dict" value="${xacro.load_yaml(driver_config)}"/>
+          <xacro:property name="control_mode" value="${driver_config_dict['robot_manager']['ros__parameters']['control_mode']}" />
+          <xacro:property name="client_ip" value="${driver_config_dict['robot_manager']['ros__parameters']['client_ip']}" />
+          <xacro:property name="controller_ip" value="${driver_config_dict['robot_manager']['ros__parameters']['controller_ip']}" />
           <!-- Read QoS profile parameters  -->
           <xacro:property name="qos_config" value="$(find kuka_iiqka_eac_driver)/config/qos_profiles.yaml" />

File: kuka_quantec_support/urdf/kr_quantec_ros2_control.xacro (robot description, xacro)
@@ -11,5 +11,5 @@
         <xacro:unless value="${use_fake_hardware}">
           <!-- Read parameters from rsi_config  -->
-          <xacro:property name="rsi_config" value="$(find kuka_kss_rsi_driver)/config/rsi_config.yaml" />
+          <xacro:property name="rsi_config" value="$(find kuka_kss_rsi_driver)/config/driver_config.yaml" />
           <xacro:property name="rsi_config_dict" value="${xacro.load_yaml(rsi_config)}"/>
           <xacro:property name="client_ip" value="${rsi_config_dict['client_ip']}" />

Commit message: remove duplicate default

File: kuka_agilus_support/urdf/kr_agilus_ros2_control.xacro (robot description, xacro)
@@ -1,5 +1,5 @@
 <?xml version="1.0" encoding="UTF-8"?>
 <robot xmlns:xacro="http://www.ros.org/wiki/xacro">
-  <xacro:macro name="kuka_agilus_ros2_control" params="name client_ip client_port prefix use_fake_hardware:=false">
+  <xacro:macro name="kuka_agilus_ros2_control" params="name client_ip client_port prefix use_fake_hardware">
     <ros2_control name="${name}" type="system">
       <hardware>

File: kuka_cybertech_support/urdf/kr_cybertech_ros2_control.xacro (robot description, xacro)
@@ -1,5 +1,5 @@
 <?xml version="1.0" encoding="UTF-8"?>
 <robot xmlns:xacro="http://www.ros.org/wiki/xacro">
-  <xacro:macro name="kuka_cybertech_ros2_control" params="name client_ip client_port prefix use_fake_hardware:=false">
+  <xacro:macro name="kuka_cybertech_ros2_control" params="name client_ip client_port prefix use_fake_hardware">
     <ros2_control name="${name}" type="system">
       <hardware>

File: kuka_lbr_iiwa_support/urdf/lbr_iiwa_ros2_control.xacro (robot description, xacro)
@@ -1,5 +1,5 @@
 <?xml version="1.0" encoding="UTF-8"?>
 <robot xmlns:xacro="http://www.ros.org/wiki/xacro">
-  <xacro:macro name="kuka_lbr_iiwa_ros2_control" params="name prefix io_access use_fake_hardware:=false">
+  <xacro:macro name="kuka_lbr_iiwa_ros2_control" params="name prefix io_access use_fake_hardware">
     <ros2_control name="${name}" type="system">
       <hardware>

File: kuka_quantec_support/urdf/kr_quantec_ros2_control.xacro (robot description, xacro)
@@ -1,5 +1,5 @@
 <?xml version="1.0" encoding="UTF-8"?>
 <robot xmlns:xacro="http://www.ros.org/wiki/xacro">
-  <xacro:macro name="kuka_quantec_ros2_control" params="name client_ip client_port prefix use_fake_hardware:=false">
+  <xacro:macro name="kuka_quantec_ros2_control" params="name client_ip client_port prefix use_fake_hardware">
     <ros2_control name="${name}" type="system">
       <hardware>
