Commit message: include ros2_control in urdf

File: kuka_agilus_support/urdf/kr6_r700_sixx_macro.xacro (robot description, xacro)
@@ -3,5 +3,14 @@
   <xacro:include filename="$(find kuka_resources)/urdf/common_constants.xacro"/>
   <xacro:include filename="$(find kuka_resources)/urdf/common_materials.xacro"/>
+  <xacro:include filename="$(find kuka_agilus_support)/urdf/kr_agilus_ros2_control.xacro" />
+  <xacro:include filename="$(find kuka_agilus_support)/urdf/kr_agilus_transmission.xacro" />
   <xacro:macro name="kuka_kr6_r700_sixx_robot" params="prefix client_ip client_port use_fake_hardware">
+    <!-- ros2 control instance -->
+    <xacro:kuka_agilus_ros2_control
+    name="KR6R700sixx"
+    prefix="${prefix}"
+    client_ip="${client_ip}"
+    client_port="${client_port}"
+    use_fake_hardware="${use_fake_hardware}" />
     <link name="${prefix}base_link">
       <visual>

File: kuka_agilus_support/urdf/kr6_r900_sixx_macro.xacro (robot description, xacro)
@@ -3,5 +3,14 @@
   <xacro:include filename="$(find kuka_resources)/urdf/common_constants.xacro"/>
   <xacro:include filename="$(find kuka_resources)/urdf/common_materials.xacro"/>
-  <xacro:macro name="kuka_kr6_r900_sixx_robot" params="prefix">
+  <xacro:include filename="$(find kuka_agilus_support)/urdf/kr_agilus_ros2_control.xacro" />
+  <xacro:include filename="$(find kuka_agilus_support)/urdf/kr_agilus_transmission.xacro" />
+  <xacro:macro name="kuka_kr6_r900_sixx_robot" params="prefix client_ip client_port use_fake_hardware">
+    <!-- ros2 control instance -->
+    <xacro:kuka_agilus_ros2_control
+    name="KR6R900sixx"
+    prefix="${prefix}"
+    client_ip="${client_ip}"
+    client_port="${client_port}"
+    use_fake_hardware="${use_fake_hardware}" />
     <link name="${prefix}base_link">
       <visual>

File: kuka_agilus_support/urdf/kr_agilus_ros2_control.xacro (robot description, xacro)
@@ -1,5 +1,5 @@
 <?xml version="1.0" encoding="UTF-8"?>
 <robot xmlns:xacro="http://www.ros.org/wiki/xacro">
-  <xacro:macro name="kuka_lbr_iisy_ros2_control" params="name prefix client_ip client_port use_fake_hardware:=false">
+  <xacro:macro name="kuka_agilus_ros2_control" params="name prefix client_ip client_port use_fake_hardware:=false">
     <ros2_control name="${name}" type="system">
       <hardware>

Commit message: base link inertia +srdf robot name fix

File: kuka_agilus_support/urdf/kr6_r700_sixx_macro.xacro (robot description, xacro)
@@ -13,5 +13,6 @@
     client_port="${client_port}"
     use_fake_hardware="${use_fake_hardware}" />
-    <link name="${prefix}base_link">
+    <link name="${prefix}base_link"/>
+    <link name="${prefix}base_link_inertia">
       <visual>
         <origin xyz="0 0 0" rpy="0 0 0" />
@@ -120,7 +121,12 @@
     <!-- Following REP199, this frame shall be use to attach EEF or other equipment -->
     <link name="${prefix}flange" />
+    <joint name="${prefix}base_link-base_link_inertia" type="fixed">
+      <parent link="${prefix}base_link" />
+      <child link="${prefix}base_link_inertia" />
+      <origin xyz="0 0 0" rpy="0 0 0" />
+    </joint>
     <joint name="${prefix}joint_a1" type="revolute">
       <origin xyz="0 0 0.4" rpy="0 0 0"/>
-      <parent link="${prefix}base_link"/>
+      <parent link="${prefix}base_link_inertia"/>
       <child link="${prefix}link_1"/>
       <axis xyz="0 0 -1"/>

File: kuka_agilus_support/urdf/kr6_r900_sixx_macro.xacro (robot description, xacro)
@@ -13,5 +13,6 @@
     client_port="${client_port}"
     use_fake_hardware="${use_fake_hardware}" />
-    <link name="${prefix}base_link">
+    <link name="${prefix}base_link"/>
+    <link name="${prefix}base_link_inertia">
       <visual>
         <origin xyz="0 0 0" rpy="0 0 0"/>
@@ -120,7 +121,12 @@
     <!-- Following REP199, this frame shall be use to attach EEF or other equipment -->
     <link name="${prefix}flange" />
+    <joint name="${prefix}base_link-base_link_inertia" type="fixed">
+      <parent link="${prefix}base_link" />
+      <child link="${prefix}base_link_inertia" />
+      <origin xyz="0 0 0" rpy="0 0 0" />
+    </joint>
     <joint name="${prefix}joint_a1" type="revolute">
       <origin xyz="0 0 0.400" rpy="0 0 0"/>
-      <parent link="${prefix}base_link"/>
+      <parent link="${prefix}base_link_inertia"/>
       <child link="${prefix}link_1"/>
       <axis xyz="0 0 -1"/>

File: kuka_kr_moveit_config/srdf/kr_arm.srdf.xacro (robot description, xacro)
@@ -4,7 +4,7 @@
     A URDF file must exist for this robot as well, where the joints and the links that are referenced are defined
 -->
-<!--TODO(Svastits): add an argument for the robot name instead of kr, as srdf model parsers logs an error now-->
-<robot xmlns:xacro="http://www.ros.org/wiki/xacro" name="kr">
+<robot xmlns:xacro="http://www.ros.org/wiki/xacro" name="$(arg robot_name)">
+  <xacro:arg name="prefix" default=""/>
   <xacro:include filename="kr_arm_macro.xacro" />
-  <xacro:kuka_kr_arm prefix=""/>
+  <xacro:kuka_kr_arm prefix="$(arg prefix)"/>
 </robot>
