Commit message: joint_ai-> joint_i

File: kuka_agilus_support/urdf/kr6_r700_sixx_macro.xacro (robot description, xacro)
@@ -124,5 +124,5 @@
       <origin xyz="0 0 0" rpy="0 0 0" />
     </joint>
-    <joint name="${prefix}joint_a1" type="revolute">
+    <joint name="${prefix}joint_1" type="revolute">
       <origin xyz="0 0 0.4" rpy="0 0 0"/>
       <parent link="${prefix}base_link_inertia"/>
@@ -131,5 +131,5 @@
       <limit lower="${radians(-170)}" upper="${radians(170)}" effort="0" velocity="${radians(360)}"/>
     </joint>
-    <joint name="${prefix}joint_a2" type="revolute">
+    <joint name="${prefix}joint_2" type="revolute">
       <origin xyz="0.025 0 0" rpy="0 0 0"/>
       <parent link="${prefix}link_1"/>
@@ -138,5 +138,5 @@
       <limit lower="${radians(-190)}" upper="${radians(45)}" effort="0" velocity="${radians(300)}"/>
     </joint>
-    <joint name="${prefix}joint_a3" type="revolute">
+    <joint name="${prefix}joint_3" type="revolute">
       <origin xyz="0.315 0 0" rpy="0 0 0"/>
       <parent link="${prefix}link_2"/>
@@ -145,5 +145,5 @@
       <limit lower="${radians(-120)}" upper="${radians(156)}" effort="0" velocity="${radians(360)}"/>
     </joint>
-    <joint name="${prefix}joint_a4" type="revolute">
+    <joint name="${prefix}joint_4" type="revolute">
       <origin xyz="0 0 0.035" rpy="0 0 0"/>
       <parent link="${prefix}link_3"/>
@@ -152,5 +152,5 @@
       <limit lower="${radians(-185)}" upper="${radians(185)}" effort="0" velocity="${radians(381)}"/>
     </joint>
-    <joint name="${prefix}joint_a5" type="revolute">
+    <joint name="${prefix}joint_5" type="revolute">
       <origin xyz="0.365 0 0" rpy="0 0 0"/>
       <parent link="${prefix}link_4"/>
@@ -159,5 +159,5 @@
       <limit lower="${radians(-120)}" upper="${radians(120)}" effort="0" velocity="${radians(388)}"/>
     </joint>
-    <joint name="${prefix}joint_a6" type="revolute">
+    <joint name="${prefix}joint_6" type="revolute">
       <origin xyz="0.080 0 0" rpy="0 0 0"/>
       <parent link="${prefix}link_5"/>
@@ -166,5 +166,5 @@
       <limit lower="${radians(-350)}" upper="${radians(350)}" effort="0" velocity="${radians(615)}"/>
     </joint>
-    <joint name="${prefix}joint_a6-flange" type="fixed">
+    <joint name="${prefix}joint_6-flange" type="fixed">
       <parent link="${prefix}link_6"/>
       <child link="${prefix}flange"/>

File: kuka_agilus_support/urdf/kr_agilus_ros2_control.xacro (robot description, xacro)
@@ -20,5 +20,5 @@
         </xacro:unless>
       </hardware>
-      <joint name="${prefix}joint_a1">
+      <joint name="${prefix}joint_1">
         <command_interface name="position"/>
       <state_interface name="position">
@@ -26,5 +26,5 @@
       </state_interface>
       </joint>
-      <joint name="${prefix}joint_a2">
+      <joint name="${prefix}joint_2">
         <command_interface name="position"/>
       <state_interface name="position">
@@ -32,5 +32,5 @@
       </state_interface>
       </joint>
-      <joint name="${prefix}joint_a3">
+      <joint name="${prefix}joint_3">
         <command_interface name="position"/>
       <state_interface name="position">
@@ -38,5 +38,5 @@
       </state_interface>
       </joint>
-      <joint name="${prefix}joint_a4">
+      <joint name="${prefix}joint_4">
         <command_interface name="position"/>
       <state_interface name="position">
@@ -44,5 +44,5 @@
       </state_interface>
       </joint>
-      <joint name="${prefix}joint_a5">
+      <joint name="${prefix}joint_5">
         <command_interface name="position"/>
       <state_interface name="position">
@@ -50,5 +50,5 @@
       </state_interface>
       </joint>
-      <joint name="${prefix}joint_a6">
+      <joint name="${prefix}joint_6">
         <command_interface name="position"/>
       <state_interface name="position">

File: kuka_cybertech_support/urdf/kr16_r2010_2_macro.xacro (robot description, xacro)
@@ -148,5 +148,5 @@
       <origin xyz="0 0 0" rpy="0 0 0" />
     </joint>
-    <joint name="${prefix}joint_a1" type="revolute">
+    <joint name="${prefix}joint_1" type="revolute">
       <axis xyz="0.0 0.0 1.0"/>
       <child link="${prefix}link_1"/>
@@ -155,5 +155,5 @@
       <parent link="${prefix}base_link_inertia"/>
     </joint>
-    <joint name="${prefix}joint_a2" type="revolute">
+    <joint name="${prefix}joint_2" type="revolute">
       <axis xyz="0.0 0.0 1.0"/>
       <child link="${prefix}link_2"/>
@@ -162,5 +162,5 @@
       <parent link="${prefix}link_1"/>
     </joint>
-    <joint name="${prefix}joint_a3" type="revolute">
+    <joint name="${prefix}joint_3" type="revolute">
       <axis xyz="0.0 0.0 1.0"/>
       <child link="${prefix}link_3"/>
@@ -169,5 +169,5 @@
       <parent link="${prefix}link_2"/>
     </joint>
-    <joint name="${prefix}joint_a4" type="revolute">
+    <joint name="${prefix}joint_4" type="revolute">
       <axis xyz="0.0 0.0 1.0"/>
       <child link="${prefix}link_4"/>
@@ -176,5 +176,5 @@
       <parent link="${prefix}link_3"/>
     </joint>
-    <joint name="${prefix}joint_a5" type="revolute">
+    <joint name="${prefix}joint_5" type="revolute">
       <axis xyz="0.0 0.0 1.0"/>
       <child link="${prefix}link_5"/>
@@ -183,5 +183,5 @@
       <parent link="${prefix}link_4"/>
     </joint>
-    <joint name="${prefix}joint_a6" type="revolute">
+    <joint name="${prefix}joint_6" type="revolute">
       <axis xyz="0.0 0.0 1.0"/>
       <child link="${prefix}link_6"/>

File: kuka_cybertech_support/urdf/kr_cybertech_ros2_control.xacro (robot description, xacro)
@@ -20,5 +20,5 @@
         </xacro:unless>
       </hardware>
-      <joint name="${prefix}joint_a1">
+      <joint name="${prefix}joint_1">
         <command_interface name="position"/>
       <state_interface name="position">
@@ -26,5 +26,5 @@
       </state_interface>
       </joint>
-      <joint name="${prefix}joint_a2">
+      <joint name="${prefix}joint_2">
         <command_interface name="position"/>
       <state_interface name="position">
@@ -32,5 +32,5 @@
       </state_interface>
       </joint>
-      <joint name="${prefix}joint_a3">
+      <joint name="${prefix}joint_3">
         <command_interface name="position"/>
       <state_interface name="position">
@@ -38,5 +38,5 @@
       </state_interface>
       </joint>
-      <joint name="${prefix}joint_a4">
+      <joint name="${prefix}joint_4">
         <command_interface name="position"/>
       <state_interface name="position">
@@ -44,5 +44,5 @@
       </state_interface>
       </joint>
-      <joint name="${prefix}joint_a5">
+      <joint name="${prefix}joint_5">
         <command_interface name="position"/>
       <state_interface name="position">
@@ -50,5 +50,5 @@
       </state_interface>
       </joint>
-      <joint name="${prefix}joint_a6">
+      <joint name="${prefix}joint_6">
         <command_interface name="position"/>
       <state_interface name="position">

File: kuka_lbr_iisy_support/urdf/lbr_iisy11_r1300_macro.xacro (robot description, xacro)
@@ -160,5 +160,5 @@
       <origin xyz="0 0 0" rpy="0 0 0" />
     </joint>
-    <joint name="${prefix}joint_a1" type="revolute">
+    <joint name="${prefix}joint_1" type="revolute">
       <axis xyz="0.0 0.0 1.0" />
       <child link="${prefix}link_1" />
@@ -167,5 +167,5 @@
       <parent link="${prefix}base_link_inertia" />
     </joint>
-    <joint name="${prefix}joint_a2" type="revolute">
+    <joint name="${prefix}joint_2" type="revolute">
       <axis xyz="0.0 0.0 1.0" />
       <child link="${prefix}link_2" />
@@ -174,5 +174,5 @@
       <parent link="${prefix}link_1" />
     </joint>
-    <joint name="${prefix}joint_a3" type="revolute">
+    <joint name="${prefix}joint_3" type="revolute">
       <axis xyz="0.0 0.0 1.0" />
       <child link="${prefix}link_3" />
@@ -181,5 +181,5 @@
       <parent link="${prefix}link_2" />
     </joint>
-    <joint name="${prefix}joint_a4" type="revolute">
+    <joint name="${prefix}joint_4" type="revolute">
       <axis xyz="0.0 0.0 1.0" />
       <child link="${prefix}link_4" />
@@ -188,5 +188,5 @@
       <parent link="${prefix}link_3" />
     </joint>
-    <joint name="${prefix}joint_a5" type="revolute">
+    <joint name="${prefix}joint_5" type="revolute">
       <axis xyz="0.0 0.0 1.0" />
       <child link="${prefix}link_5" />
@@ -195,5 +195,5 @@
       <parent link="${prefix}link_4" />
     </joint>
-    <joint name="${prefix}joint_a6" type="revolute">
+    <joint name="${prefix}joint_6" type="revolute">
       <axis xyz="0.0 0.0 1.0" />
       <child link="${prefix}link_6" />

File: kuka_lbr_iisy_support/urdf/lbr_iisy15_r930_macro.xacro (robot description, xacro)
@@ -160,5 +160,5 @@
       <origin xyz="0 0 0" rpy="0 0 0" />
     </joint>
-    <joint name="${prefix}joint_a1" type="revolute">
+    <joint name="${prefix}joint_1" type="revolute">
       <axis xyz="0.0 0.0 1.0" />
       <child link="${prefix}link_1" />
@@ -167,5 +167,5 @@
       <parent link="${prefix}base_link_inertia" />
     </joint>
-    <joint name="${prefix}joint_a2" type="revolute">
+    <joint name="${prefix}joint_2" type="revolute">
       <axis xyz="0.0 0.0 1.0" />
       <child link="${prefix}link_2" />
@@ -174,5 +174,5 @@
       <parent link="${prefix}link_1" />
     </joint>
-    <joint name="${prefix}joint_a3" type="revolute">
+    <joint name="${prefix}joint_3" type="revolute">
       <axis xyz="0.0 0.0 1.0" />
       <child link="${prefix}link_3" />
@@ -181,5 +181,5 @@
       <parent link="${prefix}link_2" />
     </joint>
-    <joint name="${prefix}joint_a4" type="revolute">
+    <joint name="${prefix}joint_4" type="revolute">
       <axis xyz="0.0 0.0 1.0" />
       <child link="${prefix}link_4" />
@@ -188,5 +188,5 @@
       <parent link="${prefix}link_3" />
     </joint>
-    <joint name="${prefix}joint_a5" type="revolute">
+    <joint name="${prefix}joint_5" type="revolute">
       <axis xyz="0.0 0.0 1.0" />
       <child link="${prefix}link_5" />
@@ -195,5 +195,5 @@
       <parent link="${prefix}link_4" />
     </joint>
-    <joint name="${prefix}joint_a6" type="revolute">
+    <joint name="${prefix}joint_6" type="revolute">
       <axis xyz="0.0 0.0 1.0" />
       <child link="${prefix}link_6" />

File: kuka_lbr_iisy_support/urdf/lbr_iisy3_r760_macro.xacro (robot description, xacro)
@@ -160,5 +160,5 @@
       <origin xyz="0 0 0" rpy="0 0 0" />
     </joint>
-    <joint name="${prefix}joint_a1" type="revolute">
+    <joint name="${prefix}joint_1" type="revolute">
       <axis xyz="0.0 0.0 -1.0" />
       <child link="${prefix}link_1" />
@@ -167,5 +167,5 @@
       <parent link="${prefix}base_link_inertia" />
     </joint>
-    <joint name="${prefix}joint_a2" type="revolute">
+    <joint name="${prefix}joint_2" type="revolute">
       <axis xyz="0.0 0.0 1.0" />
       <child link="${prefix}link_2" />
@@ -174,5 +174,5 @@
       <parent link="${prefix}link_1" />
     </joint>
-    <joint name="${prefix}joint_a3" type="revolute">
+    <joint name="${prefix}joint_3" type="revolute">
       <axis xyz="0.0 0.0 1.0" />
       <child link="${prefix}link_3" />
@@ -181,5 +181,5 @@
       <parent link="${prefix}link_2" />
     </joint>
-    <joint name="${prefix}joint_a4" type="revolute">
+    <joint name="${prefix}joint_4" type="revolute">
       <axis xyz="0.0 0.0 1.0" />
       <child link="${prefix}link_4" />
@@ -188,5 +188,5 @@
       <parent link="${prefix}link_3" />
     </joint>
-    <joint name="${prefix}joint_a5" type="revolute">
+    <joint name="${prefix}joint_5" type="revolute">
       <axis xyz="0.0 0.0 1.0" />
       <child link="${prefix}link_5" />
@@ -195,5 +195,5 @@
       <parent link="${prefix}link_4" />
     </joint>
-    <joint name="${prefix}joint_a6" type="revolute">
+    <joint name="${prefix}joint_6" type="revolute">
       <axis xyz="0.0 0.0 1.0" />
       <child link="${prefix}link_6" />

File: kuka_lbr_iisy_support/urdf/lbr_iisy_ros2_control.xacro (robot description, xacro)
@@ -32,5 +32,5 @@
       </hardware>
       <!-- define joints and command/state interfaces for each joint -->
-      <joint name="${prefix}joint_a1">
+      <joint name="${prefix}joint_1">
         <command_interface name="position"/>
         <command_interface name="stiffness"/>
@@ -40,5 +40,5 @@
         <state_interface name="effort"/>
       </joint>
-      <joint name="${prefix}joint_a2">
+      <joint name="${prefix}joint_2">
         <command_interface name="position"/>
         <command_interface name="stiffness"/>
@@ -48,5 +48,5 @@
         <state_interface name="effort"/>
       </joint>
-      <joint name="${prefix}joint_a3">
+      <joint name="${prefix}joint_3">
         <command_interface name="position"/>
         <command_interface name="stiffness"/>
@@ -56,5 +56,5 @@
         <state_interface name="effort"/>
       </joint>
-      <joint name="${prefix}joint_a4">
+      <joint name="${prefix}joint_4">
         <command_interface name="position"/>
         <command_interface name="stiffness"/>
@@ -64,5 +64,5 @@
         <state_interface name="effort"/>
       </joint>
-      <joint name="${prefix}joint_a5">
+      <joint name="${prefix}joint_5">
         <command_interface name="position"/>
         <command_interface name="stiffness"/>
@@ -72,5 +72,5 @@
         <state_interface name="effort"/>
       </joint>
-      <joint name="${prefix}joint_a6">
+      <joint name="${prefix}joint_6">
         <command_interface name="position"/>
         <command_interface name="stiffness"/>

File: kuka_lbr_iiwa_support/urdf/lbr_iiwa_ros2_control.xacro (robot description, xacro)
@@ -14,5 +14,5 @@
       </hardware>
       <!-- define joints and command/state interfaces for each joint -->
-      <joint name="${prefix}joint_a1">
+      <joint name="${prefix}joint_1">
         <command_interface name="position"/>
         <command_interface name="effort"/>
@@ -21,5 +21,5 @@
         <state_interface name="external_torque"/>
       </joint>
-      <joint name="${prefix}joint_a2">
+      <joint name="${prefix}joint_2">
         <command_interface name="position"/>
         <command_interface name="effort"/>
@@ -28,5 +28,5 @@
         <state_interface name="external_torque"/>
       </joint>
-      <joint name="${prefix}joint_a3">
+      <joint name="${prefix}joint_3">
         <command_interface name="position"/>
         <command_interface name="effort"/>
@@ -35,5 +35,5 @@
         <state_interface name="external_torque"/>
       </joint>
-      <joint name="${prefix}joint_a4">
+      <joint name="${prefix}joint_4">
         <command_interface name="position"/>
         <command_interface name="effort"/>
@@ -42,5 +42,5 @@
         <state_interface name="external_torque"/>
       </joint>
-      <joint name="${prefix}joint_a5">
+      <joint name="${prefix}joint_5">
         <command_interface name="position"/>
         <command_interface name="effort"/>
@@ -49,5 +49,5 @@
         <state_interface name="external_torque"/>
       </joint>
-      <joint name="${prefix}joint_a6">
+      <joint name="${prefix}joint_6">
         <command_interface name="position"/>
         <command_interface name="effort"/>
@@ -56,5 +56,5 @@
         <state_interface name="external_torque"/>
       </joint>
-      <joint name="${prefix}joint_a7">
+      <joint name="${prefix}joint_7">
         <command_interface name="position"/>
         <command_interface name="effort"/>

File: kuka_quantec_support/urdf/kr210_r2700_2_macro.xacro (robot description, xacro)
@@ -148,5 +148,5 @@
       <origin xyz="0 0 0" rpy="0 0 0" />
     </joint>
-    <joint name="${prefix}joint_a1" type="revolute">
+    <joint name="${prefix}joint_1" type="revolute">
       <axis xyz="0.0 0.0 1.0"/>
       <child link="${prefix}link_1"/>
@@ -155,5 +155,5 @@
       <parent link="${prefix}base_link_inertia"/>
     </joint>
-    <joint name="${prefix}joint_a2" type="revolute">
+    <joint name="${prefix}joint_2" type="revolute">
       <axis xyz="0.0 0.0 1.0"/>
       <child link="${prefix}link_2"/>
@@ -162,5 +162,5 @@
       <parent link="${prefix}link_1"/>
     </joint>
-    <joint name="${prefix}joint_a3" type="revolute">
+    <joint name="${prefix}joint_3" type="revolute">
       <axis xyz="0.0 0.0 1.0"/>
       <child link="${prefix}link_3"/>
@@ -169,5 +169,5 @@
       <parent link="${prefix}link_2"/>
     </joint>
-    <joint name="${prefix}joint_a4" type="revolute">
+    <joint name="${prefix}joint_4" type="revolute">
       <axis xyz="0.0 0.0 1.0"/>
       <child link="${prefix}link_4"/>
@@ -176,5 +176,5 @@
       <parent link="${prefix}link_3"/>
     </joint>
-    <joint name="${prefix}joint_a5" type="revolute">
+    <joint name="${prefix}joint_5" type="revolute">
       <axis xyz="0.0 0.0 1.0"/>
       <child link="${prefix}link_5"/>
@@ -183,5 +183,5 @@
       <parent link="${prefix}link_4"/>
     </joint>
-    <joint name="${prefix}joint_a6" type="revolute">
+    <joint name="${prefix}joint_6" type="revolute">
       <axis xyz="0.0 0.0 1.0"/>
       <child link="${prefix}link_6"/>

File: kuka_quantec_support/urdf/kr210_r3100_2_macro.xacro (robot description, xacro)
@@ -148,5 +148,5 @@
       <origin xyz="0 0 0" rpy="0 0 0" />
     </joint>
-    <joint name="${prefix}joint_a1" type="revolute">
+    <joint name="${prefix}joint_1" type="revolute">
       <axis xyz="0.0 0.0 1.0"/>
       <child link="${prefix}link_1"/>
@@ -155,5 +155,5 @@
       <parent link="${prefix}base_link_inertia"/>
     </joint>
-    <joint name="${prefix}joint_a2" type="revolute">
+    <joint name="${prefix}joint_2" type="revolute">
       <axis xyz="0.0 0.0 1.0"/>
       <child link="${prefix}link_2"/>
@@ -162,5 +162,5 @@
       <parent link="${prefix}link_1"/>
     </joint>
-    <joint name="${prefix}joint_a3" type="revolute">
+    <joint name="${prefix}joint_3" type="revolute">
       <axis xyz="0.0 0.0 1.0"/>
       <child link="${prefix}link_3"/>
@@ -169,5 +169,5 @@
       <parent link="${prefix}link_2"/>
     </joint>
-    <joint name="${prefix}joint_a4" type="revolute">
+    <joint name="${prefix}joint_4" type="revolute">
       <axis xyz="0.0 0.0 1.0"/>
       <child link="${prefix}link_4"/>
@@ -176,5 +176,5 @@
       <parent link="${prefix}link_3"/>
     </joint>
-    <joint name="${prefix}joint_a5" type="revolute">
+    <joint name="${prefix}joint_5" type="revolute">
       <axis xyz="0.0 0.0 1.0"/>
       <child link="${prefix}link_5"/>
@@ -183,5 +183,5 @@
       <parent link="${prefix}link_4"/>
     </joint>
-    <joint name="${prefix}joint_a6" type="revolute">
+    <joint name="${prefix}joint_6" type="revolute">
       <axis xyz="0.0 0.0 1.0"/>
       <child link="${prefix}link_6"/>

File: kuka_quantec_support/urdf/kr_quantec_ros2_control.xacro (robot description, xacro)
@@ -20,5 +20,5 @@
         </xacro:unless>
       </hardware>
-      <joint name="${prefix}joint_a1">
+      <joint name="${prefix}joint_1">
         <command_interface name="position"/>
       <state_interface name="position">
@@ -26,5 +26,5 @@
       </state_interface>
       </joint>
-      <joint name="${prefix}joint_a2">
+      <joint name="${prefix}joint_2">
         <command_interface name="position"/>
       <state_interface name="position">
@@ -32,5 +32,5 @@
       </state_interface>
       </joint>
-      <joint name="${prefix}joint_a3">
+      <joint name="${prefix}joint_3">
         <command_interface name="position"/>
       <state_interface name="position">
@@ -38,5 +38,5 @@
       </state_interface>
       </joint>
-      <joint name="${prefix}joint_a4">
+      <joint name="${prefix}joint_4">
         <command_interface name="position"/>
       <state_interface name="position">
@@ -44,5 +44,5 @@
       </state_interface>
       </joint>
-      <joint name="${prefix}joint_a5">
+      <joint name="${prefix}joint_5">
         <command_interface name="position"/>
       <state_interface name="position">
@@ -50,5 +50,5 @@
       </state_interface>
       </joint>
-      <joint name="${prefix}joint_a6">
+      <joint name="${prefix}joint_6">
         <command_interface name="position"/>
       <state_interface name="position">
