Commit message: remove incorrect inertial values from cybertech, agilus + update readme

File: kuka_agilus_support/urdf/kr6_r700_sixx_macro.xacro (robot description, xacro)
@@ -20,9 +20,4 @@
         <xacro:material_kuka_pedestal/>
       </visual>
-      <inertial>
-        <inertia ixx="0.16209200415615" ixy="0.0" ixz="0.0" iyy="0.10881181598555635" iyz="0.0" izz="0.18461591505869543"/>
-        <mass value="1.6916E1"/>
-        <origin rpy="1.6165592773339865 -1.221289277333065 3.10031147437779" xyz="-0.03713348309292976 2.6602033577676952E-5 0.10863850792149446"/>
-      </inertial>
       <collision>
         <origin xyz="0 0 0" rpy="0 0 0"/>
@@ -40,9 +35,4 @@
         <xacro:material_kuka_orange/>
       </visual>
-      <inertial>
-        <inertia ixx="0.07406183855390855" ixy="0.0" ixz="0.0" iyy="0.0890478351825312" iyz="0.0" izz="0.11039570662759429"/>
-        <mass value="8.4159999999999986E0"/>
-        <origin rpy="1.304519343134156 -0.9428616016893947 -1.4226510948637578" xyz="0.006410408745247152 -0.01626805370722434 -0.10658893773764262"/>
-      </inertial>
       <collision>
         <origin xyz="0 0 0" rpy="0 0 0"/>
@@ -60,9 +50,4 @@
         <xacro:material_kuka_orange/>
       </visual>
-      <inertial>
-        <inertia ixx="0.27913939628518236" ixy="0.0" ixz="0.0" iyy="0.08120682412128737" iyz="0.0" izz="0.31885940962560827"/>
-        <mass value="1.55659E1"/>
-        <origin rpy="-1.3903732489969973 -1.5149954424356888 -0.1998085283039958" xyz="0.09688971405443952 -0.004085391785890956 -0.07157586711979391"/>
-      </inertial>
       <collision>
         <origin xyz="0 0 0" rpy="0 0 0"/>
@@ -80,9 +65,4 @@
         <xacro:material_kuka_orange/>
       </visual>
-      <inertial>
-        <inertia ixx="0.016743444555446362" ixy="0.0" ixz="0.0" iyy="0.025482537016456808" iyz="0.0" izz="0.02822390996140248"/>
-        <mass value="5.303E0"/>
-        <origin rpy="2.3581203240627353 -0.21894199177335477 -3.004285178078088" xyz="0.022228738449934005 -0.011136149349424855 -0.06927623986422779"/>
-      </inertial>
       <collision>
         <origin xyz="0 0 0" rpy="0 0 0"/>
@@ -100,9 +80,4 @@
         <xacro:material_kuka_orange/>
       </visual>
-      <inertial>
-        <inertia ixx="0.010531272787231831" ixy="0.0" ixz="0.0" iyy="0.03425565311920862" iyz="0.0" izz="0.037359032949440756"/>
-        <mass value="4.6129999999999995E0"/>
-        <origin rpy="-2.0540104905408416 -1.5266176566842766 2.01813464445371" xyz="1.0969000650336042E-4 0.010267591588987646 -0.09163862995881207"/>
-      </inertial>
       <collision>
         <origin xyz="0 0 0" rpy="0 0 0"/>
@@ -120,9 +95,4 @@
         <xacro:material_kuka_orange/>
       </visual>
-      <inertial>
-        <inertia ixx="0.0017317756133102904" ixy="0.0" ixz="0.0" iyy="0.002219500805440681" iyz="0.0" izz="0.002467090055442975"/>
-        <mass value="1.6128E0"/>
-        <origin rpy="1.567898714902774 -0.8611716764868309 -3.100280255900493" xyz="0.009320696924603175 7.83482142857143E-4 -0.026462549603174602"/>
-      </inertial>
       <collision>
         <origin xyz="0 0 0" rpy="0 0 0"/>
@@ -140,9 +110,4 @@
         <xacro:material_kuka_pedestal/>
       </visual>
-      <inertial>
-        <inertia ixx="1.83698267603013E-4" ixy="0.0" ixz="0.0" iyy="1.8213621766783165E-4" iyz="0.0" izz="2.9589000000000004E-4"/>
-        <mass value="7.34E-1"/>
-        <origin rpy="0.0 -0.0 1.223427188696551" xyz="0.0 0.0 -0.011764604904632152"/>
-      </inertial>
       <collision>
         <origin xyz="0 0 0" rpy="0 0 0"/>

File: kuka_agilus_support/urdf/kr6_r900_sixx_macro.xacro (robot description, xacro)
@@ -20,9 +20,4 @@
         <xacro:material_kuka_pedestal/>
       </visual>
-      <inertial>
-        <inertia ixx="0.0" ixy="0.0" ixz="0.0" iyy="0.0" iyz="0.0" izz="0.0"/>
-        <mass value="6.22E0"/>
-        <origin rpy="0.0 -0.0 0.0" xyz="0.0 0.0 0.0"/>
-      </inertial>
       <collision>
         <origin xyz="0 0 0" rpy="0 0 0"/>
@@ -40,9 +35,4 @@
         <xacro:material_kuka_orange/>
       </visual>
-      <inertial>
-        <inertia ixx="0.0" ixy="0.0" ixz="0.0" iyy="0.0" iyz="0.0" izz="0.1"/>
-        <mass value="1.7555E1"/>
-        <origin rpy="0.0 -0.0 0.0" xyz="0.010625999999999998 -0.005681 -0.236731"/>
-      </inertial>
       <collision>
         <origin xyz="0 0 0" rpy="0 0 0"/>
@@ -60,9 +50,4 @@
         <xacro:material_kuka_orange/>
       </visual>
-      <inertial>
-        <inertia ixx="0.508" ixy="0.0" ixz="0.0" iyy="0.043" iyz="0.0" izz="0.522"/>
-        <mass value="1.1835E1"/>
-        <origin rpy="0.0 -1.5707963267948966 -1.5707963267948968" xyz="0.223874 0.0 0.007783"/>
-      </inertial>
       <collision>
         <origin xyz="0 0 0" rpy="0 0 0"/>
@@ -80,9 +65,4 @@
         <xacro:material_kuka_orange/>
       </visual>
-      <inertial>
-        <inertia ixx="0.007999999999999991" ixy="0.0" ixz="0.0" iyy="0.059999999999999984" iyz="0.0" izz="0.063"/>
-        <mass value="3.71E0"/>
-        <origin rpy="0.0 -0.0 3.141592653589793" xyz="0.019573999999999994 0.0 0.0014259999999999995"/>
-      </inertial>
       <collision>
         <origin xyz="0 0 0" rpy="0 0 0"/>
@@ -100,9 +80,4 @@
         <xacro:material_kuka_orange/>
       </visual>
-      <inertial>
-        <inertia ixx="0.356" ixy="0.0" ixz="0.0" iyy="0.004" iyz="0.0" izz="0.359"/>
-        <mass value="8.502E0"/>
-        <origin rpy="1.5707963267948966 -0.0 1.5707963267948966" xyz="0.0 0.0 -0.193625"/>
-      </inertial>
       <collision>
         <origin xyz="0 0 0" rpy="0 0 0"/>
@@ -120,9 +95,4 @@
         <xacro:material_kuka_orange/>
       </visual>
-      <inertial>
-        <inertia ixx="0.0" ixy="0.0" ixz="0.0" iyy="0.0" iyz="0.0" izz="0.0"/>
-        <mass value="1.0E-6"/>
-        <origin rpy="0.0 -0.0 0.0" xyz="0.0 0.0 0.0"/>
-      </inertial>
       <collision>
         <origin xyz="0 0 0" rpy="0 0 0"/>
@@ -140,9 +110,4 @@
         <xacro:material_kuka_pedestal/>
       </visual>
-      <inertial>
-        <inertia ixx="0.0" ixy="0.0" ixz="0.0" iyy="0.0" iyz="0.0" izz="0.0"/>
-        <mass value="1.0E-6"/>
-        <origin rpy="0.0 -0.0 0.0" xyz="0.0 0.0 0.0"/>
-      </inertial>
       <collision>
         <origin xyz="0 0 0" rpy="0 0 0"/>

File: kuka_cybertech_support/urdf/kr16_r2010_2_macro.xacro (robot description, xacro)
@@ -17,9 +17,4 @@
         <origin rpy="-0.0 0.0 -0.0" xyz="0.0 0.0 0.0"/>
       </collision>
-      <inertial>
-        <inertia ixx="0.0" ixy="0.0" ixz="0.0" iyy="0.0" iyz="0.0" izz="0.0"/>
-        <mass value="6.52116E1"/>
-        <origin rpy="0.0 -0.0 0.0" xyz="0.0 0.0 0.0"/>
-      </inertial>
       <visual>
         <geometry>
@@ -36,9 +31,4 @@
         <origin rpy="-0.0 0.0 -0.0" xyz="0.0 0.0 0.0"/>
       </collision>
-      <inertial>
-        <inertia ixx="0.0" ixy="0.0" ixz="0.0" iyy="0.0" iyz="0.0" izz="1.50392348"/>
-        <mass value="8.4207E1"/>
-        <origin rpy="0.0 -0.0 1.695151321341658" xyz="0.050473 0.0052792 -0.1312334"/>
-      </inertial>
       <visual>
         <geometry>
@@ -55,9 +45,4 @@
         <origin rpy="-0.0 0.0 -0.0" xyz="0.0 0.0 0.0"/>
       </collision>
-      <inertial>
-        <inertia ixx="9.85967888" ixy="0.0" ixz="0.0" iyy="0.91499458" iyz="0.0" izz="10.23026596"/>
-        <mass value="6.1775E1"/>
-        <origin rpy="0.0 -1.5707963267948966 -1.5707963267948968" xyz="0.4020773724 0.0 -0.0731476"/>
-      </inertial>
       <visual>
         <geometry>
@@ -74,9 +59,4 @@
         <origin rpy="-0.0 0.0 -0.0" xyz="0.0 0.0 0.0"/>
       </collision>
-      <inertial>
-        <inertia ixx="0.34836069" ixy="0.0" ixz="0.0" iyy="1.0268737" iyz="0.0" izz="1.13887402"/>
-        <mass value="3.5648E1"/>
-        <origin rpy="0.0 -0.0 0.0" xyz="0.10935396937 0.0 0.045030299999999995"/>
-      </inertial>
       <visual>
         <geometry>
@@ -93,9 +73,4 @@
         <origin rpy="-0.0 0.0 -0.0" xyz="0.0 0.0 0.0"/>
       </collision>
-      <inertial>
-        <inertia ixx="0.64549911" ixy="0.0" ixz="0.0" iyy="0.04236472" iyz="0.0" izz="0.6665241"/>
-        <mass value="1.64280001E1"/>
-        <origin rpy="1.5707963267948966 -0.0 1.5707963267948966" xyz="0.0 0.0 -0.32342865478"/>
-      </inertial>
       <visual>
         <geometry>
@@ -112,9 +87,4 @@
         <origin rpy="-0.0 0.0 -0.0" xyz="0.0 0.0 0.0"/>
       </collision>
-      <inertial>
-        <inertia ixx="0.0" ixy="0.0" ixz="0.0" iyy="0.0" iyz="0.0" izz="0.0"/>
-        <mass value="1.0E-6"/>
-        <origin rpy="0.0 -0.0 0.0" xyz="0.0 0.0 0.0"/>
-      </inertial>
       <visual>
         <geometry>
@@ -131,9 +101,4 @@
         <origin rpy="-0.0 0.0 -0.0" xyz="0.0 0.0 0.0"/>
       </collision>
-      <inertial>
-        <inertia ixx="0.0" ixy="0.0" ixz="0.0" iyy="0.0" iyz="0.0" izz="0.0"/>
-        <mass value="1.0E-6"/>
-        <origin rpy="0.0 -0.0 0.0" xyz="0.0 0.0 0.0"/>
-      </inertial>
       <visual>
         <geometry>
