Commit message: joint limits fix

File: kuka_agilus_support/urdf/kr10_r1100_2_macro.xacro (robot description, xacro)
@@ -163,5 +163,5 @@
       <axis xyz="0.0 0.0 1.0" />
       <child link="${prefix}link_1" />
-      <limit effort="1.0E1" lower="-2.9670597283903604E0" upper="2.9670597283903604E0" velocity="8.001E3"/>
+      <limit effort="288.36" lower="-2.9670597283903604E0" upper="2.9670597283903604E0" velocity="${radians(300)}"/>
       <origin rpy="-3.141592653589793 0.0 -0.0" xyz="0.0 0.0 0.0"/>
       <parent link="${prefix}base_link_inertia" />
@@ -170,5 +170,5 @@
       <axis xyz="0.0 0.0 1.0" />
       <child link="${prefix}link_2" />
-      <limit effort="1.0E1" lower="-3.3161255787892263E0" upper="7.853981633974483E-1" velocity="8.001E3"/>
+      <limit effort="311.954897896674" lower="-3.3161255787892263E0" upper="7.853981633974483E-1" velocity="${radians(225)}"/>
       <origin rpy="1.5707963267948963 0.0 -0.0" xyz="0.025 0.0 -0.4"/>
       <parent link="${prefix}link_1" />
@@ -177,5 +177,5 @@
       <axis xyz="0.0 0.0 1.0" />
       <child link="${prefix}link_3" />
-      <limit effort="1.0E1" lower="-2.0943951023931953E0" upper="2.722713633111154E0" velocity="8.001E3"/>
+      <limit effort="119.76245366275" lower="-2.0943951023931953E0" upper="2.722713633111154E0" velocity="${radians(330)}"/>
       <origin rpy="0.0 0.0 -1.5707963267948963" xyz="0.56 0.0 0.0"/>
       <parent link="${prefix}link_2" />
@@ -184,5 +184,5 @@
       <axis xyz="0.0 0.0 1.0" />
       <child link="${prefix}link_4" />
-      <limit effort="0.0E0" lower="-3.2288591161895095E0" upper="3.2288591161895095E0" velocity="8.001E3"/>
+      <limit effort="46.081304845791" lower="-3.2288591161895095E0" upper="3.2288591161895095E0" velocity="${radians(360)}"/>
       <origin rpy="1.5707963267948963 0.0 -0.0" xyz="0.025 0.0 0.0"/>
       <parent link="${prefix}link_3" />
@@ -191,5 +191,5 @@
       <axis xyz="0.0 0.0 1.0" />
       <child link="${prefix}link_5" />
-      <limit effort="0.0E0" lower="-2.0943951023931953E0" upper="2.0943951023931953E0" velocity="8.001E3"/>
+      <limit effort="41.6154671315968" lower="-2.0943951023931953E0" upper="2.0943951023931953E0" velocity="${radians(360)}"/>
       <origin rpy="-1.5707963267948963 0.0 -0.0" xyz="0.0 0.0 -0.515"/>
       <parent link="${prefix}link_4" />
@@ -198,5 +198,5 @@
       <axis xyz="0.0 0.0 1.0" />
       <child link="${prefix}link_6" />
-      <limit effort="5.0E2" lower="-6.1086523819801535E0" upper="6.1086523819801535E0" velocity="8.001E3"/>
+      <limit effort="28.03794" lower="-6.1086523819801535E0" upper="6.1086523819801535E0" velocity="${radians(433)}"/>
       <origin rpy="1.5707963267948963 0.0 -0.0" xyz="0.0 0.0 0.0"/>
       <parent link="${prefix}link_5" />

Commit message: fix flange trafo

File: kuka_agilus_support/urdf/kr10_r1100_2_macro.xacro (robot description, xacro)
@@ -213,5 +213,5 @@
     <joint name="${prefix}link6-flange" type="fixed">
       <child link="${prefix}flange" />
-      <origin rpy="0 ${pi} -0.0" xyz="0.0 0.0 -0.09" />
+      <origin rpy="0 ${pi/2} -0.0" xyz="0.0 0.0 -0.09" />
       <parent link="${prefix}link_6" />
     </joint>

File: kuka_cybertech_support/urdf/kr16_r2010_2_macro.xacro (robot description, xacro)
@@ -197,5 +197,5 @@
       <child link="${prefix}base"/>
     </joint>
-        <!-- ROS-Industrial 'flange' frame - attachment point for EEF models -->
+    <!-- ROS-Industrial 'flange' frame - attachment point for EEF models -->
     <link name="${prefix}flange" />
     <joint name="${prefix}link6-flange" type="fixed">

Commit message: kr macro rework

File: kuka_agilus_support/urdf/kr10_r1100_2_macro.xacro (robot description, xacro)
@@ -5,13 +5,15 @@
   <xacro:include filename="$(find kuka_agilus_support)/urdf/kr_agilus_transmission.xacro" />
   <xacro:include filename="$(find kuka_resources)/urdf/common_materials.xacro"/>
-  <xacro:macro name="kuka_kr10_r1100_2_robot" params="prefix use_fake_hardware">
+  <xacro:macro name="kuka_kr10_r1100_2_robot" params="client_ip client_port prefix use_fake_hardware *origin">
     <!-- ros2 control instance -->
     <xacro:kuka_agilus_ros2_control
-    name="kr10_r1100_2"
+    name="${prefix}kr10_r1100_2"
+    client_ip="${client_ip}"
+    client_port="${client_port}"
     prefix="${prefix}"
     use_fake_hardware="${use_fake_hardware}" />
     <!-- links - main serial chain -->
     <!-- links - root element cannot have inertia, therefore a dummy base_link is needed -->
-    <link name="${prefix}base_link"/>
+    <link name="base_link"/>
     <link name="${prefix}base_link_inertia">
       <collision>
@@ -156,7 +158,7 @@
     <!-- joints - main serial chain -->
     <joint name="${prefix}base_link-base_link_inertia" type="fixed">
-      <parent link="${prefix}base_link" />
+      <parent link="base_link" />
       <child link="${prefix}base_link_inertia" />
-      <origin xyz="0 0 0" rpy="0 0 0" />
+      <xacro:insert_block name="origin" />
     </joint>
     <joint name="${prefix}joint_1" type="revolute">
@@ -206,5 +208,5 @@
     <joint name="${prefix}base_link-base" type="fixed">
       <origin xyz="0 0 0" rpy="0 0 0"/>
-      <parent link="${prefix}base_link"/>
+      <parent link="${prefix}base_link_inertia"/>
       <child link="${prefix}base"/>
     </joint>

File: kuka_agilus_support/urdf/kr6_r700_sixx_macro.xacro (robot description, xacro)
@@ -5,11 +5,13 @@
   <xacro:include filename="$(find kuka_agilus_support)/urdf/kr_agilus_ros2_control.xacro" />
   <xacro:include filename="$(find kuka_agilus_support)/urdf/kr_agilus_transmission.xacro" />
-  <xacro:macro name="kuka_kr6_r700_sixx_robot" params="prefix use_fake_hardware">
+  <xacro:macro name="kuka_kr6_r700_sixx_robot" params="client_ip client_port prefix use_fake_hardware *origin">
     <!-- ros2 control instance -->
     <xacro:kuka_agilus_ros2_control
-    name="kr6_r700_sixx"
+    name="${prefix}kr6_r700_sixx"
+    client_ip="${client_ip}"
+    client_port="${client_port}"
     prefix="${prefix}"
     use_fake_hardware="${use_fake_hardware}" />
-    <link name="${prefix}base_link"/>
+    <link name="base_link"/>
     <link name="${prefix}base_link_inertia">
       <visual>
@@ -120,7 +122,7 @@
     <link name="${prefix}flange" />
     <joint name="${prefix}base_link-base_link_inertia" type="fixed">
-      <parent link="${prefix}base_link" />
+      <parent link="base_link" />
       <child link="${prefix}base_link_inertia" />
-      <origin xyz="0 0 0" rpy="0 0 0" />
+      <xacro:insert_block name="origin" />
     </joint>
     <joint name="${prefix}joint_1" type="revolute">
@@ -175,5 +177,5 @@
     <joint name="${prefix}base_link-base" type="fixed">
       <origin xyz="0 0 0" rpy="0 0 0"/>
-      <parent link="${prefix}base_link"/>
+      <parent link="${prefix}base_link_inertia"/>
       <child link="${prefix}base"/>
     </joint>

File: kuka_agilus_support/urdf/kr6_r900_sixx_macro.xacro (robot description, xacro)
@@ -5,11 +5,13 @@
   <xacro:include filename="$(find kuka_agilus_support)/urdf/kr_agilus_ros2_control.xacro" />
   <xacro:include filename="$(find kuka_agilus_support)/urdf/kr_agilus_transmission.xacro" />
-  <xacro:macro name="kuka_kr6_r900_sixx_robot" params="prefix use_fake_hardware">
+  <xacro:macro name="kuka_kr6_r900_sixx_robot" params="client_ip client_port prefix use_fake_hardware *origin">
     <!-- ros2 control instance -->
     <xacro:kuka_agilus_ros2_control
-    name="kr6_r900_sixx"
+    name="${prefix}kr6_r900_sixx"
+    client_ip="${client_ip}"
+    client_port="${client_port}"
     prefix="${prefix}"
     use_fake_hardware="${use_fake_hardware}" />
-    <link name="${prefix}base_link"/>
+    <link name="base_link"/>
     <link name="${prefix}base_link_inertia">
       <visual>
@@ -120,7 +122,7 @@
     <link name="${prefix}flange" />
     <joint name="${prefix}base_link-base_link_inertia" type="fixed">
-      <parent link="${prefix}base_link" />
+      <parent link="base_link" />
       <child link="${prefix}base_link_inertia" />
-      <origin xyz="0 0 0" rpy="0 0 0" />
+      <xacro:insert_block name="origin" />
     </joint>
     <joint name="${prefix}joint_1" type="revolute">
@@ -175,5 +177,5 @@
     <joint name="${prefix}base_link-base" type="fixed">
       <origin xyz="0 0 0" rpy="0 0 0"/>
-      <parent link="${prefix}base_link"/>
+      <parent link="${prefix}base_link_inertia"/>
       <child link="${prefix}base"/>
     </joint>

File: kuka_cybertech_support/urdf/kr16_r2010_2_macro.xacro (robot description, xacro)
@@ -3,11 +3,13 @@
   <xacro:include filename="$(find kuka_cybertech_support)/urdf/kr_cybertech_ros2_control.xacro" />
   <xacro:include filename="$(find kuka_cybertech_support)/urdf/kr_cybertech_transmission.xacro" />
-  <xacro:macro name="kuka_kr16_r2010_2_robot" params="prefix use_fake_hardware">
+  <xacro:macro name="kuka_kr16_r2010_2_robot" params="client_ip client_port prefix use_fake_hardware *origin">
     <!-- ros2 control instance -->
     <xacro:kuka_cybertech_ros2_control
-    name="kr16_r2010_2"
+    name="${prefix}kr16_r2010_2"
+    client_ip="${client_ip}"
+    client_port="${client_port}"
     prefix="${prefix}"
     use_fake_hardware="${use_fake_hardware}" />
-    <link name="${prefix}base_link"/>
+    <link name="base_link"/>
     <link name="${prefix}base_link_inertia">
       <collision>
@@ -144,7 +146,7 @@
     </link>
     <joint name="${prefix}base_link-base_link_inertia" type="fixed">
-      <parent link="${prefix}base_link" />
+      <parent link="base_link" />
       <child link="${prefix}base_link_inertia" />
-      <origin xyz="0 0 0" rpy="0 0 0" />
+      <xacro:insert_block name="origin" />
     </joint>
     <joint name="${prefix}joint_1" type="revolute">
@@ -194,5 +196,5 @@
     <joint name="${prefix}base_link-base" type="fixed">
       <origin xyz="0 0 0" rpy="0 0 0"/>
-      <parent link="${prefix}base_link"/>
+      <parent link="${prefix}base_link_inertia"/>
       <child link="${prefix}base"/>
     </joint>

File: kuka_quantec_support/urdf/kr210_r2700_2_macro.xacro (robot description, xacro)
@@ -3,11 +3,13 @@
   <xacro:include filename="$(find kuka_quantec_support)/urdf/kr_quantec_ros2_control.xacro" />
   <xacro:include filename="$(find kuka_quantec_support)/urdf/kr_quantec_transmission.xacro" />
-  <xacro:macro name="kuka_kr210_r2700_2_robot" params="prefix use_fake_hardware">
+  <xacro:macro name="kuka_kr210_r2700_2_robot" params="client_ip client_port prefix use_fake_hardware *origin">
     <!-- ros2 control instance -->
     <xacro:kuka_quantec_ros2_control
-    name="kr210_r2700_2"
+    name="${prefix}kr210_r2700_2"
+    client_ip="${client_ip}"
+    client_port="${client_port}"
     prefix="${prefix}"
     use_fake_hardware="${use_fake_hardware}" />
-    <link name="${prefix}base_link"/>
+    <link name="base_link"/>
     <link name="${prefix}base_link_inertia">
       <collision>
@@ -144,7 +146,7 @@
     </link>
     <joint name="${prefix}base_link-base_link_inertia" type="fixed">
-      <parent link="${prefix}base_link" />
+      <parent link="base_link" />
       <child link="${prefix}base_link_inertia" />
-      <origin xyz="0 0 0" rpy="0 0 0" />
+      <xacro:insert_block name="origin" />
     </joint>
     <joint name="${prefix}joint_1" type="revolute">
@@ -194,5 +196,5 @@
     <joint name="${prefix}base_link-base" type="fixed">
       <origin xyz="0 0 0" rpy="0 0 0"/>
-      <parent link="${prefix}base_link"/>
+      <parent link="${prefix}base_link_inertia"/>
       <child link="${prefix}base"/>
     </joint>

File: kuka_quantec_support/urdf/kr210_r3100_2_macro.xacro (robot description, xacro)
@@ -3,11 +3,13 @@
   <xacro:include filename="$(find kuka_quantec_support)/urdf/kr_quantec_ros2_control.xacro" />
   <xacro:include filename="$(find kuka_quantec_support)/urdf/kr_quantec_transmission.xacro" />
-  <xacro:macro name="kuka_kr210_r3100_2_robot" params="prefix use_fake_hardware">
+  <xacro:macro name="kuka_kr210_r3100_2_robot" params="client_ip client_port prefix use_fake_hardware *origin">
     <!-- ros2 control instance -->
     <xacro:kuka_quantec_ros2_control
-    name="kr210_r3100_2"
+    name="${prefix}kr210_r3100_2"
+    client_ip="${client_ip}"
+    client_port="${client_port}"
     prefix="${prefix}"
     use_fake_hardware="${use_fake_hardware}" />
-    <link name="${prefix}base_link"/>
+    <link name="base_link"/>
     <link name="${prefix}base_link_inertia">
       <collision>
@@ -144,7 +146,7 @@
     </link>
     <joint name="${prefix}base_link-base_link_inertia" type="fixed">
-      <parent link="${prefix}base_link" />
+      <parent link="base_link" />
       <child link="${prefix}base_link_inertia" />
-      <origin xyz="0 0 0" rpy="0 0 0" />
+      <xacro:insert_block name="origin" />
     </joint>
     <joint name="${prefix}joint_1" type="revolute">
@@ -194,5 +196,5 @@
     <joint name="${prefix}base_link-base" type="fixed">
       <origin xyz="0 0 0" rpy="0 0 0"/>
-      <parent link="${prefix}base_link"/>
+      <parent link="${prefix}base_link_inertia"/>
       <child link="${prefix}base"/>
     </joint>

Commit message: base_link->world

File: kuka_agilus_support/urdf/kr10_r1100_2_macro.xacro (robot description, xacro)
@@ -15,5 +15,5 @@
     <!-- links - main serial chain -->
     <!-- links - root element cannot have inertia, therefore a dummy base_link is needed -->
-    <link name="base_link"/>
+    <link name="world"/>
     <link name="${prefix}base_link_inertia">
       <collision>
@@ -158,5 +158,5 @@
     <!-- joints - main serial chain -->
     <joint name="${prefix}base_link-base_link_inertia" type="fixed">
-      <parent link="base_link" />
+      <parent link="world" />
       <child link="${prefix}base_link_inertia" />
       <xacro:insert_block name="origin" />

File: kuka_agilus_support/urdf/kr6_r700_sixx_macro.xacro (robot description, xacro)
@@ -13,5 +13,5 @@
     prefix="${prefix}"
     use_fake_hardware="${use_fake_hardware}" />
-    <link name="base_link"/>
+    <link name="world"/>
     <link name="${prefix}base_link_inertia">
       <visual>
@@ -122,5 +122,5 @@
     <link name="${prefix}flange" />
     <joint name="${prefix}base_link-base_link_inertia" type="fixed">
-      <parent link="base_link" />
+      <parent link="world" />
       <child link="${prefix}base_link_inertia" />
       <xacro:insert_block name="origin" />

File: kuka_agilus_support/urdf/kr6_r900_sixx_macro.xacro (robot description, xacro)
@@ -13,5 +13,5 @@
     prefix="${prefix}"
     use_fake_hardware="${use_fake_hardware}" />
-    <link name="base_link"/>
+    <link name="world"/>
     <link name="${prefix}base_link_inertia">
       <visual>
@@ -122,5 +122,5 @@
     <link name="${prefix}flange" />
     <joint name="${prefix}base_link-base_link_inertia" type="fixed">
-      <parent link="base_link" />
+      <parent link="world" />
       <child link="${prefix}base_link_inertia" />
       <xacro:insert_block name="origin" />

File: kuka_cybertech_support/urdf/kr16_r2010_2_macro.xacro (robot description, xacro)
@@ -11,5 +11,5 @@
     prefix="${prefix}"
     use_fake_hardware="${use_fake_hardware}" />
-    <link name="base_link"/>
+    <link name="world"/>
     <link name="${prefix}base_link_inertia">
       <collision>
@@ -146,5 +146,5 @@
     </link>
     <joint name="${prefix}base_link-base_link_inertia" type="fixed">
-      <parent link="base_link" />
+      <parent link="world" />
       <child link="${prefix}base_link_inertia" />
       <xacro:insert_block name="origin" />

File: kuka_lbr_iisy_moveit_config/srdf/lbr_iisy_arm.macro.xacro (robot description, xacro)
@@ -24,5 +24,5 @@
     </group_state>
     <!--VIRTUAL JOINT: Purpose: this element defines a virtual joint between a robot link and an external frame of reference (considered fixed with respect to the robot)-->
-    <!-- <virtual_joint name="world_joint" type="fixed" parent_frame="world" child_link="base_link" /> -->
+    <!-- <virtual_joint name="world_joint" type="fixed" parent_frame="world" child_link="world" /> -->
     <!--END EFFECTOR: Purpose: Represent information about an end effector.-->
     <end_effector name="${prefix}tool0" parent_link="${prefix}tool0" group="${prefix}end_effector" parent_group="${prefix}manipulator"/>

File: kuka_lbr_iisy_support/urdf/lbr_iisy11_r1300_macro.xacro (robot description, xacro)
@@ -16,5 +16,5 @@
     <!-- links - main serial chain -->
     <!-- links - root element cannot have inertia, therefore a dummy base_link is needed -->
-    <link name="base_link"/>
+    <link name="world"/>
     <link name="${prefix}base_link_inertia">
       <collision>
@@ -159,5 +159,5 @@
     <!-- joints - main serial chain -->
     <joint name="${prefix}base_link-base_link_inertia" type="fixed">
-      <parent link="base_link" />
+      <parent link="world" />
       <child link="${prefix}base_link_inertia" />
       <xacro:insert_block name="origin" />

File: kuka_lbr_iisy_support/urdf/lbr_iisy15_r930_macro.xacro (robot description, xacro)
@@ -16,5 +16,5 @@
     <!-- links - main serial chain -->
     <!-- links - root element cannot have inertia, therefore a dummy base_link is needed -->
-    <link name="base_link"/>
+    <link name="world"/>
     <link name="${prefix}base_link_inertia">
       <collision>
@@ -159,5 +159,5 @@
     <!-- joints - main serial chain -->
     <joint name="${prefix}base_link-base_link_inertia" type="fixed">
-      <parent link="base_link" />
+      <parent link="world" />
       <child link="${prefix}base_link_inertia" />
       <xacro:insert_block name="origin" />

File: kuka_lbr_iisy_support/urdf/lbr_iisy3_r760_macro.xacro (robot description, xacro)
@@ -16,5 +16,5 @@
     <!-- links - main serial chain -->
     <!-- links - root element cannot have inertia, therefore a dummy base_link is needed -->
-    <link name="base_link"/>
+    <link name="world"/>
     <link name="${prefix}base_link_inertia">
       <collision>
@@ -159,5 +159,5 @@
     <!-- joints - main serial chain -->
     <joint name="${prefix}base_link-base_link_inertia" type="fixed">
-      <parent link="base_link" />
+      <parent link="world" />
       <child link="${prefix}base_link_inertia" />
       <xacro:insert_block name="origin" />

File: kuka_lbr_iiwa_support/urdf/lbr_iiwa14_r820_macro.xacro (robot description, xacro)
@@ -14,5 +14,5 @@
     <!-- links - main serial chain -->
     <!-- links - root element cannot have inertia, therefore a dummy base_link is needed -->
-    <link name="base_link"/>
+    <link name="world"/>
     <link name="${prefix}base_link_inertia">
       <visual>
@@ -169,5 +169,5 @@
     <!-- joints - main serial chain -->
     <joint name="${prefix}base_link-base_link_inertia" type="fixed">
-      <parent link="base_link" />
+      <parent link="world" />
       <child link="${prefix}base_link_inertia" />
       <xacro:insert_block name="origin" />

File: kuka_quantec_support/urdf/kr210_r2700_2_macro.xacro (robot description, xacro)
@@ -11,5 +11,5 @@
     prefix="${prefix}"
     use_fake_hardware="${use_fake_hardware}" />
-    <link name="base_link"/>
+    <link name="world"/>
     <link name="${prefix}base_link_inertia">
       <collision>
@@ -146,5 +146,5 @@
     </link>
     <joint name="${prefix}base_link-base_link_inertia" type="fixed">
-      <parent link="base_link" />
+      <parent link="world" />
       <child link="${prefix}base_link_inertia" />
       <xacro:insert_block name="origin" />

File: kuka_quantec_support/urdf/kr210_r3100_2_macro.xacro (robot description, xacro)
@@ -11,5 +11,5 @@
     prefix="${prefix}"
     use_fake_hardware="${use_fake_hardware}" />
-    <link name="base_link"/>
+    <link name="world"/>
     <link name="${prefix}base_link_inertia">
       <collision>
@@ -146,5 +146,5 @@
     </link>
     <joint name="${prefix}base_link-base_link_inertia" type="fixed">
-      <parent link="base_link" />
+      <parent link="world" />
       <child link="${prefix}base_link_inertia" />
       <xacro:insert_block name="origin" />
