Commit message: base_link_inertia->base_link

File: kuka_agilus_support/urdf/kr10_r1100_2_macro.xacro (robot description, xacro)
@@ -14,7 +14,6 @@
     use_fake_hardware="${use_fake_hardware}" />
     <!-- links - main serial chain -->
-    <!-- links - root element cannot have inertia, therefore a dummy base_link is needed -->
     <link name="world"/>
-    <link name="${prefix}base_link_inertia">
+    <link name="${prefix}base_link">
       <collision>
         <geometry>
@@ -157,7 +156,7 @@
     </link>
     <!-- joints - main serial chain -->
-    <joint name="${prefix}base_link-base_link_inertia" type="fixed">
+    <joint name="${prefix}world-base_link" type="fixed">
       <parent link="world" />
-      <child link="${prefix}base_link_inertia" />
+      <child link="${prefix}base_link" />
       <xacro:insert_block name="origin" />
     </joint>
@@ -167,5 +166,5 @@
       <limit effort="288.36" lower="-2.9670597283903604E0" upper="2.9670597283903604E0" velocity="${radians(300)}"/>
       <origin rpy="-3.141592653589793 0.0 -0.0" xyz="0.0 0.0 0.0"/>
-      <parent link="${prefix}base_link_inertia" />
+      <parent link="${prefix}base_link" />
     </joint>
     <joint name="${prefix}joint_2" type="revolute">
@@ -208,5 +207,5 @@
     <joint name="${prefix}base_link-base" type="fixed">
       <origin xyz="0 0 0" rpy="0 0 0"/>
-      <parent link="${prefix}base_link_inertia"/>
+      <parent link="${prefix}base_link"/>
       <child link="${prefix}base"/>
     </joint>

File: kuka_agilus_support/urdf/kr6_r700_sixx_macro.xacro (robot description, xacro)
@@ -14,5 +14,5 @@
     use_fake_hardware="${use_fake_hardware}" />
     <link name="world"/>
-    <link name="${prefix}base_link_inertia">
+    <link name="${prefix}base_link">
       <visual>
         <origin xyz="0 0 0" rpy="0 0 0" />
@@ -121,12 +121,12 @@
     <!-- Following REP199, this frame shall be use to attach EEF or other equipment -->
     <link name="${prefix}flange" />
-    <joint name="${prefix}base_link-base_link_inertia" type="fixed">
+    <joint name="${prefix}world-base_link" type="fixed">
       <parent link="world" />
-      <child link="${prefix}base_link_inertia" />
+      <child link="${prefix}base_link" />
       <xacro:insert_block name="origin" />
     </joint>
     <joint name="${prefix}joint_1" type="revolute">
       <origin xyz="0 0 0.4" rpy="0 0 0"/>
-      <parent link="${prefix}base_link_inertia"/>
+      <parent link="${prefix}base_link"/>
       <child link="${prefix}link_1"/>
       <axis xyz="0 0 -1"/>
@@ -177,5 +177,5 @@
     <joint name="${prefix}base_link-base" type="fixed">
       <origin xyz="0 0 0" rpy="0 0 0"/>
-      <parent link="${prefix}base_link_inertia"/>
+      <parent link="${prefix}base_link"/>
       <child link="${prefix}base"/>
     </joint>

File: kuka_agilus_support/urdf/kr6_r900_sixx_macro.xacro (robot description, xacro)
@@ -14,5 +14,5 @@
     use_fake_hardware="${use_fake_hardware}" />
     <link name="world"/>
-    <link name="${prefix}base_link_inertia">
+    <link name="${prefix}base_link">
       <visual>
         <origin xyz="0 0 0" rpy="0 0 0"/>
@@ -121,12 +121,12 @@
     <!-- Following REP199, this frame shall be use to attach EEF or other equipment -->
     <link name="${prefix}flange" />
-    <joint name="${prefix}base_link-base_link_inertia" type="fixed">
+    <joint name="${prefix}world-base_link" type="fixed">
       <parent link="world" />
-      <child link="${prefix}base_link_inertia" />
+      <child link="${prefix}base_link" />
       <xacro:insert_block name="origin" />
     </joint>
     <joint name="${prefix}joint_1" type="revolute">
       <origin xyz="0 0 0.400" rpy="0 0 0"/>
-      <parent link="${prefix}base_link_inertia"/>
+      <parent link="${prefix}base_link"/>
       <child link="${prefix}link_1"/>
       <axis xyz="0 0 -1"/>
@@ -177,5 +177,5 @@
     <joint name="${prefix}base_link-base" type="fixed">
       <origin xyz="0 0 0" rpy="0 0 0"/>
-      <parent link="${prefix}base_link_inertia"/>
+      <parent link="${prefix}base_link"/>
       <child link="${prefix}base"/>
     </joint>

File: kuka_cybertech_support/urdf/kr16_r2010_2_macro.xacro (robot description, xacro)
@@ -12,5 +12,5 @@
     use_fake_hardware="${use_fake_hardware}" />
     <link name="world"/>
-    <link name="${prefix}base_link_inertia">
+    <link name="${prefix}base_link">
       <collision>
         <geometry>
@@ -145,7 +145,7 @@
       </visual>
     </link>
-    <joint name="${prefix}base_link-base_link_inertia" type="fixed">
+    <joint name="${prefix}world-base_link" type="fixed">
       <parent link="world" />
-      <child link="${prefix}base_link_inertia" />
+      <child link="${prefix}base_link" />
       <xacro:insert_block name="origin" />
     </joint>
@@ -155,5 +155,5 @@
       <limit effort="1905.3" lower="-3.2288591162E0" upper="3.2288591161895095E0" velocity="${radians(200)}"/>
       <origin rpy="${-pi} 0.0 -0.0" xyz="0.0 0.0 0.0"/>
-      <parent link="${prefix}base_link_inertia"/>
+      <parent link="${prefix}base_link"/>
     </joint>
     <joint name="${prefix}joint_2" type="revolute">
@@ -196,5 +196,5 @@
     <joint name="${prefix}base_link-base" type="fixed">
       <origin xyz="0 0 0" rpy="0 0 0"/>
-      <parent link="${prefix}base_link_inertia"/>
+      <parent link="${prefix}base_link"/>
       <child link="${prefix}base"/>
     </joint>

File: kuka_kr_moveit_config/srdf/kr_arm_macro.xacro (robot description, xacro)
@@ -8,5 +8,5 @@
     <!--SUBGROUPS: Groups can also be formed by referencing to already defined group names-->
     <group name="${prefix}manipulator">
-      <chain base_link="${prefix}base_link_inertia" tip_link="${prefix}tool0" />
+      <chain base_link="${prefix}base_link" tip_link="${prefix}tool0" />
     </group>
     <!--Add tool0 as end effector to be able to use moveit_visual_tools for visualising end effector path-->
@@ -26,5 +26,5 @@
     <end_effector name="${prefix}eef" parent_link="${prefix}tool0" group="${prefix}end_effector" parent_group="${prefix}manipulator"/>
     <!--DISABLE COLLISIONS: By default it is assumed that any link of the robot could potentially come into collision with any other link in the robot. This tag disables collision checking between a specified pair of links. -->
-    <disable_collisions link1="${prefix}base_link_inertia" link2="${prefix}link_1" reason="Adjacent"/>
+    <disable_collisions link1="${prefix}base_link" link2="${prefix}link_1" reason="Adjacent"/>
     <disable_collisions link1="${prefix}link_1" link2="${prefix}link_2" reason="Adjacent"/>
     <disable_collisions link1="${prefix}link_2" link2="${prefix}link_3" reason="Adjacent"/>

File: kuka_lbr_iisy_moveit_config/srdf/lbr_iisy_arm.macro.xacro (robot description, xacro)
@@ -8,5 +8,5 @@
     <!--SUBGROUPS: Groups can also be formed by referencing to already defined group names-->
     <group name="${prefix}manipulator">
-      <chain base_link="${prefix}base_link_inertia" tip_link="${prefix}tool0" />
+      <chain base_link="${prefix}base_link" tip_link="${prefix}tool0" />
     </group>
     <!--Add tool0 as end effector to be able to use moveit_visual_tools for visualising end effector path-->
@@ -28,5 +28,5 @@
     <end_effector name="${prefix}tool0" parent_link="${prefix}tool0" group="${prefix}end_effector" parent_group="${prefix}manipulator"/>
     <!--DISABLE COLLISIONS: By default it is assumed that any link of the robot could potentially come into collision with any other link in the robot. This tag disables collision checking between a specified pair of links. -->
-    <disable_collisions link1="${prefix}base_link_inertia" link2="${prefix}link_1" reason="Adjacent"/>
+    <disable_collisions link1="${prefix}base_link" link2="${prefix}link_1" reason="Adjacent"/>
     <disable_collisions link1="${prefix}link_1" link2="${prefix}link_2" reason="Adjacent"/>
     <disable_collisions link1="${prefix}link_2" link2="${prefix}link_3" reason="Adjacent"/>

File: kuka_lbr_iisy_support/urdf/lbr_iisy11_r1300_macro.xacro (robot description, xacro)
@@ -15,7 +15,6 @@
     qos_config_file="${qos_config_file}" />
     <!-- links - main serial chain -->
-    <!-- links - root element cannot have inertia, therefore a dummy base_link is needed -->
     <link name="world"/>
-    <link name="${prefix}base_link_inertia">
+    <link name="${prefix}base_link">
       <collision>
         <geometry>
@@ -158,7 +157,7 @@
     </link>
     <!-- joints - main serial chain -->
-    <joint name="${prefix}base_link-base_link_inertia" type="fixed">
+    <joint name="${prefix}world-base_link" type="fixed">
       <parent link="world" />
-      <child link="${prefix}base_link_inertia" />
+      <child link="${prefix}base_link" />
       <xacro:insert_block name="origin" />
     </joint>
@@ -168,5 +167,5 @@
       <limit effort="405.840000" lower="-3.2288591161895095E0" upper="3.2288591161895095E0" velocity="3.490656"/>
       <origin rpy="${-pi} 0.0 -0.0" xyz="0.0 0.0 0.0"/>
-      <parent link="${prefix}base_link_inertia" />
+      <parent link="${prefix}base_link" />
     </joint>
     <joint name="${prefix}joint_2" type="revolute">
@@ -209,5 +208,5 @@
     <joint name="${prefix}base_link-base" type="fixed">
       <origin xyz="0 0 0" rpy="0 0 0"/>
-      <parent link="${prefix}base_link_inertia"/>
+      <parent link="${prefix}base_link"/>
       <child link="${prefix}base"/>
     </joint>

File: kuka_lbr_iisy_support/urdf/lbr_iisy15_r930_macro.xacro (robot description, xacro)
@@ -15,7 +15,6 @@
     qos_config_file="${qos_config_file}" />
     <!-- links - main serial chain -->
-    <!-- links - root element cannot have inertia, therefore a dummy base_link is needed -->
     <link name="world"/>
-    <link name="${prefix}base_link_inertia">
+    <link name="${prefix}base_link">
       <collision>
         <geometry>
@@ -158,7 +157,7 @@
     </link>
     <!-- joints - main serial chain -->
-    <joint name="${prefix}base_link-base_link_inertia" type="fixed">
+    <joint name="${prefix}world-base_link" type="fixed">
       <parent link="world" />
-      <child link="${prefix}base_link_inertia" />
+      <child link="${prefix}base_link" />
       <xacro:insert_block name="origin" />
     </joint>
@@ -168,5 +167,5 @@
       <limit effort="398.011277" lower="-3.2288591161895095E0" upper="3.2288591161895095E0" velocity="3.490656"/>
       <origin rpy="${-pi} 0.0 -0.0" xyz="0.0 0.0 0.0"/>
-      <parent link="${prefix}base_link_inertia" />
+      <parent link="${prefix}base_link" />
     </joint>
     <joint name="${prefix}joint_2" type="revolute">
@@ -209,5 +208,5 @@
     <joint name="${prefix}base_link-base" type="fixed">
       <origin xyz="0 0 0" rpy="0 0 0"/>
-      <parent link="${prefix}base_link_inertia"/>
+      <parent link="${prefix}base_link"/>
       <child link="${prefix}base"/>
     </joint>

File: kuka_lbr_iisy_support/urdf/lbr_iisy3_r760_macro.xacro (robot description, xacro)
@@ -15,7 +15,6 @@
     qos_config_file="${qos_config_file}" />
     <!-- links - main serial chain -->
-    <!-- links - root element cannot have inertia, therefore a dummy base_link is needed -->
     <link name="world"/>
-    <link name="${prefix}base_link_inertia">
+    <link name="${prefix}base_link">
       <collision>
         <geometry>
@@ -158,7 +157,7 @@
     </link>
     <!-- joints - main serial chain -->
-    <joint name="${prefix}base_link-base_link_inertia" type="fixed">
+    <joint name="${prefix}world-base_link" type="fixed">
       <parent link="world" />
-      <child link="${prefix}base_link_inertia" />
+      <child link="${prefix}base_link" />
       <xacro:insert_block name="origin" />
     </joint>
@@ -168,5 +167,5 @@
       <limit effort="74.930405" lower="-3.2288591E0" upper="3.2288591E0" velocity="3.490656" />
       <origin rpy="-0.0 0.0 -0.0" xyz="0.0 0.0 0.1264" />
-      <parent link="${prefix}base_link_inertia" />
+      <parent link="${prefix}base_link" />
     </joint>
     <joint name="${prefix}joint_2" type="revolute">
@@ -209,5 +208,5 @@
     <joint name="${prefix}base_link-base" type="fixed">
       <origin xyz="0 0 0" rpy="0 0 0"/>
-      <parent link="${prefix}base_link_inertia"/>
+      <parent link="${prefix}base_link"/>
       <child link="${prefix}base"/>
     </joint>

File: kuka_lbr_iiwa_moveit_config/srdf/lbr_iiwa_arm.macro.xacro (robot description, xacro)
@@ -8,5 +8,5 @@
     <!--SUBGROUPS: Groups can also be formed by referencing to already defined group names-->
     <group name="${prefix}manipulator">
-      <chain base_link="${prefix}base_link_inertia" tip_link="${prefix}tool0" />
+      <chain base_link="${prefix}base_link" tip_link="${prefix}tool0" />
     </group>
     <!--Add tool0 as end effector to be able to use moveit_visual_tools for visualising end effector path-->
@@ -25,9 +25,9 @@
     </group_state>
     <!--VIRTUAL JOINT: Purpose: this element defines a virtual joint between a robot link and an external frame of reference (considered fixed with respect to the robot)-->
-    <!-- <virtual_joint name="virtual_joint" type="floating" parent_frame="world" child_link="${prefix}base_link_inertia" /> -->
+    <!-- <virtual_joint name="virtual_joint" type="floating" parent_frame="world" child_link="${prefix}base_link" /> -->
     <!--END EFFECTOR: Purpose: Represent information about an end effector.-->
     <end_effector name="tool0" parent_link="${prefix}tool0" group="end_effector" parent_group="manipulator"/>
     <!--DISABLE COLLISIONS: By default it is assumed that any link of the robot could potentially come into collision with any other link in the robot. This tag disables collision checking between a specified pair of links. -->
-    <disable_collisions link1="${prefix}base_link_inertia" link2="${prefix}link_1" reason="Adjacent"/>
+    <disable_collisions link1="${prefix}base_link" link2="${prefix}link_1" reason="Adjacent"/>
     <disable_collisions link1="${prefix}link_1" link2="${prefix}link_2" reason="Adjacent"/>
     <disable_collisions link1="${prefix}link_2" link2="${prefix}link_3" reason="Adjacent"/>
@@ -36,7 +36,7 @@
     <disable_collisions link1="${prefix}link_5" link2="${prefix}link_6" reason="Adjacent"/>
     <disable_collisions link1="${prefix}link_6" link2="${prefix}link_7" reason="Adjacent"/>
-    <disable_collisions link1="${prefix}base_link_inertia" link2="${prefix}link_1" reason="Never" />
-    <disable_collisions link1="${prefix}base_link_inertia" link2="${prefix}link_2" reason="Never" />
-    <disable_collisions link1="${prefix}base_link_inertia" link2="${prefix}link_3" reason="Never" />
+    <disable_collisions link1="${prefix}base_link" link2="${prefix}link_1" reason="Never" />
+    <disable_collisions link1="${prefix}base_link" link2="${prefix}link_2" reason="Never" />
+    <disable_collisions link1="${prefix}base_link" link2="${prefix}link_3" reason="Never" />
   </xacro:macro>
 </robot>

File: kuka_lbr_iiwa_support/urdf/lbr_iiwa14_r820_macro.xacro (robot description, xacro)
@@ -13,7 +13,6 @@
     use_fake_hardware="${use_fake_hardware}" />
     <!-- links - main serial chain -->
-    <!-- links - root element cannot have inertia, therefore a dummy base_link is needed -->
     <link name="world"/>
-    <link name="${prefix}base_link_inertia">
+    <link name="${prefix}base_link">
       <visual>
         <geometry>
@@ -168,11 +167,11 @@
     </link>
     <!-- joints - main serial chain -->
-    <joint name="${prefix}base_link-base_link_inertia" type="fixed">
+    <joint name="${prefix}world-base_link" type="fixed">
       <parent link="world" />
-      <child link="${prefix}base_link_inertia" />
+      <child link="${prefix}base_link" />
       <xacro:insert_block name="origin" />
     </joint>
     <joint name="${prefix}joint_1" type="revolute">
-      <parent link="${prefix}base_link_inertia"/>
+      <parent link="${prefix}base_link"/>
       <child link="${prefix}link_1"/>
       <origin rpy="-0.0 0.0 0.0" xyz="0.0 0.0 0.1375"/>
@@ -226,5 +225,5 @@
     <joint name="${prefix}base_link-base" type="fixed">
       <origin xyz="0 0 0" rpy="0 0 0"/>
-      <parent link="${prefix}base_link_inertia"/>
+      <parent link="${prefix}base_link"/>
       <child link="${prefix}base"/>
     </joint>

File: kuka_quantec_support/urdf/kr210_r2700_2_macro.xacro (robot description, xacro)
@@ -12,5 +12,5 @@
     use_fake_hardware="${use_fake_hardware}" />
     <link name="world"/>
-    <link name="${prefix}base_link_inertia">
+    <link name="${prefix}base_link">
       <collision>
         <geometry>
@@ -145,7 +145,7 @@
       </visual>
     </link>
-    <joint name="${prefix}base_link-base_link_inertia" type="fixed">
+    <joint name="${prefix}world-base_link" type="fixed">
       <parent link="world" />
-      <child link="${prefix}base_link_inertia" />
+      <child link="${prefix}base_link" />
       <xacro:insert_block name="origin" />
     </joint>
@@ -155,5 +155,5 @@
       <limit effort="7290" lower="-3.2288591161895095E0" upper="3.2288591161895095E0" velocity="${radians(120)}"/>
       <origin rpy="-3.141592653589793 0.0 -0.0" xyz="0.0 0.0 0.0"/>
-      <parent link="${prefix}base_link_inertia"/>
+      <parent link="${prefix}base_link"/>
     </joint>
     <joint name="${prefix}joint_2" type="revolute">
@@ -196,5 +196,5 @@
     <joint name="${prefix}base_link-base" type="fixed">
       <origin xyz="0 0 0" rpy="0 0 0"/>
-      <parent link="${prefix}base_link_inertia"/>
+      <parent link="${prefix}base_link"/>
       <child link="${prefix}base"/>
     </joint>

File: kuka_quantec_support/urdf/kr210_r3100_2_macro.xacro (robot description, xacro)
@@ -12,5 +12,5 @@
     use_fake_hardware="${use_fake_hardware}" />
     <link name="world"/>
-    <link name="${prefix}base_link_inertia">
+    <link name="${prefix}base_link">
       <collision>
         <geometry>
@@ -145,7 +145,7 @@
       </visual>
     </link>
-    <joint name="${prefix}base_link-base_link_inertia" type="fixed">
+    <joint name="${prefix}world-base_link" type="fixed">
       <parent link="world" />
-      <child link="${prefix}base_link_inertia" />
+      <child link="${prefix}base_link" />
       <xacro:insert_block name="origin" />
     </joint>
@@ -155,5 +155,5 @@
       <limit effort="7290" lower="-3.2288591161895095E0" upper="3.2288591161895095E0" velocity="${radians(105)}"/>
       <origin rpy="-3.141592653589793 0.0 -0.0" xyz="0.0 0.0 0.0"/>
-      <parent link="${prefix}base_link_inertia"/>
+      <parent link="${prefix}base_link"/>
     </joint>
     <joint name="${prefix}joint_2" type="revolute">
@@ -196,5 +196,5 @@
     <joint name="${prefix}base_link-base" type="fixed">
       <origin xyz="0 0 0" rpy="0 0 0"/>
-      <parent link="${prefix}base_link_inertia"/>
+      <parent link="${prefix}base_link"/>
       <child link="${prefix}base"/>
     </joint>

Commit message: Added a new robot model for the KUKA FORTEC family (#42)
* added fortec support

* update readme

* moveit settings

* renaming xacros

* moveit xacros done

* changed file path ref

* renaming file

* Fix flange transform in kr560_r3100_2_macro.xacro

Added a new robot model for the KUKA FORTEC family
#42

https://github.com/kroshu/kuka_robot_descriptions/pull/42#discussion_r1440587691

Co-authored-by: Svastits <49677296+Svastits@users.noreply.github.com>

* tool0 frame should be equivalent to the TCP

Fix PR comment 

https://github.com/kroshu/kuka_robot_descriptions/pull/42#discussion_r1440516921

Co-authored-by: Svastits <49677296+Svastits@users.noreply.github.com>

* revert rviz config

Reverting to using kuka_resources pkg to load rviz2 default configs: https://github.com/kroshu/kuka_robot_descriptions/pull/42#discussion_r1440507033

* mesh folder rename

https://github.com/kroshu/kuka_robot_descriptions/pull/42#discussion_r1440520754

* using joint_state_publisher_gui

solving:
- https://github.com/kroshu/kuka_robot_descriptions/pull/42#discussion_r1440508434
- https://github.com/kroshu/kuka_robot_descriptions/pull/42#discussion_r1440508710

* add ips as xacro arg

* remove prefix from base_link

* fix origin

* add all dofs to all iisys

* fix 11

* add qos config file arg

* syntax fix

* rename file

* remove pre-commit mod

* kr ros2_control+ urdf.xacro rework

* change manipulator base_link

* kr macro rework

* remove duplicate default

* iiwa fix

* format

* add missing args

* workaround for  kuka_iiqka_eac_driver

* base_link->world

* base_link_inertia->base_link

* rviz config names

* update md

* format

* rviz config cleanup

* 7axis planning scene rviz config

* fix after merge

---------

Co-authored-by: Svastits <49677296+Svastits@users.noreply.github.com>
Co-authored-by: Aron Svastits <svastits1@gmail.com>

File: kuka_agilus_support/urdf/kr10_r1100_2_macro.xacro (robot description, xacro)
@@ -5,14 +5,15 @@
   <xacro:include filename="$(find kuka_agilus_support)/urdf/kr_agilus_transmission.xacro" />
   <xacro:include filename="$(find kuka_resources)/urdf/common_materials.xacro"/>
-  <xacro:macro name="kuka_kr10_r1100_2_robot" params="prefix use_fake_hardware">
+  <xacro:macro name="kuka_kr10_r1100_2_robot" params="client_ip client_port prefix use_fake_hardware *origin">
     <!-- ros2 control instance -->
     <xacro:kuka_agilus_ros2_control
-    name="kr10_r1100_2"
+    name="${prefix}kr10_r1100_2"
+    client_ip="${client_ip}"
+    client_port="${client_port}"
     prefix="${prefix}"
     use_fake_hardware="${use_fake_hardware}" />
     <!-- links - main serial chain -->
-    <!-- links - root element cannot have inertia, therefore a dummy base_link is needed -->
-    <link name="${prefix}base_link"/>
-    <link name="${prefix}base_link_inertia">
+    <link name="world"/>
+    <link name="${prefix}base_link">
       <collision>
         <geometry>
@@ -155,8 +156,8 @@
     </link>
     <!-- joints - main serial chain -->
-    <joint name="${prefix}base_link-base_link_inertia" type="fixed">
-      <parent link="${prefix}base_link" />
-      <child link="${prefix}base_link_inertia" />
-      <origin xyz="0 0 0" rpy="0 0 0" />
+    <joint name="${prefix}world-base_link" type="fixed">
+      <parent link="world" />
+      <child link="${prefix}base_link" />
+      <xacro:insert_block name="origin" />
     </joint>
     <joint name="${prefix}joint_1" type="revolute">
@@ -165,5 +166,5 @@
       <limit effort="288.36" lower="-2.9670597283903604E0" upper="2.9670597283903604E0" velocity="${radians(300)}"/>
       <origin rpy="-3.141592653589793 0.0 -0.0" xyz="0.0 0.0 0.0"/>
-      <parent link="${prefix}base_link_inertia" />
+      <parent link="${prefix}base_link" />
     </joint>
     <joint name="${prefix}joint_2" type="revolute">
