Commit message: remove capital letters from resources

File: kuka_agilus_support/urdf/kr6_r700_sixx.urdf.xacro (robot description, xacro)
@@ -1,4 +1,4 @@
 <?xml version="1.0"?>
-<robot xmlns:xacro="http://www.ros.org/wiki/xacro" name="KR6R700sixx">
+<robot xmlns:xacro="http://www.ros.org/wiki/xacro" name="kr6_r700_sixx">
 <!-- Import urdf file  -->
 <xacro:include filename="$(find kuka_agilus_support)/urdf/kr6_r700_sixx_macro.xacro"/>

File: kuka_agilus_support/urdf/kr6_r700_sixx_macro.xacro (robot description, xacro)
@@ -8,5 +8,5 @@
     <!-- ros2 control instance -->
     <xacro:kuka_agilus_ros2_control
-    name="KR6R700sixx"
+    name="kr6_r700_sixx"
     prefix="${prefix}"
     client_ip="${client_ip}"
@@ -17,5 +17,5 @@
         <origin xyz="0 0 0" rpy="0 0 0" />
         <geometry>
-          <mesh filename="package://kuka_agilus_support/meshes/KR6R700sixx/visual/base_link.dae" />
+          <mesh filename="package://kuka_agilus_support/meshes/kr6_r700_sixx/visual/base_link.dae" />
         </geometry>
         <xacro:material_kuka_pedestal />
@@ -24,5 +24,5 @@
         <origin xyz="0 0 0" rpy="0 0 0" />
         <geometry>
-          <mesh filename="package://kuka_agilus_support/meshes/KR6R700sixx/collision/base_link.stl" />
+          <mesh filename="package://kuka_agilus_support/meshes/kr6_r700_sixx/collision/base_link.stl" />
         </geometry>
       </collision>
@@ -32,5 +32,5 @@
         <origin xyz="0 0 0" rpy="0 0 0" />
         <geometry>
-          <mesh filename="package://kuka_agilus_support/meshes/KR6R700sixx/visual/link_1.dae" />
+          <mesh filename="package://kuka_agilus_support/meshes/kr6_r700_sixx/visual/link_1.dae" />
         </geometry>
         <xacro:material_kuka_orange />
@@ -39,5 +39,5 @@
         <origin xyz="0 0 0" rpy="0 0 0" />
         <geometry>
-          <mesh filename="package://kuka_agilus_support/meshes/KR6R700sixx/collision/link_1.stl" />
+          <mesh filename="package://kuka_agilus_support/meshes/kr6_r700_sixx/collision/link_1.stl" />
         </geometry>
       </collision>
@@ -47,5 +47,5 @@
         <origin xyz="0 0 0" rpy="0 0 0" />
         <geometry>
-          <mesh filename="package://kuka_agilus_support/meshes/KR6R700sixx/visual/link_2.dae" />
+          <mesh filename="package://kuka_agilus_support/meshes/kr6_r700_sixx/visual/link_2.dae" />
         </geometry>
         <xacro:material_kuka_orange />
@@ -54,5 +54,5 @@
         <origin xyz="0 0 0" rpy="0 0 0" />
         <geometry>
-          <mesh filename="package://kuka_agilus_support/meshes/KR6R700sixx/collision/link_2.stl" />
+          <mesh filename="package://kuka_agilus_support/meshes/kr6_r700_sixx/collision/link_2.stl" />
         </geometry>
       </collision>
@@ -62,5 +62,5 @@
         <origin xyz="0 0 0" rpy="0 0 0" />
         <geometry>
-          <mesh filename="package://kuka_agilus_support/meshes/KR6R700sixx/visual/link_3.dae" />
+          <mesh filename="package://kuka_agilus_support/meshes/kr6_r700_sixx/visual/link_3.dae" />
         </geometry>
         <xacro:material_kuka_orange />
@@ -69,5 +69,5 @@
         <origin xyz="0 0 0" rpy="0 0 0" />
         <geometry>
-          <mesh filename="package://kuka_agilus_support/meshes/KR6R700sixx/collision/link_3.stl" />
+          <mesh filename="package://kuka_agilus_support/meshes/kr6_r700_sixx/collision/link_3.stl" />
         </geometry>
       </collision>
@@ -77,5 +77,5 @@
         <origin xyz="0 0 0" rpy="0 0 0" />
         <geometry>
-          <mesh filename="package://kuka_agilus_support/meshes/KR6R700sixx/visual/link_4.dae" />
+          <mesh filename="package://kuka_agilus_support/meshes/kr6_r700_sixx/visual/link_4.dae" />
         </geometry>
         <xacro:material_kuka_orange />
@@ -84,5 +84,5 @@
         <origin xyz="0 0 0" rpy="0 0 0" />
         <geometry>
-          <mesh filename="package://kuka_agilus_support/meshes/KR6R700sixx/collision/link_4.stl" />
+          <mesh filename="package://kuka_agilus_support/meshes/kr6_r700_sixx/collision/link_4.stl" />
         </geometry>
       </collision>
@@ -92,5 +92,5 @@
         <origin xyz="0 0 0" rpy="0 0 0" />
         <geometry>
-          <mesh filename="package://kuka_agilus_support/meshes/KR6R700sixx/visual/link_5.dae" />
+          <mesh filename="package://kuka_agilus_support/meshes/kr6_r700_sixx/visual/link_5.dae" />
         </geometry>
         <xacro:material_kuka_orange />
@@ -99,5 +99,5 @@
         <origin xyz="0 0 0" rpy="0 0 0" />
         <geometry>
-          <mesh filename="package://kuka_agilus_support/meshes/KR6R700sixx/collision/link_5.stl" />
+          <mesh filename="package://kuka_agilus_support/meshes/kr6_r700_sixx/collision/link_5.stl" />
         </geometry>
       </collision>
@@ -107,5 +107,5 @@
         <origin xyz="0 0 0" rpy="0 0 0" />
         <geometry>
-          <mesh filename="package://kuka_agilus_support/meshes/KR6R700sixx/visual/link_6.dae" />
+          <mesh filename="package://kuka_agilus_support/meshes/kr6_r700_sixx/visual/link_6.dae" />
         </geometry>
         <xacro:material_kuka_pedestal />
@@ -114,5 +114,5 @@
         <origin xyz="0 0 0" rpy="0 0 0" />
         <geometry>
-          <mesh filename="package://kuka_agilus_support/meshes/KR6R700sixx/collision/link_6.stl" />
+          <mesh filename="package://kuka_agilus_support/meshes/kr6_r700_sixx/collision/link_6.stl" />
         </geometry>
       </collision>

File: kuka_agilus_support/urdf/kr6_r900_sixx.urdf.xacro (robot description, xacro)
@@ -1,4 +1,4 @@
 <?xml version="1.0"?>
-<robot xmlns:xacro="http://www.ros.org/wiki/xacro" name="KR6R900sixx">
+<robot xmlns:xacro="http://www.ros.org/wiki/xacro" name="kr6_r900_sixx">
 <!-- Import urdf file  -->
 <xacro:include filename="$(find kuka_agilus_support)/urdf/kr6_r900_sixx_macro.xacro"/>

File: kuka_agilus_support/urdf/kr6_r900_sixx_macro.xacro (robot description, xacro)
@@ -8,5 +8,5 @@
     <!-- ros2 control instance -->
     <xacro:kuka_agilus_ros2_control
-    name="KR6R900sixx"
+    name="kr6_r900_sixx"
     prefix="${prefix}"
     client_ip="${client_ip}"
@@ -17,5 +17,5 @@
         <origin xyz="0 0 0" rpy="0 0 0"/>
         <geometry>
-          <mesh filename="package://kuka_agilus_support/meshes/KR6R900sixx/visual/base_link.dae" />
+          <mesh filename="package://kuka_agilus_support/meshes/kr6_r900_sixx/visual/base_link.dae" />
         </geometry>
         <xacro:material_kuka_pedestal />
@@ -24,5 +24,5 @@
         <origin xyz="0 0 0" rpy="0 0 0"/>
         <geometry>
-          <mesh filename="package://kuka_agilus_support/meshes/KR6R900sixx/collision/base_link.stl" />
+          <mesh filename="package://kuka_agilus_support/meshes/kr6_r900_sixx/collision/base_link.stl" />
         </geometry>
       </collision>
@@ -32,5 +32,5 @@
         <origin xyz="0 0 0" rpy="0 0 0"/>
         <geometry>
-          <mesh filename="package://kuka_agilus_support/meshes/KR6R900sixx/visual/link_1.dae" />
+          <mesh filename="package://kuka_agilus_support/meshes/kr6_r900_sixx/visual/link_1.dae" />
         </geometry>
         <xacro:material_kuka_orange />
@@ -39,5 +39,5 @@
         <origin xyz="0 0 0" rpy="0 0 0"/>
         <geometry>
-          <mesh filename="package://kuka_agilus_support/meshes/KR6R900sixx/collision/link_1.stl" />
+          <mesh filename="package://kuka_agilus_support/meshes/kr6_r900_sixx/collision/link_1.stl" />
         </geometry>
       </collision>
@@ -47,5 +47,5 @@
         <origin xyz="0 0 0" rpy="0 0 0"/>
         <geometry>
-          <mesh filename="package://kuka_agilus_support/meshes/KR6R900sixx/visual/link_2.dae"/>
+          <mesh filename="package://kuka_agilus_support/meshes/kr6_r900_sixx/visual/link_2.dae"/>
         </geometry>
         <xacro:material_kuka_orange />
@@ -54,5 +54,5 @@
         <origin xyz="0 0 0" rpy="0 0 0"/>
         <geometry>
-          <mesh filename="package://kuka_agilus_support/meshes/KR6R900sixx/collision/link_2.stl" />
+          <mesh filename="package://kuka_agilus_support/meshes/kr6_r900_sixx/collision/link_2.stl" />
         </geometry>
       </collision>
@@ -62,5 +62,5 @@
         <origin xyz="0 0 0" rpy="0 0 0"/>
         <geometry>
-          <mesh filename="package://kuka_agilus_support/meshes/KR6R900sixx/visual/link_3.dae" />
+          <mesh filename="package://kuka_agilus_support/meshes/kr6_r900_sixx/visual/link_3.dae" />
         </geometry>
         <xacro:material_kuka_orange />
@@ -69,5 +69,5 @@
         <origin xyz="0 0 0" rpy="0 0 0"/>
         <geometry>
-          <mesh filename="package://kuka_agilus_support/meshes/KR6R900sixx/collision/link_3.stl" />
+          <mesh filename="package://kuka_agilus_support/meshes/kr6_r900_sixx/collision/link_3.stl" />
         </geometry>
       </collision>
@@ -77,5 +77,5 @@
         <origin xyz="0 0 0" rpy="0 0 0"/>
         <geometry>
-          <mesh filename="package://kuka_agilus_support/meshes/KR6R900sixx/visual/link_4.dae" />
+          <mesh filename="package://kuka_agilus_support/meshes/kr6_r900_sixx/visual/link_4.dae" />
         </geometry>
         <xacro:material_kuka_orange />
@@ -84,5 +84,5 @@
         <origin xyz="0 0 0" rpy="0 0 0"/>
         <geometry>
-          <mesh filename="package://kuka_agilus_support/meshes/KR6R900sixx/collision/link_4.stl" />
+          <mesh filename="package://kuka_agilus_support/meshes/kr6_r900_sixx/collision/link_4.stl" />
         </geometry>
       </collision>
@@ -92,5 +92,5 @@
         <origin xyz="0 0 0" rpy="0 0 0"/>
         <geometry>
-          <mesh filename="package://kuka_agilus_support/meshes/KR6R900sixx/visual/link_5.dae" />
+          <mesh filename="package://kuka_agilus_support/meshes/kr6_r900_sixx/visual/link_5.dae" />
         </geometry>
         <xacro:material_kuka_orange />
@@ -99,5 +99,5 @@
         <origin xyz="0 0 0" rpy="0 0 0"/>
         <geometry>
-          <mesh filename="package://kuka_agilus_support/meshes/KR6R900sixx/collision/link_5.stl" />
+          <mesh filename="package://kuka_agilus_support/meshes/kr6_r900_sixx/collision/link_5.stl" />
         </geometry>
       </collision>
@@ -107,5 +107,5 @@
         <origin xyz="0 0 0" rpy="0 0 0"/>
         <geometry>
-          <mesh filename="package://kuka_agilus_support/meshes/KR6R900sixx/visual/link_6.dae" />
+          <mesh filename="package://kuka_agilus_support/meshes/kr6_r900_sixx/visual/link_6.dae" />
         </geometry>
         <xacro:material_kuka_pedestal />
@@ -114,5 +114,5 @@
         <origin xyz="0 0 0" rpy="0 0 0"/>
         <geometry>
-          <mesh filename="package://kuka_agilus_support/meshes/KR6R900sixx/collision/link_6.stl" />
+          <mesh filename="package://kuka_agilus_support/meshes/kr6_r900_sixx/collision/link_6.stl" />
         </geometry>
       </collision>
