Commit message: -sixx

File: kuka_agilus_support/urdf/kr6_r700_sixx.urdf.xacro (robot description, xacro)
@@ -1,6 +1,6 @@
 <?xml version="1.0"?>
-<robot xmlns:xacro="http://www.ros.org/wiki/xacro" name="kr6_r700_sixx">
+<robot xmlns:xacro="http://www.ros.org/wiki/xacro" name="kr6_r700-sixx">
 <!-- Import urdf file  -->
-<xacro:include filename="$(find kuka_agilus_support)/urdf/kr6_r700_sixx_macro.xacro"/>
+<xacro:include filename="$(find kuka_agilus_support)/urdf/kr6_r700-sixx_macro.xacro"/>
 <!-- Read parameters from rsi_config  -->
 <xacro:property name="rsi_config" value="$(find kuka_rsi_hw_interface)/config/rsi_config.yaml" />
@@ -10,5 +10,5 @@
 <!-- Read additional arguments  -->
 <xacro:arg name="use_fake_hardware" default="false" />
-<xacro:kuka_kr6_r700_sixx_robot prefix=""
+<xacro:kuka_kr6_r700-sixx_robot prefix=""
                   client_ip="${client_ip}"
                   client_port="${client_port}"

File: kuka_agilus_support/urdf/kr6_r700_sixx_macro.xacro (robot description, xacro)
@@ -5,8 +5,8 @@
   <xacro:include filename="$(find kuka_agilus_support)/urdf/kr_agilus_ros2_control.xacro" />
   <xacro:include filename="$(find kuka_agilus_support)/urdf/kr_agilus_transmission.xacro" />
-  <xacro:macro name="kuka_kr6_r700_sixx_robot" params="prefix client_ip client_port use_fake_hardware">
+  <xacro:macro name="kuka_kr6_r700-sixx_robot" params="prefix client_ip client_port use_fake_hardware">
     <!-- ros2 control instance -->
     <xacro:kuka_agilus_ros2_control
-    name="kr6_r700_sixx"
+    name="kr6_r700-sixx"
     prefix="${prefix}"
     client_ip="${client_ip}"
@@ -18,5 +18,5 @@
         <origin xyz="0 0 0" rpy="0 0 0" />
         <geometry>
-          <mesh filename="package://kuka_agilus_support/meshes/kr6_r700_sixx/visual/base_link.dae" />
+          <mesh filename="package://kuka_agilus_support/meshes/kr6_r700-sixx/visual/base_link.dae" />
         </geometry>
         <xacro:material_kuka_pedestal />
@@ -25,5 +25,5 @@
         <origin xyz="0 0 0" rpy="0 0 0" />
         <geometry>
-          <mesh filename="package://kuka_agilus_support/meshes/kr6_r700_sixx/collision/base_link.stl" />
+          <mesh filename="package://kuka_agilus_support/meshes/kr6_r700-sixx/collision/base_link.stl" />
         </geometry>
       </collision>
@@ -33,5 +33,5 @@
         <origin xyz="0 0 0" rpy="0 0 0" />
         <geometry>
-          <mesh filename="package://kuka_agilus_support/meshes/kr6_r700_sixx/visual/link_1.dae" />
+          <mesh filename="package://kuka_agilus_support/meshes/kr6_r700-sixx/visual/link_1.dae" />
         </geometry>
         <xacro:material_kuka_orange />
@@ -40,5 +40,5 @@
         <origin xyz="0 0 0" rpy="0 0 0" />
         <geometry>
-          <mesh filename="package://kuka_agilus_support/meshes/kr6_r700_sixx/collision/link_1.stl" />
+          <mesh filename="package://kuka_agilus_support/meshes/kr6_r700-sixx/collision/link_1.stl" />
         </geometry>
       </collision>
@@ -48,5 +48,5 @@
         <origin xyz="0 0 0" rpy="0 0 0" />
         <geometry>
-          <mesh filename="package://kuka_agilus_support/meshes/kr6_r700_sixx/visual/link_2.dae" />
+          <mesh filename="package://kuka_agilus_support/meshes/kr6_r700-sixx/visual/link_2.dae" />
         </geometry>
         <xacro:material_kuka_orange />
@@ -55,5 +55,5 @@
         <origin xyz="0 0 0" rpy="0 0 0" />
         <geometry>
-          <mesh filename="package://kuka_agilus_support/meshes/kr6_r700_sixx/collision/link_2.stl" />
+          <mesh filename="package://kuka_agilus_support/meshes/kr6_r700-sixx/collision/link_2.stl" />
         </geometry>
       </collision>
@@ -63,5 +63,5 @@
         <origin xyz="0 0 0" rpy="0 0 0" />
         <geometry>
-          <mesh filename="package://kuka_agilus_support/meshes/kr6_r700_sixx/visual/link_3.dae" />
+          <mesh filename="package://kuka_agilus_support/meshes/kr6_r700-sixx/visual/link_3.dae" />
         </geometry>
         <xacro:material_kuka_orange />
@@ -70,5 +70,5 @@
         <origin xyz="0 0 0" rpy="0 0 0" />
         <geometry>
-          <mesh filename="package://kuka_agilus_support/meshes/kr6_r700_sixx/collision/link_3.stl" />
+          <mesh filename="package://kuka_agilus_support/meshes/kr6_r700-sixx/collision/link_3.stl" />
         </geometry>
       </collision>
@@ -78,5 +78,5 @@
         <origin xyz="0 0 0" rpy="0 0 0" />
         <geometry>
-          <mesh filename="package://kuka_agilus_support/meshes/kr6_r700_sixx/visual/link_4.dae" />
+          <mesh filename="package://kuka_agilus_support/meshes/kr6_r700-sixx/visual/link_4.dae" />
         </geometry>
         <xacro:material_kuka_orange />
@@ -85,5 +85,5 @@
         <origin xyz="0 0 0" rpy="0 0 0" />
         <geometry>
-          <mesh filename="package://kuka_agilus_support/meshes/kr6_r700_sixx/collision/link_4.stl" />
+          <mesh filename="package://kuka_agilus_support/meshes/kr6_r700-sixx/collision/link_4.stl" />
         </geometry>
       </collision>
@@ -93,5 +93,5 @@
         <origin xyz="0 0 0" rpy="0 0 0" />
         <geometry>
-          <mesh filename="package://kuka_agilus_support/meshes/kr6_r700_sixx/visual/link_5.dae" />
+          <mesh filename="package://kuka_agilus_support/meshes/kr6_r700-sixx/visual/link_5.dae" />
         </geometry>
         <xacro:material_kuka_orange />
@@ -100,5 +100,5 @@
         <origin xyz="0 0 0" rpy="0 0 0" />
         <geometry>
-          <mesh filename="package://kuka_agilus_support/meshes/kr6_r700_sixx/collision/link_5.stl" />
+          <mesh filename="package://kuka_agilus_support/meshes/kr6_r700-sixx/collision/link_5.stl" />
         </geometry>
       </collision>
@@ -108,5 +108,5 @@
         <origin xyz="0 0 0" rpy="0 0 0" />
         <geometry>
-          <mesh filename="package://kuka_agilus_support/meshes/kr6_r700_sixx/visual/link_6.dae" />
+          <mesh filename="package://kuka_agilus_support/meshes/kr6_r700-sixx/visual/link_6.dae" />
         </geometry>
         <xacro:material_kuka_pedestal />
@@ -115,5 +115,5 @@
         <origin xyz="0 0 0" rpy="0 0 0" />
         <geometry>
-          <mesh filename="package://kuka_agilus_support/meshes/kr6_r700_sixx/collision/link_6.stl" />
+          <mesh filename="package://kuka_agilus_support/meshes/kr6_r700-sixx/collision/link_6.stl" />
         </geometry>
       </collision>

File: kuka_agilus_support/urdf/kr6_r900_sixx.urdf.xacro (robot description, xacro)
@@ -1,6 +1,6 @@
 <?xml version="1.0"?>
-<robot xmlns:xacro="http://www.ros.org/wiki/xacro" name="kr6_r900_sixx">
+<robot xmlns:xacro="http://www.ros.org/wiki/xacro" name="kr6_r900-sixx">
 <!-- Import urdf file  -->
-<xacro:include filename="$(find kuka_agilus_support)/urdf/kr6_r900_sixx_macro.xacro"/>
+<xacro:include filename="$(find kuka_agilus_support)/urdf/kr6_r900-sixx_macro.xacro"/>
 <!-- Read parameters from rsi_config  -->
 <xacro:property name="rsi_config" value="$(find kuka_rsi_hw_interface)/config/rsi_config.yaml" />
@@ -10,5 +10,5 @@
 <!-- Read additional arguments  -->
 <xacro:arg name="use_fake_hardware" default="false" />
-<xacro:kuka_kr6_r900_sixx_robot prefix=""
+<xacro:kuka_kr6_r900-sixx_robot prefix=""
                   client_ip="${client_ip}"
                   client_port="${client_port}"

File: kuka_agilus_support/urdf/kr6_r900_sixx_macro.xacro (robot description, xacro)
@@ -5,8 +5,8 @@
   <xacro:include filename="$(find kuka_agilus_support)/urdf/kr_agilus_ros2_control.xacro" />
   <xacro:include filename="$(find kuka_agilus_support)/urdf/kr_agilus_transmission.xacro" />
-  <xacro:macro name="kuka_kr6_r900_sixx_robot" params="prefix client_ip client_port use_fake_hardware">
+  <xacro:macro name="kuka_kr6_r900-sixx_robot" params="prefix client_ip client_port use_fake_hardware">
     <!-- ros2 control instance -->
     <xacro:kuka_agilus_ros2_control
-    name="kr6_r900_sixx"
+    name="kr6_r900-sixx"
     prefix="${prefix}"
     client_ip="${client_ip}"
@@ -18,5 +18,5 @@
         <origin xyz="0 0 0" rpy="0 0 0"/>
         <geometry>
-          <mesh filename="package://kuka_agilus_support/meshes/kr6_r900_sixx/visual/base_link.dae" />
+          <mesh filename="package://kuka_agilus_support/meshes/kr6_r900-sixx/visual/base_link.dae" />
         </geometry>
         <xacro:material_kuka_pedestal />
@@ -25,5 +25,5 @@
         <origin xyz="0 0 0" rpy="0 0 0"/>
         <geometry>
-          <mesh filename="package://kuka_agilus_support/meshes/kr6_r900_sixx/collision/base_link.stl" />
+          <mesh filename="package://kuka_agilus_support/meshes/kr6_r900-sixx/collision/base_link.stl" />
         </geometry>
       </collision>
@@ -33,5 +33,5 @@
         <origin xyz="0 0 0" rpy="0 0 0"/>
         <geometry>
-          <mesh filename="package://kuka_agilus_support/meshes/kr6_r900_sixx/visual/link_1.dae" />
+          <mesh filename="package://kuka_agilus_support/meshes/kr6_r900-sixx/visual/link_1.dae" />
         </geometry>
         <xacro:material_kuka_orange />
@@ -40,5 +40,5 @@
         <origin xyz="0 0 0" rpy="0 0 0"/>
         <geometry>
-          <mesh filename="package://kuka_agilus_support/meshes/kr6_r900_sixx/collision/link_1.stl" />
+          <mesh filename="package://kuka_agilus_support/meshes/kr6_r900-sixx/collision/link_1.stl" />
         </geometry>
       </collision>
@@ -48,5 +48,5 @@
         <origin xyz="0 0 0" rpy="0 0 0"/>
         <geometry>
-          <mesh filename="package://kuka_agilus_support/meshes/kr6_r900_sixx/visual/link_2.dae"/>
+          <mesh filename="package://kuka_agilus_support/meshes/kr6_r900-sixx/visual/link_2.dae"/>
         </geometry>
         <xacro:material_kuka_orange />
@@ -55,5 +55,5 @@
         <origin xyz="0 0 0" rpy="0 0 0"/>
         <geometry>
-          <mesh filename="package://kuka_agilus_support/meshes/kr6_r900_sixx/collision/link_2.stl" />
+          <mesh filename="package://kuka_agilus_support/meshes/kr6_r900-sixx/collision/link_2.stl" />
         </geometry>
       </collision>
@@ -63,5 +63,5 @@
         <origin xyz="0 0 0" rpy="0 0 0"/>
         <geometry>
-          <mesh filename="package://kuka_agilus_support/meshes/kr6_r900_sixx/visual/link_3.dae" />
+          <mesh filename="package://kuka_agilus_support/meshes/kr6_r900-sixx/visual/link_3.dae" />
         </geometry>
         <xacro:material_kuka_orange />
@@ -70,5 +70,5 @@
         <origin xyz="0 0 0" rpy="0 0 0"/>
         <geometry>
-          <mesh filename="package://kuka_agilus_support/meshes/kr6_r900_sixx/collision/link_3.stl" />
+          <mesh filename="package://kuka_agilus_support/meshes/kr6_r900-sixx/collision/link_3.stl" />
         </geometry>
       </collision>
@@ -78,5 +78,5 @@
         <origin xyz="0 0 0" rpy="0 0 0"/>
         <geometry>
-          <mesh filename="package://kuka_agilus_support/meshes/kr6_r900_sixx/visual/link_4.dae" />
+          <mesh filename="package://kuka_agilus_support/meshes/kr6_r900-sixx/visual/link_4.dae" />
         </geometry>
         <xacro:material_kuka_orange />
@@ -85,5 +85,5 @@
         <origin xyz="0 0 0" rpy="0 0 0"/>
         <geometry>
-          <mesh filename="package://kuka_agilus_support/meshes/kr6_r900_sixx/collision/link_4.stl" />
+          <mesh filename="package://kuka_agilus_support/meshes/kr6_r900-sixx/collision/link_4.stl" />
         </geometry>
       </collision>
@@ -93,5 +93,5 @@
         <origin xyz="0 0 0" rpy="0 0 0"/>
         <geometry>
-          <mesh filename="package://kuka_agilus_support/meshes/kr6_r900_sixx/visual/link_5.dae" />
+          <mesh filename="package://kuka_agilus_support/meshes/kr6_r900-sixx/visual/link_5.dae" />
         </geometry>
         <xacro:material_kuka_orange />
@@ -100,5 +100,5 @@
         <origin xyz="0 0 0" rpy="0 0 0"/>
         <geometry>
-          <mesh filename="package://kuka_agilus_support/meshes/kr6_r900_sixx/collision/link_5.stl" />
+          <mesh filename="package://kuka_agilus_support/meshes/kr6_r900-sixx/collision/link_5.stl" />
         </geometry>
       </collision>
@@ -108,5 +108,5 @@
         <origin xyz="0 0 0" rpy="0 0 0"/>
         <geometry>
-          <mesh filename="package://kuka_agilus_support/meshes/kr6_r900_sixx/visual/link_6.dae" />
+          <mesh filename="package://kuka_agilus_support/meshes/kr6_r900-sixx/visual/link_6.dae" />
         </geometry>
         <xacro:material_kuka_pedestal />
@@ -115,5 +115,5 @@
         <origin xyz="0 0 0" rpy="0 0 0"/>
         <geometry>
-          <mesh filename="package://kuka_agilus_support/meshes/kr6_r900_sixx/collision/link_6.stl" />
+          <mesh filename="package://kuka_agilus_support/meshes/kr6_r900-sixx/collision/link_6.stl" />
         </geometry>
       </collision>
