Commit message: Create unified structure for all support packages (#30)
* use lower case letters

* start iiwa renamings (not working yet)

* add prefix arg to iiwa

* metapackage

* mesh rename1

* mesh file rename

* iiwa urdf restruct

* iiwa fixes

* -sixx

* test launch files with fake hw

* test launc file with fake hw

* 7 axis rviz config

* extend moveit config joints for iiwa

* Update README.md

Co-authored-by: G.A. vd. Hoorn <g.a.vanderhoorn@tudelft.nl>

* remove dashes

* fix auto replace

* fix dash in readme

* manipulator for group name in srdf

* add joint_limits for iiwa

* maintainer email

* drivers rename

---------

Co-authored-by: Gergely Kovacs4 <gergely.kovacs4@kuka.com>
Co-authored-by: Aron Svastits <svastits1@gmail.com>
Co-authored-by: G.A. vd. Hoorn <g.a.vanderhoorn@tudelft.nl>

File: kuka_agilus_support/urdf/kr6_r700_sixx.urdf.xacro (robot description, xacro)
@@ -1,16 +1,8 @@
 <?xml version="1.0"?>
 <robot xmlns:xacro="http://www.ros.org/wiki/xacro" name="kr6_r700_sixx">
-<!-- Import urdf file  -->
-<xacro:include filename="$(find kuka_agilus_support)/urdf/kr6_r700_sixx_macro.xacro"/>
-<!-- Read parameters from rsi_config  -->
-<xacro:property name="rsi_config" value="$(find kuka_rsi_hw_interface)/config/rsi_config.yaml" />
-<xacro:property name="rsi_config_dict" value="${xacro.load_yaml(rsi_config)}"/>
-<xacro:property name="client_ip" value="${rsi_config_dict['client_ip']}" />
-<xacro:property name="client_port" value="${rsi_config_dict['client_port']}" />
-<!-- Read additional arguments  -->
-<xacro:arg name="use_fake_hardware" default="false" />
-<xacro:kuka_kr6_r700_sixx_robot prefix=""
-                  client_ip="${client_ip}"
-                  client_port="${client_port}"
-                  use_fake_hardware="$(arg use_fake_hardware)"/>
+  <!-- Import urdf file  -->
+  <xacro:include filename="$(find kuka_agilus_support)/urdf/kr6_r700_sixx_macro.xacro"/>
+  <!-- Read additional arguments  -->
+  <xacro:arg name="use_fake_hardware" default="false" />
+  <xacro:kuka_kr6_r700_sixx_robot prefix=""  use_fake_hardware="$(arg use_fake_hardware)"/>
 </robot>

File: kuka_agilus_support/urdf/kr6_r700_sixx_macro.xacro (robot description, xacro)
@@ -5,11 +5,9 @@
   <xacro:include filename="$(find kuka_agilus_support)/urdf/kr_agilus_ros2_control.xacro" />
   <xacro:include filename="$(find kuka_agilus_support)/urdf/kr_agilus_transmission.xacro" />
-  <xacro:macro name="kuka_kr6_r700_sixx_robot" params="prefix client_ip client_port use_fake_hardware">
+  <xacro:macro name="kuka_kr6_r700_sixx_robot" params="prefix use_fake_hardware">
     <!-- ros2 control instance -->
     <xacro:kuka_agilus_ros2_control
     name="kr6_r700_sixx"
     prefix="${prefix}"
-    client_ip="${client_ip}"
-    client_port="${client_port}"
     use_fake_hardware="${use_fake_hardware}" />
     <link name="${prefix}base_link"/>

File: kuka_agilus_support/urdf/kr6_r900_sixx.urdf.xacro (robot description, xacro)
@@ -1,16 +1,8 @@
 <?xml version="1.0"?>
 <robot xmlns:xacro="http://www.ros.org/wiki/xacro" name="kr6_r900_sixx">
-<!-- Import urdf file  -->
-<xacro:include filename="$(find kuka_agilus_support)/urdf/kr6_r900_sixx_macro.xacro"/>
-<!-- Read parameters from rsi_config  -->
-<xacro:property name="rsi_config" value="$(find kuka_rsi_hw_interface)/config/rsi_config.yaml" />
-<xacro:property name="rsi_config_dict" value="${xacro.load_yaml(rsi_config)}"/>
-<xacro:property name="client_ip" value="${rsi_config_dict['client_ip']}" />
-<xacro:property name="client_port" value="${rsi_config_dict['client_port']}" />
-<!-- Read additional arguments  -->
-<xacro:arg name="use_fake_hardware" default="false" />
-<xacro:kuka_kr6_r900_sixx_robot prefix=""
-                  client_ip="${client_ip}"
-                  client_port="${client_port}"
-                  use_fake_hardware="$(arg use_fake_hardware)"/>
+  <!-- Import urdf file  -->
+  <xacro:include filename="$(find kuka_agilus_support)/urdf/kr6_r900_sixx_macro.xacro"/>
+  <!-- Read additional arguments  -->
+  <xacro:arg name="use_fake_hardware" default="false" />
+  <xacro:kuka_kr6_r900_sixx_robot prefix="" use_fake_hardware="$(arg use_fake_hardware)"/>
 </robot>

File: kuka_agilus_support/urdf/kr6_r900_sixx_macro.xacro (robot description, xacro)
@@ -5,11 +5,9 @@
   <xacro:include filename="$(find kuka_agilus_support)/urdf/kr_agilus_ros2_control.xacro" />
   <xacro:include filename="$(find kuka_agilus_support)/urdf/kr_agilus_transmission.xacro" />
-  <xacro:macro name="kuka_kr6_r900_sixx_robot" params="prefix client_ip client_port use_fake_hardware">
+  <xacro:macro name="kuka_kr6_r900_sixx_robot" params="prefix use_fake_hardware">
     <!-- ros2 control instance -->
     <xacro:kuka_agilus_ros2_control
     name="kr6_r900_sixx"
     prefix="${prefix}"
-    client_ip="${client_ip}"
-    client_port="${client_port}"
     use_fake_hardware="${use_fake_hardware}" />
     <link name="${prefix}base_link"/>

File: kuka_lbr_iisy_support/urdf/lbr_iisy11_r1300.urdf.xacro (robot description, xacro)
@@ -1,24 +1,8 @@
 <?xml version="1.0"?>
-<robot xmlns:xacro="http://www.ros.org/wiki/xacro" name="LBRiisy11R1300">
-<!-- Import iisy urdf file  -->
-<xacro:include filename="$(find kuka_lbr_iisy_support)/urdf/lbr_iisy11_r1300_macro.xacro"/>
-<!-- Read parameters from eci_config  -->
-<xacro:property name="eci_config" value="$(find kuka_rox_hw_interface)/config/eci_config.yaml" />
-<xacro:property name="eci_config_dict" value="${xacro.load_yaml(eci_config)}"/>
-<xacro:property name="control_mode" value="${eci_config_dict['robot_manager']['ros__parameters']['control_mode']}" />
-<xacro:property name="client_ip" value="${eci_config_dict['robot_manager']['ros__parameters']['client_ip']}" />
-<xacro:property name="controller_ip" value="${eci_config_dict['robot_manager']['ros__parameters']['controller_ip']}" />
-<!-- Read QoS profile parameters  -->
-<xacro:property name="qos_config" value="$(find kuka_rox_hw_interface)/config/qos_profiles.yaml" />
-<xacro:property name="qos_config_dict" value="${xacro.load_yaml(qos_config)}"/>
-<xacro:property name="consequent_lost_packets" value="${qos_config_dict['rt_packet_loss_profile']['consequent_lost_packets']}" />
-<xacro:property name="lost_packets_in_timeframe" value="${qos_config_dict['rt_packet_loss_profile']['lost_packets_in_timeframe']}" />
-<xacro:property name="timeframe_ms" value="${qos_config_dict['rt_packet_loss_profile']['timeframe_ms']}" />
-<xacro:kuka_lbr11_r1300_robot prefix=""
-                  client_ip="${client_ip}"
-                  controller_ip="${controller_ip}"
-                  control_mode="${control_mode}"
-                  consequent_lost_packets="${consequent_lost_packets}"
-                  lost_packets_in_timeframe="${lost_packets_in_timeframe}"
-                  timeframe_ms="${timeframe_ms}"/>
+<robot xmlns:xacro="http://www.ros.org/wiki/xacro" name="lbr_iisy11_r1300">
+    <!-- Import iisy urdf file  -->
+    <xacro:include filename="$(find kuka_lbr_iisy_support)/urdf/lbr_iisy11_r1300_macro.xacro"/>
+    <!-- Read additional arguments  -->
+    <xacro:arg name="use_fake_hardware" default="false" />
+    <xacro:kuka_lbr_iisy11_r1300_robot prefix="" use_fake_hardware="$(arg use_fake_hardware)"/>
 </robot>

File: kuka_lbr_iisy_support/urdf/lbr_iisy11_r1300_macro.xacro (robot description, xacro)
@@ -1,19 +1,14 @@
 <?xml version="1.0" encoding="UTF-8"?>
-<robot xmlns:xacro="http://www.ros.org/wiki/xacro" name="LBRiisy11R1300">
+<robot xmlns:xacro="http://www.ros.org/wiki/xacro" name="lbr_iisy11_r1300">
   <!-- include helper xacros -->
   <xacro:include filename="$(find kuka_lbr_iisy_support)/urdf/lbr_iisy_ros2_control.xacro" />
   <xacro:include filename="$(find kuka_resources)/urdf/common_materials.xacro"/>
   <xacro:include filename="$(find kuka_lbr_iisy_support)/urdf/lbr_iisy_transmission.xacro" />
-  <xacro:macro name="kuka_lbr11_r1300_robot" params="prefix client_ip controller_ip control_mode consequent_lost_packets lost_packets_in_timeframe timeframe_ms">
+  <xacro:macro name="kuka_lbr_iisy11_r1300_robot" params="prefix use_fake_hardware:=false">
     <!-- ros2 control instance -->
     <xacro:kuka_lbr_iisy_ros2_control
-    name="LBRiisy11R1300"
+    name="lbr_iisy11_r1300"
     prefix="${prefix}"
-    client_ip="${client_ip}"
-    controller_ip="${controller_ip}"
-    control_mode="${control_mode}"
-    consequent_lost_packets="${consequent_lost_packets}"
-    lost_packets_in_timeframe="${lost_packets_in_timeframe}"
-    timeframe_ms="${timeframe_ms}" />
+    use_fake_hardware="${use_fake_hardware}" />
     <!-- links - main serial chain -->
     <!-- links - root element cannot have inertia, therefore a dummy base_link is needed -->
@@ -22,5 +17,5 @@
       <collision>
         <geometry>
-          <mesh filename="package://kuka_lbr_iisy_support/meshes/LBRiisy11R1300/collision/base_link.stl" />
+          <mesh filename="package://kuka_lbr_iisy_support/meshes/lbr_iisy11_r1300/collision/base_link.stl" />
         </geometry>
         <origin rpy="-0.0 0.0 -0.0" xyz="0.0 0.0 0.0" />
@@ -33,5 +28,5 @@
       <visual>
         <geometry>
-          <mesh filename="package://kuka_lbr_iisy_support/meshes/LBRiisy11R1300/visual/base_link.stl" />
+          <mesh filename="package://kuka_lbr_iisy_support/meshes/lbr_iisy11_r1300/visual/base_link.stl" />
         </geometry>
         <origin rpy="-0.0 0.0 -0.0" xyz="0.0 0.0 0.0" />
@@ -42,5 +37,5 @@
       <collision>
         <geometry>
-          <mesh filename="package://kuka_lbr_iisy_support/meshes/LBRiisy11R1300/collision/link_1.stl" />
+          <mesh filename="package://kuka_lbr_iisy_support/meshes/lbr_iisy11_r1300/collision/link_1.stl" />
         </geometry>
         <origin rpy="-0.0 0.0 -0.0" xyz="0.0 0.0 0.0" />
@@ -53,5 +48,5 @@
       <visual>
         <geometry>
-          <mesh filename="package://kuka_lbr_iisy_support/meshes/LBRiisy11R1300/visual/link_1.stl" />
+          <mesh filename="package://kuka_lbr_iisy_support/meshes/lbr_iisy11_r1300/visual/link_1.stl" />
         </geometry>
         <origin rpy="-0.0 0.0 -0.0" xyz="0.0 0.0 0.0" />
@@ -62,5 +57,5 @@
       <collision>
         <geometry>
-          <mesh filename="package://kuka_lbr_iisy_support/meshes/LBRiisy11R1300/collision/link_2.stl" />
+          <mesh filename="package://kuka_lbr_iisy_support/meshes/lbr_iisy11_r1300/collision/link_2.stl" />
         </geometry>
         <origin rpy="-0.0 0.0 -0.0" xyz="0.0 0.0 0.0" />
@@ -73,5 +68,5 @@
       <visual>
         <geometry>
-          <mesh filename="package://kuka_lbr_iisy_support/meshes/LBRiisy11R1300/visual/link_2.stl" />
+          <mesh filename="package://kuka_lbr_iisy_support/meshes/lbr_iisy11_r1300/visual/link_2.stl" />
         </geometry>
         <origin rpy="-0.0 0.0 -0.0" xyz="0.0 0.0 0.0" />
@@ -82,5 +77,5 @@
       <collision>
         <geometry>
-          <mesh filename="package://kuka_lbr_iisy_support/meshes/LBRiisy11R1300/collision/link_3.stl" />
+          <mesh filename="package://kuka_lbr_iisy_support/meshes/lbr_iisy11_r1300/collision/link_3.stl" />
         </geometry>
         <origin rpy="-0.0 0.0 -0.0" xyz="0.0 0.0 0.0" />
@@ -93,5 +88,5 @@
       <visual>
         <geometry>
-          <mesh filename="package://kuka_lbr_iisy_support/meshes/LBRiisy11R1300/visual/link_3.stl" />
+          <mesh filename="package://kuka_lbr_iisy_support/meshes/lbr_iisy11_r1300/visual/link_3.stl" />
         </geometry>
         <origin rpy="-0.0 0.0 -0.0" xyz="0.0 0.0 0.0" />
@@ -102,5 +97,5 @@
       <collision>
         <geometry>
-          <mesh filename="package://kuka_lbr_iisy_support/meshes/LBRiisy11R1300/collision/link_4.stl" />
+          <mesh filename="package://kuka_lbr_iisy_support/meshes/lbr_iisy11_r1300/collision/link_4.stl" />
         </geometry>
         <origin rpy="-0.0 0.0 -0.0" xyz="0.0 0.0 0.0" />
@@ -113,5 +108,5 @@
       <visual>
         <geometry>
-          <mesh filename="package://kuka_lbr_iisy_support/meshes/LBRiisy11R1300/visual/link_4.stl" />
+          <mesh filename="package://kuka_lbr_iisy_support/meshes/lbr_iisy11_r1300/visual/link_4.stl" />
         </geometry>
         <origin rpy="-0.0 0.0 -0.0" xyz="0.0 0.0 0.0" />
@@ -122,5 +117,5 @@
       <collision>
         <geometry>
-          <mesh filename="package://kuka_lbr_iisy_support/meshes/LBRiisy11R1300/collision/link_5.stl" />
+          <mesh filename="package://kuka_lbr_iisy_support/meshes/lbr_iisy11_r1300/collision/link_5.stl" />
         </geometry>
         <origin rpy="-0.0 0.0 -0.0" xyz="0.0 0.0 0.0" />
@@ -133,5 +128,5 @@
       <visual>
         <geometry>
-          <mesh filename="package://kuka_lbr_iisy_support/meshes/LBRiisy11R1300/visual/link_5.stl" />
+          <mesh filename="package://kuka_lbr_iisy_support/meshes/lbr_iisy11_r1300/visual/link_5.stl" />
         </geometry>
         <origin rpy="-0.0 0.0 -0.0" xyz="0.0 0.0 0.0" />
@@ -142,5 +137,5 @@
       <collision>
         <geometry>
-          <mesh filename="package://kuka_lbr_iisy_support/meshes/LBRiisy11R1300/collision/link_6.stl" />
+          <mesh filename="package://kuka_lbr_iisy_support/meshes/lbr_iisy11_r1300/collision/link_6.stl" />
         </geometry>
         <origin rpy="-0.0 0.0 -0.0" xyz="0.0 0.0 0.0" />
@@ -153,5 +148,5 @@
       <visual>
         <geometry>
-          <mesh filename="package://kuka_lbr_iisy_support/meshes/LBRiisy11R1300/visual/link_6.stl" />
+          <mesh filename="package://kuka_lbr_iisy_support/meshes/lbr_iisy11_r1300/visual/link_6.stl" />
         </geometry>
         <origin rpy="-0.0 0.0 -0.0" xyz="0.0 0.0 0.0" />

File: kuka_lbr_iisy_support/urdf/lbr_iisy15_r930.urdf.xacro (robot description, xacro)
@@ -1,24 +1,8 @@
 <?xml version="1.0"?>
-<robot xmlns:xacro="http://www.ros.org/wiki/xacro" name="LBRiisy15R930">
-<!-- Import iisy urdf file  -->
-<xacro:include filename="$(find kuka_lbr_iisy_support)/urdf/lbr_iisy15_r930_macro.xacro"/>
-<!-- Read parameters from eci_config  -->
-<xacro:property name="eci_config" value="$(find kuka_rox_hw_interface)/config/eci_config.yaml" />
-<xacro:property name="eci_config_dict" value="${xacro.load_yaml(eci_config)}"/>
-<xacro:property name="control_mode" value="${eci_config_dict['robot_manager']['ros__parameters']['control_mode']}" />
-<xacro:property name="client_ip" value="${eci_config_dict['robot_manager']['ros__parameters']['client_ip']}" />
-<xacro:property name="controller_ip" value="${eci_config_dict['robot_manager']['ros__parameters']['controller_ip']}" />
-<!-- Read QoS profile parameters  -->
-<xacro:property name="qos_config" value="$(find kuka_rox_hw_interface)/config/qos_profiles.yaml" />
-<xacro:property name="qos_config_dict" value="${xacro.load_yaml(qos_config)}"/>
-<xacro:property name="consequent_lost_packets" value="${qos_config_dict['rt_packet_loss_profile']['consequent_lost_packets']}" />
-<xacro:property name="lost_packets_in_timeframe" value="${qos_config_dict['rt_packet_loss_profile']['lost_packets_in_timeframe']}" />
-<xacro:property name="timeframe_ms" value="${qos_config_dict['rt_packet_loss_profile']['timeframe_ms']}" />
-<xacro:kuka_lbr15_r930_robot prefix=""
-                  client_ip="${client_ip}"
-                  controller_ip="${controller_ip}"
-                  control_mode="${control_mode}"
-                  consequent_lost_packets="${consequent_lost_packets}"
-                  lost_packets_in_timeframe="${lost_packets_in_timeframe}"
-                  timeframe_ms="${timeframe_ms}"/>
+<robot xmlns:xacro="http://www.ros.org/wiki/xacro" name="lbr_iisy15_r930">
+    <!-- Import iisy urdf file  -->
+    <xacro:include filename="$(find kuka_lbr_iisy_support)/urdf/lbr_iisy15_r930_macro.xacro"/>
+    <!-- Read additional arguments  -->
+    <xacro:arg name="use_fake_hardware" default="false" />
+    <xacro:kuka_lbr_iisy15_r930_robot prefix="" use_fake_hardware="$(arg use_fake_hardware)"/>
 </robot>

File: kuka_lbr_iisy_support/urdf/lbr_iisy15_r930_macro.xacro (robot description, xacro)
@@ -1,19 +1,14 @@
 <?xml version="1.0" encoding="UTF-8"?>
-<robot xmlns:xacro="http://www.ros.org/wiki/xacro" name="LBRiisy15R930">
+<robot xmlns:xacro="http://www.ros.org/wiki/xacro" name="lbr_iisy15_r930">
   <!-- include helper xacros -->
   <xacro:include filename="$(find kuka_lbr_iisy_support)/urdf/lbr_iisy_ros2_control.xacro" />
   <xacro:include filename="$(find kuka_resources)/urdf/common_materials.xacro"/>
   <xacro:include filename="$(find kuka_lbr_iisy_support)/urdf/lbr_iisy_transmission.xacro" />
-  <xacro:macro name="kuka_lbr15_r930_robot" params="prefix client_ip controller_ip control_mode consequent_lost_packets lost_packets_in_timeframe timeframe_ms">
+  <xacro:macro name="kuka_lbr_iisy15_r930_robot" params="prefix use_fake_hardware:=false">
     <!-- ros2 control instance -->
     <xacro:kuka_lbr_iisy_ros2_control
-    name="LBRiisy15R930"
+    name="lbr_iisy15_r930"
     prefix="${prefix}"
-    client_ip="${client_ip}"
-    controller_ip="${controller_ip}"
-    control_mode="${control_mode}"
-    consequent_lost_packets="${consequent_lost_packets}"
-    lost_packets_in_timeframe="${lost_packets_in_timeframe}"
-    timeframe_ms="${timeframe_ms}" />
+    use_fake_hardware="${use_fake_hardware}" />
     <!-- links - main serial chain -->
     <!-- links - root element cannot have inertia, therefore a dummy base_link is needed -->
@@ -22,5 +17,5 @@
       <collision>
         <geometry>
-          <mesh filename="package://kuka_lbr_iisy_support/meshes/LBRiisy15R930/collision/base_link.stl" />
+          <mesh filename="package://kuka_lbr_iisy_support/meshes/lbr_iisy15_r930/collision/base_link.stl" />
         </geometry>
         <origin rpy="-0.0 0.0 -0.0" xyz="0.0 0.0 0.0" />
@@ -33,5 +28,5 @@
       <visual>
         <geometry>
-          <mesh filename="package://kuka_lbr_iisy_support/meshes/LBRiisy15R930/visual/base_link.stl" />
+          <mesh filename="package://kuka_lbr_iisy_support/meshes/lbr_iisy15_r930/visual/base_link.stl" />
         </geometry>
         <origin rpy="-0.0 0.0 -0.0" xyz="0.0 0.0 0.0" />
@@ -42,5 +37,5 @@
       <collision>
         <geometry>
-          <mesh filename="package://kuka_lbr_iisy_support/meshes/LBRiisy15R930/collision/link_1.stl" />
+          <mesh filename="package://kuka_lbr_iisy_support/meshes/lbr_iisy15_r930/collision/link_1.stl" />
         </geometry>
         <origin rpy="-0.0 0.0 -0.0" xyz="0.0 0.0 0.0" />
@@ -53,5 +48,5 @@
       <visual>
         <geometry>
-          <mesh filename="package://kuka_lbr_iisy_support/meshes/LBRiisy15R930/visual/link_1.stl" />
+          <mesh filename="package://kuka_lbr_iisy_support/meshes/lbr_iisy15_r930/visual/link_1.stl" />
         </geometry>
         <origin rpy="-0.0 0.0 -0.0" xyz="0.0 0.0 0.0" />
@@ -62,5 +57,5 @@
       <collision>
         <geometry>
-          <mesh filename="package://kuka_lbr_iisy_support/meshes/LBRiisy15R930/collision/link_2.stl" />
+          <mesh filename="package://kuka_lbr_iisy_support/meshes/lbr_iisy15_r930/collision/link_2.stl" />
         </geometry>
         <origin rpy="-0.0 0.0 -0.0" xyz="0.0 0.0 0.0" />
@@ -73,5 +68,5 @@
       <visual>
         <geometry>
-          <mesh filename="package://kuka_lbr_iisy_support/meshes/LBRiisy15R930/visual/link_2.stl" />
+          <mesh filename="package://kuka_lbr_iisy_support/meshes/lbr_iisy15_r930/visual/link_2.stl" />
         </geometry>
         <origin rpy="-0.0 0.0 -0.0" xyz="0.0 0.0 0.0" />
@@ -82,5 +77,5 @@
       <collision>
         <geometry>
-          <mesh filename="package://kuka_lbr_iisy_support/meshes/LBRiisy15R930/collision/link_3.stl" />
+          <mesh filename="package://kuka_lbr_iisy_support/meshes/lbr_iisy15_r930/collision/link_3.stl" />
         </geometry>
         <origin rpy="-0.0 0.0 -0.0" xyz="0.0 0.0 0.0" />
@@ -93,5 +88,5 @@
       <visual>
         <geometry>
-          <mesh filename="package://kuka_lbr_iisy_support/meshes/LBRiisy15R930/visual/link_3.stl" />
+          <mesh filename="package://kuka_lbr_iisy_support/meshes/lbr_iisy15_r930/visual/link_3.stl" />
         </geometry>
         <origin rpy="-0.0 0.0 -0.0" xyz="0.0 0.0 0.0" />
@@ -102,5 +97,5 @@
       <collision>
         <geometry>
-          <mesh filename="package://kuka_lbr_iisy_support/meshes/LBRiisy15R930/collision/link_4.stl" />
+          <mesh filename="package://kuka_lbr_iisy_support/meshes/lbr_iisy15_r930/collision/link_4.stl" />
         </geometry>
         <origin rpy="-0.0 0.0 -0.0" xyz="0.0 0.0 0.0" />
@@ -113,5 +108,5 @@
       <visual>
         <geometry>
-          <mesh filename="package://kuka_lbr_iisy_support/meshes/LBRiisy15R930/visual/link_4.stl" />
+          <mesh filename="package://kuka_lbr_iisy_support/meshes/lbr_iisy15_r930/visual/link_4.stl" />
         </geometry>
         <origin rpy="-0.0 0.0 -0.0" xyz="0.0 0.0 0.0" />
@@ -122,5 +117,5 @@
       <collision>
         <geometry>
-          <mesh filename="package://kuka_lbr_iisy_support/meshes/LBRiisy15R930/collision/link_5.stl" />
+          <mesh filename="package://kuka_lbr_iisy_support/meshes/lbr_iisy15_r930/collision/link_5.stl" />
         </geometry>
         <origin rpy="-0.0 0.0 -0.0" xyz="0.0 0.0 0.0" />
@@ -133,5 +128,5 @@
       <visual>
         <geometry>
-          <mesh filename="package://kuka_lbr_iisy_support/meshes/LBRiisy15R930/visual/link_5.stl" />
+          <mesh filename="package://kuka_lbr_iisy_support/meshes/lbr_iisy15_r930/visual/link_5.stl" />
         </geometry>
         <origin rpy="-0.0 0.0 -0.0" xyz="0.0 0.0 0.0" />
@@ -142,5 +137,5 @@
       <collision>
         <geometry>
-          <mesh filename="package://kuka_lbr_iisy_support/meshes/LBRiisy15R930/collision/link_6.stl" />
+          <mesh filename="package://kuka_lbr_iisy_support/meshes/lbr_iisy15_r930/collision/link_6.stl" />
         </geometry>
         <origin rpy="-0.0 0.0 -0.0" xyz="0.0 0.0 0.0" />
@@ -153,5 +148,5 @@
       <visual>
         <geometry>
-          <mesh filename="package://kuka_lbr_iisy_support/meshes/LBRiisy15R930/visual/link_6.stl" />
+          <mesh filename="package://kuka_lbr_iisy_support/meshes/lbr_iisy15_r930/visual/link_6.stl" />
         </geometry>
         <origin rpy="-0.0 0.0 -0.0" xyz="0.0 0.0 0.0" />
