Commit message: Create unified structure for all support packages (#30)
* use lower case letters

* start iiwa renamings (not working yet)

* add prefix arg to iiwa

* metapackage

* mesh rename1

* mesh file rename

* iiwa urdf restruct

* iiwa fixes

* -sixx

* test launch files with fake hw

* test launc file with fake hw

* 7 axis rviz config

* extend moveit config joints for iiwa

* Update README.md

Co-authored-by: G.A. vd. Hoorn <g.a.vanderhoorn@tudelft.nl>

* remove dashes

* fix auto replace

* fix dash in readme

* manipulator for group name in srdf

* add joint_limits for iiwa

* maintainer email

* drivers rename

---------

Co-authored-by: Gergely Kovacs4 <gergely.kovacs4@kuka.com>
Co-authored-by: Aron Svastits <svastits1@gmail.com>
Co-authored-by: G.A. vd. Hoorn <g.a.vanderhoorn@tudelft.nl>

File: kuka_lbr_iisy_support/urdf/lbr_iisy3_r760.urdf.xacro (robot description, xacro)
@@ -1,27 +1,8 @@
 <?xml version="1.0"?>
-<robot xmlns:xacro="http://www.ros.org/wiki/xacro" name="LBRiisy3R760">
-<!-- Import iisy urdf file  -->
-<xacro:include filename="$(find kuka_lbr_iisy_support)/urdf/lbr_iisy3_r760_macro.xacro"/>
-<!-- Read parameters from eci_config  -->
-<xacro:property name="eci_config" value="$(find kuka_rox_hw_interface)/config/eci_config.yaml" />
-<xacro:property name="eci_config_dict" value="${xacro.load_yaml(eci_config)}"/>
-<xacro:property name="control_mode" value="${eci_config_dict['robot_manager']['ros__parameters']['control_mode']}" />
-<xacro:property name="client_ip" value="${eci_config_dict['robot_manager']['ros__parameters']['client_ip']}" />
-<xacro:property name="controller_ip" value="${eci_config_dict['robot_manager']['ros__parameters']['controller_ip']}" />
-<!-- Read QoS profile parameters  -->
-<xacro:property name="qos_config" value="$(find kuka_rox_hw_interface)/config/qos_profiles.yaml" />
-<xacro:property name="qos_config_dict" value="${xacro.load_yaml(qos_config)}"/>
-<xacro:property name="consequent_lost_packets" value="${qos_config_dict['rt_packet_loss_profile']['consequent_lost_packets']}" />
-<xacro:property name="lost_packets_in_timeframe" value="${qos_config_dict['rt_packet_loss_profile']['lost_packets_in_timeframe']}" />
-<xacro:property name="timeframe_ms" value="${qos_config_dict['rt_packet_loss_profile']['timeframe_ms']}" />
-<!-- Read additional arguments  -->
-<xacro:arg name="use_fake_hardware" default="false" />
-<xacro:kuka_lbr3_r760_robot prefix=""
-                  client_ip="${client_ip}"
-                  controller_ip="${controller_ip}"
-                  control_mode="${control_mode}"
-                  consequent_lost_packets="${consequent_lost_packets}"
-                  lost_packets_in_timeframe="${lost_packets_in_timeframe}"
-                  timeframe_ms="${timeframe_ms}"
-                  use_fake_hardware="$(arg use_fake_hardware)"/>
+<robot xmlns:xacro="http://www.ros.org/wiki/xacro" name="lbr_iisy3_r760">
+    <!-- Import iisy urdf file  -->
+    <xacro:include filename="$(find kuka_lbr_iisy_support)/urdf/lbr_iisy3_r760_macro.xacro"/>
+    <!-- Read additional arguments  -->
+    <xacro:arg name="use_fake_hardware" default="false" />
+    <xacro:kuka_lbr_iisy3_r760_robot prefix="" use_fake_hardware="$(arg use_fake_hardware)"/>
 </robot>

File: kuka_lbr_iisy_support/urdf/lbr_iisy3_r760_macro.xacro (robot description, xacro)
@@ -1,19 +1,13 @@
 <?xml version="1.0" encoding="UTF-8"?>
-<robot xmlns:xacro="http://www.ros.org/wiki/xacro" name="LBRiisy3R760">
+<robot xmlns:xacro="http://www.ros.org/wiki/xacro" name="lbr_iisy3_r760">
   <!-- include helper xacros -->
   <xacro:include filename="$(find kuka_lbr_iisy_support)/urdf/lbr_iisy_ros2_control.xacro" />
   <xacro:include filename="$(find kuka_resources)/urdf/common_materials.xacro"/>
   <xacro:include filename="$(find kuka_lbr_iisy_support)/urdf/lbr_iisy_transmission.xacro" />
-  <xacro:macro name="kuka_lbr3_r760_robot" params="prefix client_ip controller_ip control_mode consequent_lost_packets lost_packets_in_timeframe timeframe_ms use_fake_hardware:=false">
+  <xacro:macro name="kuka_lbr_iisy3_r760_robot" params="prefix use_fake_hardware:=false">
     <!-- ros2 control instance -->
     <xacro:kuka_lbr_iisy_ros2_control
-    name="LBRiisy3R760"
+    name="lbr_iisy3_r760"
     prefix="${prefix}"
-    client_ip="${client_ip}"
-    controller_ip="${controller_ip}"
-    control_mode="${control_mode}"
-    consequent_lost_packets="${consequent_lost_packets}"
-    lost_packets_in_timeframe="${lost_packets_in_timeframe}"
-    timeframe_ms="${timeframe_ms}"
     use_fake_hardware="${use_fake_hardware}" />
     <!-- links - main serial chain -->
@@ -23,5 +17,5 @@
       <collision>
         <geometry>
-          <mesh filename="package://kuka_lbr_iisy_support/meshes/LBRiisy3R760/collision/base_link.stl" />
+          <mesh filename="package://kuka_lbr_iisy_support/meshes/lbr_iisy3_r760/collision/base_link.stl" />
         </geometry>
         <origin rpy="-0.0 0.0 -0.0" xyz="0.0 0.0 0.0" />
@@ -34,5 +28,5 @@
       <visual>
         <geometry>
-          <mesh filename="package://kuka_lbr_iisy_support/meshes/LBRiisy3R760/visual/base_link.stl" />
+          <mesh filename="package://kuka_lbr_iisy_support/meshes/lbr_iisy3_r760/visual/base_link.stl" />
         </geometry>
         <origin rpy="-0.0 0.0 -0.0" xyz="0.0 0.0 0.0" />
@@ -43,5 +37,5 @@
       <collision>
         <geometry>
-          <mesh filename="package://kuka_lbr_iisy_support/meshes/LBRiisy3R760/collision/link_1.stl" />
+          <mesh filename="package://kuka_lbr_iisy_support/meshes/lbr_iisy3_r760/collision/link_1.stl" />
         </geometry>
         <origin rpy="-0.0 0.0 -0.0" xyz="0.0 0.0 0.0" />
@@ -54,5 +48,5 @@
       <visual>
         <geometry>
-          <mesh filename="package://kuka_lbr_iisy_support/meshes/LBRiisy3R760/visual/link_1.stl" />
+          <mesh filename="package://kuka_lbr_iisy_support/meshes/lbr_iisy3_r760/visual/link_1.stl" />
         </geometry>
         <origin rpy="-0.0 0.0 -0.0" xyz="0.0 0.0 0.0" />
@@ -63,5 +57,5 @@
       <collision>
         <geometry>
-          <mesh filename="package://kuka_lbr_iisy_support/meshes/LBRiisy3R760/collision/link_2.stl" />
+          <mesh filename="package://kuka_lbr_iisy_support/meshes/lbr_iisy3_r760/collision/link_2.stl" />
         </geometry>
         <origin rpy="-0.0 0.0 -0.0" xyz="0.0 0.0 0.0" />
@@ -74,5 +68,5 @@
       <visual>
         <geometry>
-          <mesh filename="package://kuka_lbr_iisy_support/meshes/LBRiisy3R760/visual/link_2.stl" />
+          <mesh filename="package://kuka_lbr_iisy_support/meshes/lbr_iisy3_r760/visual/link_2.stl" />
         </geometry>
         <origin rpy="-0.0 0.0 -0.0" xyz="0.0 0.0 0.0" />
@@ -83,5 +77,5 @@
       <collision>
         <geometry>
-          <mesh filename="package://kuka_lbr_iisy_support/meshes/LBRiisy3R760/collision/link_3.stl" />
+          <mesh filename="package://kuka_lbr_iisy_support/meshes/lbr_iisy3_r760/collision/link_3.stl" />
         </geometry>
         <origin rpy="-0.0 0.0 -0.0" xyz="0.0 0.0 0.0" />
@@ -94,5 +88,5 @@
       <visual>
         <geometry>
-          <mesh filename="package://kuka_lbr_iisy_support/meshes/LBRiisy3R760/visual/link_3.stl" />
+          <mesh filename="package://kuka_lbr_iisy_support/meshes/lbr_iisy3_r760/visual/link_3.stl" />
         </geometry>
         <origin rpy="-0.0 0.0 -0.0" xyz="0.0 0.0 0.0" />
@@ -103,5 +97,5 @@
       <collision>
         <geometry>
-          <mesh filename="package://kuka_lbr_iisy_support/meshes/LBRiisy3R760/collision/link_4.stl" />
+          <mesh filename="package://kuka_lbr_iisy_support/meshes/lbr_iisy3_r760/collision/link_4.stl" />
         </geometry>
         <origin rpy="-0.0 0.0 -0.0" xyz="0.0 0.0 0.0" />
@@ -114,5 +108,5 @@
       <visual>
         <geometry>
-          <mesh filename="package://kuka_lbr_iisy_support/meshes/LBRiisy3R760/visual/link_4.stl" />
+          <mesh filename="package://kuka_lbr_iisy_support/meshes/lbr_iisy3_r760/visual/link_4.stl" />
         </geometry>
         <origin rpy="-0.0 0.0 -0.0" xyz="0.0 0.0 0.0" />
@@ -123,5 +117,5 @@
       <collision>
         <geometry>
-          <mesh filename="package://kuka_lbr_iisy_support/meshes/LBRiisy3R760/collision/link_5.stl" />
+          <mesh filename="package://kuka_lbr_iisy_support/meshes/lbr_iisy3_r760/collision/link_5.stl" />
         </geometry>
         <origin rpy="-0.0 0.0 -0.0" xyz="0.0 0.0 0.0" />
@@ -134,5 +128,5 @@
       <visual>
         <geometry>
-          <mesh filename="package://kuka_lbr_iisy_support/meshes/LBRiisy3R760/visual/link_5.stl" />
+          <mesh filename="package://kuka_lbr_iisy_support/meshes/lbr_iisy3_r760/visual/link_5.stl" />
         </geometry>
         <origin rpy="-0.0 0.0 -0.0" xyz="0.0 0.0 0.0" />
@@ -143,5 +137,5 @@
       <collision>
         <geometry>
-          <mesh filename="package://kuka_lbr_iisy_support/meshes/LBRiisy3R760/collision/link_6.stl" />
+          <mesh filename="package://kuka_lbr_iisy_support/meshes/lbr_iisy3_r760/collision/link_6.stl" />
         </geometry>
         <origin rpy="-0.0 0.0 -0.0" xyz="0.0 0.0 0.0" />
@@ -154,5 +148,5 @@
       <visual>
         <geometry>
-          <mesh filename="package://kuka_lbr_iisy_support/meshes/LBRiisy3R760/visual/link_6.stl" />
+          <mesh filename="package://kuka_lbr_iisy_support/meshes/lbr_iisy3_r760/visual/link_6.stl" />
         </geometry>
         <origin rpy="-0.0 0.0 -0.0" xyz="0.0 0.0 0.0" />

Commit message: add external axes integration possibility for all agilus

File: kuka_agilus_support/urdf/kr6_r700_sixx.urdf.xacro (robot description, xacro)
@@ -20,7 +20,11 @@
   <xacro:arg name="pitch" default="0"/>
   <xacro:arg name="yaw" default="0"/>
-  <xacro:kuka_agilus_ros2_control name="$(arg prefix)kr6_r700_sixx" driver_version="$(arg driver_version)" client_ip="$(arg client_ip)" client_port="$(arg client_port)" controller_ip="$(arg controller_ip)" prefix="$(arg prefix)" mode="$(arg mode)" use_gpio="$(arg use_gpio)" roundtrip_time="$(arg roundtrip_time)" verify_robot_model="$(arg verify_robot_model)"/>
-  <xacro:kuka_kr6_r700_sixx_robot prefix="$(arg prefix)" package_name="kuka_agilus_support">
+  <xacro:kuka_agilus_ros2_control name="$(arg prefix)kr6_r700_sixx" driver_version="$(arg driver_version)" client_ip="$(arg client_ip)" client_port="$(arg client_port)" controller_ip="$(arg controller_ip)" prefix="$(arg prefix)" mode="$(arg mode)" use_gpio="$(arg use_gpio)" roundtrip_time="$(arg roundtrip_time)" verify_robot_model="$(arg verify_robot_model)" use_ext_axes="false">
+    <ext_axes_ros2_control_joints/>
+  </xacro:kuka_agilus_ros2_control>
+  <xacro:kuka_kr6_r700_sixx_robot prefix="$(arg prefix)" package_name="kuka_agilus_support" use_ext_axes="false">
     <origin xyz="$(arg x) $(arg y) $(arg z)" rpy="$(arg roll) $(arg pitch) $(arg yaw)"/>
+    <ext_axes_links/>
+    <ext_axes_joints/>
   </xacro:kuka_kr6_r700_sixx_robot>
 </robot>

File: kuka_agilus_support/urdf/kr6_r700_sixx_macro.xacro (robot description, xacro)
@@ -4,7 +4,10 @@
   <xacro:include filename="$(find kuka_resources)/urdf/common_constants.xacro"/>
   <xacro:include filename="$(find kuka_resources)/urdf/common_materials.xacro"/>
-  <xacro:macro name="kuka_kr6_r700_sixx_robot" params="prefix package_name *origin">
+  <xacro:macro name="kuka_kr6_r700_sixx_robot" params="prefix package_name use_ext_axes *origin **ext_axes_links **ext_axes_joints">
     <!-- links - main serial chain -->
     <link name="world"/>
+    <xacro:if value="${use_ext_axes}">
+      <xacro:insert_block name="ext_axes_links"/>
+    </xacro:if>
     <link name="${prefix}base_link">
       <visual>
@@ -114,9 +117,14 @@
     <!-- Following REP199, this frame shall be use to attach EEF or other equipment -->
     <link name="${prefix}flange"/>
-    <joint name="${prefix}world-base_link" type="fixed">
-      <parent link="world"/>
-      <child link="${prefix}base_link"/>
-      <xacro:insert_block name="origin"/>
-    </joint>
+    <xacro:if value="${use_ext_axes}">
+      <xacro:insert_block name="ext_axes_joints"/>
+    </xacro:if>
+    <xacro:unless value="${use_ext_axes}">
+      <joint name="${prefix}world-base_link" type="fixed">
+        <parent link="world"/>
+        <child link="${prefix}base_link"/>
+        <xacro:insert_block name="origin"/>
+      </joint>
+    </xacro:unless>
     <joint name="${prefix}joint_1" type="revolute">
       <origin xyz="0 0 0.4" rpy="0 0 0"/>

File: kuka_agilus_support/urdf/kr6_r900_sixx.urdf.xacro (robot description, xacro)
@@ -20,7 +20,11 @@
   <xacro:arg name="pitch" default="0"/>
   <xacro:arg name="yaw" default="0"/>
-  <xacro:kuka_agilus_ros2_control name="$(arg prefix)kr6_r900_sixx" driver_version="$(arg driver_version)" client_ip="$(arg client_ip)" client_port="$(arg client_port)" controller_ip="$(arg controller_ip)" prefix="$(arg prefix)" mode="$(arg mode)" use_gpio="$(arg use_gpio)" roundtrip_time="$(arg roundtrip_time)" verify_robot_model="$(arg verify_robot_model)"/>
-  <xacro:kuka_kr6_r900_sixx_robot prefix="$(arg prefix)" package_name="kuka_agilus_support">
+  <xacro:kuka_agilus_ros2_control name="$(arg prefix)kr6_r900_sixx" driver_version="$(arg driver_version)" client_ip="$(arg client_ip)" client_port="$(arg client_port)" controller_ip="$(arg controller_ip)" prefix="$(arg prefix)" mode="$(arg mode)" use_gpio="$(arg use_gpio)" roundtrip_time="$(arg roundtrip_time)" verify_robot_model="$(arg verify_robot_model)" use_ext_axes="false">
+    <ext_axes_ros2_control_joints/>
+  </xacro:kuka_agilus_ros2_control>
+  <xacro:kuka_kr6_r900_sixx_robot prefix="$(arg prefix)" package_name="kuka_agilus_support" use_ext_axes="false">
     <origin xyz="$(arg x) $(arg y) $(arg z)" rpy="$(arg roll) $(arg pitch) $(arg yaw)"/>
+    <ext_axes_links/>
+    <ext_axes_joints/>
   </xacro:kuka_kr6_r900_sixx_robot>
 </robot>

File: kuka_agilus_support/urdf/kr6_r900_sixx_macro.xacro (robot description, xacro)
@@ -4,7 +4,10 @@
   <xacro:include filename="$(find kuka_resources)/urdf/common_constants.xacro"/>
   <xacro:include filename="$(find kuka_resources)/urdf/common_materials.xacro"/>
-  <xacro:macro name="kuka_kr6_r900_sixx_robot" params="prefix package_name *origin">
+  <xacro:macro name="kuka_kr6_r900_sixx_robot" params="prefix package_name use_ext_axes *origin **ext_axes_links **ext_axes_joints">
     <!-- links - main serial chain -->
     <link name="world"/>
+    <xacro:if value="${use_ext_axes}">
+      <xacro:insert_block name="ext_axes_links"/>
+    </xacro:if>
     <link name="${prefix}base_link">
       <visual>
@@ -114,9 +117,14 @@
     <!-- Following REP199, this frame shall be use to attach EEF or other equipment -->
     <link name="${prefix}flange"/>
-    <joint name="${prefix}world-base_link" type="fixed">
-      <parent link="world"/>
-      <child link="${prefix}base_link"/>
-      <xacro:insert_block name="origin"/>
-    </joint>
+    <xacro:if value="${use_ext_axes}">
+      <xacro:insert_block name="ext_axes_joints"/>
+    </xacro:if>
+    <xacro:unless value="${use_ext_axes}">
+      <joint name="${prefix}world-base_link" type="fixed">
+        <parent link="world"/>
+        <child link="${prefix}base_link"/>
+        <xacro:insert_block name="origin"/>
+      </joint>
+    </xacro:unless>
     <joint name="${prefix}joint_1" type="revolute">
       <origin xyz="0 0 0.400" rpy="0 0 0"/>
