Commit message: Refactor Xacro structure (#86)
* refactor: xacro structure to conform with model generation tool

* add gazebo hw tags to cybertech and iiwa models

File: kuka_agilus_support/urdf/kr_agilus_ros2_control_macro.xacro (robot description, xacro)
@@ -1,5 +1,11 @@
 <?xml version="1.0" encoding="UTF-8"?>
 <robot xmlns:xacro="http://www.ros.org/wiki/xacro">
-  <xacro:macro name="kuka_fortec_ros2_control" params="name client_ip client_port controller_ip prefix mode roundtrip_time">
+  <xacro:macro name="kuka_agilus_ros2_control" params="name client_ip client_port controller_ip prefix mode roundtrip_time">
+    <!-- gazebo -->
+    <xacro:if value="${mode == 'gazebo'}">
+      <xacro:include filename="$(find kuka_gazebo)/gazebo/kuka_gazebo.xacro"/>
+      <xacro:kuka_gazebo controller_config_package="kuka_resources" controller_config_path="config/fake_hardware_config_6_axis.yaml"/>
+    </xacro:if>
+    <!-- ros2 control -->
     <ros2_control name="${name}" type="system">
       <hardware>

File: kuka_cybertech_support/urdf/kr_cybertech_ros2_control_macro.xacro (robot description, xacro)
@@ -2,4 +2,10 @@
 <robot xmlns:xacro="http://www.ros.org/wiki/xacro">
   <xacro:macro name="kuka_cybertech_ros2_control" params="name client_ip client_port controller_ip prefix mode roundtrip_time">
+    <!-- gazebo -->
+    <xacro:if value="${mode == 'gazebo'}">
+      <xacro:include filename="$(find kuka_gazebo)/gazebo/kuka_gazebo.xacro"/>
+      <xacro:kuka_gazebo controller_config_package="kuka_resources" controller_config_path="config/fake_hardware_config_6_axis.yaml"/>
+    </xacro:if>
+    <!-- ros2 control -->
     <ros2_control name="${name}" type="system">
       <hardware>

File: kuka_fortec_support/urdf/kr_fortec_ros2_control_macro.xacro (robot description, xacro)
@@ -1,5 +1,11 @@
 <?xml version="1.0" encoding="UTF-8"?>
 <robot xmlns:xacro="http://www.ros.org/wiki/xacro">
-  <xacro:macro name="kuka_iontec_ros2_control" params="name client_ip client_port controller_ip prefix mode roundtrip_time">
+  <xacro:macro name="kuka_fortec_ros2_control" params="name client_ip client_port controller_ip prefix mode roundtrip_time">
+    <!-- gazebo -->
+    <xacro:if value="${mode == 'gazebo'}">
+      <xacro:include filename="$(find kuka_gazebo)/gazebo/kuka_gazebo.xacro"/>
+      <xacro:kuka_gazebo controller_config_package="kuka_resources" controller_config_path="config/fake_hardware_config_6_axis.yaml"/>
+    </xacro:if>
+    <!-- ros2 control -->
     <ros2_control name="${name}" type="system">
       <hardware>

File: kuka_lbr_iiwa_support/urdf/lbr_iiwa14_r820_macro.xacro (robot description, xacro)
@@ -2,10 +2,6 @@
 <robot xmlns:xacro="http://wiki.ros.org/xacro">
   <!-- include helper xacros -->
-  <xacro:include filename="$(find kuka_lbr_iiwa_support)/urdf/lbr_iiwa_ros2_control.xacro"/>
   <xacro:include filename="$(find kuka_resources)/urdf/common_materials.xacro"/>
-  <xacro:include filename="$(find kuka_lbr_iiwa_support)/urdf/lbr_iiwa_transmission.xacro"/>
-  <xacro:macro name="kuka_lbr_iiwa14_r820_robot" params="io_access prefix mode roundtrip_time controller_ip client_ip client_port *origin">
-    <!-- ros2 control instance -->
-    <xacro:kuka_lbr_iiwa_ros2_control name="${prefix}lbr_iiwa14_r820" prefix="${prefix}" io_access="${io_access}" mode="${mode}" roundtrip_time="${roundtrip_time}" controller_ip="${controller_ip}" client_ip="${client_ip}" client_port="${client_port}"/>
+  <xacro:macro name="kuka_lbr_iiwa14_r820_robot" params="prefix package_name *origin">
     <!-- links - main serial chain -->
     <link name="world"/>
@@ -13,5 +9,5 @@
       <visual>
         <geometry>
-          <mesh filename="package://kuka_lbr_iiwa_support/meshes/lbr_iiwa14_r820/visual/base_link.stl"/>
+          <mesh filename="package://${package_name}/meshes/lbr_iiwa14_r820/visual/base_link.stl"/>
         </geometry>
         <origin rpy="-0.0 0.0 0.0" xyz="0.0 0.0 0.0"/>
@@ -20,5 +16,5 @@
         <origin rpy="-0.0 0.0 0.0" xyz="0.0 0.0 0.0"/>
         <geometry>
-          <mesh filename="package://kuka_lbr_iiwa_support/meshes/lbr_iiwa14_r820/collision/base_link.stl"/>
+          <mesh filename="package://${package_name}/meshes/lbr_iiwa14_r820/collision/base_link.stl"/>
         </geometry>
       </collision>
@@ -27,5 +23,5 @@
       <visual>
         <geometry>
-          <mesh filename="package://kuka_lbr_iiwa_support/meshes/lbr_iiwa14_r820/visual/link_1.stl"/>
+          <mesh filename="package://${package_name}/meshes/lbr_iiwa14_r820/visual/link_1.stl"/>
         </geometry>
         <origin rpy="-0.0 0.0 0.0" xyz="0.0 0.0 0.0"/>
@@ -34,5 +30,5 @@
         <origin rpy="-0.0 0.0 0.0" xyz="0.0 0.0 0.0"/>
         <geometry>
-          <mesh filename="package://kuka_lbr_iiwa_support/meshes/lbr_iiwa14_r820/collision/link_1.stl"/>
+          <mesh filename="package://${package_name}/meshes/lbr_iiwa14_r820/collision/link_1.stl"/>
         </geometry>
       </collision>
@@ -41,5 +37,5 @@
       <visual>
         <geometry>
-          <mesh filename="package://kuka_lbr_iiwa_support/meshes/lbr_iiwa14_r820/visual/link_2.stl"/>
+          <mesh filename="package://${package_name}/meshes/lbr_iiwa14_r820/visual/link_2.stl"/>
         </geometry>
         <origin rpy="-0.0 0.0 0.0" xyz="0.0 0.0 0.0"/>
@@ -48,5 +44,5 @@
         <origin rpy="-0.0 0.0 0.0" xyz="0.0 0.0 0.0"/>
         <geometry>
-          <mesh filename="package://kuka_lbr_iiwa_support/meshes/lbr_iiwa14_r820/collision/link_2.stl"/>
+          <mesh filename="package://${package_name}/meshes/lbr_iiwa14_r820/collision/link_2.stl"/>
         </geometry>
       </collision>
@@ -55,5 +51,5 @@
       <visual>
         <geometry>
-          <mesh filename="package://kuka_lbr_iiwa_support/meshes/lbr_iiwa14_r820/visual/link_3.stl"/>
+          <mesh filename="package://${package_name}/meshes/lbr_iiwa14_r820/visual/link_3.stl"/>
         </geometry>
         <origin rpy="-0.0 0.0 0.0" xyz="0.0 0.0 0.0"/>
@@ -62,5 +58,5 @@
         <origin rpy="-0.0 0.0 0.0" xyz="0.0 0.0 0.0"/>
         <geometry>
-          <mesh filename="package://kuka_lbr_iiwa_support/meshes/lbr_iiwa14_r820/collision/link_3.stl"/>
+          <mesh filename="package://${package_name}/meshes/lbr_iiwa14_r820/collision/link_3.stl"/>
         </geometry>
       </collision>
@@ -69,5 +65,5 @@
       <visual>
         <geometry>
-          <mesh filename="package://kuka_lbr_iiwa_support/meshes/lbr_iiwa14_r820/visual/link_4.stl"/>
+          <mesh filename="package://${package_name}/meshes/lbr_iiwa14_r820/visual/link_4.stl"/>
         </geometry>
         <origin rpy="-0.0 0.0 0.0" xyz="0.0 0.0 0.0"/>
@@ -76,5 +72,5 @@
         <origin rpy="-0.0 0.0 0.0" xyz="0.0 0.0 0.0"/>
         <geometry>
-          <mesh filename="package://kuka_lbr_iiwa_support/meshes/lbr_iiwa14_r820/collision/link_4.stl"/>
+          <mesh filename="package://${package_name}/meshes/lbr_iiwa14_r820/collision/link_4.stl"/>
         </geometry>
       </collision>
@@ -83,5 +79,5 @@
       <visual>
         <geometry>
-          <mesh filename="package://kuka_lbr_iiwa_support/meshes/lbr_iiwa14_r820/visual/link_5.stl"/>
+          <mesh filename="package://${package_name}/meshes/lbr_iiwa14_r820/visual/link_5.stl"/>
         </geometry>
         <origin rpy="-0.0 0.0 0.0" xyz="0.0 0.0 0.0"/>
@@ -90,5 +86,5 @@
         <origin rpy="-0.0 0.0 0.0" xyz="0.0 0.0 0.0"/>
         <geometry>
-          <mesh filename="package://kuka_lbr_iiwa_support/meshes/lbr_iiwa14_r820/collision/link_5.stl"/>
+          <mesh filename="package://${package_name}/meshes/lbr_iiwa14_r820/collision/link_5.stl"/>
         </geometry>
       </collision>
@@ -97,5 +93,5 @@
       <visual>
         <geometry>
-          <mesh filename="package://kuka_lbr_iiwa_support/meshes/lbr_iiwa14_r820/visual/link_6.stl"/>
+          <mesh filename="package://${package_name}/meshes/lbr_iiwa14_r820/visual/link_6.stl"/>
         </geometry>
         <origin rpy="-0.0 0.0 0.0" xyz="0.0 0.0 0.0"/>
@@ -104,5 +100,5 @@
         <origin rpy="-0.0 0.0 0.0" xyz="0.0 0.0 0.0"/>
         <geometry>
-          <mesh filename="package://kuka_lbr_iiwa_support/meshes/lbr_iiwa14_r820/collision/link_6.stl"/>
+          <mesh filename="package://${package_name}/meshes/lbr_iiwa14_r820/collision/link_6.stl"/>
         </geometry>
       </collision>
@@ -111,5 +107,5 @@
       <visual>
         <geometry>
-          <mesh filename="package://kuka_lbr_iiwa_support/meshes/lbr_iiwa14_r820/visual/link_7.stl"/>
+          <mesh filename="package://${package_name}/meshes/lbr_iiwa14_r820/visual/link_7.stl"/>
         </geometry>
         <origin rpy="-0.0 0.0 0.0" xyz="0.0 0.0 0.0"/>
@@ -118,5 +114,5 @@
         <origin rpy="-0.0 0.0 0.0" xyz="0.0 0.0 0.0"/>
         <geometry>
-          <mesh filename="package://kuka_lbr_iiwa_support/meshes/lbr_iiwa14_r820/collision/link_7.stl"/>
+          <mesh filename="package://${package_name}/meshes/lbr_iiwa14_r820/collision/link_7.stl"/>
         </geometry>
       </collision>

File: kuka_lbr_iiwa_support/urdf/lbr_iiwa_ros2_control_macro.xacro (robot description, xacro)
@@ -2,4 +2,10 @@
 <robot xmlns:xacro="http://www.ros.org/wiki/xacro">
   <xacro:macro name="kuka_lbr_iiwa_ros2_control" params="name prefix io_access mode roundtrip_time controller_ip client_ip client_port">
+    <!-- gazebo -->
+    <xacro:if value="${mode == 'gazebo'}">
+      <xacro:include filename="$(find kuka_gazebo)/gazebo/kuka_gazebo.xacro"/>
+      <xacro:kuka_gazebo controller_config_package="kuka_resources" controller_config_path="config/fake_hardware_config_7_axis.yaml"/>
+    </xacro:if>
+    <!-- ros2 control -->
     <ros2_control name="${name}" type="system">
       <hardware>
@@ -17,11 +23,16 @@
           <param name="client_port">${client_port}</param>
         </xacro:if>
+        <xacro:if value="${mode == 'gazebo'}">
+          <plugin>gz_ros2_control/GazeboSimSystem</plugin>
+        </xacro:if>
       </hardware>
       <!-- define joints and command/state interfaces for each joint -->
       <joint name="${prefix}joint_1">
         <command_interface name="position"/>
-        <command_interface name="stiffness"/>
-        <command_interface name="damping"/>
-        <command_interface name="effort"/>
+        <xacro:unless value="${mode == 'gazebo'}">
+          <command_interface name="stiffness"/>
+          <command_interface name="damping"/>
+          <command_interface name="effort"/>
+        </xacro:unless>
         <state_interface name="position">
           <param name="initial_value">0.0</param>
@@ -36,7 +47,9 @@
       <joint name="${prefix}joint_2">
         <command_interface name="position"/>
-        <command_interface name="stiffness"/>
-        <command_interface name="damping"/>
-        <command_interface name="effort"/>
+        <xacro:unless value="${mode == 'gazebo'}">
+          <command_interface name="stiffness"/>
+          <command_interface name="damping"/>
+          <command_interface name="effort"/>
+        </xacro:unless>
         <state_interface name="position">
           <param name="initial_value">0.0</param>
@@ -51,7 +64,9 @@
       <joint name="${prefix}joint_3">
         <command_interface name="position"/>
-        <command_interface name="stiffness"/>
-        <command_interface name="damping"/>
-        <command_interface name="effort"/>
+        <xacro:unless value="${mode == 'gazebo'}">
+          <command_interface name="stiffness"/>
+          <command_interface name="damping"/>
+          <command_interface name="effort"/>
+        </xacro:unless>
         <state_interface name="position">
           <param name="initial_value">0.0</param>
@@ -66,7 +81,9 @@
       <joint name="${prefix}joint_4">
         <command_interface name="position"/>
-        <command_interface name="stiffness"/>
-        <command_interface name="damping"/>
-        <command_interface name="effort"/>
+        <xacro:unless value="${mode == 'gazebo'}">
+          <command_interface name="stiffness"/>
+          <command_interface name="damping"/>
+          <command_interface name="effort"/>
+        </xacro:unless>
         <state_interface name="position">
           <param name="initial_value">0.0</param>
@@ -81,7 +98,9 @@
       <joint name="${prefix}joint_5">
         <command_interface name="position"/>
-        <command_interface name="stiffness"/>
-        <command_interface name="damping"/>
-        <command_interface name="effort"/>
+        <xacro:unless value="${mode == 'gazebo'}">
+          <command_interface name="stiffness"/>
+          <command_interface name="damping"/>
+          <command_interface name="effort"/>
+        </xacro:unless>
         <state_interface name="position">
           <param name="initial_value">0.0</param>
@@ -96,7 +115,9 @@
       <joint name="${prefix}joint_6">
         <command_interface name="position"/>
-        <command_interface name="stiffness"/>
-        <command_interface name="damping"/>
-        <command_interface name="effort"/>
+        <xacro:unless value="${mode == 'gazebo'}">
+          <command_interface name="stiffness"/>
+          <command_interface name="damping"/>
+          <command_interface name="effort"/>
+        </xacro:unless>
         <state_interface name="position">
           <param name="initial_value">0.0</param>
@@ -111,7 +132,9 @@
       <joint name="${prefix}joint_7">
         <command_interface name="position"/>
-        <command_interface name="stiffness"/>
-        <command_interface name="damping"/>
-        <command_interface name="effort"/>
+        <xacro:unless value="${mode == 'gazebo'}">
+          <command_interface name="stiffness"/>
+          <command_interface name="damping"/>
+          <command_interface name="effort"/>
+        </xacro:unless>
         <state_interface name="position">
           <param name="initial_value">0.0</param>

Commit message: Add mxa hardware interface to ros2_control xacros (#138)
* extend xacros

* client port to xacros

* add new state interfaces to mock hw if

* more hwif

* mxa_client_port

* format

---------

Co-authored-by: Svastits <49677296+Svastits@users.noreply@github.com>

File: kuka_agilus_support/urdf/kr_agilus_ros2_control_macro.xacro (robot description, xacro)
@@ -1,5 +1,5 @@
 <?xml version="1.0" encoding="UTF-8"?>
 <robot xmlns:xacro="http://www.ros.org/wiki/xacro">
-  <xacro:macro name="kuka_agilus_ros2_control" params="name driver_version client_ip client_port controller_ip prefix mode use_gpio roundtrip_time verify_robot_model">
+  <xacro:macro name="kuka_agilus_ros2_control" params="name driver_version client_ip client_port mxa_client_port controller_ip prefix mode use_gpio roundtrip_time verify_robot_model">
     <!-- gazebo -->
     <xacro:if value="${mode == 'gazebo'}">
@@ -22,4 +22,11 @@
             <param name="controller_ip">${controller_ip}</param>
             <param name="name">${name}</param>
+            <param name="verify_robot_model">${verify_robot_model}</param>
+          </xacro:if>
+          <xacro:if value="${driver_version == 'mxa_rsi'}">
+            <plugin>kuka_rsi_driver::KukaMxaRsiHardwareInterface</plugin>
+            <param name="controller_ip">${controller_ip}</param>
+            <param name="client_port">${client_port}</param>
+            <param name="mxa_client_port">${mxa_client_port}</param>
             <param name="verify_robot_model">${verify_robot_model}</param>
           </xacro:if>

File: kuka_cybertech_support/urdf/kr_cybertech_ros2_control_macro.xacro (robot description, xacro)
@@ -1,5 +1,5 @@
 <?xml version="1.0" encoding="UTF-8"?>
 <robot xmlns:xacro="http://www.ros.org/wiki/xacro">
-  <xacro:macro name="kuka_cybertech_ros2_control" params="name driver_version client_ip client_port controller_ip prefix mode use_gpio roundtrip_time verify_robot_model">
+  <xacro:macro name="kuka_cybertech_ros2_control" params="name driver_version client_ip client_port mxa_client_port controller_ip prefix mode use_gpio roundtrip_time verify_robot_model">
     <!-- gazebo -->
     <xacro:if value="${mode == 'gazebo'}">
@@ -22,4 +22,11 @@
             <param name="controller_ip">${controller_ip}</param>
             <param name="name">${name}</param>
+            <param name="verify_robot_model">${verify_robot_model}</param>
+          </xacro:if>
+          <xacro:if value="${driver_version == 'mxa_rsi'}">
+            <plugin>kuka_rsi_driver::KukaMxaRsiHardwareInterface</plugin>
+            <param name="controller_ip">${controller_ip}</param>
+            <param name="client_port">${client_port}</param>
+            <param name="mxa_client_port">${mxa_client_port}</param>
             <param name="verify_robot_model">${verify_robot_model}</param>
           </xacro:if>

File: kuka_fortec_support/urdf/kr_fortec_ros2_control_macro.xacro (robot description, xacro)
@@ -1,5 +1,5 @@
 <?xml version="1.0" encoding="UTF-8"?>
 <robot xmlns:xacro="http://www.ros.org/wiki/xacro">
-  <xacro:macro name="kuka_fortec_ros2_control" params="name driver_version client_ip client_port controller_ip prefix mode use_gpio roundtrip_time verify_robot_model">
+  <xacro:macro name="kuka_fortec_ros2_control" params="name driver_version client_ip client_port mxa_client_port controller_ip prefix mode use_gpio roundtrip_time verify_robot_model">
     <!-- gazebo -->
     <xacro:if value="${mode == 'gazebo'}">
@@ -22,4 +22,11 @@
             <param name="controller_ip">${controller_ip}</param>
             <param name="name">${name}</param>
+            <param name="verify_robot_model">${verify_robot_model}</param>
+          </xacro:if>
+          <xacro:if value="${driver_version == 'mxa_rsi'}">
+            <plugin>kuka_rsi_driver::KukaMxaRsiHardwareInterface</plugin>
+            <param name="controller_ip">${controller_ip}</param>
+            <param name="client_port">${client_port}</param>
+            <param name="mxa_client_port">${mxa_client_port}</param>
             <param name="verify_robot_model">${verify_robot_model}</param>
           </xacro:if>

File: kuka_iontec_support/urdf/kr70_r2100.urdf.xacro (robot description, xacro)
@@ -11,4 +11,5 @@
   <xacro:arg name="client_ip" default="0.0.0.0"/>
   <xacro:arg name="client_port" default="59152"/>
+  <xacro:arg name="mxa_client_port" default="1337"/>
   <xacro:arg name="controller_ip" default="0.0.0.0"/>
   <xacro:arg name="verify_robot_model" default="true"/>
@@ -20,5 +21,5 @@
   <xacro:arg name="pitch" default="0"/>
   <xacro:arg name="yaw" default="0"/>
-  <xacro:kuka_iontec_ros2_control name="$(arg prefix)kr70_r2100" driver_version="$(arg driver_version)" client_ip="$(arg client_ip)" controller_ip="$(arg controller_ip)" client_port="$(arg client_port)" prefix="$(arg prefix)" mode="$(arg mode)" use_gpio="$(arg use_gpio)" roundtrip_time="$(arg roundtrip_time)" verify_robot_model="$(arg verify_robot_model)"/>
+  <xacro:kuka_iontec_ros2_control name="$(arg prefix)kr70_r2100" driver_version="$(arg driver_version)" client_ip="$(arg client_ip)" controller_ip="$(arg controller_ip)" client_port="$(arg client_port)" mxa_client_port="$(arg mxa_client_port)" prefix="$(arg prefix)" mode="$(arg mode)" use_gpio="$(arg use_gpio)" roundtrip_time="$(arg roundtrip_time)" verify_robot_model="$(arg verify_robot_model)"/>
   <xacro:kuka_kr70_r2100_robot prefix="$(arg prefix)" package_name="kuka_iontec_support">
     <origin xyz="$(arg x) $(arg y) $(arg z)" rpy="$(arg roll) $(arg pitch) $(arg yaw)"/>

File: kuka_iontec_support/urdf/kr_iontec_ros2_control_macro.xacro (robot description, xacro)
@@ -1,5 +1,5 @@
 <?xml version="1.0" encoding="UTF-8"?>
 <robot xmlns:xacro="http://www.ros.org/wiki/xacro">
-  <xacro:macro name="kuka_iontec_ros2_control" params="name driver_version client_ip client_port controller_ip prefix mode use_gpio roundtrip_time verify_robot_model">
+  <xacro:macro name="kuka_iontec_ros2_control" params="name driver_version client_ip client_port mxa_client_port controller_ip prefix mode use_gpio roundtrip_time verify_robot_model">
     <!-- gazebo -->
     <xacro:if value="${mode == 'gazebo'}">
@@ -22,4 +22,11 @@
             <param name="controller_ip">${controller_ip}</param>
             <param name="name">${name}</param>
+            <param name="verify_robot_model">${verify_robot_model}</param>
+          </xacro:if>
+          <xacro:if value="${driver_version == 'mxa_rsi'}">
+            <plugin>kuka_rsi_driver::KukaMxaRsiHardwareInterface</plugin>
+            <param name="controller_ip">${controller_ip}</param>
+            <param name="client_port">${client_port}</param>
+            <param name="mxa_client_port">${mxa_client_port}</param>
             <param name="verify_robot_model">${verify_robot_model}</param>
           </xacro:if>

File: kuka_quantec_support/urdf/kr_quantec_ros2_control_macro.xacro (robot description, xacro)
@@ -1,5 +1,5 @@
 <?xml version="1.0" encoding="UTF-8"?>
 <robot xmlns:xacro="http://www.ros.org/wiki/xacro">
-  <xacro:macro name="kuka_quantec_ros2_control" params="name driver_version client_ip client_port controller_ip prefix mode use_gpio roundtrip_time verify_robot_model">
+  <xacro:macro name="kuka_quantec_ros2_control" params="name driver_version client_ip client_port mxa_client_port controller_ip prefix mode use_gpio roundtrip_time verify_robot_model">
     <!-- gazebo -->
     <xacro:if value="${mode == 'gazebo'}">
@@ -22,4 +22,11 @@
             <param name="controller_ip">${controller_ip}</param>
             <param name="name">${name}</param>
+            <param name="verify_robot_model">${verify_robot_model}</param>
+          </xacro:if>
+          <xacro:if value="${driver_version == 'mxa_rsi'}">
+            <plugin>kuka_rsi_driver::KukaMxaRsiHardwareInterface</plugin>
+            <param name="controller_ip">${controller_ip}</param>
+            <param name="client_port">${client_port}</param>
+            <param name="mxa_client_port">${mxa_client_port}</param>
             <param name="verify_robot_model">${verify_robot_model}</param>
           </xacro:if>
