Commit message: Add rsi_xml_config_file parameter to control macros

File: kuka_agilus_support/urdf/kr_agilus_ros2_control_macro.xacro (robot description, xacro)
@@ -1,5 +1,5 @@
 <?xml version="1.0" encoding="UTF-8"?>
 <robot xmlns:xacro="http://www.ros.org/wiki/xacro">
-  <xacro:macro name="kuka_agilus_ros2_control" params="name driver_version client_ip client_port mxa_client_port controller_ip prefix mode use_gpio roundtrip_time verify_robot_model **ext_axes_ros2_control_joints">
+  <xacro:macro name="kuka_agilus_ros2_control" params="name driver_version client_ip client_port mxa_client_port controller_ip prefix mode use_gpio roundtrip_time verify_robot_model rsi_xml_config_file:='' **ext_axes_ros2_control_joints">
     <!-- gazebo -->
     <xacro:if value="${mode == 'gazebo'}">
@@ -25,4 +25,5 @@
             <param name="name">${name}</param>
             <param name="verify_robot_model">${verify_robot_model}</param>
+            <param name="rsi_xml_config_file">${rsi_xml_config_file}</param>
           </xacro:if>
           <xacro:if value="${driver_version == 'mxa_rsi'}">
@@ -33,4 +34,5 @@
             <param name="mxa_client_port">${mxa_client_port}</param>
             <param name="verify_robot_model">${verify_robot_model}</param>
+            <param name="rsi_xml_config_file">${rsi_xml_config_file}</param>
           </xacro:if>
           <xacro:if value="${driver_version == 'rsi_only'}">
@@ -38,4 +40,5 @@
             <param name="client_ip">${client_ip}</param>
             <param name="client_port">${client_port}</param>
+            <param name="rsi_xml_config_file">${rsi_xml_config_file}</param>
           </xacro:if>
         </xacro:if>

File: kuka_cybertech_support/urdf/kr_cybertech_ros2_control_macro.xacro (robot description, xacro)
@@ -1,5 +1,5 @@
 <?xml version="1.0" encoding="UTF-8"?>
 <robot xmlns:xacro="http://www.ros.org/wiki/xacro">
-  <xacro:macro name="kuka_cybertech_ros2_control" params="name driver_version client_ip client_port mxa_client_port controller_ip prefix mode use_gpio roundtrip_time verify_robot_model **ext_axes_ros2_control_joints">
+  <xacro:macro name="kuka_cybertech_ros2_control" params="name driver_version client_ip client_port mxa_client_port controller_ip prefix mode use_gpio roundtrip_time verify_robot_model rsi_xml_config_file:='' **ext_axes_ros2_control_joints">
     <!-- gazebo -->
     <xacro:if value="${mode == 'gazebo'}">
@@ -25,4 +25,5 @@
             <param name="name">${name}</param>
             <param name="verify_robot_model">${verify_robot_model}</param>
+            <param name="rsi_xml_config_file">${rsi_xml_config_file}</param>
           </xacro:if>
           <xacro:if value="${driver_version == 'mxa_rsi'}">
@@ -33,4 +34,5 @@
             <param name="mxa_client_port">${mxa_client_port}</param>
             <param name="verify_robot_model">${verify_robot_model}</param>
+            <param name="rsi_xml_config_file">${rsi_xml_config_file}</param>
           </xacro:if>
           <xacro:if value="${driver_version == 'rsi_only'}">
@@ -38,4 +40,5 @@
             <param name="client_ip">${client_ip}</param>
             <param name="client_port">${client_port}</param>
+            <param name="rsi_xml_config_file">${rsi_xml_config_file}</param>
           </xacro:if>
         </xacro:if>

File: kuka_fortec_support/urdf/kr_fortec_ros2_control_macro.xacro (robot description, xacro)
@@ -1,5 +1,5 @@
 <?xml version="1.0" encoding="UTF-8"?>
 <robot xmlns:xacro="http://www.ros.org/wiki/xacro">
-  <xacro:macro name="kuka_fortec_ros2_control" params="name driver_version client_ip client_port mxa_client_port controller_ip prefix mode use_gpio roundtrip_time verify_robot_model **ext_axes_ros2_control_joints">
+  <xacro:macro name="kuka_fortec_ros2_control" params="name driver_version client_ip client_port mxa_client_port controller_ip prefix mode use_gpio roundtrip_time verify_robot_model rsi_xml_config_file:='' **ext_axes_ros2_control_joints">
     <!-- gazebo -->
     <xacro:if value="${mode == 'gazebo'}">
@@ -25,4 +25,5 @@
             <param name="name">${name}</param>
             <param name="verify_robot_model">${verify_robot_model}</param>
+            <param name="rsi_xml_config_file">${rsi_xml_config_file}</param>
           </xacro:if>
           <xacro:if value="${driver_version == 'mxa_rsi'}">
@@ -33,4 +34,5 @@
             <param name="mxa_client_port">${mxa_client_port}</param>
             <param name="verify_robot_model">${verify_robot_model}</param>
+            <param name="rsi_xml_config_file">${rsi_xml_config_file}</param>
           </xacro:if>
           <xacro:if value="${driver_version == 'rsi_only'}">
@@ -38,4 +40,5 @@
             <param name="client_ip">${client_ip}</param>
             <param name="client_port">${client_port}</param>
+            <param name="rsi_xml_config_file">${rsi_xml_config_file}</param>
           </xacro:if>
         </xacro:if>

File: kuka_iontec_support/urdf/kr_iontec_ros2_control_macro.xacro (robot description, xacro)
@@ -1,5 +1,5 @@
 <?xml version="1.0" encoding="UTF-8"?>
 <robot xmlns:xacro="http://www.ros.org/wiki/xacro">
-  <xacro:macro name="kuka_iontec_ros2_control" params="name driver_version client_ip client_port mxa_client_port controller_ip prefix mode use_gpio roundtrip_time verify_robot_model **ext_axes_ros2_control_joints">
+  <xacro:macro name="kuka_iontec_ros2_control" params="name driver_version client_ip client_port mxa_client_port controller_ip prefix mode use_gpio roundtrip_time verify_robot_model rsi_xml_config_file:='' **ext_axes_ros2_control_joints">
     <!-- gazebo -->
     <xacro:if value="${mode == 'gazebo'}">
@@ -25,4 +25,5 @@
             <param name="name">${name}</param>
             <param name="verify_robot_model">${verify_robot_model}</param>
+            <param name="rsi_xml_config_file">${rsi_xml_config_file}</param>
           </xacro:if>
           <xacro:if value="${driver_version == 'mxa_rsi'}">
@@ -33,4 +34,5 @@
             <param name="mxa_client_port">${mxa_client_port}</param>
             <param name="verify_robot_model">${verify_robot_model}</param>
+            <param name="rsi_xml_config_file">${rsi_xml_config_file}</param>
           </xacro:if>
           <xacro:if value="${driver_version == 'rsi_only'}">
@@ -38,4 +40,5 @@
             <param name="client_ip">${client_ip}</param>
             <param name="client_port">${client_port}</param>
+            <param name="rsi_xml_config_file">${rsi_xml_config_file}</param>
           </xacro:if>
         </xacro:if>

File: kuka_lbr_iisy_support/urdf/lbr_iisy_ros2_control_macro.xacro (robot description, xacro)
@@ -1,5 +1,5 @@
 <?xml version="1.0" encoding="UTF-8"?>
 <robot xmlns:xacro="http://www.ros.org/wiki/xacro">
-  <xacro:macro name="kuka_lbr_iisy_ros2_control" params="name driver_version prefix client_ip client_port mxa_client_port controller_ip use_gpio mode qos_config_file roundtrip_time verify_robot_model **ext_axes_ros2_control_joints">
+  <xacro:macro name="kuka_lbr_iisy_ros2_control" params="name driver_version prefix client_ip client_port mxa_client_port controller_ip use_gpio mode qos_config_file roundtrip_time verify_robot_model rsi_xml_config_file:='' **ext_axes_ros2_control_joints">
     <!-- gazebo -->
     <xacro:if value="${mode == 'gazebo'}">
@@ -46,4 +46,5 @@
             <param name="name">${name}</param>
             <param name="verify_robot_model">${verify_robot_model}</param>
+            <param name="rsi_xml_config_file">${rsi_xml_config_file}</param>
           </xacro:if>
           <xacro:if value="${driver_version == 'mxa_rsi'}">
@@ -54,4 +55,5 @@
             <param name="mxa_client_port">${mxa_client_port}</param>
             <param name="verify_robot_model">${verify_robot_model}</param>
+            <param name="rsi_xml_config_file">${rsi_xml_config_file}</param>
           </xacro:if>
           <xacro:if value="${driver_version == 'rsi_only'}">
@@ -59,4 +61,5 @@
             <param name="client_ip">${client_ip}</param>
             <param name="client_port">${client_port}</param>
+            <param name="rsi_xml_config_file">${rsi_xml_config_file}</param>
           </xacro:if>
         </xacro:if>

File: kuka_quantec_support/urdf/kr_quantec_ros2_control_macro.xacro (robot description, xacro)
@@ -1,5 +1,5 @@
 <?xml version="1.0" encoding="UTF-8"?>
 <robot xmlns:xacro="http://www.ros.org/wiki/xacro">
-  <xacro:macro name="kuka_quantec_ros2_control" params="name driver_version client_ip client_port mxa_client_port controller_ip prefix mode use_gpio roundtrip_time verify_robot_model **ext_axes_ros2_control_joints">
+  <xacro:macro name="kuka_quantec_ros2_control" params="name driver_version client_ip client_port mxa_client_port controller_ip prefix mode use_gpio roundtrip_time verify_robot_model rsi_xml_config_file:='' **ext_axes_ros2_control_joints">
     <!-- gazebo -->
     <xacro:if value="${mode == 'gazebo'}">
@@ -25,4 +25,5 @@
             <param name="name">${name}</param>
             <param name="verify_robot_model">${verify_robot_model}</param>
+            <param name="rsi_xml_config_file">${rsi_xml_config_file}</param>
           </xacro:if>
           <xacro:if value="${driver_version == 'mxa_rsi'}">
@@ -33,4 +34,5 @@
             <param name="mxa_client_port">${mxa_client_port}</param>
             <param name="verify_robot_model">${verify_robot_model}</param>
+            <param name="rsi_xml_config_file">${rsi_xml_config_file}</param>
           </xacro:if>
           <xacro:if value="${driver_version == 'rsi_only'}">
@@ -38,4 +40,5 @@
             <param name="client_ip">${client_ip}</param>
             <param name="client_port">${client_port}</param>
+            <param name="rsi_xml_config_file">${rsi_xml_config_file}</param>
           </xacro:if>
         </xacro:if>

Commit message: is_async with default value

File: kuka_agilus_support/urdf/kr_agilus_ros2_control_macro.xacro (robot description, xacro)
@@ -1,5 +1,5 @@
 <?xml version="1.0" encoding="UTF-8"?>
 <robot xmlns:xacro="http://www.ros.org/wiki/xacro">
-  <xacro:macro name="kuka_agilus_ros2_control" params="name driver_version client_ip client_port mxa_client_port controller_ip prefix mode use_gpio roundtrip_time verify_robot_model **ext_axes_ros2_control_joints">
+  <xacro:macro name="kuka_agilus_ros2_control" params="name driver_version client_ip client_port mxa_client_port controller_ip prefix mode use_gpio roundtrip_time verify_robot_model is_async:=true **ext_axes_ros2_control_joints">
     <!-- gazebo -->
     <xacro:if value="${mode == 'gazebo'}">
@@ -8,8 +8,12 @@
     </xacro:if>
     <!-- ros2 control -->
-    <ros2_control name="${name}" type="system">
+    <ros2_control name="${name}" type="system" is_async="${is_async}">
+      <properties>
+        <async scheduling_policy="detached" print_warnings="false" thread_priority="50"/>
+      </properties>
       <hardware>
         <xacro:if value="${mode == 'mock'}">
           <plugin>kuka_mock_hardware_interface::KukaMockHardwareInterface</plugin>
+          <param name="interface_prefix">${prefix}</param>
           <param name="cycle_time_ms">4</param>
           <param name="roundtrip_time_micro">${roundtrip_time}</param>

Commit message: scheduling parametrization

File: kuka_agilus_support/urdf/kr_agilus_ros2_control_macro.xacro (robot description, xacro)
@@ -1,5 +1,5 @@
 <?xml version="1.0" encoding="UTF-8"?>
 <robot xmlns:xacro="http://www.ros.org/wiki/xacro">
-  <xacro:macro name="kuka_agilus_ros2_control" params="name driver_version client_ip client_port mxa_client_port controller_ip prefix mode use_gpio roundtrip_time verify_robot_model is_async **ext_axes_ros2_control_joints">
+  <xacro:macro name="kuka_agilus_ros2_control" params="name driver_version client_ip client_port mxa_client_port controller_ip prefix mode use_gpio roundtrip_time verify_robot_model is_async async_thread_priority async_affinity **ext_axes_ros2_control_joints">
     <!-- gazebo -->
     <xacro:if value="${mode == 'gazebo'}">
@@ -10,5 +10,5 @@
     <ros2_control name="${name}" type="system" is_async="${is_async}">
       <properties>
-        <async scheduling_policy="detached" print_warnings="false" thread_priority="69"/>
+        <async affinity="${async_affinity}" scheduling_policy="detached" print_warnings="false" thread_priority="${async_thread_priority}"/>
       </properties>
       <hardware>

File: kuka_cybertech_support/urdf/kr_cybertech_ros2_control_macro.xacro (robot description, xacro)
@@ -1,5 +1,5 @@
 <?xml version="1.0" encoding="UTF-8"?>
 <robot xmlns:xacro="http://www.ros.org/wiki/xacro">
-  <xacro:macro name="kuka_cybertech_ros2_control" params="name driver_version client_ip client_port mxa_client_port controller_ip prefix mode use_gpio roundtrip_time verify_robot_model is_async **ext_axes_ros2_control_joints">
+  <xacro:macro name="kuka_cybertech_ros2_control" params="name driver_version client_ip client_port mxa_client_port controller_ip prefix mode use_gpio roundtrip_time verify_robot_model is_async async_thread_priority:=69 async_affinity:='' **ext_axes_ros2_control_joints">
     <!-- gazebo -->
     <xacro:if value="${mode == 'gazebo'}">
@@ -10,5 +10,5 @@
     <ros2_control name="${name}" type="system" is_async="${is_async}">
       <properties>
-        <async scheduling_policy="detached" print_warnings="false" thread_priority="69"/>
+        <async affinity="${async_affinity}" scheduling_policy="detached" print_warnings="false" thread_priority="${async_thread_priority}"/>
       </properties>
       <hardware>

File: kuka_fortec_support/urdf/kr_fortec_ros2_control_macro.xacro (robot description, xacro)
@@ -1,5 +1,5 @@
 <?xml version="1.0" encoding="UTF-8"?>
 <robot xmlns:xacro="http://www.ros.org/wiki/xacro">
-  <xacro:macro name="kuka_fortec_ros2_control" params="name driver_version client_ip client_port mxa_client_port controller_ip prefix mode use_gpio roundtrip_time verify_robot_model is_async **ext_axes_ros2_control_joints">
+  <xacro:macro name="kuka_fortec_ros2_control" params="name driver_version client_ip client_port mxa_client_port controller_ip prefix mode use_gpio roundtrip_time verify_robot_model is_async async_thread_priority:=69 async_affinity:='' **ext_axes_ros2_control_joints">
     <!-- gazebo -->
     <xacro:if value="${mode == 'gazebo'}">
@@ -10,5 +10,5 @@
     <ros2_control name="${name}" type="system" is_async="${is_async}">
       <properties>
-        <async scheduling_policy="detached" print_warnings="false" thread_priority="69"/>
+        <async affinity="${async_affinity}" scheduling_policy="detached" print_warnings="false" thread_priority="${async_thread_priority}"/>
       </properties>
       <hardware>

File: kuka_iontec_support/urdf/kr_iontec_ros2_control_macro.xacro (robot description, xacro)
@@ -1,5 +1,5 @@
 <?xml version="1.0" encoding="UTF-8"?>
 <robot xmlns:xacro="http://www.ros.org/wiki/xacro">
-  <xacro:macro name="kuka_iontec_ros2_control" params="name driver_version client_ip client_port mxa_client_port controller_ip prefix mode use_gpio roundtrip_time verify_robot_model is_async **ext_axes_ros2_control_joints">
+  <xacro:macro name="kuka_iontec_ros2_control" params="name driver_version client_ip client_port mxa_client_port controller_ip prefix mode use_gpio roundtrip_time verify_robot_model is_async async_thread_priority:=69 async_affinity:='' **ext_axes_ros2_control_joints">
     <!-- gazebo -->
     <xacro:if value="${mode == 'gazebo'}">
@@ -10,5 +10,5 @@
     <ros2_control name="${name}" type="system" is_async="${is_async}">
       <properties>
-        <async scheduling_policy="detached" print_warnings="false" thread_priority="69"/>
+        <async affinity="${async_affinity}" scheduling_policy="detached" print_warnings="false" thread_priority="${async_thread_priority}"/>
       </properties>
       <hardware>

File: kuka_lbr_iisy_support/urdf/lbr_iisy_ros2_control_macro.xacro (robot description, xacro)
@@ -1,5 +1,5 @@
 <?xml version="1.0" encoding="UTF-8"?>
 <robot xmlns:xacro="http://www.ros.org/wiki/xacro">
-  <xacro:macro name="kuka_lbr_iisy_ros2_control" params="name driver_version prefix client_ip client_port mxa_client_port controller_ip use_gpio mode qos_config_file roundtrip_time verify_robot_model is_async **ext_axes_ros2_control_joints">
+  <xacro:macro name="kuka_lbr_iisy_ros2_control" params="name driver_version prefix client_ip client_port mxa_client_port controller_ip use_gpio mode qos_config_file roundtrip_time verify_robot_model is_async async_thread_priority:=69 async_affinity:='' **ext_axes_ros2_control_joints">
     <!-- gazebo -->
     <xacro:if value="${mode == 'gazebo'}">
@@ -10,5 +10,5 @@
     <ros2_control name="${name}" type="system" is_async="${is_async}">
       <properties>
-        <async scheduling_policy="detached" print_warnings="false" thread_priority="69"/>
+        <async affinity="${async_affinity}" scheduling_policy="detached" print_warnings="false" thread_priority="${async_thread_priority}"/>
       </properties>
       <hardware>

File: kuka_lbr_iiwa_support/urdf/lbr_iiwa_ros2_control_macro.xacro (robot description, xacro)
@@ -1,5 +1,5 @@
 <?xml version="1.0" encoding="UTF-8"?>
 <robot xmlns:xacro="http://www.ros.org/wiki/xacro">
-  <xacro:macro name="kuka_lbr_iiwa_ros2_control" params="name prefix io_access mode roundtrip_time controller_ip client_ip client_port is_async **ext_axes_ros2_control_joints">
+  <xacro:macro name="kuka_lbr_iiwa_ros2_control" params="name prefix io_access mode roundtrip_time controller_ip client_ip client_port is_async async_thread_priority:=69 async_affinity:='' **ext_axes_ros2_control_joints">
     <!-- gazebo -->
     <xacro:if value="${mode == 'gazebo'}">
@@ -10,5 +10,5 @@
     <ros2_control name="${name}" type="system" is_async="${is_async}">
       <properties>
-        <async scheduling_policy="detached" print_warnings="false" thread_priority="69"/>
+        <async affinity="${async_affinity}" scheduling_policy="detached" print_warnings="false" thread_priority="${async_thread_priority}"/>
       </properties>
       <hardware>

File: kuka_quantec_support/urdf/kr_quantec_ros2_control_macro.xacro (robot description, xacro)
@@ -1,5 +1,5 @@
 <?xml version="1.0" encoding="UTF-8"?>
 <robot xmlns:xacro="http://www.ros.org/wiki/xacro">
-  <xacro:macro name="kuka_quantec_ros2_control" params="name driver_version client_ip client_port mxa_client_port controller_ip prefix mode use_gpio roundtrip_time verify_robot_model is_async **ext_axes_ros2_control_joints">
+  <xacro:macro name="kuka_quantec_ros2_control" params="name driver_version client_ip client_port mxa_client_port controller_ip prefix mode use_gpio roundtrip_time verify_robot_model is_async async_thread_priority:=69 async_affinity:='' **ext_axes_ros2_control_joints">
     <!-- gazebo -->
     <xacro:if value="${mode == 'gazebo'}">
@@ -10,5 +10,5 @@
     <ros2_control name="${name}" type="system" is_async="${is_async}">
       <properties>
-        <async scheduling_policy="detached" print_warnings="false" thread_priority="69"/>
+        <async affinity="${async_affinity}" scheduling_policy="detached" print_warnings="false" thread_priority="${async_thread_priority}"/>
       </properties>
       <hardware>
