Commit message: Custom RSI XML parsing (#216)
* Add rsi_xml_config_file parameter to control macros

* Add rsi_xml_config_file to robot URDFs

* Refactor driver version handling in control macro

* Pre-commit

* Update KR 120 R2700-2

File: kuka_agilus_support/urdf/kr_agilus_ros2_control_macro.xacro (robot description, xacro)
@@ -1,5 +1,5 @@
 <?xml version="1.0" encoding="UTF-8"?>
 <robot xmlns:xacro="http://www.ros.org/wiki/xacro">
-  <xacro:macro name="kuka_agilus_ros2_control" params="name driver_version client_ip client_port mxa_client_port controller_ip prefix mode use_gpio roundtrip_time verify_robot_model **ext_axes_ros2_control_joints">
+  <xacro:macro name="kuka_agilus_ros2_control" params="name driver_version client_ip client_port mxa_client_port controller_ip prefix mode use_gpio roundtrip_time verify_robot_model rsi_xml_config_file **ext_axes_ros2_control_joints">
     <!-- gazebo -->
     <xacro:if value="${mode == 'gazebo'}">
@@ -25,4 +25,5 @@
             <param name="name">${name}</param>
             <param name="verify_robot_model">${verify_robot_model}</param>
+            <param name="rsi_xml_config_file">${rsi_xml_config_file}</param>
           </xacro:if>
           <xacro:if value="${driver_version == 'mxa_rsi'}">
@@ -33,4 +34,5 @@
             <param name="mxa_client_port">${mxa_client_port}</param>
             <param name="verify_robot_model">${verify_robot_model}</param>
+            <param name="rsi_xml_config_file">${rsi_xml_config_file}</param>
           </xacro:if>
           <xacro:if value="${driver_version == 'rsi_only'}">
@@ -38,4 +40,5 @@
             <param name="client_ip">${client_ip}</param>
             <param name="client_port">${client_port}</param>
+            <param name="rsi_xml_config_file">${rsi_xml_config_file}</param>
           </xacro:if>
         </xacro:if>

File: kuka_cybertech_support/urdf/kr_cybertech_ros2_control_macro.xacro (robot description, xacro)
@@ -1,5 +1,5 @@
 <?xml version="1.0" encoding="UTF-8"?>
 <robot xmlns:xacro="http://www.ros.org/wiki/xacro">
-  <xacro:macro name="kuka_cybertech_ros2_control" params="name driver_version client_ip client_port mxa_client_port controller_ip prefix mode use_gpio roundtrip_time verify_robot_model **ext_axes_ros2_control_joints">
+  <xacro:macro name="kuka_cybertech_ros2_control" params="name driver_version client_ip client_port mxa_client_port controller_ip prefix mode use_gpio roundtrip_time verify_robot_model rsi_xml_config_file **ext_axes_ros2_control_joints">
     <!-- gazebo -->
     <xacro:if value="${mode == 'gazebo'}">
@@ -25,4 +25,5 @@
             <param name="name">${name}</param>
             <param name="verify_robot_model">${verify_robot_model}</param>
+            <param name="rsi_xml_config_file">${rsi_xml_config_file}</param>
           </xacro:if>
           <xacro:if value="${driver_version == 'mxa_rsi'}">
@@ -33,4 +34,5 @@
             <param name="mxa_client_port">${mxa_client_port}</param>
             <param name="verify_robot_model">${verify_robot_model}</param>
+            <param name="rsi_xml_config_file">${rsi_xml_config_file}</param>
           </xacro:if>
           <xacro:if value="${driver_version == 'rsi_only'}">
@@ -38,4 +40,5 @@
             <param name="client_ip">${client_ip}</param>
             <param name="client_port">${client_port}</param>
+            <param name="rsi_xml_config_file">${rsi_xml_config_file}</param>
           </xacro:if>
         </xacro:if>

File: kuka_fortec_support/urdf/kr_fortec_ros2_control_macro.xacro (robot description, xacro)
@@ -1,5 +1,5 @@
 <?xml version="1.0" encoding="UTF-8"?>
 <robot xmlns:xacro="http://www.ros.org/wiki/xacro">
-  <xacro:macro name="kuka_fortec_ros2_control" params="name driver_version client_ip client_port mxa_client_port controller_ip prefix mode use_gpio roundtrip_time verify_robot_model **ext_axes_ros2_control_joints">
+  <xacro:macro name="kuka_fortec_ros2_control" params="name driver_version client_ip client_port mxa_client_port controller_ip prefix mode use_gpio roundtrip_time verify_robot_model rsi_xml_config_file **ext_axes_ros2_control_joints">
     <!-- gazebo -->
     <xacro:if value="${mode == 'gazebo'}">
@@ -25,4 +25,5 @@
             <param name="name">${name}</param>
             <param name="verify_robot_model">${verify_robot_model}</param>
+            <param name="rsi_xml_config_file">${rsi_xml_config_file}</param>
           </xacro:if>
           <xacro:if value="${driver_version == 'mxa_rsi'}">
@@ -33,4 +34,5 @@
             <param name="mxa_client_port">${mxa_client_port}</param>
             <param name="verify_robot_model">${verify_robot_model}</param>
+            <param name="rsi_xml_config_file">${rsi_xml_config_file}</param>
           </xacro:if>
           <xacro:if value="${driver_version == 'rsi_only'}">
@@ -38,4 +40,5 @@
             <param name="client_ip">${client_ip}</param>
             <param name="client_port">${client_port}</param>
+            <param name="rsi_xml_config_file">${rsi_xml_config_file}</param>
           </xacro:if>
         </xacro:if>

File: kuka_iontec_support/urdf/kr_iontec_ros2_control_macro.xacro (robot description, xacro)
@@ -1,5 +1,5 @@
 <?xml version="1.0" encoding="UTF-8"?>
 <robot xmlns:xacro="http://www.ros.org/wiki/xacro">
-  <xacro:macro name="kuka_iontec_ros2_control" params="name driver_version client_ip client_port mxa_client_port controller_ip prefix mode use_gpio roundtrip_time verify_robot_model **ext_axes_ros2_control_joints">
+  <xacro:macro name="kuka_iontec_ros2_control" params="name driver_version client_ip client_port mxa_client_port controller_ip prefix mode use_gpio roundtrip_time verify_robot_model rsi_xml_config_file **ext_axes_ros2_control_joints">
     <!-- gazebo -->
     <xacro:if value="${mode == 'gazebo'}">
@@ -25,4 +25,5 @@
             <param name="name">${name}</param>
             <param name="verify_robot_model">${verify_robot_model}</param>
+            <param name="rsi_xml_config_file">${rsi_xml_config_file}</param>
           </xacro:if>
           <xacro:if value="${driver_version == 'mxa_rsi'}">
@@ -33,4 +34,5 @@
             <param name="mxa_client_port">${mxa_client_port}</param>
             <param name="verify_robot_model">${verify_robot_model}</param>
+            <param name="rsi_xml_config_file">${rsi_xml_config_file}</param>
           </xacro:if>
           <xacro:if value="${driver_version == 'rsi_only'}">
@@ -38,4 +40,5 @@
             <param name="client_ip">${client_ip}</param>
             <param name="client_port">${client_port}</param>
+            <param name="rsi_xml_config_file">${rsi_xml_config_file}</param>
           </xacro:if>
         </xacro:if>

File: kuka_lbr_iisy_support/urdf/lbr_iisy_ros2_control_macro.xacro (robot description, xacro)
@@ -1,5 +1,5 @@
 <?xml version="1.0" encoding="UTF-8"?>
 <robot xmlns:xacro="http://www.ros.org/wiki/xacro">
-  <xacro:macro name="kuka_lbr_iisy_ros2_control" params="name driver_version prefix client_ip client_port mxa_client_port controller_ip use_gpio mode qos_config_file roundtrip_time verify_robot_model **ext_axes_ros2_control_joints">
+  <xacro:macro name="kuka_lbr_iisy_ros2_control" params="name driver_version prefix client_ip client_port mxa_client_port controller_ip use_gpio mode qos_config_file roundtrip_time verify_robot_model rsi_xml_config_file **ext_axes_ros2_control_joints">
     <!-- gazebo -->
     <xacro:if value="${mode == 'gazebo'}">
@@ -39,25 +39,26 @@
             <param name="timeframe_ms">${timeframe_ms}</param>
           </xacro:if>
-          <xacro:if value="${driver_version == 'eki_rsi'}">
-            <plugin>kuka_rsi_driver::KukaEkiRsiHardwareInterface</plugin>
-            <param name="controller_ip">${controller_ip}</param>
+          <xacro:unless value="${driver_version == 'eac'}">
+            <!-- Common params for all three KSS drivers -->
             <param name="client_ip">${client_ip}</param>
             <param name="client_port">${client_port}</param>
-            <param name="name">${name}</param>
-            <param name="verify_robot_model">${verify_robot_model}</param>
-          </xacro:if>
-          <xacro:if value="${driver_version == 'mxa_rsi'}">
-            <plugin>kuka_rsi_driver::KukaMxaRsiHardwareInterface</plugin>
-            <param name="controller_ip">${controller_ip}</param>
-            <param name="client_ip">${client_ip}</param>
-            <param name="client_port">${client_port}</param>
-            <param name="mxa_client_port">${mxa_client_port}</param>
-            <param name="verify_robot_model">${verify_robot_model}</param>
-          </xacro:if>
-          <xacro:if value="${driver_version == 'rsi_only'}">
-            <plugin>kuka_rsi_driver::KukaRSIHardwareInterface</plugin>
-            <param name="client_ip">${client_ip}</param>
-            <param name="client_port">${client_port}</param>
-          </xacro:if>
+            <param name="rsi_xml_config_file">${rsi_xml_config_file}</param>
+            <xacro:if value="${driver_version == 'rsi_only'}">
+              <plugin>kuka_rsi_driver::KukaRSIHardwareInterface</plugin>
+            </xacro:if>
+            <xacro:unless value="${driver_version == 'rsi_only'}">
+              <!-- Common params for the EKI and mxAutomation drivers -->
+              <param name="controller_ip">${controller_ip}</param>
+              <param name="verify_robot_model">${verify_robot_model}</param>
+              <xacro:if value="${driver_version == 'eki_rsi'}">
+                <plugin>kuka_rsi_driver::KukaEkiRsiHardwareInterface</plugin>
+                <param name="name">${name}</param>
+              </xacro:if>
+              <xacro:if value="${driver_version == 'mxa_rsi'}">
+                <plugin>kuka_rsi_driver::KukaMxaRsiHardwareInterface</plugin>
+                <param name="mxa_client_port">${mxa_client_port}</param>
+              </xacro:if>
+            </xacro:unless>
+          </xacro:unless>
         </xacro:if>
         <xacro:if value="${mode == 'gazebo'}">

File: kuka_quantec_support/urdf/kr_quantec_ros2_control_macro.xacro (robot description, xacro)
@@ -1,5 +1,5 @@
 <?xml version="1.0" encoding="UTF-8"?>
 <robot xmlns:xacro="http://www.ros.org/wiki/xacro">
-  <xacro:macro name="kuka_quantec_ros2_control" params="name driver_version client_ip client_port mxa_client_port controller_ip prefix mode use_gpio roundtrip_time verify_robot_model **ext_axes_ros2_control_joints">
+  <xacro:macro name="kuka_quantec_ros2_control" params="name driver_version client_ip client_port mxa_client_port controller_ip prefix mode use_gpio roundtrip_time verify_robot_model rsi_xml_config_file **ext_axes_ros2_control_joints">
     <!-- gazebo -->
     <xacro:if value="${mode == 'gazebo'}">
@@ -25,4 +25,5 @@
             <param name="name">${name}</param>
             <param name="verify_robot_model">${verify_robot_model}</param>
+            <param name="rsi_xml_config_file">${rsi_xml_config_file}</param>
           </xacro:if>
           <xacro:if value="${driver_version == 'mxa_rsi'}">
@@ -33,4 +34,5 @@
             <param name="mxa_client_port">${mxa_client_port}</param>
             <param name="verify_robot_model">${verify_robot_model}</param>
+            <param name="rsi_xml_config_file">${rsi_xml_config_file}</param>
           </xacro:if>
           <xacro:if value="${driver_version == 'rsi_only'}">
@@ -38,4 +40,5 @@
             <param name="client_ip">${client_ip}</param>
             <param name="client_port">${client_port}</param>
+            <param name="rsi_xml_config_file">${rsi_xml_config_file}</param>
           </xacro:if>
         </xacro:if>
