Commit message: Add conditional velocity and effort interfaces

File: kuka_lbr_iisy_support/urdf/lbr_iisy_ros2_control_macro.xacro (robot description, xacro)
@@ -70,163 +70,151 @@
       <joint name="${prefix}joint_1">
         <command_interface name="position"/>
-        <xacro:unless value="${driver_version == 'eac'}">
-          <command_interface name="velocity"/>
-          <command_interface name="effort"/>
-        </xacro:unless>
-        <xacro:if value="${driver_version == 'eac' and mode != 'gazebo'}">
-          <command_interface name="stiffness"/>
-          <command_interface name="damping"/>
-          <command_interface name="effort"/>
-        </xacro:if>
-        <state_interface name="position">
-          <param name="initial_value">0.0</param>
-        </state_interface>
-        <xacro:unless value="${driver_version == 'eac'}">
-          <state_interface name="velocity"/>
-          <state_interface name="effort"/>
-        </xacro:unless>
-        <xacro:if value="${driver_version == 'eac'}">
-          <state_interface name="effort">
-            <param name="initial_value">0.0</param>
-          </state_interface>
-          <state_interface name="commanded_position">
-            <param name="initial_value">0.0</param>
-          </state_interface>
-        </xacro:if>
+        <state_interface name="position">
+          <param name="initial_value">0.0</param>
+        </state_interface>
+        <xacro:unless value="${mode == 'gazebo'}">
+          <command_interface name="effort"/>
+          <state_interface name="effort">
+            <param name="initial_value">0.0</param>
+          </state_interface>
+          <xacro:if value="${driver_version == 'eac'}">
+            <command_interface name="stiffness"/>
+            <command_interface name="damping"/>
+            <state_interface name="commanded_position">
+              <param name="initial_value">0.0</param>
+            </state_interface>
+          </xacro:if>
+          <xacro:unless value="${driver_version == 'eac'}">
+            <command_interface name="velocity"/>
+            <state_interface name="velocity">
+              <param name="initial_value">0.0</param>
+            </state_interface>
+          </xacro:unless>
+        </xacro:unless>
       </joint>
       <joint name="${prefix}joint_2">
         <command_interface name="position"/>
-        <xacro:unless value="${driver_version == 'eac'}">
-          <command_interface name="velocity"/>
-          <command_interface name="effort"/>
-        </xacro:unless>
-        <xacro:if value="${driver_version == 'eac' and mode != 'gazebo'}">
-          <command_interface name="stiffness"/>
-          <command_interface name="damping"/>
-          <command_interface name="effort"/>
-        </xacro:if>
         <state_interface name="position">
           <param name="initial_value">-1.5708</param>
         </state_interface>
-        <xacro:unless value="${driver_version == 'eac'}">
-          <state_interface name="velocity"/>
-          <state_interface name="effort"/>
-        </xacro:unless>
-        <xacro:if value="${driver_version == 'eac'}">
-          <state_interface name="effort">
-            <param name="initial_value">0.0</param>
-          </state_interface>
-          <state_interface name="commanded_position">
-            <param name="initial_value">0.0</param>
-          </state_interface>
-        </xacro:if>
+        <xacro:unless value="${mode == 'gazebo'}">
+          <command_interface name="effort"/>
+          <state_interface name="effort">
+            <param name="initial_value">0.0</param>
+          </state_interface>
+          <xacro:if value="${driver_version == 'eac'}">
+            <command_interface name="stiffness"/>
+            <command_interface name="damping"/>
+            <state_interface name="commanded_position">
+              <param name="initial_value">0.0</param>
+            </state_interface>
+          </xacro:if>
+          <xacro:unless value="${driver_version == 'eac'}">
+            <command_interface name="velocity"/>
+            <state_interface name="velocity">
+              <param name="initial_value">0.0</param>
+            </state_interface>
+          </xacro:unless>
+        </xacro:unless>
       </joint>
       <joint name="${prefix}joint_3">
         <command_interface name="position"/>
-        <xacro:unless value="${driver_version == 'eac'}">
-          <command_interface name="velocity"/>
-          <command_interface name="effort"/>
-        </xacro:unless>
-        <xacro:if value="${driver_version == 'eac' and mode != 'gazebo'}">
-          <command_interface name="stiffness"/>
-          <command_interface name="damping"/>
-          <command_interface name="effort"/>
-        </xacro:if>
         <state_interface name="position">
           <param name="initial_value">1.5708</param>
         </state_interface>
-        <xacro:unless value="${driver_version == 'eac'}">
-          <state_interface name="velocity"/>
-          <state_interface name="effort"/>
-        </xacro:unless>
-        <xacro:if value="${driver_version == 'eac'}">
-          <state_interface name="effort">
-            <param name="initial_value">0.0</param>
-          </state_interface>
-          <state_interface name="commanded_position">
-            <param name="initial_value">0.0</param>
-          </state_interface>
-        </xacro:if>
+        <xacro:unless value="${mode == 'gazebo'}">
+          <command_interface name="effort"/>
+          <state_interface name="effort">
+            <param name="initial_value">0.0</param>
+          </state_interface>
+          <xacro:if value="${driver_version == 'eac'}">
+            <command_interface name="stiffness"/>
+            <command_interface name="damping"/>
+            <state_interface name="commanded_position">
+              <param name="initial_value">0.0</param>
+            </state_interface>
+          </xacro:if>
+          <xacro:unless value="${driver_version == 'eac'}">
+            <command_interface name="velocity"/>
+            <state_interface name="velocity">
+              <param name="initial_value">0.0</param>
+            </state_interface>
+          </xacro:unless>
+        </xacro:unless>
       </joint>
       <joint name="${prefix}joint_4">
         <command_interface name="position"/>
-        <xacro:unless value="${driver_version == 'eac'}">
-          <command_interface name="velocity"/>
-          <command_interface name="effort"/>
-        </xacro:unless>
-        <xacro:if value="${driver_version == 'eac' and mode != 'gazebo'}">
-          <command_interface name="stiffness"/>
-          <command_interface name="damping"/>
-          <command_interface name="effort"/>
-        </xacro:if>
-        <state_interface name="position">
-          <param name="initial_value">0.0</param>
-        </state_interface>
-        <xacro:unless value="${driver_version == 'eac'}">
-          <state_interface name="velocity"/>
-          <state_interface name="effort"/>
-        </xacro:unless>
-        <xacro:if value="${driver_version == 'eac'}">
-          <state_interface name="effort">
-            <param name="initial_value">0.0</param>
-          </state_interface>
-          <state_interface name="commanded_position">
-            <param name="initial_value">0.0</param>
-          </state_interface>
-        </xacro:if>
+        <state_interface name="position">
+          <param name="initial_value">0.0</param>
+        </state_interface>
+        <xacro:unless value="${mode == 'gazebo'}">
+          <command_interface name="effort"/>
+          <state_interface name="effort">
+            <param name="initial_value">0.0</param>
+          </state_interface>
+          <xacro:if value="${driver_version == 'eac'}">
+            <command_interface name="stiffness"/>
+            <command_interface name="damping"/>
+            <state_interface name="commanded_position">
+              <param name="initial_value">0.0</param>
+            </state_interface>
+          </xacro:if>
+          <xacro:unless value="${driver_version == 'eac'}">
+            <command_interface name="velocity"/>
+            <state_interface name="velocity">
+              <param name="initial_value">0.0</param>
+            </state_interface>
+          </xacro:unless>
+        </xacro:unless>
       </joint>
       <joint name="${prefix}joint_5">
         <command_interface name="position"/>
-        <xacro:unless value="${driver_version == 'eac'}">
-          <command_interface name="velocity"/>
-          <command_interface name="effort"/>
-        </xacro:unless>
-        <xacro:if value="${driver_version == 'eac' and mode != 'gazebo'}">
-          <command_interface name="stiffness"/>
-          <command_interface name="damping"/>
-          <command_interface name="effort"/>
-        </xacro:if>
-        <state_interface name="position">
-          <param name="initial_value">0.0</param>
-        </state_interface>
-        <xacro:unless value="${driver_version == 'eac'}">
-          <state_interface name="velocity"/>
-          <state_interface name="effort"/>
-        </xacro:unless>
-        <xacro:if value="${driver_version == 'eac'}">
-          <state_interface name="effort">
-            <param name="initial_value">0.0</param>
-          </state_interface>
-          <state_interface name="commanded_position">
-            <param name="initial_value">0.0</param>
-          </state_interface>
-        </xacro:if>
+        <state_interface name="position">
+          <param name="initial_value">0.0</param>
+        </state_interface>
+        <xacro:unless value="${mode == 'gazebo'}">
+          <command_interface name="effort"/>
+          <state_interface name="effort">
+            <param name="initial_value">0.0</param>
+          </state_interface>
+          <xacro:if value="${driver_version == 'eac'}">
+            <command_interface name="stiffness"/>
+            <command_interface name="damping"/>
+            <state_interface name="commanded_position">
+              <param name="initial_value">0.0</param>
+            </state_interface>
+          </xacro:if>
+          <xacro:unless value="${driver_version == 'eac'}">
+            <command_interface name="velocity"/>
+            <state_interface name="velocity">
+              <param name="initial_value">0.0</param>
+            </state_interface>
+          </xacro:unless>
+        </xacro:unless>
       </joint>
       <joint name="${prefix}joint_6">
         <command_interface name="position"/>
-        <xacro:unless value="${driver_version == 'eac'}">
-          <command_interface name="velocity"/>
-          <command_interface name="effort"/>
-        </xacro:unless>
-        <xacro:if value="${driver_version == 'eac' and mode != 'gazebo'}">
-          <command_interface name="stiffness"/>
-          <command_interface name="damping"/>
-          <command_interface name="effort"/>
-        </xacro:if>
-        <state_interface name="position">
-          <param name="initial_value">0.0</param>
-        </state_interface>
-        <xacro:unless value="${driver_version == 'eac'}">
-          <state_interface name="velocity"/>
-          <state_interface name="effort"/>
-        </xacro:unless>
-        <xacro:if value="${driver_version == 'eac'}">
-          <state_interface name="effort">
-            <param name="initial_value">0.0</param>
-          </state_interface>
-          <state_interface name="commanded_position">
-            <param name="initial_value">0.0</param>
-          </state_interface>
-        </xacro:if>
+        <state_interface name="position">
+          <param name="initial_value">0.0</param>
+        </state_interface>
+        <xacro:unless value="${mode == 'gazebo'}">
+          <command_interface name="effort"/>
+          <state_interface name="effort">
+            <param name="initial_value">0.0</param>
+          </state_interface>
+          <xacro:if value="${driver_version == 'eac'}">
+            <command_interface name="stiffness"/>
+            <command_interface name="damping"/>
+            <state_interface name="commanded_position">
+              <param name="initial_value">0.0</param>
+            </state_interface>
+          </xacro:if>
+          <xacro:unless value="${driver_version == 'eac'}">
+            <command_interface name="velocity"/>
+            <state_interface name="velocity">
+              <param name="initial_value">0.0</param>
+            </state_interface>
+          </xacro:unless>
+        </xacro:unless>
       </joint>
       <xacro:if value="${use_gpio}">

File: kuka_quantec_support/urdf/kr_quantec_ros2_control_macro.xacro (robot description, xacro)
@@ -50,61 +50,97 @@
       <joint name="${prefix}joint_1">
         <command_interface name="position"/>
-        <command_interface name="velocity"/>
-        <command_interface name="effort"/>
         <state_interface name="position">
           <param name="initial_value">0.0</param>
         </state_interface>
-        <state_interface name="velocity"/>
-        <state_interface name="effort"/>
+        <xacro:unless value="${mode == 'gazebo'}">
+          <command_interface name="velocity"/>
+          <command_interface name="effort"/>
+          <state_interface name="velocity">
+            <param name="initial_value">0.0</param>
+          </state_interface>
+          <state_interface name="effort">
+            <param name="initial_value">0.0</param>
+          </state_interface>
+        </xacro:unless>
       </joint>
       <joint name="${prefix}joint_2">
         <command_interface name="position"/>
-        <command_interface name="velocity"/>
-        <command_interface name="effort"/>
         <state_interface name="position">
           <param name="initial_value">-1.5708</param>
         </state_interface>
-        <state_interface name="velocity"/>
-        <state_interface name="effort"/>
+        <xacro:unless value="${mode == 'gazebo'}">
+          <command_interface name="velocity"/>
+          <command_interface name="effort"/>
+          <state_interface name="velocity">
+            <param name="initial_value">0.0</param>
+          </state_interface>
+          <state_interface name="effort">
+            <param name="initial_value">0.0</param>
+          </state_interface>
+        </xacro:unless>
       </joint>
       <joint name="${prefix}joint_3">
         <command_interface name="position"/>
-        <command_interface name="velocity"/>
-        <command_interface name="effort"/>
         <state_interface name="position">
           <param name="initial_value">1.5708</param>
         </state_interface>
-        <state_interface name="velocity"/>
-        <state_interface name="effort"/>
+        <xacro:unless value="${mode == 'gazebo'}">
+          <command_interface name="velocity"/>
+          <command_interface name="effort"/>
+          <state_interface name="velocity">
+            <param name="initial_value">0.0</param>
+          </state_interface>
+          <state_interface name="effort">
+            <param name="initial_value">0.0</param>
+          </state_interface>
+        </xacro:unless>
       </joint>
       <joint name="${prefix}joint_4">
         <command_interface name="position"/>
-        <command_interface name="velocity"/>
-        <command_interface name="effort"/>
         <state_interface name="position">
           <param name="initial_value">0.0</param>
         </state_interface>
-        <state_interface name="velocity"/>
-        <state_interface name="effort"/>
+        <xacro:unless value="${mode == 'gazebo'}">
+          <command_interface name="velocity"/>
+          <command_interface name="effort"/>
+          <state_interface name="velocity">
+            <param name="initial_value">0.0</param>
+          </state_interface>
+          <state_interface name="effort">
+            <param name="initial_value">0.0</param>
+          </state_interface>
+        </xacro:unless>
       </joint>
       <joint name="${prefix}joint_5">
         <command_interface name="position"/>
-        <command_interface name="velocity"/>
-        <command_interface name="effort"/>
         <state_interface name="position">
           <param name="initial_value">0.0</param>
         </state_interface>
-        <state_interface name="velocity"/>
-        <state_interface name="effort"/>
+        <xacro:unless value="${mode == 'gazebo'}">
+          <command_interface name="velocity"/>
+          <command_interface name="effort"/>
+          <state_interface name="velocity">
+            <param name="initial_value">0.0</param>
+          </state_interface>
+          <state_interface name="effort">
+            <param name="initial_value">0.0</param>
+          </state_interface>
+        </xacro:unless>
       </joint>
       <joint name="${prefix}joint_6">
         <command_interface name="position"/>
-        <command_interface name="velocity"/>
-        <command_interface name="effort"/>
         <state_interface name="position">
           <param name="initial_value">0.0</param>
         </state_interface>
-        <state_interface name="velocity"/>
-        <state_interface name="effort"/>
+        <xacro:unless value="${mode == 'gazebo'}">
+          <command_interface name="velocity"/>
+          <command_interface name="effort"/>
+          <state_interface name="velocity">
+            <param name="initial_value">0.0</param>
+          </state_interface>
+          <state_interface name="effort">
+            <param name="initial_value">0.0</param>
+          </state_interface>
+        </xacro:unless>
       </joint>
       <xacro:if value="${use_gpio}">
