Commit message: add ext axis gazebo integration - mesh not ok in gz yet

File: kuka_agilus_support/urdf/kr_agilus_ros2_control_macro.xacro (robot description, xacro)
@@ -1,9 +1,9 @@
 <?xml version="1.0" encoding="UTF-8"?>
 <robot xmlns:xacro="http://www.ros.org/wiki/xacro">
-  <xacro:macro name="kuka_agilus_ros2_control" params="name driver_version client_ip client_port mxa_client_port controller_ip prefix mode use_gpio roundtrip_time verify_robot_model **ext_axes_ros2_control_joints">
+  <xacro:macro name="kuka_agilus_ros2_control" params="name driver_version client_ip client_port mxa_client_port controller_ip prefix mode use_gpio roundtrip_time verify_robot_model gazebo_controller_config_path:=config/fake_hardware_config_6_axis.yaml **ext_axes_ros2_control_joints">
     <!-- gazebo -->
     <xacro:if value="${mode == 'gazebo'}">
       <xacro:include filename="$(find kuka_gazebo)/gazebo/kuka_gazebo.xacro"/>
-      <xacro:kuka_gazebo controller_config_package="kuka_resources" controller_config_path="config/fake_hardware_config_6_axis.yaml"/>
+      <xacro:kuka_gazebo controller_config_package="kuka_resources" controller_config_path="${gazebo_controller_config_path}"/>
     </xacro:if>
     <!-- ros2 control -->

File: kuka_cybertech_support/urdf/kr_cybertech_ros2_control_macro.xacro (robot description, xacro)
@@ -1,9 +1,9 @@
 <?xml version="1.0" encoding="UTF-8"?>
 <robot xmlns:xacro="http://www.ros.org/wiki/xacro">
-  <xacro:macro name="kuka_cybertech_ros2_control" params="name driver_version client_ip client_port mxa_client_port controller_ip prefix mode use_gpio roundtrip_time verify_robot_model **ext_axes_ros2_control_joints">
+  <xacro:macro name="kuka_cybertech_ros2_control" params="name driver_version client_ip client_port mxa_client_port controller_ip prefix mode use_gpio roundtrip_time verify_robot_model gazebo_controller_config_path:=config/fake_hardware_config_6_axis.yaml **ext_axes_ros2_control_joints">
     <!-- gazebo -->
     <xacro:if value="${mode == 'gazebo'}">
       <xacro:include filename="$(find kuka_gazebo)/gazebo/kuka_gazebo.xacro"/>
-      <xacro:kuka_gazebo controller_config_package="kuka_resources" controller_config_path="config/fake_hardware_config_6_axis.yaml"/>
+      <xacro:kuka_gazebo controller_config_package="kuka_resources" controller_config_path="${gazebo_controller_config_path}"/>
     </xacro:if>
     <!-- ros2 control -->

File: kuka_fortec_support/urdf/kr_fortec_ros2_control_macro.xacro (robot description, xacro)
@@ -1,9 +1,9 @@
 <?xml version="1.0" encoding="UTF-8"?>
 <robot xmlns:xacro="http://www.ros.org/wiki/xacro">
-  <xacro:macro name="kuka_fortec_ros2_control" params="name driver_version client_ip client_port mxa_client_port controller_ip prefix mode use_gpio roundtrip_time verify_robot_model **ext_axes_ros2_control_joints">
+  <xacro:macro name="kuka_fortec_ros2_control" params="name driver_version client_ip client_port mxa_client_port controller_ip prefix mode use_gpio roundtrip_time verify_robot_model gazebo_controller_config_path:=config/fake_hardware_config_6_axis.yaml **ext_axes_ros2_control_joints">
     <!-- gazebo -->
     <xacro:if value="${mode == 'gazebo'}">
       <xacro:include filename="$(find kuka_gazebo)/gazebo/kuka_gazebo.xacro"/>
-      <xacro:kuka_gazebo controller_config_package="kuka_resources" controller_config_path="config/fake_hardware_config_6_axis.yaml"/>
+      <xacro:kuka_gazebo controller_config_package="kuka_resources" controller_config_path="${gazebo_controller_config_path}"/>
     </xacro:if>
     <!-- ros2 control -->

File: kuka_iontec_support/urdf/kr_iontec_ros2_control_macro.xacro (robot description, xacro)
@@ -1,9 +1,9 @@
 <?xml version="1.0" encoding="UTF-8"?>
 <robot xmlns:xacro="http://www.ros.org/wiki/xacro">
-  <xacro:macro name="kuka_iontec_ros2_control" params="name driver_version client_ip client_port mxa_client_port controller_ip prefix mode use_gpio roundtrip_time verify_robot_model **ext_axes_ros2_control_joints">
+  <xacro:macro name="kuka_iontec_ros2_control" params="name driver_version client_ip client_port mxa_client_port controller_ip prefix mode use_gpio roundtrip_time verify_robot_model gazebo_controller_config_path:=config/fake_hardware_config_6_axis.yaml **ext_axes_ros2_control_joints">
     <!-- gazebo -->
     <xacro:if value="${mode == 'gazebo'}">
       <xacro:include filename="$(find kuka_gazebo)/gazebo/kuka_gazebo.xacro"/>
-      <xacro:kuka_gazebo controller_config_package="kuka_resources" controller_config_path="config/fake_hardware_config_6_axis.yaml"/>
+      <xacro:kuka_gazebo controller_config_package="kuka_resources" controller_config_path="${gazebo_controller_config_path}"/>
     </xacro:if>
     <!-- ros2 control -->

File: kuka_kl_support/urdf/kl100_2_macro.xacro (robot description, xacro)
@@ -1,27 +1,37 @@
 <?xml version="1.0" encoding="UTF-8"?>
 <robot xmlns:xacro="http://www.ros.org/wiki/xacro">
-  <xacro:macro name="kl100_2_links" params="prefix">
+  <xacro:macro name="kl100_2_links" params="prefix package_name">
     <!-- links -->
     <link name="${prefix}base_link">
+      <inertial>
+        <origin rpy="0.0 0.0 0.0" xyz="0.0 0.0 0.0"/>
+        <mass value="500.0"/>
+        <inertia ixx="8" ixy="0.0" ixz="0.0" iyy="190" iyz="0.0" izz="190"/>
+      </inertial>
       <visual>
         <geometry>
-          <mesh filename="package://kuka_kl_support/meshes/kl100_2/visual/rail_base_link.dae"/>
+          <mesh filename="package://${package_name}/meshes/kl100_2/visual/rail_base_link.dae"/>
         </geometry>
       </visual>
       <collision>
         <geometry>
-          <mesh filename="package://kuka_kl_support/meshes/kl100_2/collision/rail_base_link.stl"/>
+          <mesh filename="package://${package_name}/meshes/kl100_2/collision/rail_base_link.stl"/>
         </geometry>
       </collision>
     </link>
     <link name="${prefix}link_1">
+      <inertial>
+        <origin rpy="0.0 0.0 0.0" xyz="0.0 0.0 0.0"/>
+        <mass value="43.0"/>
+        <inertia ixx="1.03" ixy="0.0" ixz="0.0" iyy="1.135" iyz="0.0" izz="1.517"/>
+      </inertial>
       <visual>
         <geometry>
-          <mesh filename="package://kuka_kl_support/meshes/kl100_2/visual/rail_moving_link.dae"/>
+          <mesh filename="package://${package_name}/meshes/kl100_2/visual/rail_moving_link.dae"/>
         </geometry>
       </visual>
       <collision>
         <geometry>
-          <mesh filename="package://kuka_kl_support/meshes/kl100_2/collision/rail_moving_link.stl"/>
+          <mesh filename="package://${package_name}/meshes/kl100_2/collision/rail_moving_link.stl"/>
         </geometry>
       </collision>
@@ -30,9 +40,4 @@
   <xacro:macro name="kl100_2_joints" params="prefix robot_base_link *origin">
     <!-- joints -->
-    <joint name="world-${prefix}base_link" type="fixed">
-      <parent link="world"/>
-      <child link="${prefix}base_link"/>
-      <xacro:insert_block name="origin"/>
-    </joint>
     <joint name="${prefix}joint_1" type="prismatic">
       <parent link="${prefix}base_link"/>

File: kuka_lbr_iisy_support/urdf/lbr_iisy_ros2_control_macro.xacro (robot description, xacro)
@@ -1,9 +1,9 @@
 <?xml version="1.0" encoding="UTF-8"?>
 <robot xmlns:xacro="http://www.ros.org/wiki/xacro">
-  <xacro:macro name="kuka_lbr_iisy_ros2_control" params="name driver_version prefix client_ip client_port mxa_client_port controller_ip use_gpio mode qos_config_file roundtrip_time verify_robot_model **ext_axes_ros2_control_joints">
+  <xacro:macro name="kuka_lbr_iisy_ros2_control" params="name driver_version prefix client_ip client_port mxa_client_port controller_ip use_gpio mode qos_config_file roundtrip_time verify_robot_model gazebo_controller_config_path:=config/fake_hardware_config_6_axis.yaml **ext_axes_ros2_control_joints">
     <!-- gazebo -->
     <xacro:if value="${mode == 'gazebo'}">
       <xacro:include filename="$(find kuka_gazebo)/gazebo/kuka_gazebo.xacro"/>
-      <xacro:kuka_gazebo controller_config_package="kuka_resources" controller_config_path="config/fake_hardware_config_6_axis.yaml"/>
+      <xacro:kuka_gazebo controller_config_package="kuka_resources" controller_config_path="${gazebo_controller_config_path}"/>
     </xacro:if>
     <!-- ros2 control -->

File: kuka_quantec_support/urdf/kr_quantec_ros2_control_macro.xacro (robot description, xacro)
@@ -1,9 +1,9 @@
 <?xml version="1.0" encoding="UTF-8"?>
 <robot xmlns:xacro="http://www.ros.org/wiki/xacro">
-  <xacro:macro name="kuka_quantec_ros2_control" params="name driver_version client_ip client_port mxa_client_port controller_ip prefix mode use_gpio roundtrip_time verify_robot_model **ext_axes_ros2_control_joints">
+  <xacro:macro name="kuka_quantec_ros2_control" params="name driver_version client_ip client_port mxa_client_port controller_ip prefix mode use_gpio roundtrip_time verify_robot_model gazebo_controller_config_path:=config/fake_hardware_config_6_axis.yaml **ext_axes_ros2_control_joints">
     <!-- gazebo -->
     <xacro:if value="${mode == 'gazebo'}">
       <xacro:include filename="$(find kuka_gazebo)/gazebo/kuka_gazebo.xacro"/>
-      <xacro:kuka_gazebo controller_config_package="kuka_resources" controller_config_path="config/fake_hardware_config_6_axis.yaml"/>
+      <xacro:kuka_gazebo controller_config_package="kuka_resources" controller_config_path="${gazebo_controller_config_path}"/>
     </xacro:if>
     <!-- ros2 control -->

File: kuka_resources/urdf/robot_with_external_axis_template.urdf.xacro (robot description, xacro)
@@ -26,4 +26,5 @@
   <xacro:arg name="robot_ros2_control_macro_file" default="kr_agilus_ros2_control_macro.xacro"/>
   <xacro:arg name="kl_model" default="kl100_2"/>
+  <xacro:arg name="gazebo_controller_config_path" default="config/fake_hardware_config_6_axis_kl.yaml"/>
   <!-- Define properties for dynamic macro and package resolution -->
   <xacro:property name="robot_family_value" value="$(arg robot_family)"/>
@@ -59,10 +60,4 @@
    />
   <xacro:property name="kl_full_prefix" value="${prefix_value + kl_prefix_value}"/>
-  <!-- gazebo -->
-  <xacro:property name="mode_value" value="$(arg mode)"/>
-  <xacro:if value="${mode_value == 'gazebo'}">
-    <xacro:include filename="$(find kuka_gazebo)/gazebo/kuka_gazebo.xacro"/>
-    <xacro:kuka_gazebo controller_config_package="kuka_resources" controller_config_path="config/fake_hardware_config_6_axis_kl.yaml"/>
-  </xacro:if>
   <!-- Include urdf macro files -->
   <xacro:include filename="${robot_support_urdf_dir}/${robot_model_value}_macro.xacro"/>
@@ -84,5 +79,6 @@
       qos_config_file=""
       roundtrip_time="$(arg roundtrip_time)"
-      verify_robot_model="$(arg verify_robot_model)">
+      verify_robot_model="$(arg verify_robot_model)"
+      gazebo_controller_config_path="$(arg gazebo_controller_config_path)">
       <ext_axes_ros2_control_joints>
         <xacro:kuka_kl_ros2_control_joints prefix="${kl_full_prefix}"/>
@@ -102,5 +98,6 @@
       mode="$(arg mode)"
       roundtrip_time="$(arg roundtrip_time)"
-      verify_robot_model="$(arg verify_robot_model)">
+      verify_robot_model="$(arg verify_robot_model)"
+      gazebo_controller_config_path="$(arg gazebo_controller_config_path)">
       <ext_axes_ros2_control_joints>
         <xacro:kuka_kl_ros2_control_joints prefix="${kl_full_prefix}"/>
@@ -109,7 +106,17 @@
   </xacro:unless>
   <!-- world link -->
-  <link name="world"/>
+    <link name="world"/>
+  <!-- default world - external-axis base joint -->
+    <joint name="world-${kl_full_prefix}base_link" type="fixed">
+      <parent link="world"/>
+      <child link="${kl_full_prefix}base_link"/>
+      <origin xyz="$(arg x) $(arg y) $(arg z)" rpy="$(arg roll) $(arg pitch) $(arg yaw)"/>
+    </joint>
   <!-- external axis links -->
-  <xacro:call macro="${kl_model_links_macro_name}" prefix="${kl_full_prefix}"/>
+  <xacro:call
+    macro="${kl_model_links_macro_name}"
+    prefix="${kl_full_prefix}"
+    package_name="${kl_urdf_package_value}"
+  />
   <!-- robot links -->
   <xacro:call
