Commit message: Add scheduling_policy argument to all robot models
Expose scheduling_policy as a top-level xacro argument, wired through
each per-model urdf.xacro into the family ros2_control macro, instead
of a hardcoded "detached" value. The async properties block is now
gated behind is_async, and read/write rate is made explicit on the
ros2_control tag for every family macro.

Co-Authored-By: Claude Sonnet 5 <noreply@anthropic.com>

File: kuka_agilus_support/urdf/kr_agilus_ros2_control_macro.xacro (robot description, xacro)
@@ -1,5 +1,5 @@
 <?xml version="1.0" encoding="UTF-8"?>
 <robot xmlns:xacro="http://www.ros.org/wiki/xacro">
-  <xacro:macro name="kuka_agilus_ros2_control" params="name driver_version client_ip client_port mxa_client_port controller_ip prefix mode use_gpio roundtrip_time verify_robot_model rsi_xml_config_file is_async async_thread_priority async_affinity gazebo_controller_config_path:=config/fake_hardware_config_6_axis.yaml **ext_axes_ros2_control_joints">
+  <xacro:macro name="kuka_agilus_ros2_control" params="name driver_version client_ip client_port mxa_client_port controller_ip prefix mode use_gpio roundtrip_time verify_robot_model rsi_xml_config_file is_async async_thread_priority async_affinity gazebo_controller_config_path:=config/fake_hardware_config_6_axis.yaml **ext_axes_ros2_control_joints scheduling_policy:=detached">
     <!-- gazebo -->
     <xacro:if value="${mode == 'gazebo'}">
@@ -8,8 +8,10 @@
     </xacro:if>
     <!-- ros2 control -->
-    <ros2_control name="${name}" type="system" is_async="${is_async}">
-      <properties>
-        <async affinity="${async_affinity}" scheduling_policy="detached" print_warnings="false" thread_priority="${async_thread_priority}"/>
-      </properties>
+    <ros2_control name="${name}" type="system" is_async="${is_async}" rw_rate="250">
+      <xacro:if value="${is_async}">
+        <properties>
+          <async affinity="${async_affinity}" scheduling_policy="${scheduling_policy}" print_warnings="false" thread_priority="${async_thread_priority}"/>
+        </properties>
+      </xacro:if>
       <hardware>
         <param name="interface_prefix">${prefix}</param>

File: kuka_cybertech_support/urdf/kr_cybertech_ros2_control_macro.xacro (robot description, xacro)
@@ -1,5 +1,5 @@
 <?xml version="1.0" encoding="UTF-8"?>
 <robot xmlns:xacro="http://www.ros.org/wiki/xacro">
-  <xacro:macro name="kuka_cybertech_ros2_control" params="name driver_version client_ip client_port mxa_client_port controller_ip prefix mode use_gpio roundtrip_time verify_robot_model rsi_xml_config_file is_async async_thread_priority async_affinity gazebo_controller_config_path:=config/fake_hardware_config_6_axis.yaml **ext_axes_ros2_control_joints">
+  <xacro:macro name="kuka_cybertech_ros2_control" params="name driver_version client_ip client_port mxa_client_port controller_ip prefix mode use_gpio roundtrip_time verify_robot_model rsi_xml_config_file is_async async_thread_priority async_affinity gazebo_controller_config_path:=config/fake_hardware_config_6_axis.yaml **ext_axes_ros2_control_joints scheduling_policy:=detached">
     <!-- gazebo -->
     <xacro:if value="${mode == 'gazebo'}">
@@ -9,7 +9,9 @@
     <!-- ros2 control -->
     <ros2_control name="${name}" type="system" is_async="${is_async}">
-      <properties>
-        <async affinity="${async_affinity}" scheduling_policy="detached" print_warnings="false" thread_priority="${async_thread_priority}"/>
-      </properties>
+      <xacro:if value="${is_async}">
+        <properties>
+          <async affinity="${async_affinity}" scheduling_policy="${scheduling_policy}" print_warnings="false" thread_priority="${async_thread_priority}"/>
+        </properties>
+      </xacro:if>
       <hardware>
         <param name="interface_prefix">${prefix}</param>

File: kuka_fortec_support/urdf/kr_fortec_ros2_control_macro.xacro (robot description, xacro)
@@ -1,5 +1,5 @@
 <?xml version="1.0" encoding="UTF-8"?>
 <robot xmlns:xacro="http://www.ros.org/wiki/xacro">
-  <xacro:macro name="kuka_fortec_ros2_control" params="name driver_version client_ip client_port mxa_client_port controller_ip prefix mode use_gpio roundtrip_time verify_robot_model rsi_xml_config_file is_async async_thread_priority async_affinity gazebo_controller_config_path:=config/fake_hardware_config_6_axis.yaml **ext_axes_ros2_control_joints">
+  <xacro:macro name="kuka_fortec_ros2_control" params="name driver_version client_ip client_port mxa_client_port controller_ip prefix mode use_gpio roundtrip_time verify_robot_model rsi_xml_config_file is_async async_thread_priority async_affinity gazebo_controller_config_path:=config/fake_hardware_config_6_axis.yaml **ext_axes_ros2_control_joints scheduling_policy:=detached">
     <!-- gazebo -->
     <xacro:if value="${mode == 'gazebo'}">
@@ -8,8 +8,10 @@
     </xacro:if>
     <!-- ros2 control -->
-    <ros2_control name="${name}" type="system" is_async="${is_async}">
-      <properties>
-        <async affinity="${async_affinity}" scheduling_policy="detached" print_warnings="false" thread_priority="${async_thread_priority}"/>
-      </properties>
+    <ros2_control name="${name}" type="system" is_async="${is_async}" rw_rate="250">
+      <xacro:if value="${is_async}">
+        <properties>
+          <async affinity="${async_affinity}" scheduling_policy="${scheduling_policy}" print_warnings="false" thread_priority="${async_thread_priority}"/>
+        </properties>
+      </xacro:if>
       <hardware>
         <param name="interface_prefix">${prefix}</param>

File: kuka_iontec_support/urdf/kr_iontec_ros2_control_macro.xacro (robot description, xacro)
@@ -1,5 +1,5 @@
 <?xml version="1.0" encoding="UTF-8"?>
 <robot xmlns:xacro="http://www.ros.org/wiki/xacro">
-  <xacro:macro name="kuka_iontec_ros2_control" params="name driver_version client_ip client_port mxa_client_port controller_ip prefix mode use_gpio roundtrip_time verify_robot_model rsi_xml_config_file is_async async_thread_priority async_affinity gazebo_controller_config_path:=config/fake_hardware_config_6_axis.yaml **ext_axes_ros2_control_joints">
+  <xacro:macro name="kuka_iontec_ros2_control" params="name driver_version client_ip client_port mxa_client_port controller_ip prefix mode use_gpio roundtrip_time verify_robot_model rsi_xml_config_file is_async async_thread_priority async_affinity gazebo_controller_config_path:=config/fake_hardware_config_6_axis.yaml **ext_axes_ros2_control_joints scheduling_policy:=detached">
     <!-- gazebo -->
     <xacro:if value="${mode == 'gazebo'}">
@@ -8,8 +8,10 @@
     </xacro:if>
     <!-- ros2 control -->
-    <ros2_control name="${name}" type="system" is_async="${is_async}">
-      <properties>
-        <async affinity="${async_affinity}" scheduling_policy="detached" print_warnings="false" thread_priority="${async_thread_priority}"/>
-      </properties>
+    <ros2_control name="${name}" type="system" is_async="${is_async}" rw_rate="250">
+      <xacro:if value="${is_async}">
+        <properties>
+          <async affinity="${async_affinity}" scheduling_policy="${scheduling_policy}" print_warnings="false" thread_priority="${async_thread_priority}"/>
+        </properties>
+      </xacro:if>
       <hardware>
         <param name="interface_prefix">${prefix}</param>

File: kuka_lbr_iico_support/urdf/lbr_iico_ros2_control_macro.xacro (robot description, xacro)
@@ -1,5 +1,5 @@
 <?xml version="1.0" encoding="UTF-8"?>
 <robot xmlns:xacro="http://www.ros.org/wiki/xacro">
-  <xacro:macro name="kuka_lbr_iico_ros2_control" params="name driver_version client_ip client_port mxa_client_port controller_ip prefix mode use_gpio roundtrip_time verify_robot_model rsi_xml_config_file is_async async_thread_priority async_affinity gazebo_controller_config_path:=config/fake_hardware_config_6_axis.yaml **ext_axes_ros2_control_joints">
+  <xacro:macro name="kuka_lbr_iico_ros2_control" params="name driver_version client_ip client_port mxa_client_port controller_ip prefix mode use_gpio roundtrip_time verify_robot_model rsi_xml_config_file is_async async_thread_priority async_affinity gazebo_controller_config_path:=config/fake_hardware_config_6_axis.yaml **ext_axes_ros2_control_joints scheduling_policy:=detached">
     <!-- gazebo -->
     <xacro:if value="${mode == 'gazebo'}">
@@ -8,8 +8,10 @@
     </xacro:if>
     <!-- ros2 control -->
-    <ros2_control name="${name}" type="system" is_async="${is_async}">
-      <properties>
-        <async affinity="${async_affinity}" scheduling_policy="detached" print_warnings="false" thread_priority="${async_thread_priority}"/>
-      </properties>
+    <ros2_control name="${name}" type="system" is_async="${is_async}" rw_rate="250">
+      <xacro:if value="${is_async}">
+        <properties>
+          <async affinity="${async_affinity}" scheduling_policy="${scheduling_policy}" print_warnings="false" thread_priority="${async_thread_priority}"/>
+        </properties>
+      </xacro:if>
       <hardware>
         <param name="interface_prefix">${prefix}</param>

File: kuka_lbr_iisy_support/urdf/lbr_iisy_ros2_control_macro.xacro (robot description, xacro)
@@ -1,5 +1,5 @@
 <?xml version="1.0" encoding="UTF-8"?>
 <robot xmlns:xacro="http://www.ros.org/wiki/xacro">
-  <xacro:macro name="kuka_lbr_iisy_ros2_control" params="name driver_version prefix client_ip client_port mxa_client_port controller_ip use_gpio mode qos_config_file='' roundtrip_time verify_robot_model rsi_xml_config_file is_async async_thread_priority async_affinity gazebo_controller_config_path:=config/fake_hardware_config_6_axis.yaml **ext_axes_ros2_control_joints">
+  <xacro:macro name="kuka_lbr_iisy_ros2_control" params="name driver_version prefix client_ip client_port mxa_client_port controller_ip use_gpio mode qos_config_file='' roundtrip_time verify_robot_model rsi_xml_config_file is_async async_thread_priority async_affinity gazebo_controller_config_path:=config/fake_hardware_config_6_axis.yaml **ext_axes_ros2_control_joints scheduling_policy:=detached">
     <!-- gazebo -->
     <xacro:if value="${mode == 'gazebo'}">
@@ -8,8 +8,10 @@
     </xacro:if>
     <!-- ros2 control -->
-    <ros2_control name="${name}" type="system" is_async="${is_async}">
-      <properties>
-        <async affinity="${async_affinity}" scheduling_policy="detached" print_warnings="false" thread_priority="${async_thread_priority}"/>
-      </properties>
+    <ros2_control name="${name}" type="system" is_async="${is_async}" rw_rate="250">
+      <xacro:if value="${is_async}">
+        <properties>
+          <async affinity="${async_affinity}" scheduling_policy="${scheduling_policy}" print_warnings="false" thread_priority="${async_thread_priority}"/>
+        </properties>
+      </xacro:if>
       <hardware>
         <param name="interface_prefix">${prefix}</param>

File: kuka_lbr_iiwa_support/urdf/lbr_iiwa_ros2_control_macro.xacro (robot description, xacro)
@@ -1,5 +1,5 @@
 <?xml version="1.0" encoding="UTF-8"?>
 <robot xmlns:xacro="http://www.ros.org/wiki/xacro">
-  <xacro:macro name="kuka_lbr_iiwa_ros2_control" params="name prefix io_access mode roundtrip_time controller_ip client_ip client_port is_async async_thread_priority async_affinity gazebo_controller_config_path:=config/fake_hardware_config_7_axis.yaml **ext_axes_ros2_control_joints">
+  <xacro:macro name="kuka_lbr_iiwa_ros2_control" params="name prefix io_access mode roundtrip_time controller_ip client_ip client_port is_async async_thread_priority async_affinity gazebo_controller_config_path:=config/fake_hardware_config_7_axis.yaml **ext_axes_ros2_control_joints scheduling_policy:=detached">
     <!-- gazebo -->
     <xacro:if value="${mode == 'gazebo'}">
@@ -8,8 +8,10 @@
     </xacro:if>
     <!-- ros2 control -->
-    <ros2_control name="${name}" type="system" is_async="${is_async}">
-      <properties>
-        <async affinity="${async_affinity}" scheduling_policy="detached" print_warnings="false" thread_priority="${async_thread_priority}"/>
-      </properties>
+    <ros2_control name="${name}" type="system" is_async="${is_async}" rw_rate="1000">
+      <xacro:if value="${is_async}">
+        <properties>
+          <async affinity="${async_affinity}" scheduling_policy="${scheduling_policy}" print_warnings="false" thread_priority="${async_thread_priority}"/>
+        </properties>
+      </xacro:if>
       <hardware>
         <param name="interface_prefix">${prefix}</param>

File: kuka_quantec_support/urdf/kr_quantec_ros2_control_macro.xacro (robot description, xacro)
@@ -1,5 +1,5 @@
 <?xml version="1.0" encoding="UTF-8"?>
 <robot xmlns:xacro="http://www.ros.org/wiki/xacro">
-  <xacro:macro name="kuka_quantec_ros2_control" params="name driver_version client_ip client_port mxa_client_port controller_ip prefix mode use_gpio roundtrip_time verify_robot_model rsi_xml_config_file is_async async_thread_priority async_affinity gazebo_controller_config_path:=config/fake_hardware_config_6_axis.yaml **ext_axes_ros2_control_joints">
+  <xacro:macro name="kuka_quantec_ros2_control" params="name driver_version client_ip client_port mxa_client_port controller_ip prefix mode use_gpio roundtrip_time verify_robot_model rsi_xml_config_file is_async async_thread_priority async_affinity gazebo_controller_config_path:=config/fake_hardware_config_6_axis.yaml **ext_axes_ros2_control_joints scheduling_policy:=detached">
     <!-- gazebo -->
     <xacro:if value="${mode == 'gazebo'}">
@@ -9,7 +9,9 @@
     <!-- ros2 control -->
     <ros2_control name="${name}" type="system" is_async="${is_async}">
-      <properties>
-        <async affinity="${async_affinity}" scheduling_policy="detached" print_warnings="false" thread_priority="${async_thread_priority}"/>
-      </properties>
+      <xacro:if value="${is_async}">
+        <properties>
+          <async affinity="${async_affinity}" scheduling_policy="${scheduling_policy}" print_warnings="false" thread_priority="${async_thread_priority}"/>
+        </properties>
+      </xacro:if>
       <hardware>
         <param name="interface_prefix">${prefix}</param>
