Commit message: adapt to conventions

File: kuka_agilus_support/urdf/kr10_r1100_2.urdf.xacro (robot description, xacro)
@@ -1,16 +1,8 @@
 <?xml version="1.0"?>
 <robot xmlns:xacro="http://www.ros.org/wiki/xacro" name="kr10_r1100_2">
-<!-- Import urdf file  -->
-<xacro:include filename="$(find kuka_agilus_support)/urdf/kr10_r1100_2_macro.xacro"/>
-<!-- Read parameters from rsi_config  -->
-<xacro:property name="rsi_config" value="$(find kuka_rsi_hw_interface)/config/rsi_config.yaml" />
-<xacro:property name="rsi_config_dict" value="${xacro.load_yaml(rsi_config)}"/>
-<xacro:property name="client_ip" value="${rsi_config_dict['client_ip']}" />
-<xacro:property name="client_port" value="${rsi_config_dict['client_port']}" />
-<!-- Read additional arguments  -->
-<xacro:arg name="use_fake_hardware" default="false" />
-<xacro:kuka_kr10_r1100_2_robot prefix=""
-                  client_ip="${client_ip}"
-                  client_port="${client_port}"
-                  use_fake_hardware="$(arg use_fake_hardware)"/>
+  <!-- Import urdf file  -->
+  <xacro:include filename="$(find kuka_agilus_support)/urdf/kr10_r1100_2_macro.xacro"/>
+  <!-- Read additional arguments  -->
+  <xacro:arg name="use_fake_hardware" default="false" />
+  <xacro:kuka_kr10_r1100_2_robot prefix="" use_fake_hardware="$(arg use_fake_hardware)"/>
 </robot>

File: kuka_agilus_support/urdf/kr10_r1100_2_macro.xacro (robot description, xacro)
@@ -5,11 +5,9 @@
   <xacro:include filename="$(find kuka_agilus_support)/urdf/kr_agilus_transmission.xacro" />
   <xacro:include filename="$(find kuka_resources)/urdf/common_materials.xacro"/>
-  <xacro:macro name="kuka_kr10_r1100_2_robot" params="prefix client_ip client_port use_fake_hardware">
+  <xacro:macro name="kuka_kr10_r1100_2_robot" params="prefix use_fake_hardware">
     <!-- ros2 control instance -->
     <xacro:kuka_agilus_ros2_control
     name="kr10_r1100_2"
     prefix="${prefix}"
-    client_ip="${client_ip}"
-    client_port="${client_port}"
     use_fake_hardware="${use_fake_hardware}" />
     <!-- links - main serial chain -->
@@ -162,5 +160,5 @@
       <origin xyz="0 0 0" rpy="0 0 0" />
     </joint>
-    <joint name="${prefix}joint_a1" type="revolute">
+    <joint name="${prefix}joint_1" type="revolute">
       <axis xyz="0.0 0.0 1.0" />
       <child link="${prefix}link_1" />
@@ -169,5 +167,5 @@
       <parent link="${prefix}base_link_inertia" />
     </joint>
-    <joint name="${prefix}joint_a2" type="revolute">
+    <joint name="${prefix}joint_2" type="revolute">
       <axis xyz="0.0 0.0 1.0" />
       <child link="${prefix}link_2" />
@@ -176,5 +174,5 @@
       <parent link="${prefix}link_1" />
     </joint>
-    <joint name="${prefix}joint_a3" type="revolute">
+    <joint name="${prefix}joint_3" type="revolute">
       <axis xyz="0.0 0.0 1.0" />
       <child link="${prefix}link_3" />
@@ -183,5 +181,5 @@
       <parent link="${prefix}link_2" />
     </joint>
-    <joint name="${prefix}joint_a4" type="revolute">
+    <joint name="${prefix}joint_4" type="revolute">
       <axis xyz="0.0 0.0 1.0" />
       <child link="${prefix}link_4" />
@@ -190,5 +188,5 @@
       <parent link="${prefix}link_3" />
     </joint>
-    <joint name="${prefix}joint_a5" type="revolute">
+    <joint name="${prefix}joint_5" type="revolute">
       <axis xyz="0.0 0.0 1.0" />
       <child link="${prefix}link_5" />
@@ -197,5 +195,5 @@
       <parent link="${prefix}link_4" />
     </joint>
-    <joint name="${prefix}joint_a6" type="revolute">
+    <joint name="${prefix}joint_6" type="revolute">
       <axis xyz="0.0 0.0 1.0" />
       <child link="${prefix}link_6" />

Commit message: kr ros2_control+ urdf.xacro rework

File: kuka_agilus_support/urdf/kr10_r1100_2.urdf.xacro (robot description, xacro)
@@ -5,4 +5,19 @@
   <!-- Read additional arguments  -->
   <xacro:arg name="use_fake_hardware" default="false" />
-  <xacro:kuka_kr10_r1100_2_robot prefix="" use_fake_hardware="$(arg use_fake_hardware)"/>
+  <xacro:arg name="client_ip" default="0.0.0.0" />
+  <xacro:arg name="client_port" default="59152" />
+  <xacro:arg name="prefix" default="" />
+  <xacro:arg name="x" default="0" />
+  <xacro:arg name="y" default="0" />
+  <xacro:arg name="z" default="0" />
+  <xacro:arg name="roll" default="0" />
+  <xacro:arg name="pitch" default="0" />
+  <xacro:arg name="yaw" default="0" />
+  <xacro:kuka_kr10_r1100_2_robot
+    client_ip="$(arg client_ip)"
+    client_port="$(arg client_port)"
+    prefix="$(arg prefix)"
+    use_fake_hardware="$(arg use_fake_hardware)">
+    <origin xyz="$(arg x) $(arg y) $(arg z)" rpy="$(arg roll) $(arg pitch) $(arg yaw)" />
+  </xacro:kuka_kr10_r1100_2_robot>
 </robot>

File: kuka_agilus_support/urdf/kr6_r700_sixx.urdf.xacro (robot description, xacro)
@@ -5,4 +5,19 @@
   <!-- Read additional arguments  -->
   <xacro:arg name="use_fake_hardware" default="false" />
-  <xacro:kuka_kr6_r700_sixx_robot prefix=""  use_fake_hardware="$(arg use_fake_hardware)"/>
+  <xacro:arg name="client_ip" default="0.0.0.0" />
+  <xacro:arg name="client_port" default="59152" />
+  <xacro:arg name="prefix" default="" />
+  <xacro:arg name="x" default="0" />
+  <xacro:arg name="y" default="0" />
+  <xacro:arg name="z" default="0" />
+  <xacro:arg name="roll" default="0" />
+  <xacro:arg name="pitch" default="0" />
+  <xacro:arg name="yaw" default="0" />
+  <xacro:kuka_kr6_r700_sixx_robot
+    client_ip="$(arg client_ip)"
+    client_port="$(arg client_port)"
+    prefix="$(arg prefix)"
+    use_fake_hardware="$(arg use_fake_hardware)">
+    <origin xyz="$(arg x) $(arg y) $(arg z)" rpy="$(arg roll) $(arg pitch) $(arg yaw)" />
+  </xacro:kuka_kr6_r700_sixx_robot>
 </robot>

File: kuka_agilus_support/urdf/kr6_r900_sixx.urdf.xacro (robot description, xacro)
@@ -5,4 +5,19 @@
   <!-- Read additional arguments  -->
   <xacro:arg name="use_fake_hardware" default="false" />
-  <xacro:kuka_kr6_r900_sixx_robot prefix="" use_fake_hardware="$(arg use_fake_hardware)"/>
+  <xacro:arg name="client_ip" default="0.0.0.0" />
+  <xacro:arg name="client_port" default="59152" />
+  <xacro:arg name="prefix" default="" />
+  <xacro:arg name="x" default="0" />
+  <xacro:arg name="y" default="0" />
+  <xacro:arg name="z" default="0" />
+  <xacro:arg name="roll" default="0" />
+  <xacro:arg name="pitch" default="0" />
+  <xacro:arg name="yaw" default="0" />
+  <xacro:kuka_kr6_r900_sixx_robot
+    client_ip="$(arg client_ip)"
+    client_port="$(arg client_port)"
+    prefix="$(arg prefix)"
+    use_fake_hardware="$(arg use_fake_hardware)">
+    <origin xyz="$(arg x) $(arg y) $(arg z)" rpy="$(arg roll) $(arg pitch) $(arg yaw)" />
+  </xacro:kuka_kr6_r900_sixx_robot>
 </robot>

File: kuka_agilus_support/urdf/kr_agilus_ros2_control.xacro (robot description, xacro)
@@ -1,5 +1,5 @@
 <?xml version="1.0" encoding="UTF-8"?>
 <robot xmlns:xacro="http://www.ros.org/wiki/xacro">
-  <xacro:macro name="kuka_agilus_ros2_control" params="name prefix use_fake_hardware:=false">
+  <xacro:macro name="kuka_agilus_ros2_control" params="name client_ip client_port prefix use_fake_hardware:=false">
     <ros2_control name="${name}" type="system">
       <hardware>
@@ -10,9 +10,4 @@
         </xacro:if>
         <xacro:unless value="${use_fake_hardware}">
-          <!-- Read parameters from rsi_config  -->
-          <xacro:property name="rsi_config" value="$(find kuka_kss_rsi_driver)/config/driver_config.yaml" />
-          <xacro:property name="rsi_config_dict" value="${xacro.load_yaml(rsi_config)}"/>
-          <xacro:property name="client_ip" value="${rsi_config_dict['client_ip']}" />
-          <xacro:property name="client_port" value="${rsi_config_dict['client_port']}" />
           <plugin>kuka_kss_rsi_driver::KukaRSIHardwareInterface</plugin>
           <param name="client_ip">${client_ip}</param>

File: kuka_cybertech_support/urdf/kr16_r2010_2.urdf.xacro (robot description, xacro)
@@ -5,4 +5,19 @@
   <!-- Read additional arguments  -->
   <xacro:arg name="use_fake_hardware" default="false" />
-  <xacro:kuka_kr16_r2010_2_robot prefix="" use_fake_hardware="$(arg use_fake_hardware)"/>
+  <xacro:arg name="client_ip" default="0.0.0.0" />
+  <xacro:arg name="client_port" default="59152" />
+  <xacro:arg name="prefix" default="" />
+  <xacro:arg name="x" default="0" />
+  <xacro:arg name="y" default="0" />
+  <xacro:arg name="z" default="0" />
+  <xacro:arg name="roll" default="0" />
+  <xacro:arg name="pitch" default="0" />
+  <xacro:arg name="yaw" default="0" />
+  <xacro:kuka_kr16_r2010_2_robot
+    client_ip="$(arg client_ip)"
+    client_port="$(arg client_port)"
+    prefix="$(arg prefix)"
+    use_fake_hardware="$(arg use_fake_hardware)">
+    <origin xyz="$(arg x) $(arg y) $(arg z)" rpy="$(arg roll) $(arg pitch) $(arg yaw)" />
+  </xacro:kuka_kr16_r2010_2_robot>
 </robot>

File: kuka_cybertech_support/urdf/kr_cybertech_ros2_control.xacro (robot description, xacro)
@@ -1,5 +1,5 @@
 <?xml version="1.0" encoding="UTF-8"?>
 <robot xmlns:xacro="http://www.ros.org/wiki/xacro">
-  <xacro:macro name="kuka_cybertech_ros2_control" params="name prefix use_fake_hardware:=false">
+  <xacro:macro name="kuka_cybertech_ros2_control" params="name client_ip client_port prefix use_fake_hardware:=false">
     <ros2_control name="${name}" type="system">
       <hardware>
@@ -10,9 +10,4 @@
         </xacro:if>
         <xacro:unless value="${use_fake_hardware}">
-          <!-- Read parameters from rsi_config  -->
-          <xacro:property name="rsi_config" value="$(find kuka_kss_rsi_driver)/config/driver_config.yaml" />
-          <xacro:property name="rsi_config_dict" value="${xacro.load_yaml(rsi_config)}"/>
-          <xacro:property name="client_ip" value="${rsi_config_dict['client_ip']}" />
-          <xacro:property name="client_port" value="${rsi_config_dict['client_port']}" />
           <plugin>kuka_kss_rsi_driver::KukaRSIHardwareInterface</plugin>
           <param name="client_ip">${client_ip}</param>

File: kuka_quantec_support/urdf/kr210_r2700_2.urdf.xacro (robot description, xacro)
@@ -5,4 +5,19 @@
   <!-- Read additional arguments  -->
   <xacro:arg name="use_fake_hardware" default="false" />
-  <xacro:kuka_kr210_r2700_2_robot prefix="" use_fake_hardware="$(arg use_fake_hardware)"/>
+  <xacro:arg name="client_ip" default="0.0.0.0" />
+  <xacro:arg name="client_port" default="59152" />
+  <xacro:arg name="prefix" default="" />
+  <xacro:arg name="x" default="0" />
+  <xacro:arg name="y" default="0" />
+  <xacro:arg name="z" default="0" />
+  <xacro:arg name="roll" default="0" />
+  <xacro:arg name="pitch" default="0" />
+  <xacro:arg name="yaw" default="0" />
+  <xacro:kuka_kr210_r2700_2_robot
+    client_ip="$(arg client_ip)"
+    client_port="$(arg client_port)"
+    prefix="$(arg prefix)"
+    use_fake_hardware="$(arg use_fake_hardware)">
+    <origin xyz="$(arg x) $(arg y) $(arg z)" rpy="$(arg roll) $(arg pitch) $(arg yaw)" />
+  </xacro:kuka_kr210_r2700_2_robot>
 </robot>

File: kuka_quantec_support/urdf/kr210_r3100_2.urdf.xacro (robot description, xacro)
@@ -5,4 +5,19 @@
   <!-- Read additional arguments  -->
   <xacro:arg name="use_fake_hardware" default="false" />
-  <xacro:kuka_kr210_r3100_2_robot prefix="" use_fake_hardware="$(arg use_fake_hardware)"/>
+  <xacro:arg name="client_ip" default="0.0.0.0" />
+  <xacro:arg name="client_port" default="59152" />
+  <xacro:arg name="prefix" default="" />
+  <xacro:arg name="x" default="0" />
+  <xacro:arg name="y" default="0" />
+  <xacro:arg name="z" default="0" />
+  <xacro:arg name="roll" default="0" />
+  <xacro:arg name="pitch" default="0" />
+  <xacro:arg name="yaw" default="0" />
+  <xacro:kuka_kr210_r3100_2_robot
+    client_ip="$(arg client_ip)"
+    client_port="$(arg client_port)"
+    prefix="$(arg prefix)"
+    use_fake_hardware="$(arg use_fake_hardware)">
+    <origin xyz="$(arg x) $(arg y) $(arg z)" rpy="$(arg roll) $(arg pitch) $(arg yaw)" />
+  </xacro:kuka_kr210_r3100_2_robot>
 </robot>

File: kuka_quantec_support/urdf/kr_quantec_ros2_control.xacro (robot description, xacro)
@@ -1,5 +1,5 @@
 <?xml version="1.0" encoding="UTF-8"?>
 <robot xmlns:xacro="http://www.ros.org/wiki/xacro">
-  <xacro:macro name="kuka_quantec_ros2_control" params="name prefix use_fake_hardware:=false">
+  <xacro:macro name="kuka_quantec_ros2_control" params="name client_ip client_port prefix use_fake_hardware:=false">
     <ros2_control name="${name}" type="system">
       <hardware>
@@ -10,9 +10,4 @@
         </xacro:if>
         <xacro:unless value="${use_fake_hardware}">
-          <!-- Read parameters from rsi_config  -->
-          <xacro:property name="rsi_config" value="$(find kuka_kss_rsi_driver)/config/driver_config.yaml" />
-          <xacro:property name="rsi_config_dict" value="${xacro.load_yaml(rsi_config)}"/>
-          <xacro:property name="client_ip" value="${rsi_config_dict['client_ip']}" />
-          <xacro:property name="client_port" value="${rsi_config_dict['client_port']}" />
           <plugin>kuka_kss_rsi_driver::KukaRSIHardwareInterface</plugin>
           <param name="client_ip">${client_ip}</param>

Commit message: Rename fake hardware naming

File: kuka_agilus_support/urdf/kr10_r1100_2.urdf.xacro (robot description, xacro)
@@ -5,5 +5,5 @@
   <!-- Read additional arguments  -->
   <xacro:arg name="use_fake_hardware" default="false"/>
-  <xacro:arg name="enable_isaac_sim" default="false"/>
+  <xacro:arg name="fake_hardware_type" default="false"/>
   <xacro:arg name="client_ip" default="0.0.0.0"/>
   <xacro:arg name="client_port" default="59152"/>
@@ -15,5 +15,5 @@
   <xacro:arg name="pitch" default="0"/>
   <xacro:arg name="yaw" default="0"/>
-  <xacro:kuka_kr10_r1100_2_robot client_ip="$(arg client_ip)" client_port="$(arg client_port)" prefix="$(arg prefix)" use_fake_hardware="$(arg use_fake_hardware)" enable_isaac_sim="$(arg enable_isaac_sim)">
+  <xacro:kuka_kr10_r1100_2_robot client_ip="$(arg client_ip)" client_port="$(arg client_port)" prefix="$(arg prefix)" use_fake_hardware="$(arg use_fake_hardware)" fake_hardware_type="$(arg fake_hardware_type)">
     <origin xyz="$(arg x) $(arg y) $(arg z)" rpy="$(arg roll) $(arg pitch) $(arg yaw)"/>
   </xacro:kuka_kr10_r1100_2_robot>

File: kuka_agilus_support/urdf/kr10_r1100_2_macro.xacro (robot description, xacro)
@@ -5,7 +5,7 @@
   <xacro:include filename="$(find kuka_agilus_support)/urdf/kr_agilus_transmission.xacro"/>
   <xacro:include filename="$(find kuka_resources)/urdf/common_materials.xacro"/>
-  <xacro:macro name="kuka_kr10_r1100_2_robot" params="client_ip client_port prefix use_fake_hardware enable_isaac_sim *origin">
+  <xacro:macro name="kuka_kr10_r1100_2_robot" params="client_ip client_port prefix use_fake_hardware fake_hardware_type *origin">
     <!-- ros2 control instance -->
-    <xacro:kuka_agilus_ros2_control name="${prefix}kr10_r1100_2" client_ip="${client_ip}" client_port="${client_port}" prefix="${prefix}" use_fake_hardware="${use_fake_hardware}" enable_isaac_sim="${enable_isaac_sim}"/>
+    <xacro:kuka_agilus_ros2_control name="${prefix}kr10_r1100_2" client_ip="${client_ip}" client_port="${client_port}" prefix="${prefix}" use_fake_hardware="${use_fake_hardware}" fake_hardware_type="${fake_hardware_type}"/>
     <!-- links - main serial chain -->
     <link name="world"/>

File: kuka_agilus_support/urdf/kr6_r700_sixx.urdf.xacro (robot description, xacro)
@@ -5,5 +5,5 @@
   <!-- Read additional arguments  -->
   <xacro:arg name="use_fake_hardware" default="false"/>
-  <xacro:arg name="enable_isaac_sim" default="false"/>
+  <xacro:arg name="fake_hardware_type" default="false"/>
   <xacro:arg name="client_ip" default="0.0.0.0"/>
   <xacro:arg name="client_port" default="59152"/>
@@ -15,5 +15,5 @@
   <xacro:arg name="pitch" default="0"/>
   <xacro:arg name="yaw" default="0"/>
-  <xacro:kuka_kr6_r700_sixx_robot client_ip="$(arg client_ip)" client_port="$(arg client_port)" prefix="$(arg prefix)" use_fake_hardware="$(arg use_fake_hardware)" enable_isaac_sim="$(arg enable_isaac_sim)">
+  <xacro:kuka_kr6_r700_sixx_robot client_ip="$(arg client_ip)" client_port="$(arg client_port)" prefix="$(arg prefix)" use_fake_hardware="$(arg use_fake_hardware)" fake_hardware_type="$(arg fake_hardware_type)">
     <origin xyz="$(arg x) $(arg y) $(arg z)" rpy="$(arg roll) $(arg pitch) $(arg yaw)"/>
   </xacro:kuka_kr6_r700_sixx_robot>

File: kuka_agilus_support/urdf/kr6_r700_sixx_macro.xacro (robot description, xacro)
@@ -5,7 +5,7 @@
   <xacro:include filename="$(find kuka_agilus_support)/urdf/kr_agilus_ros2_control.xacro"/>
   <xacro:include filename="$(find kuka_agilus_support)/urdf/kr_agilus_transmission.xacro"/>
-  <xacro:macro name="kuka_kr6_r700_sixx_robot" params="client_ip client_port prefix use_fake_hardware enable_isaac_sim *origin">
+  <xacro:macro name="kuka_kr6_r700_sixx_robot" params="client_ip client_port prefix use_fake_hardware fake_hardware_type *origin">
     <!-- ros2 control instance -->
-    <xacro:kuka_agilus_ros2_control name="${prefix}kr6_r700_sixx" client_ip="${client_ip}" client_port="${client_port}" prefix="${prefix}" use_fake_hardware="${use_fake_hardware}" enable_isaac_sim="${enable_isaac_sim}"/>
+    <xacro:kuka_agilus_ros2_control name="${prefix}kr6_r700_sixx" client_ip="${client_ip}" client_port="${client_port}" prefix="${prefix}" use_fake_hardware="${use_fake_hardware}" fake_hardware_type="${fake_hardware_type}"/>
     <link name="world"/>
     <link name="${prefix}base_link">

File: kuka_agilus_support/urdf/kr6_r900_sixx.urdf.xacro (robot description, xacro)
@@ -5,5 +5,5 @@
   <!-- Read additional arguments  -->
   <xacro:arg name="use_fake_hardware" default="false"/>
-  <xacro:arg name="enable_isaac_sim" default="false"/>
+  <xacro:arg name="fake_hardware_type" default="false"/>
   <xacro:arg name="client_ip" default="0.0.0.0"/>
   <xacro:arg name="client_port" default="59152"/>
@@ -15,5 +15,5 @@
   <xacro:arg name="pitch" default="0"/>
   <xacro:arg name="yaw" default="0"/>
-  <xacro:kuka_kr6_r900_sixx_robot client_ip="$(arg client_ip)" client_port="$(arg client_port)" prefix="$(arg prefix)" use_fake_hardware="$(arg use_fake_hardware)" enable_isaac_sim="$(arg enable_isaac_sim)">
+  <xacro:kuka_kr6_r900_sixx_robot client_ip="$(arg client_ip)" client_port="$(arg client_port)" prefix="$(arg prefix)" use_fake_hardware="$(arg use_fake_hardware)" fake_hardware_type="$(arg fake_hardware_type)">
     <origin xyz="$(arg x) $(arg y) $(arg z)" rpy="$(arg roll) $(arg pitch) $(arg yaw)"/>
   </xacro:kuka_kr6_r900_sixx_robot>

File: kuka_agilus_support/urdf/kr6_r900_sixx_macro.xacro (robot description, xacro)
@@ -5,7 +5,7 @@
   <xacro:include filename="$(find kuka_agilus_support)/urdf/kr_agilus_ros2_control.xacro"/>
   <xacro:include filename="$(find kuka_agilus_support)/urdf/kr_agilus_transmission.xacro"/>
-  <xacro:macro name="kuka_kr6_r900_sixx_robot" params="client_ip client_port prefix use_fake_hardware enable_isaac_sim *origin">
+  <xacro:macro name="kuka_kr6_r900_sixx_robot" params="client_ip client_port prefix use_fake_hardware fake_hardware_type *origin">
     <!-- ros2 control instance -->
-    <xacro:kuka_agilus_ros2_control name="${prefix}kr6_r900_sixx" client_ip="${client_ip}" client_port="${client_port}" prefix="${prefix}" use_fake_hardware="${use_fake_hardware}" enable_isaac_sim="${enable_isaac_sim}"/>
+    <xacro:kuka_agilus_ros2_control name="${prefix}kr6_r900_sixx" client_ip="${client_ip}" client_port="${client_port}" prefix="${prefix}" use_fake_hardware="${use_fake_hardware}" fake_hardware_type="${fake_hardware_type}"/>
     <link name="world"/>
     <link name="${prefix}base_link">

File: kuka_agilus_support/urdf/kr_agilus_ros2_control.xacro (robot description, xacro)
@@ -1,14 +1,14 @@
 <?xml version="1.0" encoding="UTF-8"?>
 <robot xmlns:xacro="http://www.ros.org/wiki/xacro">
-  <xacro:macro name="kuka_agilus_ros2_control" params="name client_ip client_port prefix use_fake_hardware enable_isaac_sim">
+  <xacro:macro name="kuka_agilus_ros2_control" params="name client_ip client_port prefix use_fake_hardware fake_hardware_type">
     <ros2_control name="${name}" type="system">
       <hardware>
         <xacro:if value="${use_fake_hardware}">
-          <xacro:if value="${enable_isaac_sim}">
+          <xacro:if value="${fake_hardware_type}">
             <plugin>topic_based_ros2_control/TopicBasedSystem</plugin>
             <param name="joint_commands_topic">/joint_commands</param>
             <param name="joint_states_topic">/joint_states</param>
           </xacro:if>
-          <xacro:unless value="${enable_isaac_sim}">
+          <xacro:unless value="${fake_hardware_type}">
             <plugin>mock_components/GenericSystem</plugin>
             <param name="mock_sensor_commands">false</param>
