Commit message: initial go at integrating ext axes, TODO find the pkg structure that fits best

File: kuka_agilus_support/urdf/kr10_r1100_2.urdf.xacro (robot description, xacro)
@@ -4,8 +4,10 @@
   <xacro:include filename="$(find kuka_agilus_support)/urdf/kr10_r1100_2_macro.xacro"/>
   <xacro:include filename="$(find kuka_agilus_support)/urdf/kr_agilus_ros2_control_macro.xacro"/>
+  <xacro:include filename="$(find kuka_agilus_support)/urdf/dummy_rail.xacro"/>
   <!-- Read additional arguments  -->
   <xacro:arg name="driver_version" default="rsi_only"/>
   <xacro:arg name="mode" default="hardware"/>
   <xacro:arg name="use_gpio" default="false"/>
+  <xacro:arg name="use_ext_axes" default="true"/>
   <xacro:arg name="roundtrip_time" default="0"/>
   <xacro:arg name="client_ip" default="0.0.0.0"/>
@@ -20,7 +22,17 @@
   <xacro:arg name="pitch" default="0"/>
   <xacro:arg name="yaw" default="0"/>
-  <xacro:kuka_agilus_ros2_control name="$(arg prefix)kr10_r1100_2" driver_version="$(arg driver_version)" client_ip="$(arg client_ip)" client_port="$(arg client_port)" controller_ip="$(arg controller_ip)" prefix="$(arg prefix)" mode="$(arg mode)" use_gpio="$(arg use_gpio)" roundtrip_time="$(arg roundtrip_time)" verify_robot_model="$(arg verify_robot_model)"/>
-  <xacro:kuka_kr10_r1100_2_robot prefix="$(arg prefix)" package_name="kuka_agilus_support">
+  <xacro:kuka_agilus_ros2_control name="$(arg prefix)kr10_r1100_2" driver_version="$(arg driver_version)" client_ip="$(arg client_ip)" client_port="$(arg client_port)" controller_ip="$(arg controller_ip)" prefix="$(arg prefix)" mode="$(arg mode)" use_gpio="$(arg use_gpio)" roundtrip_time="$(arg roundtrip_time)" verify_robot_model="$(arg verify_robot_model)" use_ext_axes="$(arg use_ext_axes)">
+    <ext_axes_ros2_control_joints>
+      <xacro:dummy_rail_ext_axes_ros2_control_joints/>
+    </ext_axes_ros2_control_joints>
+  </xacro:kuka_agilus_ros2_control>
+  <xacro:kuka_kr10_r1100_2_robot prefix="$(arg prefix)" package_name="kuka_agilus_support" use_ext_axes="$(arg use_ext_axes)">
     <origin xyz="$(arg x) $(arg y) $(arg z)" rpy="$(arg roll) $(arg pitch) $(arg yaw)"/>
+    <ext_axes_links>
+      <xacro:dummy_rail_ext_axes_links/>
+    </ext_axes_links>
+    <ext_axes_joints>
+      <xacro:dummy_rail_ext_axes_joints robot_base_link="$(arg prefix)base_link"/>
+    </ext_axes_joints>
   </xacro:kuka_kr10_r1100_2_robot>
 </robot>

File: kuka_agilus_support/urdf/kr10_r1100_2_macro.xacro (robot description, xacro)
@@ -3,7 +3,10 @@
   <!-- include helper xacros -->
   <xacro:include filename="$(find kuka_resources)/urdf/common_materials.xacro"/>
-  <xacro:macro name="kuka_kr10_r1100_2_robot" params="prefix package_name *origin">
+  <xacro:macro name="kuka_kr10_r1100_2_robot" params="prefix package_name use_ext_axes *origin **ext_axes_links **ext_axes_joints">
     <!-- links - main serial chain -->
     <link name="world"/>
+    <xacro:if value="${use_ext_axes}">
+      <xacro:insert_block name="ext_axes_links"/>
+    </xacro:if>
     <link name="${prefix}base_link">
       <collision>
@@ -147,9 +150,14 @@
     </link>
     <!-- joints - main serial chain -->
-    <joint name="${prefix}world-base_link" type="fixed">
-      <parent link="world"/>
-      <child link="${prefix}base_link"/>
-      <xacro:insert_block name="origin"/>
-    </joint>
+    <xacro:if value="${use_ext_axes}">
+      <xacro:insert_block name="ext_axes_joints"/>
+    </xacro:if>
+    <xacro:unless value="${use_ext_axes}">
+      <joint name="${prefix}world-base_link" type="fixed">
+        <parent link="world"/>
+        <child link="${prefix}base_link"/>
+        <xacro:insert_block name="origin"/>
+      </joint>
+    </xacro:unless>
     <joint name="${prefix}joint_1" type="revolute">
       <axis xyz="0.0 0.0 1.0"/>

File: kuka_agilus_support/urdf/kr_agilus_ros2_control_macro.xacro (robot description, xacro)
@@ -1,5 +1,5 @@
 <?xml version="1.0" encoding="UTF-8"?>
 <robot xmlns:xacro="http://www.ros.org/wiki/xacro">
-  <xacro:macro name="kuka_agilus_ros2_control" params="name driver_version client_ip client_port controller_ip prefix mode use_gpio roundtrip_time verify_robot_model">
+  <xacro:macro name="kuka_agilus_ros2_control" params="name driver_version client_ip client_port controller_ip prefix mode use_gpio roundtrip_time verify_robot_model use_ext_axes **ext_axes_ros2_control_joints">
     <!-- gazebo -->
     <xacro:if value="${mode == 'gazebo'}">
@@ -32,4 +32,7 @@
         </xacro:if>
       </hardware>
+      <xacro:if value="${use_ext_axes}">
+        <xacro:insert_block name="ext_axes_ros2_control_joints"/>
+      </xacro:if>
       <joint name="${prefix}joint_1">
         <command_interface name="position"/>
