Commit message: Fix KR 10 R1100-2 mesh

File: kuka_agilus_support/urdf/kr10_r1100_2.urdf.xacro (robot description, xacro)
@@ -21,5 +21,5 @@
   <xacro:arg name="pitch" default="0"/>
   <xacro:arg name="yaw" default="0"/>
-  <xacro:kuka_agilus_ros2_control name="$(arg prefix)kr10_r1100_2" driver_version="$(arg driver_version)" client_ip="$(arg client_ip)" client_port="$(arg client_port)" controller_ip="$(arg controller_ip)" prefix="$(arg prefix)" mode="$(arg mode)" use_gpio="$(arg use_gpio)" roundtrip_time="$(arg roundtrip_time)" verify_robot_model="$(arg verify_robot_model)">
+  <xacro:kuka_agilus_ros2_control name="$(arg prefix)kr10_r1100_2" driver_version="$(arg driver_version)" client_ip="$(arg client_ip)" client_port="$(arg client_port)" mxa_client_port="$(arg mxa_client_port)" controller_ip="$(arg controller_ip)" prefix="$(arg prefix)" mode="$(arg mode)" use_gpio="$(arg use_gpio)" roundtrip_time="$(arg roundtrip_time)" verify_robot_model="$(arg verify_robot_model)">
     <ext_axes_ros2_control_joints/>
   </xacro:kuka_agilus_ros2_control>

File: kuka_agilus_support/urdf/kr10_r1100_2_macro.xacro (robot description, xacro)
@@ -1,8 +1,6 @@
-<?xml version="1.0" encoding="UTF-8"?>
+<?xml version='1.0' encoding='UTF-8'?>
 <robot xmlns:xacro="http://www.ros.org/wiki/xacro" name="kr10_r1100_2">
-  <!-- include helper xacros -->
-  <xacro:include filename="$(find kuka_resources)/urdf/common_materials.xacro"/>
   <xacro:macro name="kuka_kr10_r1100_2_robot" params="prefix package_name">
-    <!-- links - main serial chain -->
+    <link name="${prefix}base"/>
     <link name="${prefix}base_link">
       <collision>
@@ -10,5 +8,5 @@
           <mesh filename="package://${package_name}/meshes/kr10_r1100_2/collision/base_link.stl"/>
         </geometry>
-        <origin rpy="-0.0 0.0 -0.0" xyz="0.0 0.0 0.0"/>
+        <origin rpy="0.0 -0.0 0.0" xyz="0.0 0.0 0.0"/>
       </collision>
       <inertial>
@@ -19,10 +17,10 @@
       <visual>
         <geometry>
-          <mesh filename="package://${package_name}/meshes/kr10_r1100_2/visual/base_link.stl"/>
+          <mesh filename="package://${package_name}/meshes/kr10_r1100_2/visual/base_link.dae"/>
         </geometry>
-        <origin rpy="-0.0 0.0 -0.0" xyz="0.0 0.0 0.0"/>
-        <xacro:material_kuka_ral_pure_white/>
+        <origin rpy="0.0 -0.0 0.0" xyz="0.0 0.0 0.0"/>
       </visual>
     </link>
+    <link name="${prefix}flange"/>
     <link name="${prefix}link_1">
       <collision>
@@ -30,17 +28,16 @@
           <mesh filename="package://${package_name}/meshes/kr10_r1100_2/collision/link_1.stl"/>
         </geometry>
-        <origin rpy="-0.0 0.0 -0.0" xyz="0.0 0.0 0.0"/>
+        <origin rpy="-3.141592653589793 0.0 -0.0" xyz="0.0 -2.547265342226495e-17 0.20800000000000002"/>
       </collision>
       <inertial>
-        <inertia ixx="0.07406183855390855" ixy="0.0" ixz="0.0" iyy="0.0890478351825312" iyz="0.0" izz="0.11039570662759429"/>
-        <mass value="8.4159999999999986E0"/>
-        <origin rpy="1.304519343134156 -0.9428616016893947 -1.4226510948637578" xyz="0.006410408745247152 -0.01626805370722434 -0.10658893773764262"/>
+        <inertia ixx="0.07406183855390856" ixy="0.0" ixz="0.0" iyy="0.0890478351825312" iyz="0.0" izz="0.11039570662759428"/>
+        <mass value="8.416E0"/>
+        <origin rpy="1.304519343134156 -0.9428616016893944 -1.4226510948637578" xyz="0.00641040874524715 -0.016268053707224336 -0.1065889377376426"/>
       </inertial>
       <visual>
         <geometry>
-          <mesh filename="package://${package_name}/meshes/kr10_r1100_2/visual/link_1.stl"/>
+          <mesh filename="package://${package_name}/meshes/kr10_r1100_2/visual/link_1.dae"/>
         </geometry>
-        <origin rpy="-0.0 0.0 -0.0" xyz="0.0 0.0 0.0"/>
-        <xacro:material_kuka_ral_pure_white/>
+        <origin rpy="-3.141592653589793 0.0 -0.0" xyz="0.0 -2.547265342226495e-17 0.20800000000000002"/>
       </visual>
     </link>
@@ -50,17 +47,16 @@
           <mesh filename="package://${package_name}/meshes/kr10_r1100_2/collision/link_2.stl"/>
         </geometry>
-        <origin rpy="-0.0 0.0 -0.0" xyz="0.0 0.0 0.0"/>
+        <origin rpy="1.5707963267948968 -0.0 1.5707963267948966" xyz="-0.4 -0.024999999999999977 -0.09069999999999996"/>
       </collision>
       <inertial>
-        <inertia ixx="0.8751595055066254" ixy="0.0" ixz="0.0" iyy="0.09215049446198915" iyz="0.0" izz="0.9157117764876721"/>
+        <inertia ixx="0.8751595055066256" ixy="0.0" ixz="0.0" iyy="0.09215049446198954" iyz="0.0" izz="0.9157117764876714"/>
         <mass value="1.78369E1"/>
-        <origin rpy="1.9524873827550635 -1.5422358773344043 -0.3902815673307173" xyz="0.191160133767639 -0.004651344123698628 -0.07520541854245974"/>
+        <origin rpy="1.9524873827550724 -1.5422358773344043 -0.3902815673307255" xyz="0.19116013376763902 -0.004651344123698628 -0.07520541854245974"/>
       </inertial>
       <visual>
         <geometry>
-          <mesh filename="package://${package_name}/meshes/kr10_r1100_2/visual/link_2.stl"/>
+          <mesh filename="package://${package_name}/meshes/kr10_r1100_2/visual/link_2.dae"/>
         </geometry>
-        <origin rpy="-0.0 0.0 -0.0" xyz="0.0 0.0 0.0"/>
-        <xacro:material_kuka_ral_pure_white/>
+        <origin rpy="1.5707963267948968 -0.0 1.5707963267948966" xyz="-0.4 -0.024999999999999977 -0.09069999999999996"/>
       </visual>
     </link>
@@ -70,17 +66,16 @@
           <mesh filename="package://${package_name}/meshes/kr10_r1100_2/collision/link_3.stl"/>
         </geometry>
-        <origin rpy="-0.0 0.0 -0.0" xyz="0.0 0.0 0.0"/>
+        <origin rpy="1.5707963267948968 -0.0 -0.0" xyz="-0.025000000000000036 0.96 -0.08649999999999995"/>
       </collision>
       <inertial>
-        <inertia ixx="0.04469381119929391" ixy="0.0" ixz="0.0" iyy="0.018969508933922696" iyz="0.0" izz="0.0498412586885908"/>
-        <mass value="6.075E0"/>
-        <origin rpy="-2.676930368410595 -1.321895859309871 1.1860920267202666" xyz="0.04386106995884774 -0.012506995884773664 -0.06825142386831277"/>
+        <inertia ixx="0.04469381119929391" ixy="0.0" ixz="0.0" iyy="0.018969508933922692" iyz="0.0" izz="0.049841258688590774"/>
+        <mass value="6.0749999999999993E0"/>
+        <origin rpy="-2.6769303684105967 -1.3218958593098697 1.186092026720268" xyz="0.043861069958847754 -0.012506995884773666 -0.06825142386831277"/>
       </inertial>
       <visual>
         <geometry>
-          <mesh filename="package://${package_name}/meshes/kr10_r1100_2/visual/link_3.stl"/>
+          <mesh filename="package://${package_name}/meshes/kr10_r1100_2/visual/link_3.dae"/>
         </geometry>
-        <origin rpy="-0.0 0.0 -0.0" xyz="0.0 0.0 0.0"/>
-        <xacro:material_kuka_ral_pure_white/>
+        <origin rpy="1.5707963267948968 -0.0 -0.0" xyz="-0.025000000000000036 0.96 -0.08649999999999995"/>
       </visual>
     </link>
@@ -90,17 +85,16 @@
           <mesh filename="package://${package_name}/meshes/kr10_r1100_2/collision/link_4.stl"/>
         </geometry>
-        <origin rpy="-0.0 0.0 -0.0" xyz="0.0 0.0 0.0"/>
+        <origin rpy="1.8369701987210297e-16 1.5707963267948966 0.0" xyz="-0.9850000000000001 3.0620797726250457e-17 0.22099999999999997"/>
       </collision>
       <inertial>
-        <inertia ixx="0.012301413884477554" ixy="0.0" ixz="0.0" iyy="0.08469612193319441" iyz="0.0" izz="0.08739834186747329"/>
-        <mass value="5.1623807059999995E0"/>
-        <origin rpy="-2.228094247436686 -1.5326119469267911 2.179783954730353" xyz="0.0013191433102012267 0.008607757626765767 -0.14098161935749579"/>
+        <inertia ixx="0.012301413884477554" ixy="0.0" ixz="0.0" iyy="0.0846961219331944" iyz="0.0" izz="0.08739834186747328"/>
+        <mass value="5.162380706E0"/>
+        <origin rpy="-2.228094247436686 -1.5326119469267911 2.179783954730353" xyz="0.0013191433102012265 0.008607757626765767 -0.14098161935749576"/>
       </inertial>
       <visual>
         <geometry>
-          <mesh filename="package://${package_name}/meshes/kr10_r1100_2/visual/link_4.stl"/>
+          <mesh filename="package://${package_name}/meshes/kr10_r1100_2/visual/link_4.dae"/>
         </geometry>
-        <origin rpy="-0.0 0.0 -0.0" xyz="0.0 0.0 0.0"/>
-        <xacro:material_kuka_ral_pure_white/>
+        <origin rpy="1.8369701987210297e-16 1.5707963267948966 0.0" xyz="-0.9850000000000001 3.0620797726250457e-17 0.22099999999999997"/>
       </visual>
     </link>
@@ -110,17 +104,16 @@
           <mesh filename="package://${package_name}/meshes/kr10_r1100_2/collision/link_5.stl"/>
         </geometry>
-        <origin rpy="-0.0 0.0 -0.0" xyz="0.0 0.0 0.0"/>
+        <origin rpy="1.5707963267948968 -3.749399456654644e-33 -6.123233995736766e-17" xyz="-0.5399999999999999 0.9850000000000001 -0.05049999999999999"/>
       </collision>
       <inertial>
-        <inertia ixx="0.0017317756133102904" ixy="0.0" ixz="0.0" iyy="0.002219500805440681" iyz="0.0" izz="0.002467090055442975"/>
+        <inertia ixx="0.0017317756133102906" ixy="0.0" ixz="0.0" iyy="0.0022195008054406813" iyz="0.0" izz="0.0024670900554429774"/>
         <mass value="1.6128E0"/>
-        <origin rpy="1.567898714902774 -0.8611716764868309 -3.100280255900493" xyz="0.009320696924603175 7.83482142857143E-4 -0.026462549603174602"/>
+        <origin rpy="1.5678987149027706 -0.8611716764868321 -3.100280255900495" xyz="0.009320696924603177 7.83482142857143E-4 -0.026462549603174602"/>
       </inertial>
       <visual>
         <geometry>
-          <mesh filename="package://${package_name}/meshes/kr10_r1100_2/visual/link_5.stl"/>
+          <mesh filename="package://${package_name}/meshes/kr10_r1100_2/visual/link_5.dae"/>
         </geometry>
-        <origin rpy="-0.0 0.0 -0.0" xyz="0.0 0.0 0.0"/>
-        <xacro:material_kuka_ral_pure_white/>
+        <origin rpy="1.5707963267948968 -3.749399456654644e-33 -6.123233995736766e-17" xyz="-0.5399999999999999 0.9850000000000001 -0.05049999999999999"/>
       </visual>
     </link>
@@ -130,25 +123,28 @@
           <mesh filename="package://${package_name}/meshes/kr10_r1100_2/collision/link_6.stl"/>
         </geometry>
-        <origin rpy="-0.0 0.0 -0.0" xyz="0.0 0.0 0.0"/>
+        <origin rpy="1.2246467991473532e-16 1.5707963267948966 0.0" xyz="-0.9850000000000002 -3.9114174677720623e-17 0.6014999999999999"/>
       </collision>
       <inertial>
         <inertia ixx="1.83698267603013E-4" ixy="0.0" ixz="0.0" iyy="1.8213621766783165E-4" iyz="0.0" izz="2.9589000000000004E-4"/>
         <mass value="7.34E-1"/>
-        <origin rpy="0.0 -0.0 1.223427188696551" xyz="0.0 0.0 -0.011764604904632152"/>
+        <origin rpy="0.0 -0.0 1.2234271886965395" xyz="0.0 0.0 -0.011764604904632152"/>
       </inertial>
       <visual>
         <geometry>
-          <mesh filename="package://${package_name}/meshes/kr10_r1100_2/visual/link_6.stl"/>
+          <mesh filename="package://${package_name}/meshes/kr10_r1100_2/visual/link_6.dae"/>
         </geometry>
-        <origin rpy="-0.0 0.0 -0.0" xyz="0.0 0.0 0.0"/>
-        <xacro:material_kuka_ral_pure_white/>
+        <origin rpy="1.2246467991473532e-16 1.5707963267948966 0.0" xyz="-0.9850000000000002 -3.9114174677720623e-17 0.6014999999999999"/>
       </visual>
     </link>
-    <!-- joints - main serial chain -->
+    <link name="${prefix}tool0"/>
+    <joint name="${prefix}base_link-base" type="fixed">
+      <child link="${prefix}base"/>
+      <parent link="${prefix}base_link"/>
+    </joint>
     <joint name="${prefix}joint_1" type="revolute">
       <axis xyz="0.0 0.0 1.0"/>
       <child link="${prefix}link_1"/>
-      <limit effort="288.36" lower="-2.9670597283903604E0" upper="2.9670597283903604E0" velocity="${radians(300)}"/>
-      <origin rpy="-3.141592653589793 0.0 -0.0" xyz="0.0 0.0 0.0"/>
+      <limit effort="2.8836E2" lower="-2.967059725E0" upper="2.967059725E0" velocity="5.23598775598299E0"/>
+      <origin rpy="3.141592653589793 -0.0 0.0" xyz="0.0 0.0 0.20800000000000002"/>
       <parent link="${prefix}base_link"/>
     </joint>
@@ -156,6 +152,6 @@
       <axis xyz="0.0 0.0 1.0"/>
       <child link="${prefix}link_2"/>
-      <limit effort="311.954897896674" lower="-3.3161255787892263E0" upper="7.853981633974483E-1" velocity="${radians(225)}"/>
-      <origin rpy="1.5707963267948963 0.0 -0.0" xyz="0.025 0.0 -0.4"/>
+      <limit effort="3.1199661990909851E2" lower="-3.316125575E0" upper="7.853981625E-1" velocity="3.92699081698724E0"/>
+      <origin rpy="1.5707963267948966 -0.0 0.0" xyz="0.025 -0.0907 -0.192"/>
       <parent link="${prefix}link_1"/>
     </joint>
@@ -163,6 +159,6 @@
       <axis xyz="0.0 0.0 1.0"/>
       <child link="${prefix}link_3"/>
-      <limit effort="119.76245366275" lower="-2.0943951023931953E0" upper="2.722713633111154E0" velocity="${radians(330)}"/>
-      <origin rpy="0.0 0.0 -1.5707963267948963" xyz="0.56 0.0 0.0"/>
+      <limit effort="1.1975898206876661E2" lower="-2.0943951E0" upper="2.72271363E0" velocity="5.75958653158129E0"/>
+      <origin rpy="0.0 -0.0 0.0" xyz="0.56 0.0 -0.004200000000000001"/>
       <parent link="${prefix}link_2"/>
     </joint>
@@ -170,6 +166,6 @@
       <axis xyz="0.0 0.0 1.0"/>
       <child link="${prefix}link_4"/>
-      <limit effort="46.081304845791" lower="-3.2288591161895095E0" upper="3.2288591161895095E0" velocity="${radians(360)}"/>
-      <origin rpy="1.5707963267948963 0.0 -0.0" xyz="0.025 0.0 0.0"/>
+      <limit effort="4.6080276297203334E1" lower="-3.2288591125E0" upper="3.2288591125E0" velocity="6.28318530717959E0"/>
+      <origin rpy="1.5707963267948966 -0.0 -1.5707963267948966" xyz="0.196 -0.025 -0.08650000000000001"/>
       <parent link="${prefix}link_3"/>
     </joint>
@@ -177,6 +173,6 @@
       <axis xyz="0.0 0.0 1.0"/>
       <child link="${prefix}link_5"/>
-      <limit effort="41.6154671315968" lower="-2.0943951023931953E0" upper="2.0943951023931953E0" velocity="${radians(360)}"/>
-      <origin rpy="-1.5707963267948963 0.0 -0.0" xyz="0.0 0.0 -0.515"/>
+      <limit effort="4.1613521240808865E1" lower="-2.0943951E0" upper="2.0943951E0" velocity="6.28318530717959E0"/>
+      <origin rpy="0.0 1.5707963267948966 1.5707963267948966" xyz="0.0 0.0505 -0.319"/>
       <parent link="${prefix}link_4"/>
     </joint>
@@ -184,27 +180,16 @@
       <axis xyz="0.0 0.0 1.0"/>
       <child link="${prefix}link_6"/>
-      <limit effort="28.03794" lower="-6.1086523819801535E0" upper="6.1086523819801535E0" velocity="${radians(433)}"/>
-      <origin rpy="1.5707963267948963 0.0 -0.0" xyz="0.0 0.0 0.0"/>
+      <limit effort="2.8038609999999991E1" lower="-6.108652375E0" upper="6.108652375E0" velocity="7.55727566113545E0"/>
+      <origin rpy="1.5707963267948966 -0.0 -1.5707963267948966" xyz="0.0615 0.0 -0.0505"/>
       <parent link="${prefix}link_5"/>
     </joint>
-    <!-- ROS-Industrial 'base' frame - equivalent of 'KUKA ROBROOT'-->
-    <link name="${prefix}base"/>
-    <joint name="${prefix}base_link-base" type="fixed">
-      <origin xyz="0 0 0" rpy="0 0 0"/>
-      <parent link="${prefix}base_link"/>
-      <child link="${prefix}base"/>
-    </joint>
-    <!-- ROS-Industrial 'flange' frame - attachment point for EEF models -->
-    <link name="${prefix}flange"/>
     <joint name="${prefix}link6-flange" type="fixed">
       <child link="${prefix}flange"/>
-      <origin rpy="0 ${pi/2} -0.0" xyz="0.0 0.0 -0.09"/>
+      <origin rpy="0.0 1.5707963267948966 0.0" xyz="0.0 0.0 -0.0285"/>
       <parent link="${prefix}link_6"/>
     </joint>
-    <!-- ROS-Industrial 'tool0' frame - all-zeros tool frame -->
-    <link name="${prefix}tool0"/>
     <joint name="${prefix}link6-tool0" type="fixed">
       <child link="${prefix}tool0"/>
-      <origin rpy="0 ${pi} -0.0" xyz="0.0 0.0 -0.09"/>
+      <origin rpy="3.141592653589793 1.2246467991473532E-16 3.141592653589793" xyz="0.0 0.0 -0.0285"/>
       <parent link="${prefix}link_6"/>
     </joint>
