Commit message: Expose gpio_config as a configurable xacro argument
Add a gpio_config argument to every ros2_control macro that supports
use_gpio, defaulting to the existing kuka_rsi_driver gpio_config.xacro
when left empty. This lets a launch file point use_gpio at a custom
GPIO xacro file, for example to describe external IOs, instead of
always including the driver's default config.

Wire the argument through every per-model urdf.xacro so it can be set
from the top level.

Co-Authored-By: Claude Sonnet 5 <noreply@anthropic.com>

File: kuka_agilus_support/urdf/kr10_r1100_2.urdf.xacro (robot description, xacro)
@@ -8,4 +8,5 @@
   <xacro:arg name="mode" default="hardware"/>
   <xacro:arg name="use_gpio" default="false"/>
+  <xacro:arg name="gpio_config" default=""/>
   <xacro:arg name="roundtrip_time" default="0"/>
   <xacro:arg name="client_ip" default="0.0.0.0"/>
@@ -25,5 +26,5 @@
   <xacro:arg name="yaw" default="0"/>
   <xacro:arg name="rsi_xml_config_file" default=""/>
-  <xacro:kuka_agilus_ros2_control name="$(arg prefix)kr10_r1100_2" driver_version="$(arg driver_version)" client_ip="$(arg client_ip)" client_port="$(arg client_port)" mxa_client_port="$(arg mxa_client_port)" controller_ip="$(arg controller_ip)" prefix="$(arg prefix)" mode="$(arg mode)" use_gpio="$(arg use_gpio)" roundtrip_time="$(arg roundtrip_time)" verify_robot_model="$(arg verify_robot_model)" rsi_xml_config_file="$(arg rsi_xml_config_file)" is_async="$(arg is_async)" async_thread_priority="$(arg async_thread_priority)" async_affinity="$(arg async_affinity)">
+  <xacro:kuka_agilus_ros2_control name="$(arg prefix)kr10_r1100_2" driver_version="$(arg driver_version)" client_ip="$(arg client_ip)" client_port="$(arg client_port)" mxa_client_port="$(arg mxa_client_port)" controller_ip="$(arg controller_ip)" prefix="$(arg prefix)" mode="$(arg mode)" use_gpio="$(arg use_gpio)" gpio_config="$(arg gpio_config)" roundtrip_time="$(arg roundtrip_time)" verify_robot_model="$(arg verify_robot_model)" rsi_xml_config_file="$(arg rsi_xml_config_file)" is_async="$(arg is_async)" async_thread_priority="$(arg async_thread_priority)" async_affinity="$(arg async_affinity)">
     <ext_axes_ros2_control_joints/>
   </xacro:kuka_agilus_ros2_control>

File: kuka_agilus_support/urdf/kr10_r1100_3.urdf.xacro (robot description, xacro)
@@ -20,4 +20,5 @@
   <xacro:arg name="mode" default="hardware"/>
   <xacro:arg name="use_gpio" default="false"/>
+  <xacro:arg name="gpio_config" default=""/>
   <xacro:arg name="roundtrip_time" default="0"/>
   <xacro:arg name="client_ip" default="0.0.0.0"/>
@@ -26,5 +27,5 @@
   <xacro:arg name="controller_ip" default="0.0.0.0"/>
   <xacro:arg name="verify_robot_model" default="true"/>
-  <xacro:kuka_agilus_ros2_control name="$(arg prefix)kr10_r1100_3" driver_version="$(arg driver_version)" client_ip="$(arg client_ip)" client_port="$(arg client_port)" mxa_client_port="$(arg mxa_client_port)" controller_ip="$(arg controller_ip)" prefix="$(arg prefix)" mode="$(arg mode)" use_gpio="$(arg use_gpio)" roundtrip_time="$(arg roundtrip_time)" verify_robot_model="$(arg verify_robot_model)" rsi_xml_config_file="$(arg rsi_xml_config_file)" is_async="$(arg is_async)" async_thread_priority="$(arg async_thread_priority)" async_affinity="$(arg async_affinity)">
+  <xacro:kuka_agilus_ros2_control name="$(arg prefix)kr10_r1100_3" driver_version="$(arg driver_version)" client_ip="$(arg client_ip)" client_port="$(arg client_port)" mxa_client_port="$(arg mxa_client_port)" controller_ip="$(arg controller_ip)" prefix="$(arg prefix)" mode="$(arg mode)" use_gpio="$(arg use_gpio)" gpio_config="$(arg gpio_config)" roundtrip_time="$(arg roundtrip_time)" verify_robot_model="$(arg verify_robot_model)" rsi_xml_config_file="$(arg rsi_xml_config_file)" is_async="$(arg is_async)" async_thread_priority="$(arg async_thread_priority)" async_affinity="$(arg async_affinity)">
     <ext_axes_ros2_control_joints/>
   </xacro:kuka_agilus_ros2_control>

File: kuka_agilus_support/urdf/kr10_r900_2.urdf.xacro (robot description, xacro)
@@ -8,4 +8,5 @@
   <xacro:arg name="mode" default="hardware"/>
   <xacro:arg name="use_gpio" default="false"/>
+  <xacro:arg name="gpio_config" default=""/>
   <xacro:arg name="roundtrip_time" default="0"/>
   <xacro:arg name="client_ip" default="0.0.0.0"/>
@@ -25,5 +26,5 @@
   <xacro:arg name="yaw" default="0"/>
   <xacro:arg name="rsi_xml_config_file" default=""/>
-  <xacro:kuka_agilus_ros2_control name="$(arg prefix)kr10_r900_2" driver_version="$(arg driver_version)" client_ip="$(arg client_ip)" client_port="$(arg client_port)" mxa_client_port="$(arg mxa_client_port)" controller_ip="$(arg controller_ip)" prefix="$(arg prefix)" mode="$(arg mode)" use_gpio="$(arg use_gpio)" roundtrip_time="$(arg roundtrip_time)" verify_robot_model="$(arg verify_robot_model)" rsi_xml_config_file="$(arg rsi_xml_config_file)" is_async="$(arg is_async)" async_thread_priority="$(arg async_thread_priority)" async_affinity="$(arg async_affinity)">
+  <xacro:kuka_agilus_ros2_control name="$(arg prefix)kr10_r900_2" driver_version="$(arg driver_version)" client_ip="$(arg client_ip)" client_port="$(arg client_port)" mxa_client_port="$(arg mxa_client_port)" controller_ip="$(arg controller_ip)" prefix="$(arg prefix)" mode="$(arg mode)" use_gpio="$(arg use_gpio)" gpio_config="$(arg gpio_config)" roundtrip_time="$(arg roundtrip_time)" verify_robot_model="$(arg verify_robot_model)" rsi_xml_config_file="$(arg rsi_xml_config_file)" is_async="$(arg is_async)" async_thread_priority="$(arg async_thread_priority)" async_affinity="$(arg async_affinity)">
     <ext_axes_ros2_control_joints/>
   </xacro:kuka_agilus_ros2_control>

File: kuka_agilus_support/urdf/kr13_r900_3.urdf.xacro (robot description, xacro)
@@ -20,4 +20,5 @@
   <xacro:arg name="mode" default="hardware"/>
   <xacro:arg name="use_gpio" default="false"/>
+  <xacro:arg name="gpio_config" default=""/>
   <xacro:arg name="roundtrip_time" default="0"/>
   <xacro:arg name="client_ip" default="0.0.0.0"/>
@@ -26,5 +27,5 @@
   <xacro:arg name="controller_ip" default="0.0.0.0"/>
   <xacro:arg name="verify_robot_model" default="true"/>
-  <xacro:kuka_agilus_ros2_control name="$(arg prefix)kr13_r900_3" driver_version="$(arg driver_version)" client_ip="$(arg client_ip)" client_port="$(arg client_port)" mxa_client_port="$(arg mxa_client_port)" controller_ip="$(arg controller_ip)" prefix="$(arg prefix)" mode="$(arg mode)" use_gpio="$(arg use_gpio)" roundtrip_time="$(arg roundtrip_time)" verify_robot_model="$(arg verify_robot_model)" rsi_xml_config_file="$(arg rsi_xml_config_file)" is_async="$(arg is_async)" async_thread_priority="$(arg async_thread_priority)" async_affinity="$(arg async_affinity)">
+  <xacro:kuka_agilus_ros2_control name="$(arg prefix)kr13_r900_3" driver_version="$(arg driver_version)" client_ip="$(arg client_ip)" client_port="$(arg client_port)" mxa_client_port="$(arg mxa_client_port)" controller_ip="$(arg controller_ip)" prefix="$(arg prefix)" mode="$(arg mode)" use_gpio="$(arg use_gpio)" gpio_config="$(arg gpio_config)" roundtrip_time="$(arg roundtrip_time)" verify_robot_model="$(arg verify_robot_model)" rsi_xml_config_file="$(arg rsi_xml_config_file)" is_async="$(arg is_async)" async_thread_priority="$(arg async_thread_priority)" async_affinity="$(arg async_affinity)">
     <ext_axes_ros2_control_joints/>
   </xacro:kuka_agilus_ros2_control>

File: kuka_agilus_support/urdf/kr16_r1100_3.urdf.xacro (robot description, xacro)
@@ -20,4 +20,5 @@
   <xacro:arg name="mode" default="hardware"/>
   <xacro:arg name="use_gpio" default="false"/>
+  <xacro:arg name="gpio_config" default=""/>
   <xacro:arg name="roundtrip_time" default="0"/>
   <xacro:arg name="client_ip" default="0.0.0.0"/>
@@ -26,5 +27,5 @@
   <xacro:arg name="controller_ip" default="0.0.0.0"/>
   <xacro:arg name="verify_robot_model" default="true"/>
-  <xacro:kuka_agilus_ros2_control name="$(arg prefix)kr16_r1100_3" driver_version="$(arg driver_version)" client_ip="$(arg client_ip)" client_port="$(arg client_port)" mxa_client_port="$(arg mxa_client_port)" controller_ip="$(arg controller_ip)" prefix="$(arg prefix)" mode="$(arg mode)" use_gpio="$(arg use_gpio)" roundtrip_time="$(arg roundtrip_time)" verify_robot_model="$(arg verify_robot_model)" rsi_xml_config_file="$(arg rsi_xml_config_file)" is_async="$(arg is_async)" async_thread_priority="$(arg async_thread_priority)" async_affinity="$(arg async_affinity)">
+  <xacro:kuka_agilus_ros2_control name="$(arg prefix)kr16_r1100_3" driver_version="$(arg driver_version)" client_ip="$(arg client_ip)" client_port="$(arg client_port)" mxa_client_port="$(arg mxa_client_port)" controller_ip="$(arg controller_ip)" prefix="$(arg prefix)" mode="$(arg mode)" use_gpio="$(arg use_gpio)" gpio_config="$(arg gpio_config)" roundtrip_time="$(arg roundtrip_time)" verify_robot_model="$(arg verify_robot_model)" rsi_xml_config_file="$(arg rsi_xml_config_file)" is_async="$(arg is_async)" async_thread_priority="$(arg async_thread_priority)" async_affinity="$(arg async_affinity)">
     <ext_axes_ros2_control_joints/>
   </xacro:kuka_agilus_ros2_control>

File: kuka_agilus_support/urdf/kr4_r600.urdf.xacro (robot description, xacro)
@@ -8,4 +8,5 @@
   <xacro:arg name="mode" default="hardware"/>
   <xacro:arg name="use_gpio" default="false"/>
+  <xacro:arg name="gpio_config" default=""/>
   <xacro:arg name="roundtrip_time" default="0"/>
   <xacro:arg name="client_ip" default="0.0.0.0"/>
@@ -25,5 +26,5 @@
   <xacro:arg name="yaw" default="0"/>
   <xacro:arg name="rsi_xml_config_file" default=""/>
-  <xacro:kuka_agilus_ros2_control name="$(arg prefix)kr4_r600" driver_version="$(arg driver_version)" client_ip="$(arg client_ip)" client_port="$(arg client_port)" mxa_client_port="$(arg mxa_client_port)" controller_ip="$(arg controller_ip)" prefix="$(arg prefix)" mode="$(arg mode)" use_gpio="$(arg use_gpio)" roundtrip_time="$(arg roundtrip_time)" verify_robot_model="$(arg verify_robot_model)" rsi_xml_config_file="$(arg rsi_xml_config_file)" is_async="$(arg is_async)" async_thread_priority="$(arg async_thread_priority)" async_affinity="$(arg async_affinity)">
+  <xacro:kuka_agilus_ros2_control name="$(arg prefix)kr4_r600" driver_version="$(arg driver_version)" client_ip="$(arg client_ip)" client_port="$(arg client_port)" mxa_client_port="$(arg mxa_client_port)" controller_ip="$(arg controller_ip)" prefix="$(arg prefix)" mode="$(arg mode)" use_gpio="$(arg use_gpio)" gpio_config="$(arg gpio_config)" roundtrip_time="$(arg roundtrip_time)" verify_robot_model="$(arg verify_robot_model)" rsi_xml_config_file="$(arg rsi_xml_config_file)" is_async="$(arg is_async)" async_thread_priority="$(arg async_thread_priority)" async_affinity="$(arg async_affinity)">
     <ext_axes_ros2_control_joints/>
   </xacro:kuka_agilus_ros2_control>

File: kuka_agilus_support/urdf/kr6_r700_2.urdf.xacro (robot description, xacro)
@@ -8,4 +8,5 @@
   <xacro:arg name="mode" default="hardware"/>
   <xacro:arg name="use_gpio" default="false"/>
+  <xacro:arg name="gpio_config" default=""/>
   <xacro:arg name="roundtrip_time" default="0"/>
   <xacro:arg name="client_ip" default="0.0.0.0"/>
@@ -25,5 +26,5 @@
   <xacro:arg name="yaw" default="0"/>
   <xacro:arg name="rsi_xml_config_file" default=""/>
-  <xacro:kuka_agilus_ros2_control name="$(arg prefix)kr6_r700_2" driver_version="$(arg driver_version)" client_ip="$(arg client_ip)" client_port="$(arg client_port)" mxa_client_port="$(arg mxa_client_port)" controller_ip="$(arg controller_ip)" prefix="$(arg prefix)" mode="$(arg mode)" use_gpio="$(arg use_gpio)" roundtrip_time="$(arg roundtrip_time)" verify_robot_model="$(arg verify_robot_model)" rsi_xml_config_file="$(arg rsi_xml_config_file)" is_async="$(arg is_async)" async_thread_priority="$(arg async_thread_priority)" async_affinity="$(arg async_affinity)">
+  <xacro:kuka_agilus_ros2_control name="$(arg prefix)kr6_r700_2" driver_version="$(arg driver_version)" client_ip="$(arg client_ip)" client_port="$(arg client_port)" mxa_client_port="$(arg mxa_client_port)" controller_ip="$(arg controller_ip)" prefix="$(arg prefix)" mode="$(arg mode)" use_gpio="$(arg use_gpio)" gpio_config="$(arg gpio_config)" roundtrip_time="$(arg roundtrip_time)" verify_robot_model="$(arg verify_robot_model)" rsi_xml_config_file="$(arg rsi_xml_config_file)" is_async="$(arg is_async)" async_thread_priority="$(arg async_thread_priority)" async_affinity="$(arg async_affinity)">
     <ext_axes_ros2_control_joints/>
   </xacro:kuka_agilus_ros2_control>

File: kuka_agilus_support/urdf/kr6_r700_sixx.urdf.xacro (robot description, xacro)
@@ -8,4 +8,5 @@
   <xacro:arg name="mode" default="hardware"/>
   <xacro:arg name="use_gpio" default="false"/>
+  <xacro:arg name="gpio_config" default=""/>
   <xacro:arg name="roundtrip_time" default="0"/>
   <xacro:arg name="client_ip" default="0.0.0.0"/>
@@ -25,5 +26,5 @@
   <xacro:arg name="yaw" default="0"/>
   <xacro:arg name="rsi_xml_config_file" default=""/>
-  <xacro:kuka_agilus_ros2_control name="$(arg prefix)kr6_r700_sixx" driver_version="$(arg driver_version)" client_ip="$(arg client_ip)" client_port="$(arg client_port)" mxa_client_port="$(arg mxa_client_port)" controller_ip="$(arg controller_ip)" prefix="$(arg prefix)" mode="$(arg mode)" use_gpio="$(arg use_gpio)" roundtrip_time="$(arg roundtrip_time)" verify_robot_model="$(arg verify_robot_model)" rsi_xml_config_file="$(arg rsi_xml_config_file)" is_async="$(arg is_async)" async_thread_priority="$(arg async_thread_priority)" async_affinity="$(arg async_affinity)">
+  <xacro:kuka_agilus_ros2_control name="$(arg prefix)kr6_r700_sixx" driver_version="$(arg driver_version)" client_ip="$(arg client_ip)" client_port="$(arg client_port)" mxa_client_port="$(arg mxa_client_port)" controller_ip="$(arg controller_ip)" prefix="$(arg prefix)" mode="$(arg mode)" use_gpio="$(arg use_gpio)" gpio_config="$(arg gpio_config)" roundtrip_time="$(arg roundtrip_time)" verify_robot_model="$(arg verify_robot_model)" rsi_xml_config_file="$(arg rsi_xml_config_file)" is_async="$(arg is_async)" async_thread_priority="$(arg async_thread_priority)" async_affinity="$(arg async_affinity)">
     <ext_axes_ros2_control_joints/>
   </xacro:kuka_agilus_ros2_control>

File: kuka_agilus_support/urdf/kr6_r900_2.urdf.xacro (robot description, xacro)
@@ -8,4 +8,5 @@
   <xacro:arg name="mode" default="hardware"/>
   <xacro:arg name="use_gpio" default="false"/>
+  <xacro:arg name="gpio_config" default=""/>
   <xacro:arg name="roundtrip_time" default="0"/>
   <xacro:arg name="client_ip" default="0.0.0.0"/>
@@ -25,5 +26,5 @@
   <xacro:arg name="yaw" default="0"/>
   <xacro:arg name="rsi_xml_config_file" default=""/>
-  <xacro:kuka_agilus_ros2_control name="$(arg prefix)kr6_r900_2" driver_version="$(arg driver_version)" client_ip="$(arg client_ip)" client_port="$(arg client_port)" mxa_client_port="$(arg mxa_client_port)" controller_ip="$(arg controller_ip)" prefix="$(arg prefix)" mode="$(arg mode)" use_gpio="$(arg use_gpio)" roundtrip_time="$(arg roundtrip_time)" verify_robot_model="$(arg verify_robot_model)" rsi_xml_config_file="$(arg rsi_xml_config_file)" is_async="$(arg is_async)" async_thread_priority="$(arg async_thread_priority)" async_affinity="$(arg async_affinity)">
+  <xacro:kuka_agilus_ros2_control name="$(arg prefix)kr6_r900_2" driver_version="$(arg driver_version)" client_ip="$(arg client_ip)" client_port="$(arg client_port)" mxa_client_port="$(arg mxa_client_port)" controller_ip="$(arg controller_ip)" prefix="$(arg prefix)" mode="$(arg mode)" use_gpio="$(arg use_gpio)" gpio_config="$(arg gpio_config)" roundtrip_time="$(arg roundtrip_time)" verify_robot_model="$(arg verify_robot_model)" rsi_xml_config_file="$(arg rsi_xml_config_file)" is_async="$(arg is_async)" async_thread_priority="$(arg async_thread_priority)" async_affinity="$(arg async_affinity)">
     <ext_axes_ros2_control_joints/>
   </xacro:kuka_agilus_ros2_control>

File: kuka_agilus_support/urdf/kr6_r900_sixx.urdf.xacro (robot description, xacro)
@@ -8,4 +8,5 @@
   <xacro:arg name="mode" default="hardware"/>
   <xacro:arg name="use_gpio" default="false"/>
+  <xacro:arg name="gpio_config" default=""/>
   <xacro:arg name="roundtrip_time" default="0"/>
   <xacro:arg name="client_ip" default="0.0.0.0"/>
@@ -25,5 +26,5 @@
   <xacro:arg name="yaw" default="0"/>
   <xacro:arg name="rsi_xml_config_file" default=""/>
-  <xacro:kuka_agilus_ros2_control name="$(arg prefix)kr6_r900_sixx" driver_version="$(arg driver_version)" client_ip="$(arg client_ip)" client_port="$(arg client_port)" mxa_client_port="$(arg mxa_client_port)" controller_ip="$(arg controller_ip)" prefix="$(arg prefix)" mode="$(arg mode)" use_gpio="$(arg use_gpio)" roundtrip_time="$(arg roundtrip_time)" verify_robot_model="$(arg verify_robot_model)" rsi_xml_config_file="$(arg rsi_xml_config_file)" is_async="$(arg is_async)" async_thread_priority="$(arg async_thread_priority)" async_affinity="$(arg async_affinity)">
+  <xacro:kuka_agilus_ros2_control name="$(arg prefix)kr6_r900_sixx" driver_version="$(arg driver_version)" client_ip="$(arg client_ip)" client_port="$(arg client_port)" mxa_client_port="$(arg mxa_client_port)" controller_ip="$(arg controller_ip)" prefix="$(arg prefix)" mode="$(arg mode)" use_gpio="$(arg use_gpio)" gpio_config="$(arg gpio_config)" roundtrip_time="$(arg roundtrip_time)" verify_robot_model="$(arg verify_robot_model)" rsi_xml_config_file="$(arg rsi_xml_config_file)" is_async="$(arg is_async)" async_thread_priority="$(arg async_thread_priority)" async_affinity="$(arg async_affinity)">
     <ext_axes_ros2_control_joints/>
   </xacro:kuka_agilus_ros2_control>

File: kuka_agilus_support/urdf/kr7_r900_3.urdf.xacro (robot description, xacro)
@@ -20,4 +20,5 @@
   <xacro:arg name="mode" default="hardware"/>
   <xacro:arg name="use_gpio" default="false"/>
+  <xacro:arg name="gpio_config" default=""/>
   <xacro:arg name="roundtrip_time" default="0"/>
   <xacro:arg name="client_ip" default="0.0.0.0"/>
@@ -26,5 +27,5 @@
   <xacro:arg name="controller_ip" default="0.0.0.0"/>
   <xacro:arg name="verify_robot_model" default="true"/>
-  <xacro:kuka_agilus_ros2_control name="$(arg prefix)kr7_r900_3" driver_version="$(arg driver_version)" client_ip="$(arg client_ip)" client_port="$(arg client_port)" mxa_client_port="$(arg mxa_client_port)" controller_ip="$(arg controller_ip)" prefix="$(arg prefix)" mode="$(arg mode)" use_gpio="$(arg use_gpio)" roundtrip_time="$(arg roundtrip_time)" verify_robot_model="$(arg verify_robot_model)" rsi_xml_config_file="$(arg rsi_xml_config_file)" is_async="$(arg is_async)" async_thread_priority="$(arg async_thread_priority)" async_affinity="$(arg async_affinity)">
+  <xacro:kuka_agilus_ros2_control name="$(arg prefix)kr7_r900_3" driver_version="$(arg driver_version)" client_ip="$(arg client_ip)" client_port="$(arg client_port)" mxa_client_port="$(arg mxa_client_port)" controller_ip="$(arg controller_ip)" prefix="$(arg prefix)" mode="$(arg mode)" use_gpio="$(arg use_gpio)" gpio_config="$(arg gpio_config)" roundtrip_time="$(arg roundtrip_time)" verify_robot_model="$(arg verify_robot_model)" rsi_xml_config_file="$(arg rsi_xml_config_file)" is_async="$(arg is_async)" async_thread_priority="$(arg async_thread_priority)" async_affinity="$(arg async_affinity)">
     <ext_axes_ros2_control_joints/>
   </xacro:kuka_agilus_ros2_control>

File: kuka_agilus_support/urdf/kr_agilus_ros2_control_macro.xacro (robot description, xacro)
@@ -1,5 +1,8 @@
 <?xml version="1.0" encoding="UTF-8"?>
 <robot xmlns:xacro="http://www.ros.org/wiki/xacro">
-  <xacro:macro name="kuka_agilus_ros2_control" params="name driver_version client_ip client_port mxa_client_port controller_ip prefix mode use_gpio roundtrip_time verify_robot_model rsi_xml_config_file is_async async_thread_priority async_affinity gazebo_controller_config_path:=config/fake_hardware_config_6_axis.yaml **ext_axes_ros2_control_joints">
+  <xacro:macro name="kuka_agilus_ros2_control" params="name driver_version client_ip client_port mxa_client_port controller_ip prefix mode use_gpio roundtrip_time verify_robot_model rsi_xml_config_file is_async async_thread_priority async_affinity gazebo_controller_config_path:=config/fake_hardware_config_6_axis.yaml gpio_config:='' **ext_axes_ros2_control_joints">
+    <xacro:if value="${gpio_config == ''}">
+      <xacro:property name="gpio_config" value="$(find kuka_rsi_driver)/config/gpio_config.xacro"/>
+    </xacro:if>
     <!-- gazebo -->
     <xacro:if value="${mode == 'gazebo'}">
@@ -149,5 +152,5 @@
       </joint>
       <xacro:if value="${use_gpio}">
-        <xacro:include filename="$(find kuka_rsi_driver)/config/gpio_config.xacro"/>
+        <xacro:include filename="${gpio_config}"/>
         <xacro:gpio_config/>
       </xacro:if>

File: kuka_cybertech_support/urdf/kr12_r1450_3_hw.urdf.xacro (robot description, xacro)
@@ -8,4 +8,5 @@
   <xacro:arg name="mode" default="hardware"/>
   <xacro:arg name="use_gpio" default="false"/>
+  <xacro:arg name="gpio_config" default=""/>
   <xacro:arg name="roundtrip_time" default="0"/>
   <xacro:arg name="client_ip" default="0.0.0.0"/>
@@ -25,5 +26,5 @@
   <xacro:arg name="yaw" default="0"/>
   <xacro:arg name="rsi_xml_config_file" default=""/>
-  <xacro:kuka_cybertech_ros2_control name="$(arg prefix)kr12_r1450_3_hw" driver_version="$(arg driver_version)" client_ip="$(arg client_ip)" client_port="$(arg client_port)" mxa_client_port="$(arg mxa_client_port)" controller_ip="$(arg controller_ip)" prefix="$(arg prefix)" mode="$(arg mode)" use_gpio="$(arg use_gpio)" roundtrip_time="$(arg roundtrip_time)" verify_robot_model="$(arg verify_robot_model)" rsi_xml_config_file="$(arg rsi_xml_config_file)" is_async="$(arg is_async)" async_thread_priority="$(arg async_thread_priority)" async_affinity="$(arg async_affinity)">
+  <xacro:kuka_cybertech_ros2_control name="$(arg prefix)kr12_r1450_3_hw" driver_version="$(arg driver_version)" client_ip="$(arg client_ip)" client_port="$(arg client_port)" mxa_client_port="$(arg mxa_client_port)" controller_ip="$(arg controller_ip)" prefix="$(arg prefix)" mode="$(arg mode)" use_gpio="$(arg use_gpio)" gpio_config="$(arg gpio_config)" roundtrip_time="$(arg roundtrip_time)" verify_robot_model="$(arg verify_robot_model)" rsi_xml_config_file="$(arg rsi_xml_config_file)" is_async="$(arg is_async)" async_thread_priority="$(arg async_thread_priority)" async_affinity="$(arg async_affinity)">
     <ext_axes_ros2_control_joints/>
   </xacro:kuka_cybertech_ros2_control>
