Commit message: Drop use_gpio in favour of gpio_config alone
Remove the use_gpio argument from every ros2_control macro and
per-model urdf.xacro. Whether GPIO is enabled is now derived from
gpio_config: empty means no GPIO, a path means include and instantiate
that GPIO xacro file. This also drops the unconditional
$(find kuka_rsi_driver) fallback resolution for the disabled case.

Co-Authored-By: Claude Sonnet 5 <noreply@anthropic.com>

File: kuka_agilus_support/urdf/kr10_r1100_2.urdf.xacro (robot description, xacro)
@@ -7,5 +7,4 @@
   <xacro:arg name="driver_version" default="rsi_only"/>
   <xacro:arg name="mode" default="hardware"/>
-  <xacro:arg name="use_gpio" default="false"/>
   <xacro:arg name="gpio_config" default=""/>
   <xacro:arg name="roundtrip_time" default="0"/>
@@ -26,5 +25,5 @@
   <xacro:arg name="yaw" default="0"/>
   <xacro:arg name="rsi_xml_config_file" default=""/>
-  <xacro:kuka_agilus_ros2_control name="$(arg prefix)kr10_r1100_2" driver_version="$(arg driver_version)" client_ip="$(arg client_ip)" client_port="$(arg client_port)" mxa_client_port="$(arg mxa_client_port)" controller_ip="$(arg controller_ip)" prefix="$(arg prefix)" mode="$(arg mode)" use_gpio="$(arg use_gpio)" gpio_config="$(arg gpio_config)" roundtrip_time="$(arg roundtrip_time)" verify_robot_model="$(arg verify_robot_model)" rsi_xml_config_file="$(arg rsi_xml_config_file)" is_async="$(arg is_async)" async_thread_priority="$(arg async_thread_priority)" async_affinity="$(arg async_affinity)">
+  <xacro:kuka_agilus_ros2_control name="$(arg prefix)kr10_r1100_2" driver_version="$(arg driver_version)" client_ip="$(arg client_ip)" client_port="$(arg client_port)" mxa_client_port="$(arg mxa_client_port)" controller_ip="$(arg controller_ip)" prefix="$(arg prefix)" mode="$(arg mode)" gpio_config="$(arg gpio_config)" roundtrip_time="$(arg roundtrip_time)" verify_robot_model="$(arg verify_robot_model)" rsi_xml_config_file="$(arg rsi_xml_config_file)" is_async="$(arg is_async)" async_thread_priority="$(arg async_thread_priority)" async_affinity="$(arg async_affinity)">
     <ext_axes_ros2_control_joints/>
   </xacro:kuka_agilus_ros2_control>

File: kuka_agilus_support/urdf/kr10_r1100_3.urdf.xacro (robot description, xacro)
@@ -19,5 +19,4 @@
   <xacro:arg name="driver_version" default="rsi_only"/>
   <xacro:arg name="mode" default="hardware"/>
-  <xacro:arg name="use_gpio" default="false"/>
   <xacro:arg name="gpio_config" default=""/>
   <xacro:arg name="roundtrip_time" default="0"/>
@@ -27,5 +26,5 @@
   <xacro:arg name="controller_ip" default="0.0.0.0"/>
   <xacro:arg name="verify_robot_model" default="true"/>
-  <xacro:kuka_agilus_ros2_control name="$(arg prefix)kr10_r1100_3" driver_version="$(arg driver_version)" client_ip="$(arg client_ip)" client_port="$(arg client_port)" mxa_client_port="$(arg mxa_client_port)" controller_ip="$(arg controller_ip)" prefix="$(arg prefix)" mode="$(arg mode)" use_gpio="$(arg use_gpio)" gpio_config="$(arg gpio_config)" roundtrip_time="$(arg roundtrip_time)" verify_robot_model="$(arg verify_robot_model)" rsi_xml_config_file="$(arg rsi_xml_config_file)" is_async="$(arg is_async)" async_thread_priority="$(arg async_thread_priority)" async_affinity="$(arg async_affinity)">
+  <xacro:kuka_agilus_ros2_control name="$(arg prefix)kr10_r1100_3" driver_version="$(arg driver_version)" client_ip="$(arg client_ip)" client_port="$(arg client_port)" mxa_client_port="$(arg mxa_client_port)" controller_ip="$(arg controller_ip)" prefix="$(arg prefix)" mode="$(arg mode)" gpio_config="$(arg gpio_config)" roundtrip_time="$(arg roundtrip_time)" verify_robot_model="$(arg verify_robot_model)" rsi_xml_config_file="$(arg rsi_xml_config_file)" is_async="$(arg is_async)" async_thread_priority="$(arg async_thread_priority)" async_affinity="$(arg async_affinity)">
     <ext_axes_ros2_control_joints/>
   </xacro:kuka_agilus_ros2_control>

File: kuka_agilus_support/urdf/kr10_r900_2.urdf.xacro (robot description, xacro)
@@ -7,5 +7,4 @@
   <xacro:arg name="driver_version" default="rsi_only"/>
   <xacro:arg name="mode" default="hardware"/>
-  <xacro:arg name="use_gpio" default="false"/>
   <xacro:arg name="gpio_config" default=""/>
   <xacro:arg name="roundtrip_time" default="0"/>
@@ -26,5 +25,5 @@
   <xacro:arg name="yaw" default="0"/>
   <xacro:arg name="rsi_xml_config_file" default=""/>
-  <xacro:kuka_agilus_ros2_control name="$(arg prefix)kr10_r900_2" driver_version="$(arg driver_version)" client_ip="$(arg client_ip)" client_port="$(arg client_port)" mxa_client_port="$(arg mxa_client_port)" controller_ip="$(arg controller_ip)" prefix="$(arg prefix)" mode="$(arg mode)" use_gpio="$(arg use_gpio)" gpio_config="$(arg gpio_config)" roundtrip_time="$(arg roundtrip_time)" verify_robot_model="$(arg verify_robot_model)" rsi_xml_config_file="$(arg rsi_xml_config_file)" is_async="$(arg is_async)" async_thread_priority="$(arg async_thread_priority)" async_affinity="$(arg async_affinity)">
+  <xacro:kuka_agilus_ros2_control name="$(arg prefix)kr10_r900_2" driver_version="$(arg driver_version)" client_ip="$(arg client_ip)" client_port="$(arg client_port)" mxa_client_port="$(arg mxa_client_port)" controller_ip="$(arg controller_ip)" prefix="$(arg prefix)" mode="$(arg mode)" gpio_config="$(arg gpio_config)" roundtrip_time="$(arg roundtrip_time)" verify_robot_model="$(arg verify_robot_model)" rsi_xml_config_file="$(arg rsi_xml_config_file)" is_async="$(arg is_async)" async_thread_priority="$(arg async_thread_priority)" async_affinity="$(arg async_affinity)">
     <ext_axes_ros2_control_joints/>
   </xacro:kuka_agilus_ros2_control>

File: kuka_agilus_support/urdf/kr13_r900_3.urdf.xacro (robot description, xacro)
@@ -19,5 +19,4 @@
   <xacro:arg name="driver_version" default="rsi_only"/>
   <xacro:arg name="mode" default="hardware"/>
-  <xacro:arg name="use_gpio" default="false"/>
   <xacro:arg name="gpio_config" default=""/>
   <xacro:arg name="roundtrip_time" default="0"/>
@@ -27,5 +26,5 @@
   <xacro:arg name="controller_ip" default="0.0.0.0"/>
   <xacro:arg name="verify_robot_model" default="true"/>
-  <xacro:kuka_agilus_ros2_control name="$(arg prefix)kr13_r900_3" driver_version="$(arg driver_version)" client_ip="$(arg client_ip)" client_port="$(arg client_port)" mxa_client_port="$(arg mxa_client_port)" controller_ip="$(arg controller_ip)" prefix="$(arg prefix)" mode="$(arg mode)" use_gpio="$(arg use_gpio)" gpio_config="$(arg gpio_config)" roundtrip_time="$(arg roundtrip_time)" verify_robot_model="$(arg verify_robot_model)" rsi_xml_config_file="$(arg rsi_xml_config_file)" is_async="$(arg is_async)" async_thread_priority="$(arg async_thread_priority)" async_affinity="$(arg async_affinity)">
+  <xacro:kuka_agilus_ros2_control name="$(arg prefix)kr13_r900_3" driver_version="$(arg driver_version)" client_ip="$(arg client_ip)" client_port="$(arg client_port)" mxa_client_port="$(arg mxa_client_port)" controller_ip="$(arg controller_ip)" prefix="$(arg prefix)" mode="$(arg mode)" gpio_config="$(arg gpio_config)" roundtrip_time="$(arg roundtrip_time)" verify_robot_model="$(arg verify_robot_model)" rsi_xml_config_file="$(arg rsi_xml_config_file)" is_async="$(arg is_async)" async_thread_priority="$(arg async_thread_priority)" async_affinity="$(arg async_affinity)">
     <ext_axes_ros2_control_joints/>
   </xacro:kuka_agilus_ros2_control>

File: kuka_agilus_support/urdf/kr16_r1100_3.urdf.xacro (robot description, xacro)
@@ -19,5 +19,4 @@
   <xacro:arg name="driver_version" default="rsi_only"/>
   <xacro:arg name="mode" default="hardware"/>
-  <xacro:arg name="use_gpio" default="false"/>
   <xacro:arg name="gpio_config" default=""/>
   <xacro:arg name="roundtrip_time" default="0"/>
@@ -27,5 +26,5 @@
   <xacro:arg name="controller_ip" default="0.0.0.0"/>
   <xacro:arg name="verify_robot_model" default="true"/>
-  <xacro:kuka_agilus_ros2_control name="$(arg prefix)kr16_r1100_3" driver_version="$(arg driver_version)" client_ip="$(arg client_ip)" client_port="$(arg client_port)" mxa_client_port="$(arg mxa_client_port)" controller_ip="$(arg controller_ip)" prefix="$(arg prefix)" mode="$(arg mode)" use_gpio="$(arg use_gpio)" gpio_config="$(arg gpio_config)" roundtrip_time="$(arg roundtrip_time)" verify_robot_model="$(arg verify_robot_model)" rsi_xml_config_file="$(arg rsi_xml_config_file)" is_async="$(arg is_async)" async_thread_priority="$(arg async_thread_priority)" async_affinity="$(arg async_affinity)">
+  <xacro:kuka_agilus_ros2_control name="$(arg prefix)kr16_r1100_3" driver_version="$(arg driver_version)" client_ip="$(arg client_ip)" client_port="$(arg client_port)" mxa_client_port="$(arg mxa_client_port)" controller_ip="$(arg controller_ip)" prefix="$(arg prefix)" mode="$(arg mode)" gpio_config="$(arg gpio_config)" roundtrip_time="$(arg roundtrip_time)" verify_robot_model="$(arg verify_robot_model)" rsi_xml_config_file="$(arg rsi_xml_config_file)" is_async="$(arg is_async)" async_thread_priority="$(arg async_thread_priority)" async_affinity="$(arg async_affinity)">
     <ext_axes_ros2_control_joints/>
   </xacro:kuka_agilus_ros2_control>

File: kuka_agilus_support/urdf/kr4_r600.urdf.xacro (robot description, xacro)
@@ -7,5 +7,4 @@
   <xacro:arg name="driver_version" default="rsi_only"/>
   <xacro:arg name="mode" default="hardware"/>
-  <xacro:arg name="use_gpio" default="false"/>
   <xacro:arg name="gpio_config" default=""/>
   <xacro:arg name="roundtrip_time" default="0"/>
@@ -26,5 +25,5 @@
   <xacro:arg name="yaw" default="0"/>
   <xacro:arg name="rsi_xml_config_file" default=""/>
-  <xacro:kuka_agilus_ros2_control name="$(arg prefix)kr4_r600" driver_version="$(arg driver_version)" client_ip="$(arg client_ip)" client_port="$(arg client_port)" mxa_client_port="$(arg mxa_client_port)" controller_ip="$(arg controller_ip)" prefix="$(arg prefix)" mode="$(arg mode)" use_gpio="$(arg use_gpio)" gpio_config="$(arg gpio_config)" roundtrip_time="$(arg roundtrip_time)" verify_robot_model="$(arg verify_robot_model)" rsi_xml_config_file="$(arg rsi_xml_config_file)" is_async="$(arg is_async)" async_thread_priority="$(arg async_thread_priority)" async_affinity="$(arg async_affinity)">
+  <xacro:kuka_agilus_ros2_control name="$(arg prefix)kr4_r600" driver_version="$(arg driver_version)" client_ip="$(arg client_ip)" client_port="$(arg client_port)" mxa_client_port="$(arg mxa_client_port)" controller_ip="$(arg controller_ip)" prefix="$(arg prefix)" mode="$(arg mode)" gpio_config="$(arg gpio_config)" roundtrip_time="$(arg roundtrip_time)" verify_robot_model="$(arg verify_robot_model)" rsi_xml_config_file="$(arg rsi_xml_config_file)" is_async="$(arg is_async)" async_thread_priority="$(arg async_thread_priority)" async_affinity="$(arg async_affinity)">
     <ext_axes_ros2_control_joints/>
   </xacro:kuka_agilus_ros2_control>

File: kuka_agilus_support/urdf/kr6_r700_2.urdf.xacro (robot description, xacro)
@@ -7,5 +7,4 @@
   <xacro:arg name="driver_version" default="rsi_only"/>
   <xacro:arg name="mode" default="hardware"/>
-  <xacro:arg name="use_gpio" default="false"/>
   <xacro:arg name="gpio_config" default=""/>
   <xacro:arg name="roundtrip_time" default="0"/>
@@ -26,5 +25,5 @@
   <xacro:arg name="yaw" default="0"/>
   <xacro:arg name="rsi_xml_config_file" default=""/>
-  <xacro:kuka_agilus_ros2_control name="$(arg prefix)kr6_r700_2" driver_version="$(arg driver_version)" client_ip="$(arg client_ip)" client_port="$(arg client_port)" mxa_client_port="$(arg mxa_client_port)" controller_ip="$(arg controller_ip)" prefix="$(arg prefix)" mode="$(arg mode)" use_gpio="$(arg use_gpio)" gpio_config="$(arg gpio_config)" roundtrip_time="$(arg roundtrip_time)" verify_robot_model="$(arg verify_robot_model)" rsi_xml_config_file="$(arg rsi_xml_config_file)" is_async="$(arg is_async)" async_thread_priority="$(arg async_thread_priority)" async_affinity="$(arg async_affinity)">
+  <xacro:kuka_agilus_ros2_control name="$(arg prefix)kr6_r700_2" driver_version="$(arg driver_version)" client_ip="$(arg client_ip)" client_port="$(arg client_port)" mxa_client_port="$(arg mxa_client_port)" controller_ip="$(arg controller_ip)" prefix="$(arg prefix)" mode="$(arg mode)" gpio_config="$(arg gpio_config)" roundtrip_time="$(arg roundtrip_time)" verify_robot_model="$(arg verify_robot_model)" rsi_xml_config_file="$(arg rsi_xml_config_file)" is_async="$(arg is_async)" async_thread_priority="$(arg async_thread_priority)" async_affinity="$(arg async_affinity)">
     <ext_axes_ros2_control_joints/>
   </xacro:kuka_agilus_ros2_control>

File: kuka_agilus_support/urdf/kr6_r700_sixx.urdf.xacro (robot description, xacro)
@@ -7,5 +7,4 @@
   <xacro:arg name="driver_version" default="rsi_only"/>
   <xacro:arg name="mode" default="hardware"/>
-  <xacro:arg name="use_gpio" default="false"/>
   <xacro:arg name="gpio_config" default=""/>
   <xacro:arg name="roundtrip_time" default="0"/>
@@ -26,5 +25,5 @@
   <xacro:arg name="yaw" default="0"/>
   <xacro:arg name="rsi_xml_config_file" default=""/>
-  <xacro:kuka_agilus_ros2_control name="$(arg prefix)kr6_r700_sixx" driver_version="$(arg driver_version)" client_ip="$(arg client_ip)" client_port="$(arg client_port)" mxa_client_port="$(arg mxa_client_port)" controller_ip="$(arg controller_ip)" prefix="$(arg prefix)" mode="$(arg mode)" use_gpio="$(arg use_gpio)" gpio_config="$(arg gpio_config)" roundtrip_time="$(arg roundtrip_time)" verify_robot_model="$(arg verify_robot_model)" rsi_xml_config_file="$(arg rsi_xml_config_file)" is_async="$(arg is_async)" async_thread_priority="$(arg async_thread_priority)" async_affinity="$(arg async_affinity)">
+  <xacro:kuka_agilus_ros2_control name="$(arg prefix)kr6_r700_sixx" driver_version="$(arg driver_version)" client_ip="$(arg client_ip)" client_port="$(arg client_port)" mxa_client_port="$(arg mxa_client_port)" controller_ip="$(arg controller_ip)" prefix="$(arg prefix)" mode="$(arg mode)" gpio_config="$(arg gpio_config)" roundtrip_time="$(arg roundtrip_time)" verify_robot_model="$(arg verify_robot_model)" rsi_xml_config_file="$(arg rsi_xml_config_file)" is_async="$(arg is_async)" async_thread_priority="$(arg async_thread_priority)" async_affinity="$(arg async_affinity)">
     <ext_axes_ros2_control_joints/>
   </xacro:kuka_agilus_ros2_control>

File: kuka_agilus_support/urdf/kr6_r900_2.urdf.xacro (robot description, xacro)
@@ -7,5 +7,4 @@
   <xacro:arg name="driver_version" default="rsi_only"/>
   <xacro:arg name="mode" default="hardware"/>
-  <xacro:arg name="use_gpio" default="false"/>
   <xacro:arg name="gpio_config" default=""/>
   <xacro:arg name="roundtrip_time" default="0"/>
@@ -26,5 +25,5 @@
   <xacro:arg name="yaw" default="0"/>
   <xacro:arg name="rsi_xml_config_file" default=""/>
-  <xacro:kuka_agilus_ros2_control name="$(arg prefix)kr6_r900_2" driver_version="$(arg driver_version)" client_ip="$(arg client_ip)" client_port="$(arg client_port)" mxa_client_port="$(arg mxa_client_port)" controller_ip="$(arg controller_ip)" prefix="$(arg prefix)" mode="$(arg mode)" use_gpio="$(arg use_gpio)" gpio_config="$(arg gpio_config)" roundtrip_time="$(arg roundtrip_time)" verify_robot_model="$(arg verify_robot_model)" rsi_xml_config_file="$(arg rsi_xml_config_file)" is_async="$(arg is_async)" async_thread_priority="$(arg async_thread_priority)" async_affinity="$(arg async_affinity)">
+  <xacro:kuka_agilus_ros2_control name="$(arg prefix)kr6_r900_2" driver_version="$(arg driver_version)" client_ip="$(arg client_ip)" client_port="$(arg client_port)" mxa_client_port="$(arg mxa_client_port)" controller_ip="$(arg controller_ip)" prefix="$(arg prefix)" mode="$(arg mode)" gpio_config="$(arg gpio_config)" roundtrip_time="$(arg roundtrip_time)" verify_robot_model="$(arg verify_robot_model)" rsi_xml_config_file="$(arg rsi_xml_config_file)" is_async="$(arg is_async)" async_thread_priority="$(arg async_thread_priority)" async_affinity="$(arg async_affinity)">
     <ext_axes_ros2_control_joints/>
   </xacro:kuka_agilus_ros2_control>

File: kuka_agilus_support/urdf/kr6_r900_sixx.urdf.xacro (robot description, xacro)
@@ -7,5 +7,4 @@
   <xacro:arg name="driver_version" default="rsi_only"/>
   <xacro:arg name="mode" default="hardware"/>
-  <xacro:arg name="use_gpio" default="false"/>
   <xacro:arg name="gpio_config" default=""/>
   <xacro:arg name="roundtrip_time" default="0"/>
@@ -26,5 +25,5 @@
   <xacro:arg name="yaw" default="0"/>
   <xacro:arg name="rsi_xml_config_file" default=""/>
-  <xacro:kuka_agilus_ros2_control name="$(arg prefix)kr6_r900_sixx" driver_version="$(arg driver_version)" client_ip="$(arg client_ip)" client_port="$(arg client_port)" mxa_client_port="$(arg mxa_client_port)" controller_ip="$(arg controller_ip)" prefix="$(arg prefix)" mode="$(arg mode)" use_gpio="$(arg use_gpio)" gpio_config="$(arg gpio_config)" roundtrip_time="$(arg roundtrip_time)" verify_robot_model="$(arg verify_robot_model)" rsi_xml_config_file="$(arg rsi_xml_config_file)" is_async="$(arg is_async)" async_thread_priority="$(arg async_thread_priority)" async_affinity="$(arg async_affinity)">
+  <xacro:kuka_agilus_ros2_control name="$(arg prefix)kr6_r900_sixx" driver_version="$(arg driver_version)" client_ip="$(arg client_ip)" client_port="$(arg client_port)" mxa_client_port="$(arg mxa_client_port)" controller_ip="$(arg controller_ip)" prefix="$(arg prefix)" mode="$(arg mode)" gpio_config="$(arg gpio_config)" roundtrip_time="$(arg roundtrip_time)" verify_robot_model="$(arg verify_robot_model)" rsi_xml_config_file="$(arg rsi_xml_config_file)" is_async="$(arg is_async)" async_thread_priority="$(arg async_thread_priority)" async_affinity="$(arg async_affinity)">
     <ext_axes_ros2_control_joints/>
   </xacro:kuka_agilus_ros2_control>

File: kuka_agilus_support/urdf/kr7_r900_3.urdf.xacro (robot description, xacro)
@@ -19,5 +19,4 @@
   <xacro:arg name="driver_version" default="rsi_only"/>
   <xacro:arg name="mode" default="hardware"/>
-  <xacro:arg name="use_gpio" default="false"/>
   <xacro:arg name="gpio_config" default=""/>
   <xacro:arg name="roundtrip_time" default="0"/>
@@ -27,5 +26,5 @@
   <xacro:arg name="controller_ip" default="0.0.0.0"/>
   <xacro:arg name="verify_robot_model" default="true"/>
-  <xacro:kuka_agilus_ros2_control name="$(arg prefix)kr7_r900_3" driver_version="$(arg driver_version)" client_ip="$(arg client_ip)" client_port="$(arg client_port)" mxa_client_port="$(arg mxa_client_port)" controller_ip="$(arg controller_ip)" prefix="$(arg prefix)" mode="$(arg mode)" use_gpio="$(arg use_gpio)" gpio_config="$(arg gpio_config)" roundtrip_time="$(arg roundtrip_time)" verify_robot_model="$(arg verify_robot_model)" rsi_xml_config_file="$(arg rsi_xml_config_file)" is_async="$(arg is_async)" async_thread_priority="$(arg async_thread_priority)" async_affinity="$(arg async_affinity)">
+  <xacro:kuka_agilus_ros2_control name="$(arg prefix)kr7_r900_3" driver_version="$(arg driver_version)" client_ip="$(arg client_ip)" client_port="$(arg client_port)" mxa_client_port="$(arg mxa_client_port)" controller_ip="$(arg controller_ip)" prefix="$(arg prefix)" mode="$(arg mode)" gpio_config="$(arg gpio_config)" roundtrip_time="$(arg roundtrip_time)" verify_robot_model="$(arg verify_robot_model)" rsi_xml_config_file="$(arg rsi_xml_config_file)" is_async="$(arg is_async)" async_thread_priority="$(arg async_thread_priority)" async_affinity="$(arg async_affinity)">
     <ext_axes_ros2_control_joints/>
   </xacro:kuka_agilus_ros2_control>

File: kuka_agilus_support/urdf/kr_agilus_ros2_control_macro.xacro (robot description, xacro)
@@ -1,8 +1,5 @@
 <?xml version="1.0" encoding="UTF-8"?>
 <robot xmlns:xacro="http://www.ros.org/wiki/xacro">
-  <xacro:macro name="kuka_agilus_ros2_control" params="name driver_version client_ip client_port mxa_client_port controller_ip prefix mode use_gpio roundtrip_time verify_robot_model rsi_xml_config_file is_async async_thread_priority async_affinity gazebo_controller_config_path:=config/fake_hardware_config_6_axis.yaml gpio_config:='' **ext_axes_ros2_control_joints">
-    <xacro:if value="${gpio_config == ''}">
-      <xacro:property name="gpio_config" value="$(find kuka_rsi_driver)/config/gpio_config.xacro"/>
-    </xacro:if>
+  <xacro:macro name="kuka_agilus_ros2_control" params="name driver_version client_ip client_port mxa_client_port controller_ip prefix mode roundtrip_time verify_robot_model rsi_xml_config_file is_async async_thread_priority async_affinity gazebo_controller_config_path:=config/fake_hardware_config_6_axis.yaml gpio_config:='' **ext_axes_ros2_control_joints">
     <!-- gazebo -->
     <xacro:if value="${mode == 'gazebo'}">
@@ -151,11 +148,11 @@
         </xacro:unless>
       </joint>
-      <xacro:if value="${use_gpio}">
+      <xacro:unless value="${gpio_config == ''}">
         <xacro:include filename="${gpio_config}"/>
         <xacro:gpio_config/>
+      </xacro:unless>
+      <xacro:if value="${gpio_config == ''}">
+        <gpio name="gpio"/>
       </xacro:if>
-      <xacro:unless value="${use_gpio}">
-        <gpio name="gpio"/>
-      </xacro:unless>
     </ros2_control>
   </xacro:macro>

File: kuka_cybertech_support/urdf/kr12_r1450_3_hw.urdf.xacro (robot description, xacro)
@@ -7,5 +7,4 @@
   <xacro:arg name="driver_version" default="eki_rsi"/>
   <xacro:arg name="mode" default="hardware"/>
-  <xacro:arg name="use_gpio" default="false"/>
   <xacro:arg name="gpio_config" default=""/>
   <xacro:arg name="roundtrip_time" default="0"/>
@@ -26,5 +25,5 @@
   <xacro:arg name="yaw" default="0"/>
   <xacro:arg name="rsi_xml_config_file" default=""/>
-  <xacro:kuka_cybertech_ros2_control name="$(arg prefix)kr12_r1450_3_hw" driver_version="$(arg driver_version)" client_ip="$(arg client_ip)" client_port="$(arg client_port)" mxa_client_port="$(arg mxa_client_port)" controller_ip="$(arg controller_ip)" prefix="$(arg prefix)" mode="$(arg mode)" use_gpio="$(arg use_gpio)" gpio_config="$(arg gpio_config)" roundtrip_time="$(arg roundtrip_time)" verify_robot_model="$(arg verify_robot_model)" rsi_xml_config_file="$(arg rsi_xml_config_file)" is_async="$(arg is_async)" async_thread_priority="$(arg async_thread_priority)" async_affinity="$(arg async_affinity)">
+  <xacro:kuka_cybertech_ros2_control name="$(arg prefix)kr12_r1450_3_hw" driver_version="$(arg driver_version)" client_ip="$(arg client_ip)" client_port="$(arg client_port)" mxa_client_port="$(arg mxa_client_port)" controller_ip="$(arg controller_ip)" prefix="$(arg prefix)" mode="$(arg mode)" gpio_config="$(arg gpio_config)" roundtrip_time="$(arg roundtrip_time)" verify_robot_model="$(arg verify_robot_model)" rsi_xml_config_file="$(arg rsi_xml_config_file)" is_async="$(arg is_async)" async_thread_priority="$(arg async_thread_priority)" async_affinity="$(arg async_affinity)">
     <ext_axes_ros2_control_joints/>
   </xacro:kuka_cybertech_ros2_control>
