Commit message: Drop use_gpio in favour of gpio_config alone
Remove the use_gpio argument from every ros2_control macro and
per-model urdf.xacro. Whether GPIO is enabled is now derived from
gpio_config: empty means no GPIO, a path means include and instantiate
that GPIO xacro file. This also drops the unconditional
$(find kuka_rsi_driver) fallback resolution for the disabled case.

Co-Authored-By: Claude Sonnet 5 <noreply@anthropic.com>

File: kuka_cybertech_support/urdf/kr16_r1610_2.urdf.xacro (robot description, xacro)
@@ -7,5 +7,4 @@
   <xacro:arg name="driver_version" default="eki_rsi"/>
   <xacro:arg name="mode" default="hardware"/>
-  <xacro:arg name="use_gpio" default="false"/>
   <xacro:arg name="gpio_config" default=""/>
   <xacro:arg name="roundtrip_time" default="0"/>
@@ -26,5 +25,5 @@
   <xacro:arg name="yaw" default="0"/>
   <xacro:arg name="rsi_xml_config_file" default=""/>
-  <xacro:kuka_cybertech_ros2_control name="$(arg prefix)kr16_r1610_2" driver_version="$(arg driver_version)" client_ip="$(arg client_ip)" client_port="$(arg client_port)" mxa_client_port="$(arg mxa_client_port)" controller_ip="$(arg controller_ip)" prefix="$(arg prefix)" mode="$(arg mode)" use_gpio="$(arg use_gpio)" gpio_config="$(arg gpio_config)" roundtrip_time="$(arg roundtrip_time)" verify_robot_model="$(arg verify_robot_model)" rsi_xml_config_file="$(arg rsi_xml_config_file)" is_async="$(arg is_async)" async_thread_priority="$(arg async_thread_priority)" async_affinity="$(arg async_affinity)">
+  <xacro:kuka_cybertech_ros2_control name="$(arg prefix)kr16_r1610_2" driver_version="$(arg driver_version)" client_ip="$(arg client_ip)" client_port="$(arg client_port)" mxa_client_port="$(arg mxa_client_port)" controller_ip="$(arg controller_ip)" prefix="$(arg prefix)" mode="$(arg mode)" gpio_config="$(arg gpio_config)" roundtrip_time="$(arg roundtrip_time)" verify_robot_model="$(arg verify_robot_model)" rsi_xml_config_file="$(arg rsi_xml_config_file)" is_async="$(arg is_async)" async_thread_priority="$(arg async_thread_priority)" async_affinity="$(arg async_affinity)">
     <ext_axes_ros2_control_joints/>
   </xacro:kuka_cybertech_ros2_control>

File: kuka_cybertech_support/urdf/kr16_r2010_2.urdf.xacro (robot description, xacro)
@@ -7,5 +7,4 @@
   <xacro:arg name="driver_version" default="eki_rsi"/>
   <xacro:arg name="mode" default="hardware"/>
-  <xacro:arg name="use_gpio" default="false"/>
   <xacro:arg name="gpio_config" default=""/>
   <xacro:arg name="roundtrip_time" default="0"/>
@@ -26,5 +25,5 @@
   <xacro:arg name="yaw" default="0"/>
   <xacro:arg name="rsi_xml_config_file" default=""/>
-  <xacro:kuka_cybertech_ros2_control name="$(arg prefix)kr16_r2010_2" driver_version="$(arg driver_version)" client_ip="$(arg client_ip)" client_port="$(arg client_port)" mxa_client_port="$(arg mxa_client_port)" controller_ip="$(arg controller_ip)" prefix="$(arg prefix)" mode="$(arg mode)" use_gpio="$(arg use_gpio)" gpio_config="$(arg gpio_config)" roundtrip_time="$(arg roundtrip_time)" verify_robot_model="$(arg verify_robot_model)" rsi_xml_config_file="$(arg rsi_xml_config_file)" is_async="$(arg is_async)" async_thread_priority="$(arg async_thread_priority)" async_affinity="$(arg async_affinity)">
+  <xacro:kuka_cybertech_ros2_control name="$(arg prefix)kr16_r2010_2" driver_version="$(arg driver_version)" client_ip="$(arg client_ip)" client_port="$(arg client_port)" mxa_client_port="$(arg mxa_client_port)" controller_ip="$(arg controller_ip)" prefix="$(arg prefix)" mode="$(arg mode)" gpio_config="$(arg gpio_config)" roundtrip_time="$(arg roundtrip_time)" verify_robot_model="$(arg verify_robot_model)" rsi_xml_config_file="$(arg rsi_xml_config_file)" is_async="$(arg is_async)" async_thread_priority="$(arg async_thread_priority)" async_affinity="$(arg async_affinity)">
     <ext_axes_ros2_control_joints/>
   </xacro:kuka_cybertech_ros2_control>

File: kuka_cybertech_support/urdf/kr20_r1810_2.urdf.xacro (robot description, xacro)
@@ -7,5 +7,4 @@
   <xacro:arg name="driver_version" default="eki_rsi"/>
   <xacro:arg name="mode" default="hardware"/>
-  <xacro:arg name="use_gpio" default="false"/>
   <xacro:arg name="gpio_config" default=""/>
   <xacro:arg name="roundtrip_time" default="0"/>
@@ -26,5 +25,5 @@
   <xacro:arg name="yaw" default="0"/>
   <xacro:arg name="rsi_xml_config_file" default=""/>
-  <xacro:kuka_cybertech_ros2_control name="$(arg prefix)kr20_r1810_2" driver_version="$(arg driver_version)" client_ip="$(arg client_ip)" client_port="$(arg client_port)" mxa_client_port="$(arg mxa_client_port)" controller_ip="$(arg controller_ip)" prefix="$(arg prefix)" mode="$(arg mode)" use_gpio="$(arg use_gpio)" gpio_config="$(arg gpio_config)" roundtrip_time="$(arg roundtrip_time)" verify_robot_model="$(arg verify_robot_model)" rsi_xml_config_file="$(arg rsi_xml_config_file)" is_async="$(arg is_async)" async_thread_priority="$(arg async_thread_priority)" async_affinity="$(arg async_affinity)">
+  <xacro:kuka_cybertech_ros2_control name="$(arg prefix)kr20_r1810_2" driver_version="$(arg driver_version)" client_ip="$(arg client_ip)" client_port="$(arg client_port)" mxa_client_port="$(arg mxa_client_port)" controller_ip="$(arg controller_ip)" prefix="$(arg prefix)" mode="$(arg mode)" gpio_config="$(arg gpio_config)" roundtrip_time="$(arg roundtrip_time)" verify_robot_model="$(arg verify_robot_model)" rsi_xml_config_file="$(arg rsi_xml_config_file)" is_async="$(arg is_async)" async_thread_priority="$(arg async_thread_priority)" async_affinity="$(arg async_affinity)">
     <ext_axes_ros2_control_joints/>
   </xacro:kuka_cybertech_ros2_control>

File: kuka_cybertech_support/urdf/kr20_r1820_2_e.urdf.xacro (robot description, xacro)
@@ -19,5 +19,4 @@
   <xacro:arg name="driver_version" default="rsi_only"/>
   <xacro:arg name="mode" default="hardware"/>
-  <xacro:arg name="use_gpio" default="false"/>
   <xacro:arg name="gpio_config" default=""/>
   <xacro:arg name="roundtrip_time" default="0"/>
@@ -27,5 +26,5 @@
   <xacro:arg name="controller_ip" default="0.0.0.0"/>
   <xacro:arg name="verify_robot_model" default="true"/>
-  <xacro:kuka_cybertech_ros2_control name="$(arg prefix)kr20_r1820_2_e" driver_version="$(arg driver_version)" client_ip="$(arg client_ip)" client_port="$(arg client_port)" mxa_client_port="$(arg mxa_client_port)" controller_ip="$(arg controller_ip)" prefix="$(arg prefix)" mode="$(arg mode)" use_gpio="$(arg use_gpio)" gpio_config="$(arg gpio_config)" roundtrip_time="$(arg roundtrip_time)" verify_robot_model="$(arg verify_robot_model)" rsi_xml_config_file="$(arg rsi_xml_config_file)" is_async="$(arg is_async)" async_thread_priority="$(arg async_thread_priority)" async_affinity="$(arg async_affinity)">
+  <xacro:kuka_cybertech_ros2_control name="$(arg prefix)kr20_r1820_2_e" driver_version="$(arg driver_version)" client_ip="$(arg client_ip)" client_port="$(arg client_port)" mxa_client_port="$(arg mxa_client_port)" controller_ip="$(arg controller_ip)" prefix="$(arg prefix)" mode="$(arg mode)" gpio_config="$(arg gpio_config)" roundtrip_time="$(arg roundtrip_time)" verify_robot_model="$(arg verify_robot_model)" rsi_xml_config_file="$(arg rsi_xml_config_file)" is_async="$(arg is_async)" async_thread_priority="$(arg async_thread_priority)" async_affinity="$(arg async_affinity)">
     <ext_axes_ros2_control_joints/>
   </xacro:kuka_cybertech_ros2_control>

File: kuka_cybertech_support/urdf/kr35_r1840_3.urdf.xacro (robot description, xacro)
@@ -18,5 +18,4 @@
   <xacro:arg name="driver_version" default="rsi_only"/>
   <xacro:arg name="mode" default="hardware"/>
-  <xacro:arg name="use_gpio" default="false"/>
   <xacro:arg name="gpio_config" default=""/>
   <xacro:arg name="roundtrip_time" default="0"/>
@@ -27,5 +26,5 @@
   <xacro:arg name="verify_robot_model" default="true"/>
   <xacro:arg name="rsi_xml_config_file" default=""/>
-  <xacro:kuka_cybertech_ros2_control name="$(arg prefix)kr35_r1840_3" driver_version="$(arg driver_version)" client_ip="$(arg client_ip)" client_port="$(arg client_port)" mxa_client_port="$(arg mxa_client_port)" controller_ip="$(arg controller_ip)" prefix="$(arg prefix)" mode="$(arg mode)" use_gpio="$(arg use_gpio)" gpio_config="$(arg gpio_config)" roundtrip_time="$(arg roundtrip_time)" verify_robot_model="$(arg verify_robot_model)" rsi_xml_config_file="$(arg rsi_xml_config_file)" is_async="$(arg is_async)" async_thread_priority="$(arg async_thread_priority)" async_affinity="$(arg async_affinity)">
+  <xacro:kuka_cybertech_ros2_control name="$(arg prefix)kr35_r1840_3" driver_version="$(arg driver_version)" client_ip="$(arg client_ip)" client_port="$(arg client_port)" mxa_client_port="$(arg mxa_client_port)" controller_ip="$(arg controller_ip)" prefix="$(arg prefix)" mode="$(arg mode)" gpio_config="$(arg gpio_config)" roundtrip_time="$(arg roundtrip_time)" verify_robot_model="$(arg verify_robot_model)" rsi_xml_config_file="$(arg rsi_xml_config_file)" is_async="$(arg is_async)" async_thread_priority="$(arg async_thread_priority)" async_affinity="$(arg async_affinity)">
     <ext_axes_ros2_control_joints/>
   </xacro:kuka_cybertech_ros2_control>

File: kuka_cybertech_support/urdf/kr35_r1840_3_hw.urdf.xacro (robot description, xacro)
@@ -18,5 +18,4 @@
   <xacro:arg name="driver_version" default="rsi_only"/>
   <xacro:arg name="mode" default="hardware"/>
-  <xacro:arg name="use_gpio" default="false"/>
   <xacro:arg name="gpio_config" default=""/>
   <xacro:arg name="roundtrip_time" default="0"/>
@@ -27,5 +26,5 @@
   <xacro:arg name="verify_robot_model" default="true"/>
   <xacro:arg name="rsi_xml_config_file" default=""/>
-  <xacro:kuka_cybertech_ros2_control name="$(arg prefix)kr35_r1840_3_hw" driver_version="$(arg driver_version)" client_ip="$(arg client_ip)" client_port="$(arg client_port)" mxa_client_port="$(arg mxa_client_port)" controller_ip="$(arg controller_ip)" prefix="$(arg prefix)" mode="$(arg mode)" use_gpio="$(arg use_gpio)" gpio_config="$(arg gpio_config)" roundtrip_time="$(arg roundtrip_time)" verify_robot_model="$(arg verify_robot_model)" rsi_xml_config_file="$(arg rsi_xml_config_file)" is_async="$(arg is_async)" async_thread_priority="$(arg async_thread_priority)" async_affinity="$(arg async_affinity)">
+  <xacro:kuka_cybertech_ros2_control name="$(arg prefix)kr35_r1840_3_hw" driver_version="$(arg driver_version)" client_ip="$(arg client_ip)" client_port="$(arg client_port)" mxa_client_port="$(arg mxa_client_port)" controller_ip="$(arg controller_ip)" prefix="$(arg prefix)" mode="$(arg mode)" gpio_config="$(arg gpio_config)" roundtrip_time="$(arg roundtrip_time)" verify_robot_model="$(arg verify_robot_model)" rsi_xml_config_file="$(arg rsi_xml_config_file)" is_async="$(arg is_async)" async_thread_priority="$(arg async_thread_priority)" async_affinity="$(arg async_affinity)">
     <ext_axes_ros2_control_joints/>
   </xacro:kuka_cybertech_ros2_control>

File: kuka_cybertech_support/urdf/kr8_r1440_2_arc_hw.urdf.xacro (robot description, xacro)
@@ -7,5 +7,4 @@
   <xacro:arg name="driver_version" default="eki_rsi"/>
   <xacro:arg name="mode" default="hardware"/>
-  <xacro:arg name="use_gpio" default="false"/>
   <xacro:arg name="gpio_config" default=""/>
   <xacro:arg name="roundtrip_time" default="0"/>
@@ -26,5 +25,5 @@
   <xacro:arg name="yaw" default="0"/>
   <xacro:arg name="rsi_xml_config_file" default=""/>
-  <xacro:kuka_cybertech_ros2_control name="$(arg prefix)kr8_r1440_2_arc_hw" driver_version="$(arg driver_version)" client_ip="$(arg client_ip)" client_port="$(arg client_port)" mxa_client_port="$(arg mxa_client_port)" controller_ip="$(arg controller_ip)" prefix="$(arg prefix)" mode="$(arg mode)" use_gpio="$(arg use_gpio)" gpio_config="$(arg gpio_config)" roundtrip_time="$(arg roundtrip_time)" verify_robot_model="$(arg verify_robot_model)" rsi_xml_config_file="$(arg rsi_xml_config_file)" is_async="$(arg is_async)" async_thread_priority="$(arg async_thread_priority)" async_affinity="$(arg async_affinity)">
+  <xacro:kuka_cybertech_ros2_control name="$(arg prefix)kr8_r1440_2_arc_hw" driver_version="$(arg driver_version)" client_ip="$(arg client_ip)" client_port="$(arg client_port)" mxa_client_port="$(arg mxa_client_port)" controller_ip="$(arg controller_ip)" prefix="$(arg prefix)" mode="$(arg mode)" gpio_config="$(arg gpio_config)" roundtrip_time="$(arg roundtrip_time)" verify_robot_model="$(arg verify_robot_model)" rsi_xml_config_file="$(arg rsi_xml_config_file)" is_async="$(arg is_async)" async_thread_priority="$(arg async_thread_priority)" async_affinity="$(arg async_affinity)">
     <ext_axes_ros2_control_joints/>
   </xacro:kuka_cybertech_ros2_control>
