Commit message: Expose gpio_config as a configurable xacro argument (backport #287) (#288)
* Expose gpio_config as a configurable xacro argument (#287)

* Expose gpio_config as a configurable xacro argument

Add a gpio_config argument to every ros2_control macro that supports
use_gpio, defaulting to the existing kuka_rsi_driver gpio_config.xacro
when left empty. This lets a launch file point use_gpio at a custom
GPIO xacro file, for example to describe external IOs, instead of
always including the driver's default config.

Wire the argument through every per-model urdf.xacro so it can be set
from the top level.

Co-Authored-By: Claude Sonnet 5 <noreply@anthropic.com>

* Drop use_gpio in favour of gpio_config alone

Remove the use_gpio argument from every ros2_control macro and
per-model urdf.xacro. Whether GPIO is enabled is now derived from
gpio_config: empty means no GPIO, a path means include and instantiate
that GPIO xacro file. This also drops the unconditional
$(find kuka_rsi_driver) fallback resolution for the disabled case.

Co-Authored-By: Claude Sonnet 5 <noreply@anthropic.com>

* Fix drive_package typo in README GPIO section

Co-Authored-By: Claude Sonnet 5 <noreply@anthropic.com>

* new kr210 + templates

---------

Co-authored-by: Dr. Denis <denis.stogl@b-robotized.com>
Co-authored-by: Claude Sonnet 5 <noreply@anthropic.com>
(cherry picked from commit f0202b281d40d16c90ceeed23d1a9548dd0c3981)

# Conflicts:
#	kuka_agilus_support/urdf/kr10_r1100_2.urdf.xacro
#	kuka_agilus_support/urdf/kr10_r1100_3.urdf.xacro
#	kuka_agilus_support/urdf/kr10_r900_2.urdf.xacro
#	kuka_agilus_support/urdf/kr13_r900_3.urdf.xacro
#	kuka_agilus_support/urdf/kr16_r1100_3.urdf.xacro
#	kuka_agilus_support/urdf/kr4_r600.urdf.xacro
#	kuka_agilus_support/urdf/kr6_r700_2.urdf.xacro
#	kuka_agilus_support/urdf/kr6_r700_sixx.urdf.xacro
#	kuka_agilus_support/urdf/kr6_r900_2.urdf.xacro
#	kuka_agilus_support/urdf/kr6_r900_sixx.urdf.xacro
#	kuka_agilus_support/urdf/kr7_r900_3.urdf.xacro
#	kuka_agilus_support/urdf/kr_agilus_ros2_control_macro.xacro
#	kuka_cybertech_support/urdf/kr12_r1450_3_hw.urdf.xacro
#	kuka_cybertech_support/urdf/kr16_r1610_2.urdf.xacro
#	kuka_cybertech_support/urdf/kr16_r2010_2.urdf.xacro
#	kuka_cybertech_support/urdf/kr20_r1810_2.urdf.xacro
#	kuka_cybertech_support/urdf/kr20_r1820_2_e.urdf.xacro
#	kuka_cybertech_support/urdf/kr35_r1840_3.urdf.xacro
#	kuka_cybertech_support/urdf/kr35_r1840_3_hw.urdf.xacro
#	kuka_cybertech_support/urdf/kr8_r1440_2_arc_hw.urdf.xacro
#	kuka_cybertech_support/urdf/kr8_r2100_2_arc_hw.urdf.xacro
#	kuka_cybertech_support/urdf/kr_cybertech_ros2_control_macro.xacro
#	kuka_fortec_support/urdf/kr240_r3330.urdf.xacro
#	kuka_fortec_support/urdf/kr300_r2800_2_mt.urdf.xacro
#	kuka_fortec_support/urdf/kr340_r3400_2.urdf.xacro
#	kuka_fortec_support/urdf/kr360_r2830.urdf.xacro
#	kuka_fortec_support/urdf/kr500_r2800_2.urdf.xacro
#	kuka_fortec_support/urdf/kr560_r3100_2.urdf.xacro
#	kuka_fortec_support/urdf/kr600_r2830.urdf.xacro
#	kuka_fortec_support/urdf/kr800_r2800_2.urdf.xacro
#	kuka_fortec_support/urdf/kr_fortec_ros2_control_macro.xacro
#	kuka_iontec_support/urdf/kr20_r3100.urdf.xacro
#	kuka_iontec_support/urdf/kr30_r2100.urdf.xacro
#	kuka_iontec_support/urdf/kr50_r2100.urdf.xacro
#	kuka_iontec_support/urdf/kr50_r2500.urdf.xacro
#	kuka_iontec_support/urdf/kr70_r2100.urdf.xacro
#	kuka_iontec_support/urdf/kr_iontec_ros2_control_macro.xacro
#	kuka_lbr_iico_support/urdf/lbr_iico12_r1260.urdf.xacro
#	kuka_lbr_iico_support/urdf/lbr_iico7_r900.urdf.xacro
#	kuka_lbr_iico_support/urdf/lbr_iico_ros2_control_macro.xacro
#	kuka_lbr_iisy_support/urdf/lbr_iisy11_r1300.urdf.xacro
#	kuka_lbr_iisy_support/urdf/lbr_iisy15_r930.urdf.xacro
#	kuka_lbr_iisy_support/urdf/lbr_iisy3_r760.urdf.xacro
#	kuka_lbr_iisy_support/urdf/lbr_iisy8_r930.urdf.xacro
#	kuka_lbr_iisy_support/urdf/lbr_iisy_ros2_control_macro.xacro
#	kuka_quantec_support/urdf/kr120_r2700_2.urdf.xacro
#	kuka_quantec_support/urdf/kr150_r3100_2.urdf.xacro
#	kuka_quantec_support/urdf/kr210_r2700_2.urdf.xacro
#	kuka_quantec_support/urdf/kr210_r2700_extra.urdf.xacro
#	kuka_quantec_support/urdf/kr210_r3100_2.urdf.xacro
#	kuka_quantec_support/urdf/kr210_r3100_ultra.urdf.xacro
#	kuka_quantec_support/urdf/kr210_r3300_2_k.urdf.xacro
#	kuka_quantec_support/urdf/kr240_r2900_2.urdf.xacro
#	kuka_quantec_support/urdf/kr300_r2700_2.urdf.xacro
#	kuka_quantec_support/urdf/kr_quantec_ros2_control_macro.xacro
#	kuka_resources/urdf/dual_arm_template.urdf.xacro
#	kuka_resources/urdf/robot_with_external_axis_template.urdf.xacro

* merge conflicts

* no dual arm for humble

---------

Co-authored-by: Áron Svastits <49677296+Svastits@users.noreply.github.com>

File: kuka_agilus_support/urdf/kr10_r1100_2.urdf.xacro (robot description, xacro)
@@ -7,5 +7,5 @@
   <xacro:arg name="driver_version" default="rsi_only"/>
   <xacro:arg name="mode" default="hardware"/>
-  <xacro:arg name="use_gpio" default="false"/>
+  <xacro:arg name="gpio_config" default=""/>
   <xacro:arg name="roundtrip_time" default="0"/>
   <xacro:arg name="client_ip" default="0.0.0.0"/>
@@ -22,5 +22,5 @@
   <xacro:arg name="yaw" default="0"/>
   <xacro:arg name="rsi_xml_config_file" default=""/>
-  <xacro:kuka_agilus_ros2_control name="$(arg prefix)kr10_r1100_2" driver_version="$(arg driver_version)" client_ip="$(arg client_ip)" client_port="$(arg client_port)" mxa_client_port="$(arg mxa_client_port)" controller_ip="$(arg controller_ip)" prefix="$(arg prefix)" mode="$(arg mode)" use_gpio="$(arg use_gpio)" roundtrip_time="$(arg roundtrip_time)" verify_robot_model="$(arg verify_robot_model)" rsi_xml_config_file="$(arg rsi_xml_config_file)">
+  <xacro:kuka_agilus_ros2_control name="$(arg prefix)kr10_r1100_2" driver_version="$(arg driver_version)" client_ip="$(arg client_ip)" client_port="$(arg client_port)" mxa_client_port="$(arg mxa_client_port)" controller_ip="$(arg controller_ip)" prefix="$(arg prefix)" mode="$(arg mode)" gpio_config="$(arg gpio_config)" roundtrip_time="$(arg roundtrip_time)" verify_robot_model="$(arg verify_robot_model)" rsi_xml_config_file="$(arg rsi_xml_config_file)">
     <ext_axes_ros2_control_joints/>
   </xacro:kuka_agilus_ros2_control>

File: kuka_agilus_support/urdf/kr10_r1100_3.urdf.xacro (robot description, xacro)
@@ -16,5 +16,5 @@
   <xacro:arg name="driver_version" default="rsi_only"/>
   <xacro:arg name="mode" default="hardware"/>
-  <xacro:arg name="use_gpio" default="false"/>
+  <xacro:arg name="gpio_config" default=""/>
   <xacro:arg name="roundtrip_time" default="0"/>
   <xacro:arg name="client_ip" default="0.0.0.0"/>
@@ -23,5 +23,5 @@
   <xacro:arg name="controller_ip" default="0.0.0.0"/>
   <xacro:arg name="verify_robot_model" default="true"/>
-  <xacro:kuka_agilus_ros2_control name="$(arg prefix)kr10_r1100_3" driver_version="$(arg driver_version)" client_ip="$(arg client_ip)" client_port="$(arg client_port)" mxa_client_port="$(arg mxa_client_port)" controller_ip="$(arg controller_ip)" prefix="$(arg prefix)" mode="$(arg mode)" use_gpio="$(arg use_gpio)" roundtrip_time="$(arg roundtrip_time)" verify_robot_model="$(arg verify_robot_model)" rsi_xml_config_file="$(arg rsi_xml_config_file)">
+  <xacro:kuka_agilus_ros2_control name="$(arg prefix)kr10_r1100_3" driver_version="$(arg driver_version)" client_ip="$(arg client_ip)" client_port="$(arg client_port)" mxa_client_port="$(arg mxa_client_port)" controller_ip="$(arg controller_ip)" prefix="$(arg prefix)" mode="$(arg mode)" gpio_config="$(arg gpio_config)" roundtrip_time="$(arg roundtrip_time)" verify_robot_model="$(arg verify_robot_model)" rsi_xml_config_file="$(arg rsi_xml_config_file)">
     <ext_axes_ros2_control_joints/>
   </xacro:kuka_agilus_ros2_control>

File: kuka_agilus_support/urdf/kr10_r900_2.urdf.xacro (robot description, xacro)
@@ -7,5 +7,5 @@
   <xacro:arg name="driver_version" default="rsi_only"/>
   <xacro:arg name="mode" default="hardware"/>
-  <xacro:arg name="use_gpio" default="false"/>
+  <xacro:arg name="gpio_config" default=""/>
   <xacro:arg name="roundtrip_time" default="0"/>
   <xacro:arg name="client_ip" default="0.0.0.0"/>
@@ -22,5 +22,5 @@
   <xacro:arg name="yaw" default="0"/>
   <xacro:arg name="rsi_xml_config_file" default=""/>
-  <xacro:kuka_agilus_ros2_control name="$(arg prefix)kr10_r900_2" driver_version="$(arg driver_version)" client_ip="$(arg client_ip)" client_port="$(arg client_port)" mxa_client_port="$(arg mxa_client_port)" controller_ip="$(arg controller_ip)" prefix="$(arg prefix)" mode="$(arg mode)" use_gpio="$(arg use_gpio)" roundtrip_time="$(arg roundtrip_time)" verify_robot_model="$(arg verify_robot_model)" rsi_xml_config_file="$(arg rsi_xml_config_file)">
+  <xacro:kuka_agilus_ros2_control name="$(arg prefix)kr10_r900_2" driver_version="$(arg driver_version)" client_ip="$(arg client_ip)" client_port="$(arg client_port)" mxa_client_port="$(arg mxa_client_port)" controller_ip="$(arg controller_ip)" prefix="$(arg prefix)" mode="$(arg mode)" gpio_config="$(arg gpio_config)" roundtrip_time="$(arg roundtrip_time)" verify_robot_model="$(arg verify_robot_model)" rsi_xml_config_file="$(arg rsi_xml_config_file)">
     <ext_axes_ros2_control_joints/>
   </xacro:kuka_agilus_ros2_control>

File: kuka_agilus_support/urdf/kr13_r900_3.urdf.xacro (robot description, xacro)
@@ -16,5 +16,5 @@
   <xacro:arg name="driver_version" default="rsi_only"/>
   <xacro:arg name="mode" default="hardware"/>
-  <xacro:arg name="use_gpio" default="false"/>
+  <xacro:arg name="gpio_config" default=""/>
   <xacro:arg name="roundtrip_time" default="0"/>
   <xacro:arg name="client_ip" default="0.0.0.0"/>
@@ -23,5 +23,5 @@
   <xacro:arg name="controller_ip" default="0.0.0.0"/>
   <xacro:arg name="verify_robot_model" default="true"/>
-  <xacro:kuka_agilus_ros2_control name="$(arg prefix)kr13_r900_3" driver_version="$(arg driver_version)" client_ip="$(arg client_ip)" client_port="$(arg client_port)" mxa_client_port="$(arg mxa_client_port)" controller_ip="$(arg controller_ip)" prefix="$(arg prefix)" mode="$(arg mode)" use_gpio="$(arg use_gpio)" roundtrip_time="$(arg roundtrip_time)" verify_robot_model="$(arg verify_robot_model)" rsi_xml_config_file="$(arg rsi_xml_config_file)">
+  <xacro:kuka_agilus_ros2_control name="$(arg prefix)kr13_r900_3" driver_version="$(arg driver_version)" client_ip="$(arg client_ip)" client_port="$(arg client_port)" mxa_client_port="$(arg mxa_client_port)" controller_ip="$(arg controller_ip)" prefix="$(arg prefix)" mode="$(arg mode)" gpio_config="$(arg gpio_config)" roundtrip_time="$(arg roundtrip_time)" verify_robot_model="$(arg verify_robot_model)" rsi_xml_config_file="$(arg rsi_xml_config_file)">
     <ext_axes_ros2_control_joints/>
   </xacro:kuka_agilus_ros2_control>

File: kuka_agilus_support/urdf/kr16_r1100_3.urdf.xacro (robot description, xacro)
@@ -16,5 +16,5 @@
   <xacro:arg name="driver_version" default="rsi_only"/>
   <xacro:arg name="mode" default="hardware"/>
-  <xacro:arg name="use_gpio" default="false"/>
+  <xacro:arg name="gpio_config" default=""/>
   <xacro:arg name="roundtrip_time" default="0"/>
   <xacro:arg name="client_ip" default="0.0.0.0"/>
@@ -23,5 +23,5 @@
   <xacro:arg name="controller_ip" default="0.0.0.0"/>
   <xacro:arg name="verify_robot_model" default="true"/>
-  <xacro:kuka_agilus_ros2_control name="$(arg prefix)kr16_r1100_3" driver_version="$(arg driver_version)" client_ip="$(arg client_ip)" client_port="$(arg client_port)" mxa_client_port="$(arg mxa_client_port)" controller_ip="$(arg controller_ip)" prefix="$(arg prefix)" mode="$(arg mode)" use_gpio="$(arg use_gpio)" roundtrip_time="$(arg roundtrip_time)" verify_robot_model="$(arg verify_robot_model)" rsi_xml_config_file="$(arg rsi_xml_config_file)">
+  <xacro:kuka_agilus_ros2_control name="$(arg prefix)kr16_r1100_3" driver_version="$(arg driver_version)" client_ip="$(arg client_ip)" client_port="$(arg client_port)" mxa_client_port="$(arg mxa_client_port)" controller_ip="$(arg controller_ip)" prefix="$(arg prefix)" mode="$(arg mode)" gpio_config="$(arg gpio_config)" roundtrip_time="$(arg roundtrip_time)" verify_robot_model="$(arg verify_robot_model)" rsi_xml_config_file="$(arg rsi_xml_config_file)">
     <ext_axes_ros2_control_joints/>
   </xacro:kuka_agilus_ros2_control>

File: kuka_agilus_support/urdf/kr4_r600.urdf.xacro (robot description, xacro)
@@ -7,5 +7,5 @@
   <xacro:arg name="driver_version" default="rsi_only"/>
   <xacro:arg name="mode" default="hardware"/>
-  <xacro:arg name="use_gpio" default="false"/>
+  <xacro:arg name="gpio_config" default=""/>
   <xacro:arg name="roundtrip_time" default="0"/>
   <xacro:arg name="client_ip" default="0.0.0.0"/>
@@ -22,5 +22,5 @@
   <xacro:arg name="yaw" default="0"/>
   <xacro:arg name="rsi_xml_config_file" default=""/>
-  <xacro:kuka_agilus_ros2_control name="$(arg prefix)kr4_r600" driver_version="$(arg driver_version)" client_ip="$(arg client_ip)" client_port="$(arg client_port)" mxa_client_port="$(arg mxa_client_port)" controller_ip="$(arg controller_ip)" prefix="$(arg prefix)" mode="$(arg mode)" use_gpio="$(arg use_gpio)" roundtrip_time="$(arg roundtrip_time)" verify_robot_model="$(arg verify_robot_model)" rsi_xml_config_file="$(arg rsi_xml_config_file)">
+  <xacro:kuka_agilus_ros2_control name="$(arg prefix)kr4_r600" driver_version="$(arg driver_version)" client_ip="$(arg client_ip)" client_port="$(arg client_port)" mxa_client_port="$(arg mxa_client_port)" controller_ip="$(arg controller_ip)" prefix="$(arg prefix)" mode="$(arg mode)" gpio_config="$(arg gpio_config)" roundtrip_time="$(arg roundtrip_time)" verify_robot_model="$(arg verify_robot_model)" rsi_xml_config_file="$(arg rsi_xml_config_file)">
     <ext_axes_ros2_control_joints/>
   </xacro:kuka_agilus_ros2_control>

File: kuka_agilus_support/urdf/kr6_r700_2.urdf.xacro (robot description, xacro)
@@ -7,5 +7,5 @@
   <xacro:arg name="driver_version" default="rsi_only"/>
   <xacro:arg name="mode" default="hardware"/>
-  <xacro:arg name="use_gpio" default="false"/>
+  <xacro:arg name="gpio_config" default=""/>
   <xacro:arg name="roundtrip_time" default="0"/>
   <xacro:arg name="client_ip" default="0.0.0.0"/>
@@ -22,5 +22,5 @@
   <xacro:arg name="yaw" default="0"/>
   <xacro:arg name="rsi_xml_config_file" default=""/>
-  <xacro:kuka_agilus_ros2_control name="$(arg prefix)kr6_r700_2" driver_version="$(arg driver_version)" client_ip="$(arg client_ip)" client_port="$(arg client_port)" mxa_client_port="$(arg mxa_client_port)" controller_ip="$(arg controller_ip)" prefix="$(arg prefix)" mode="$(arg mode)" use_gpio="$(arg use_gpio)" roundtrip_time="$(arg roundtrip_time)" verify_robot_model="$(arg verify_robot_model)" rsi_xml_config_file="$(arg rsi_xml_config_file)">
+  <xacro:kuka_agilus_ros2_control name="$(arg prefix)kr6_r700_2" driver_version="$(arg driver_version)" client_ip="$(arg client_ip)" client_port="$(arg client_port)" mxa_client_port="$(arg mxa_client_port)" controller_ip="$(arg controller_ip)" prefix="$(arg prefix)" mode="$(arg mode)" gpio_config="$(arg gpio_config)" roundtrip_time="$(arg roundtrip_time)" verify_robot_model="$(arg verify_robot_model)" rsi_xml_config_file="$(arg rsi_xml_config_file)">
     <ext_axes_ros2_control_joints/>
   </xacro:kuka_agilus_ros2_control>

File: kuka_agilus_support/urdf/kr6_r700_sixx.urdf.xacro (robot description, xacro)
@@ -7,5 +7,5 @@
   <xacro:arg name="driver_version" default="rsi_only"/>
   <xacro:arg name="mode" default="hardware"/>
-  <xacro:arg name="use_gpio" default="false"/>
+  <xacro:arg name="gpio_config" default=""/>
   <xacro:arg name="roundtrip_time" default="0"/>
   <xacro:arg name="client_ip" default="0.0.0.0"/>
@@ -22,5 +22,5 @@
   <xacro:arg name="yaw" default="0"/>
   <xacro:arg name="rsi_xml_config_file" default=""/>
-  <xacro:kuka_agilus_ros2_control name="$(arg prefix)kr6_r700_sixx" driver_version="$(arg driver_version)" client_ip="$(arg client_ip)" client_port="$(arg client_port)" mxa_client_port="$(arg mxa_client_port)" controller_ip="$(arg controller_ip)" prefix="$(arg prefix)" mode="$(arg mode)" use_gpio="$(arg use_gpio)" roundtrip_time="$(arg roundtrip_time)" verify_robot_model="$(arg verify_robot_model)" rsi_xml_config_file="$(arg rsi_xml_config_file)">
+  <xacro:kuka_agilus_ros2_control name="$(arg prefix)kr6_r700_sixx" driver_version="$(arg driver_version)" client_ip="$(arg client_ip)" client_port="$(arg client_port)" mxa_client_port="$(arg mxa_client_port)" controller_ip="$(arg controller_ip)" prefix="$(arg prefix)" mode="$(arg mode)" gpio_config="$(arg gpio_config)" roundtrip_time="$(arg roundtrip_time)" verify_robot_model="$(arg verify_robot_model)" rsi_xml_config_file="$(arg rsi_xml_config_file)">
     <ext_axes_ros2_control_joints/>
   </xacro:kuka_agilus_ros2_control>

File: kuka_agilus_support/urdf/kr6_r900_2.urdf.xacro (robot description, xacro)
@@ -7,5 +7,5 @@
   <xacro:arg name="driver_version" default="rsi_only"/>
   <xacro:arg name="mode" default="hardware"/>
-  <xacro:arg name="use_gpio" default="false"/>
+  <xacro:arg name="gpio_config" default=""/>
   <xacro:arg name="roundtrip_time" default="0"/>
   <xacro:arg name="client_ip" default="0.0.0.0"/>
@@ -22,5 +22,5 @@
   <xacro:arg name="yaw" default="0"/>
   <xacro:arg name="rsi_xml_config_file" default=""/>
-  <xacro:kuka_agilus_ros2_control name="$(arg prefix)kr6_r900_2" driver_version="$(arg driver_version)" client_ip="$(arg client_ip)" client_port="$(arg client_port)" mxa_client_port="$(arg mxa_client_port)" controller_ip="$(arg controller_ip)" prefix="$(arg prefix)" mode="$(arg mode)" use_gpio="$(arg use_gpio)" roundtrip_time="$(arg roundtrip_time)" verify_robot_model="$(arg verify_robot_model)" rsi_xml_config_file="$(arg rsi_xml_config_file)">
+  <xacro:kuka_agilus_ros2_control name="$(arg prefix)kr6_r900_2" driver_version="$(arg driver_version)" client_ip="$(arg client_ip)" client_port="$(arg client_port)" mxa_client_port="$(arg mxa_client_port)" controller_ip="$(arg controller_ip)" prefix="$(arg prefix)" mode="$(arg mode)" gpio_config="$(arg gpio_config)" roundtrip_time="$(arg roundtrip_time)" verify_robot_model="$(arg verify_robot_model)" rsi_xml_config_file="$(arg rsi_xml_config_file)">
     <ext_axes_ros2_control_joints/>
   </xacro:kuka_agilus_ros2_control>

File: kuka_agilus_support/urdf/kr6_r900_sixx.urdf.xacro (robot description, xacro)
@@ -7,5 +7,5 @@
   <xacro:arg name="driver_version" default="rsi_only"/>
   <xacro:arg name="mode" default="hardware"/>
-  <xacro:arg name="use_gpio" default="false"/>
+  <xacro:arg name="gpio_config" default=""/>
   <xacro:arg name="roundtrip_time" default="0"/>
   <xacro:arg name="client_ip" default="0.0.0.0"/>
@@ -22,5 +22,5 @@
   <xacro:arg name="yaw" default="0"/>
   <xacro:arg name="rsi_xml_config_file" default=""/>
-  <xacro:kuka_agilus_ros2_control name="$(arg prefix)kr6_r900_sixx" driver_version="$(arg driver_version)" client_ip="$(arg client_ip)" client_port="$(arg client_port)" mxa_client_port="$(arg mxa_client_port)" controller_ip="$(arg controller_ip)" prefix="$(arg prefix)" mode="$(arg mode)" use_gpio="$(arg use_gpio)" roundtrip_time="$(arg roundtrip_time)" verify_robot_model="$(arg verify_robot_model)" rsi_xml_config_file="$(arg rsi_xml_config_file)">
+  <xacro:kuka_agilus_ros2_control name="$(arg prefix)kr6_r900_sixx" driver_version="$(arg driver_version)" client_ip="$(arg client_ip)" client_port="$(arg client_port)" mxa_client_port="$(arg mxa_client_port)" controller_ip="$(arg controller_ip)" prefix="$(arg prefix)" mode="$(arg mode)" gpio_config="$(arg gpio_config)" roundtrip_time="$(arg roundtrip_time)" verify_robot_model="$(arg verify_robot_model)" rsi_xml_config_file="$(arg rsi_xml_config_file)">
     <ext_axes_ros2_control_joints/>
   </xacro:kuka_agilus_ros2_control>

File: kuka_agilus_support/urdf/kr7_r900_3.urdf.xacro (robot description, xacro)
@@ -16,5 +16,5 @@
   <xacro:arg name="driver_version" default="rsi_only"/>
   <xacro:arg name="mode" default="hardware"/>
-  <xacro:arg name="use_gpio" default="false"/>
+  <xacro:arg name="gpio_config" default=""/>
   <xacro:arg name="roundtrip_time" default="0"/>
   <xacro:arg name="client_ip" default="0.0.0.0"/>
@@ -23,5 +23,5 @@
   <xacro:arg name="controller_ip" default="0.0.0.0"/>
   <xacro:arg name="verify_robot_model" default="true"/>
-  <xacro:kuka_agilus_ros2_control name="$(arg prefix)kr7_r900_3" driver_version="$(arg driver_version)" client_ip="$(arg client_ip)" client_port="$(arg client_port)" mxa_client_port="$(arg mxa_client_port)" controller_ip="$(arg controller_ip)" prefix="$(arg prefix)" mode="$(arg mode)" use_gpio="$(arg use_gpio)" roundtrip_time="$(arg roundtrip_time)" verify_robot_model="$(arg verify_robot_model)" rsi_xml_config_file="$(arg rsi_xml_config_file)">
+  <xacro:kuka_agilus_ros2_control name="$(arg prefix)kr7_r900_3" driver_version="$(arg driver_version)" client_ip="$(arg client_ip)" client_port="$(arg client_port)" mxa_client_port="$(arg mxa_client_port)" controller_ip="$(arg controller_ip)" prefix="$(arg prefix)" mode="$(arg mode)" gpio_config="$(arg gpio_config)" roundtrip_time="$(arg roundtrip_time)" verify_robot_model="$(arg verify_robot_model)" rsi_xml_config_file="$(arg rsi_xml_config_file)">
     <ext_axes_ros2_control_joints/>
   </xacro:kuka_agilus_ros2_control>

File: kuka_agilus_support/urdf/kr_agilus_ros2_control_macro.xacro (robot description, xacro)
@@ -1,5 +1,5 @@
 <?xml version="1.0" encoding="UTF-8"?>
 <robot xmlns:xacro="http://www.ros.org/wiki/xacro">
-  <xacro:macro name="kuka_agilus_ros2_control" params="name driver_version client_ip client_port mxa_client_port controller_ip prefix mode use_gpio roundtrip_time verify_robot_model rsi_xml_config_file gazebo_controller_config_path:=config/fake_hardware_config_6_axis.yaml **ext_axes_ros2_control_joints">
+  <xacro:macro name="kuka_agilus_ros2_control" params="name driver_version client_ip client_port mxa_client_port controller_ip prefix mode roundtrip_time verify_robot_model rsi_xml_config_file gazebo_controller_config_path:=config/fake_hardware_config_6_axis.yaml gpio_config:='' **ext_axes_ros2_control_joints">
     <!-- gazebo -->
     <xacro:if value="${mode == 'gazebo'}">
@@ -144,11 +144,11 @@
         </xacro:unless>
       </joint>
-      <xacro:if value="${use_gpio}">
-        <xacro:include filename="$(find kuka_rsi_driver)/config/gpio_config.xacro"/>
+      <xacro:unless value="${gpio_config == ''}">
+        <xacro:include filename="${gpio_config}"/>
         <xacro:gpio_config/>
+      </xacro:unless>
+      <xacro:if value="${gpio_config == ''}">
+        <gpio name="gpio"/>
       </xacro:if>
-      <xacro:unless value="${use_gpio}">
-        <gpio name="gpio"/>
-      </xacro:unless>
     </ros2_control>
   </xacro:macro>
