Commit message: Add robot model for issue #236

File: kuka_agilus_support/urdf/kr6_r900_2.urdf.xacro (robot description, xacro)
@@ -1,17 +1,8 @@
 <?xml version="1.0" encoding="UTF-8"?>
-<robot xmlns:xacro="http://ros.org/wiki/xacro" name="kr6_r900_2">
-  <!-- Import macro files  -->
+<robot xmlns:xacro="http://www.ros.org/wiki/xacro" name="kr6_r900_2">
+  <!-- Import urdf files  -->
   <xacro:include filename="$(find kuka_agilus_support)/urdf/kr6_r900_2_macro.xacro"/>
   <xacro:include filename="$(find kuka_agilus_support)/urdf/kr_agilus_ros2_control_macro.xacro"/>
-  <!-- Read additional arguments  -->
-  <xacro:arg name="driver_version" default="rsi_only"/>
-  <xacro:arg name="mode" default="hardware"/>
-  <xacro:arg name="use_gpio" default="false"/>
-  <xacro:arg name="roundtrip_time" default="0"/>
-  <xacro:arg name="client_ip" default="0.0.0.0"/>
-  <xacro:arg name="client_port" default="59152"/>
-  <xacro:arg name="mxa_client_port" default="1337"/>
-  <xacro:arg name="controller_ip" default="0.0.0.0"/>
-  <xacro:arg name="verify_robot_model" default="true"/>
+  <!-- Basic arguments  -->
   <xacro:arg name="prefix" default=""/>
   <xacro:arg name="is_async" default="false"/>
@@ -24,4 +15,14 @@
   <xacro:arg name="pitch" default="0"/>
   <xacro:arg name="yaw" default="0"/>
+  <!-- kroshu-specific arguments -->
+  <xacro:arg name="driver_version" default="rsi_only"/>
+  <xacro:arg name="mode" default="hardware"/>
+  <xacro:arg name="use_gpio" default="false"/>
+  <xacro:arg name="roundtrip_time" default="0"/>
+  <xacro:arg name="client_ip" default="0.0.0.0"/>
+  <xacro:arg name="client_port" default="59152"/>
+  <xacro:arg name="mxa_client_port" default="1337"/>
+  <xacro:arg name="controller_ip" default="0.0.0.0"/>
+  <xacro:arg name="verify_robot_model" default="true"/>
   <xacro:arg name="rsi_xml_config_file" default=""/>
   <xacro:kuka_agilus_ros2_control name="$(arg prefix)kr6_r900_2" driver_version="$(arg driver_version)" client_ip="$(arg client_ip)" client_port="$(arg client_port)" mxa_client_port="$(arg mxa_client_port)" controller_ip="$(arg controller_ip)" prefix="$(arg prefix)" mode="$(arg mode)" use_gpio="$(arg use_gpio)" roundtrip_time="$(arg roundtrip_time)" verify_robot_model="$(arg verify_robot_model)" rsi_xml_config_file="$(arg rsi_xml_config_file)" is_async="$(arg is_async)" async_thread_priority="$(arg async_thread_priority)" async_affinity="$(arg async_affinity)">

File: kuka_agilus_support/urdf/kr6_r900_2_macro.xacro (robot description, xacro)
@@ -8,10 +8,10 @@
           <mesh filename="package://${package_name}/meshes/kr6_r900_2/collision/base_link.stl"/>
         </geometry>
-        <origin rpy="0.0 -0.0 0.0" xyz="0.0 0.0 0.0"/>
+        <origin rpy="0.0 0.0 0.0" xyz="0.0 0.0 0.0"/>
       </collision>
       <inertial>
-        <inertia ixx="0.16209200415615" ixy="0.0" ixz="0.0" iyy="0.10881181598555635" iyz="0.0" izz="0.18461591505869543"/>
-        <mass value="1.6916E1"/>
-        <origin rpy="1.6165592773339865 -1.221289277333065 3.10031147437779" xyz="-0.03713348309292976 2.6602033577676952E-5 0.10863850792149446"/>
+        <inertia ixx="0.1621" ixy="0.0" ixz="0.0" iyy="0.1088" iyz="0.0" izz="0.1846"/>
+        <mass value="16.916"/>
+        <origin rpy="1.6166 -1.2213 3.1003" xyz="-0.0371 0.0 0.1086"/>
       </inertial>
       <visual>
@@ -19,5 +19,5 @@
           <mesh filename="package://${package_name}/meshes/kr6_r900_2/visual/base_link.dae"/>
         </geometry>
-        <origin rpy="0.0 -0.0 0.0" xyz="0.0 0.0 0.0"/>
+        <origin rpy="0.0 0.0 0.0" xyz="0.0 0.0 0.0"/>
       </visual>
     </link>
@@ -28,10 +28,10 @@
           <mesh filename="package://${package_name}/meshes/kr6_r900_2/collision/link_1.stl"/>
         </geometry>
-        <origin rpy="-3.141592653589793 0.0 -0.0" xyz="0.0 -2.547265342226495e-17 0.20800000000000002"/>
+        <origin rpy="-3.1415853071795867 0.0 -0.0" xyz="0.0 -1.528053322981866e-06 0.20799999999438715"/>
       </collision>
       <inertial>
-        <inertia ixx="0.07406183855390855" ixy="0.0" ixz="0.0" iyy="0.0890478351825312" iyz="0.0" izz="0.11039570662759429"/>
-        <mass value="8.4159999999999986E0"/>
-        <origin rpy="1.304519343134156 -0.9428616016893947 -1.4226510948637578" xyz="0.006410408745247152 -0.01626805370722434 -0.10658893773764262"/>
+        <inertia ixx="0.0741" ixy="0.0" ixz="0.0" iyy="0.089" iyz="0.0" izz="0.1104"/>
+        <mass value="8.416"/>
+        <origin rpy="1.3045 -0.9429 -1.4227" xyz="0.0064 -0.0163 -0.1066"/>
       </inertial>
       <visual>
@@ -39,5 +39,5 @@
           <mesh filename="package://${package_name}/meshes/kr6_r900_2/visual/link_1.dae"/>
         </geometry>
-        <origin rpy="-3.141592653589793 0.0 -0.0" xyz="0.0 -2.547265342226495e-17 0.20800000000000002"/>
+        <origin rpy="-3.1415853071795867 0.0 -0.0" xyz="0.0 -1.528053322981866e-06 0.20799999999438715"/>
       </visual>
     </link>
@@ -47,10 +47,10 @@
           <mesh filename="package://${package_name}/meshes/kr6_r900_2/collision/link_2.stl"/>
         </geometry>
-        <origin rpy="1.5707963267948968 -0.0 1.5707963267948966" xyz="-0.4 -0.024999999999999977 -0.09069999999999996"/>
+        <origin rpy="1.5708 4.70197740325743e-38 1.5707963267948966" xyz="-0.39999966683759874 -0.024999999999999977 -0.09069994122810648"/>
       </collision>
       <inertial>
-        <inertia ixx="0.548306118225302" ixy="0.0" ixz="0.0" iyy="0.0872309454394033" iyz="0.0" izz="0.5885170960694246"/>
-        <mass value="1.67929E1"/>
-        <origin rpy="1.8410866125641745 -1.5373992728262285 -0.2834226607733986" xyz="0.14741713998177805 -0.004477319760136727 -0.07370278248545517"/>
+        <inertia ixx="0.5483" ixy="0.0" ixz="0.0" iyy="0.0872" iyz="0.0" izz="0.5885"/>
+        <mass value="16.7929"/>
+        <origin rpy="1.8411 -1.5374 -0.2834" xyz="0.1474 -0.0045 -0.0737"/>
       </inertial>
       <visual>
@@ -58,5 +58,5 @@
           <mesh filename="package://${package_name}/meshes/kr6_r900_2/visual/link_2.dae"/>
         </geometry>
-        <origin rpy="1.5707963267948968 -0.0 1.5707963267948966" xyz="-0.4 -0.024999999999999977 -0.09069999999999996"/>
+        <origin rpy="1.5708 4.70197740325743e-38 1.5707963267948966" xyz="-0.39999966683759874 -0.024999999999999977 -0.09069994122810648"/>
       </visual>
     </link>
@@ -66,10 +66,10 @@
           <mesh filename="package://${package_name}/meshes/kr6_r900_2/collision/link_3.stl"/>
         </geometry>
-        <origin rpy="1.5707963267948968 -0.0 -0.0" xyz="-0.02500000000000003 0.855 -0.08649999999999997"/>
+        <origin rpy="1.5708 -0.0 -0.0" xyz="-0.02500000000000003 0.8549996668375988 -0.08649994122810648"/>
       </collision>
       <inertial>
-        <inertia ixx="0.04261164351414989" ixy="0.0" ixz="0.0" iyy="0.01892041629125804" iyz="0.0" izz="0.04780021844065417"/>
-        <mass value="5.988E0"/>
-        <origin rpy="-2.675092481056456 -1.3258514256524945 1.194666577454412" xyz="0.04165063460253841 -0.012325484301937206 -0.06798628924515698"/>
+        <inertia ixx="0.0426" ixy="0.0" ixz="0.0" iyy="0.0189" iyz="0.0" izz="0.0478"/>
+        <mass value="5.988"/>
+        <origin rpy="-2.6751 -1.3259 1.1947" xyz="0.0417 -0.0123 -0.068"/>
       </inertial>
       <visual>
@@ -77,5 +77,5 @@
           <mesh filename="package://${package_name}/meshes/kr6_r900_2/visual/link_3.dae"/>
         </geometry>
-        <origin rpy="1.5707963267948968 -0.0 -0.0" xyz="-0.02500000000000003 0.855 -0.08649999999999997"/>
+        <origin rpy="1.5708 -0.0 -0.0" xyz="-0.02500000000000003 0.8549996668375988 -0.08649994122810648"/>
       </visual>
     </link>
@@ -85,10 +85,10 @@
           <mesh filename="package://${package_name}/meshes/kr6_r900_2/collision/link_4.stl"/>
         </geometry>
-        <origin rpy="1.8369701987210297e-16 1.5707963267948966 0.0" xyz="-0.8800000000000001 3.806918983854133e-17 0.22099999999999997"/>
+        <origin rpy="-2.3561908169838683 1.570791132098422 -2.356194490195718" xyz="-0.8799988550533341 8.705620946852126e-07 0.2210032324160695"/>
       </collision>
       <inertial>
-        <inertia ixx="0.010489707545547112" ixy="0.0" ixz="0.0" iyy="0.04423898136862264" iyz="0.0" izz="0.04721253436329341"/>
-        <mass value="4.69985262E0"/>
-        <origin rpy="-2.330109287924748 -1.5210980103983611 2.285952535622045" xyz="0.0014479693417065146 0.009426192930537397 -0.08164304521000952"/>
+        <inertia ixx="0.0105" ixy="0.0" ixz="0.0" iyy="0.0442" iyz="0.0" izz="0.0472"/>
+        <mass value="4.6999"/>
+        <origin rpy="-2.3301 -1.5211 2.286" xyz="0.0014 0.0094 -0.0816"/>
       </inertial>
       <visual>
@@ -96,5 +96,5 @@
           <mesh filename="package://${package_name}/meshes/kr6_r900_2/visual/link_4.dae"/>
         </geometry>
-        <origin rpy="1.8369701987210297e-16 1.5707963267948966 0.0" xyz="-0.8800000000000001 3.806918983854133e-17 0.22099999999999997"/>
+        <origin rpy="-2.3561908169838683 1.570791132098422 -2.356194490195718" xyz="-0.8799988550533341 8.705620946852126e-07 0.2210032324160695"/>
       </visual>
     </link>
@@ -104,10 +104,10 @@
           <mesh filename="package://${package_name}/meshes/kr6_r900_2/collision/link_5.stl"/>
         </geometry>
-        <origin rpy="1.5707963267948968 -3.749399456654644e-33 -6.123233995736766e-17" xyz="-0.44500000000000006 0.8800000000000001 -0.05049999999999998"/>
+        <origin rpy="1.5708036732051034 -1.3492460511333462e-11 3.673218595765785e-06" xyz="-0.44500304693128084 0.8799990405410575 -0.05049753160908297"/>
       </collision>
       <inertial>
-        <inertia ixx="0.0017317756133102904" ixy="0.0" ixz="0.0" iyy="0.002219500805440681" iyz="0.0" izz="0.002467090055442975"/>
-        <mass value="1.6128E0"/>
-        <origin rpy="1.567898714902774 -0.8611716764868309 -3.100280255900493" xyz="0.009320696924603175 7.83482142857143E-4 -0.026462549603174602"/>
+        <inertia ixx="0.0017" ixy="0.0" ixz="0.0" iyy="0.0022" iyz="0.0" izz="0.0025"/>
+        <mass value="1.6128"/>
+        <origin rpy="1.5679 -0.8612 -3.1003" xyz="0.0093 0.0008 -0.0265"/>
       </inertial>
       <visual>
@@ -115,5 +115,5 @@
           <mesh filename="package://${package_name}/meshes/kr6_r900_2/visual/link_5.dae"/>
         </geometry>
-        <origin rpy="1.5707963267948968 -3.749399456654644e-33 -6.123233995736766e-17" xyz="-0.44500000000000006 0.8800000000000001 -0.05049999999999998"/>
+        <origin rpy="1.5708036732051034 -1.3492460511333462e-11 3.673218595765785e-06" xyz="-0.44500304693128084 0.8799990405410575 -0.05049753160908297"/>
       </visual>
     </link>
@@ -123,10 +123,10 @@
           <mesh filename="package://${package_name}/meshes/kr6_r900_2/collision/link_6.stl"/>
         </geometry>
-        <origin rpy="1.2246467991473532e-16 1.5707963267948966 0.0" xyz="-0.88 -1.941931457395624e-17 0.5065"/>
+        <origin rpy="-2.6779399020961754 1.5707881132525563 -2.6779472485198745" xyz="-0.879997180045544 4.3288923671780846e-06 0.5065062793323466"/>
       </collision>
       <inertial>
-        <inertia ixx="1.83698267603013E-4" ixy="0.0" ixz="0.0" iyy="1.8213621766783165E-4" iyz="0.0" izz="2.9589000000000004E-4"/>
-        <mass value="7.34E-1"/>
-        <origin rpy="0.0 -0.0 1.223427188696551" xyz="0.0 0.0 -0.011764604904632152"/>
+        <inertia ixx="0.0002" ixy="0.0" ixz="0.0" iyy="0.0002" iyz="0.0" izz="0.0003"/>
+        <mass value="0.734"/>
+        <origin rpy="0.0 0.0 1.2234" xyz="0.0 0.0 -0.0118"/>
       </inertial>
       <visual>
@@ -134,5 +134,5 @@
           <mesh filename="package://${package_name}/meshes/kr6_r900_2/visual/link_6.dae"/>
         </geometry>
-        <origin rpy="1.2246467991473532e-16 1.5707963267948966 0.0" xyz="-0.88 -1.941931457395624e-17 0.5065"/>
+        <origin rpy="-2.6779399020961754 1.5707881132525563 -2.6779472485198745" xyz="-0.879997180045544 4.3288923671780846e-06 0.5065062793323466"/>
       </visual>
     </link>
@@ -140,4 +140,5 @@
     <joint name="${prefix}base_link-base" type="fixed">
       <child link="${prefix}base"/>
+      <origin rpy="0.0 0.0 0.0" xyz="0.0 0.0 0.0"/>
       <parent link="${prefix}base_link"/>
     </joint>
@@ -145,6 +146,6 @@
       <axis xyz="0.0 0.0 1.0"/>
       <child link="${prefix}link_1"/>
-      <limit effort="3.3480000000000007E2" lower="-2.967059725E0" upper="2.967059725E0" velocity="6.2831853071795862E0"/>
-      <origin rpy="3.141592653589793 -0.0 0.0" xyz="0.0 0.0 0.20800000000000002"/>
+      <limit effort="334.8" lower="-2.9671" upper="2.9671" velocity="6.2832"/>
+      <origin rpy="-3.1416 0.0 0.0" xyz="0.0 0.0 0.208"/>
       <parent link="${prefix}base_link"/>
     </joint>
@@ -152,6 +153,6 @@
       <axis xyz="0.0 0.0 1.0"/>
       <child link="${prefix}link_2"/>
-      <limit effort="2.6065652967616722E2" lower="-3.316125575E0" upper="7.853981625E-1" velocity="5.2359877559829888E0"/>
-      <origin rpy="1.5707963267948966 -0.0 0.0" xyz="0.025 -0.0907 -0.192"/>
+      <limit effort="260.6565" lower="-3.3161" upper="0.7854" velocity="5.236"/>
+      <origin rpy="1.5708 0.0 0.0" xyz="0.025 -0.0907 -0.192"/>
       <parent link="${prefix}link_1"/>
     </joint>
@@ -159,6 +160,6 @@
       <axis xyz="0.0 0.0 1.0"/>
       <child link="${prefix}link_3"/>
-      <limit effort="1.3782737531209466E2" lower="-2.0943951E0" upper="2.72271363E0" velocity="6.2831853071795862E0"/>
-      <origin rpy="0.0 -0.0 0.0" xyz="0.455 0.0 -0.004200000000000001"/>
+      <limit effort="137.8274" lower="-2.0944" upper="2.7227" velocity="6.2832"/>
+      <origin rpy="0.0 0.0 0.0" xyz="0.455 0.0 -0.0042"/>
       <parent link="${prefix}link_2"/>
     </joint>
@@ -166,6 +167,6 @@
       <axis xyz="0.0 0.0 1.0"/>
       <child link="${prefix}link_4"/>
-      <limit effort="4.3282069018283245E1" lower="-3.2288591125E0" upper="3.2288591125E0" velocity="7.8539816339744828E0"/>
-      <origin rpy="1.5707963267948966 -0.0 -1.5707963267948966" xyz="0.196 -0.025 -0.08650000000000001"/>
+      <limit effort="43.2821" lower="-3.2289" upper="3.2289" velocity="7.854"/>
+      <origin rpy="1.5708 0.0 -1.5708" xyz="0.196 -0.025 -0.0865"/>
       <parent link="${prefix}link_3"/>
     </joint>
@@ -173,6 +174,6 @@
       <axis xyz="0.0 0.0 1.0"/>
       <child link="${prefix}link_5"/>
-      <limit effort="4.5669606843995879E1" lower="-2.0943951E0" upper="2.0943951E0" velocity="7.8539816339744828E0"/>
-      <origin rpy="0.0 1.5707963267948966 1.5707963267948966" xyz="0.0 0.0505 -0.224"/>
+      <limit effort="45.6696" lower="-2.0944" upper="2.0944" velocity="7.854"/>
+      <origin rpy="0.0 1.5708 1.5708" xyz="0.0 0.0505 -0.224"/>
       <parent link="${prefix}link_4"/>
     </joint>
@@ -180,16 +181,16 @@
       <axis xyz="0.0 0.0 1.0"/>
       <child link="${prefix}link_6"/>
-      <limit effort="2.32939212E1" lower="-6.108652375E0" upper="6.108652375E0" velocity="9.42477796076938E0"/>
-      <origin rpy="1.5707963267948966 -0.0 -1.5707963267948966" xyz="0.0615 0.0 -0.0505"/>
+      <limit effort="23.2939" lower="-6.1087" upper="6.1087" velocity="9.4248"/>
+      <origin rpy="1.5708 0.0 -1.5708" xyz="0.0615 0.0 -0.0505"/>
       <parent link="${prefix}link_5"/>
     </joint>
-    <joint name="${prefix}link6-flange" type="fixed">
+    <joint name="${prefix}link_6-flange" type="fixed">
       <child link="${prefix}flange"/>
-      <origin rpy="0.0 1.5707963267948966 0.0" xyz="0.0 0.0 -0.0285"/>
+      <origin rpy="0.0 1.5708 0.0" xyz="0.0 0.0 -0.0285"/>
       <parent link="${prefix}link_6"/>
     </joint>
-    <joint name="${prefix}link6-tool0" type="fixed">
+    <joint name="${prefix}link_6-tool0" type="fixed">
       <child link="${prefix}tool0"/>
-      <origin rpy="3.141592653589793 1.2246467991473532E-16 3.141592653589793" xyz="0.0 0.0 -0.0285"/>
+      <origin rpy="3.1416 -0.0 3.1416" xyz="0.0 0.0 -0.0285"/>
       <parent link="${prefix}link_6"/>
     </joint>
