Commit message: fix

File: kuka_quantec_support/urdf/kr210_r2700-2_macro.xacro (robot description, xacro)
@@ -15,5 +15,5 @@
       <collision>
         <geometry>
-          <mesh filename="package://kr210_r2700-2/meshes/collision/base_link.stl"/>
+          <mesh filename="package://kuka_quantec_support/meshes/kr210_r2700-2/collision/base_link.stl"/>
         </geometry>
         <origin rpy="-0.0 0.0 -0.0" xyz="0.0 0.0 0.0"/>
@@ -26,5 +26,5 @@
       <visual>
         <geometry>
-          <mesh filename="package://kr210_r2700-2/meshes/visual/base_link.stl"/>
+          <mesh filename="package://kuka_quantec_support/meshes/kr210_r2700-2/visual/base_link.stl"/>
         </geometry>
         <origin rpy="-0.0 0.0 -0.0" xyz="0.0 0.0 0.0"/>
@@ -34,5 +34,5 @@
       <collision>
         <geometry>
-          <mesh filename="package://kr210_r2700-2/meshes/collision/link_1.stl"/>
+          <mesh filename="package://kuka_quantec_support/meshes/kr210_r2700-2/collision/link_1.stl"/>
         </geometry>
         <origin rpy="-0.0 0.0 -0.0" xyz="0.0 0.0 0.0"/>
@@ -45,5 +45,5 @@
       <visual>
         <geometry>
-          <mesh filename="package://kr210_r2700-2/meshes/visual/link_1.stl"/>
+          <mesh filename="package://kuka_quantec_support/meshes/kr210_r2700-2/visual/link_1.stl"/>
         </geometry>
         <origin rpy="-0.0 0.0 -0.0" xyz="0.0 0.0 0.0"/>
@@ -53,5 +53,5 @@
       <collision>
         <geometry>
-          <mesh filename="package://kr210_r2700-2/meshes/collision/link_2.stl"/>
+          <mesh filename="package://kuka_quantec_support/meshes/kr210_r2700-2/collision/link_2.stl"/>
         </geometry>
         <origin rpy="-0.0 0.0 -0.0" xyz="0.0 0.0 0.0"/>
@@ -64,5 +64,5 @@
       <visual>
         <geometry>
-          <mesh filename="package://kr210_r2700-2/meshes/visual/link_2.stl"/>
+          <mesh filename="package://kuka_quantec_support/meshes/kr210_r2700-2/visual/link_2.stl"/>
         </geometry>
         <origin rpy="-0.0 0.0 -0.0" xyz="0.0 0.0 0.0"/>
@@ -72,5 +72,5 @@
       <collision>
         <geometry>
-          <mesh filename="package://kr210_r2700-2/meshes/collision/link_3.stl"/>
+          <mesh filename="package://kuka_quantec_support/meshes/kr210_r2700-2/collision/link_3.stl"/>
         </geometry>
         <origin rpy="-0.0 0.0 -0.0" xyz="0.0 0.0 0.0"/>
@@ -83,5 +83,5 @@
       <visual>
         <geometry>
-          <mesh filename="package://kr210_r2700-2/meshes/visual/link_3.stl"/>
+          <mesh filename="package://kuka_quantec_support/meshes/kr210_r2700-2/visual/link_3.stl"/>
         </geometry>
         <origin rpy="-0.0 0.0 -0.0" xyz="0.0 0.0 0.0"/>
@@ -91,5 +91,5 @@
       <collision>
         <geometry>
-          <mesh filename="package://kr210_r2700-2/meshes/collision/link_4.stl"/>
+          <mesh filename="package://kuka_quantec_support/meshes/kr210_r2700-2/collision/link_4.stl"/>
         </geometry>
         <origin rpy="-0.0 0.0 -0.0" xyz="0.0 0.0 0.0"/>
@@ -102,5 +102,5 @@
       <visual>
         <geometry>
-          <mesh filename="package://kr210_r2700-2/meshes/visual/link_4.stl"/>
+          <mesh filename="package://kuka_quantec_support/meshes/kr210_r2700-2/visual/link_4.stl"/>
         </geometry>
         <origin rpy="-0.0 0.0 -0.0" xyz="0.0 0.0 0.0"/>
@@ -110,5 +110,5 @@
       <collision>
         <geometry>
-          <mesh filename="package://kr210_r2700-2/meshes/collision/link_5.stl"/>
+          <mesh filename="package://kuka_quantec_support/meshes/kr210_r2700-2/collision/link_5.stl"/>
         </geometry>
         <origin rpy="-0.0 0.0 -0.0" xyz="0.0 0.0 0.0"/>
@@ -121,5 +121,5 @@
       <visual>
         <geometry>
-          <mesh filename="package://kr210_r2700-2/meshes/visual/link_5.stl"/>
+          <mesh filename="package://kuka_quantec_support/meshes/kr210_r2700-2/visual/link_5.stl"/>
         </geometry>
         <origin rpy="-0.0 0.0 -0.0" xyz="0.0 0.0 0.0"/>
@@ -129,5 +129,5 @@
       <collision>
         <geometry>
-          <mesh filename="package://kr210_r2700-2/meshes/collision/link_6.stl"/>
+          <mesh filename="package://kuka_quantec_support/meshes/kr210_r2700-2/collision/link_6.stl"/>
         </geometry>
         <origin rpy="-0.0 0.0 -0.0" xyz="0.0 0.0 0.0"/>
@@ -136,137 +136,4 @@
         <inertia ixx="0.03694113" ixy="0.0" ixz="0.0" iyy="0.03695315" iyz="0.0" izz="0.048251"/>
         <mass value="6.6E0"/>
-        <origin rpy="-0.0 0.0 -0.0" xyz="0.0 0.0 0.0"/>
-      </inertial>
-      <visual>
-        <geometry>
-          <mesh filename="package://kr210_r2700-2/meshes/visual/link_6.stl"/>
-        </geometry>
-        <origin rpy="-0.0 0.0 -0.0" xyz="0.0 0.0 0.0"/>
-      </visual>
-    </link>
-    <link name="${prefix}base_link_inertia">
-      <collision>
-        <geometry>
-          <mesh filename="package://kuka_quantec_support/meshes/kr210_r2700-2/collision/base_link.stl"/>
-        </geometry>
-        <origin rpy="-0.0 0.0 -0.0" xyz="0.0 0.0 0.0"/>
-      </collision>
-      <inertial>
-        <inertia ixx="0.0" ixy="0.0" ixz="0.0" iyy="0.0" iyz="0.0" izz="0.0"/>
-        <mass value="6.5212E1"/>
-        <origin rpy="-0.0 0.0 -0.0" xyz="0.0 0.0 0.0"/>
-      </inertial>
-      <visual>
-        <geometry>
-          <mesh filename="package://kuka_quantec_support/meshes/kr210_r2700-2/visual/base_link.stl"/>
-        </geometry>
-        <origin rpy="-0.0 0.0 -0.0" xyz="0.0 0.0 0.0"/>
-      </visual>
-    </link>
-    <link name="${prefix}link_1">
-      <collision>
-        <geometry>
-          <mesh filename="package://kuka_quantec_support/meshes/kr210_r2700-2/collision/link_1.stl"/>
-        </geometry>
-        <origin rpy="-0.0 0.0 -0.0" xyz="0.0 0.0 0.0"/>
-      </collision>
-      <inertial>
-        <inertia ixx="9.85967888" ixy="0.0" ixz="0.0" iyy="0.91499458" iyz="0.0" izz="10.23026596"/>
-        <mass value="8.4207E1"/>
-        <origin rpy="-0.0 0.0 -0.0" xyz="0.0 0.0 0.0"/>
-      </inertial>
-      <visual>
-        <geometry>
-          <mesh filename="package://kuka_quantec_support/meshes/kr210_r2700-2/visual/link_1.stl"/>
-        </geometry>
-        <origin rpy="-0.0 0.0 -0.0" xyz="0.0 0.0 0.0"/>
-      </visual>
-    </link>
-    <link name="${prefix}link_2">
-      <collision>
-        <geometry>
-          <mesh filename="package://kuka_quantec_support/meshes/kr210_r2700-2/collision/link_2.stl"/>
-        </geometry>
-        <origin rpy="-0.0 0.0 -0.0" xyz="0.0 0.0 0.0"/>
-      </collision>
-      <inertial>
-        <inertia ixx="0.34836069" ixy="0.0" ixz="0.0" iyy="1.0268737" iyz="0.0" izz="1.13887402"/>
-        <mass value="6.1775E1"/>
-        <origin rpy="-0.0 0.0 -0.0" xyz="0.0 0.0 0.0"/>
-      </inertial>
-      <visual>
-        <geometry>
-          <mesh filename="package://kuka_quantec_support/meshes/kr210_r2700-2/visual/link_2.stl"/>
-        </geometry>
-        <origin rpy="-0.0 0.0 -0.0" xyz="0.0 0.0 0.0"/>
-      </visual>
-    </link>
-    <link name="${prefix}link_3">
-      <collision>
-        <geometry>
-          <mesh filename="package://kuka_quantec_support/meshes/kr210_r2700-2/collision/link_3.stl"/>
-        </geometry>
-        <origin rpy="-0.0 0.0 -0.0" xyz="0.0 0.0 0.0"/>
-      </collision>
-      <inertial>
-        <inertia ixx="0.64549911" ixy="0.0" ixz="0.0" iyy="0.04236472" iyz="0.0" izz="0.6665241"/>
-        <mass value="3.5648E1"/>
-        <origin rpy="-0.0 0.0 -0.0" xyz="0.0 0.0 0.0"/>
-      </inertial>
-      <visual>
-        <geometry>
-          <mesh filename="package://kuka_quantec_support/meshes/kr210_r2700-2/visual/link_3.stl"/>
-        </geometry>
-        <origin rpy="-0.0 0.0 -0.0" xyz="0.0 0.0 0.0"/>
-      </visual>
-    </link>
-    <link name="${prefix}link_4">
-      <collision>
-        <geometry>
-          <mesh filename="package://kuka_quantec_support/meshes/kr210_r2700-2/collision/link_4.stl"/>
-        </geometry>
-        <origin rpy="-0.0 0.0 -0.0" xyz="0.0 0.0 0.0"/>
-      </collision>
-      <inertial>
-        <inertia ixx="0.64549911" ixy="0.0" ixz="0.0" iyy="0.04236472" iyz="0.0" izz="0.6665241"/>
-        <mass value="1.6428E1"/>
-        <origin rpy="-0.0 0.0 -0.0" xyz="0.0 0.0 0.0"/>
-      </inertial>
-      <visual>
-        <geometry>
-          <mesh filename="package://kuka_quantec_support/meshes/kr210_r2700-2/visual/link_4.stl"/>
-        </geometry>
-        <origin rpy="-0.0 0.0 -0.0" xyz="0.0 0.0 0.0"/>
-      </visual>
-    </link>
-    <link name="${prefix}link_5">
-      <collision>
-        <geometry>
-          <mesh filename="package://kuka_quantec_support/meshes/kr210_r2700-2/collision/link_5.stl"/>
-        </geometry>
-        <origin rpy="-0.0 0.0 -0.0" xyz="0.0 0.0 0.0"/>
-      </collision>
-      <inertial>
-        <inertia ixx="1.0E-8" ixy="0.0" ixz="0.0" iyy="1.0E-8" iyz="0.0" izz="1.0E-8"/>
-        <mass value="1.0E-6"/>
-        <origin rpy="-0.0 0.0 -0.0" xyz="0.0 0.0 0.0"/>
-      </inertial>
-      <visual>
-        <geometry>
-          <mesh filename="package://kuka_quantec_support/meshes/kr210_r2700-2/visual/link_5.stl"/>
-        </geometry>
-        <origin rpy="-0.0 0.0 -0.0" xyz="0.0 0.0 0.0"/>
-      </visual>
-    </link>
-    <link name="${prefix}link_6">
-      <collision>
-        <geometry>
-          <mesh filename="package://kuka_quantec_support/meshes/kr210_r2700-2/collision/link_6.stl"/>
-        </geometry>
-        <origin rpy="-0.0 0.0 -0.0" xyz="0.0 0.0 0.0"/>
-      </collision>
-      <inertial>
-        <inertia ixx="1.0E-8" ixy="0.0" ixz="0.0" iyy="1.0E-8" iyz="0.0" izz="1.0E-8"/>
-        <mass value="1.0E-6"/>
         <origin rpy="-0.0 0.0 -0.0" xyz="0.0 0.0 0.0"/>
       </inertial>

File: kuka_quantec_support/urdf/kr_quantec_ros2_control.xacro (robot description, xacro)
@@ -1,5 +1,5 @@
 <?xml version="1.0" encoding="UTF-8"?>
 <robot xmlns:xacro="http://www.ros.org/wiki/xacro">
-  <xacro:macro name="kuka_cybertech_ros2_control" params="name prefix client_ip client_port use_fake_hardware:=false">
+  <xacro:macro name="kuka_quantec_ros2_control" params="name prefix client_ip client_port use_fake_hardware:=false">
     <ros2_control name="${name}" type="system">
       <hardware>

File: kuka_quantec_support/urdf/kr_quantec_transmission.xacro (robot description, xacro)
@@ -1,5 +1,5 @@
 <?xml version="1.0" encoding="UTF-8"?>
 <robot xmlns:xacro="http://wiki.ros.org/xacro">
-  <xacro:macro name="kuka_cybertech_transmission" params="prefix">
+  <xacro:macro name="kuka_quantec_transmission" params="prefix">
     <transmission name="${prefix}joint_a1_trans">
       <actuator name="${prefix}joint_a1_motor">

Commit message: link6-flange trafos

File: kuka_quantec_support/urdf/kr210_r2700-2_macro.xacro (robot description, xacro)
@@ -203,5 +203,5 @@
     <joint name="${prefix}link6-flange" type="fixed">
       <child link="${prefix}flange" />
-      <origin rpy="0 ${pi} -0.0" xyz="0.0 0.0 -0.153" />
+      <origin rpy="0 ${pi} -0.0" xyz="0.0 0.0 -0.215" />
       <parent link="${prefix}link_6" />
     </joint>
@@ -210,5 +210,5 @@
     <joint name="${prefix}link6-tool0" type="fixed">
       <child link="${prefix}tool0" />
-      <origin rpy="0 ${pi} -0.0" xyz="0.0 0.0 -0.153" />
+      <origin rpy="0 ${pi} -0.0" xyz="0.0 0.0 -0.215" />
       <parent link="${prefix}link_6" />
     </joint>

File: kuka_quantec_support/urdf/kr210_r3100-2_macro.xacro (robot description, xacro)
@@ -203,5 +203,5 @@
     <joint name="${prefix}link6-flange" type="fixed">
       <child link="${prefix}flange" />
-      <origin rpy="0 ${pi} -0.0" xyz="0.0 0.0 -0.153" />
+      <origin rpy="0 ${pi} -0.0" xyz="0.0 0.0 -0.240" />
       <parent link="${prefix}link_6" />
     </joint>
@@ -210,5 +210,5 @@
     <joint name="${prefix}link6-tool0" type="fixed">
       <child link="${prefix}tool0" />
-      <origin rpy="0 ${pi} -0.0" xyz="0.0 0.0 -0.153" />
+      <origin rpy="0 ${pi} -0.0" xyz="0.0 0.0 -0.240" />
       <parent link="${prefix}link_6" />
     </joint>

Commit message: invalidate vel torque lims

File: kuka_quantec_support/urdf/kr210_r2700-2_macro.xacro (robot description, xacro)
@@ -153,5 +153,5 @@
       <axis xyz="0.0 0.0 1.0"/>
       <child link="${prefix}link_1"/>
-      <limit effort="0" lower="-3.2288591161895095E0" upper="3.2288591161895095E0" velocity="5.501E3"/>
+      <limit effort="0" lower="-3.2288591161895095E0" upper="3.2288591161895095E0" velocity="0"/>
       <origin rpy="-3.141592653589793 0.0 -0.0" xyz="0.0 0.0 0.0"/>
       <parent link="${prefix}base_link_inertia"/>
@@ -160,5 +160,5 @@
       <axis xyz="0.0 0.0 1.0"/>
       <child link="${prefix}link_2"/>
-      <limit effort="0" lower="-2.443460952792061E0" upper="-8.726646259971647E-2" velocity="5.001E3"/>
+      <limit effort="0" lower="-2.443460952792061E0" upper="-8.726646259971647E-2" velocity="0"/>
       <origin rpy="1.5707963267948963 0.0 -0.0" xyz="0.33 0.0 -0.645"/>
       <parent link="${prefix}link_1"/>
@@ -167,5 +167,5 @@
       <axis xyz="0.0 0.0 1.0"/>
       <child link="${prefix}link_3"/>
-      <limit effort="0" lower="-2.0943951023931953E0" upper="2.9321531433504737E0" velocity="5.001E3"/>
+      <limit effort="0" lower="-2.0943951023931953E0" upper="2.9321531433504737E0" velocity="0"/>
       <origin rpy="0.0 0.0 -1.5707963267948963" xyz="1.15 0.0 0.0"/>
       <parent link="${prefix}link_2"/>
@@ -174,5 +174,5 @@
       <axis xyz="0.0 0.0 1.0"/>
       <child link="${prefix}link_4"/>
-      <limit effort="0" lower="-6.1086523819801535E0" upper="6.1086523819801535E0" velocity="6.001E3"/>
+      <limit effort="0" lower="-6.1086523819801535E0" upper="6.1086523819801535E0" velocity="0"/>
       <origin rpy="1.5707963267948963 0.0 -0.0" xyz="0.115 0.0 0.0"/>
       <parent link="${prefix}link_3"/>
@@ -181,5 +181,5 @@
       <axis xyz="0.0 0.0 1.0"/>
       <child link="${prefix}link_5"/>
-      <limit effort="0" lower="-2.181661564992912E0" upper="2.181661564992912E0" velocity="6.001E3"/>
+      <limit effort="0" lower="-2.181661564992912E0" upper="2.181661564992912E0" velocity="0"/>
       <origin rpy="-1.5707963267948963 0.0 -0.0" xyz="0.0 0.0 -1.22"/>
       <parent link="${prefix}link_4"/>
@@ -188,5 +188,5 @@
       <axis xyz="0.0 0.0 1.0"/>
       <child link="${prefix}link_6"/>
-      <limit effort="0" lower="-6.1086523819801535E0" upper="6.1086523819801535E0" velocity="6.001E3"/>
+      <limit effort="0" lower="-6.1086523819801535E0" upper="6.1086523819801535E0" velocity="0"/>
       <origin rpy="1.5707963267948963 0.0 -0.0" xyz="0.0 0.0 0.0"/>
       <parent link="${prefix}link_5"/>

File: kuka_quantec_support/urdf/kr210_r3100-2_macro.xacro (robot description, xacro)
@@ -153,5 +153,5 @@
       <axis xyz="0.0 0.0 1.0"/>
       <child link="${prefix}link_1"/>
-      <limit effort="0" lower="-3.2288591161895095E0" upper="3.2288591161895095E0" velocity="5.001E3"/>
+      <limit effort="0" lower="-3.2288591161895095E0" upper="3.2288591161895095E0" velocity="0"/>
       <origin rpy="-3.141592653589793 0.0 -0.0" xyz="0.0 0.0 0.0"/>
       <parent link="${prefix}base_link_inertia"/>
@@ -160,5 +160,5 @@
       <axis xyz="0.0 0.0 1.0"/>
       <child link="${prefix}link_2"/>
-      <limit effort="0" lower="-2.443460952792061E0" upper="-8.726646259971647E-2" velocity="4.783E3"/>
+      <limit effort="0" lower="-2.443460952792061E0" upper="-8.726646259971647E-2" velocity="0"/>
       <origin rpy="1.5707963267948963 0.0 -0.0" xyz="0.33 0.0 -0.645"/>
       <parent link="${prefix}link_1"/>
@@ -167,5 +167,5 @@
       <axis xyz="0.0 0.0 1.0"/>
       <child link="${prefix}link_3"/>
-      <limit effort="0" lower="-2.0943951023931953E0" upper="2.9321531433504737E0" velocity="4.783E3"/>
+      <limit effort="0" lower="-2.0943951023931953E0" upper="2.9321531433504737E0" velocity="0"/>
       <origin rpy="0.0 0.0 -1.5707963267948963" xyz="1.35 0.0 0.0"/>
       <parent link="${prefix}link_2"/>
@@ -174,5 +174,5 @@
       <axis xyz="0.0 0.0 1.0"/>
       <child link="${prefix}link_4"/>
-      <limit effort="0" lower="-6.1086523819801535E0" upper="6.1086523819801535E0" velocity="6.001E3"/>
+      <limit effort="0" lower="-6.1086523819801535E0" upper="6.1086523819801535E0" velocity="0"/>
       <origin rpy="1.5707963267948963 0.0 -0.0" xyz="0.115 0.0 0.0"/>
       <parent link="${prefix}link_3"/>
@@ -181,5 +181,5 @@
       <axis xyz="0.0 0.0 1.0"/>
       <child link="${prefix}link_5"/>
-      <limit effort="0" lower="-2.138028333693054E0" upper="2.138028333693054E0" velocity="6.001E3"/>
+      <limit effort="0" lower="-2.138028333693054E0" upper="2.138028333693054E0" velocity="0"/>
       <origin rpy="-1.5707963267948963 0.0 -0.0" xyz="0.0 0.0 -1.42"/>
       <parent link="${prefix}link_4"/>
@@ -188,5 +188,5 @@
       <axis xyz="0.0 0.0 1.0"/>
       <child link="${prefix}link_6"/>
-      <limit effort="0" lower="-6.1086523819801535E0" upper="6.1086523819801535E0" velocity="6.001E3"/>
+      <limit effort="0" lower="-6.1086523819801535E0" upper="6.1086523819801535E0" velocity="0"/>
       <origin rpy="1.5707963267948963 0.0 -0.0" xyz="0.0 0.0 0.0"/>
       <parent link="${prefix}link_5"/>

Commit message: velocity limits

File: kuka_quantec_support/urdf/kr210_r2700-2_macro.xacro (robot description, xacro)
@@ -153,5 +153,5 @@
       <axis xyz="0.0 0.0 1.0"/>
       <child link="${prefix}link_1"/>
-      <limit effort="0" lower="-3.2288591161895095E0" upper="3.2288591161895095E0" velocity="0"/>
+      <limit effort="0" lower="-3.2288591161895095E0" upper="3.2288591161895095E0" velocity="${radians(120)}"/>
       <origin rpy="-3.141592653589793 0.0 -0.0" xyz="0.0 0.0 0.0"/>
       <parent link="${prefix}base_link_inertia"/>
@@ -160,5 +160,5 @@
       <axis xyz="0.0 0.0 1.0"/>
       <child link="${prefix}link_2"/>
-      <limit effort="0" lower="-2.443460952792061E0" upper="-8.726646259971647E-2" velocity="0"/>
+      <limit effort="0" lower="-2.443460952792061E0" upper="-8.726646259971647E-2" velocity="${radians(115)}"/>
       <origin rpy="1.5707963267948963 0.0 -0.0" xyz="0.33 0.0 -0.645"/>
       <parent link="${prefix}link_1"/>
@@ -167,5 +167,5 @@
       <axis xyz="0.0 0.0 1.0"/>
       <child link="${prefix}link_3"/>
-      <limit effort="0" lower="-2.0943951023931953E0" upper="2.9321531433504737E0" velocity="0"/>
+      <limit effort="0" lower="-2.0943951023931953E0" upper="2.9321531433504737E0" velocity="${radians(112)}"/>
       <origin rpy="0.0 0.0 -1.5707963267948963" xyz="1.15 0.0 0.0"/>
       <parent link="${prefix}link_2"/>
@@ -174,5 +174,5 @@
       <axis xyz="0.0 0.0 1.0"/>
       <child link="${prefix}link_4"/>
-      <limit effort="0" lower="-6.1086523819801535E0" upper="6.1086523819801535E0" velocity="0"/>
+      <limit effort="0" lower="-6.1086523819801535E0" upper="6.1086523819801535E0" velocity="${radians(179)}"/>
       <origin rpy="1.5707963267948963 0.0 -0.0" xyz="0.115 0.0 0.0"/>
       <parent link="${prefix}link_3"/>
@@ -181,5 +181,5 @@
       <axis xyz="0.0 0.0 1.0"/>
       <child link="${prefix}link_5"/>
-      <limit effort="0" lower="-2.181661564992912E0" upper="2.181661564992912E0" velocity="0"/>
+      <limit effort="0" lower="-2.181661564992912E0" upper="2.181661564992912E0" velocity="${radians(172)}"/>
       <origin rpy="-1.5707963267948963 0.0 -0.0" xyz="0.0 0.0 -1.22"/>
       <parent link="${prefix}link_4"/>
@@ -188,5 +188,5 @@
       <axis xyz="0.0 0.0 1.0"/>
       <child link="${prefix}link_6"/>
-      <limit effort="0" lower="-6.1086523819801535E0" upper="6.1086523819801535E0" velocity="0"/>
+      <limit effort="0" lower="-6.1086523819801535E0" upper="6.1086523819801535E0" velocity="${radians(220)}"/>
       <origin rpy="1.5707963267948963 0.0 -0.0" xyz="0.0 0.0 0.0"/>
       <parent link="${prefix}link_5"/>

File: kuka_quantec_support/urdf/kr210_r3100-2_macro.xacro (robot description, xacro)
@@ -153,5 +153,5 @@
       <axis xyz="0.0 0.0 1.0"/>
       <child link="${prefix}link_1"/>
-      <limit effort="0" lower="-3.2288591161895095E0" upper="3.2288591161895095E0" velocity="0"/>
+      <limit effort="0" lower="-3.2288591161895095E0" upper="3.2288591161895095E0" velocity="${radians(105)}"/>
       <origin rpy="-3.141592653589793 0.0 -0.0" xyz="0.0 0.0 0.0"/>
       <parent link="${prefix}base_link_inertia"/>
@@ -160,5 +160,5 @@
       <axis xyz="0.0 0.0 1.0"/>
       <child link="${prefix}link_2"/>
-      <limit effort="0" lower="-2.443460952792061E0" upper="-8.726646259971647E-2" velocity="0"/>
+      <limit effort="0" lower="-2.443460952792061E0" upper="-8.726646259971647E-2" velocity="${radians(94)}"/>
       <origin rpy="1.5707963267948963 0.0 -0.0" xyz="0.33 0.0 -0.645"/>
       <parent link="${prefix}link_1"/>
@@ -167,5 +167,5 @@
       <axis xyz="0.0 0.0 1.0"/>
       <child link="${prefix}link_3"/>
-      <limit effort="0" lower="-2.0943951023931953E0" upper="2.9321531433504737E0" velocity="0"/>
+      <limit effort="0" lower="-2.0943951023931953E0" upper="2.9321531433504737E0" velocity="${radians(100)}"/>
       <origin rpy="0.0 0.0 -1.5707963267948963" xyz="1.35 0.0 0.0"/>
       <parent link="${prefix}link_2"/>
@@ -174,5 +174,5 @@
       <axis xyz="0.0 0.0 1.0"/>
       <child link="${prefix}link_4"/>
-      <limit effort="0" lower="-6.1086523819801535E0" upper="6.1086523819801535E0" velocity="0"/>
+      <limit effort="0" lower="-6.1086523819801535E0" upper="6.1086523819801535E0" velocity="${radians(136)}"/>
       <origin rpy="1.5707963267948963 0.0 -0.0" xyz="0.115 0.0 0.0"/>
       <parent link="${prefix}link_3"/>
@@ -181,5 +181,5 @@
       <axis xyz="0.0 0.0 1.0"/>
       <child link="${prefix}link_5"/>
-      <limit effort="0" lower="-2.138028333693054E0" upper="2.138028333693054E0" velocity="0"/>
+      <limit effort="0" lower="-2.138028333693054E0" upper="2.138028333693054E0" velocity="${radians(129)}"/>
       <origin rpy="-1.5707963267948963 0.0 -0.0" xyz="0.0 0.0 -1.42"/>
       <parent link="${prefix}link_4"/>
@@ -188,5 +188,5 @@
       <axis xyz="0.0 0.0 1.0"/>
       <child link="${prefix}link_6"/>
-      <limit effort="0" lower="-6.1086523819801535E0" upper="6.1086523819801535E0" velocity="0"/>
+      <limit effort="0" lower="-6.1086523819801535E0" upper="6.1086523819801535E0" velocity="${radians(206)}"/>
       <origin rpy="1.5707963267948963 0.0 -0.0" xyz="0.0 0.0 0.0"/>
       <parent link="${prefix}link_5"/>
