Commit message: effort limits

File: kuka_quantec_support/urdf/kr210_r2700-2_macro.xacro (robot description, xacro)
@@ -153,5 +153,5 @@
       <axis xyz="0.0 0.0 1.0"/>
       <child link="${prefix}link_1"/>
-      <limit effort="0" lower="-3.2288591161895095E0" upper="3.2288591161895095E0" velocity="${radians(120)}"/>
+      <limit effort="7290" lower="-3.2288591161895095E0" upper="3.2288591161895095E0" velocity="${radians(120)}"/>
       <origin rpy="-3.141592653589793 0.0 -0.0" xyz="0.0 0.0 0.0"/>
       <parent link="${prefix}base_link_inertia"/>
@@ -160,5 +160,5 @@
       <axis xyz="0.0 0.0 1.0"/>
       <child link="${prefix}link_2"/>
-      <limit effort="0" lower="-2.443460952792061E0" upper="-8.726646259971647E-2" velocity="${radians(115)}"/>
+      <limit effort="8910" lower="-2.443460952792061E0" upper="-8.726646259971647E-2" velocity="${radians(115)}"/>
       <origin rpy="1.5707963267948963 0.0 -0.0" xyz="0.33 0.0 -0.645"/>
       <parent link="${prefix}link_1"/>
@@ -167,5 +167,5 @@
       <axis xyz="0.0 0.0 1.0"/>
       <child link="${prefix}link_3"/>
-      <limit effort="0" lower="-2.0943951023931953E0" upper="2.9321531433504737E0" velocity="${radians(112)}"/>
+      <limit effort="6988.84717" lower="-2.0943951023931953E0" upper="2.9321531433504737E0" velocity="${radians(112)}"/>
       <origin rpy="0.0 0.0 -1.5707963267948963" xyz="1.15 0.0 0.0"/>
       <parent link="${prefix}link_2"/>
@@ -174,5 +174,5 @@
       <axis xyz="0.0 0.0 1.0"/>
       <child link="${prefix}link_4"/>
-      <limit effort="0" lower="-6.1086523819801535E0" upper="6.1086523819801535E0" velocity="${radians(179)}"/>
+      <limit effort="2274.29199" lower="-6.1086523819801535E0" upper="6.1086523819801535E0" velocity="${radians(179)}"/>
       <origin rpy="1.5707963267948963 0.0 -0.0" xyz="0.115 0.0 0.0"/>
       <parent link="${prefix}link_3"/>
@@ -181,5 +181,5 @@
       <axis xyz="0.0 0.0 1.0"/>
       <child link="${prefix}link_5"/>
-      <limit effort="0" lower="-2.181661564992912E0" upper="2.181661564992912E0" velocity="${radians(172)}"/>
+      <limit effort="1398.30298" lower="-2.181661564992912E0" upper="2.181661564992912E0" velocity="${radians(172)}"/>
       <origin rpy="-1.5707963267948963 0.0 -0.0" xyz="0.0 0.0 -1.22"/>
       <parent link="${prefix}link_4"/>
@@ -188,5 +188,5 @@
       <axis xyz="0.0 0.0 1.0"/>
       <child link="${prefix}link_6"/>
-      <limit effort="0" lower="-6.1086523819801535E0" upper="6.1086523819801535E0" velocity="${radians(220)}"/>
+      <limit effort="781.554626" lower="-6.1086523819801535E0" upper="6.1086523819801535E0" velocity="${radians(220)}"/>
       <origin rpy="1.5707963267948963 0.0 -0.0" xyz="0.0 0.0 0.0"/>
       <parent link="${prefix}link_5"/>

File: kuka_quantec_support/urdf/kr210_r3100-2_macro.xacro (robot description, xacro)
@@ -153,5 +153,5 @@
       <axis xyz="0.0 0.0 1.0"/>
       <child link="${prefix}link_1"/>
-      <limit effort="0" lower="-3.2288591161895095E0" upper="3.2288591161895095E0" velocity="${radians(105)}"/>
+      <limit effort="7290" lower="-3.2288591161895095E0" upper="3.2288591161895095E0" velocity="${radians(105)}"/>
       <origin rpy="-3.141592653589793 0.0 -0.0" xyz="0.0 0.0 0.0"/>
       <parent link="${prefix}base_link_inertia"/>
@@ -160,5 +160,5 @@
       <axis xyz="0.0 0.0 1.0"/>
       <child link="${prefix}link_2"/>
-      <limit effort="0" lower="-2.443460952792061E0" upper="-8.726646259971647E-2" velocity="${radians(94)}"/>
+      <limit effort="8910" lower="-2.443460952792061E0" upper="-8.726646259971647E-2" velocity="${radians(94)}"/>
       <origin rpy="1.5707963267948963 0.0 -0.0" xyz="0.33 0.0 -0.645"/>
       <parent link="${prefix}link_1"/>
@@ -167,5 +167,5 @@
       <axis xyz="0.0 0.0 1.0"/>
       <child link="${prefix}link_3"/>
-      <limit effort="0" lower="-2.0943951023931953E0" upper="2.9321531433504737E0" velocity="${radians(100)}"/>
+      <limit effort="7251.2876" lower="-2.0943951023931953E0" upper="2.9321531433504737E0" velocity="${radians(100)}"/>
       <origin rpy="0.0 0.0 -1.5707963267948963" xyz="1.35 0.0 0.0"/>
       <parent link="${prefix}link_2"/>
@@ -174,5 +174,5 @@
       <axis xyz="0.0 0.0 1.0"/>
       <child link="${prefix}link_4"/>
-      <limit effort="0" lower="-6.1086523819801535E0" upper="6.1086523819801535E0" velocity="${radians(136)}"/>
+      <limit effort="2356.12598" lower="-6.1086523819801535E0" upper="6.1086523819801535E0" velocity="${radians(136)}"/>
       <origin rpy="1.5707963267948963 0.0 -0.0" xyz="0.115 0.0 0.0"/>
       <parent link="${prefix}link_3"/>
@@ -181,5 +181,5 @@
       <axis xyz="0.0 0.0 1.0"/>
       <child link="${prefix}link_5"/>
-      <limit effort="0" lower="-2.138028333693054E0" upper="2.138028333693054E0" velocity="${radians(129)}"/>
+      <limit effort="2358.44531" lower="-2.138028333693054E0" upper="2.138028333693054E0" velocity="${radians(129)}"/>
       <origin rpy="-1.5707963267948963 0.0 -0.0" xyz="0.0 0.0 -1.42"/>
       <parent link="${prefix}link_4"/>
@@ -188,5 +188,5 @@
       <axis xyz="0.0 0.0 1.0"/>
       <child link="${prefix}link_6"/>
-      <limit effort="0" lower="-6.1086523819801535E0" upper="6.1086523819801535E0" velocity="${radians(206)}"/>
+      <limit effort="1508.75476" lower="-6.1086523819801535E0" upper="6.1086523819801535E0" velocity="${radians(206)}"/>
       <origin rpy="1.5707963267948963 0.0 -0.0" xyz="0.0 0.0 0.0"/>
       <parent link="${prefix}link_5"/>
