Commit message: add updated velocity limit on joint_1 for kr210_r2700_2 in urdf

File: kuka_quantec_support/urdf/kr210_r2700_2_macro.xacro (robot description, xacro)
@@ -113,5 +113,5 @@
       <axis xyz="0.0 0.0 1.0"/>
       <child link="${prefix}link_1"/>
-      <limit effort="7290" lower="-3.2288591161895095E0" upper="3.2288591161895095E0" velocity="${radians(120)}"/>
+      <limit effort="7290" lower="-3.2288591161895095E0" upper="3.2288591161895095E0" velocity="2.0384"/>
       <origin rpy="-3.141592653589793 0.0 -0.0" xyz="0.0 0.0 0.0"/>
       <parent link="${prefix}base_link"/>

Commit message: fix joint2 velocity limit for kr210r2700-2

File: kuka_quantec_support/urdf/kr210_r2700_2_macro.xacro (robot description, xacro)
@@ -120,5 +120,5 @@
       <axis xyz="0.0 0.0 1.0"/>
       <child link="${prefix}link_2"/>
-      <limit effort="8910" lower="-2.443460952792061E0" upper="-8.726646259971647E-2" velocity="${radians(115)}"/>
+      <limit effort="8910" lower="-2.443460952792061E0" upper="-8.726646259971647E-2" velocity="1.9451"/>
       <origin rpy="1.5707963267948963 0.0 -0.0" xyz="0.33 0.0 -0.645"/>
       <parent link="${prefix}link_1"/>
