Commit message: Align link6-tool0 orientation with convention

File: kuka_quantec_support/urdf/kr210_r3100_ultra_macro.xacro (robot description, xacro)
@@ -191,5 +191,5 @@
     <joint name="${prefix}link6-tool0" type="fixed">
       <child link="${prefix}tool0"/>
-      <origin rpy="0.0 -0.0 0.0" xyz="0.0 0.0 -0.24"/>
+      <origin rpy="0.0 ${pi} 0.0" xyz="0.0 0.0 -0.24"/>
       <parent link="${prefix}link_6"/>
     </joint>
