Commit message: add gazebo support, fix urdf issues

File: kuka_mobile_robot_support/gazebo/diffbot.gazebo.xacro (robot description, xacro)
@@ -5,74 +5,74 @@
 -->
 <robot xmlns:xacro="http://ros.org/wiki/xacro">
-  <xacro:macro name="diffbot_gazebo" params="prefix">
-    <!-- Link1 -->
-    <gazebo reference="${prefix}base_link">
-      <material>Gazebo/Blue</material>
+  <xacro:macro name="diffbot_gazebo" params="prefix ros2_control_sim:=false">
+    <!-- left wheel -->
+    <gazebo reference="${prefix}left_wheel">
+      <mu1>0.95</mu1>
+      <mu2>0.95</mu2>
+      <material>Gazebo/Red</material>
     </gazebo>
-    <!-- Link2 -->
-    <gazebo reference="${prefix}link1">
-      <mu1>0.2</mu1>
-      <mu2>0.2</mu2>
+    <!-- right wheel -->
+    <gazebo reference="${prefix}right_wheel">
+      <mu1>0.95</mu1>
+      <mu2>0.95</mu2>
+      <material>Gazebo/Red</material>
+    </gazebo>
+     <!-- Base link -->
+    <gazebo reference="${prefix}generic_mr_body">
+      <material>Gazebo/Orange</material>
+    </gazebo>
+    <!-- Caster links -->
+    <gazebo reference="${prefix}caster_wheel_fl_link">
+      <mu1>0.001</mu1>
+      <mu2>0.001</mu2>
       <material>Gazebo/Black</material>
     </gazebo>
-    <!-- Link3 -->
-    <gazebo reference="${prefix}link2">
-      <mu1>0.2</mu1>
-      <mu2>0.2</mu2>
+    <gazebo reference="${prefix}caster_wheel_rl_link">
+      <mu1>0.001</mu1>
+      <mu2>0.001</mu2>
       <material>Gazebo/Black</material>
     </gazebo>
-    <!-- camera_link -->
-    <gazebo reference="${prefix}camera_link">
-      <mu1>0.2</mu1>
-      <mu2>0.2</mu2>
-      <material>Gazebo/Red</material>
+    <gazebo reference="${prefix}caster_wheel_bl_link">
+      <mu1>0.001</mu1>
+      <mu2>0.001</mu2>
+      <material>Gazebo/Black</material>
     </gazebo>
-    <!-- camera -->
-    <gazebo reference="${prefix}camera_link">
-      <sensor type="camera" name="camera1">
-        <update_rate>30.0</update_rate>
-        <camera name="head">
-          <horizontal_fov>1.3962634</horizontal_fov>
-          <image>
-            <width>800</width>
-            <height>800</height>
-            <format>R8G8B8</format>
-          </image>
-          <clip>
-            <near>0.02</near>
-            <far>300</far>
-          </clip>
-          <noise>
-            <type>gaussian</type>
-            <!-- Noise is sampled independently per pixel on each frame.
-            That pixel's noise value is added to each of its color
-            channels, which at that point lie in the range [0,1]. -->
-            <mean>0.0</mean>
-            <stddev>0.007</stddev>
-          </noise>
-        </camera>
-        <plugin name="camera_controller" filename="libgazebo_ros_camera.so">
-          <alwaysOn>true</alwaysOn>
-          <updateRate>0.0</updateRate>
-          <cameraName>diffbot/camera1</cameraName>
-          <imageTopicName>image_raw</imageTopicName>
-          <cameraInfoTopicName>camera_info</cameraInfoTopicName>
-          <frameName>camera_link_optical</frameName>
-          <!-- setting hackBaseline to anything but 0.0 will cause a misalignment
-          between the gazebo sensor image and the frame it is supposed to
-          be attached to -->
-          <hackBaseline>0.0</hackBaseline>
-          <distortionK1>0.0</distortionK1>
-          <distortionK2>0.0</distortionK2>
-          <distortionK3>0.0</distortionK3>
-          <distortionT1>0.0</distortionT1>
-          <distortionT2>0.0</distortionT2>
-          <CxPrime>0</CxPrime>
-          <Cx>0.0</Cx>
-          <Cy>0.0</Cy>
-          <focalLength>0.0</focalLength>
+    <gazebo reference="${prefix}caster_wheel_br_link">
+      <mu1>0.001</mu1>
+      <mu2>0.001</mu2>
+      <material>Gazebo/Black</material>
+    </gazebo>
+    <xacro:if value="${ros2_control_sim}">
+      <gazebo>
+        <!-- Joint state publisher -->
+        <plugin name="gazebo_ros2_control" filename="libgazebo_ros2_control.so" >
+          <robot_param>robot_description</robot_param>
+          <robot_param_node>robot_state_publisher</robot_param_node>
+          <parameters>$(find kuka_rox_hw_interface)/config/ros2_controller_config.yaml</parameters>
+          <parameters>$(find kuka_rox_hw_interface)/config/diff_drive_controller_config.yaml</parameters>
         </plugin>
-      </sensor>
-    </gazebo>
+      </gazebo>
+      <!-- diff drive controller plugin without ros2_control -->
+    </xacro:if>
+     <xacro:unless value="${ros2_control_sim}">
+      <gazebo>
+              <plugin name="diff_drive" filename="libgazebo_ros_diff_drive.so">
+                   <!-- Wheel Information  -->
+                  <left_joint>left_wheel_motor</left_joint>
+                  <right_joint>right_wheel_motor</right_joint>
+                  <wheel_separation>0.64</wheel_separation>
+                  <wheel_diameter>0.06</wheel_diameter>
+                    <!-- Limits  -->
+                  <max_wheel_torque>400</max_wheel_torque>
+                  <max_wheel_acceleration>1.0</max_wheel_acceleration>
+                    <!-- Output  -->
+                  <odometry_frame>odom</odometry_frame>
+                  <robot_base_frame>generic_mr_body_dummy</robot_base_frame>
+                  <publish_odom>true</publish_odom>
+                  <publish_odom_tf>true</publish_odom_tf>
+                  <publish_wheel_tf>true</publish_wheel_tf>
+              </plugin>
+          </gazebo>
+      </xacro:unless>
   </xacro:macro>
 </robot>

File: kuka_mobile_robot_support/ros2_control/mrob_kuka.ros2_control.xacro (robot description, xacro)
@@ -1,48 +1,66 @@
 <?xml version="1.0"?>
 <robot xmlns:xacro="http://www.ros.org/wiki/xacro">
-  <xacro:macro name="mrob_kuka_ros2_control" params="name prefix client_ip controller_ip control_mode consequent_lost_packets lost_packets_in_timeframe timeframe_ms">
+  <xacro:macro name="mrob_kuka_ros2_control" params="name prefix client_ip controller_ip control_mode consequent_lost_packets lost_packets_in_timeframe timeframe_ms use_fake_hardware:=false gazebo_sim:=false">
     <ros2_control name="${name}" type="system">
       <hardware>
-        <plugin>kuka_rox::KukaRoXHardwareInterface</plugin>
-        <param name="client_ip">${client_ip}</param>
-        <param name="controller_ip">${controller_ip}</param>
-        <param name="control_mode">${control_mode}</param>
-        <param name="consequent_lost_packets">${consequent_lost_packets}</param>
-        <param name="lost_packets_in_timeframe">${lost_packets_in_timeframe}</param>
-        <param name="timeframe_ms">${timeframe_ms}</param>
-        <param name="example_param_hw_start_duration_sec">0</param>
-        <param name="example_param_hw_stop_duration_sec">3.0</param>
+        <xacro:if value="${use_fake_hardware}">
+          <plugin>mock_components/GenericSystem</plugin>
+          <param name="fake_sensor_commands">false</param>
+          <param name="state_following_offset">0.0</param>
+        </xacro:if>
+        <xacro:unless value="${use_fake_hardware}">
+          <xacro:if value="${gazebo_sim}">
+            <plugin>gazebo_ros2_control/GazeboSystem</plugin>
+          </xacro:if>
+          <xacro:unless value="${gazebo_sim}">
+            <plugin>kuka_rox::KukaRoXHardwareInterface</plugin>
+            <param name="client_ip">${client_ip}</param>
+            <param name="controller_ip">${controller_ip}</param>
+            <param name="control_mode">${control_mode}</param>
+            <param name="consequent_lost_packets">${consequent_lost_packets}</param>
+            <param name="lost_packets_in_timeframe">${lost_packets_in_timeframe}</param>
+            <param name="timeframe_ms">${timeframe_ms}</param>
+          </xacro:unless>
+        </xacro:unless>
+        <plugin>gazebo_ros2_control/GazeboSystem</plugin>
       </hardware>
-      <joint name="${prefix}linear/x">
-        <command_interface name="velocity"/>
-        <state_interface name="position"/>
-        <state_interface name="velocity"/>
+      <joint name="${prefix}twist/linear">
+        <command_interface name="x"/>
+        <command_interface name="y"/>
+        <command_interface name="z"/>
+        <state_interface name="x"/>
+        <state_interface name="y"/>
+        <state_interface name="z"/>
       </joint>
-      <joint name="${prefix}linear/y">
-        <command_interface name="velocity"/>
-        <state_interface name="position"/>
-        <state_interface name="velocity"/>
+      <joint name="${prefix}twist/angular">
+        <command_interface name="x"/>
+        <command_interface name="y"/>
+        <command_interface name="z"/>
+        <state_interface name="x"/>
+        <state_interface name="y"/>
+        <state_interface name="z"/>
       </joint>
-      <joint name="${prefix}linear/z">
-        <command_interface name="velocity"/>
-        <state_interface name="position"/>
-        <state_interface name="velocity"/>
-      </joint>
-      <joint name="${prefix}angular/x">
-        <command_interface name="velocity"/>
-        <state_interface name="position"/>
-        <state_interface name="velocity"/>
-      </joint>
-      <joint name="${prefix}angular/y">
-        <command_interface name="velocity"/>
-        <state_interface name="position"/>
-        <state_interface name="velocity"/>
-      </joint>
-      <joint name="${prefix}angular/z">
-        <command_interface name="velocity"/>
-        <state_interface name="position"/>
-        <state_interface name="velocity"/>
-      </joint>
+      <joint name="left_wheel_motor">
+          <command_interface name="velocity">
+            <param name="min">-1</param>
+            <param name="max">1</param>
+          </command_interface>
+          <state_interface name="position"/>
+          <state_interface name="velocity"/>
+        </joint>
+        <joint name="right_wheel_motor">
+          <command_interface name="velocity">
+            <param name="min">-1</param>
+            <param name="max">1</param>
+          </command_interface>
+          <state_interface name="position"/>
+          <state_interface name="velocity"/>
+        </joint>
     </ros2_control>
+ <xacro:if value="${gazebo_sim}">
+<!-- config file with gazebo parameters-->
+            <xacro:include filename="$(find kuka_mobile_robot_support)/gazebo/diffbot.gazebo.xacro" />
+            <xacro:diffbot_gazebo  prefix="" ros2_control_sim="true"/>
+ </xacro:if>
   </xacro:macro>
 </robot>

File: kuka_mobile_robot_support/urdf/KUKA_MR.urdf.xacro (robot description, xacro)
@@ -4,5 +4,5 @@
   <xacro:arg name="prefix" default="" />
 <!-- Import diffbot urdf file  -->
-  <xacro:include filename="$(find kuka_mobile_robot_support)/urdf/diffbot_kuka_macro.xacro" />
+  <!-- <xacro:include filename="$(find kuka_mobile_robot_support)/urdf/diffbot_kuka_macro.xacro" /> -->
   <xacro:include filename="$(find kuka_mobile_robot_support)/urdf/mrob_kuka_macro.xacro" />
   <!-- Read parameters from eci_config  -->
@@ -25,4 +25,7 @@
                   lost_packets_in_timeframe="${lost_packets_in_timeframe}"
                   timeframe_ms="${timeframe_ms}"/>  -->
+  <!-- Read additional arguments  -->
+  <xacro:arg name="use_fake_hardware" default="false" />
+  <xacro:arg name="gazebo_sim" default="false" />
   <xacro:mrob_kuka prefix=""
                   client_ip="${client_ip}"
@@ -31,4 +34,6 @@
                   consequent_lost_packets="${consequent_lost_packets}"
                   lost_packets_in_timeframe="${lost_packets_in_timeframe}"
-                  timeframe_ms="${timeframe_ms}"/>
+                  timeframe_ms="${timeframe_ms}"
+                  use_fake_hardware="$(arg use_fake_hardware)"
+                  gazebo_sim="$(arg gazebo_sim)" />
 </robot>

File: kuka_mobile_robot_support/urdf/mrob_kuka_macro.xacro (robot description, xacro)
@@ -1,8 +1,8 @@
 <?xml version="1.0" encoding="UTF-8"?>
-<robot xmlns:xacro="http://www.ros.org/wiki/xacro" name="LBRiisy15R930">
+<robot xmlns:xacro="http://www.ros.org/wiki/xacro" name="">
   <!-- include helper xacros -->
   <xacro:include filename="$(find kuka_mobile_robot_support)/ros2_control/mrob_kuka.ros2_control.xacro" />
   <xacro:include filename="$(find kuka_resources)/urdf/common_materials.xacro"/>
-  <xacro:macro name="mrob_kuka" params="prefix client_ip controller_ip control_mode consequent_lost_packets lost_packets_in_timeframe timeframe_ms">
+  <xacro:macro name="mrob_kuka" params="prefix client_ip controller_ip control_mode consequent_lost_packets lost_packets_in_timeframe timeframe_ms use_fake_hardware:=false gazebo_sim:=false">
     <!-- ros2 control instance -->
     <xacro:mrob_kuka_ros2_control
@@ -14,5 +14,7 @@
       consequent_lost_packets="${consequent_lost_packets}"
       lost_packets_in_timeframe="${lost_packets_in_timeframe}"
-      timeframe_ms="${timeframe_ms}" />
+      timeframe_ms="${timeframe_ms}"
+      use_fake_hardware="${use_fake_hardware}"
+      gazebo_sim="${gazebo_sim}"/>
     <!-- Include and instatiate diffbot description urdf file-->
     <xacro:include filename="$(find kuka_mobile_robot_support)/urdf/diffbot_description.urdf.xacro" />
@@ -33,5 +35,5 @@
           <child link="left_wheel"/>
           <limit effort="5.0E2" velocity="1.0E2"/>
-          <origin rpy="-0.0 0.0 -0.0" xyz="0.0 0.325 0.06"/>
+          <origin rpy="-0.0 0.0 -0.0" xyz="0.0 0.325 0.028"/>  <!-- 0.06 -->
           <parent link="generic_mr_body"/>
         </joint>
@@ -40,5 +42,5 @@
           <child link="right_wheel"/>
           <limit effort="5.0E2" velocity="1.0E1"/>
-          <origin rpy="-0.0 0.0 -0.0" xyz="0.0 -0.325 0.0"/>
+          <origin rpy="-0.0 0.0 -0.0" xyz="0.0 -0.325 0.028"/>  <!-- 0.06 -->
           <parent link="generic_mr_body"/>
         </joint>
@@ -95,5 +97,5 @@
           <inertial>
             <inertia ixx="5.0" ixy="0.0" ixz="0.0" iyy="10.0" iyz="0.0" izz="10.0"/>
-            <mass value="1.0E1"/>
+            <mass value="1.0E2"/>
             <origin rpy="-0.0 0.0 -0.0" xyz="0.0 0.0 0.325"/>
           </inertial>
@@ -129,5 +131,5 @@
               <mesh filename="package://kuka_mobile_robot_support/meshes/37153975930.stl"/>
             </geometry>
-            <origin rpy="1.5707963267948963 0.0 -0.0" xyz="0.0 0.0 0.0"/>
+            <origin rpy="0.0 0.0 -1.5707963267948963" xyz="0.0 -0.02 0.0"/>
           </collision>
           <inertial>
@@ -205,5 +207,5 @@
               <mesh filename="package://kuka_mobile_robot_support/meshes/37154306984.stl"/>
             </geometry>
-            <origin rpy="1.5707963267948963 0.0 -0.0" xyz="0.0 0.0 0.0"/>
+            <origin rpy="-0.0 0.0 1.5707963267948963" xyz="0.0 0.02 0.0"/>
           </collision>
           <inertial>
