Commit message: iiwa fixes

File: kuka_lbr_iiwa_moveit_config/srdf/lbr_iiwa_arm.macro.xacro (robot description, xacro)
@@ -25,5 +25,5 @@
     </group_state>
     <!--VIRTUAL JOINT: Purpose: this element defines a virtual joint between a robot link and an external frame of reference (considered fixed with respect to the robot)-->
-    <virtual_joint name="virtual_joint" type="floating" parent_frame="world" child_link="${prefix}base_link_inertia" />
+    <!-- <virtual_joint name="virtual_joint" type="floating" parent_frame="world" child_link="${prefix}base_link_inertia" /> -->
     <!--END EFFECTOR: Purpose: Represent information about an end effector.-->
     <end_effector name="flange" parent_link="${prefix}flange" group="end_effector" parent_group="lbr_iiwa_arm"/>

File: kuka_lbr_iiwa_support/urdf/lbr_iiwa14_r820_macro.xacro (robot description, xacro)
@@ -169,4 +169,9 @@
     </link>
     <!-- joints - main serial chain -->
+    <joint name="${prefix}base_link-base_link_inertia" type="fixed">
+      <parent link="${prefix}base_link" />
+      <child link="${prefix}base_link_inertia" />
+      <origin xyz="0 0 0" rpy="0 0 0" />
+    </joint>
     <joint name="${prefix}joint_a1" type="revolute">
       <parent link="${prefix}base_link_inertia"/>
@@ -236,5 +241,5 @@
     <joint name="${prefix}link7-tool0" type="fixed">
       <parent link="${prefix}link_7"/>
-      <child link="${prefix}flange"/>
+      <child link="${prefix}tool0"/>
       <origin rpy="-0.0 0.0 0.0" xyz="0.0 0.0 0.071"/>
     </joint>

File: kuka_lbr_iiwa_support/urdf/lbr_iiwa_ros2_control.xacro (robot description, xacro)
@@ -1,5 +1,5 @@
 <?xml version="1.0" encoding="UTF-8"?>
 <robot xmlns:xacro="http://www.ros.org/wiki/xacro">
-  <xacro:macro name="kuka_lbr_iisy_ros2_control" params="name prefix use_fake_hardware:=false gazebo_sim:=false">
+  <xacro:macro name="kuka_lbr_iiwa_ros2_control" params="name prefix io_access use_fake_hardware:=false gazebo_sim:=false">
     <ros2_control name="${name}" type="system">
       <hardware>
