Commit message: Fix flange transform in kr560_r3100_2_macro.xacro
Added a new robot model for the KUKA FORTEC family
#42

https://github.com/kroshu/kuka_robot_descriptions/pull/42#discussion_r1440587691

Co-authored-by: Svastits <49677296+Svastits@users.noreply.github.com>

File: kuka_fortec_support/urdf/kr560_r3100_2_macro.xacro (robot description, xacro)
@@ -198,5 +198,5 @@
         <joint name="${prefix}link6-flange" type="fixed">
             <child link="${prefix}flange" />
-            <origin rpy="${pi/2} 0.0 -0.0" xyz="0.0 0.0 -0.0899" />
+            <origin rpy="0 ${pi/2} -0.0" xyz="0.0 0.0 -0.305" />
             <parent link="${prefix}link_6" />
         </joint>

Commit message: tool0 frame should be equivalent to the TCP
Fix PR comment 

https://github.com/kroshu/kuka_robot_descriptions/pull/42#discussion_r1440516921

Co-authored-by: Svastits <49677296+Svastits@users.noreply.github.com>

File: kuka_fortec_support/urdf/kr560_r3100_2_macro.xacro (robot description, xacro)
@@ -205,5 +205,5 @@
         <joint name="${prefix}link6-tool0" type="fixed">
             <child link="${prefix}tool0" />
-            <origin rpy="${pi/2} 0.0 -0.0" xyz="0.0 0.0 -0.0899" />
+            <origin rpy="0 ${pi} -0.0" xyz="0.0 0.0 -0.305" />
             <parent link="${prefix}link_6" />
         </joint>

Commit message: mesh folder rename
https://github.com/kroshu/kuka_robot_descriptions/pull/42#discussion_r1440520754

File: kuka_fortec_support/urdf/kr560_r3100_2_macro.xacro (robot description, xacro)
@@ -10,5 +10,5 @@
             <collision>
                 <geometry>
-                    <mesh filename="package://kuka_fortec_support/meshes/kr560_r3100-2/collision/base_link.stl"/>
+                    <mesh filename="package://kuka_fortec_support/meshes/kr560_r3100_2/collision/base_link.stl"/>
                 </geometry>
                 <origin rpy="-0.0 0.0 -0.0" xyz="0.0 0.0 0.0"/>
@@ -21,5 +21,5 @@
             <visual>
                 <geometry>
-                    <mesh filename="package://kuka_fortec_support/meshes/kr560_r3100-2/visual/base_link.dae" />
+                    <mesh filename="package://kuka_fortec_support/meshes/kr560_r3100_2/visual/base_link.dae" />
                 </geometry>
                 <origin rpy="-0.0 0.0 -0.0" xyz="0.0 0.0 0.0" />
@@ -29,5 +29,5 @@
             <collision>
                 <geometry>
-                    <mesh filename="package://kuka_fortec_support/meshes/kr560_r3100-2/collision/link_1.stl"/>
+                    <mesh filename="package://kuka_fortec_support/meshes/kr560_r3100_2/collision/link_1.stl"/>
                 </geometry>
                 <origin rpy="-0.0 0.0 -0.0" xyz="0.0 0.0 0.0"/>
@@ -40,5 +40,5 @@
             <visual>
                 <geometry>
-                    <mesh filename="package://kuka_fortec_support/meshes/kr560_r3100-2/visual/link_1.dae" />
+                    <mesh filename="package://kuka_fortec_support/meshes/kr560_r3100_2/visual/link_1.dae" />
                 </geometry>
                 <origin rpy="-0.0 0.0 -0.0" xyz="0.0 0.0 0.0" />
@@ -48,5 +48,5 @@
             <collision>
                 <geometry>
-                    <mesh filename="package://kuka_fortec_support/meshes/kr560_r3100-2/collision/link_2.stl"/>
+                    <mesh filename="package://kuka_fortec_support/meshes/kr560_r3100_2/collision/link_2.stl"/>
                 </geometry>
                 <origin rpy="-0.0 0.0 -0.0" xyz="0.0 0.0 0.0"/>
@@ -59,5 +59,5 @@
             <visual>
                 <geometry>
-                    <mesh filename="package://kuka_fortec_support/meshes/kr560_r3100-2/visual/link_2.dae" />
+                    <mesh filename="package://kuka_fortec_support/meshes/kr560_r3100_2/visual/link_2.dae" />
                 </geometry>
                 <origin rpy="-0.0 0.0 -0.0" xyz="0.0 0.0 0.0" />
@@ -67,5 +67,5 @@
             <collision>
                 <geometry>
-                    <mesh filename="package://kuka_fortec_support/meshes/kr560_r3100-2/collision/link_3.stl"/>
+                    <mesh filename="package://kuka_fortec_support/meshes/kr560_r3100_2/collision/link_3.stl"/>
                 </geometry>
                 <origin rpy="-0.0 0.0 -0.0" xyz="0.0 0.0 0.0"/>
@@ -78,5 +78,5 @@
             <visual>
                 <geometry>
-                    <mesh filename="package://kuka_fortec_support/meshes/kr560_r3100-2/visual/link_3.dae" />
+                    <mesh filename="package://kuka_fortec_support/meshes/kr560_r3100_2/visual/link_3.dae" />
                 </geometry>
                 <origin rpy="-0.0 0.0 -0.0" xyz="0.0 0.0 0.0" />
@@ -86,5 +86,5 @@
             <collision>
                 <geometry>
-                    <mesh filename="package://kuka_fortec_support/meshes/kr560_r3100-2/collision/link_4.stl"/>
+                    <mesh filename="package://kuka_fortec_support/meshes/kr560_r3100_2/collision/link_4.stl"/>
                 </geometry>
                 <origin rpy="-0.0 0.0 -0.0" xyz="0.0 0.0 0.0"/>
@@ -97,5 +97,5 @@
             <visual>
                 <geometry>
-                    <mesh filename="package://kuka_fortec_support/meshes/kr560_r3100-2/visual/link_4.dae" />
+                    <mesh filename="package://kuka_fortec_support/meshes/kr560_r3100_2/visual/link_4.dae" />
                 </geometry>
                 <origin rpy="-0.0 0.0 -0.0" xyz="0.0 0.0 0.0" />
@@ -105,5 +105,5 @@
             <collision>
                 <geometry>
-                    <mesh filename="package://kuka_fortec_support/meshes/kr560_r3100-2/collision/link_5.stl"/>
+                    <mesh filename="package://kuka_fortec_support/meshes/kr560_r3100_2/collision/link_5.stl"/>
                 </geometry>
                 <origin rpy="-0.0 0.0 -0.0" xyz="0.0 0.0 0.0"/>
@@ -116,5 +116,5 @@
             <visual>
                 <geometry>
-                    <mesh filename="package://kuka_fortec_support/meshes/kr560_r3100-2/visual/link_5.dae" />
+                    <mesh filename="package://kuka_fortec_support/meshes/kr560_r3100_2/visual/link_5.dae" />
                 </geometry>
                 <origin rpy="-0.0 0.0 -0.0" xyz="0.0 0.0 0.0" />
@@ -124,5 +124,5 @@
             <collision>
                 <geometry>
-                    <mesh filename="package://kuka_fortec_support/meshes/kr560_r3100-2/collision/link_6.stl"/>
+                    <mesh filename="package://kuka_fortec_support/meshes/kr560_r3100_2/collision/link_6.stl"/>
                 </geometry>
                 <origin rpy="-0.0 0.0 -0.0" xyz="0.0 0.0 0.0"/>
@@ -135,5 +135,5 @@
             <visual>
                 <geometry>
-                    <mesh filename="package://kuka_fortec_support/meshes/kr560_r3100-2/visual/link_6.dae" />
+                    <mesh filename="package://kuka_fortec_support/meshes/kr560_r3100_2/visual/link_6.dae" />
                 </geometry>
                 <origin rpy="-0.0 0.0 -0.0" xyz="0.0 0.0 0.0" />
