Commit message: fix after merge

File: kuka_fortec_support/urdf/kr560_r3100_2.urdf.xacro (robot description, xacro)
@@ -5,4 +5,15 @@
     <!-- Read additional arguments  -->
     <xacro:arg name="use_fake_hardware" default="false" />
-    <xacro:kuka_kr560_r3100_2_robot prefix="" use_fake_hardware="$(arg use_fake_hardware)" />
+    <xacro:arg name="client_ip" default="0.0.0.0" />
+    <xacro:arg name="client_port" default="59152" />
+    <xacro:arg name="prefix" default="" />
+    <xacro:arg name="x" default="0" />
+    <xacro:arg name="y" default="0" />
+    <xacro:arg name="z" default="0" />
+    <xacro:arg name="roll" default="0" />
+    <xacro:arg name="pitch" default="0" />
+    <xacro:arg name="yaw" default="0" />
+    <xacro:kuka_kr560_r3100_2_robot client_ip="$(arg client_ip)" client_port="$(arg client_port)" prefix="$(arg prefix)" use_fake_hardware="$(arg use_fake_hardware)">
+        <origin xyz="$(arg x) $(arg y) $(arg z)" rpy="$(arg roll) $(arg pitch) $(arg yaw)" />
+    </xacro:kuka_kr560_r3100_2_robot>
 </robot>

File: kuka_fortec_support/urdf/kr560_r3100_2_macro.xacro (robot description, xacro)
@@ -1,11 +1,11 @@
-<?xml version="1.0" encoding="UTF-8"?>
+<?xml version="1.0"?>
 <robot xmlns:xacro="http://wiki.ros.org/xacro">
-    <xacro:include filename="$(find kuka_fortec_support)/urdf/kr_fortec_ros2_control.xacro"/>
+    <xacro:include filename="$(find kuka_fortec_support)/urdf/kr_fortec_ros2_control.xacro" />
     <xacro:include filename="$(find kuka_fortec_support)/urdf/kr_fortec_transmission.xacro" />
-    <xacro:macro name="kuka_kr560_r3100_2_robot" params="prefix use_fake_hardware">
+    <xacro:macro name="kuka_kr560_r3100_2_robot" params="client_ip client_port prefix use_fake_hardware *origin">
         <!-- ros2 control instance -->
-        <xacro:kuka_fortec_ros2_control name="kr560_r3100_2" prefix="${prefix}" use_fake_hardware="${use_fake_hardware}" />
-        <link name="${prefix}base_link" />
-        <link name="${prefix}base_link_inertia">
+        <xacro:kuka_fortec_ros2_control name="${prefix}kr560_r3100_2" client_ip="${client_ip}" client_port="${client_port}" prefix="${prefix}" use_fake_hardware="${use_fake_hardware}"/>
+        <link name="world"/>
+        <link name="${prefix}base_link">
             <collision>
                 <geometry>
@@ -15,13 +15,13 @@
             </collision>
             <inertial>
-                <inertia ixx="68.88717275" ixy="0.0" ixz="0.0" iyy="31.94793234" iyz="0.0" izz="84.55633739" />
-                <mass value="4.3839E2" />
-                <origin rpy="-0.0 0.0 -0.0" xyz="0.0 0.0 0.0" />
-            </inertial>
-            <visual>
-                <geometry>
-                    <mesh filename="package://kuka_fortec_support/meshes/kr560_r3100_2/visual/base_link.dae" />
-                </geometry>
-                <origin rpy="-0.0 0.0 -0.0" xyz="0.0 0.0 0.0" />
+                <inertia ixx="68.88717275" ixy="0.0" ixz="0.0" iyy="31.94793234" iyz="0.0" izz="84.55633739"/>
+                <mass value="4.3839E2"/>
+                <origin rpy="-0.0 0.0 -0.0" xyz="0.0 0.0 0.0"/>
+            </inertial>
+            <visual>
+                <geometry>
+                    <mesh filename="package://kuka_fortec_support/meshes/kr560_r3100_2/visual/base_link.dae"/>
+                </geometry>
+                <origin rpy="-0.0 0.0 -0.0" xyz="0.0 0.0 0.0"/>
             </visual>
         </link>
@@ -34,13 +34,13 @@
             </collision>
             <inertial>
-                <inertia ixx="344.90558565" ixy="0.0" ixz="0.0" iyy="45.43063965" iyz="0.0" izz="376.57742569" />
-                <mass value="5.5748E2" />
-                <origin rpy="-0.0 0.0 -0.0" xyz="0.0 0.0 0.0" />
-            </inertial>
-            <visual>
-                <geometry>
-                    <mesh filename="package://kuka_fortec_support/meshes/kr560_r3100_2/visual/link_1.dae" />
-                </geometry>
-                <origin rpy="-0.0 0.0 -0.0" xyz="0.0 0.0 0.0" />
+                <inertia ixx="344.90558565" ixy="0.0" ixz="0.0" iyy="45.43063965" iyz="0.0" izz="376.57742569"/>
+                <mass value="5.5748E2"/>
+                <origin rpy="-0.0 0.0 -0.0" xyz="0.0 0.0 0.0"/>
+            </inertial>
+            <visual>
+                <geometry>
+                    <mesh filename="package://kuka_fortec_support/meshes/kr560_r3100_2/visual/link_1.dae"/>
+                </geometry>
+                <origin rpy="-0.0 0.0 -0.0" xyz="0.0 0.0 0.0"/>
             </visual>
         </link>
@@ -53,13 +53,13 @@
             </collision>
             <inertial>
-                <inertia ixx="6.30840213" ixy="0.0" ixz="0.0" iyy="26.6876282" iyz="0.0" izz="29.5636589" />
-                <mass value="7.4023E2" />
-                <origin rpy="-0.0 0.0 -0.0" xyz="0.0 0.0 0.0" />
-            </inertial>
-            <visual>
-                <geometry>
-                    <mesh filename="package://kuka_fortec_support/meshes/kr560_r3100_2/visual/link_2.dae" />
-                </geometry>
-                <origin rpy="-0.0 0.0 -0.0" xyz="0.0 0.0 0.0" />
+                <inertia ixx="6.30840213" ixy="0.0" ixz="0.0" iyy="26.6876282" iyz="0.0" izz="29.5636589"/>
+                <mass value="7.4023E2"/>
+                <origin rpy="-0.0 0.0 -0.0" xyz="0.0 0.0 0.0"/>
+            </inertial>
+            <visual>
+                <geometry>
+                    <mesh filename="package://kuka_fortec_support/meshes/kr560_r3100_2/visual/link_2.dae"/>
+                </geometry>
+                <origin rpy="-0.0 0.0 -0.0" xyz="0.0 0.0 0.0"/>
             </visual>
         </link>
@@ -72,13 +72,13 @@
             </collision>
             <inertial>
-                <inertia ixx="0.69367801" ixy="0.0" ixz="0.0" iyy="2.78506558" iyz="0.0" izz="2.86251005" />
-                <mass value="2.41307E2" />
-                <origin rpy="-0.0 0.0 -0.0" xyz="0.0 0.0 0.0" />
-            </inertial>
-            <visual>
-                <geometry>
-                    <mesh filename="package://kuka_fortec_support/meshes/kr560_r3100_2/visual/link_3.dae" />
-                </geometry>
-                <origin rpy="-0.0 0.0 -0.0" xyz="0.0 0.0 0.0" />
+                <inertia ixx="0.69367801" ixy="0.0" ixz="0.0" iyy="2.78506558" iyz="0.0" izz="2.86251005"/>
+                <mass value="2.41307E2"/>
+                <origin rpy="-0.0 0.0 -0.0" xyz="0.0 0.0 0.0"/>
+            </inertial>
+            <visual>
+                <geometry>
+                    <mesh filename="package://kuka_fortec_support/meshes/kr560_r3100_2/visual/link_3.dae"/>
+                </geometry>
+                <origin rpy="-0.0 0.0 -0.0" xyz="0.0 0.0 0.0"/>
             </visual>
         </link>
@@ -91,13 +91,13 @@
             </collision>
             <inertial>
-                <inertia ixx="1.10203833" ixy="0.0" ixz="0.0" iyy="0.78393869" iyz="0.0" izz="1.20828475" />
-                <mass value="9.7442E1" />
-                <origin rpy="-0.0 0.0 -0.0" xyz="0.0 0.0 0.0" />
-            </inertial>
-            <visual>
-                <geometry>
-                    <mesh filename="package://kuka_fortec_support/meshes/kr560_r3100_2/visual/link_4.dae" />
-                </geometry>
-                <origin rpy="-0.0 0.0 -0.0" xyz="0.0 0.0 0.0" />
+                <inertia ixx="1.10203833" ixy="0.0" ixz="0.0" iyy="0.78393869" iyz="0.0" izz="1.20828475"/>
+                <mass value="9.7442E1"/>
+                <origin rpy="-0.0 0.0 -0.0" xyz="0.0 0.0 0.0"/>
+            </inertial>
+            <visual>
+                <geometry>
+                    <mesh filename="package://kuka_fortec_support/meshes/kr560_r3100_2/visual/link_4.dae"/>
+                </geometry>
+                <origin rpy="-0.0 0.0 -0.0" xyz="0.0 0.0 0.0"/>
             </visual>
         </link>
@@ -110,13 +110,13 @@
             </collision>
             <inertial>
-                <inertia ixx="0.15462725" ixy="0.0" ixz="0.0" iyy="0.15475987" iyz="0.0" izz="0.18961138" />
-                <mass value="5.36088E1" />
-                <origin rpy="-0.0 0.0 -0.0" xyz="0.0 0.0 0.0" />
-            </inertial>
-            <visual>
-                <geometry>
-                    <mesh filename="package://kuka_fortec_support/meshes/kr560_r3100_2/visual/link_5.dae" />
-                </geometry>
-                <origin rpy="-0.0 0.0 -0.0" xyz="0.0 0.0 0.0" />
+                <inertia ixx="0.15462725" ixy="0.0" ixz="0.0" iyy="0.15475987" iyz="0.0" izz="0.18961138"/>
+                <mass value="5.36088E1"/>
+                <origin rpy="-0.0 0.0 -0.0" xyz="0.0 0.0 0.0"/>
+            </inertial>
+            <visual>
+                <geometry>
+                    <mesh filename="package://kuka_fortec_support/meshes/kr560_r3100_2/visual/link_5.dae"/>
+                </geometry>
+                <origin rpy="-0.0 0.0 -0.0" xyz="0.0 0.0 0.0"/>
             </visual>
         </link>
@@ -129,68 +129,68 @@
             </collision>
             <inertial>
-                <inertia ixx="0.15462725" ixy="0.0" ixz="0.0" iyy="0.15475987" iyz="0.0" izz="0.18961138" />
-                <mass value="3.202E1" />
-                <origin rpy="-0.0 0.0 -0.0" xyz="0.0 0.0 0.0" />
-            </inertial>
-            <visual>
-                <geometry>
-                    <mesh filename="package://kuka_fortec_support/meshes/kr560_r3100_2/visual/link_6.dae" />
-                </geometry>
-                <origin rpy="-0.0 0.0 -0.0" xyz="0.0 0.0 0.0" />
-            </visual>
-        </link>
-        <joint name="${prefix}base_link-base_link_inertia" type="fixed">
-            <parent link="${prefix}base_link" />
-            <child link="${prefix}base_link_inertia" />
-            <origin xyz="0 0 0" rpy="0 0 0" />
+                <inertia ixx="0.15462725" ixy="0.0" ixz="0.0" iyy="0.15475987" iyz="0.0" izz="0.18961138"/>
+                <mass value="3.202E1"/>
+                <origin rpy="-0.0 0.0 -0.0" xyz="0.0 0.0 0.0"/>
+            </inertial>
+            <visual>
+                <geometry>
+                    <mesh filename="package://kuka_fortec_support/meshes/kr560_r3100_2/visual/link_6.dae"/>
+                </geometry>
+                <origin rpy="-0.0 0.0 -0.0" xyz="0.0 0.0 0.0"/>
+            </visual>
+        </link>
+        <joint name="${prefix}world-base_link" type="fixed">
+            <parent link="world" />
+            <child link="${prefix}base_link" />
+            <xacro:insert_block name="origin" />
         </joint>
         <joint name="${prefix}joint_1" type="revolute">
-            <axis xyz="0.0 0.0 1.0" />
-            <child link="${prefix}link_1" />
-            <limit effort="15000.0E0" lower="-3.2288591161895095E0" upper="3.2288591161895095E0" velocity="${radians(90)}" />
-            <origin rpy="-3.141592653589793 0.0 -0.0" xyz="0.0 0.0 0.0" />
-            <parent link="${prefix}base_link_inertia" />
+            <axis xyz="0.0 0.0 1.0"/>
+            <child link="${prefix}link_1"/>
+            <limit effort="15000.0E0" lower="-3.2288591161895095E0" upper="3.2288591161895095E0" velocity="${radians(90)}"/>
+            <origin rpy="-3.141592653589793 0.0 -0.0" xyz="0.0 0.0 0.0"/>
+            <parent link="${prefix}base_link"/>
         </joint>
         <joint name="${prefix}joint_2" type="revolute">
-            <axis xyz="0.0 0.0 1.0" />
-            <child link="${prefix}link_2" />
-            <limit effort="17880.0E0" lower="-2.2689280275926285E0" upper="3.490658503988659E-1" velocity="${radians(80)}" />
-            <origin rpy="${pi/2.0} 0.0 -0.0" xyz="0.5 0.0 -0.86" />
-            <parent link="${prefix}link_1" />
+            <axis xyz="0.0 0.0 1.0"/>
+            <child link="${prefix}link_2"/>
+            <limit effort="17880.0E0" lower="-2.2689280275926285E0" upper="3.490658503988659E-1" velocity="${radians(80)}"/>
+            <origin rpy="${pi/2.0} 0.0 -0.0" xyz="0.5 0.0 -0.86"/>
+            <parent link="${prefix}link_1"/>
         </joint>
         <joint name="${prefix}joint_3" type="revolute">
-            <axis xyz="0.0 0.0 1.0" />
-            <child link="${prefix}link_3" />
-            <limit effort="15315.272850848E0" lower="-1.7453292519943295E0" upper="2.8797932657906435E0" velocity="${radians(75)}" />
-            <origin rpy="0.0 0.0 -${pi/2.0}" xyz="1.55 0.0 0.0" />
-            <parent link="${prefix}link_2" />
+            <axis xyz="0.0 0.0 1.0"/>
+            <child link="${prefix}link_3"/>
+            <limit effort="15315.272850848E0" lower="-1.7453292519943295E0" upper="2.8797932657906435E0" velocity="${radians(75)}"/>
+            <origin rpy="0.0 0.0 -${pi/2.0}" xyz="1.55 0.0 0.0"/>
+            <parent link="${prefix}link_2"/>
         </joint>
         <joint name="${prefix}joint_4" type="revolute">
-            <axis xyz="0.0 0.0 1.0" />
-            <child link="${prefix}link_4" />
-            <limit effort="4847.11596436905E0" lower="-6.1086523819801535E0" upper="6.1086523819801535E0" velocity="${radians(90)}" />
-            <origin rpy="${pi/2.0} 0.0 -0.0" xyz="0.18 0.0 0.0" />
-            <parent link="${prefix}link_3" />
+            <axis xyz="0.0 0.0 1.0"/>
+            <child link="${prefix}link_4"/>
+            <limit effort="4847.11596436905E0" lower="-6.1086523819801535E0" upper="6.1086523819801535E0" velocity="${radians(90)}"/>
+            <origin rpy="${pi/2.0} 0.0 -0.0" xyz="0.18 0.0 0.0"/>
+            <parent link="${prefix}link_3"/>
         </joint>
         <joint name="${prefix}joint_5" type="revolute">
-            <axis xyz="0.0 0.0 1.0" />
-            <child link="${prefix}link_5" />
-            <limit effort="4852.96953685247E0" lower="-2.0943951023931953E0" upper="2.0943951023931953E0" velocity="${radians(90)}" />
-            <origin rpy="-${pi/2.0} 0.0 -0.0" xyz="0.0 0.0 -1.0345" />
-            <parent link="${prefix}link_4" />
+            <axis xyz="0.0 0.0 1.0"/>
+            <child link="${prefix}link_5"/>
+            <limit effort="4852.96953685247E0" lower="-2.0943951023931953E0" upper="2.0943951023931953E0" velocity="${radians(90)}"/>
+            <origin rpy="-${pi/2.0} 0.0 -0.0" xyz="0.0 0.0 -1.0345"/>
+            <parent link="${prefix}link_4"/>
         </joint>
         <joint name="${prefix}joint_6" type="revolute">
-            <axis xyz="0.0 0.0 1.0" />
-            <child link="${prefix}link_6" />
-            <limit effort="2675.4449432041E0" lower="-6.1086523819801535E0" upper="6.1086523819801535E0" velocity="${radians(130)}" />
-            <origin rpy="${pi/2.0} 0.0 -0.0" xyz="0.0 0.0 0.0" />
-            <parent link="${prefix}link_5" />
+            <axis xyz="0.0 0.0 1.0"/>
+            <child link="${prefix}link_6"/>
+            <limit effort="2675.4449432041E0" lower="-6.1086523819801535E0" upper="6.1086523819801535E0" velocity="${radians(130)}"/>
+            <origin rpy="${pi/2.0} 0.0 -0.0" xyz="0.0 0.0 0.0"/>
+            <parent link="${prefix}link_5"/>
         </joint>
         <!-- ROS-Industrial 'base' frame - equivalent of 'KUKA ROBROOT'-->
         <link name="${prefix}base" />
         <joint name="${prefix}base_link-base" type="fixed">
-            <origin xyz="0 0 0" rpy="0 0 0" />
-            <parent link="${prefix}base_link" />
-            <child link="${prefix}base" />
+            <origin xyz="0 0 0" rpy="0 0 0"/>
+            <parent link="${prefix}base_link"/>
+            <child link="${prefix}base"/>
         </joint>
         <!-- ROS-Industrial 'flange' frame - attachment point for EEF models -->

File: kuka_fortec_support/urdf/kr_fortec_ros2_control.xacro (robot description, xacro)
@@ -1,5 +1,5 @@
 <?xml version="1.0" encoding="UTF-8"?>
 <robot xmlns:xacro="http://www.ros.org/wiki/xacro">
-  <xacro:macro name="kuka_fortec_ros2_control" params="name prefix use_fake_hardware:=false">
+  <xacro:macro name="kuka_fortec_ros2_control" params="name client_ip client_port prefix use_fake_hardware">
     <ros2_control name="${name}" type="system">
       <hardware>
@@ -10,9 +10,4 @@
         </xacro:if>
         <xacro:unless value="${use_fake_hardware}">
-          <!-- Read parameters from rsi_config  -->
-          <xacro:property name="rsi_config" value="$(find kuka_kss_rsi_driver)/config/driver_config.yaml" />
-          <xacro:property name="rsi_config_dict" value="${xacro.load_yaml(rsi_config)}"/>
-          <xacro:property name="client_ip" value="${rsi_config_dict['client_ip']}" />
-          <xacro:property name="client_port" value="${rsi_config_dict['client_port']}" />
           <plugin>kuka_kss_rsi_driver::KukaRSIHardwareInterface</plugin>
           <param name="client_ip">${client_ip}</param>
@@ -22,37 +17,37 @@
       <joint name="${prefix}joint_1">
         <command_interface name="position"/>
-      <state_interface name="position">
-        <param name="initial_value">0.0</param>
-      </state_interface>
+        <state_interface name="position">
+          <param name="initial_value">0.0</param>
+        </state_interface>
       </joint>
       <joint name="${prefix}joint_2">
         <command_interface name="position"/>
-      <state_interface name="position">
-        <param name="initial_value">0.0</param>
-      </state_interface>
+        <state_interface name="position">
+          <param name="initial_value">0.0</param>
+        </state_interface>
       </joint>
       <joint name="${prefix}joint_3">
         <command_interface name="position"/>
-      <state_interface name="position">
-        <param name="initial_value">0.0</param>
-      </state_interface>
+        <state_interface name="position">
+          <param name="initial_value">0.0</param>
+        </state_interface>
       </joint>
       <joint name="${prefix}joint_4">
         <command_interface name="position"/>
-      <state_interface name="position">
-        <param name="initial_value">0.0</param>
-      </state_interface>
+        <state_interface name="position">
+          <param name="initial_value">0.0</param>
+        </state_interface>
       </joint>
       <joint name="${prefix}joint_5">
         <command_interface name="position"/>
-      <state_interface name="position">
-        <param name="initial_value">0.0</param>
-      </state_interface>
+        <state_interface name="position">
+          <param name="initial_value">0.0</param>
+        </state_interface>
       </joint>
       <joint name="${prefix}joint_6">
         <command_interface name="position"/>
-      <state_interface name="position">
-        <param name="initial_value">0.0</param>
-      </state_interface>
+        <state_interface name="position">
+          <param name="initial_value">0.0</param>
+        </state_interface>
       </joint>
     </ros2_control>

Commit message: Add gpio config to kr fortec

File: kuka_fortec_support/urdf/kr560_r3100_2.urdf.xacro (robot description, xacro)
@@ -5,4 +5,5 @@
   <!-- Read additional arguments  -->
   <xacro:arg name="use_fake_hardware" default="false"/>
+  <xacro:arg name="use_gpio" default="true"/>
   <xacro:arg name="roundtrip_time" default="0"/>
   <xacro:arg name="client_ip" default="0.0.0.0"/>
@@ -16,5 +17,5 @@
   <xacro:arg name="pitch" default="0"/>
   <xacro:arg name="yaw" default="0"/>
-  <xacro:kuka_kr560_r3100_2_robot client_ip="$(arg client_ip)" client_port="$(arg client_port)" controller_ip="$(arg controller_ip)" prefix="$(arg prefix)" use_fake_hardware="$(arg use_fake_hardware)" roundtrip_time="$(arg roundtrip_time)">
+  <xacro:kuka_kr560_r3100_2_robot client_ip="$(arg client_ip)" client_port="$(arg client_port)" controller_ip="$(arg controller_ip)" prefix="$(arg prefix)" use_fake_hardware="$(arg use_fake_hardware)" use_gpio="$(arg use_gpio)" roundtrip_time="$(arg roundtrip_time)">
     <origin xyz="$(arg x) $(arg y) $(arg z)" rpy="$(arg roll) $(arg pitch) $(arg yaw)"/>
   </xacro:kuka_kr560_r3100_2_robot>

File: kuka_fortec_support/urdf/kr560_r3100_2_macro.xacro (robot description, xacro)
@@ -3,7 +3,7 @@
   <xacro:include filename="$(find kuka_fortec_support)/urdf/kr_fortec_ros2_control.xacro"/>
   <xacro:include filename="$(find kuka_fortec_support)/urdf/kr_fortec_transmission.xacro"/>
-  <xacro:macro name="kuka_kr560_r3100_2_robot" params="client_ip client_port controller_ip prefix use_fake_hardware roundtrip_time *origin">
+  <xacro:macro name="kuka_kr560_r3100_2_robot" params="client_ip client_port controller_ip prefix use_fake_hardware use_gpio roundtrip_time *origin">
     <!-- ros2 control instance -->
-    <xacro:kuka_fortec_ros2_control name="${prefix}kr560_r3100_2" client_ip="${client_ip}" client_port="${client_port}" controller_ip="${controller_ip}" prefix="${prefix}" use_fake_hardware="${use_fake_hardware}" roundtrip_time="${roundtrip_time}"/>
+    <xacro:kuka_fortec_ros2_control name="${prefix}kr560_r3100_2" client_ip="${client_ip}" client_port="${client_port}" controller_ip="${controller_ip}" prefix="${prefix}" use_fake_hardware="${use_fake_hardware}" use_gpio="${use_gpio}" roundtrip_time="${roundtrip_time}"/>
     <link name="world"/>
     <link name="${prefix}base_link">

File: kuka_fortec_support/urdf/kr_fortec_ros2_control.xacro (robot description, xacro)
@@ -1,5 +1,5 @@
 <?xml version="1.0" encoding="UTF-8"?>
 <robot xmlns:xacro="http://www.ros.org/wiki/xacro">
-  <xacro:macro name="kuka_fortec_ros2_control" params="name client_ip client_port controller_ip prefix use_fake_hardware roundtrip_time">
+  <xacro:macro name="kuka_fortec_ros2_control" params="name client_ip client_port controller_ip prefix use_fake_hardware use_gpio roundtrip_time">
     <ros2_control name="${name}" type="system">
       <hardware>
@@ -54,4 +54,8 @@
         </state_interface>
       </joint>
+      <xacro:if value="${use_gpio}">
+        <xacro:include filename="$(find kuka_fortec_support)/urdf/kr_fortec_gpio_config.xacro"/>
+        <xacro:kr_fortec_gpio_config/>
+      </xacro:if>
     </ros2_control>
   </xacro:macro>
