Commit message: remove world + world-base_link from macro

File: kuka_fortec_support/urdf/kr360_r2830_macro.xacro (robot description, xacro)
@@ -138,5 +138,4 @@
     </link>
     <link name="${prefix}tool0"/>
-    <link name="world"/>
     <joint name="${prefix}base_link-base" type="fixed">
       <child link="${prefix}base"/>
@@ -195,9 +194,4 @@
       <parent link="${prefix}link_6"/>
     </joint>
-    <joint name="${prefix}world-base_link" type="fixed">
-      <child link="${prefix}base_link"/>
-      <parent link="world"/>
-      <xacro:insert_block name="origin"/>
-    </joint>
   </xacro:macro>
 </robot>
