Commit message: Add world-base link as fixed

File: kuka_fortec_support/urdf/kr360_r2830.urdf.xacro (robot description, xacro)
@@ -11,4 +11,5 @@
   <xacro:arg name="client_ip" default="0.0.0.0"/>
   <xacro:arg name="client_port" default="59152"/>
+  <xacro:arg name="mxa_client_port" default="1337"/>
   <xacro:arg name="controller_ip" default="0.0.0.0"/>
   <xacro:arg name="verify_robot_model" default="true"/>
@@ -21,7 +22,18 @@
   <xacro:arg name="yaw" default="0"/>
   <xacro:kuka_fortec_ros2_control name="$(arg prefix)kr360_r2830" driver_version="$(arg driver_version)" client_ip="$(arg client_ip)" client_port="$(arg client_port)" controller_ip="$(arg controller_ip)" prefix="$(arg prefix)" mode="$(arg mode)" use_gpio="$(arg use_gpio)" roundtrip_time="$(arg roundtrip_time)" verify_robot_model="$(arg verify_robot_model)"/>
+  <ext_axes_ros2_control_joints/>
+  </xacro:kuka_fortec_ros2_control>
+  <!-- world link -->
+  <link name="world"/>
+  <!-- robot links, joints -->
   <xacro:kuka_kr360_r2830_robot prefix="$(arg prefix)" package_name="kuka_fortec_support">
     <origin xyz="$(arg x) $(arg y) $(arg z)" rpy="$(arg roll) $(arg pitch) $(arg yaw)"/>
   </xacro:kuka_kr360_r2830_robot>
+   <!-- default world - base_link joint -->
+  <joint name="$(arg prefix)world-base_link" type="fixed">
+    <parent link="world"/>
+    <child link="$(arg prefix)base_link"/>
+    <origin xyz="$(arg x) $(arg y) $(arg z)" rpy="$(arg roll) $(arg pitch) $(arg yaw)"/>
+  </joint>
   <version>2025-09-17_13-38-40</version>
 </robot>

Commit message: Remove wrong origin tag

File: kuka_fortec_support/urdf/kr360_r2830.urdf.xacro (robot description, xacro)
@@ -27,8 +27,6 @@
   <link name="world"/>
   <!-- robot links, joints -->
-  <xacro:kuka_kr360_r2830_robot prefix="$(arg prefix)" package_name="kuka_fortec_support">
-    <origin xyz="$(arg x) $(arg y) $(arg z)" rpy="$(arg roll) $(arg pitch) $(arg yaw)"/>
-  </xacro:kuka_kr360_r2830_robot>
-   <!-- default world - base_link joint -->
+  <xacro:kuka_kr360_r2830_robot prefix="$(arg prefix)" package_name="kuka_fortec_support"/>
+  <!-- default world - base_link joint -->
   <joint name="$(arg prefix)world-base_link" type="fixed">
     <parent link="world"/>

Commit message: URDF fix

File: kuka_fortec_support/urdf/kr360_r2830.urdf.xacro (robot description, xacro)
@@ -21,5 +21,5 @@
   <xacro:arg name="pitch" default="0"/>
   <xacro:arg name="yaw" default="0"/>
-  <xacro:kuka_fortec_ros2_control name="$(arg prefix)kr360_r2830" driver_version="$(arg driver_version)" client_ip="$(arg client_ip)" client_port="$(arg client_port)" controller_ip="$(arg controller_ip)" prefix="$(arg prefix)" mode="$(arg mode)" use_gpio="$(arg use_gpio)" roundtrip_time="$(arg roundtrip_time)" verify_robot_model="$(arg verify_robot_model)">
+  <xacro:kuka_fortec_ros2_control name="$(arg prefix)kr360_r2830" driver_version="$(arg driver_version)" client_ip="$(arg client_ip)" client_port="$(arg client_port)" mxa_client_port="$(arg mxa_client_port)" controller_ip="$(arg controller_ip)" prefix="$(arg prefix)" mode="$(arg mode)" use_gpio="$(arg use_gpio)" roundtrip_time="$(arg roundtrip_time)" verify_robot_model="$(arg verify_robot_model)">
     <ext_axes_ros2_control_joints/>
   </xacro:kuka_fortec_ros2_control>

File: kuka_fortec_support/urdf/kr360_r2830_macro.xacro (robot description, xacro)
@@ -1,5 +1,5 @@
-<?xml version="1.0"?>
+<?xml version="1.0" encoding="UTF-8"?>
 <robot xmlns:xacro="http://www.ros.org/wiki/xacro" name="kr360_r2830">
-  <xacro:macro name="kuka_kr360_r2830_robot" params="prefix package_name *origin">
+  <xacro:macro name="kuka_kr360_r2830_robot" params="prefix package_name">
     <link name="${prefix}base"/>
     <link name="${prefix}base_link">
