Commit message: update xacro files

File: kuka_mobile_robot_support/ros2_control/mrob_kuka.ros2_control.xacro (robot description, xacro)
@@ -1,28 +1,39 @@
 <?xml version="1.0"?>
 <robot xmlns:xacro="http://www.ros.org/wiki/xacro">
-  <xacro:macro name="mrob_kuka_ros2_control" params="name prefix client_ip controller_ip control_mode consequent_lost_packets lost_packets_in_timeframe timeframe_ms use_fake_hardware:=false gazebo_sim:=false">
+  <xacro:macro name="mrob_kuka_ros2_control" params="name prefix client_ip controller_ip use_fake_hardware qos_config_file roundtrip_time">
     <ros2_control name="${name}" type="system">
       <hardware>
         <xacro:if value="${use_fake_hardware}">
-          <plugin>mock_components/GenericSystem</plugin>
-          <param name="fake_sensor_commands">false</param>
+          <plugin>kuka_mock_hardware_interface::KukaMockHardwareInterface</plugin>
+          <param name="cycle_time_ms">4</param>
+          <param name="roundtrip_time_micro">${roundtrip_time}</param>
+          <param name="mock_sensor_commands">false</param>
           <param name="state_following_offset">0.0</param>
+          <!--<xacro:if value="${gazebo_sim}">
+            <plugin>kuka_eac::KukaEACHardwareInterface</plugin>
+            <plugin>gazebo_ros2_control/GazeboSystem</plugin>
+          </xacro:if> -->
         </xacro:if>
         <xacro:unless value="${use_fake_hardware}">
-          <xacro:if value="${gazebo_sim}">
-            <plugin>gazebo_ros2_control/GazeboSystem</plugin>
+          <!-- Read QoS profile parameters  -->
+          <xacro:if value="${qos_config_file == ''}">
+            <xacro:property name="qos_config" value="$(find kuka_iiqka_eac_driver)/config/qos_config.yaml"/>
           </xacro:if>
-          <xacro:unless value="${gazebo_sim}">
-            <plugin>kuka_rox::KukaRoXHardwareInterface</plugin>
-            <param name="client_ip">${client_ip}</param>
-            <param name="controller_ip">${controller_ip}</param>
-            <param name="control_mode">${control_mode}</param>
-            <param name="consequent_lost_packets">${consequent_lost_packets}</param>
-            <param name="lost_packets_in_timeframe">${lost_packets_in_timeframe}</param>
-            <param name="timeframe_ms">${timeframe_ms}</param>
+          <xacro:unless value="${qos_config_file == ''}">
+            <xacro:property name="qos_config" value="${qos_config_file}"/>
           </xacro:unless>
+          <xacro:property name="qos_config_dict" value="${xacro.load_yaml(qos_config)}"/>
+          <xacro:property name="consequent_lost_packets" value="${qos_config_dict['rt_packet_loss_profile']['consequent_lost_packets']}"/>
+          <xacro:property name="lost_packets_in_timeframe" value="${qos_config_dict['rt_packet_loss_profile']['lost_packets_in_timeframe']}"/>
+          <xacro:property name="timeframe_ms" value="${qos_config_dict['rt_packet_loss_profile']['timeframe_ms']}"/>
+          <plugin>kuka_eac::KukaEACHardwareInterface</plugin>
+          <param name="client_ip">${client_ip}</param>
+          <param name="controller_ip">${controller_ip}</param>
+          <param name="consequent_lost_packets">${consequent_lost_packets}</param>
+          <param name="lost_packets_in_timeframe">${lost_packets_in_timeframe}</param>
+          <param name="timeframe_ms">${timeframe_ms}</param>
         </xacro:unless>
-        <plugin>gazebo_ros2_control/GazeboSystem</plugin>
       </hardware>
+      <!-- define joints and command/state interfaces for each joint -->
       <joint name="${prefix}twist/linear">
         <command_interface name="x"/>
@@ -30,6 +41,9 @@
         <command_interface name="z"/>
         <state_interface name="x"/>
+          <param name="initial_value">0.0</param>
         <state_interface name="y"/>
+          <param name="initial_value">0.0</param>
         <state_interface name="z"/>
+          <param name="initial_value">0.0</param>
       </joint>
       <joint name="${prefix}twist/angular">
@@ -38,8 +52,11 @@
         <command_interface name="z"/>
         <state_interface name="x"/>
+          <param name="initial_value">0.0</param>
         <state_interface name="y"/>
+          <param name="initial_value">0.0</param>
         <state_interface name="z"/>
+          <param name="initial_value">0.0</param>
       </joint>
-      <joint name="left_wheel_motor">
+      <!--<joint name="left_wheel_motor">
           <command_interface name="velocity">
             <param name="min">-1</param>
@@ -47,5 +64,7 @@
           </command_interface>
           <state_interface name="position"/>
+            <param name="initial_value">0.0</param>
           <state_interface name="velocity"/>
+            <param name="initial_value">0.0</param>
         </joint>
         <joint name="right_wheel_motor">
@@ -55,12 +74,14 @@
           </command_interface>
           <state_interface name="position"/>
+            <param name="initial_value">0.0</param>
           <state_interface name="velocity"/>
-        </joint>
+            <param name="initial_value">0.0</param>
+        </joint>  -->
     </ros2_control>
- <xacro:if value="${gazebo_sim}">
-<!-- config file with gazebo parameters-->
+ <!--<xacro:if value="${gazebo_sim}">
+ config file with gazebo parameters
             <xacro:include filename="$(find kuka_mobile_robot_support)/gazebo/diffbot.gazebo.xacro" />
             <xacro:diffbot_gazebo  prefix="" ros2_control_sim="true"/>
- </xacro:if>
+ </xacro:if>-->
   </xacro:macro>
 </robot>

File: kuka_mobile_robot_support/urdf/KUKA_MR.urdf.xacro (robot description, xacro)
@@ -1,39 +1,24 @@
 <?xml version="1.0"?>
-<!-- Basic differential drive mobile base -->
-<robot xmlns:xacro="http://www.ros.org/wiki/xacro" name="diffdrive_robot">
-  <xacro:arg name="prefix" default="" />
-<!-- Import diffbot urdf file  -->
+<!-- Basic KUKA mobile base -->
+<robot xmlns:xacro="http://www.ros.org/wiki/xacro" name="KUKA_MR">
+<!-- Import mrob urdf file  -->
   <!-- <xacro:include filename="$(find kuka_mobile_robot_support)/urdf/diffbot_kuka_macro.xacro" /> -->
   <xacro:include filename="$(find kuka_mobile_robot_support)/urdf/mrob_kuka_macro.xacro" />
-  <!-- Read parameters from eci_config  -->
-  <xacro:property name="eci_config" value="$(find kuka_rox_hw_interface)/config/eci_config.yaml" />
-  <xacro:property name="eci_config_dict" value="${xacro.load_yaml(eci_config)}"/>
-  <xacro:property name="control_mode" value="${eci_config_dict['robot_manager']['ros__parameters']['control_mode']}" />
-  <xacro:property name="client_ip" value="${eci_config_dict['robot_manager']['ros__parameters']['client_ip']}" />
-  <xacro:property name="controller_ip" value="${eci_config_dict['robot_manager']['ros__parameters']['controller_ip']}" />
-  <!-- Read QoS profile parameters  -->
-  <xacro:property name="qos_config" value="$(find kuka_rox_hw_interface)/config/qos_profiles.yaml" />
-  <xacro:property name="qos_config_dict" value="${xacro.load_yaml(qos_config)}"/>
-  <xacro:property name="consequent_lost_packets" value="${qos_config_dict['rt_packet_loss_profile']['consequent_lost_packets']}" />
-  <xacro:property name="lost_packets_in_timeframe" value="${qos_config_dict['rt_packet_loss_profile']['lost_packets_in_timeframe']}" />
-  <xacro:property name="timeframe_ms" value="${qos_config_dict['rt_packet_loss_profile']['timeframe_ms']}" />
-  <!-- <xacro:diffbot_kuka_robot prefix=""
-                  client_ip="${client_ip}"
-                  controller_ip="${controller_ip}"
-                  control_mode="${control_mode}"
-                  consequent_lost_packets="${consequent_lost_packets}"
-                  lost_packets_in_timeframe="${lost_packets_in_timeframe}"
-                  timeframe_ms="${timeframe_ms}"/>  -->
-  <!-- Read additional arguments  -->
-  <xacro:arg name="use_fake_hardware" default="false" />
+   <!-- Read additional arguments  -->
   <xacro:arg name="gazebo_sim" default="false" />
-  <xacro:mrob_kuka prefix=""
-                  client_ip="${client_ip}"
-                  controller_ip="${controller_ip}"
-                  control_mode="${control_mode}"
-                  consequent_lost_packets="${consequent_lost_packets}"
-                  lost_packets_in_timeframe="${lost_packets_in_timeframe}"
-                  timeframe_ms="${timeframe_ms}"
-                  use_fake_hardware="$(arg use_fake_hardware)"
-                  gazebo_sim="$(arg gazebo_sim)" />
+  <xacro:arg name="prefix" default=""/>
+  <xacro:arg name="controller_ip" default="0.0.0.0"/>
+  <xacro:arg name="client_ip" default="0.0.0.0"/>
+  <xacro:arg name="use_fake_hardware" default="false"/>
+  <xacro:arg name="roundtrip_time" default="0"/>
+  <xacro:arg name="qos_config_file" default=""/>
+  <xacro:arg name="x" default="0"/>
+  <xacro:arg name="y" default="0"/>
+  <xacro:arg name="z" default="0"/>
+  <xacro:arg name="roll" default="0"/>
+  <xacro:arg name="pitch" default="0"/>
+  <xacro:arg name="yaw" default="0"/>
+  <xacro:mrob_kuka prefix="$(arg prefix)" controller_ip="$(arg controller_ip)" client_ip="$(arg client_ip)" use_fake_hardware="$(arg use_fake_hardware)" roundtrip_time="$(arg roundtrip_time)" qos_config_file="$(arg qos_config_file)">
+    <origin xyz="$(arg x) $(arg y) $(arg z)" rpy="$(arg roll) $(arg pitch) $(arg yaw)"/>
+  </xacro:mrob_kuka>
 </robot>

File: kuka_mobile_robot_support/urdf/mrob_kuka_macro.xacro (robot description, xacro)
@@ -4,18 +4,8 @@
   <xacro:include filename="$(find kuka_mobile_robot_support)/ros2_control/mrob_kuka.ros2_control.xacro" />
   <xacro:include filename="$(find kuka_resources)/urdf/common_materials.xacro"/>
-  <xacro:macro name="mrob_kuka" params="prefix client_ip controller_ip control_mode consequent_lost_packets lost_packets_in_timeframe timeframe_ms use_fake_hardware:=false gazebo_sim:=false">
+  <xacro:macro name="mrob_kuka" params="prefix controller_ip client_ip use_fake_hardware roundtrip_time qos_config_file *origin">
     <!-- ros2 control instance -->
-    <xacro:mrob_kuka_ros2_control
-      name="KUKA_MR"
-      prefix="${prefix}"
-      client_ip="${client_ip}"
-      controller_ip="${controller_ip}"
-      control_mode="${control_mode}"
-      consequent_lost_packets="${consequent_lost_packets}"
-      lost_packets_in_timeframe="${lost_packets_in_timeframe}"
-      timeframe_ms="${timeframe_ms}"
-      use_fake_hardware="${use_fake_hardware}"
-      gazebo_sim="${gazebo_sim}"/>
-     <joint name="odom_joint" type="planar">
+    <xacro:mrob_kuka_ros2_control name="KUKA_MR" prefix="${prefix}" client_ip="${client_ip}" controller_ip="${controller_ip}" use_fake_hardware="${use_fake_hardware}" roundtrip_time="${roundtrip_time}" qos_config_file="${qos_config_file}"/>
+     <joint name="odom_joint" type="fixed">
             <axis xyz="0.0 1.0 0.0"/>
             <parent link="odom" />
