Commit message: renamed package and meshes, deleted unnecesary files

File: kuka_kmr_iisy_support/urdf/kmr_iisy.urdf.xacro (robot description, xacro)
@@ -1,10 +1,8 @@
 <?xml version="1.0"?>
 <!-- Basic KUKA mobile base -->
-<robot xmlns:xacro="http://www.ros.org/wiki/xacro" name="KUKA_MR">
+<robot xmlns:xacro="http://www.ros.org/wiki/xacro" name="kmr_iisy">
 <!-- Import mrob urdf file  -->
-  <!-- <xacro:include filename="$(find kuka_mobile_robot_support)/urdf/diffbot_kuka_macro.xacro" /> -->
-  <xacro:include filename="$(find kuka_mobile_robot_support)/urdf/mrob_kuka_macro.xacro" />
+  <xacro:include filename="$(find kuka_kmr_iisy_support)/urdf/kmr_iisy_macro.xacro" />
    <!-- Read additional arguments  -->
-  <xacro:arg name="gazebo_sim" default="false" />
   <xacro:arg name="prefix" default=""/>
   <xacro:arg name="controller_ip" default="0.0.0.0"/>

File: kuka_kmr_iisy_support/urdf/kmr_iisy_macro.xacro (robot description, xacro)
@@ -2,18 +2,18 @@
 <robot xmlns:xacro="http://www.ros.org/wiki/xacro" name="">
   <!-- include helper xacros -->
-  <xacro:include filename="$(find kuka_mobile_robot_support)/ros2_control/mrob_kuka.ros2_control.xacro" />
+  <xacro:include filename="$(find kuka_kmr_iisy_support)/urdf/kmr_iisy_ros2_control.xacro" />
   <xacro:include filename="$(find kuka_resources)/urdf/common_materials.xacro"/>
   <xacro:macro name="mrob_kuka" params="prefix controller_ip client_ip use_fake_hardware roundtrip_time qos_config_file *origin">
     <!-- ros2 control instance -->
-    <xacro:mrob_kuka_ros2_control name="KUKA_MR" prefix="${prefix}" client_ip="${client_ip}" controller_ip="${controller_ip}" use_fake_hardware="${use_fake_hardware}" roundtrip_time="${roundtrip_time}" qos_config_file="${qos_config_file}"/>
-     <joint name="odom_joint" type="fixed">
+    <xacro:mrob_kuka_ros2_control name="kmr_iisy" prefix="${prefix}" client_ip="${client_ip}" controller_ip="${controller_ip}" use_fake_hardware="${use_fake_hardware}" roundtrip_time="${roundtrip_time}" qos_config_file="${qos_config_file}"/>
+     <joint name="twist" type="fixed">
             <axis xyz="0.0 1.0 0.0"/>
             <parent link="odom" />
-            <child link="generic_mr_body_dummy" />
+            <child link="kmr_iisy_body_dummy" />
             <origin xyz="0 0 0" rpy="0 0 0" />
           </joint>
-      <joint name="generic_mr_body_dummy" type="fixed">
-            <parent link="generic_mr_body_dummy" />
-            <child link="generic_mr_body" />
+      <joint name="kmr_iisy_body_dummy" type="fixed">
+            <parent link="kmr_iisy_body_dummy" />
+            <child link="kmr_iisy_body" />
             <origin xyz="0 0 0" rpy="0 0 0" />
           </joint>
@@ -29,5 +29,5 @@
           <limit effort="5.0E2" velocity="1.0E2"/>
           <origin rpy="-0.0 0.0 -0.0" xyz="0.0 0.325 0.028"/>  <!-- 0.06 -->
-          <parent link="generic_mr_body"/>
+          <parent link="kmr_iisy_body"/>
         </joint>
         <joint name="right_wheel_motor" type="fixed">
@@ -36,5 +36,5 @@
           <limit effort="5.0E2" velocity="1.0E1"/>
           <origin rpy="-0.0 0.0 -0.0" xyz="0.0 -0.325 0.028"/>  <!-- 0.06 -->
-          <parent link="generic_mr_body"/>
+          <parent link="kmr_iisy_body"/>
         </joint>
         <joint name="caster_base_fl_joint" type="fixed">
@@ -42,5 +42,5 @@
           <child link="caster_base_fl_link"/>
           <origin rpy="-0.0 0.0 -0.0" xyz="0.48 0.27 0.055"/>
-          <parent link="generic_mr_body"/>
+          <parent link="kmr_iisy_body"/>
         </joint>
         <joint name="caster_base_rl_joint" type="fixed">
@@ -48,5 +48,5 @@
           <child link="caster_base_rl_link"/>
           <origin rpy="-0.0 0.0 -0.0" xyz="0.48 -0.27 0.055"/>
-          <parent link="generic_mr_body"/>
+          <parent link="kmr_iisy_body"/>
         </joint>
         <joint name="caster_base_bl_joint" type="fixed">
@@ -54,5 +54,5 @@
           <child link="caster_base_bl_link"/>
           <origin rpy="-0.0 0.0 -0.0" xyz="-0.48 0.27 0.055"/>
-          <parent link="generic_mr_body"/>
+          <parent link="kmr_iisy_body"/>
         </joint>
         <joint name="caster_base_br_joint" type="fixed">
@@ -60,5 +60,5 @@
           <child link="caster_base_br_link"/>
           <origin rpy="-0.0 0.0 -0.0" xyz="-0.48 -0.27 0.055"/>
-          <parent link="generic_mr_body"/>
+          <parent link="kmr_iisy_body"/>
         </joint>
         <joint name="caster_wheel_fl_joint" type="fixed">
@@ -80,10 +80,10 @@
           <parent link="caster_base_bl_link"/>
         </joint>
-        <link name="generic_mr_body_dummy"/>
+        <link name="kmr_iisy_body_dummy"/>
         <link name="odom"/>
-        <link name="generic_mr_body">
-          <collision>
-            <geometry>
-              <mesh filename="package://kuka_mobile_robot_support/meshes/37156934227.stl"/>
+        <link name="kmr_iisy_body">
+          <collision>
+            <geometry>
+              <mesh filename="package://kuka_kmr_iisy_support/meshes/collision/body.stl"/>
             </geometry>
             <origin rpy="-0.0 0.0 -0.0" xyz="0.0 0.0 0.0"/>
@@ -96,7 +96,8 @@
           <visual>
             <geometry>
-              <mesh filename="package://kuka_mobile_robot_support/meshes/37156942086.stl"/>
-            </geometry>
-            <origin rpy="-0.0 0.0 -0.0" xyz="0.0 0.0 0.0"/>
+              <mesh filename="package://kuka_kmr_iisy_support/meshes/visual/body.stl"/>
+            </geometry>
+            <origin rpy="-0.0 0.0 -0.0" xyz="0.0 0.0 0.0"/>
+            <xacro:material_kuka_ral_pure_white/>
           </visual>
         </link>
@@ -104,18 +105,19 @@
           <collision>
             <geometry>
-              <mesh filename="package://kuka_mobile_robot_support/meshes/37149321854.stl"/>
-            </geometry>
-            <origin rpy="1.5707963267948963 0.0 -0.0" xyz="0.0 0.0 0.0"/>
-          </collision>
-          <inertial>
-            <inertia ixx="1.0E-4" ixy="0.0" ixz="0.0" iyy="1.0E-4" iyz="0.0" izz="1.0E-4"/>
-            <mass value="1.0E-1"/>
-            <origin rpy="-0.0 0.0 -0.0" xyz="0.0 0.0 0.0"/>
-          </inertial>
-          <visual>
-            <geometry>
-              <mesh filename="package://kuka_mobile_robot_support/meshes/37149329314.stl"/>
-            </geometry>
-            <origin rpy="1.5707963267948963 0.0 -0.0" xyz="0.0 0.0 0.0"/>
+              <mesh filename="package://kuka_kmr_iisy_support/meshes/collision/caster_wheel_link.stl"/>
+            </geometry>
+            <origin rpy="1.5707963267948963 0.0 -0.0" xyz="0.0 0.0 0.0"/>
+          </collision>
+          <inertial>
+            <inertia ixx="1.0E-4" ixy="0.0" ixz="0.0" iyy="1.0E-4" iyz="0.0" izz="1.0E-4"/>
+            <mass value="1.0E-1"/>
+            <origin rpy="-0.0 0.0 -0.0" xyz="0.0 0.0 0.0"/>
+          </inertial>
+          <visual>
+            <geometry>
+              <mesh filename="package://kuka_kmr_iisy_support/meshes/visual/caster_wheel_link.stl"/>
+            </geometry>
+            <origin rpy="1.5707963267948963 0.0 -0.0" xyz="0.0 0.0 0.0"/>
+            <xacro:material_kuka_ral_gray_white/>
           </visual>
         </link>
@@ -123,5 +125,5 @@
           <collision>
             <geometry>
-              <mesh filename="package://kuka_mobile_robot_support/meshes/37153975930.stl"/>
+              <mesh filename="package://kuka_kmr_iisy_support/meshes/collision/left_wheel.stl"/>
             </geometry>
             <origin rpy="0.0 0.0 -1.5707963267948963" xyz="0.0 -0.02 0.0"/>
@@ -134,7 +136,8 @@
           <visual>
             <geometry>
-              <mesh filename="package://kuka_mobile_robot_support/meshes/37153983406.stl"/>
+              <mesh filename="package://kuka_kmr_iisy_support/meshes/visual/left_wheel.stl"/>
             </geometry>
             <origin rpy="0.0 0.0 -1.5707963267948963" xyz="0.0 -0.02 0.0"/>
+             <xacro:material_kuka_black/>
           </visual>
         </link>
@@ -142,18 +145,19 @@
           <collision>
             <geometry>
-              <mesh filename="package://kuka_mobile_robot_support/meshes/37153528620.stl"/>
-            </geometry>
-            <origin rpy="-0.0 0.0 -0.0" xyz="0.0 0.0 0.0"/>
-          </collision>
-          <inertial>
-            <inertia ixx="1.0E-4" ixy="0.0" ixz="0.0" iyy="1.0E-4" iyz="0.0" izz="1.0E-4"/>
-            <mass value="1.0E-1"/>
-            <origin rpy="-0.0 0.0 -0.0" xyz="0.0 0.0 0.0"/>
-          </inertial>
-          <visual>
-            <geometry>
-              <mesh filename="package://kuka_mobile_robot_support/meshes/37153537063.stl"/>
-            </geometry>
-            <origin rpy="-0.0 0.0 -0.0" xyz="0.0 0.0 0.0"/>
+              <mesh filename="package://kuka_kmr_iisy_support/meshes/collision/caster_base_fl_link.stl"/>
+            </geometry>
+            <origin rpy="-0.0 0.0 -0.0" xyz="0.0 0.0 0.0"/>
+          </collision>
+          <inertial>
+            <inertia ixx="1.0E-4" ixy="0.0" ixz="0.0" iyy="1.0E-4" iyz="0.0" izz="1.0E-4"/>
+            <mass value="1.0E-1"/>
+            <origin rpy="-0.0 0.0 -0.0" xyz="0.0 0.0 0.0"/>
+          </inertial>
+          <visual>
+            <geometry>
+              <mesh filename="package://kuka_kmr_iisy_support/meshes/visual/caster_base_fl_link.stl"/>
+            </geometry>
+            <origin rpy="-0.0 0.0 -0.0" xyz="0.0 0.0 0.0"/>
+            <xacro:material_kuka_ral_gray_white/>
           </visual>
         </link>
@@ -161,18 +165,19 @@
           <collision>
             <geometry>
-              <mesh filename="package://kuka_mobile_robot_support/meshes/37149321854.stl"/>
-            </geometry>
-            <origin rpy="1.5707963267948963 0.0 -0.0" xyz="0.0 0.0 0.0"/>
-          </collision>
-          <inertial>
-            <inertia ixx="1.0E-4" ixy="0.0" ixz="0.0" iyy="1.0E-4" iyz="0.0" izz="1.0E-4"/>
-            <mass value="1.0E-1"/>
-            <origin rpy="-0.0 0.0 -0.0" xyz="0.0 0.0 0.0"/>
-          </inertial>
-          <visual>
-            <geometry>
-              <mesh filename="package://kuka_mobile_robot_support/meshes/37149329314.stl"/>
-            </geometry>
-            <origin rpy="1.5707963267948963 0.0 -0.0" xyz="0.0 0.0 0.0"/>
+              <mesh filename="package://kuka_kmr_iisy_support/meshes/collision/caster_wheel_link.stl"/>
+            </geometry>
+            <origin rpy="1.5707963267948963 0.0 -0.0" xyz="0.0 0.0 0.0"/>
+          </collision>
+          <inertial>
+            <inertia ixx="1.0E-4" ixy="0.0" ixz="0.0" iyy="1.0E-4" iyz="0.0" izz="1.0E-4"/>
+            <mass value="1.0E-1"/>
+            <origin rpy="-0.0 0.0 -0.0" xyz="0.0 0.0 0.0"/>
+          </inertial>
+          <visual>
+            <geometry>
+              <mesh filename="package://kuka_kmr_iisy_support/meshes/visual/caster_wheel_link.stl"/>
+            </geometry>
+            <origin rpy="1.5707963267948963 0.0 -0.0" xyz="0.0 0.0 0.0"/>
+            <xacro:material_kuka_ral_gray_white/>
           </visual>
         </link>
@@ -180,18 +185,19 @@
           <collision>
             <geometry>
-              <mesh filename="package://kuka_mobile_robot_support/meshes/37153636399.stl"/>
-            </geometry>
-            <origin rpy="-0.0 0.0 -0.0" xyz="0.0 0.0 0.0"/>
-          </collision>
-          <inertial>
-            <inertia ixx="1.0E-4" ixy="0.0" ixz="0.0" iyy="1.0E-4" iyz="0.0" izz="1.0E-4"/>
-            <mass value="1.0E-1"/>
-            <origin rpy="-0.0 0.0 -0.0" xyz="0.0 0.0 0.0"/>
-          </inertial>
-          <visual>
-            <geometry>
-              <mesh filename="package://kuka_mobile_robot_support/meshes/37153643851.stl"/>
-            </geometry>
-            <origin rpy="-0.0 0.0 -0.0" xyz="0.0 0.0 0.0"/>
+              <mesh filename="package://kuka_kmr_iisy_support/meshes/collision/caster_base_rl_link.stl"/>
+            </geometry>
+            <origin rpy="-0.0 0.0 -0.0" xyz="0.0 0.0 0.0"/>
+          </collision>
+          <inertial>
+            <inertia ixx="1.0E-4" ixy="0.0" ixz="0.0" iyy="1.0E-4" iyz="0.0" izz="1.0E-4"/>
+            <mass value="1.0E-1"/>
+            <origin rpy="-0.0 0.0 -0.0" xyz="0.0 0.0 0.0"/>
+          </inertial>
+          <visual>
+            <geometry>
+              <mesh filename="package://kuka_kmr_iisy_support/meshes/visual/caster_base_rl_link.stl"/>
+            </geometry>
+            <origin rpy="-0.0 0.0 -0.0" xyz="0.0 0.0 0.0"/>
+            <xacro:material_kuka_ral_gray_white/>
           </visual>
         </link>
@@ -199,5 +205,5 @@
           <collision>
             <geometry>
-              <mesh filename="package://kuka_mobile_robot_support/meshes/37154306984.stl"/>
+              <mesh filename="package://kuka_kmr_iisy_support/meshes/collision/right_wheel.stl"/>
             </geometry>
             <origin rpy="-0.0 0.0 1.5707963267948963" xyz="0.0 0.02 0.0"/>
@@ -210,7 +216,8 @@
           <visual>
             <geometry>
-              <mesh filename="package://kuka_mobile_robot_support/meshes/37154317878.stl"/>
+              <mesh filename="package://kuka_kmr_iisy_support/meshes/visual/right_wheel.stl"/>
             </geometry>
             <origin rpy="-0.0 0.0 1.5707963267948963" xyz="0.0 0.02 0.0"/>
+            <xacro:material_kuka_black/>
           </visual>
         </link>
@@ -218,18 +225,19 @@
           <collision>
             <geometry>
-              <mesh filename="package://kuka_mobile_robot_support/meshes/37149321854.stl"/>
-            </geometry>
-            <origin rpy="1.5707963267948963 0.0 -0.0" xyz="0.0 0.0 0.0"/>
-          </collision>
-          <inertial>
-            <inertia ixx="1.0E-4" ixy="0.0" ixz="0.0" iyy="1.0E-4" iyz="0.0" izz="1.0E-4"/>
-            <mass value="1.0E-1"/>
-            <origin rpy="-0.0 0.0 -0.0" xyz="0.0 0.0 0.0"/>
-          </inertial>
-          <visual>
-            <geometry>
-              <mesh filename="package://kuka_mobile_robot_support/meshes/37149329314.stl"/>
-            </geometry>
-            <origin rpy="1.5707963267948963 0.0 -0.0" xyz="0.0 0.0 0.0"/>
+              <mesh filename="package://kuka_kmr_iisy_support/meshes/collision/caster_wheel_link.stl"/>
+            </geometry>
+            <origin rpy="1.5707963267948963 0.0 -0.0" xyz="0.0 0.0 0.0"/>
+          </collision>
+          <inertial>
+            <inertia ixx="1.0E-4" ixy="0.0" ixz="0.0" iyy="1.0E-4" iyz="0.0" izz="1.0E-4"/>
+            <mass value="1.0E-1"/>
+            <origin rpy="-0.0 0.0 -0.0" xyz="0.0 0.0 0.0"/>
+          </inertial>
+          <visual>
+            <geometry>
+              <mesh filename="package://kuka_kmr_iisy_support/meshes/visual/caster_wheel_link.stl"/>
+            </geometry>
+            <origin rpy="1.5707963267948963 0.0 -0.0" xyz="0.0 0.0 0.0"/>
+            <xacro:material_kuka_ral_gray_white/>
           </visual>
         </link>
@@ -237,18 +245,19 @@
           <collision>
             <geometry>
-              <mesh filename="package://kuka_mobile_robot_support/meshes/37152976775.stl"/>
-            </geometry>
-            <origin rpy="-0.0 0.0 -0.0" xyz="0.0 0.0 0.0"/>
-          </collision>
-          <inertial>
-            <inertia ixx="1.0E-4" ixy="0.0" ixz="0.0" iyy="1.0E-4" iyz="0.0" izz="1.0E-4"/>
-            <mass value="1.0E-1"/>
-            <origin rpy="-0.0 0.0 -0.0" xyz="0.0 0.0 0.0"/>
-          </inertial>
-          <visual>
-            <geometry>
-              <mesh filename="package://kuka_mobile_robot_support/meshes/37152984509.stl"/>
-            </geometry>
-            <origin rpy="-0.0 0.0 -0.0" xyz="0.0 0.0 0.0"/>
+              <mesh filename="package://kuka_kmr_iisy_support/meshes/collision/caster_base_bl_link.stl"/>
+            </geometry>
+            <origin rpy="-0.0 0.0 -0.0" xyz="0.0 0.0 0.0"/>
+          </collision>
+          <inertial>
+            <inertia ixx="1.0E-4" ixy="0.0" ixz="0.0" iyy="1.0E-4" iyz="0.0" izz="1.0E-4"/>
+            <mass value="1.0E-1"/>
+            <origin rpy="-0.0 0.0 -0.0" xyz="0.0 0.0 0.0"/>
+          </inertial>
+          <visual>
+            <geometry>
+              <mesh filename="package://kuka_kmr_iisy_support/meshes/visual/caster_base_bl_link.stl"/>
+            </geometry>
+            <origin rpy="-0.0 0.0 -0.0" xyz="0.0 0.0 0.0"/>
+            <xacro:material_kuka_ral_gray_white/>
           </visual>
         </link>
@@ -256,18 +265,19 @@
           <collision>
             <geometry>
-              <mesh filename="package://kuka_mobile_robot_support/meshes/37149321854.stl"/>
-            </geometry>
-            <origin rpy="1.5707963267948963 0.0 -0.0" xyz="0.0 0.0 0.0"/>
-          </collision>
-          <inertial>
-            <inertia ixx="1.0E-4" ixy="0.0" ixz="0.0" iyy="1.0E-4" iyz="0.0" izz="1.0E-4"/>
-            <mass value="1.0E-1"/>
-            <origin rpy="-0.0 0.0 -0.0" xyz="0.0 0.0 0.0"/>
-          </inertial>
-          <visual>
-            <geometry>
-              <mesh filename="package://kuka_mobile_robot_support/meshes/37149329314.stl"/>
-            </geometry>
-            <origin rpy="1.5707963267948963 0.0 -0.0" xyz="0.0 0.0 0.0"/>
+              <mesh filename="package://kuka_kmr_iisy_support/meshes/collision/caster_wheel_link.stl"/>
+            </geometry>
+            <origin rpy="1.5707963267948963 0.0 -0.0" xyz="0.0 0.0 0.0"/>
+          </collision>
+          <inertial>
+            <inertia ixx="1.0E-4" ixy="0.0" ixz="0.0" iyy="1.0E-4" iyz="0.0" izz="1.0E-4"/>
+            <mass value="1.0E-1"/>
+            <origin rpy="-0.0 0.0 -0.0" xyz="0.0 0.0 0.0"/>
+          </inertial>
+          <visual>
+            <geometry>
+              <mesh filename="package://kuka_kmr_iisy_support/meshes/visual/caster_wheel_link.stl"/>
+            </geometry>
+            <origin rpy="1.5707963267948963 0.0 -0.0" xyz="0.0 0.0 0.0"/>
+            <xacro:material_kuka_ral_gray_white/>
           </visual>
         </link>
@@ -275,18 +285,19 @@
           <collision>
             <geometry>
-              <mesh filename="package://kuka_mobile_robot_support/meshes/37153311411.stl"/>
-            </geometry>
-            <origin rpy="-0.0 0.0 -0.0" xyz="0.0 0.0 0.0"/>
-          </collision>
-          <inertial>
-            <inertia ixx="1.0E-4" ixy="0.0" ixz="0.0" iyy="1.0E-4" iyz="0.0" izz="1.0E-4"/>
-            <mass value="1.0E-1"/>
-            <origin rpy="-0.0 0.0 -0.0" xyz="0.0 0.0 0.0"/>
-          </inertial>
-          <visual>
-            <geometry>
-              <mesh filename="package://kuka_mobile_robot_support/meshes/37153318102.stl"/>
-            </geometry>
-            <origin rpy="-0.0 0.0 -0.0" xyz="0.0 0.0 0.0"/>
+              <mesh filename="package://kuka_kmr_iisy_support/meshes/collision/caster_base_br_link.stl"/>
+            </geometry>
+            <origin rpy="-0.0 0.0 -0.0" xyz="0.0 0.0 0.0"/>
+          </collision>
+          <inertial>
+            <inertia ixx="1.0E-4" ixy="0.0" ixz="0.0" iyy="1.0E-4" iyz="0.0" izz="1.0E-4"/>
+            <mass value="1.0E-1"/>
+            <origin rpy="-0.0 0.0 -0.0" xyz="0.0 0.0 0.0"/>
+          </inertial>
+          <visual>
+            <geometry>
+              <mesh filename="package://kuka_kmr_iisy_support/meshes/visual/caster_base_br_link.stl"/>
+            </geometry>
+            <origin rpy="-0.0 0.0 -0.0" xyz="0.0 0.0 0.0"/>
+            <xacro:material_kuka_ral_gray_white/>
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