Commit message: renamed package and meshes, deleted unnecesary files

File: kuka_kmr_iisy_support/urdf/kmr_iisy_ros2_control.xacro (robot description, xacro)
@@ -10,13 +10,9 @@
           <param name="mock_sensor_commands">false</param>
           <param name="state_following_offset">0.0</param>
-          <!--<xacro:if value="${gazebo_sim}">
-            <plugin>kuka_eac::KukaEACHardwareInterface</plugin>
-            <plugin>gazebo_ros2_control/GazeboSystem</plugin>
-          </xacro:if> -->
         </xacro:if>
         <xacro:unless value="${use_fake_hardware}">
           <!-- Read QoS profile parameters  -->
           <xacro:if value="${qos_config_file == ''}">
-            <xacro:property name="qos_config" value="$(find kuka_iiqka_eac_driver)/config/qos_config.yaml"/>
+            <xacro:property name="qos_config" value="$(find kuka_kmr_iisy_eac_driver)/config/qos_config.yaml"/>
           </xacro:if>
           <xacro:unless value="${qos_config_file == ''}">
@@ -27,5 +23,5 @@
           <xacro:property name="lost_packets_in_timeframe" value="${qos_config_dict['rt_packet_loss_profile']['lost_packets_in_timeframe']}"/>
           <xacro:property name="timeframe_ms" value="${qos_config_dict['rt_packet_loss_profile']['timeframe_ms']}"/>
-          <plugin>kuka_eac::KukaEACHardwareInterface</plugin>
+          <plugin>kuka_eac::KukaKMRiisyEACHardwareInterface</plugin>
           <param name="client_ip">${client_ip}</param>
           <param name="controller_ip">${controller_ip}</param>
@@ -36,52 +32,25 @@
       </hardware>
       <!-- define joints and command/state interfaces for each joint -->
-      <joint name="${prefix}twist/linear">
-        <command_interface name="x"/>
-        <command_interface name="y"/>
-        <command_interface name="z"/>
-        <state_interface name="x"/>
+      <joint name="${prefix}twist">
+        <command_interface name="linear/x"/>
+        <command_interface name="linear/y"/>
+        <command_interface name="linear/z"/>
+        <command_interface name="angular/x"/>
+        <command_interface name="angular/y"/>
+        <command_interface name="angular/z"/>
+        <state_interface name="linear/x"/>
           <param name="initial_value">0.0</param>
-        <state_interface name="y"/>
+        <state_interface name="linear/y"/>
           <param name="initial_value">0.0</param>
-        <state_interface name="z"/>
+        <state_interface name="linear/z"/>
+          <param name="initial_value">0.0</param>
+        <state_interface name="angular/x"/>
+          <param name="initial_value">0.0</param>
+        <state_interface name="angular/y"/>
+          <param name="initial_value">0.0</param>
+        <state_interface name="angular/z"/>
           <param name="initial_value">0.0</param>
       </joint>
-      <joint name="${prefix}twist/angular">
-        <command_interface name="x"/>
-        <command_interface name="y"/>
-        <command_interface name="z"/>
-        <state_interface name="x"/>
-          <param name="initial_value">0.0</param>
-        <state_interface name="y"/>
-          <param name="initial_value">0.0</param>
-        <state_interface name="z"/>
-          <param name="initial_value">0.0</param>
-      </joint>
-      <!--<joint name="left_wheel_motor">
-          <command_interface name="velocity">
-            <param name="min">-1</param>
-            <param name="max">1</param>
-          </command_interface>
-          <state_interface name="position"/>
-            <param name="initial_value">0.0</param>
-          <state_interface name="velocity"/>
-            <param name="initial_value">0.0</param>
-        </joint>
-        <joint name="right_wheel_motor">
-          <command_interface name="velocity">
-            <param name="min">-1</param>
-            <param name="max">1</param>
-          </command_interface>
-          <state_interface name="position"/>
-            <param name="initial_value">0.0</param>
-          <state_interface name="velocity"/>
-            <param name="initial_value">0.0</param>
-        </joint>  -->
     </ros2_control>
- <!--<xacro:if value="${gazebo_sim}">
- config file with gazebo parameters
-            <xacro:include filename="$(find kuka_mobile_robot_support)/gazebo/diffbot.gazebo.xacro" />
-            <xacro:diffbot_gazebo  prefix="" ros2_control_sim="true"/>
- </xacro:if>-->
   </xacro:macro>
 </robot>

Commit message: remove config dir, typo, remove unused args

File: kuka_kmr_iisy_support/urdf/kmr_iisy.urdf.xacro (robot description, xacro)
@@ -11,12 +11,5 @@
   <xacro:arg name="roundtrip_time" default="0"/>
   <xacro:arg name="qos_config_file" default=""/>
-  <xacro:arg name="x" default="0"/>
-  <xacro:arg name="y" default="0"/>
-  <xacro:arg name="z" default="0"/>
-  <xacro:arg name="roll" default="0"/>
-  <xacro:arg name="pitch" default="0"/>
-  <xacro:arg name="yaw" default="0"/>
   <xacro:mrob_kuka prefix="$(arg prefix)" controller_ip="$(arg controller_ip)" client_ip="$(arg client_ip)" use_fake_hardware="$(arg use_fake_hardware)" roundtrip_time="$(arg roundtrip_time)" qos_config_file="$(arg qos_config_file)">
-    <origin xyz="$(arg x) $(arg y) $(arg z)" rpy="$(arg roll) $(arg pitch) $(arg yaw)"/>
   </xacro:mrob_kuka>
 </robot>

File: kuka_kmr_iisy_support/urdf/kmr_iisy_macro.xacro (robot description, xacro)
@@ -4,5 +4,5 @@
   <xacro:include filename="$(find kuka_kmr_iisy_support)/urdf/kmr_iisy_ros2_control.xacro" />
   <xacro:include filename="$(find kuka_resources)/urdf/common_materials.xacro"/>
-  <xacro:macro name="mrob_kuka" params="prefix controller_ip client_ip use_fake_hardware roundtrip_time qos_config_file *origin">
+  <xacro:macro name="mrob_kuka" params="prefix controller_ip client_ip use_fake_hardware roundtrip_time qos_config_file">
     <!-- ros2 control instance -->
     <xacro:mrob_kuka_ros2_control name="kmr_iisy" prefix="${prefix}" client_ip="${client_ip}" controller_ip="${controller_ip}" use_fake_hardware="${use_fake_hardware}" roundtrip_time="${roundtrip_time}" qos_config_file="${qos_config_file}"/>
