Commit message: add cart joints to mock hardware

File: kuka_lbr_iiwa_support/urdf/lbr_iiwa_ros2_control.xacro (robot description, xacro)
@@ -124,4 +124,36 @@
         </state_interface>
       </joint>
+      <xacro:if value="${use_fake_hardware}">
+        <joint name="${prefix}dummy_cart_joint/x">
+          <command_interface name="stiffness"/>
+          <command_interface name="damping"/>
+          <command_interface name="effort"/>
+        </joint>
+        <joint name="${prefix}dummy_cart_joint/y">
+          <command_interface name="stiffness"/>
+          <command_interface name="damping"/>
+          <command_interface name="effort"/>
+        </joint>
+        <joint name="${prefix}dummy_cart_joint/z">
+          <command_interface name="stiffness"/>
+          <command_interface name="damping"/>
+          <command_interface name="effort"/>
+        </joint>
+        <joint name="${prefix}dummy_cart_joint/a">
+          <command_interface name="stiffness"/>
+          <command_interface name="damping"/>
+          <command_interface name="effort"/>
+        </joint>
+        <joint name="${prefix}dummy_cart_joint/b">
+          <command_interface name="stiffness"/>
+          <command_interface name="damping"/>
+          <command_interface name="effort"/>
+        </joint>
+        <joint name="${prefix}dummy_cart_joint/c">
+          <command_interface name="stiffness"/>
+          <command_interface name="damping"/>
+          <command_interface name="effort"/>
+        </joint>
+      </xacro:if>
       <xacro:unless value="${use_fake_hardware}">
         <xacro:if value="${io_access}">

Commit message: add quaternion mock joints and position

File: kuka_lbr_iiwa_support/urdf/lbr_iiwa_ros2_control.xacro (robot description, xacro)
@@ -126,4 +126,5 @@
       <xacro:if value="${use_fake_hardware}">
         <joint name="${prefix}dummy_cart_joint/x">
+          <command_interface name="position"/>
           <command_interface name="stiffness"/>
           <command_interface name="damping"/>
@@ -131,4 +132,5 @@
         </joint>
         <joint name="${prefix}dummy_cart_joint/y">
+          <command_interface name="position"/>
           <command_interface name="stiffness"/>
           <command_interface name="damping"/>
@@ -136,7 +138,20 @@
         </joint>
         <joint name="${prefix}dummy_cart_joint/z">
+          <command_interface name="position"/>
           <command_interface name="stiffness"/>
           <command_interface name="damping"/>
           <command_interface name="effort"/>
+        </joint>
+        <joint name="${prefix}dummy_cart_joint/qx">
+          <command_interface name="position"/>
+        </joint>
+        <joint name="${prefix}dummy_cart_joint/qy">
+          <command_interface name="position"/>
+        </joint>
+        <joint name="${prefix}dummy_cart_joint/qz">
+          <command_interface name="position"/>
+        </joint>
+        <joint name="${prefix}dummy_cart_joint/qw">
+          <command_interface name="position"/>
         </joint>
         <joint name="${prefix}dummy_cart_joint/a">
