Commit message: iiwa urdf restruct

File: kuka_lbr_iiwa_support/urdf/lbr_iiwa14_r820.urdf.xacro (robot description, xacro)
@@ -3,4 +3,7 @@
 <!-- Import iiwa urdf file  -->
 <xacro:include filename="$(find kuka_lbr_iiwa_support)/urdf/lbr_iiwa14_r820_macro.xacro"/>
-<xacro:kuka_lbr_iiwa14_r820_robot prefix="" io_access="false"/>
+<!-- Read additional arguments  -->
+<xacro:arg name="use_fake_hardware" default="false" />
+<xacro:arg name="gazebo_sim" default="false" />
+<xacro:kuka_lbr_iiwa14_r820_robot prefix="" io_access="false" use_fake_hardware="$(arg use_fake_hardware)" gazebo_sim="$(arg gazebo_sim)"/>
 </robot>

File: kuka_lbr_iiwa_support/urdf/lbr_iiwa14_r820_macro.xacro (robot description, xacro)
@@ -1,431 +1,242 @@
 <?xml version="1.0"?>
 <robot xmlns:xacro="http://wiki.ros.org/xacro">
-  <xacro:macro name="kuka_lbr_iiwa14_r820_robot" params="io_access prefix">
-  <ros2_control name="iiwa_hardware" type="system">
-    <hardware>
-      <plugin>kuka_sunrise::KUKAFRIHardwareInterface</plugin>
-    </hardware>
-    <!-- define joints and command/state interfaces for each joint -->
-    <joint name="${prefix}joint_a1">
-      <command_interface name="position">
-        <param name="min">-1</param>
-        <param name="max"> 1</param>
-      </command_interface>
-      <command_interface name="effort">
-        <param name="min">-1</param>
-        <param name="max"> 1</param>
-      </command_interface>
-      <state_interface name="position"/>
-      <state_interface name="effort"/>
-      <state_interface name="external_torque"/>
-    </joint>
-    <joint name="${prefix}joint_a2">
-      <command_interface name="position">
-        <param name="min">-1</param>
-        <param name="max"> 1</param>
-      </command_interface>
-      <command_interface name="effort">
-        <param name="min">-1</param>
-        <param name="max"> 1</param>
-      </command_interface>
-      <state_interface name="position"/>
-      <state_interface name="effort"/>
-      <state_interface name="external_torque"/>
-    </joint>
-    <joint name="${prefix}joint_a3">
-      <command_interface name="position">
-        <param name="min">-1</param>
-        <param name="max"> 1</param>
-      </command_interface>
-      <command_interface name="effort">
-        <param name="min">-1</param>
-        <param name="max"> 1</param>
-      </command_interface>
-      <state_interface name="position"/>
-      <state_interface name="effort"/>
-      <state_interface name="external_torque"/>
-    </joint>
-    <joint name="${prefix}joint_a4">
-      <command_interface name="position">
-        <param name="min">-1</param>
-        <param name="max"> 1</param>
-      </command_interface>
-      <command_interface name="effort">
-        <param name="min">-1</param>
-        <param name="max"> 1</param>
-      </command_interface>
-      <state_interface name="position"/>
-      <state_interface name="effort"/>
-      <state_interface name="external_torque"/>
-    </joint>
-    <joint name="${prefix}joint_a5">
-      <command_interface name="position">
-        <param name="min">-1</param>
-        <param name="max"> 1</param>
-      </command_interface>
-      <command_interface name="effort">
-        <param name="min">-1</param>
-        <param name="max"> 1</param>
-      </command_interface>
-      <state_interface name="position"/>
-      <state_interface name="effort"/>
-      <state_interface name="external_torque"/>
-    </joint>
-    <joint name="${prefix}joint_a6">
-      <command_interface name="position">
-        <param name="min">-1</param>
-        <param name="max"> 1</param>
-      </command_interface>
-      <command_interface name="effort">
-        <param name="min">-1</param>
-        <param name="max"> 1</param>
-      </command_interface>
-      <state_interface name="position"/>
-      <state_interface name="effort"/>
-      <state_interface name="external_torque"/>
-    </joint>
-    <joint name="${prefix}joint_a7">
-      <command_interface name="position">
-        <param name="min">-1</param>
-        <param name="max"> 1</param>
-      </command_interface>
-      <command_interface name="effort">
-        <param name="min">-1</param>
-        <param name="max"> 1</param>
-      </command_interface>
-      <state_interface name="position"/>
-      <state_interface name="effort"/>
-      <state_interface name="external_torque"/>
-    </joint>
-    <!-- TODO(Svastits): update GPIO list from config file-->
-    <xacro:if value="${io_access}">
-      <xacro:include filename="$(find kuka_sunrise)/config/gpio_config.xacro" />
-      <xacro:fri_gpio_config/>
-    </xacro:if>
-    <xacro:unless value="${io_access}">
-      <gpio name="gpio"/>
-    </xacro:unless>
-  </ros2_control>
-  <gazebo>
-    <plugin name="gazebo_ros2_control" filename="libgazebo_ros2_control.so">
-      <robotSimType>gazebo_ros2_control/DefaultRobotHWSim</robotSimType>
-      <parameters>$(find kuka_lbr_iiwa_support)/config/lbriiwa_control.yaml</parameters>
-    </plugin>
-  </gazebo>
-  <gazebo reference="${prefix}base_link">
-    <selfCollide>true</selfCollide>
-    <material>Gazebo/Orange</material>
-  </gazebo>
-  <gazebo reference="${prefix}link_1">
-    <selfCollide>true</selfCollide>
-    <material>Gazebo/Orange</material>
-  </gazebo>
-  <gazebo reference="${prefix}link_2">
-    <selfCollide>true</selfCollide>
-    <material>Gazebo/Orange</material>
-  </gazebo>
-  <gazebo reference="${prefix}link_3">
-    <selfCollide>true</selfCollide>
-    <material>Gazebo/Orange</material>
-  </gazebo>
-  <gazebo reference="${prefix}link_4">
-    <selfCollide>true</selfCollide>
-    <material>Gazebo/Orange</material>
-  </gazebo>
-  <gazebo reference="${prefix}link_5">
-    <selfCollide>true</selfCollide>
-    <material>Gazebo/Orange</material>
-  </gazebo>
-  <gazebo reference="${prefix}link_6">
-    <selfCollide>true</selfCollide>
-    <material>Gazebo/Orange</material>
-  </gazebo>
-  <gazebo reference="${prefix}link_7">
-    <selfCollide>true</selfCollide>
-    <material>Gazebo/Orange</material>
-  </gazebo>
-  <link name="world"/>
-  <link name="${prefix}base_link">
-    <visual>
-      <geometry>
-        <mesh filename="package://kuka_lbr_iiwa_support/lbr_iiwa14_r820/meshes/visual/base_link.stl"/>
-      </geometry>
-      <origin rpy="-0.0 0.0 0.0" xyz="0.0 0.0 0.0"/>
-    </visual>
-    <collision>
-      <origin rpy="-0.0 0.0 0.0" xyz="0.0 0.0 0.0"/>
-      <geometry>
-        <mesh filename="package://kuka_lbr_iiwa_support/lbr_iiwa14_r820/meshes/collision/base_link.stl"/>
-      </geometry>
-    </collision>
-    <inertial>
-      <mass value="3.2832"/>
-      <origin rpy="0 0 0" xyz="0.0 0.0 0.0"/>
-      <inertia ixx="5.0E-4" ixy="0.0" ixz="0.0" iyy="5.0E-4" iyz="0.0" izz="5.0E-4"/>
-    </inertial>
-  </link>
-  <link name="${prefix}link_1">
-    <visual>
-      <geometry>
-        <mesh filename="package://kuka_lbr_iiwa_support/lbr_iiwa14_r820/meshes/visual/link_1.stl"/>
-      </geometry>
-      <origin rpy="-0.0 0.0 0.0" xyz="0.0 0.0 0.0"/>
-    </visual>
-    <collision>
-      <origin rpy="-0.0 0.0 0.0" xyz="0.0 0.0 0.0"/>
-      <geometry>
-        <mesh filename="package://kuka_lbr_iiwa_support/lbr_iiwa14_r820/meshes/collision/link_1.stl"/>
-      </geometry>
-    </collision>
-    <inertial>
-      <mass value="6.495"/>
-      <origin rpy="0 0 0" xyz="0.0 0.0 0.0"/>
-      <inertia ixx="0.06907" ixy="0.0" ixz="0.0" iyy="0.0711" iyz="0.0" izz="0.02"/>
-    </inertial>
-  </link>
-  <link name="${prefix}link_2">
-    <visual>
-      <geometry>
-        <mesh filename="package://kuka_lbr_iiwa_support/lbr_iiwa14_r820/meshes/visual/link_2.stl"/>
-      </geometry>
-      <origin rpy="-0.0 0.0 0.0" xyz="0.0 0.0 0.0"/>
-    </visual>
-    <collision>
-      <origin rpy="-0.0 0.0 0.0" xyz="0.0 0.0 0.0"/>
-      <geometry>
-        <mesh filename="package://kuka_lbr_iiwa_support/lbr_iiwa14_r820/meshes/collision/link_2.stl"/>
-      </geometry>
-    </collision>
-    <inertial>
-      <mass value="8.365"/>
-      <origin rpy="0 0 0" xyz="0.0 0.0 0.0"/>
-      <inertia ixx="0.08" ixy="0.0" ixz="0.0" iyy="0.08" iyz="0.0" izz="0.01"/>
-    </inertial>
-  </link>
-  <link name="${prefix}link_3">
-    <visual>
-      <geometry>
-        <mesh filename="package://kuka_lbr_iiwa_support/lbr_iiwa14_r820/meshes/visual/link_3.stl"/>
-      </geometry>
-      <origin rpy="-0.0 0.0 0.0" xyz="0.0 0.0 0.0"/>
-    </visual>
-    <collision>
-      <origin rpy="-0.0 0.0 0.0" xyz="0.0 0.0 0.0"/>
-      <geometry>
-        <mesh filename="package://kuka_lbr_iiwa_support/lbr_iiwa14_r820/meshes/collision/link_3.stl"/>
-      </geometry>
-    </collision>
-    <inertial>
-      <mass value="2.5697"/>
-      <origin rpy="0 0 0" xyz="0.0 0.0 0.0"/>
-      <inertia ixx="0.02" ixy="0.0" ixz="0.0" iyy="0.02" iyz="0.0" izz="0.06"/>
-    </inertial>
-  </link>
-  <link name="${prefix}link_4">
-    <visual>
-      <geometry>
-        <mesh filename="package://kuka_lbr_iiwa_support/lbr_iiwa14_r820/meshes/visual/link_4.stl"/>
-      </geometry>
-      <origin rpy="-0.0 0.0 0.0" xyz="0.0 0.0 0.0"/>
-    </visual>
-    <collision>
-      <origin rpy="-0.0 0.0 0.0" xyz="0.0 0.0 0.0"/>
-      <geometry>
-        <mesh filename="package://kuka_lbr_iiwa_support/lbr_iiwa14_r820/meshes/collision/link_4.stl"/>
-      </geometry>
-    </collision>
-    <inertial>
-      <mass value="5.41"/>
-      <origin rpy="0 0 0" xyz="0.0 0.0 0.0"/>
-      <inertia ixx="0.04" ixy="0.0" ixz="0.0" iyy="0.03" iyz="0.0" izz="0.01"/>
-    </inertial>
-  </link>
-  <link name="${prefix}link_5">
-    <visual>
-      <geometry>
-        <mesh filename="package://kuka_lbr_iiwa_support/lbr_iiwa14_r820/meshes/visual/link_5.stl"/>
-      </geometry>
-      <origin rpy="-0.0 0.0 0.0" xyz="0.0 0.0 0.0"/>
-    </visual>
-    <collision>
-      <origin rpy="-0.0 0.0 0.0" xyz="0.0 0.0 0.0"/>
-      <geometry>
-        <mesh filename="package://kuka_lbr_iiwa_support/lbr_iiwa14_r820/meshes/collision/link_5.stl"/>
-      </geometry>
-    </collision>
-    <inertial>
-      <mass value="1.867"/>
-      <origin rpy="0 0 0" xyz="0.0 0.0 0.0"/>
-      <inertia ixx="0.01" ixy="0.0" ixz="0.0" iyy="0.01" iyz="0.0" izz="0.01"/>
-    </inertial>
-  </link>
-  <link name="${prefix}link_6">
-    <visual>
-      <geometry>
-        <mesh filename="package://kuka_lbr_iiwa_support/lbr_iiwa14_r820/meshes/visual/link_6.stl"/>
-      </geometry>
-      <origin rpy="-0.0 0.0 0.0" xyz="0.0 0.0 0.0"/>
-    </visual>
-    <collision>
-      <origin rpy="-0.0 0.0 0.0" xyz="0.0 0.0 0.0"/>
-      <geometry>
-        <mesh filename="package://kuka_lbr_iiwa_support/lbr_iiwa14_r820/meshes/collision/link_6.stl"/>
-      </geometry>
-    </collision>
-    <inertial>
-      <mass value="2.458"/>
-      <origin rpy="0 0 0" xyz="0.0 0.0 0.0"/>
-      <inertia ixx="0.007" ixy="0.0" ixz="0.0" iyy="0.006" iyz="0.0" izz="0.005"/>
-    </inertial>
-  </link>
-  <link name="${prefix}link_7">
-    <visual>
-      <geometry>
-        <mesh filename="package://kuka_lbr_iiwa_support/lbr_iiwa14_r820/meshes/visual/link_7.stl"/>
-      </geometry>
-      <origin rpy="-0.0 0.0 0.0" xyz="0.0 0.0 0.0"/>
-    </visual>
-    <collision>
-      <origin rpy="-0.0 0.0 0.0" xyz="0.0 0.0 0.0"/>
-      <geometry>
-        <mesh filename="package://kuka_lbr_iiwa_support/lbr_iiwa14_r820/meshes/collision/link_7.stl"/>
-      </geometry>
-    </collision>
-    <inertial>
-      <mass value="0.627"/>
-      <origin rpy="0 0 0" xyz="0.0 0.0 0.0"/>
-      <inertia ixx="3.0E-4" ixy="0.0" ixz="0.0" iyy="3.0E-4" iyz="0.0" izz="5.0E-4"/>
-    </inertial>
-  </link>
-  <link name="LBRiiwaFlange"></link>
-  <joint name="${prefix}base_linkJoint" type="fixed">
-    <parent link="world"/>
-    <child link="${prefix}base_link"/>
-  </joint>
-  <joint name="${prefix}joint_a1" type="revolute">
-    <parent link="${prefix}base_link"/>
-    <child link="${prefix}link_1"/>
-    <origin rpy="-0.0 0.0 0.0" xyz="0.0 0.0 0.1375"/>
-    <axis xyz="0.0 0.0 1.0"/>
-    <limit effort="158.4" lower="-2.67035" upper="2.67035" velocity="6.283"/>
-  </joint>
-  <joint name="${prefix}joint_a2" type="revolute">
-    <parent link="${prefix}link_1"/>
-    <child link="${prefix}link_2"/>
-    <origin rpy="-0.0 0.0 0.0" xyz="0.0 0.0 0.2025"/>
-    <axis xyz="0.0 1.0 0.0"/>
-    <limit effort="158.4" lower="-1.8849" upper="1.8849" velocity="6.283"/>
-  </joint>
-  <joint name="${prefix}joint_a3" type="revolute">
-    <parent link="${prefix}link_2"/>
-    <child link="${prefix}link_3"/>
-    <origin rpy="-0.0 0.0 0.0" xyz="0.0 0.0 0.1845"/>
-    <axis xyz="0.0 0.0 1.0"/>
-    <limit effort="99" lower="-2.67035" upper="2.67035" velocity="6.283"/>
-  </joint>
-  <joint name="${prefix}joint_a4" type="revolute">
-    <parent link="${prefix}link_3"/>
-    <child link="${prefix}link_4"/>
-    <origin rpy="-0.0 0.0 0.0" xyz="0.0 0.0 0.2155"/>
-    <axis xyz="0.0 -1.0 0.0"/>
-    <limit effort="99" lower="-1.8849" upper="1.8849" velocity="6.283"/>
-  </joint>
-  <joint name="${prefix}joint_a5" type="revolute">
-    <parent link="${prefix}link_4"/>
-    <child link="${prefix}link_5"/>
-    <origin rpy="-0.0 0.0 0.0" xyz="0.0 0.0 0.1845"/>
-    <axis xyz="0.0 0.0 1.0"/>
-    <limit effort="99" lower="-2.67035" upper="2.67035" velocity="6.283"/>
-  </joint>
-  <joint name="${prefix}joint_a6" type="revolute">
-    <parent link="${prefix}link_5"/>
-    <child link="${prefix}link_6"/>
-    <origin rpy="-0.0 0.0 0.0" xyz="0.0 0.0 0.2155"/>
-    <axis xyz="0.0 1.0 0.0"/>
-    <limit effort="36" lower="-1.8849" upper="1.8849" velocity="6.283"/>
-  </joint>
-  <joint name="${prefix}joint_a7" type="revolute">
-    <parent link="${prefix}link_6"/>
-    <child link="${prefix}link_7"/>
-    <origin rpy="-0.0 0.0 0.0" xyz="0.0 0.0 0.081"/>
-    <axis xyz="0.0 0.0 1.0"/>
-    <limit effort="36" lower="-2.74889" upper="2.74889" velocity="6.283"/>
-  </joint>
-  <joint name="LBRiiwaTCP" type="fixed">
-    <parent link="${prefix}link_7"/>
-    <child link="LBRiiwaFlange"/>
-    <origin rpy="-0.0 0.0 0.0" xyz="0.0 0.0 0.071"/>
-    <axis xyz="0.0 0.0 1.0"/>
-  </joint>
-  <transmission name="Transmission_${prefix}joint_a1">
-    <type>transmission_interface/SimpleTransmission</type>
-    <joint name="${prefix}joint_a1">
-      <hardwareInterface>hardware_interface/EffortJointInterface</hardwareInterface>
-    </joint>
-    <actuator name="motor_${prefix}joint_a1">
-      <hardwareInterface>EffortJointInterface</hardwareInterface>
-      <mechanicalReduction>1.0</mechanicalReduction>
-    </actuator>
-  </transmission>
-  <transmission name="Transmission_${prefix}joint_a2">
-    <type>transmission_interface/SimpleTransmission</type>
-    <joint name="${prefix}joint_a2">
-      <hardwareInterface>hardware_interface/EffortJointInterface</hardwareInterface>
-    </joint>
-    <actuator name="motor_${prefix}joint_a2">
-      <hardwareInterface>EffortJointInterface</hardwareInterface>
-      <mechanicalReduction>1.0</mechanicalReduction>
-    </actuator>
-  </transmission>
-  <transmission name="Transmission_${prefix}joint_a3">
-    <type>transmission_interface/SimpleTransmission</type>
-    <joint name="${prefix}joint_a3">
-      <hardwareInterface>hardware_interface/EffortJointInterface</hardwareInterface>
-    </joint>
-    <actuator name="motor_${prefix}joint_a3">
-      <hardwareInterface>EffortJointInterface</hardwareInterface>
-      <mechanicalReduction>1.0</mechanicalReduction>
-    </actuator>
-  </transmission>
-  <transmission name="Transmission_${prefix}joint_a4">
-    <type>transmission_interface/SimpleTransmission</type>
-    <joint name="${prefix}joint_a4">
-      <hardwareInterface>hardware_interface/EffortJointInterface</hardwareInterface>
-    </joint>
-    <actuator name="motor_${prefix}joint_a4">
-      <hardwareInterface>EffortJointInterface</hardwareInterface>
-      <mechanicalReduction>1.0</mechanicalReduction>
-    </actuator>
-  </transmission>
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
Commit message: add missing args

File: kuka_lbr_iiwa_support/urdf/lbr_iiwa14_r820.urdf.xacro (robot description, xacro)
@@ -5,4 +5,15 @@
 <!-- Read additional arguments  -->
 <xacro:arg name="use_fake_hardware" default="false" />
-<xacro:kuka_lbr_iiwa14_r820_robot prefix="" io_access="false" use_fake_hardware="$(arg use_fake_hardware)"/>
+<xacro:arg name="x" default="0" />
+<xacro:arg name="y" default="0" />
+<xacro:arg name="z" default="0" />
+<xacro:arg name="roll" default="0" />
+<xacro:arg name="pitch" default="0" />
+<xacro:arg name="yaw" default="0" />
+<xacro:kuka_lbr_iiwa14_r820_robot
+  prefix=""
+  io_access="false"
+  use_fake_hardware="$(arg use_fake_hardware)">
+  <origin xyz="$(arg x) $(arg y) $(arg z)" rpy="$(arg roll) $(arg pitch) $(arg yaw)" />
+</xacro:kuka_lbr_iiwa14_r820_robot>
 </robot>

Commit message: add controller_ip to urdf

File: kuka_lbr_iiwa_support/urdf/lbr_iiwa14_r820.urdf.xacro (robot description, xacro)
@@ -4,4 +4,5 @@
   <xacro:include filename="$(find kuka_lbr_iiwa_support)/urdf/lbr_iiwa14_r820_macro.xacro"/>
   <!-- Read additional arguments  -->
+  <xacro:arg name="controller_ip" default="0.0.0.0"/>
   <xacro:arg name="use_fake_hardware" default="false"/>
   <xacro:arg name="x" default="0"/>
@@ -12,5 +13,5 @@
   <xacro:arg name="yaw" default="0"/>
   <xacro:arg name="prefix" default=""/>
-  <xacro:kuka_lbr_iiwa14_r820_robot prefix="$(arg prefix)" io_access="false" use_fake_hardware="$(arg use_fake_hardware)">
+  <xacro:kuka_lbr_iiwa14_r820_robot prefix="$(arg prefix)" io_access="false" use_fake_hardware="$(arg use_fake_hardware)" controller_ip="$(arg controller_ip)">
     <origin xyz="$(arg x) $(arg y) $(arg z)" rpy="$(arg roll) $(arg pitch) $(arg yaw)"/>
   </xacro:kuka_lbr_iiwa14_r820_robot>

File: kuka_lbr_iiwa_support/urdf/lbr_iiwa14_r820_macro.xacro (robot description, xacro)
@@ -5,7 +5,7 @@
   <xacro:include filename="$(find kuka_resources)/urdf/common_materials.xacro"/>
   <xacro:include filename="$(find kuka_lbr_iiwa_support)/urdf/lbr_iiwa_transmission.xacro"/>
-  <xacro:macro name="kuka_lbr_iiwa14_r820_robot" params="io_access prefix use_fake_hardware *origin">
+  <xacro:macro name="kuka_lbr_iiwa14_r820_robot" params="io_access prefix use_fake_hardware controller_ip *origin">
     <!-- ros2 control instance -->
-    <xacro:kuka_lbr_iiwa_ros2_control name="${prefix}lbr_iiwa14_r820" prefix="${prefix}" io_access="${io_access}" use_fake_hardware="${use_fake_hardware}"/>
+    <xacro:kuka_lbr_iiwa_ros2_control name="${prefix}lbr_iiwa14_r820" prefix="${prefix}" io_access="${io_access}" use_fake_hardware="${use_fake_hardware}" controller_ip="${controller_ip}"/>
     <!-- links - main serial chain -->
     <link name="world"/>

File: kuka_lbr_iiwa_support/urdf/lbr_iiwa_ros2_control.xacro (robot description, xacro)
@@ -1,5 +1,5 @@
 <?xml version="1.0" encoding="UTF-8"?>
 <robot xmlns:xacro="http://www.ros.org/wiki/xacro">
-  <xacro:macro name="kuka_lbr_iiwa_ros2_control" params="name prefix io_access use_fake_hardware">
+  <xacro:macro name="kuka_lbr_iiwa_ros2_control" params="name prefix io_access use_fake_hardware controller_ip">
     <ros2_control name="${name}" type="system">
       <hardware>
@@ -11,4 +11,5 @@
         <xacro:unless value="${use_fake_hardware}">
           <plugin>kuka_sunrise_fri_driver::KukaFRIHardwareInterface</plugin>
+          <param name="controller_ip">${controller_ip}</param>
         </xacro:unless>
       </hardware>

Commit message: client ip port

File: kuka_lbr_iiwa_support/urdf/lbr_iiwa14_r820.urdf.xacro (robot description, xacro)
@@ -5,4 +5,6 @@
   <!-- Read additional arguments  -->
   <xacro:arg name="controller_ip" default="0.0.0.0"/>
+  <xacro:arg name="client_ip" default="0.0.0.0"/>
+  <xacro:arg name="client_port" default="30200"/>
   <xacro:arg name="use_fake_hardware" default="false"/>
   <xacro:arg name="x" default="0"/>
@@ -13,5 +15,5 @@
   <xacro:arg name="yaw" default="0"/>
   <xacro:arg name="prefix" default=""/>
-  <xacro:kuka_lbr_iiwa14_r820_robot prefix="$(arg prefix)" io_access="false" use_fake_hardware="$(arg use_fake_hardware)" controller_ip="$(arg controller_ip)">
+  <xacro:kuka_lbr_iiwa14_r820_robot prefix="$(arg prefix)" io_access="false" use_fake_hardware="$(arg use_fake_hardware)" controller_ip="$(arg controller_ip)" client_ip="$(arg client_ip)" client_port="$(arg client_port)">
     <origin xyz="$(arg x) $(arg y) $(arg z)" rpy="$(arg roll) $(arg pitch) $(arg yaw)"/>
   </xacro:kuka_lbr_iiwa14_r820_robot>

File: kuka_lbr_iiwa_support/urdf/lbr_iiwa14_r820_macro.xacro (robot description, xacro)
@@ -5,7 +5,7 @@
   <xacro:include filename="$(find kuka_resources)/urdf/common_materials.xacro"/>
   <xacro:include filename="$(find kuka_lbr_iiwa_support)/urdf/lbr_iiwa_transmission.xacro"/>
-  <xacro:macro name="kuka_lbr_iiwa14_r820_robot" params="io_access prefix use_fake_hardware controller_ip *origin">
+  <xacro:macro name="kuka_lbr_iiwa14_r820_robot" params="io_access prefix use_fake_hardware controller_ip client_ip client_port *origin">
     <!-- ros2 control instance -->
-    <xacro:kuka_lbr_iiwa_ros2_control name="${prefix}lbr_iiwa14_r820" prefix="${prefix}" io_access="${io_access}" use_fake_hardware="${use_fake_hardware}" controller_ip="${controller_ip}"/>
+    <xacro:kuka_lbr_iiwa_ros2_control name="${prefix}lbr_iiwa14_r820" prefix="${prefix}" io_access="${io_access}" use_fake_hardware="${use_fake_hardware}" controller_ip="${controller_ip}" client_ip="${client_ip}" client_port="${client_port}"/>
     <!-- links - main serial chain -->
     <link name="world"/>

File: kuka_lbr_iiwa_support/urdf/lbr_iiwa_ros2_control.xacro (robot description, xacro)
@@ -1,5 +1,5 @@
 <?xml version="1.0" encoding="UTF-8"?>
 <robot xmlns:xacro="http://www.ros.org/wiki/xacro">
-  <xacro:macro name="kuka_lbr_iiwa_ros2_control" params="name prefix io_access use_fake_hardware controller_ip">
+  <xacro:macro name="kuka_lbr_iiwa_ros2_control" params="name prefix io_access use_fake_hardware controller_ip client_ip client_port">
     <ros2_control name="${name}" type="system">
       <hardware>
@@ -12,4 +12,6 @@
           <plugin>kuka_sunrise_fri_driver::KukaFRIHardwareInterface</plugin>
           <param name="controller_ip">${controller_ip}</param>
+          <param name="client_ip">${client_ip}</param>
+          <param name="client_port">${client_port}</param>
         </xacro:unless>
       </hardware>
