Commit message: update doc

File: kuka_lbr_iiwa_support/urdf/lbr_iiwa14_r820.urdf.xacro (robot description, xacro)
@@ -4,4 +4,7 @@
   <xacro:include filename="$(find kuka_lbr_iiwa_support)/urdf/lbr_iiwa14_r820_macro.xacro"/>
   <!-- Read additional arguments  -->
+  <xacro:arg name="controller_ip" default="0.0.0.0"/>
+  <xacro:arg name="client_ip" default="0.0.0.0"/>
+  <xacro:arg name="client_port" default="30200"/>
   <xacro:arg name="use_fake_hardware" default="false"/>
   <xacro:arg name="x" default="0"/>
@@ -12,5 +15,5 @@
   <xacro:arg name="yaw" default="0"/>
   <xacro:arg name="prefix" default=""/>
-  <xacro:kuka_lbr_iiwa14_r820_robot prefix="$(arg prefix)" io_access="false" use_fake_hardware="$(arg use_fake_hardware)">
+  <xacro:kuka_lbr_iiwa14_r820_robot prefix="$(arg prefix)" io_access="false" use_fake_hardware="$(arg use_fake_hardware)" controller_ip="$(arg controller_ip)" client_ip="$(arg client_ip)" client_port="$(arg client_port)">
     <origin xyz="$(arg x) $(arg y) $(arg z)" rpy="$(arg roll) $(arg pitch) $(arg yaw)"/>
   </xacro:kuka_lbr_iiwa14_r820_robot>

File: kuka_lbr_iiwa_support/urdf/lbr_iiwa14_r820_macro.xacro (robot description, xacro)
@@ -5,7 +5,7 @@
   <xacro:include filename="$(find kuka_resources)/urdf/common_materials.xacro"/>
   <xacro:include filename="$(find kuka_lbr_iiwa_support)/urdf/lbr_iiwa_transmission.xacro"/>
-  <xacro:macro name="kuka_lbr_iiwa14_r820_robot" params="io_access prefix use_fake_hardware *origin">
+  <xacro:macro name="kuka_lbr_iiwa14_r820_robot" params="io_access prefix use_fake_hardware controller_ip client_ip client_port *origin">
     <!-- ros2 control instance -->
-    <xacro:kuka_lbr_iiwa_ros2_control name="${prefix}lbr_iiwa14_r820" prefix="${prefix}" io_access="${io_access}" use_fake_hardware="${use_fake_hardware}"/>
+    <xacro:kuka_lbr_iiwa_ros2_control name="${prefix}lbr_iiwa14_r820" prefix="${prefix}" io_access="${io_access}" use_fake_hardware="${use_fake_hardware}" controller_ip="${controller_ip}" client_ip="${client_ip}" client_port="${client_port}"/>
     <!-- links - main serial chain -->
     <link name="world"/>

File: kuka_lbr_iiwa_support/urdf/lbr_iiwa_ros2_control.xacro (robot description, xacro)
@@ -1,5 +1,5 @@
 <?xml version="1.0" encoding="UTF-8"?>
 <robot xmlns:xacro="http://www.ros.org/wiki/xacro">
-  <xacro:macro name="kuka_lbr_iiwa_ros2_control" params="name prefix io_access use_fake_hardware">
+  <xacro:macro name="kuka_lbr_iiwa_ros2_control" params="name prefix io_access use_fake_hardware controller_ip client_ip client_port">
     <ros2_control name="${name}" type="system">
       <hardware>
@@ -11,4 +11,7 @@
         <xacro:unless value="${use_fake_hardware}">
           <plugin>kuka_sunrise_fri_driver::KukaFRIHardwareInterface</plugin>
+          <param name="controller_ip">${controller_ip}</param>
+          <param name="client_ip">${client_ip}</param>
+          <param name="client_port">${client_port}</param>
         </xacro:unless>
       </hardware>
@@ -16,4 +19,6 @@
       <joint name="${prefix}joint_1">
         <command_interface name="position"/>
+        <command_interface name="stiffness"/>
+        <command_interface name="damping"/>
         <command_interface name="effort"/>
         <state_interface name="position">
@@ -29,4 +34,6 @@
       <joint name="${prefix}joint_2">
         <command_interface name="position"/>
+        <command_interface name="stiffness"/>
+        <command_interface name="damping"/>
         <command_interface name="effort"/>
         <state_interface name="position">
@@ -42,4 +49,6 @@
       <joint name="${prefix}joint_3">
         <command_interface name="position"/>
+        <command_interface name="stiffness"/>
+        <command_interface name="damping"/>
         <command_interface name="effort"/>
         <state_interface name="position">
@@ -55,4 +64,6 @@
       <joint name="${prefix}joint_4">
         <command_interface name="position"/>
+        <command_interface name="stiffness"/>
+        <command_interface name="damping"/>
         <command_interface name="effort"/>
         <state_interface name="position">
@@ -68,4 +79,6 @@
       <joint name="${prefix}joint_5">
         <command_interface name="position"/>
+        <command_interface name="stiffness"/>
+        <command_interface name="damping"/>
         <command_interface name="effort"/>
         <state_interface name="position">
@@ -81,4 +94,6 @@
       <joint name="${prefix}joint_6">
         <command_interface name="position"/>
+        <command_interface name="stiffness"/>
+        <command_interface name="damping"/>
         <command_interface name="effort"/>
         <state_interface name="position">
@@ -94,4 +109,6 @@
       <joint name="${prefix}joint_7">
         <command_interface name="position"/>
+        <command_interface name="stiffness"/>
+        <command_interface name="damping"/>
         <command_interface name="effort"/>
         <state_interface name="position">
@@ -105,5 +122,4 @@
         </state_interface>
       </joint>
-      <!-- TODO(Svastits): update GPIO list from config file-->
       <xacro:unless value="${use_fake_hardware}">
         <xacro:if value="${io_access}">

Commit message: Revert "update doc"
This reverts commit b055d0a64a7ebcf39ed1aae3e9fb3d874765a4be.

File: kuka_lbr_iiwa_support/urdf/lbr_iiwa14_r820.urdf.xacro (robot description, xacro)
@@ -4,7 +4,4 @@
   <xacro:include filename="$(find kuka_lbr_iiwa_support)/urdf/lbr_iiwa14_r820_macro.xacro"/>
   <!-- Read additional arguments  -->
-  <xacro:arg name="controller_ip" default="0.0.0.0"/>
-  <xacro:arg name="client_ip" default="0.0.0.0"/>
-  <xacro:arg name="client_port" default="30200"/>
   <xacro:arg name="use_fake_hardware" default="false"/>
   <xacro:arg name="x" default="0"/>
@@ -15,5 +12,5 @@
   <xacro:arg name="yaw" default="0"/>
   <xacro:arg name="prefix" default=""/>
-  <xacro:kuka_lbr_iiwa14_r820_robot prefix="$(arg prefix)" io_access="false" use_fake_hardware="$(arg use_fake_hardware)" controller_ip="$(arg controller_ip)" client_ip="$(arg client_ip)" client_port="$(arg client_port)">
+  <xacro:kuka_lbr_iiwa14_r820_robot prefix="$(arg prefix)" io_access="false" use_fake_hardware="$(arg use_fake_hardware)">
     <origin xyz="$(arg x) $(arg y) $(arg z)" rpy="$(arg roll) $(arg pitch) $(arg yaw)"/>
   </xacro:kuka_lbr_iiwa14_r820_robot>

File: kuka_lbr_iiwa_support/urdf/lbr_iiwa14_r820_macro.xacro (robot description, xacro)
@@ -5,7 +5,7 @@
   <xacro:include filename="$(find kuka_resources)/urdf/common_materials.xacro"/>
   <xacro:include filename="$(find kuka_lbr_iiwa_support)/urdf/lbr_iiwa_transmission.xacro"/>
-  <xacro:macro name="kuka_lbr_iiwa14_r820_robot" params="io_access prefix use_fake_hardware controller_ip client_ip client_port *origin">
+  <xacro:macro name="kuka_lbr_iiwa14_r820_robot" params="io_access prefix use_fake_hardware *origin">
     <!-- ros2 control instance -->
-    <xacro:kuka_lbr_iiwa_ros2_control name="${prefix}lbr_iiwa14_r820" prefix="${prefix}" io_access="${io_access}" use_fake_hardware="${use_fake_hardware}" controller_ip="${controller_ip}" client_ip="${client_ip}" client_port="${client_port}"/>
+    <xacro:kuka_lbr_iiwa_ros2_control name="${prefix}lbr_iiwa14_r820" prefix="${prefix}" io_access="${io_access}" use_fake_hardware="${use_fake_hardware}"/>
     <!-- links - main serial chain -->
     <link name="world"/>

File: kuka_lbr_iiwa_support/urdf/lbr_iiwa_ros2_control.xacro (robot description, xacro)
@@ -1,5 +1,5 @@
 <?xml version="1.0" encoding="UTF-8"?>
 <robot xmlns:xacro="http://www.ros.org/wiki/xacro">
-  <xacro:macro name="kuka_lbr_iiwa_ros2_control" params="name prefix io_access use_fake_hardware controller_ip client_ip client_port">
+  <xacro:macro name="kuka_lbr_iiwa_ros2_control" params="name prefix io_access use_fake_hardware">
     <ros2_control name="${name}" type="system">
       <hardware>
@@ -11,7 +11,4 @@
         <xacro:unless value="${use_fake_hardware}">
           <plugin>kuka_sunrise_fri_driver::KukaFRIHardwareInterface</plugin>
-          <param name="controller_ip">${controller_ip}</param>
-          <param name="client_ip">${client_ip}</param>
-          <param name="client_port">${client_port}</param>
         </xacro:unless>
       </hardware>
@@ -19,6 +16,4 @@
       <joint name="${prefix}joint_1">
         <command_interface name="position"/>
-        <command_interface name="stiffness"/>
-        <command_interface name="damping"/>
         <command_interface name="effort"/>
         <state_interface name="position">
@@ -34,6 +29,4 @@
       <joint name="${prefix}joint_2">
         <command_interface name="position"/>
-        <command_interface name="stiffness"/>
-        <command_interface name="damping"/>
         <command_interface name="effort"/>
         <state_interface name="position">
@@ -49,6 +42,4 @@
       <joint name="${prefix}joint_3">
         <command_interface name="position"/>
-        <command_interface name="stiffness"/>
-        <command_interface name="damping"/>
         <command_interface name="effort"/>
         <state_interface name="position">
@@ -64,6 +55,4 @@
       <joint name="${prefix}joint_4">
         <command_interface name="position"/>
-        <command_interface name="stiffness"/>
-        <command_interface name="damping"/>
         <command_interface name="effort"/>
         <state_interface name="position">
@@ -79,6 +68,4 @@
       <joint name="${prefix}joint_5">
         <command_interface name="position"/>
-        <command_interface name="stiffness"/>
-        <command_interface name="damping"/>
         <command_interface name="effort"/>
         <state_interface name="position">
@@ -94,6 +81,4 @@
       <joint name="${prefix}joint_6">
         <command_interface name="position"/>
-        <command_interface name="stiffness"/>
-        <command_interface name="damping"/>
         <command_interface name="effort"/>
         <state_interface name="position">
@@ -109,6 +94,4 @@
       <joint name="${prefix}joint_7">
         <command_interface name="position"/>
-        <command_interface name="stiffness"/>
-        <command_interface name="damping"/>
         <command_interface name="effort"/>
         <state_interface name="position">
@@ -122,4 +105,5 @@
         </state_interface>
       </joint>
+      <!-- TODO(Svastits): update GPIO list from config file-->
       <xacro:unless value="${use_fake_hardware}">
         <xacro:if value="${io_access}">

Commit message: Add IP arg and impedance attributes to iiwa URDF (#55)
* unnecessary args

* add controller_ip to urdf

* add stifness, damping ifs

* Revert "add stifness, damping ifs"

This reverts commit 6b6d43fe1bac8b522e50b64b89d9e227012fe813.

* Revert "Revert "add stifness, damping ifs""

This reverts commit 98bd40ab5cba92bda2fb44deef986c3383fce7cb.

* client ip port

* add kuka mock hw if (only copy)

* extend metapackage

* export kuka-specific interfaces

* use kuka mock hw

* add server_state

* format

* add wait_unitl + fix folder names

* format

* warning for timeout

---------

Co-authored-by: Aron Svastits <svastits1@gmail.com>

File: kuka_lbr_iiwa_support/urdf/lbr_iiwa14_r820.urdf.xacro (robot description, xacro)
@@ -4,4 +4,7 @@
   <xacro:include filename="$(find kuka_lbr_iiwa_support)/urdf/lbr_iiwa14_r820_macro.xacro"/>
   <!-- Read additional arguments  -->
+  <xacro:arg name="controller_ip" default="0.0.0.0"/>
+  <xacro:arg name="client_ip" default="0.0.0.0"/>
+  <xacro:arg name="client_port" default="30200"/>
   <xacro:arg name="use_fake_hardware" default="false"/>
   <xacro:arg name="roundtrip_time" default="0"/>
@@ -13,5 +16,5 @@
   <xacro:arg name="yaw" default="0"/>
   <xacro:arg name="prefix" default=""/>
-  <xacro:kuka_lbr_iiwa14_r820_robot prefix="$(arg prefix)" io_access="false" use_fake_hardware="$(arg use_fake_hardware)" roundtrip_time="$(arg roundtrip_time)">
+  <xacro:kuka_lbr_iiwa14_r820_robot prefix="$(arg prefix)" io_access="false" use_fake_hardware="$(arg use_fake_hardware)" roundtrip_time="$(arg roundtrip_time)" controller_ip="$(arg controller_ip)" client_ip="$(arg client_ip)" client_port="$(arg client_port)">
     <origin xyz="$(arg x) $(arg y) $(arg z)" rpy="$(arg roll) $(arg pitch) $(arg yaw)"/>
   </xacro:kuka_lbr_iiwa14_r820_robot>

File: kuka_lbr_iiwa_support/urdf/lbr_iiwa14_r820_macro.xacro (robot description, xacro)
@@ -5,7 +5,7 @@
   <xacro:include filename="$(find kuka_resources)/urdf/common_materials.xacro"/>
   <xacro:include filename="$(find kuka_lbr_iiwa_support)/urdf/lbr_iiwa_transmission.xacro"/>
-  <xacro:macro name="kuka_lbr_iiwa14_r820_robot" params="io_access prefix use_fake_hardware roundtrip_time *origin">
+  <xacro:macro name="kuka_lbr_iiwa14_r820_robot" params="io_access prefix use_fake_hardware roundtrip_time controller_ip client_ip client_port *origin">
     <!-- ros2 control instance -->
-    <xacro:kuka_lbr_iiwa_ros2_control name="${prefix}lbr_iiwa14_r820" prefix="${prefix}" io_access="${io_access}" use_fake_hardware="${use_fake_hardware}" roundtrip_time="${roundtrip_time}"/>
+    <xacro:kuka_lbr_iiwa_ros2_control name="${prefix}lbr_iiwa14_r820" prefix="${prefix}" io_access="${io_access}" use_fake_hardware="${use_fake_hardware}" roundtrip_time="${roundtrip_time}" controller_ip="${controller_ip}" client_ip="${client_ip}" client_port="${client_port}"/>
     <!-- links - main serial chain -->
     <link name="world"/>

File: kuka_lbr_iiwa_support/urdf/lbr_iiwa_ros2_control.xacro (robot description, xacro)
@@ -1,5 +1,5 @@
 <?xml version="1.0" encoding="UTF-8"?>
 <robot xmlns:xacro="http://www.ros.org/wiki/xacro">
-  <xacro:macro name="kuka_lbr_iiwa_ros2_control" params="name prefix io_access use_fake_hardware roundtrip_time">
+  <xacro:macro name="kuka_lbr_iiwa_ros2_control" params="name prefix io_access use_fake_hardware roundtrip_time controller_ip client_ip client_port">
     <ros2_control name="${name}" type="system">
       <hardware>
@@ -13,4 +13,7 @@
         <xacro:unless value="${use_fake_hardware}">
           <plugin>kuka_sunrise_fri_driver::KukaFRIHardwareInterface</plugin>
+          <param name="controller_ip">${controller_ip}</param>
+          <param name="client_ip">${client_ip}</param>
+          <param name="client_port">${client_port}</param>
         </xacro:unless>
       </hardware>
@@ -18,4 +21,6 @@
       <joint name="${prefix}joint_1">
         <command_interface name="position"/>
+        <command_interface name="stiffness"/>
+        <command_interface name="damping"/>
         <command_interface name="effort"/>
         <state_interface name="position">
@@ -31,4 +36,6 @@
       <joint name="${prefix}joint_2">
         <command_interface name="position"/>
+        <command_interface name="stiffness"/>
+        <command_interface name="damping"/>
         <command_interface name="effort"/>
         <state_interface name="position">
@@ -44,4 +51,6 @@
       <joint name="${prefix}joint_3">
         <command_interface name="position"/>
+        <command_interface name="stiffness"/>
+        <command_interface name="damping"/>
         <command_interface name="effort"/>
         <state_interface name="position">
@@ -57,4 +66,6 @@
       <joint name="${prefix}joint_4">
         <command_interface name="position"/>
+        <command_interface name="stiffness"/>
+        <command_interface name="damping"/>
         <command_interface name="effort"/>
         <state_interface name="position">
@@ -70,4 +81,6 @@
       <joint name="${prefix}joint_5">
         <command_interface name="position"/>
+        <command_interface name="stiffness"/>
+        <command_interface name="damping"/>
         <command_interface name="effort"/>
         <state_interface name="position">
@@ -83,4 +96,6 @@
       <joint name="${prefix}joint_6">
         <command_interface name="position"/>
+        <command_interface name="stiffness"/>
+        <command_interface name="damping"/>
         <command_interface name="effort"/>
         <state_interface name="position">
@@ -96,4 +111,6 @@
       <joint name="${prefix}joint_7">
         <command_interface name="position"/>
+        <command_interface name="stiffness"/>
+        <command_interface name="damping"/>
         <command_interface name="effort"/>
         <state_interface name="position">
@@ -107,5 +124,4 @@
         </state_interface>
       </joint>
-      <!-- TODO(Svastits): update GPIO list from config file-->
       <xacro:unless value="${use_fake_hardware}">
         <xacro:if value="${io_access}">

Commit message: replace remaining use_fake_hardware with mode

File: kuka_lbr_iiwa_support/urdf/lbr_iiwa14_r820.urdf.xacro (robot description, xacro)
@@ -7,5 +7,5 @@
   <xacro:arg name="client_ip" default="0.0.0.0"/>
   <xacro:arg name="client_port" default="30200"/>
-  <xacro:arg name="use_fake_hardware" default="false"/>
+  <xacro:arg name="mode" default="hardware"/>
   <xacro:arg name="roundtrip_time" default="0"/>
   <xacro:arg name="x" default="0"/>
@@ -16,5 +16,5 @@
   <xacro:arg name="yaw" default="0"/>
   <xacro:arg name="prefix" default=""/>
-  <xacro:kuka_lbr_iiwa14_r820_robot prefix="$(arg prefix)" io_access="false" use_fake_hardware="$(arg use_fake_hardware)" roundtrip_time="$(arg roundtrip_time)" controller_ip="$(arg controller_ip)" client_ip="$(arg client_ip)" client_port="$(arg client_port)">
+  <xacro:kuka_lbr_iiwa14_r820_robot prefix="$(arg prefix)" io_access="false" mode="$(arg mode)" roundtrip_time="$(arg roundtrip_time)" controller_ip="$(arg controller_ip)" client_ip="$(arg client_ip)" client_port="$(arg client_port)">
     <origin xyz="$(arg x) $(arg y) $(arg z)" rpy="$(arg roll) $(arg pitch) $(arg yaw)"/>
   </xacro:kuka_lbr_iiwa14_r820_robot>

File: kuka_lbr_iiwa_support/urdf/lbr_iiwa14_r820_macro.xacro (robot description, xacro)
@@ -5,7 +5,7 @@
   <xacro:include filename="$(find kuka_resources)/urdf/common_materials.xacro"/>
   <xacro:include filename="$(find kuka_lbr_iiwa_support)/urdf/lbr_iiwa_transmission.xacro"/>
-  <xacro:macro name="kuka_lbr_iiwa14_r820_robot" params="io_access prefix use_fake_hardware roundtrip_time controller_ip client_ip client_port *origin">
+  <xacro:macro name="kuka_lbr_iiwa14_r820_robot" params="io_access prefix mode roundtrip_time controller_ip client_ip client_port *origin">
     <!-- ros2 control instance -->
-    <xacro:kuka_lbr_iiwa_ros2_control name="${prefix}lbr_iiwa14_r820" prefix="${prefix}" io_access="${io_access}" use_fake_hardware="${use_fake_hardware}" roundtrip_time="${roundtrip_time}" controller_ip="${controller_ip}" client_ip="${client_ip}" client_port="${client_port}"/>
+    <xacro:kuka_lbr_iiwa_ros2_control name="${prefix}lbr_iiwa14_r820" prefix="${prefix}" io_access="${io_access}" mode="${mode}" roundtrip_time="${roundtrip_time}" controller_ip="${controller_ip}" client_ip="${client_ip}" client_port="${client_port}"/>
     <!-- links - main serial chain -->
     <link name="world"/>

File: kuka_lbr_iiwa_support/urdf/lbr_iiwa_ros2_control.xacro (robot description, xacro)
@@ -1,8 +1,8 @@
 <?xml version="1.0" encoding="UTF-8"?>
 <robot xmlns:xacro="http://www.ros.org/wiki/xacro">
-  <xacro:macro name="kuka_lbr_iiwa_ros2_control" params="name prefix io_access use_fake_hardware roundtrip_time controller_ip client_ip client_port">
+  <xacro:macro name="kuka_lbr_iiwa_ros2_control" params="name prefix io_access mode roundtrip_time controller_ip client_ip client_port">
     <ros2_control name="${name}" type="system">
       <hardware>
-        <xacro:if value="${use_fake_hardware}">
+        <xacro:if value="${mode == 'mock'}">
           <plugin>kuka_mock_hardware_interface::KukaMockHardwareInterface</plugin>
           <param name="cycle_time_ms">5</param>
@@ -11,5 +11,5 @@
           <param name="state_following_offset">0.0</param>
         </xacro:if>
-        <xacro:unless value="${use_fake_hardware}">
+        <xacro:unless value="${mode != 'hardware'}">
           <plugin>kuka_sunrise_fri_driver::KukaFRIHardwareInterface</plugin>
           <param name="controller_ip">${controller_ip}</param>
@@ -124,5 +124,5 @@
         </state_interface>
       </joint>
-      <xacro:unless value="${use_fake_hardware}">
+      <xacro:unless value="${mode != 'hardware'}">
         <xacro:if value="${io_access}">
           <xacro:include filename="$(find kuka_sunrise_fri_driver)/config/gpio_config.xacro"/>
