Commit message: add prefix arg to iiwa

File: kuka_lbr_iiwa_support/urdf/lbr_iiwa14_r820_macro.xacro (robot description, xacro)
@@ -1,5 +1,5 @@
 <?xml version="1.0"?>
 <robot xmlns:xacro="http://wiki.ros.org/xacro">
-  <xacro:macro name="kuka_lbr_iiwa14_r820_robot" params="io_access">
+  <xacro:macro name="kuka_lbr_iiwa14_r820_robot" params="io_access prefix">
   <ros2_control name="iiwa_hardware" type="system">
     <hardware>

Commit message: mesh rename1

File: kuka_lbr_iiwa_support/urdf/lbr_iiwa14_r820_macro.xacro (robot description, xacro)
@@ -149,12 +149,12 @@
     <visual>
       <geometry>
-        <mesh filename="package://kuka_lbr_iiwa_support/meshes/visual/iiwa_r820_link_0_hull_v0.1_iiwa_r820_link_0_hull.stl"/>
-      </geometry>
-      <origin rpy="-0.0 0.0 0.0" xyz="0.0 0.0 0.0"/>
-    </visual>
-    <collision>
-      <origin rpy="-0.0 0.0 0.0" xyz="0.0 0.0 0.0"/>
-      <geometry>
-        <mesh filename="package://kuka_lbr_iiwa_support/meshes/collision/iiwa_r820_link_0_collision_v0.1_iiwa_r820_link_0_collision.stl"/>
+        <mesh filename="package://kuka_lbr_iiwa_support/lbr_iiwa14_r820/meshes/visual/base_link.stl"/>
+      </geometry>
+      <origin rpy="-0.0 0.0 0.0" xyz="0.0 0.0 0.0"/>
+    </visual>
+    <collision>
+      <origin rpy="-0.0 0.0 0.0" xyz="0.0 0.0 0.0"/>
+      <geometry>
+        <mesh filename="package://kuka_lbr_iiwa_support/lbr_iiwa14_r820/meshes/collision/base_link.stl"/>
       </geometry>
     </collision>
@@ -168,12 +168,12 @@
     <visual>
       <geometry>
-        <mesh filename="package://kuka_lbr_iiwa_support/meshes/visual/iiwa_r820_link_1_hull_v0.1_iiwa_r820_link_1_hull.stl"/>
-      </geometry>
-      <origin rpy="-0.0 0.0 0.0" xyz="0.0 0.0 0.0"/>
-    </visual>
-    <collision>
-      <origin rpy="-0.0 0.0 0.0" xyz="0.0 0.0 0.0"/>
-      <geometry>
-        <mesh filename="package://kuka_lbr_iiwa_support/meshes/collision/iiwa_r820_link_1_collision_v0.1_iiwa_r820_link_1_collision.stl"/>
+        <mesh filename="package://kuka_lbr_iiwa_support/lbr_iiwa14_r820/meshes/visual/link_1.stl"/>
+      </geometry>
+      <origin rpy="-0.0 0.0 0.0" xyz="0.0 0.0 0.0"/>
+    </visual>
+    <collision>
+      <origin rpy="-0.0 0.0 0.0" xyz="0.0 0.0 0.0"/>
+      <geometry>
+        <mesh filename="package://kuka_lbr_iiwa_support/lbr_iiwa14_r820/meshes/collision/link_1.stl"/>
       </geometry>
     </collision>
@@ -187,12 +187,12 @@
     <visual>
       <geometry>
-        <mesh filename="package://kuka_lbr_iiwa_support/meshes/visual/iiwa_r820_link_2_hull_v0.1_iiwa_r820_link_2_hull.stl"/>
-      </geometry>
-      <origin rpy="-0.0 0.0 0.0" xyz="0.0 0.0 0.0"/>
-    </visual>
-    <collision>
-      <origin rpy="-0.0 0.0 0.0" xyz="0.0 0.0 0.0"/>
-      <geometry>
-        <mesh filename="package://kuka_lbr_iiwa_support/meshes/collision/iiwa_r820_link_2_collision_v0.1_iiwa_r820_link_2_collision.stl"/>
+        <mesh filename="package://kuka_lbr_iiwa_support/lbr_iiwa14_r820/meshes/visual/link_2.stl"/>
+      </geometry>
+      <origin rpy="-0.0 0.0 0.0" xyz="0.0 0.0 0.0"/>
+    </visual>
+    <collision>
+      <origin rpy="-0.0 0.0 0.0" xyz="0.0 0.0 0.0"/>
+      <geometry>
+        <mesh filename="package://kuka_lbr_iiwa_support/lbr_iiwa14_r820/meshes/collision/link_2.stl"/>
       </geometry>
     </collision>
@@ -206,12 +206,12 @@
     <visual>
       <geometry>
-        <mesh filename="package://kuka_lbr_iiwa_support/meshes/visual/iiwa_r820_link_3_hull_v0.1_iiwa_r820_link_3_hull.stl"/>
-      </geometry>
-      <origin rpy="-0.0 0.0 0.0" xyz="0.0 0.0 0.0"/>
-    </visual>
-    <collision>
-      <origin rpy="-0.0 0.0 0.0" xyz="0.0 0.0 0.0"/>
-      <geometry>
-        <mesh filename="package://kuka_lbr_iiwa_support/meshes/collision/iiwa_r820_link_3_collision_v0.1_iiwa_r820_link_3_collision.stl"/>
+        <mesh filename="package://kuka_lbr_iiwa_support/lbr_iiwa14_r820/meshes/visual/link_3.stl"/>
+      </geometry>
+      <origin rpy="-0.0 0.0 0.0" xyz="0.0 0.0 0.0"/>
+    </visual>
+    <collision>
+      <origin rpy="-0.0 0.0 0.0" xyz="0.0 0.0 0.0"/>
+      <geometry>
+        <mesh filename="package://kuka_lbr_iiwa_support/lbr_iiwa14_r820/meshes/collision/link_3.stl"/>
       </geometry>
     </collision>
@@ -225,12 +225,12 @@
     <visual>
       <geometry>
-        <mesh filename="package://kuka_lbr_iiwa_support/meshes/visual/iiwa_r820_link_4_hull_v0.1_iiwa_r820_link_4_hull.stl"/>
-      </geometry>
-      <origin rpy="-0.0 0.0 0.0" xyz="0.0 0.0 0.0"/>
-    </visual>
-    <collision>
-      <origin rpy="-0.0 0.0 0.0" xyz="0.0 0.0 0.0"/>
-      <geometry>
-        <mesh filename="package://kuka_lbr_iiwa_support/meshes/collision/iiwa_r820_link_4_collision_v0.1_iiwa_r820_link_4_collision.stl"/>
+        <mesh filename="package://kuka_lbr_iiwa_support/lbr_iiwa14_r820/meshes/visual/link_4.stl"/>
+      </geometry>
+      <origin rpy="-0.0 0.0 0.0" xyz="0.0 0.0 0.0"/>
+    </visual>
+    <collision>
+      <origin rpy="-0.0 0.0 0.0" xyz="0.0 0.0 0.0"/>
+      <geometry>
+        <mesh filename="package://kuka_lbr_iiwa_support/lbr_iiwa14_r820/meshes/collision/link_4.stl"/>
       </geometry>
     </collision>
@@ -244,12 +244,12 @@
     <visual>
       <geometry>
-        <mesh filename="package://kuka_lbr_iiwa_support/meshes/visual/iiwa_r820_link_5_hull_v0.1_iiwa_r820_link_5_hull.stl"/>
-      </geometry>
-      <origin rpy="-0.0 0.0 0.0" xyz="0.0 0.0 0.0"/>
-    </visual>
-    <collision>
-      <origin rpy="-0.0 0.0 0.0" xyz="0.0 0.0 0.0"/>
-      <geometry>
-        <mesh filename="package://kuka_lbr_iiwa_support/meshes/collision/iiwa_r820_link_5_collision_v0.1_iiwa_r820_link_5_collision.stl"/>
+        <mesh filename="package://kuka_lbr_iiwa_support/lbr_iiwa14_r820/meshes/visual/link_5.stl"/>
+      </geometry>
+      <origin rpy="-0.0 0.0 0.0" xyz="0.0 0.0 0.0"/>
+    </visual>
+    <collision>
+      <origin rpy="-0.0 0.0 0.0" xyz="0.0 0.0 0.0"/>
+      <geometry>
+        <mesh filename="package://kuka_lbr_iiwa_support/lbr_iiwa14_r820/meshes/collision/link_5.stl"/>
       </geometry>
     </collision>
@@ -263,12 +263,12 @@
     <visual>
       <geometry>
-        <mesh filename="package://kuka_lbr_iiwa_support/meshes/visual/iiwa_r820_link_6_hull_v0.1_iiwa_r820_link_6_hull.stl"/>
-      </geometry>
-      <origin rpy="-0.0 0.0 0.0" xyz="0.0 0.0 0.0"/>
-    </visual>
-    <collision>
-      <origin rpy="-0.0 0.0 0.0" xyz="0.0 0.0 0.0"/>
-      <geometry>
-        <mesh filename="package://kuka_lbr_iiwa_support/meshes/collision/iiwa_r820_link_6_collision_v0.1_iiwa_r820_link_6_collision.stl"/>
+        <mesh filename="package://kuka_lbr_iiwa_support/lbr_iiwa14_r820/meshes/visual/link_6.stl"/>
+      </geometry>
+      <origin rpy="-0.0 0.0 0.0" xyz="0.0 0.0 0.0"/>
+    </visual>
+    <collision>
+      <origin rpy="-0.0 0.0 0.0" xyz="0.0 0.0 0.0"/>
+      <geometry>
+        <mesh filename="package://kuka_lbr_iiwa_support/lbr_iiwa14_r820/meshes/collision/link_6.stl"/>
       </geometry>
     </collision>
@@ -282,12 +282,12 @@
     <visual>
       <geometry>
-        <mesh filename="package://kuka_lbr_iiwa_support/meshes/visual/iiwa_r820_link_7_hull_v0.1_iiwa_r820_link_7_hull.stl"/>
-      </geometry>
-      <origin rpy="-0.0 0.0 0.0" xyz="0.0 0.0 0.0"/>
-    </visual>
-    <collision>
-      <origin rpy="-0.0 0.0 0.0" xyz="0.0 0.0 0.0"/>
-      <geometry>
-        <mesh filename="package://kuka_lbr_iiwa_support/meshes/collision/iiwa_r820_link_7_collision_v0.1_iiwa_r820_link_7_collision.stl"/>
+        <mesh filename="package://kuka_lbr_iiwa_support/lbr_iiwa14_r820/meshes/visual/link_7.stl"/>
+      </geometry>
+      <origin rpy="-0.0 0.0 0.0" xyz="0.0 0.0 0.0"/>
+    </visual>
+    <collision>
+      <origin rpy="-0.0 0.0 0.0" xyz="0.0 0.0 0.0"/>
+      <geometry>
+        <mesh filename="package://kuka_lbr_iiwa_support/lbr_iiwa14_r820/meshes/collision/link_7.stl"/>
       </geometry>
     </collision>

Commit message: iiwa fix

File: kuka_lbr_iiwa_support/urdf/lbr_iiwa14_r820_macro.xacro (robot description, xacro)
@@ -5,8 +5,8 @@
   <xacro:include filename="$(find kuka_resources)/urdf/common_materials.xacro"/>
   <xacro:include filename="$(find kuka_lbr_iiwa_support)/urdf/lbr_iiwa_transmission.xacro" />
-  <xacro:macro name="kuka_lbr_iiwa14_r820_robot" params="io_access prefix use_fake_hardware:=false">
+  <xacro:macro name="kuka_lbr_iiwa14_r820_robot" params="io_access prefix use_fake_hardware *origin">
     <!-- ros2 control instance -->
     <xacro:kuka_lbr_iiwa_ros2_control
-    name="lbr_iiwa14_r820"
+    name="${prefix}lbr_iiwa14_r820"
     prefix="${prefix}"
     io_access = "${io_access}"
@@ -14,5 +14,5 @@
     <!-- links - main serial chain -->
     <!-- links - root element cannot have inertia, therefore a dummy base_link is needed -->
-    <link name="${prefix}base_link"/>
+    <link name="base_link"/>
     <link name="${prefix}base_link_inertia">
       <visual>
@@ -169,7 +169,7 @@
     <!-- joints - main serial chain -->
     <joint name="${prefix}base_link-base_link_inertia" type="fixed">
-      <parent link="${prefix}base_link" />
+      <parent link="base_link" />
       <child link="${prefix}base_link_inertia" />
-      <origin xyz="0 0 0" rpy="0 0 0" />
+      <xacro:insert_block name="origin" />
     </joint>
     <joint name="${prefix}joint_1" type="revolute">
@@ -226,5 +226,5 @@
     <joint name="${prefix}base_link-base" type="fixed">
       <origin xyz="0 0 0" rpy="0 0 0"/>
-      <parent link="${prefix}base_link"/>
+      <parent link="${prefix}base_link_inertia"/>
       <child link="${prefix}base"/>
     </joint>

Commit message: fix iiwa limits

File: kuka_lbr_iiwa_support/urdf/lbr_iiwa14_r820_macro.xacro (robot description, xacro)
@@ -173,5 +173,5 @@
       <origin rpy="-0.0 0.0 0.0" xyz="0.0 0.0 0.1375"/>
       <axis xyz="0.0 0.0 1.0"/>
-      <limit effort="158.4" lower="-2.67035" upper="2.67035" velocity="6.283"/>
+      <limit effort="0" lower="${radians(-170)}" upper="${radians(170)}" velocity="${radians(85)}"/>
     </joint>
     <joint name="${prefix}joint_2" type="revolute">
@@ -180,5 +180,5 @@
       <origin rpy="-0.0 0.0 0.0" xyz="0.0 0.0 0.2025"/>
       <axis xyz="0.0 1.0 0.0"/>
-      <limit effort="158.4" lower="-1.8849" upper="1.8849" velocity="6.283"/>
+      <limit effort="0" lower="${radians(-120)}" upper="${radians(120)}" velocity="${radians(85)}"/>
     </joint>
     <joint name="${prefix}joint_3" type="revolute">
@@ -187,5 +187,5 @@
       <origin rpy="-0.0 0.0 0.0" xyz="0.0 0.0 0.1845"/>
       <axis xyz="0.0 0.0 1.0"/>
-      <limit effort="99" lower="-2.67035" upper="2.67035" velocity="6.283"/>
+      <limit effort="0" lower="${radians(-170)}" upper="${radians(170)}" velocity="${radians(100)}"/>
     </joint>
     <joint name="${prefix}joint_4" type="revolute">
@@ -194,5 +194,5 @@
       <origin rpy="-0.0 0.0 0.0" xyz="0.0 0.0 0.2155"/>
       <axis xyz="0.0 -1.0 0.0"/>
-      <limit effort="99" lower="-1.8849" upper="1.8849" velocity="6.283"/>
+      <limit effort="0" lower="${radians(-120)}" upper="${radians(120)}" velocity="${radians(75)}"/>
     </joint>
     <joint name="${prefix}joint_5" type="revolute">
@@ -201,5 +201,5 @@
       <origin rpy="-0.0 0.0 0.0" xyz="0.0 0.0 0.1845"/>
       <axis xyz="0.0 0.0 1.0"/>
-      <limit effort="99" lower="-2.67035" upper="2.67035" velocity="6.283"/>
+      <limit effort="0" lower="${radians(-170)}" upper="${radians(170)}" velocity="${radians(130)}"/>
     </joint>
     <joint name="${prefix}joint_6" type="revolute">
@@ -208,5 +208,5 @@
       <origin rpy="-0.0 0.0 0.0" xyz="0.0 0.0 0.2155"/>
       <axis xyz="0.0 1.0 0.0"/>
-      <limit effort="36" lower="-1.8849" upper="1.8849" velocity="6.283"/>
+      <limit effort="0" lower="${radians(-120)}" upper="${radians(120)}" velocity="${radians(135)}"/>
     </joint>
     <joint name="${prefix}joint_7" type="revolute">
@@ -215,5 +215,5 @@
       <origin rpy="-0.0 0.0 0.0" xyz="0.0 0.0 0.081"/>
       <axis xyz="0.0 0.0 1.0"/>
-      <limit effort="36" lower="-2.74889" upper="2.74889" velocity="6.283"/>
+      <limit effort="0" lower="${radians(-175)}" upper="${radians(175)}" velocity="${radians(135)}"/>
     </joint>
     <!-- ROS-Industrial 'base' frame - equivalent of 'KUKA ROBROOT'-->

Commit message: Prepare first ROS2 release (#57)
* fix iiwa limits

* remove invalid info

* fix md

* collision iisy15

* collision iiwa14

* collision kr10

* collision kr16

* collision kr210r2700

* collision kr210r3100

* update md

* generate changelogs

* format

---------

Co-authored-by: Aron Svastits <svastits1@gmail.com>

File: kuka_lbr_iiwa_support/urdf/lbr_iiwa14_r820_macro.xacro (robot description, xacro)
@@ -23,9 +23,4 @@
         </geometry>
       </collision>
-      <inertial>
-        <mass value="3.2832"/>
-        <origin rpy="0 0 0" xyz="0.0 0.0 0.0"/>
-        <inertia ixx="5.0E-4" ixy="0.0" ixz="0.0" iyy="5.0E-4" iyz="0.0" izz="5.0E-4"/>
-      </inertial>
     </link>
     <link name="${prefix}link_1">
@@ -42,9 +37,4 @@
         </geometry>
       </collision>
-      <inertial>
-        <mass value="6.495"/>
-        <origin rpy="0 0 0" xyz="0.0 0.0 0.0"/>
-        <inertia ixx="0.06907" ixy="0.0" ixz="0.0" iyy="0.0711" iyz="0.0" izz="0.02"/>
-      </inertial>
     </link>
     <link name="${prefix}link_2">
@@ -61,9 +51,4 @@
         </geometry>
       </collision>
-      <inertial>
-        <mass value="8.365"/>
-        <origin rpy="0 0 0" xyz="0.0 0.0 0.0"/>
-        <inertia ixx="0.08" ixy="0.0" ixz="0.0" iyy="0.08" iyz="0.0" izz="0.01"/>
-      </inertial>
     </link>
     <link name="${prefix}link_3">
@@ -80,9 +65,4 @@
         </geometry>
       </collision>
-      <inertial>
-        <mass value="2.5697"/>
-        <origin rpy="0 0 0" xyz="0.0 0.0 0.0"/>
-        <inertia ixx="0.02" ixy="0.0" ixz="0.0" iyy="0.02" iyz="0.0" izz="0.06"/>
-      </inertial>
     </link>
     <link name="${prefix}link_4">
@@ -99,9 +79,4 @@
         </geometry>
       </collision>
-      <inertial>
-        <mass value="5.41"/>
-        <origin rpy="0 0 0" xyz="0.0 0.0 0.0"/>
-        <inertia ixx="0.04" ixy="0.0" ixz="0.0" iyy="0.03" iyz="0.0" izz="0.01"/>
-      </inertial>
     </link>
     <link name="${prefix}link_5">
@@ -118,9 +93,4 @@
         </geometry>
       </collision>
-      <inertial>
-        <mass value="1.867"/>
-        <origin rpy="0 0 0" xyz="0.0 0.0 0.0"/>
-        <inertia ixx="0.01" ixy="0.0" ixz="0.0" iyy="0.01" iyz="0.0" izz="0.01"/>
-      </inertial>
     </link>
     <link name="${prefix}link_6">
@@ -137,9 +107,4 @@
         </geometry>
       </collision>
-      <inertial>
-        <mass value="2.458"/>
-        <origin rpy="0 0 0" xyz="0.0 0.0 0.0"/>
-        <inertia ixx="0.007" ixy="0.0" ixz="0.0" iyy="0.006" iyz="0.0" izz="0.005"/>
-      </inertial>
     </link>
     <link name="${prefix}link_7">
@@ -156,9 +121,4 @@
         </geometry>
       </collision>
-      <inertial>
-        <mass value="0.627"/>
-        <origin rpy="0 0 0" xyz="0.0 0.0 0.0"/>
-        <inertia ixx="3.0E-4" ixy="0.0" ixz="0.0" iyy="3.0E-4" iyz="0.0" izz="5.0E-4"/>
-      </inertial>
     </link>
     <!-- joints - main serial chain -->
@@ -173,5 +133,5 @@
       <origin rpy="-0.0 0.0 0.0" xyz="0.0 0.0 0.1375"/>
       <axis xyz="0.0 0.0 1.0"/>
-      <limit effort="158.4" lower="-2.67035" upper="2.67035" velocity="6.283"/>
+      <limit effort="0" lower="${radians(-170)}" upper="${radians(170)}" velocity="${radians(85)}"/>
     </joint>
     <joint name="${prefix}joint_2" type="revolute">
@@ -180,5 +140,5 @@
       <origin rpy="-0.0 0.0 0.0" xyz="0.0 0.0 0.2025"/>
       <axis xyz="0.0 1.0 0.0"/>
-      <limit effort="158.4" lower="-1.8849" upper="1.8849" velocity="6.283"/>
+      <limit effort="0" lower="${radians(-120)}" upper="${radians(120)}" velocity="${radians(85)}"/>
     </joint>
     <joint name="${prefix}joint_3" type="revolute">
@@ -187,5 +147,5 @@
       <origin rpy="-0.0 0.0 0.0" xyz="0.0 0.0 0.1845"/>
       <axis xyz="0.0 0.0 1.0"/>
-      <limit effort="99" lower="-2.67035" upper="2.67035" velocity="6.283"/>
+      <limit effort="0" lower="${radians(-170)}" upper="${radians(170)}" velocity="${radians(100)}"/>
     </joint>
     <joint name="${prefix}joint_4" type="revolute">
@@ -194,5 +154,5 @@
       <origin rpy="-0.0 0.0 0.0" xyz="0.0 0.0 0.2155"/>
       <axis xyz="0.0 -1.0 0.0"/>
-      <limit effort="99" lower="-1.8849" upper="1.8849" velocity="6.283"/>
+      <limit effort="0" lower="${radians(-120)}" upper="${radians(120)}" velocity="${radians(75)}"/>
     </joint>
     <joint name="${prefix}joint_5" type="revolute">
@@ -201,5 +161,5 @@
       <origin rpy="-0.0 0.0 0.0" xyz="0.0 0.0 0.1845"/>
       <axis xyz="0.0 0.0 1.0"/>
-      <limit effort="99" lower="-2.67035" upper="2.67035" velocity="6.283"/>
+      <limit effort="0" lower="${radians(-170)}" upper="${radians(170)}" velocity="${radians(130)}"/>
     </joint>
     <joint name="${prefix}joint_6" type="revolute">
@@ -208,5 +168,5 @@
       <origin rpy="-0.0 0.0 0.0" xyz="0.0 0.0 0.2155"/>
       <axis xyz="0.0 1.0 0.0"/>
-      <limit effort="36" lower="-1.8849" upper="1.8849" velocity="6.283"/>
+      <limit effort="0" lower="${radians(-120)}" upper="${radians(120)}" velocity="${radians(135)}"/>
     </joint>
     <joint name="${prefix}joint_7" type="revolute">
@@ -215,5 +175,5 @@
       <origin rpy="-0.0 0.0 0.0" xyz="0.0 0.0 0.081"/>
       <axis xyz="0.0 0.0 1.0"/>
-      <limit effort="36" lower="-2.74889" upper="2.74889" velocity="6.283"/>
+      <limit effort="0" lower="${radians(-175)}" upper="${radians(175)}" velocity="${radians(135)}"/>
     </joint>
     <!-- ROS-Industrial 'base' frame - equivalent of 'KUKA ROBROOT'-->

Commit message: add dummy cart joint to urdf, jazzy requirement

File: kuka_lbr_iiwa_support/urdf/lbr_iiwa14_r820_macro.xacro (robot description, xacro)
@@ -198,4 +198,44 @@
       <origin rpy="-0.0 0.0 0.0" xyz="0.0 0.0 0.071"/>
     </joint>
+    <joint name="${prefix}dummy_cart_joint/x" type="continuous">
+      <parent link="world"/>
+      <child link="${prefix}base_link"/>
+    </joint>
+    <joint name="${prefix}dummy_cart_joint/y" type="continuous">
+      <parent link="world"/>
+      <child link="${prefix}base_link"/>
+    </joint>
+    <joint name="${prefix}dummy_cart_joint/z" type="continuous">
+      <parent link="world"/>
+      <child link="${prefix}base_link"/>
+    </joint>
+    <joint name="${prefix}dummy_cart_joint/a" type="continuous">
+      <parent link="world"/>
+      <child link="${prefix}base_link"/>
+    </joint>
+    <joint name="${prefix}dummy_cart_joint/b" type="continuous">
+      <parent link="world"/>
+      <child link="${prefix}base_link"/>
+    </joint>
+    <joint name="${prefix}dummy_cart_joint/c" type="continuous">
+      <parent link="world"/>
+      <child link="${prefix}base_link"/>
+    </joint>
+    <joint name="${prefix}dummy_cart_joint/qw" type="continuous">
+      <parent link="world"/>
+      <child link="${prefix}base_link"/>
+    </joint>
+    <joint name="${prefix}dummy_cart_joint/qx" type="continuous">
+      <parent link="world"/>
+      <child link="${prefix}base_link"/>
+    </joint>
+    <joint name="${prefix}dummy_cart_joint/qy" type="continuous">
+      <parent link="world"/>
+      <child link="${prefix}base_link"/>
+    </joint>
+    <joint name="${prefix}dummy_cart_joint/qz" type="continuous">
+      <parent link="world"/>
+      <child link="${prefix}base_link"/>
+    </joint>
   </xacro:macro>
 </robot>

Commit message: Fix iiwa 14 dimensions

File: kuka_lbr_iiwa_support/urdf/lbr_iiwa14_r820_macro.xacro (robot description, xacro)
@@ -131,5 +131,5 @@
       <parent link="${prefix}base_link"/>
       <child link="${prefix}link_1"/>
-      <origin rpy="-0.0 0.0 0.0" xyz="0.0 0.0 0.1375"/>
+      <origin rpy="-0.0 0.0 0.0" xyz="0.0 0.0 0.1575"/>
       <axis xyz="0.0 0.0 1.0"/>
       <limit effort="0" lower="${radians(-170)}" upper="${radians(170)}" velocity="${radians(85)}"/>
@@ -145,5 +145,5 @@
       <parent link="${prefix}link_2"/>
       <child link="${prefix}link_3"/>
-      <origin rpy="-0.0 0.0 0.0" xyz="0.0 0.0 0.1845"/>
+      <origin rpy="-0.0 0.0 0.0" xyz="0.0 0.0 0.2045"/>
       <axis xyz="0.0 0.0 1.0"/>
       <limit effort="0" lower="${radians(-170)}" upper="${radians(170)}" velocity="${radians(100)}"/>
