Commit message: Add gpio config to kr iontec

File: kuka_iontec_support/urdf/kr70_r2100.urdf.xacro (robot description, xacro)
@@ -5,4 +5,5 @@
   <!-- Read additional arguments  -->
   <xacro:arg name="use_fake_hardware" default="false"/>
+  <xacro:arg name="use_gpio" default="true"/>
   <xacro:arg name="roundtrip_time" default="0"/>
   <xacro:arg name="client_ip" default="0.0.0.0"/>
@@ -16,5 +17,5 @@
   <xacro:arg name="pitch" default="0"/>
   <xacro:arg name="yaw" default="0"/>
-  <xacro:kuka_kr70_r2100_robot client_ip="$(arg client_ip)" client_port="$(arg client_port)" controller_ip="$(arg controller_ip)" prefix="$(arg prefix)" use_fake_hardware="$(arg use_fake_hardware)" roundtrip_time="$(arg roundtrip_time)">
+  <xacro:kuka_kr70_r2100_robot client_ip="$(arg client_ip)" client_port="$(arg client_port)" controller_ip="$(arg controller_ip)" prefix="$(arg prefix)" use_fake_hardware="$(arg use_fake_hardware)" use_gpio="$(arg use_gpio)" roundtrip_time="$(arg roundtrip_time)">
     <origin xyz="$(arg x) $(arg y) $(arg z)" rpy="$(arg roll) $(arg pitch) $(arg yaw)"/>
   </xacro:kuka_kr70_r2100_robot>

File: kuka_iontec_support/urdf/kr70_r2100_macro.xacro (robot description, xacro)
@@ -3,7 +3,7 @@
   <xacro:include filename="$(find kuka_iontec_support)/urdf/kr_iontec_ros2_control.xacro"/>
   <xacro:include filename="$(find kuka_iontec_support)/urdf/kr_iontec_transmission.xacro"/>
-  <xacro:macro name="kuka_kr70_r2100_robot" params="client_ip client_port controller_ip prefix use_fake_hardware roundtrip_time *origin">
+  <xacro:macro name="kuka_kr70_r2100_robot" params="client_ip client_port controller_ip prefix use_fake_hardware use_gpio roundtrip_time *origin">
     <!-- ros2 control instance -->
-    <xacro:kuka_iontec_ros2_control name="${prefix}kr70_r2100" client_ip="${client_ip}" controller_ip="${controller_ip}" client_port="${client_port}" prefix="${prefix}" use_fake_hardware="${use_fake_hardware}" roundtrip_time="${roundtrip_time}"/>
+    <xacro:kuka_iontec_ros2_control name="${prefix}kr70_r2100" client_ip="${client_ip}" controller_ip="${controller_ip}" client_port="${client_port}" prefix="${prefix}" use_fake_hardware="${use_fake_hardware}" use_gpio="${use_gpio}" roundtrip_time="${roundtrip_time}"/>
     <link name="world"/>
     <link name="${prefix}base_link">

File: kuka_iontec_support/urdf/kr_iontec_ros2_control.xacro (robot description, xacro)
@@ -1,5 +1,5 @@
 <?xml version="1.0" encoding="UTF-8"?>
 <robot xmlns:xacro="http://www.ros.org/wiki/xacro">
-  <xacro:macro name="kuka_iontec_ros2_control" params="name client_ip client_port controller_ip prefix use_fake_hardware roundtrip_time">
+  <xacro:macro name="kuka_iontec_ros2_control" params="name client_ip client_port controller_ip prefix use_fake_hardware use_gpio roundtrip_time">
     <ros2_control name="${name}" type="system">
       <hardware>
@@ -54,4 +54,8 @@
         </state_interface>
       </joint>
+      <xacro:if value="${use_gpio}">
+        <xacro:include filename="$(find kuka_iontec_support)/urdf/kr_iontec_gpio_config.xacro"/>
+        <xacro:kr_iontec_gpio_config/>
+      </xacro:if>
     </ros2_control>
   </xacro:macro>
