Commit message: add rest of necessary files, separate to moveit+non-moveit pkgs - TODO not ok yet

File: ext_axis_examples/urdf/dummy_rail.xacro (robot description, xacro)
@@ -1,5 +1,5 @@
 <?xml version="1.0" encoding="UTF-8"?>
 <robot xmlns:xacro="http://www.ros.org/wiki/xacro">
-  <xacro:macro name="dummy_rail_ext_axes_links" params="">
+  <xacro:macro name="dummy_rail_links" params="">
     <!-- links -->
     <link name="rail_link">
@@ -12,5 +12,5 @@
     </link>
   </xacro:macro>
-  <xacro:macro name="dummy_rail_ext_axes_joints" params="robot_base_link">
+  <xacro:macro name="dummy_rail_joints" params="robot_base_link">
     <!-- joints -->
     <joint name="world-rail_link" type="fixed">
@@ -27,5 +27,5 @@
     </joint>
   </xacro:macro>
-  <xacro:macro name="dummy_rail_ext_axes_ros2_control_joints" params="">
+  <xacro:macro name="dummy_rail_ros2_control_joints" params="">
     <!-- ros2 control joints -->
     <joint name="rail_joint">
@@ -36,3 +36,11 @@
     </joint>
   </xacro:macro>
+  <xacro::macro name="dummy_rail_srdf_adjacent_links" params="">
+    <!-- adjacent links -->
+    <disable_collisions link1="rail_link" link2="base_link" reason="Adjacent"/>
+  </xacro::macro>
+  <xacro:macro name="dummy_rail_srdf_joints" params="">
+    <!-- srdf joints TODO remove redundancy -->
+    <joint name="rail_joint" value="0"/>
+  </xacro:macro>
 </robot>

File: ext_axis_examples/urdf/kr10_r1100_2_with_dummy_rail.urdf.xacro (robot description, xacro)
@@ -23,5 +23,5 @@
   <xacro:kuka_agilus_ros2_control name="$(arg prefix)kr10_r1100_2_with_dummy_rail" driver_version="$(arg driver_version)" client_ip="$(arg client_ip)" client_port="$(arg client_port)" controller_ip="$(arg controller_ip)" prefix="$(arg prefix)" mode="$(arg mode)" use_gpio="$(arg use_gpio)" roundtrip_time="$(arg roundtrip_time)" verify_robot_model="$(arg verify_robot_model)" use_ext_axes="true">
     <ext_axes_ros2_control_joints>
-      <xacro:dummy_rail_ext_axes_ros2_control_joints/>
+      <xacro:dummy_rail_ros2_control_joints/>
     </ext_axes_ros2_control_joints>
   </xacro:kuka_agilus_ros2_control>
@@ -29,8 +29,8 @@
     <origin xyz="$(arg x) $(arg y) $(arg z)" rpy="$(arg roll) $(arg pitch) $(arg yaw)"/>
     <ext_axes_links>
-      <xacro:dummy_rail_ext_axes_links/>
+      <xacro:dummy_rail_links/>
     </ext_axes_links>
     <ext_axes_joints>
-      <xacro:dummy_rail_ext_axes_joints robot_base_link="$(arg prefix)base_link"/>
+      <xacro:dummy_rail_joints robot_base_link="$(arg prefix)base_link"/>
     </ext_axes_joints>
   </xacro:kuka_kr10_r1100_2_robot>

Commit message: fix issues in ext axis moveit config

File: ext_axis_examples/urdf/dummy_rail.xacro (robot description, xacro)
@@ -36,8 +36,8 @@
     </joint>
   </xacro:macro>
-  <xacro::macro name="dummy_rail_srdf_adjacent_links" params="">
+  <xacro:macro name="dummy_rail_srdf_adjacent_links" params="">
     <!-- adjacent links -->
     <disable_collisions link1="rail_link" link2="base_link" reason="Adjacent"/>
-  </xacro::macro>
+  </xacro:macro>
   <xacro:macro name="dummy_rail_srdf_joints" params="">
     <!-- srdf joints TODO remove redundancy -->

File: ext_axis_examples_moveit_config/srdf/6_axis_macro.xacro (robot description, xacro)
@@ -16,5 +16,5 @@
     <!--GROUP STATES: Purpose: Define a named state for a particular group, in terms of joint values. This is useful to define states like 'folded arms'-->
     <group_state name="home" group="${prefix}manipulator">
-      <xacro::insert_block name="ext_joints"/>
+      <xacro:insert_block name="ext_joints"/>
       <joint name="${prefix}joint_1" value="0"/>
       <joint name="${prefix}joint_2" value="${-pi/2}"/>
@@ -27,5 +27,5 @@
     <end_effector name="${prefix}eef" parent_link="${prefix}tool0" group="${prefix}end_effector" parent_group="${prefix}manipulator"/>
     <!--DISABLE COLLISIONS: By default it is assumed that any link of the robot could potentially come into collision with any other link in the robot. This tag disables collision checking between a specified pair of links. -->
-    <xacro::insert_block name="ext_adjacent_links"/>
+    <xacro:insert_block name="ext_adjacent_links"/>
     <disable_collisions link1="${prefix}base_link" link2="${prefix}link_1" reason="Adjacent"/>
     <disable_collisions link1="${prefix}link_1" link2="${prefix}link_2" reason="Adjacent"/>

Commit message: fix formatting

File: ext_axis_examples/urdf/dummy_rail.xacro (robot description, xacro)
@@ -6,5 +6,5 @@
       <visual>
         <geometry>
-           <box size="2 0.2 0.2"/>
+          <box size="2 0.2 0.2"/>
         </geometry>
         <xacro:material_kuka_black/>

Commit message: add ext axes support for kr16_r2010_2, fix upcoming issues

File: ext_axis_examples/urdf/dummy_rail.xacro (robot description, xacro)
@@ -1,4 +1,5 @@
 <?xml version="1.0" encoding="UTF-8"?>
 <robot xmlns:xacro="http://www.ros.org/wiki/xacro">
+  <xacro:include filename="$(find kuka_resources)/urdf/common_materials.xacro"/>
   <xacro:macro name="dummy_rail_links" params="">
     <!-- links -->

File: kuka_cybertech_support/urdf/kr16_r2010_2.urdf.xacro (robot description, xacro)
@@ -20,7 +20,11 @@
   <xacro:arg name="pitch" default="0"/>
   <xacro:arg name="yaw" default="0"/>
-  <xacro:kuka_cybertech_ros2_control name="$(arg prefix)kr16_r2010_2" driver_version="$(arg driver_version)" client_ip="$(arg client_ip)" client_port="$(arg client_port)" controller_ip="$(arg controller_ip)" prefix="$(arg prefix)" mode="$(arg mode)" use_gpio="$(arg use_gpio)" roundtrip_time="$(arg roundtrip_time)" verify_robot_model="$(arg verify_robot_model)"/>
-  <xacro:kuka_kr16_r2010_2_robot prefix="$(arg prefix)" package_name="kuka_cybertech_support">
+  <xacro:kuka_cybertech_ros2_control name="$(arg prefix)kr10_r1100_2" driver_version="$(arg driver_version)" client_ip="$(arg client_ip)" client_port="$(arg client_port)" controller_ip="$(arg controller_ip)" prefix="$(arg prefix)" mode="$(arg mode)" use_gpio="$(arg use_gpio)" roundtrip_time="$(arg roundtrip_time)" verify_robot_model="$(arg verify_robot_model)" use_ext_axes="false">
+    <ext_axes_ros2_control_joints/>
+  </xacro:kuka_cybertech_ros2_control>
+  <xacro:kuka_kr16_r2010_2_robot prefix="$(arg prefix)" package_name="kuka_cybertech_support" use_ext_axes="false">
     <origin xyz="$(arg x) $(arg y) $(arg z)" rpy="$(arg roll) $(arg pitch) $(arg yaw)"/>
+    <ext_axes_links/>
+    <ext_axes_joints/>
   </xacro:kuka_kr16_r2010_2_robot>
 </robot>

File: kuka_cybertech_support/urdf/kr16_r2010_2_macro.xacro (robot description, xacro)
@@ -1,7 +1,10 @@
 <?xml version="1.0"?>
 <robot xmlns:xacro="http://wiki.ros.org/xacro">
-  <xacro:macro name="kuka_kr16_r2010_2_robot" params="prefix package_name *origin">
+  <xacro:macro name="kuka_kr16_r2010_2_robot" params="prefix package_name use_ext_axes *origin **ext_axes_links **ext_axes_joints">
     <!-- links - main serial chain -->
     <link name="world"/>
+    <xacro:if value="${use_ext_axes}">
+      <xacro:insert_block name="ext_axes_links"/>
+    </xacro:if>
     <link name="${prefix}base_link">
       <collision>
@@ -102,9 +105,14 @@
       </visual>
     </link>
-    <joint name="${prefix}world-base_link" type="fixed">
-      <parent link="world"/>
-      <child link="${prefix}base_link"/>
-      <xacro:insert_block name="origin"/>
-    </joint>
+    <xacro:if value="${use_ext_axes}">
+      <xacro:insert_block name="ext_axes_joints"/>
+    </xacro:if>
+    <xacro:unless value="${use_ext_axes}">
+      <joint name="${prefix}world-base_link" type="fixed">
+        <parent link="world"/>
+        <child link="${prefix}base_link"/>
+        <xacro:insert_block name="origin"/>
+      </joint>
+    </xacro:unless>
     <joint name="${prefix}joint_1" type="revolute">
       <axis xyz="0.0 0.0 1.0"/>

File: kuka_cybertech_support/urdf/kr_cybertech_ros2_control_macro.xacro (robot description, xacro)
@@ -1,5 +1,5 @@
 <?xml version="1.0" encoding="UTF-8"?>
 <robot xmlns:xacro="http://www.ros.org/wiki/xacro">
-  <xacro:macro name="kuka_cybertech_ros2_control" params="name driver_version client_ip client_port controller_ip prefix mode use_gpio roundtrip_time verify_robot_model">
+  <xacro:macro name="kuka_cybertech_ros2_control" params="name driver_version client_ip client_port controller_ip prefix mode use_gpio roundtrip_time verify_robot_model use_ext_axes **ext_axes_ros2_control_joints">
     <!-- gazebo -->
     <xacro:if value="${mode == 'gazebo'}">
@@ -32,4 +32,7 @@
         </xacro:if>
       </hardware>
+      <xacro:if value="${use_ext_axes}">
+        <xacro:insert_block name="ext_axes_ros2_control_joints"/>
+      </xacro:if>
       <joint name="${prefix}joint_1">
         <command_interface name="position"/>
