Commit message: refactor - rm use_ext_axes xacro param for urdfs

File: ext_axis_examples/urdf/dummy_rail.xacro (robot description, xacro)
@@ -13,10 +13,10 @@
     </link>
   </xacro:macro>
-  <xacro:macro name="dummy_rail_joints" params="robot_base_link">
+  <xacro:macro name="dummy_rail_joints" params="robot_base_link *origin">
     <!-- joints -->
     <joint name="world-rail_link" type="fixed">
       <parent link="world"/>
       <child link="rail_link"/>
-      <origin rpy="0.0 0.0 0.0" xyz="0.0 0.0 0.0"/>
+      <xacro:insert_block name="origin"/>
     </joint>
     <joint name="rail_joint" type="prismatic">

File: ext_axis_examples/urdf/kr10_r1100_2_with_dummy_rail.urdf.xacro (robot description, xacro)
@@ -21,16 +21,17 @@
   <xacro:arg name="pitch" default="0"/>
   <xacro:arg name="yaw" default="0"/>
-  <xacro:kuka_agilus_ros2_control name="$(arg prefix)kr10_r1100_2_with_dummy_rail" driver_version="$(arg driver_version)" client_ip="$(arg client_ip)" client_port="$(arg client_port)" controller_ip="$(arg controller_ip)" prefix="$(arg prefix)" mode="$(arg mode)" use_gpio="$(arg use_gpio)" roundtrip_time="$(arg roundtrip_time)" verify_robot_model="$(arg verify_robot_model)" use_ext_axes="true">
+  <xacro:kuka_agilus_ros2_control name="$(arg prefix)kr10_r1100_2_with_dummy_rail" driver_version="$(arg driver_version)" client_ip="$(arg client_ip)" client_port="$(arg client_port)" controller_ip="$(arg controller_ip)" prefix="$(arg prefix)" mode="$(arg mode)" use_gpio="$(arg use_gpio)" roundtrip_time="$(arg roundtrip_time)" verify_robot_model="$(arg verify_robot_model)">
     <ext_axes_ros2_control_joints>
       <xacro:dummy_rail_ros2_control_joints/>
     </ext_axes_ros2_control_joints>
   </xacro:kuka_agilus_ros2_control>
-  <xacro:kuka_kr10_r1100_2_robot prefix="$(arg prefix)" package_name="kuka_agilus_support" use_ext_axes="true">
-    <origin xyz="$(arg x) $(arg y) $(arg z)" rpy="$(arg roll) $(arg pitch) $(arg yaw)"/>
+  <xacro:kuka_kr10_r1100_2_robot prefix="$(arg prefix)" package_name="kuka_agilus_support">
     <ext_axes_links>
       <xacro:dummy_rail_links/>
     </ext_axes_links>
     <ext_axes_joints>
-      <xacro:dummy_rail_joints robot_base_link="$(arg prefix)base_link"/>
+      <xacro:dummy_rail_joints robot_base_link="$(arg prefix)base_link">
+        <origin xyz="$(arg x) $(arg y) $(arg z)" rpy="$(arg roll) $(arg pitch) $(arg yaw)"/>
+      </xacro:dummy_rail_joints>
     </ext_axes_joints>
   </xacro:kuka_kr10_r1100_2_robot>

File: ext_axis_examples/urdf/kr16_r2010_2_with_dummy_rail.urdf.xacro (robot description, xacro)
@@ -21,17 +21,18 @@
   <xacro:arg name="pitch" default="0"/>
   <xacro:arg name="yaw" default="0"/>
-  <xacro:kuka_cybertech_ros2_control name="$(arg prefix)kr16_r2010_2_with_dummy_rail" driver_version="$(arg driver_version)" client_ip="$(arg client_ip)" client_port="$(arg client_port)" controller_ip="$(arg controller_ip)" prefix="$(arg prefix)" mode="$(arg mode)" use_gpio="$(arg use_gpio)" roundtrip_time="$(arg roundtrip_time)" verify_robot_model="$(arg verify_robot_model)" use_ext_axes="true">
+  <xacro:kuka_cybertech_ros2_control name="$(arg prefix)kr16_r2010_2_with_dummy_rail" driver_version="$(arg driver_version)" client_ip="$(arg client_ip)" client_port="$(arg client_port)" controller_ip="$(arg controller_ip)" prefix="$(arg prefix)" mode="$(arg mode)" use_gpio="$(arg use_gpio)" roundtrip_time="$(arg roundtrip_time)" verify_robot_model="$(arg verify_robot_model)">
     <ext_axes_ros2_control_joints>
       <xacro:dummy_rail_ros2_control_joints/>
     </ext_axes_ros2_control_joints>
   </xacro:kuka_cybertech_ros2_control>
-  <xacro:kuka_kr16_r2010_2_robot prefix="$(arg prefix)" package_name="kuka_cybertech_support" use_ext_axes="true">
-    <origin xyz="$(arg x) $(arg y) $(arg z)" rpy="$(arg roll) $(arg pitch) $(arg yaw)"/>
+  <xacro:kuka_kr16_r2010_2_robot prefix="$(arg prefix)" package_name="kuka_cybertech_support">
     <ext_axes_links>
       <xacro:dummy_rail_links/>
     </ext_axes_links>
-    <ext_axes_joints>
-      <xacro:dummy_rail_joints robot_base_link="$(arg prefix)base_link"/>
-    </ext_axes_joints>
+    <world-base_link_joints>
+      <xacro:dummy_rail_joints robot_base_link="$(arg prefix)base_link">
+        <origin xyz="$(arg x) $(arg y) $(arg z)" rpy="$(arg roll) $(arg pitch) $(arg yaw)"/>
+      </xacro:dummy_rail_joints>
+    </world-base_link_joints>
   </xacro:kuka_kr16_r2010_2_robot>
 </robot>

File: kuka_agilus_support/urdf/kr10_r1100_2.urdf.xacro (robot description, xacro)
@@ -20,11 +20,16 @@
   <xacro:arg name="pitch" default="0"/>
   <xacro:arg name="yaw" default="0"/>
-  <xacro:kuka_agilus_ros2_control name="$(arg prefix)kr10_r1100_2" driver_version="$(arg driver_version)" client_ip="$(arg client_ip)" client_port="$(arg client_port)" controller_ip="$(arg controller_ip)" prefix="$(arg prefix)" mode="$(arg mode)" use_gpio="$(arg use_gpio)" roundtrip_time="$(arg roundtrip_time)" verify_robot_model="$(arg verify_robot_model)" use_ext_axes="false">
+  <xacro:kuka_agilus_ros2_control name="$(arg prefix)kr10_r1100_2" driver_version="$(arg driver_version)" client_ip="$(arg client_ip)" client_port="$(arg client_port)" controller_ip="$(arg controller_ip)" prefix="$(arg prefix)" mode="$(arg mode)" use_gpio="$(arg use_gpio)" roundtrip_time="$(arg roundtrip_time)" verify_robot_model="$(arg verify_robot_model)">
     <ext_axes_ros2_control_joints/>
   </xacro:kuka_agilus_ros2_control>
-  <xacro:kuka_kr10_r1100_2_robot prefix="$(arg prefix)" package_name="kuka_agilus_support" use_ext_axes="false">
-    <origin xyz="$(arg x) $(arg y) $(arg z)" rpy="$(arg roll) $(arg pitch) $(arg yaw)"/>
+  <xacro:kuka_kr10_r1100_2_robot prefix="$(arg prefix)" package_name="kuka_agilus_support">
     <ext_axes_links/>
-    <ext_axes_joints/>
+    <world-base_link_joints>
+      <joint name="$(arg prefix)world-base_link" type="fixed">
+        <parent link="world"/>
+        <child link="$(arg prefix)base_link"/>
+        <origin xyz="$(arg x) $(arg y) $(arg z)" rpy="$(arg roll) $(arg pitch) $(arg yaw)"/>
+      </joint>
+    </world-base_link_joints>
   </xacro:kuka_kr10_r1100_2_robot>
 </robot>

File: kuka_agilus_support/urdf/kr10_r1100_2_macro.xacro (robot description, xacro)
@@ -3,10 +3,8 @@
   <!-- include helper xacros -->
   <xacro:include filename="$(find kuka_resources)/urdf/common_materials.xacro"/>
-  <xacro:macro name="kuka_kr10_r1100_2_robot" params="prefix package_name use_ext_axes *origin **ext_axes_links **ext_axes_joints">
+  <xacro:macro name="kuka_kr10_r1100_2_robot" params="prefix package_name **ext_axes_links **world-base_link_joints">
     <!-- links - main serial chain -->
     <link name="world"/>
-    <xacro:if value="${use_ext_axes}">
-      <xacro:insert_block name="ext_axes_links"/>
-    </xacro:if>
+    <xacro:insert_block name="ext_axes_links"/>
     <link name="${prefix}base_link">
       <collision>
@@ -150,14 +148,5 @@
     </link>
     <!-- joints - main serial chain -->
-    <xacro:if value="${use_ext_axes}">
-      <xacro:insert_block name="ext_axes_joints"/>
-    </xacro:if>
-    <xacro:unless value="${use_ext_axes}">
-      <joint name="${prefix}world-base_link" type="fixed">
-        <parent link="world"/>
-        <child link="${prefix}base_link"/>
-        <xacro:insert_block name="origin"/>
-      </joint>
-    </xacro:unless>
+    <xacro:insert_block name="world-base_link_joints"/>
     <joint name="${prefix}joint_1" type="revolute">
       <axis xyz="0.0 0.0 1.0"/>

File: kuka_agilus_support/urdf/kr6_r700_2.urdf.xacro (robot description, xacro)
@@ -20,7 +20,16 @@
   <xacro:arg name="pitch" default="0"/>
   <xacro:arg name="yaw" default="0"/>
-  <xacro:kuka_agilus_ros2_control name="$(arg prefix)kr6_r700_2" driver_version="$(arg driver_version)" client_ip="$(arg client_ip)" client_port="$(arg client_port)" controller_ip="$(arg controller_ip)" prefix="$(arg prefix)" mode="$(arg mode)" use_gpio="$(arg use_gpio)" roundtrip_time="$(arg roundtrip_time)" verify_robot_model="$(arg verify_robot_model)"/>
+  <xacro:kuka_agilus_ros2_control name="$(arg prefix)kr6_r700_2" driver_version="$(arg driver_version)" client_ip="$(arg client_ip)" client_port="$(arg client_port)" controller_ip="$(arg controller_ip)" prefix="$(arg prefix)" mode="$(arg mode)" use_gpio="$(arg use_gpio)" roundtrip_time="$(arg roundtrip_time)" verify_robot_model="$(arg verify_robot_model)">
+    <ext_axes_ros2_control_joints/>
+  </xacro:kuka_agilus_ros2_control>
   <xacro:kuka_kr6_r700_2_robot prefix="$(arg prefix)" package_name="kuka_agilus_support">
-    <origin xyz="$(arg x) $(arg y) $(arg z)" rpy="$(arg roll) $(arg pitch) $(arg yaw)"/>
+    <ext_axes_links/>
+    <world-base_link_joints>
+      <joint name="$(arg prefix)world-base_link" type="fixed">
+        <parent link="world"/>
+        <child link="$(arg prefix)base_link"/>
+        <origin xyz="$(arg x) $(arg y) $(arg z)" rpy="$(arg roll) $(arg pitch) $(arg yaw)"/>
+      </joint>
+    </world-base_link_joints>
   </xacro:kuka_kr6_r700_2_robot>
 </robot>

File: kuka_agilus_support/urdf/kr6_r700_2_macro.xacro (robot description, xacro)
@@ -1,5 +1,6 @@
 <?xml version="1.0" encoding="UTF-8"?>
 <robot xmlns:xacro="http://www.ros.org/wiki/xacro" name="kr6_r700_2">
-  <xacro:macro name="kuka_kr6_r700_2_robot" params="prefix package_name *origin">
+  <xacro:macro name="kuka_kr6_r700_2_robot" params="prefix package_name **ext_axes_links **world-base_link_joints">
+    <xacro:insert_block name="ext_axes_links"/>
     <link name="${prefix}base"/>
     <link name="${prefix}base_link">
@@ -139,4 +140,5 @@
     <link name="${prefix}tool0"/>
     <link name="world"/>
+    <xacro:insert_block name="world-base_link_joints"/>
     <joint name="${prefix}base_link-base" type="fixed">
       <child link="${prefix}base"/>
@@ -195,9 +197,4 @@
       <parent link="${prefix}link_6"/>
     </joint>
-    <joint name="${prefix}world-base_link" type="fixed">
-      <child link="${prefix}base_link"/>
-      <parent link="world"/>
-      <xacro:insert_block name="origin"/>
-    </joint>
   </xacro:macro>
 </robot>

File: kuka_agilus_support/urdf/kr6_r700_sixx.urdf.xacro (robot description, xacro)
@@ -20,11 +20,16 @@
   <xacro:arg name="pitch" default="0"/>
   <xacro:arg name="yaw" default="0"/>
-  <xacro:kuka_agilus_ros2_control name="$(arg prefix)kr6_r700_sixx" driver_version="$(arg driver_version)" client_ip="$(arg client_ip)" client_port="$(arg client_port)" controller_ip="$(arg controller_ip)" prefix="$(arg prefix)" mode="$(arg mode)" use_gpio="$(arg use_gpio)" roundtrip_time="$(arg roundtrip_time)" verify_robot_model="$(arg verify_robot_model)" use_ext_axes="false">
+  <xacro:kuka_agilus_ros2_control name="$(arg prefix)kr6_r700_sixx" driver_version="$(arg driver_version)" client_ip="$(arg client_ip)" client_port="$(arg client_port)" controller_ip="$(arg controller_ip)" prefix="$(arg prefix)" mode="$(arg mode)" use_gpio="$(arg use_gpio)" roundtrip_time="$(arg roundtrip_time)" verify_robot_model="$(arg verify_robot_model)">
     <ext_axes_ros2_control_joints/>
   </xacro:kuka_agilus_ros2_control>
-  <xacro:kuka_kr6_r700_sixx_robot prefix="$(arg prefix)" package_name="kuka_agilus_support" use_ext_axes="false">
-    <origin xyz="$(arg x) $(arg y) $(arg z)" rpy="$(arg roll) $(arg pitch) $(arg yaw)"/>
+  <xacro:kuka_kr6_r700_sixx_robot prefix="$(arg prefix)" package_name="kuka_agilus_support">
     <ext_axes_links/>
-    <ext_axes_joints/>
+    <world-base_link_joints>
+      <joint name="$(arg prefix)world-base_link" type="fixed">
+        <parent link="world"/>
+        <child link="$(arg prefix)base_link"/>
+        <origin xyz="$(arg x) $(arg y) $(arg z)" rpy="$(arg roll) $(arg pitch) $(arg yaw)"/>
+      </joint>
+    </world-base_link_joints>
   </xacro:kuka_kr6_r700_sixx_robot>
 </robot>

File: kuka_agilus_support/urdf/kr6_r700_sixx_macro.xacro (robot description, xacro)
@@ -4,10 +4,8 @@
   <xacro:include filename="$(find kuka_resources)/urdf/common_constants.xacro"/>
   <xacro:include filename="$(find kuka_resources)/urdf/common_materials.xacro"/>
-  <xacro:macro name="kuka_kr6_r700_sixx_robot" params="prefix package_name use_ext_axes *origin **ext_axes_links **ext_axes_joints">
+  <xacro:macro name="kuka_kr6_r700_sixx_robot" params="prefix package_name **ext_axes_links **world-base_link_joints">
     <!-- links - main serial chain -->
     <link name="world"/>
-    <xacro:if value="${use_ext_axes}">
-      <xacro:insert_block name="ext_axes_links"/>
-    </xacro:if>
+    <xacro:insert_block name="ext_axes_links"/>
     <link name="${prefix}base_link">
       <visual>
@@ -117,14 +115,5 @@
     <!-- Following REP199, this frame shall be use to attach EEF or other equipment -->
     <link name="${prefix}flange"/>
-    <xacro:if value="${use_ext_axes}">
-      <xacro:insert_block name="ext_axes_joints"/>
-    </xacro:if>
-    <xacro:unless value="${use_ext_axes}">
-      <joint name="${prefix}world-base_link" type="fixed">
-        <parent link="world"/>
-        <child link="${prefix}base_link"/>
-        <xacro:insert_block name="origin"/>
-      </joint>
-    </xacro:unless>
+    <xacro:insert_block name="world-base_link_joints"/>
     <joint name="${prefix}joint_1" type="revolute">
       <origin xyz="0 0 0.4" rpy="0 0 0"/>

File: kuka_agilus_support/urdf/kr6_r900_2.urdf.xacro (robot description, xacro)
@@ -20,7 +20,16 @@
   <xacro:arg name="pitch" default="0"/>
   <xacro:arg name="yaw" default="0"/>
-  <xacro:kuka_agilus_ros2_control name="$(arg prefix)kr6_r900_2" driver_version="$(arg driver_version)" client_ip="$(arg client_ip)" client_port="$(arg client_port)" controller_ip="$(arg controller_ip)" prefix="$(arg prefix)" mode="$(arg mode)" use_gpio="$(arg use_gpio)" roundtrip_time="$(arg roundtrip_time)" verify_robot_model="$(arg verify_robot_model)"/>
+  <xacro:kuka_agilus_ros2_control name="$(arg prefix)kr6_r900_2" driver_version="$(arg driver_version)" client_ip="$(arg client_ip)" client_port="$(arg client_port)" controller_ip="$(arg controller_ip)" prefix="$(arg prefix)" mode="$(arg mode)" use_gpio="$(arg use_gpio)" roundtrip_time="$(arg roundtrip_time)" verify_robot_model="$(arg verify_robot_model)">
+    <ext_axes_ros2_control_joints/>
+  </xacro:kuka_agilus_ros2_control>
   <xacro:kuka_kr6_r900_2_robot prefix="$(arg prefix)" package_name="kuka_agilus_support">
-    <origin xyz="$(arg x) $(arg y) $(arg z)" rpy="$(arg roll) $(arg pitch) $(arg yaw)"/>
+    <ext_axes_links/>
+    <world-base_link_joints>
+      <joint name="$(arg prefix)world-base_link" type="fixed">
+        <parent link="world"/>
+        <child link="$(arg prefix)base_link"/>
+        <origin xyz="$(arg x) $(arg y) $(arg z)" rpy="$(arg roll) $(arg pitch) $(arg yaw)"/>
+      </joint>
+    </world-base_link_joints>
   </xacro:kuka_kr6_r900_2_robot>
 </robot>

File: kuka_agilus_support/urdf/kr6_r900_2_macro.xacro (robot description, xacro)
@@ -1,5 +1,6 @@
 <?xml version="1.0" encoding="UTF-8"?>
 <robot xmlns:xacro="http://www.ros.org/wiki/xacro" name="kr6_r900_2">
-  <xacro:macro name="kuka_kr6_r900_2_robot" params="prefix package_name *origin">
+  <xacro:macro name="kuka_kr6_r900_2_robot" params="prefix package_name **ext_axes_links **world-base_link_joints">
+    <xacro:insert_block name="ext_axes_links"/>
     <link name="${prefix}base"/>
     <link name="${prefix}base_link">
@@ -139,4 +140,5 @@
     <link name="${prefix}tool0"/>
     <link name="world"/>
+    <xacro:insert_block name="world-base_link_joints"/>
     <joint name="${prefix}base_link-base" type="fixed">
       <child link="${prefix}base"/>
@@ -195,9 +197,4 @@
       <parent link="${prefix}link_6"/>
     </joint>
-    <joint name="${prefix}world-base_link" type="fixed">
-      <child link="${prefix}base_link"/>
-      <parent link="world"/>
-      <xacro:insert_block name="origin"/>
-    </joint>
   </xacro:macro>
 </robot>

File: kuka_agilus_support/urdf/kr6_r900_sixx.urdf.xacro (robot description, xacro)
@@ -20,11 +20,16 @@
   <xacro:arg name="pitch" default="0"/>
   <xacro:arg name="yaw" default="0"/>
-  <xacro:kuka_agilus_ros2_control name="$(arg prefix)kr6_r900_sixx" driver_version="$(arg driver_version)" client_ip="$(arg client_ip)" client_port="$(arg client_port)" controller_ip="$(arg controller_ip)" prefix="$(arg prefix)" mode="$(arg mode)" use_gpio="$(arg use_gpio)" roundtrip_time="$(arg roundtrip_time)" verify_robot_model="$(arg verify_robot_model)" use_ext_axes="false">
+  <xacro:kuka_agilus_ros2_control name="$(arg prefix)kr6_r900_sixx" driver_version="$(arg driver_version)" client_ip="$(arg client_ip)" client_port="$(arg client_port)" controller_ip="$(arg controller_ip)" prefix="$(arg prefix)" mode="$(arg mode)" use_gpio="$(arg use_gpio)" roundtrip_time="$(arg roundtrip_time)" verify_robot_model="$(arg verify_robot_model)">
     <ext_axes_ros2_control_joints/>
   </xacro:kuka_agilus_ros2_control>
-  <xacro:kuka_kr6_r900_sixx_robot prefix="$(arg prefix)" package_name="kuka_agilus_support" use_ext_axes="false">
-    <origin xyz="$(arg x) $(arg y) $(arg z)" rpy="$(arg roll) $(arg pitch) $(arg yaw)"/>
+  <xacro:kuka_kr6_r900_sixx_robot prefix="$(arg prefix)" package_name="kuka_agilus_support">
     <ext_axes_links/>
-    <ext_axes_joints/>
+    <world-base_link_joints>
+      <joint name="$(arg prefix)world-base_link" type="fixed">
+        <parent link="world"/>
+        <child link="$(arg prefix)base_link"/>
+        <origin xyz="$(arg x) $(arg y) $(arg z)" rpy="$(arg roll) $(arg pitch) $(arg yaw)"/>
+      </joint>
+    </world-base_link_joints>
   </xacro:kuka_kr6_r900_sixx_robot>
 </robot>

File: kuka_agilus_support/urdf/kr6_r900_sixx_macro.xacro (robot description, xacro)
@@ -4,10 +4,8 @@
   <xacro:include filename="$(find kuka_resources)/urdf/common_constants.xacro"/>
   <xacro:include filename="$(find kuka_resources)/urdf/common_materials.xacro"/>
-  <xacro:macro name="kuka_kr6_r900_sixx_robot" params="prefix package_name use_ext_axes *origin **ext_axes_links **ext_axes_joints">
+  <xacro:macro name="kuka_kr6_r900_sixx_robot" params="prefix package_name **ext_axes_links **world-base_link_joints">
     <!-- links - main serial chain -->
     <link name="world"/>
-    <xacro:if value="${use_ext_axes}">
-      <xacro:insert_block name="ext_axes_links"/>
-    </xacro:if>
+    <xacro:insert_block name="ext_axes_links"/>
     <link name="${prefix}base_link">
       <visual>
@@ -117,14 +115,5 @@
     <!-- Following REP199, this frame shall be use to attach EEF or other equipment -->
     <link name="${prefix}flange"/>
-    <xacro:if value="${use_ext_axes}">
-      <xacro:insert_block name="ext_axes_joints"/>
-    </xacro:if>
-    <xacro:unless value="${use_ext_axes}">
-      <joint name="${prefix}world-base_link" type="fixed">
-        <parent link="world"/>
-        <child link="${prefix}base_link"/>
-        <xacro:insert_block name="origin"/>
-      </joint>
-    </xacro:unless>
+    <xacro:insert_block name="world-base_link_joints"/>
     <joint name="${prefix}joint_1" type="revolute">
       <origin xyz="0 0 0.400" rpy="0 0 0"/>

File: kuka_agilus_support/urdf/kr_agilus_ros2_control_macro.xacro (robot description, xacro)
@@ -1,5 +1,5 @@
 <?xml version="1.0" encoding="UTF-8"?>
 <robot xmlns:xacro="http://www.ros.org/wiki/xacro">
-  <xacro:macro name="kuka_agilus_ros2_control" params="name driver_version client_ip client_port controller_ip prefix mode use_gpio roundtrip_time verify_robot_model use_ext_axes **ext_axes_ros2_control_joints">
+  <xacro:macro name="kuka_agilus_ros2_control" params="name driver_version client_ip client_port controller_ip prefix mode use_gpio roundtrip_time verify_robot_model **ext_axes_ros2_control_joints">
     <!-- gazebo -->
     <xacro:if value="${mode == 'gazebo'}">
@@ -32,7 +32,5 @@
         </xacro:if>
       </hardware>
-      <xacro:if value="${use_ext_axes}">
-        <xacro:insert_block name="ext_axes_ros2_control_joints"/>
-      </xacro:if>
+      <xacro:insert_block name="ext_axes_ros2_control_joints"/>
       <joint name="${prefix}joint_1">
         <command_interface name="position"/>

File: kuka_cybertech_support/urdf/kr16_r1610_2.urdf.xacro (robot description, xacro)
@@ -20,7 +20,16 @@
   <xacro:arg name="pitch" default="0"/>
   <xacro:arg name="yaw" default="0"/>
-  <xacro:kuka_cybertech_ros2_control name="$(arg prefix)kr16_r1610_2" driver_version="$(arg driver_version)" client_ip="$(arg client_ip)" client_port="$(arg client_port)" controller_ip="$(arg controller_ip)" prefix="$(arg prefix)" mode="$(arg mode)" use_gpio="$(arg use_gpio)" roundtrip_time="$(arg roundtrip_time)" verify_robot_model="$(arg verify_robot_model)"/>
+  <xacro:kuka_cybertech_ros2_control name="$(arg prefix)kr16_r1610_2" driver_version="$(arg driver_version)" client_ip="$(arg client_ip)" client_port="$(arg client_port)" controller_ip="$(arg controller_ip)" prefix="$(arg prefix)" mode="$(arg mode)" use_gpio="$(arg use_gpio)" roundtrip_time="$(arg roundtrip_time)" verify_robot_model="$(arg verify_robot_model)">
+    <ext_axes_ros2_control_joints/>
+  </xacro:kuka_cybertech_ros2_control>
   <xacro:kuka_kr16_r1610_2_robot prefix="$(arg prefix)" package_name="kuka_cybertech_support">
-    <origin xyz="$(arg x) $(arg y) $(arg z)" rpy="$(arg roll) $(arg pitch) $(arg yaw)"/>
+    <ext_axes_links/>
+    <world-base_link_joints>
+      <joint name="$(arg prefix)world-base_link" type="fixed">
+        <parent link="world"/>
+        <child link="$(arg prefix)base_link"/>
+        <origin xyz="$(arg x) $(arg y) $(arg z)" rpy="$(arg roll) $(arg pitch) $(arg yaw)"/>
+      </joint>
+    </world-base_link_joints>
   </xacro:kuka_kr16_r1610_2_robot>
 </robot>

File: kuka_cybertech_support/urdf/kr16_r1610_2_macro.xacro (robot description, xacro)
@@ -1,5 +1,6 @@
 <?xml version="1.0" encoding="UTF-8"?>
 <robot xmlns:xacro="http://www.ros.org/wiki/xacro" name="kr16_r1610_2">
-  <xacro:macro name="kuka_kr16_r1610_2_robot" params="prefix package_name *origin">
+  <xacro:macro name="kuka_kr16_r1610_2_robot" params="prefix package_name **ext_axes_links **world-base_link_joints">
+    <xacro:insert_block name="ext_axes_links"/>
     <link name="${prefix}base"/>
     <link name="${prefix}base_link">
@@ -139,4 +140,5 @@
     <link name="${prefix}tool0"/>
     <link name="world"/>
+    <xacro:insert_block name="world-base_link_joints"/>
     <joint name="${prefix}base_link-base" type="fixed">
       <child link="${prefix}base"/>
@@ -195,9 +197,4 @@
       <parent link="${prefix}link_6"/>
     </joint>
-    <joint name="${prefix}world-base_link" type="fixed">
-      <child link="${prefix}base_link"/>
-      <parent link="world"/>
-      <xacro:insert_block name="origin"/>
-    </joint>
   </xacro:macro>
 </robot>
