Commit message: refactor - rm use_ext_axes xacro param for urdfs

File: kuka_cybertech_support/urdf/kr16_r2010_2.urdf.xacro (robot description, xacro)
@@ -20,11 +20,16 @@
   <xacro:arg name="pitch" default="0"/>
   <xacro:arg name="yaw" default="0"/>
-  <xacro:kuka_cybertech_ros2_control name="$(arg prefix)kr10_r1100_2" driver_version="$(arg driver_version)" client_ip="$(arg client_ip)" client_port="$(arg client_port)" controller_ip="$(arg controller_ip)" prefix="$(arg prefix)" mode="$(arg mode)" use_gpio="$(arg use_gpio)" roundtrip_time="$(arg roundtrip_time)" verify_robot_model="$(arg verify_robot_model)" use_ext_axes="false">
+  <xacro:kuka_cybertech_ros2_control name="$(arg prefix)kr10_r1100_2" driver_version="$(arg driver_version)" client_ip="$(arg client_ip)" client_port="$(arg client_port)" controller_ip="$(arg controller_ip)" prefix="$(arg prefix)" mode="$(arg mode)" use_gpio="$(arg use_gpio)" roundtrip_time="$(arg roundtrip_time)" verify_robot_model="$(arg verify_robot_model)">
     <ext_axes_ros2_control_joints/>
   </xacro:kuka_cybertech_ros2_control>
-  <xacro:kuka_kr16_r2010_2_robot prefix="$(arg prefix)" package_name="kuka_cybertech_support" use_ext_axes="false">
-    <origin xyz="$(arg x) $(arg y) $(arg z)" rpy="$(arg roll) $(arg pitch) $(arg yaw)"/>
+  <xacro:kuka_kr16_r2010_2_robot prefix="$(arg prefix)" package_name="kuka_cybertech_support">
     <ext_axes_links/>
-    <ext_axes_joints/>
+    <world-base_link_joints>
+      <joint name="$(arg prefix)world-base_link" type="fixed">
+        <parent link="world"/>
+        <child link="$(arg prefix)base_link"/>
+        <origin xyz="$(arg x) $(arg y) $(arg z)" rpy="$(arg roll) $(arg pitch) $(arg yaw)"/>
+      </joint>
+    </world-base_link_joints>
   </xacro:kuka_kr16_r2010_2_robot>
 </robot>

File: kuka_cybertech_support/urdf/kr16_r2010_2_macro.xacro (robot description, xacro)
@@ -1,10 +1,8 @@
 <?xml version="1.0"?>
 <robot xmlns:xacro="http://wiki.ros.org/xacro">
-  <xacro:macro name="kuka_kr16_r2010_2_robot" params="prefix package_name use_ext_axes *origin **ext_axes_links **ext_axes_joints">
+  <xacro:macro name="kuka_kr16_r2010_2_robot" params="prefix package_name **ext_axes_links **world-base_link_joints">
     <!-- links - main serial chain -->
     <link name="world"/>
-    <xacro:if value="${use_ext_axes}">
-      <xacro:insert_block name="ext_axes_links"/>
-    </xacro:if>
+    <xacro:insert_block name="ext_axes_links"/>
     <link name="${prefix}base_link">
       <collision>
@@ -105,14 +103,5 @@
       </visual>
     </link>
-    <xacro:if value="${use_ext_axes}">
-      <xacro:insert_block name="ext_axes_joints"/>
-    </xacro:if>
-    <xacro:unless value="${use_ext_axes}">
-      <joint name="${prefix}world-base_link" type="fixed">
-        <parent link="world"/>
-        <child link="${prefix}base_link"/>
-        <xacro:insert_block name="origin"/>
-      </joint>
-    </xacro:unless>
+    <xacro:insert_block name="world-base_link_joints"/>
     <joint name="${prefix}joint_1" type="revolute">
       <axis xyz="0.0 0.0 1.0"/>

File: kuka_cybertech_support/urdf/kr_cybertech_ros2_control_macro.xacro (robot description, xacro)
@@ -1,5 +1,5 @@
 <?xml version="1.0" encoding="UTF-8"?>
 <robot xmlns:xacro="http://www.ros.org/wiki/xacro">
-  <xacro:macro name="kuka_cybertech_ros2_control" params="name driver_version client_ip client_port controller_ip prefix mode use_gpio roundtrip_time verify_robot_model use_ext_axes **ext_axes_ros2_control_joints">
+  <xacro:macro name="kuka_cybertech_ros2_control" params="name driver_version client_ip client_port controller_ip prefix mode use_gpio roundtrip_time verify_robot_model **ext_axes_ros2_control_joints">
     <!-- gazebo -->
     <xacro:if value="${mode == 'gazebo'}">
@@ -32,7 +32,5 @@
         </xacro:if>
       </hardware>
-      <xacro:if value="${use_ext_axes}">
-        <xacro:insert_block name="ext_axes_ros2_control_joints"/>
-      </xacro:if>
+      <xacro:insert_block name="ext_axes_ros2_control_joints"/>
       <joint name="${prefix}joint_1">
         <command_interface name="position"/>
