Commit message: refactor: move world link + ext axis links + world-base joint/ext axes joints to urdf.xacro from macro.xacro

File: ext_axis_examples/urdf/kr10_r1100_2_with_dummy_rail.urdf.xacro (robot description, xacro)
@@ -26,13 +26,12 @@
     </ext_axes_ros2_control_joints>
   </xacro:kuka_agilus_ros2_control>
-  <xacro:kuka_kr10_r1100_2_robot prefix="$(arg prefix)" package_name="kuka_agilus_support">
-    <ext_axes_links>
-      <xacro:dummy_rail_links/>
-    </ext_axes_links>
-    <ext_axes_joints>
-      <xacro:dummy_rail_joints robot_base_link="$(arg prefix)base_link">
-        <origin xyz="$(arg x) $(arg y) $(arg z)" rpy="$(arg roll) $(arg pitch) $(arg yaw)"/>
-      </xacro:dummy_rail_joints>
-    </ext_axes_joints>
-  </xacro:kuka_kr10_r1100_2_robot>
+  <!-- world link -->
+  <link name="world"/>
+  <!-- dummy rail links -->
+  <xacro:dummy_rail_links/>
+  <xacro:kuka_kr10_r1100_2_robot prefix="$(arg prefix)" package_name="kuka_agilus_support"/>
+  <!-- dummy rail joints -->
+  <xacro:dummy_rail_joints robot_base_link="$(arg prefix)base_link">
+    <origin xyz="$(arg x) $(arg y) $(arg z)" rpy="$(arg roll) $(arg pitch) $(arg yaw)"/>
+  </xacro:dummy_rail_joints>
 </robot>

File: ext_axis_examples/urdf/kr16_r2010_2_with_dummy_rail.urdf.xacro (robot description, xacro)
@@ -26,13 +26,12 @@
     </ext_axes_ros2_control_joints>
   </xacro:kuka_cybertech_ros2_control>
-  <xacro:kuka_kr16_r2010_2_robot prefix="$(arg prefix)" package_name="kuka_cybertech_support">
-    <ext_axes_links>
-      <xacro:dummy_rail_links/>
-    </ext_axes_links>
-    <world-base_link_joints>
-      <xacro:dummy_rail_joints robot_base_link="$(arg prefix)base_link">
-        <origin xyz="$(arg x) $(arg y) $(arg z)" rpy="$(arg roll) $(arg pitch) $(arg yaw)"/>
-      </xacro:dummy_rail_joints>
-    </world-base_link_joints>
-  </xacro:kuka_kr16_r2010_2_robot>
+  <!-- world link -->
+  <link name="world"/>
+  <!-- dummy rail links -->
+  <xacro:dummy_rail_links/>
+  <xacro:kuka_kr16_r2010_2_robot prefix="$(arg prefix)" package_name="kuka_cybertech_support"/>
+  <!-- dummy rail joints -->
+  <xacro:dummy_rail_joints robot_base_link="$(arg prefix)base_link">
+    <origin xyz="$(arg x) $(arg y) $(arg z)" rpy="$(arg roll) $(arg pitch) $(arg yaw)"/>
+  </xacro:dummy_rail_joints>
 </robot>

File: kuka_agilus_support/urdf/kr10_r1100_2.urdf.xacro (robot description, xacro)
@@ -23,13 +23,13 @@
     <ext_axes_ros2_control_joints/>
   </xacro:kuka_agilus_ros2_control>
-  <xacro:kuka_kr10_r1100_2_robot prefix="$(arg prefix)" package_name="kuka_agilus_support">
-    <ext_axes_links/>
-    <world-base_link_joints>
-      <joint name="$(arg prefix)world-base_link" type="fixed">
-        <parent link="world"/>
-        <child link="$(arg prefix)base_link"/>
-        <origin xyz="$(arg x) $(arg y) $(arg z)" rpy="$(arg roll) $(arg pitch) $(arg yaw)"/>
-      </joint>
-    </world-base_link_joints>
-  </xacro:kuka_kr10_r1100_2_robot>
+  <!-- world link -->
+  <link name="world"/>
+  <!-- robot links, joints -->
+  <xacro:kuka_kr10_r1100_2_robot prefix="$(arg prefix)" package_name="kuka_agilus_support"/>
+  <!-- default world - base_link joint -->
+  <joint name="$(arg prefix)world-base_link" type="fixed">
+    <parent link="world"/>
+    <child link="$(arg prefix)base_link"/>
+    <origin xyz="$(arg x) $(arg y) $(arg z)" rpy="$(arg roll) $(arg pitch) $(arg yaw)"/>
+  </joint>
 </robot>

File: kuka_agilus_support/urdf/kr10_r1100_2_macro.xacro (robot description, xacro)
@@ -3,8 +3,6 @@
   <!-- include helper xacros -->
   <xacro:include filename="$(find kuka_resources)/urdf/common_materials.xacro"/>
-  <xacro:macro name="kuka_kr10_r1100_2_robot" params="prefix package_name **ext_axes_links **world-base_link_joints">
+  <xacro:macro name="kuka_kr10_r1100_2_robot" params="prefix package_name">
     <!-- links - main serial chain -->
-    <link name="world"/>
-    <xacro:insert_block name="ext_axes_links"/>
     <link name="${prefix}base_link">
       <collision>
@@ -148,5 +146,4 @@
     </link>
     <!-- joints - main serial chain -->
-    <xacro:insert_block name="world-base_link_joints"/>
     <joint name="${prefix}joint_1" type="revolute">
       <axis xyz="0.0 0.0 1.0"/>

File: kuka_agilus_support/urdf/kr6_r700_2.urdf.xacro (robot description, xacro)
@@ -23,13 +23,13 @@
     <ext_axes_ros2_control_joints/>
   </xacro:kuka_agilus_ros2_control>
-  <xacro:kuka_kr6_r700_2_robot prefix="$(arg prefix)" package_name="kuka_agilus_support">
-    <ext_axes_links/>
-    <world-base_link_joints>
-      <joint name="$(arg prefix)world-base_link" type="fixed">
-        <parent link="world"/>
-        <child link="$(arg prefix)base_link"/>
-        <origin xyz="$(arg x) $(arg y) $(arg z)" rpy="$(arg roll) $(arg pitch) $(arg yaw)"/>
-      </joint>
-    </world-base_link_joints>
-  </xacro:kuka_kr6_r700_2_robot>
+  <!-- world link -->
+  <link name="world"/>
+  <!-- robot links, joints -->
+  <xacro:kuka_kr6_r700_2_robot prefix="$(arg prefix)" package_name="kuka_agilus_support"/>
+  <!-- default world - base_link joint -->
+  <joint name="$(arg prefix)world-base_link" type="fixed">
+    <parent link="world"/>
+    <child link="$(arg prefix)base_link"/>
+    <origin xyz="$(arg x) $(arg y) $(arg z)" rpy="$(arg roll) $(arg pitch) $(arg yaw)"/>
+  </joint>
 </robot>

File: kuka_agilus_support/urdf/kr6_r700_2_macro.xacro (robot description, xacro)
@@ -1,6 +1,5 @@
 <?xml version="1.0" encoding="UTF-8"?>
 <robot xmlns:xacro="http://www.ros.org/wiki/xacro" name="kr6_r700_2">
-  <xacro:macro name="kuka_kr6_r700_2_robot" params="prefix package_name **ext_axes_links **world-base_link_joints">
-    <xacro:insert_block name="ext_axes_links"/>
+  <xacro:macro name="kuka_kr6_r700_2_robot" params="prefix package_name">
     <link name="${prefix}base"/>
     <link name="${prefix}base_link">
@@ -139,6 +138,4 @@
     </link>
     <link name="${prefix}tool0"/>
-    <link name="world"/>
-    <xacro:insert_block name="world-base_link_joints"/>
     <joint name="${prefix}base_link-base" type="fixed">
       <child link="${prefix}base"/>

File: kuka_agilus_support/urdf/kr6_r700_sixx.urdf.xacro (robot description, xacro)
@@ -23,13 +23,13 @@
     <ext_axes_ros2_control_joints/>
   </xacro:kuka_agilus_ros2_control>
-  <xacro:kuka_kr6_r700_sixx_robot prefix="$(arg prefix)" package_name="kuka_agilus_support">
-    <ext_axes_links/>
-    <world-base_link_joints>
-      <joint name="$(arg prefix)world-base_link" type="fixed">
-        <parent link="world"/>
-        <child link="$(arg prefix)base_link"/>
-        <origin xyz="$(arg x) $(arg y) $(arg z)" rpy="$(arg roll) $(arg pitch) $(arg yaw)"/>
-      </joint>
-    </world-base_link_joints>
-  </xacro:kuka_kr6_r700_sixx_robot>
+  <!-- world link -->
+  <link name="world"/>
+  <!-- robot links, joints -->
+  <xacro:kuka_kr6_r700_sixx_robot prefix="$(arg prefix)" package_name="kuka_agilus_support"/>
+  <!-- default world - base_link joint -->
+  <joint name="$(arg prefix)world-base_link" type="fixed">
+    <parent link="world"/>
+    <child link="$(arg prefix)base_link"/>
+    <origin xyz="$(arg x) $(arg y) $(arg z)" rpy="$(arg roll) $(arg pitch) $(arg yaw)"/>
+  </joint>
 </robot>

File: kuka_agilus_support/urdf/kr6_r700_sixx_macro.xacro (robot description, xacro)
@@ -4,8 +4,6 @@
   <xacro:include filename="$(find kuka_resources)/urdf/common_constants.xacro"/>
   <xacro:include filename="$(find kuka_resources)/urdf/common_materials.xacro"/>
-  <xacro:macro name="kuka_kr6_r700_sixx_robot" params="prefix package_name **ext_axes_links **world-base_link_joints">
+  <xacro:macro name="kuka_kr6_r700_sixx_robot" params="prefix package_name">
     <!-- links - main serial chain -->
-    <link name="world"/>
-    <xacro:insert_block name="ext_axes_links"/>
     <link name="${prefix}base_link">
       <visual>
@@ -115,5 +113,4 @@
     <!-- Following REP199, this frame shall be use to attach EEF or other equipment -->
     <link name="${prefix}flange"/>
-    <xacro:insert_block name="world-base_link_joints"/>
     <joint name="${prefix}joint_1" type="revolute">
       <origin xyz="0 0 0.4" rpy="0 0 0"/>

File: kuka_agilus_support/urdf/kr6_r900_2.urdf.xacro (robot description, xacro)
@@ -23,13 +23,13 @@
     <ext_axes_ros2_control_joints/>
   </xacro:kuka_agilus_ros2_control>
-  <xacro:kuka_kr6_r900_2_robot prefix="$(arg prefix)" package_name="kuka_agilus_support">
-    <ext_axes_links/>
-    <world-base_link_joints>
-      <joint name="$(arg prefix)world-base_link" type="fixed">
-        <parent link="world"/>
-        <child link="$(arg prefix)base_link"/>
-        <origin xyz="$(arg x) $(arg y) $(arg z)" rpy="$(arg roll) $(arg pitch) $(arg yaw)"/>
-      </joint>
-    </world-base_link_joints>
-  </xacro:kuka_kr6_r900_2_robot>
+  <!-- world link -->
+  <link name="world"/>
+  <!-- robot links, joints -->
+  <xacro:kuka_kr6_r900_2_robot prefix="$(arg prefix)" package_name="kuka_agilus_support"/>
+  <!-- default world - base_link joint -->
+  <joint name="$(arg prefix)world-base_link" type="fixed">
+    <parent link="world"/>
+    <child link="$(arg prefix)base_link"/>
+    <origin xyz="$(arg x) $(arg y) $(arg z)" rpy="$(arg roll) $(arg pitch) $(arg yaw)"/>
+  </joint>
 </robot>

File: kuka_agilus_support/urdf/kr6_r900_2_macro.xacro (robot description, xacro)
@@ -1,6 +1,5 @@
 <?xml version="1.0" encoding="UTF-8"?>
 <robot xmlns:xacro="http://www.ros.org/wiki/xacro" name="kr6_r900_2">
-  <xacro:macro name="kuka_kr6_r900_2_robot" params="prefix package_name **ext_axes_links **world-base_link_joints">
-    <xacro:insert_block name="ext_axes_links"/>
+  <xacro:macro name="kuka_kr6_r900_2_robot" params="prefix package_name">
     <link name="${prefix}base"/>
     <link name="${prefix}base_link">
@@ -139,6 +138,4 @@
     </link>
     <link name="${prefix}tool0"/>
-    <link name="world"/>
-    <xacro:insert_block name="world-base_link_joints"/>
     <joint name="${prefix}base_link-base" type="fixed">
       <child link="${prefix}base"/>

File: kuka_agilus_support/urdf/kr6_r900_sixx.urdf.xacro (robot description, xacro)
@@ -23,13 +23,13 @@
     <ext_axes_ros2_control_joints/>
   </xacro:kuka_agilus_ros2_control>
-  <xacro:kuka_kr6_r900_sixx_robot prefix="$(arg prefix)" package_name="kuka_agilus_support">
-    <ext_axes_links/>
-    <world-base_link_joints>
-      <joint name="$(arg prefix)world-base_link" type="fixed">
-        <parent link="world"/>
-        <child link="$(arg prefix)base_link"/>
-        <origin xyz="$(arg x) $(arg y) $(arg z)" rpy="$(arg roll) $(arg pitch) $(arg yaw)"/>
-      </joint>
-    </world-base_link_joints>
-  </xacro:kuka_kr6_r900_sixx_robot>
+  <!-- world link -->
+  <link name="world"/>
+  <!-- robot links, joints -->
+  <xacro:kuka_kr6_r900_sixx_robot prefix="$(arg prefix)" package_name="kuka_agilus_support"/>
+  <!-- default world - base_link joint -->
+  <joint name="$(arg prefix)world-base_link" type="fixed">
+    <parent link="world"/>
+    <child link="$(arg prefix)base_link"/>
+    <origin xyz="$(arg x) $(arg y) $(arg z)" rpy="$(arg roll) $(arg pitch) $(arg yaw)"/>
+  </joint>
 </robot>

File: kuka_agilus_support/urdf/kr6_r900_sixx_macro.xacro (robot description, xacro)
@@ -4,8 +4,6 @@
   <xacro:include filename="$(find kuka_resources)/urdf/common_constants.xacro"/>
   <xacro:include filename="$(find kuka_resources)/urdf/common_materials.xacro"/>
-  <xacro:macro name="kuka_kr6_r900_sixx_robot" params="prefix package_name **ext_axes_links **world-base_link_joints">
+  <xacro:macro name="kuka_kr6_r900_sixx_robot" params="prefix package_name">
     <!-- links - main serial chain -->
-    <link name="world"/>
-    <xacro:insert_block name="ext_axes_links"/>
     <link name="${prefix}base_link">
       <visual>
@@ -115,5 +113,4 @@
     <!-- Following REP199, this frame shall be use to attach EEF or other equipment -->
     <link name="${prefix}flange"/>
-    <xacro:insert_block name="world-base_link_joints"/>
     <joint name="${prefix}joint_1" type="revolute">
       <origin xyz="0 0 0.400" rpy="0 0 0"/>

File: kuka_cybertech_support/urdf/kr16_r1610_2.urdf.xacro (robot description, xacro)
@@ -23,13 +23,13 @@
     <ext_axes_ros2_control_joints/>
   </xacro:kuka_cybertech_ros2_control>
-  <xacro:kuka_kr16_r1610_2_robot prefix="$(arg prefix)" package_name="kuka_cybertech_support">
-    <ext_axes_links/>
-    <world-base_link_joints>
-      <joint name="$(arg prefix)world-base_link" type="fixed">
-        <parent link="world"/>
-        <child link="$(arg prefix)base_link"/>
-        <origin xyz="$(arg x) $(arg y) $(arg z)" rpy="$(arg roll) $(arg pitch) $(arg yaw)"/>
-      </joint>
-    </world-base_link_joints>
-  </xacro:kuka_kr16_r1610_2_robot>
+  <!-- world link -->
+  <link name="world"/>
+  <!-- robot links, joints -->
+  <xacro:kuka_kr16_r1610_2_robot prefix="$(arg prefix)" package_name="kuka_cybertech_support"/>
+  <!-- default world - base_link joint -->
+  <joint name="$(arg prefix)world-base_link" type="fixed">
+    <parent link="world"/>
+    <child link="$(arg prefix)base_link"/>
+    <origin xyz="$(arg x) $(arg y) $(arg z)" rpy="$(arg roll) $(arg pitch) $(arg yaw)"/>
+  </joint>
 </robot>

File: kuka_cybertech_support/urdf/kr16_r1610_2_macro.xacro (robot description, xacro)
@@ -1,6 +1,5 @@
 <?xml version="1.0" encoding="UTF-8"?>
 <robot xmlns:xacro="http://www.ros.org/wiki/xacro" name="kr16_r1610_2">
-  <xacro:macro name="kuka_kr16_r1610_2_robot" params="prefix package_name **ext_axes_links **world-base_link_joints">
-    <xacro:insert_block name="ext_axes_links"/>
+  <xacro:macro name="kuka_kr16_r1610_2_robot" params="prefix package_name">
     <link name="${prefix}base"/>
     <link name="${prefix}base_link">
@@ -139,6 +138,4 @@
     </link>
     <link name="${prefix}tool0"/>
-    <link name="world"/>
-    <xacro:insert_block name="world-base_link_joints"/>
     <joint name="${prefix}base_link-base" type="fixed">
       <child link="${prefix}base"/>

File: kuka_cybertech_support/urdf/kr16_r2010_2.urdf.xacro (robot description, xacro)
@@ -23,13 +23,13 @@
     <ext_axes_ros2_control_joints/>
   </xacro:kuka_cybertech_ros2_control>
-  <xacro:kuka_kr16_r2010_2_robot prefix="$(arg prefix)" package_name="kuka_cybertech_support">
-    <ext_axes_links/>
-    <world-base_link_joints>
-      <joint name="$(arg prefix)world-base_link" type="fixed">
-        <parent link="world"/>
-        <child link="$(arg prefix)base_link"/>
-        <origin xyz="$(arg x) $(arg y) $(arg z)" rpy="$(arg roll) $(arg pitch) $(arg yaw)"/>
-      </joint>
-    </world-base_link_joints>
-  </xacro:kuka_kr16_r2010_2_robot>
+  <!-- world link -->
+  <link name="world"/>
+  <!-- robot links, joints -->
+  <xacro:kuka_kr16_r2010_2_robot prefix="$(arg prefix)" package_name="kuka_cybertech_support"/>
+  <!-- default world - base_link joint -->
+  <joint name="$(arg prefix)world-base_link" type="fixed">
+    <parent link="world"/>
+    <child link="$(arg prefix)base_link"/>
+    <origin xyz="$(arg x) $(arg y) $(arg z)" rpy="$(arg roll) $(arg pitch) $(arg yaw)"/>
+  </joint>
 </robot>

File: kuka_cybertech_support/urdf/kr16_r2010_2_macro.xacro (robot description, xacro)
@@ -1,8 +1,6 @@
 <?xml version="1.0"?>
 <robot xmlns:xacro="http://wiki.ros.org/xacro">
-  <xacro:macro name="kuka_kr16_r2010_2_robot" params="prefix package_name **ext_axes_links **world-base_link_joints">
+  <xacro:macro name="kuka_kr16_r2010_2_robot" params="prefix package_name">
     <!-- links - main serial chain -->
-    <link name="world"/>
-    <xacro:insert_block name="ext_axes_links"/>
     <link name="${prefix}base_link">
       <collision>
@@ -103,5 +101,4 @@
       </visual>
     </link>
-    <xacro:insert_block name="world-base_link_joints"/>
     <joint name="${prefix}joint_1" type="revolute">
       <axis xyz="0.0 0.0 1.0"/>
