Commit message: fix formatting issues

File: kuka_kl_support/urdf/kl100_macro.xacro (robot description, xacro)
@@ -10,5 +10,5 @@
       </visual>
     </link>
-    <link name="rail_moving_link" >
+    <link name="rail_moving_link">
       <visual>
         <geometry>

File: kuka_kl_support/urdf/kl_ros2_control_macro.xacro (robot description, xacro)
@@ -2,5 +2,5 @@
 <robot xmlns:xacro="http://www.ros.org/wiki/xacro">
   <xacro:macro name="kuka_kl_ros2_control_joints" params="">
-   <joint name="rail_joint">
+    <joint name="rail_joint">
       <command_interface name="position"/>
       <state_interface name="position">

Commit message: Add visual mesh to KL 100

File: kuka_kl_support/urdf/kl100_macro.xacro (robot description, xacro)
@@ -9,4 +9,9 @@
         </geometry>
       </visual>
+      <collision>
+        <geometry>
+          <mesh filename="package://kuka_kl_support/meshes/kl100/collision/rail_base_link.stl"/>
+        </geometry>
+      </collision>
     </link>
     <link name="rail_moving_link">
@@ -16,4 +21,9 @@
         </geometry>
       </visual>
+      <collision>
+        <geometry>
+          <mesh filename="package://kuka_kl_support/meshes/kl100/collision/rail_moving_link.stl"/>
+        </geometry>
+      </collision>
     </link>
   </xacro:macro>

Commit message: Add KL100 height offset to Xacro

File: kuka_kl_support/urdf/kl100_macro.xacro (robot description, xacro)
@@ -45,5 +45,5 @@
       <parent link="rail_moving_link"/>
       <child link="${robot_base_link}"/>
-      <origin rpy="0.0 0.0 0.0" xyz="0.0 0.0 0.0"/>
+      <origin rpy="0.0 0.0 0.0" xyz="0.0 0.0 0.35"/>
     </joint>
   </xacro:macro>
