Commit message: kl_support - move rail_ to general prefixing

File: kuka_kl_support/urdf/kl100_2_macro.xacro (robot description, xacro)
@@ -1,7 +1,7 @@
 <?xml version="1.0" encoding="UTF-8"?>
 <robot xmlns:xacro="http://www.ros.org/wiki/xacro">
-  <xacro:macro name="kl100_2_links" params="">
+  <xacro:macro name="kl100_2_links" params="prefix">
     <!-- links -->
-    <link name="rail_base_link">
+    <link name="${prefix}base_link">
       <visual>
         <geometry>
@@ -15,5 +15,5 @@
       </collision>
     </link>
-    <link name="rail_moving_link">
+    <link name="${prefix}link_1">
       <visual>
         <geometry>
@@ -28,20 +28,20 @@
     </link>
   </xacro:macro>
-  <xacro:macro name="kl100_2_joints" params="robot_base_link *origin">
+  <xacro:macro name="kl100_2_joints" params="prefix robot_base_link *origin">
     <!-- joints -->
-    <joint name="world-rail_base" type="fixed">
+    <joint name="world-${prefix}base_link" type="fixed">
       <parent link="world"/>
-      <child link="rail_base_link"/>
+      <child link="${prefix}base_link"/>
       <xacro:insert_block name="origin"/>
     </joint>
-    <joint name="rail_joint" type="prismatic">
-      <parent link="rail_base_link"/>
-      <child link="rail_moving_link"/>
+    <joint name="${prefix}joint_1" type="prismatic">
+      <parent link="${prefix}base_link"/>
+      <child link="${prefix}link_1"/>
       <origin rpy="0.0 0.0 0.0" xyz="0.0 0.0 0.0"/>
       <axis xyz="1 0 0"/>
       <limit lower="-1.0" upper="1.0" effort="702.0" velocity="2.5"/>
     </joint>
-    <joint name="rail-robot_base" type="fixed">
-      <parent link="rail_moving_link"/>
+    <joint name="${prefix}link_1-${robot_base_link}" type="fixed">
+      <parent link="${prefix}link_1"/>
       <child link="${robot_base_link}"/>
       <origin rpy="0.0 0.0 0.0" xyz="0.0 0.0 0.356"/>

File: kuka_kl_support/urdf/kl_ros2_control_macro.xacro (robot description, xacro)
@@ -1,6 +1,6 @@
 <?xml version="1.0" encoding="UTF-8"?>
 <robot xmlns:xacro="http://www.ros.org/wiki/xacro">
-  <xacro:macro name="kuka_kl_ros2_control_joints" params="">
-    <joint name="rail_joint">
+  <xacro:macro name="kuka_kl_ros2_control_joints" params="prefix">
+    <joint name="${prefix}joint_1">
       <param name="type">prismatic</param>
       <param name="is_external">true</param>

Commit message: format + rename meshes to fit prefixing

File: kuka_kl_support/urdf/kl100_2_macro.xacro (robot description, xacro)
@@ -11,10 +11,10 @@
       <visual>
         <geometry>
-          <mesh filename="package://${package_name}/meshes/kl100_2/visual/rail_base_link.dae"/>
+          <mesh filename="package://${package_name}/meshes/kl100_2/visual/base_link.dae"/>
         </geometry>
       </visual>
       <collision>
         <geometry>
-          <mesh filename="package://${package_name}/meshes/kl100_2/collision/rail_base_link.stl"/>
+          <mesh filename="package://${package_name}/meshes/kl100_2/collision/base_link.stl"/>
         </geometry>
       </collision>
@@ -28,10 +28,10 @@
       <visual>
         <geometry>
-          <mesh filename="package://${package_name}/meshes/kl100_2/visual/rail_moving_link.dae"/>
+          <mesh filename="package://${package_name}/meshes/kl100_2/visual/link_1.dae"/>
         </geometry>
       </visual>
       <collision>
         <geometry>
-          <mesh filename="package://${package_name}/meshes/kl100_2/collision/rail_moving_link.stl"/>
+          <mesh filename="package://${package_name}/meshes/kl100_2/collision/link_1.stl"/>
         </geometry>
       </collision>

Commit message: rm unnec package arg

File: kuka_kl_support/urdf/kl100_2_macro.xacro (robot description, xacro)
@@ -1,5 +1,5 @@
 <?xml version="1.0" encoding="UTF-8"?>
 <robot xmlns:xacro="http://www.ros.org/wiki/xacro">
-  <xacro:macro name="kl100_2_links" params="prefix package_name">
+  <xacro:macro name="kl100_2_links" params="prefix">
     <!-- links -->
     <link name="${prefix}base_link">
@@ -11,10 +11,10 @@
       <visual>
         <geometry>
-          <mesh filename="package://${package_name}/meshes/kl100_2/visual/base_link.dae"/>
+          <mesh filename="package://kuka_kl_support/meshes/kl100_2/visual/base_link.dae"/>
         </geometry>
       </visual>
       <collision>
         <geometry>
-          <mesh filename="package://${package_name}/meshes/kl100_2/collision/base_link.stl"/>
+          <mesh filename="package://kuka_kl_support/meshes/kl100_2/collision/base_link.stl"/>
         </geometry>
       </collision>
@@ -28,10 +28,10 @@
       <visual>
         <geometry>
-          <mesh filename="package://${package_name}/meshes/kl100_2/visual/link_1.dae"/>
+          <mesh filename="package://kuka_kl_support/meshes/kl100_2/visual/link_1.dae"/>
         </geometry>
       </visual>
       <collision>
         <geometry>
-          <mesh filename="package://${package_name}/meshes/kl100_2/collision/link_1.stl"/>
+          <mesh filename="package://kuka_kl_support/meshes/kl100_2/collision/link_1.stl"/>
         </geometry>
       </collision>

File: kuka_resources/urdf/robot_with_external_axis_template.urdf.xacro (robot description, xacro)
@@ -71,5 +71,5 @@
   </joint>
   <!-- external axis links -->
-  <xacro:call macro="${kl_model_links_macro_name}" prefix="${kl_full_prefix}" package_name="${kl_urdf_package_value}"/>
+  <xacro:call macro="${kl_model_links_macro_name}" prefix="${kl_full_prefix}"/>
   <!-- robot links -->
   <xacro:call macro="${robot_model_macro_name}" prefix="$(arg prefix)" package_name="$(arg robot_support_package)"/>
