Commit message: Remove default value

File: kuka_kl_support/urdf/kl_ros2_control_macro.xacro (robot description, xacro)
@@ -1,5 +1,5 @@
 <?xml version="1.0" encoding="UTF-8"?>
 <robot xmlns:xacro="http://www.ros.org/wiki/xacro">
-  <xacro:macro name="kuka_kl_ros2_control_joints" params="mode:='hardware'">
+  <xacro:macro name="kuka_kl_ros2_control_joints" params="">
     <joint name="rail_joint">
       <param name="type">prismatic</param>

Commit message: fix missing mode in macro, add config for rviz launch

File: kuka_kl_support/urdf/kl_ros2_control_macro.xacro (robot description, xacro)
@@ -1,5 +1,5 @@
 <?xml version="1.0" encoding="UTF-8"?>
 <robot xmlns:xacro="http://www.ros.org/wiki/xacro">
-  <xacro:macro name="kuka_kl_ros2_control_joints" params="prefix">
+  <xacro:macro name="kuka_kl_ros2_control_joints" params="prefix mode">
     <joint name="${prefix}joint_1">
       <param name="type">prismatic</param>

File: kuka_resources/urdf/robot_with_external_axis_template.urdf.xacro (robot description, xacro)
@@ -55,5 +55,5 @@
     <xacro:call macro="${robot_ros2_control_macro_name}" name="$(arg prefix)$(arg composed_model)" driver_version="$(arg driver_version)" client_ip="$(arg client_ip)" client_port="$(arg client_port)" mxa_client_port="$(arg mxa_client_port)" controller_ip="$(arg controller_ip)" prefix="$(arg prefix)" use_gpio="$(arg use_gpio)" mode="$(arg mode)" qos_config_file="" roundtrip_time="$(arg roundtrip_time)" verify_robot_model="$(arg verify_robot_model)" rsi_xml_config_file="$(arg rsi_xml_config_file)" gazebo_controller_config_path="$(arg gazebo_controller_config_path)">
       <ext_axes_ros2_control_joints>
-        <xacro:call macro="${kl_ros2_control_joints_macro_name}" prefix="${kl_full_prefix}"/>
+        <xacro:call macro="${kl_ros2_control_joints_macro_name}" prefix="${kl_full_prefix}" mode="$(arg mode)"/>
       </ext_axes_ros2_control_joints>
     </xacro:call>
@@ -62,5 +62,5 @@
     <xacro:call macro="${robot_ros2_control_macro_name}" name="$(arg prefix)$(arg composed_model)" driver_version="$(arg driver_version)" client_ip="$(arg client_ip)" client_port="$(arg client_port)" mxa_client_port="$(arg mxa_client_port)" controller_ip="$(arg controller_ip)" prefix="$(arg prefix)" use_gpio="$(arg use_gpio)" mode="$(arg mode)" roundtrip_time="$(arg roundtrip_time)" verify_robot_model="$(arg verify_robot_model)" rsi_xml_config_file="$(arg rsi_xml_config_file)" gazebo_controller_config_path="$(arg gazebo_controller_config_path)">
       <ext_axes_ros2_control_joints>
-        <xacro:call macro="${kl_ros2_control_joints_macro_name}" prefix="${kl_full_prefix}"/>
+        <xacro:call macro="${kl_ros2_control_joints_macro_name}" prefix="${kl_full_prefix}" mode="$(arg mode)"/>
       </ext_axes_ros2_control_joints>
     </xacro:call>
