Commit message: add missing formatting

File: kuka_resources/srdf/robot_with_external_axis_template.srdf.xacro (robot description, xacro)
@@ -13,7 +13,4 @@
   <xacro:property name="kl_prefix_value" value="$(arg kl_prefix)"/>
   <xacro:include filename="robot_arm_macro.xacro"/>
-  <xacro:robot_with_external_axis_srdf
-    prefix="${prefix_value}"
-    kl_prefix="${kl_prefix_value}"
-    kl_urdf_package="${kl_urdf_package_value}"/>
+  <xacro:robot_with_external_axis_srdf prefix="${prefix_value}" kl_prefix="${kl_prefix_value}" kl_urdf_package="${kl_urdf_package_value}"/>
 </robot>

File: kuka_resources/urdf/robot_with_external_axis_template.urdf.xacro (robot description, xacro)
@@ -35,28 +35,10 @@
   <xacro:property name="kl_prefix_value" value="$(arg kl_prefix)"/>
   <xacro:property name="prefix_value" value="$(arg prefix)"/>
-  <xacro:property
-    name="robot_support_urdf_dir"
-    value="$(find ${robot_support_package_value})/urdf"
-  />
-  <xacro:property
-    name="kl_support_urdf_dir"
-    value="$(find ${kl_urdf_package_value})/urdf"
-  />
-  <xacro:property
-    name="robot_model_macro_name"
-    value="${'kuka_' + robot_model_value + '_robot'}"
-  />
-  <xacro:property
-    name="robot_ros2_control_macro_name"
-    value="${'kuka_' + robot_family_value + '_ros2_control'}"
-  />
-  <xacro:property
-    name="kl_model_links_macro_name"
-    value="${kl_model_value + '_links'}"
-  />
-  <xacro:property
-    name="kl_model_joints_macro_name"
-    value="${kl_model_value + '_joints'}"
-   />
+  <xacro:property name="robot_support_urdf_dir" value="$(find ${robot_support_package_value})/urdf"/>
+  <xacro:property name="kl_support_urdf_dir" value="$(find ${kl_urdf_package_value})/urdf"/>
+  <xacro:property name="robot_model_macro_name" value="${'kuka_' + robot_model_value + '_robot'}"/>
+  <xacro:property name="robot_ros2_control_macro_name" value="${'kuka_' + robot_family_value + '_ros2_control'}"/>
+  <xacro:property name="kl_model_links_macro_name" value="${kl_model_value + '_links'}"/>
+  <xacro:property name="kl_model_joints_macro_name" value="${kl_model_value + '_joints'}"/>
   <xacro:property name="kl_full_prefix" value="${prefix_value + kl_prefix_value}"/>
   <!-- Include urdf macro files -->
@@ -67,18 +49,5 @@
   <!-- ros2 control configuration -->
   <xacro:if value="${robot_ros2_control_macro_name == 'kuka_lbr_iisy_ros2_control'}">
-    <xacro:call macro="${robot_ros2_control_macro_name}"
-      name="$(arg prefix)$(arg composed_model)"
-      driver_version="$(arg driver_version)"
-      client_ip="$(arg client_ip)"
-      client_port="$(arg client_port)"
-      mxa_client_port="$(arg mxa_client_port)"
-      controller_ip="$(arg controller_ip)"
-      prefix="$(arg prefix)"
-      use_gpio="$(arg use_gpio)"
-      mode="$(arg mode)"
-      qos_config_file=""
-      roundtrip_time="$(arg roundtrip_time)"
-      verify_robot_model="$(arg verify_robot_model)"
-      gazebo_controller_config_path="$(arg gazebo_controller_config_path)">
+    <xacro:call macro="${robot_ros2_control_macro_name}" name="$(arg prefix)$(arg composed_model)" driver_version="$(arg driver_version)" client_ip="$(arg client_ip)" client_port="$(arg client_port)" mxa_client_port="$(arg mxa_client_port)" controller_ip="$(arg controller_ip)" prefix="$(arg prefix)" use_gpio="$(arg use_gpio)" mode="$(arg mode)" qos_config_file="" roundtrip_time="$(arg roundtrip_time)" verify_robot_model="$(arg verify_robot_model)" gazebo_controller_config_path="$(arg gazebo_controller_config_path)">
       <ext_axes_ros2_control_joints>
         <xacro:kuka_kl_ros2_control_joints prefix="${kl_full_prefix}"/>
@@ -87,17 +56,5 @@
   </xacro:if>
   <xacro:unless value="${robot_ros2_control_macro_name == 'kuka_lbr_iisy_ros2_control'}">
-    <xacro:call macro="${robot_ros2_control_macro_name}"
-      name="$(arg prefix)$(arg composed_model)"
-      driver_version="$(arg driver_version)"
-      client_ip="$(arg client_ip)"
-      client_port="$(arg client_port)"
-      mxa_client_port="$(arg mxa_client_port)"
-      controller_ip="$(arg controller_ip)"
-      prefix="$(arg prefix)"
-      use_gpio="$(arg use_gpio)"
-      mode="$(arg mode)"
-      roundtrip_time="$(arg roundtrip_time)"
-      verify_robot_model="$(arg verify_robot_model)"
-      gazebo_controller_config_path="$(arg gazebo_controller_config_path)">
+    <xacro:call macro="${robot_ros2_control_macro_name}" name="$(arg prefix)$(arg composed_model)" driver_version="$(arg driver_version)" client_ip="$(arg client_ip)" client_port="$(arg client_port)" mxa_client_port="$(arg mxa_client_port)" controller_ip="$(arg controller_ip)" prefix="$(arg prefix)" use_gpio="$(arg use_gpio)" mode="$(arg mode)" roundtrip_time="$(arg roundtrip_time)" verify_robot_model="$(arg verify_robot_model)" gazebo_controller_config_path="$(arg gazebo_controller_config_path)">
       <ext_axes_ros2_control_joints>
         <xacro:kuka_kl_ros2_control_joints prefix="${kl_full_prefix}"/>
@@ -106,28 +63,17 @@
   </xacro:unless>
   <!-- world link -->
-    <link name="world"/>
+  <link name="world"/>
   <!-- default world - external-axis base joint -->
-    <joint name="world-${kl_full_prefix}base_link" type="fixed">
-      <parent link="world"/>
-      <child link="${kl_full_prefix}base_link"/>
-      <origin xyz="$(arg x) $(arg y) $(arg z)" rpy="$(arg roll) $(arg pitch) $(arg yaw)"/>
-    </joint>
+  <joint name="world-${kl_full_prefix}base_link" type="fixed">
+    <parent link="world"/>
+    <child link="${kl_full_prefix}base_link"/>
+    <origin xyz="$(arg x) $(arg y) $(arg z)" rpy="$(arg roll) $(arg pitch) $(arg yaw)"/>
+  </joint>
   <!-- external axis links -->
-  <xacro:call
-    macro="${kl_model_links_macro_name}"
-    prefix="${kl_full_prefix}"
-    package_name="${kl_urdf_package_value}"
-  />
+  <xacro:call macro="${kl_model_links_macro_name}" prefix="${kl_full_prefix}" package_name="${kl_urdf_package_value}"/>
   <!-- robot links -->
-  <xacro:call
-    macro="${robot_model_macro_name}"
-    prefix="$(arg prefix)"
-    package_name="$(arg robot_support_package)"
-  />
+  <xacro:call macro="${robot_model_macro_name}" prefix="$(arg prefix)" package_name="$(arg robot_support_package)"/>
   <!-- external axis joints -->
-  <xacro:call
-    macro="${kl_model_joints_macro_name}"
-    prefix="${kl_full_prefix}"
-    robot_base_link="$(arg prefix)base_link">
+  <xacro:call macro="${kl_model_joints_macro_name}" prefix="${kl_full_prefix}" robot_base_link="$(arg prefix)base_link">
     <origin xyz="$(arg x) $(arg y) $(arg z)" rpy="$(arg roll) $(arg pitch) $(arg yaw)"/>
   </xacro:call>
