Commit message: rename kl_urdf_package to kl_support_package, add extra args needed for generalization

File: kuka_resources/srdf/robot_arm_macro.xacro (robot description, xacro)
@@ -5,13 +5,13 @@
 -->
 <robot xmlns:xacro="http://www.ros.org/wiki/xacro">
-  <xacro:macro name="robot_with_external_axis_srdf" params="prefix kl_prefix kl_urdf_package">
-    <xacro:include filename="$(find ${kl_urdf_package})/srdf/kl_macro.xacro"/>
+  <xacro:macro name="robot_with_external_axis_srdf" params="prefix kl_prefix kl_support_package kl_srdf_macro_file:=kl_macro.xacro kl_srdf_joints_macro:=kl_srdf_joints kl_srdf_adjacent_links_macro:=kl_srdf_adjacent_links">
+    <xacro:include filename="$(find ${kl_support_package})/srdf/${kl_srdf_macro_file}"/>
     <xacro:include filename="robot_arm_group_macro.xacro"/>
     <xacro:srdf_robot_with_ext_axes prefix="${prefix}" kl_prefix="${kl_prefix}">
       <ext_joints>
-        <xacro:kl_srdf_joints prefix="${prefix}${kl_prefix}"/>
+        <xacro:call macro="${kl_srdf_joints_macro}" prefix="${prefix}${kl_prefix}"/>
       </ext_joints>
       <ext_adjacent_links>
-        <xacro:kl_srdf_adjacent_links robot_base_link="${prefix}base_link" prefix="${prefix}${kl_prefix}"/>
+        <xacro:call macro="${kl_srdf_adjacent_links_macro}" robot_base_link="${prefix}base_link" prefix="${prefix}${kl_prefix}"/>
       </ext_adjacent_links>
     </xacro:srdf_robot_with_ext_axes>

File: kuka_resources/srdf/robot_with_external_axis_template.srdf.xacro (robot description, xacro)
@@ -6,11 +6,23 @@
 <robot xmlns:xacro="http://www.ros.org/wiki/xacro" name="$(arg composed_model)">
   <xacro:arg name="composed_model" default="robot_with_external_axis"/>
-  <xacro:arg name="kl_urdf_package" default="kuka_kl_support"/>
+  <xacro:arg name="kl_support_package" default="kuka_kl_support"/>
+  <xacro:arg name="kl_srdf_macro_file" default="kl_macro.xacro"/>
+  <xacro:arg name="kl_srdf_joints_macro" default="kl_srdf_joints"/>
+  <xacro:arg name="kl_srdf_adjacent_links_macro" default="kl_srdf_adjacent_links"/>
   <xacro:arg name="prefix" default=""/>
   <xacro:arg name="kl_prefix" default="rail_"/>
-  <xacro:property name="kl_urdf_package_value" value="$(arg kl_urdf_package)"/>
+  <xacro:property name="kl_support_package_value" value="$(arg kl_support_package)"/>
+  <xacro:property name="kl_srdf_macro_file_value" value="$(arg kl_srdf_macro_file)"/>
+  <xacro:property name="kl_srdf_joints_macro_value" value="$(arg kl_srdf_joints_macro)"/>
+  <xacro:property name="kl_srdf_adjacent_links_macro_value" value="$(arg kl_srdf_adjacent_links_macro)"/>
   <xacro:property name="prefix_value" value="$(arg prefix)"/>
   <xacro:property name="kl_prefix_value" value="$(arg kl_prefix)"/>
   <xacro:include filename="robot_arm_macro.xacro"/>
-  <xacro:robot_with_external_axis_srdf prefix="${prefix_value}" kl_prefix="${kl_prefix_value}" kl_urdf_package="${kl_urdf_package_value}"/>
+  <xacro:robot_with_external_axis_srdf
+    prefix="${prefix_value}"
+    kl_prefix="${kl_prefix_value}"
+    kl_support_package="${kl_support_package_value}"
+    kl_srdf_macro_file="${kl_srdf_macro_file_value}"
+    kl_srdf_joints_macro="${kl_srdf_joints_macro_value}"
+    kl_srdf_adjacent_links_macro="${kl_srdf_adjacent_links_macro_value}"/>
 </robot>

File: kuka_resources/urdf/robot_with_external_axis_template.urdf.xacro (robot description, xacro)
@@ -23,7 +23,9 @@
   <xacro:arg name="robot_model" default="kr10_r1100_2"/>
   <xacro:arg name="robot_support_package" default="kuka_agilus_support"/>
-  <xacro:arg name="kl_urdf_package" default="kuka_kl_support"/>
+  <xacro:arg name="kl_support_package" default="kuka_kl_support"/>
   <xacro:arg name="robot_ros2_control_macro_file" default="kr_agilus_ros2_control_macro.xacro"/>
+  <xacro:arg name="kl_ros2_control_macro_file" default="kl_ros2_control_macro.xacro"/>
   <xacro:arg name="kl_model" default="kl100_2"/>
+  <xacro:arg name="kl_ros2_control_joints_macro" default="kuka_kl_ros2_control_joints"/>
   <xacro:arg name="rsi_xml_config_file" default=""/>
   <xacro:arg name="gazebo_controller_config_path" default="config/fake_hardware_config_6_axis_kl.yaml"/>
@@ -32,14 +34,15 @@
   <xacro:property name="robot_model_value" value="$(arg robot_model)"/>
   <xacro:property name="robot_support_package_value" value="$(arg robot_support_package)"/>
-  <xacro:property name="kl_urdf_package_value" value="$(arg kl_urdf_package)"/>
+  <xacro:property name="kl_support_package_value" value="$(arg kl_support_package)"/>
   <xacro:property name="kl_model_value" value="$(arg kl_model)"/>
   <xacro:property name="kl_prefix_value" value="$(arg kl_prefix)"/>
   <xacro:property name="prefix_value" value="$(arg prefix)"/>
   <xacro:property name="robot_support_urdf_dir" value="$(find ${robot_support_package_value})/urdf"/>
-  <xacro:property name="kl_support_urdf_dir" value="$(find ${kl_urdf_package_value})/urdf"/>
+  <xacro:property name="kl_support_urdf_dir" value="$(find ${kl_support_package_value})/urdf"/>
   <xacro:property name="robot_model_macro_name" value="${'kuka_' + robot_model_value + '_robot'}"/>
   <xacro:property name="robot_ros2_control_macro_name" value="${'kuka_' + robot_family_value + '_ros2_control'}"/>
   <xacro:property name="kl_model_links_macro_name" value="${kl_model_value + '_links'}"/>
   <xacro:property name="kl_model_joints_macro_name" value="${kl_model_value + '_joints'}"/>
+  <xacro:property name="kl_ros2_control_joints_macro_name" value="$(arg kl_ros2_control_joints_macro)"/>
   <xacro:property name="kl_full_prefix" value="${prefix_value + kl_prefix_value}"/>
   <!-- Include urdf macro files -->
@@ -47,10 +50,10 @@
   <xacro:include filename="${robot_support_urdf_dir}/$(arg robot_ros2_control_macro_file)"/>
   <xacro:include filename="${kl_support_urdf_dir}/${kl_model_value}_macro.xacro"/>
-  <xacro:include filename="${kl_support_urdf_dir}/kl_ros2_control_macro.xacro"/>
+  <xacro:include filename="${kl_support_urdf_dir}/$(arg kl_ros2_control_macro_file)"/>
   <!-- ros2 control configuration -->
   <xacro:if value="${robot_ros2_control_macro_name == 'kuka_lbr_iisy_ros2_control'}">
     <xacro:call macro="${robot_ros2_control_macro_name}" name="$(arg prefix)$(arg composed_model)" driver_version="$(arg driver_version)" client_ip="$(arg client_ip)" client_port="$(arg client_port)" mxa_client_port="$(arg mxa_client_port)" controller_ip="$(arg controller_ip)" prefix="$(arg prefix)" use_gpio="$(arg use_gpio)" mode="$(arg mode)" qos_config_file="" roundtrip_time="$(arg roundtrip_time)" verify_robot_model="$(arg verify_robot_model)" rsi_xml_config_file="$(arg rsi_xml_config_file)" gazebo_controller_config_path="$(arg gazebo_controller_config_path)">
       <ext_axes_ros2_control_joints>
-        <xacro:kuka_kl_ros2_control_joints prefix="${kl_full_prefix}"/>
+        <xacro:call macro="${kl_ros2_control_joints_macro_name}" prefix="${kl_full_prefix}"/>
       </ext_axes_ros2_control_joints>
     </xacro:call>
@@ -59,5 +62,5 @@
     <xacro:call macro="${robot_ros2_control_macro_name}" name="$(arg prefix)$(arg composed_model)" driver_version="$(arg driver_version)" client_ip="$(arg client_ip)" client_port="$(arg client_port)" mxa_client_port="$(arg mxa_client_port)" controller_ip="$(arg controller_ip)" prefix="$(arg prefix)" use_gpio="$(arg use_gpio)" mode="$(arg mode)" roundtrip_time="$(arg roundtrip_time)" verify_robot_model="$(arg verify_robot_model)" rsi_xml_config_file="$(arg rsi_xml_config_file)" gazebo_controller_config_path="$(arg gazebo_controller_config_path)">
       <ext_axes_ros2_control_joints>
-        <xacro:kuka_kl_ros2_control_joints prefix="${kl_full_prefix}"/>
+        <xacro:call macro="${kl_ros2_control_joints_macro_name}" prefix="${kl_full_prefix}"/>
       </ext_axes_ros2_control_joints>
     </xacro:call>
